Commit message: fixed rotation directions of wheels

File: control/urdf/rover.urdf (robot description, URDF)
Before this commit: robot Rover, 11 links, 10 joints
Links:
- link chassis: mass None -> 2.6545367242346
Joints:
- joint back_left_pivot_to_leg: limit lower=-1.570796327 upper=1.570796327 effort=1 velocity=1 -> lower=0 upper=3.142 effort=1 velocity=1
- joint back_left_wheel_to_pivot: origin xyz=0 0.21 0 rpy=0 0 0 -> xyz=0 0.21 0 rpy=2.618 0.7854 0
- joint back_right_pivot_to_leg: limit lower=-1.570796327 upper=1.570796327 effort=1 velocity=1 -> lower=0 upper=3.142 effort=1 velocity=1
- joint back_right_wheel_to_pivot: origin xyz=0 0.21 0 rpy=0 0 0 -> xyz=0 0.21 0 rpy=2.618 0.7854 0
- joint front_left_pivot_to_leg: limit lower=-1.570796327 upper=1.570796327 effort=1 velocity=1 -> lower=0 upper=3.142 effort=1 velocity=1
- joint front_left_wheel_to_pivot: origin xyz=0 0.21 0 rpy=0 0 0 -> xyz=0 0.21 0 rpy=2.618 0.7854 0
- joint front_right_pivot_to_leg: limit lower=-1.570796327 upper=1.570796327 effort=1 velocity=1 -> lower=0 upper=3.142 effort=1 velocity=1
- joint front_right_wheel_to_pivot: origin xyz=0 0.21 0 rpy=0 0 0 -> xyz=0 0.21 0 rpy=2.618 0.7854 0
- joint right_leg_to_chassis: origin xyz=0.38331 -0.45807 0.025086 rpy=0.241692654 -1.5117 1.5708 -> xyz=0.38331 -0.45807 0.025086 rpy=-2.8999 -1.5117 1.5708

Commit message: Improved control scheme

File: control/urdf/rover.urdf (robot description, URDF)
Before this commit: robot rover, 11 links, 10 joints
Joints:
- joint back_left_pivot_to_leg: limit lower=0 upper=3.142 effort=1 velocity=1 -> lower=-1.570796327 upper=1.570796327 effort=1 velocity=1
- joint back_right_pivot_to_leg: limit lower=0 upper=3.142 effort=1 velocity=1 -> lower=-1.570796327 upper=1.570796327 effort=1 velocity=1
- joint front_left_pivot_to_leg: limit lower=0 upper=3.142 effort=1 velocity=1 -> lower=-1.570796327 upper=1.570796327 effort=1 velocity=1
- joint front_right_pivot_to_leg: limit lower=0 upper=3.142 effort=1 velocity=1 -> lower=-1.570796327 upper=1.570796327 effort=1 velocity=1
