Commit message: moved everything to core

File: core/urdf/rover.urdf (robot description, URDF)
Before this commit: robot rover, 11 links, 10 joints
Links:
- added link base_link
Joints:
- added joint base_to_chassis: type fixed, parent base_link, child chassis, origin xyz=0. -0. 0.38 rpy=0. 0. ${-pi/2}

Commit message: moving urdf mesh location to core

File: core/urdf/rover.urdf (robot description, URDF)
Before this commit: robot rover, 12 links, 11 joints
Links:
- link back_left_pivot: geometry collision mesh filename=package://core/meshes/back_left_pivot.STL; visual mesh filename=package://core/meshes/back_left_pivot.STL
- link back_left_wheel: geometry collision mesh filename=package://core/meshes/back_left_wheel.STL; visual mesh filename=package://core/meshes/back_left_wheel.STL
- link back_right_pivot: geometry collision mesh filename=package://core/meshes/back_right_pivot.STL; visual mesh filename=package://core/meshes/back_right_pivot.STL
- link back_right_wheel: geometry collision mesh filename=package://core/meshes/back_right_wheel.STL; visual mesh filename=package://core/meshes/back_right_wheel.STL
- link chassis: geometry collision mesh filename=package://core/meshes/chassis.STL; visual mesh filename=package://core/meshes/chassis.STL
- link front_left_pivot: geometry collision mesh filename=package://core/meshes/front_left_pivot.STL; visual mesh filename=package://core/meshes/front_left_pivot.STL
- link front_left_wheel: geometry collision mesh filename=package://core/meshes/front_left_wheel.STL; visual mesh filename=package://core/meshes/front_left_wheel.STL
- link front_right_pivot: geometry collision mesh filename=package://core/meshes/front_right_pivot.STL; visual mesh filename=package://core/meshes/front_right_pivot.STL
- link front_right_wheel: geometry collision mesh filename=package://core/meshes/front_right_wheel.STL; visual mesh filename=package://core/meshes/front_right_wheel.STL
- link left_leg: geometry collision mesh filename=package://core/meshes/left_leg.STL; visual mesh filename=package://core/meshes/left_leg.STL
- link right_leg: geometry collision mesh filename=package://core/meshes/right_leg.STL; visual mesh filename=package://core/meshes/right_leg.STL
