Commit message: added imu, gps, and depth cam transforms to urdf file

File: src/ros/rover/core/urdf/rover.urdf (robot description, URDF)
Before this commit: robot rover, 12 links, 11 joints
Links:
- added link d435_1
- added link d435_1_forward
- added link gps_link
- added link imu_link
Joints:
- added joint base_to_depth_forward: type fixed, parent base_link, child d435_1_forward, origin xyz=0.46 0. 0.45 rpy=0. 0. 0.
- added joint base_to_gps: type fixed, parent base_link, child gps_link, origin xyz=0. 0. 0.38 rpy=0. 0. ${-5 * pi / 18}
- added joint base_to_imu: type fixed, parent base_link, child imu_link, origin xyz=0. 0. 0.38 rpy=0. 0. 0.
- added joint depth_forward_to_depth: type fixed, parent d435_1_forward, child d435_1, origin xyz=0. 0. 0. rpy=${-49 * pi / 90} 0. ${-pi / 2}

Commit message: fixed urdf rotations for tracking and depth cameras

File: src/ros/rover/core/urdf/rover.urdf (robot description, URDF)
Before this commit: robot rover, 16 links, 15 joints
Links:
- added link t265
- added link t265_footprint
- added link t265_forward
Joints:
- added joint base_to_t265_forward: type fixed, parent base_link, child t265_forward, origin xyz=0.45 0. 0.49 rpy=0. 0. 0.
- added joint t265_forward_to_footprint: type fixed, parent t265_forward, child t265_footprint, origin xyz=0. 0. 0. rpy=${pi / 2} 0. ${-pi / 2}
- added joint t265_forward_to_t265: type fixed, parent t265_forward, child t265, origin xyz=0. 0. 0. rpy=${41 * pi / 90} 0. ${-pi / 2}

Commit message: fixed gps orientation in urdf and switched pitch and roll angles

File: src/ros/rover/core/urdf/rover.urdf (robot description, URDF)
Before this commit: robot rover, 19 links, 18 joints
Joints:
- joint base_to_gps: origin xyz=0. 0. 0.38 rpy=0. 0. ${-5 * pi / 18} -> xyz=0. 0. 0.38 rpy=0. 0. ${-5.35 * pi / 18}

Commit message: extracting useful tested changes for field test 06/05

File: src/ros/rover/core/urdf/rover.urdf (robot description, URDF)
Before this commit: robot rover, 12 links, 11 joints
Links:
- added link d435_1
- added link d435_1_forward
- added link gps_link
- added link imu_link
- added link t265
- added link t265_footprint
- added link t265_forward
Joints:
- added joint base_to_depth_forward: type fixed, parent base_link, child d435_1_forward, origin xyz=0.46 0. 0.45 rpy=0. 0. 0.
- added joint base_to_gps: type fixed, parent base_link, child gps_link, origin xyz=0. 0. 0.38 rpy=0. 0. ${-5.35 * pi / 18}
- added joint base_to_imu: type fixed, parent base_link, child imu_link, origin xyz=0. 0. 0.38 rpy=0. 0. 0.
- added joint base_to_t265_forward: type fixed, parent base_link, child t265_forward, origin xyz=0.45 0. 0.49 rpy=0. 0. 0.
- added joint depth_forward_to_depth: type fixed, parent d435_1_forward, child d435_1, origin xyz=0. 0. 0. rpy=${-49 * pi / 90} 0. ${-pi / 2}
- added joint t265_forward_to_footprint: type fixed, parent t265_forward, child t265_footprint, origin xyz=0. 0. 0. rpy=${pi / 2} 0. ${-pi / 2}
- added joint t265_forward_to_t265: type fixed, parent t265_forward, child t265, origin xyz=0. 0. 0. rpy=${41 * pi / 90} 0. ${-pi / 2}

Commit message: added both gps modules to urdf

File: src/ros/rover/core/urdf/rover.urdf (robot description, URDF)
Before this commit: robot rover, 19 links, 18 joints
Links:
- added link gps_secondary
Joints:
- added joint gps_link_to_gps_secondary: type fixed, parent gps_link, child gps_secondary, origin xyz=0.33 0.46 0. rpy=0. 0. 0.
- joint base_to_gps: origin xyz=0. 0. 0.38 rpy=0. 0. ${-5.35 * pi / 18} -> xyz=-0.33 0.23 0.38 rpy=0. 0. 0.

Commit message: fixed transforms and build dependencies

File: src/ros/rover/core/urdf/rover.urdf (robot description, URDF)
Before this commit: robot rover, 20 links, 19 joints
Joints:
- joint gps_link_to_gps_secondary: origin xyz=0.33 0.46 0. rpy=0. 0. 0. -> xyz=0.33 -0.46 0. rpy=0. 0. 0.

Commit message: fixed pitch cutoff for mapping

File: src/ros/rover/core/urdf/rover.urdf (robot description, URDF)
Before this commit: robot rover, 20 links, 19 joints
Joints:
- joint depth_forward_to_depth: origin xyz=0. 0. 0. rpy=${-49 * pi / 90} 0. ${-pi / 2} -> xyz=0. 0. 0. rpy=${-pi / 2} 0. ${-pi / 2}
