Commit message: Implemented basic approximation of d455 depth camera for gazebo.

File: src/ros/rover/core/urdf/depth_camera.xacro (robot description, xacro)
@@ -1,53 +1,50 @@
 <?xml version="1.0" encoding="utf-8"?>
-<!--Hello! This is a file coding up the depth camera for the rover in gazebo. This file is referenced at the bottom of rover.urdf.xacro,
+<!--This is a file coding up the depth camera for the rover in gazebo. This file is referenced at the bottom of rover.urdf.xacro,
 which is how it gets added to the gazebo sim. Author/s: Victor Bartlinski-->
 <robot xmlns:xacro="http://www.ros.org/wiki/xacro" >
-    <joint name="camera_joint" type="fixed">
-        <parent link="chassis"/>
-        <child link="camera_link"/>
-        <origin xyz="0 1 0.3" rpy="0 0 0"/>
-    </joint>
-    <link name="camera_link">
-        <visual>
-            <geometry>
-                <box size="0.2 0.2 0.2"/>
-            </geometry>
-        </visual>
-    </link>
-    <joint name="camera_joint_optical" type="fixed">
-        <parent link="camera_link"/>
-        <child link="camera_link_optical"/>
-        <origin xyz="0 0 0" rpy="${-pi/2} 0 ${-pi/2}"/>
-    </joint>
-    <link name="camera_link_optical"></link>
-    <gazebo reference="camera_link">
-        <sensor name="camera" type="depth">
-            <pose> 0 0 0 0 0 0 </pose>
-            <visualize>true</visualize>
-            <update_rate>10</update_rate>
-            <camera>
-                <horizontal_fov>1.089</horizontal_fov>
-                <image>
-                    <format>B8G8R8</format>
-                    <width>640</width>
-                    <height>480</height>
-                </image>
-                <clip>
-                    <near>0.05</near>
-                    <far>8.0</far>
-                </clip>
-            </camera>
-            <plugin name="camera_controller" filename="libgazebo_ros_camera.so">
-                <frame_name>camera_link_optical</frame_name>
-                <min_depth>0.1</min_depth>
-                <max_depth>100.0</max_depth>
-                <imageTopicName>image_raw</imageTopicName>
-                <pointCloudTopicName>points</pointCloudTopicName>
-                <depthImageTopicName>image_depth</depthImageTopicName>
-                <depthImageCameraInfoTopicName>depth_camera_info</depthImageCameraInfoTopicName>
-                <pointCloudCutoff>0.001</pointCloudCutoff>
-                <cameraName>camera_controller</cameraName>
-            </plugin>
-        </sensor>
-    </gazebo>
+  <joint name="camera_joint" type="fixed">
+    <origin xyz="0 0 0.48" rpy="0 0 0" />
+    <parent link="base_link" />
+    <child link="camera_link" />
+  </joint>
+  <link name='camera_link'>
+    <visual>
+      <origin xyz="0 0 0" rpy="${pi/2} 0 ${pi/2}" />
+      <geometry>
+        <mesh
+          filename="file:///$(find core)/meshes/d455.STL"
+          scale="0.001 0.001 0.001" />
+      </geometry>
+    </visual>
+  </link>
+  <joint name="camera_frame_joint" type="fixed">
+    <origin xyz="0 0 0" rpy="${-pi/2} 0 ${-pi/2}" />
+    <parent link="camera_link" />
+    <child link="camera_link_frame" />
+  </joint>
+  <link name="camera_link_frame"></link>
+  <gazebo reference="camera_link">
+    <sensor type="depth" name="camera">
+      <pose>0 0 0 0 0 0</pose>
+      <visualize>true</visualize>
+      <update_rate>10</update_rate>
+      <camera>
+        <horizontal_fov>${radians(87)}</horizontal_fov>
+        <image>
+          <width>1280</width>
+          <height>720</height>
+          <format>B8G8R8</format>
+        </image>
+        <clip>
+          <near>0.4</near>
+          <far>6.0</far>
+        </clip>
+      </camera>
+      <plugin name="camera_controller" filename="libgazebo_ros_camera.so">
+        <frame_name>camera_link_frame</frame_name>
+        <min_depth>0.1</min_depth>
+        <max_depth>100.0</max_depth>
+      </plugin>
+    </sensor>
+  </gazebo>
 </robot>

Commit message: updated depth camera pos and orientation

File: src/ros/rover/core/urdf/depth_camera.xacro (robot description, xacro)
@@ -4,12 +4,12 @@
 <robot xmlns:xacro="http://www.ros.org/wiki/xacro" >
     <joint name="camera_joint" type="fixed">
-        <parent link="chassis"/>
+        <parent link="base_link"/>
         <child link="camera_link"/>
-        <origin xyz="0 1 0.3" rpy="0 0 0"/>
+        <origin xyz="0.46 0 0.45" rpy="0 0 0"/>
     </joint>
     <link name="camera_link">
         <visual>
             <geometry>
-                <box size="0.2 0.2 0.2"/>
+                <box size="0.05 0.2 0.05"/>
             </geometry>
         </visual>
@@ -27,5 +27,5 @@
             <update_rate>10</update_rate>
             <camera>
-                <horizontal_fov>1.089</horizontal_fov>
+                <horizontal_fov>1.5</horizontal_fov>
                 <image>
                     <format>B8G8R8</format>
@@ -35,5 +35,5 @@
                 <clip>
                     <near>0.05</near>
-                    <far>8.0</far>
+                    <far>100.0</far>
                 </clip>
             </camera>
@@ -41,5 +41,5 @@
                 <frame_name>camera_link_optical</frame_name>
                 <min_depth>0.1</min_depth>
-                <max_depth>100.0</max_depth>
+                <max_depth>6.0</max_depth>
                 <imageTopicName>image_raw</imageTopicName>
                 <pointCloudTopicName>points</pointCloudTopicName>

Commit message: depth camera improvements

File: src/ros/rover/core/urdf/depth_camera.xacro (robot description, xacro)
@@ -4,5 +4,5 @@
 <robot xmlns:xacro="http://www.ros.org/wiki/xacro" >
   <joint name="camera_joint" type="fixed">
-    <origin xyz="0 0 0.48" rpy="0 0 0" />
+    <origin xyz="0.49 0 0.48" rpy="0 0 0" />
     <parent link="base_link" />
     <child link="camera_link" />
@@ -38,11 +38,11 @@
         <clip>
           <near>0.4</near>
-          <far>6.0</far>
+          <far>100.0</far>
         </clip>
       </camera>
       <plugin name="camera_controller" filename="libgazebo_ros_camera.so">
         <frame_name>camera_link_frame</frame_name>
-        <min_depth>0.1</min_depth>
-        <max_depth>100.0</max_depth>
+        <min_depth>0.6</min_depth>
+        <max_depth>6.0</max_depth>
       </plugin>
     </sensor>
