Commit message: seperate gazebo_ros2_control and non-gazebo ros2_control in urdf

File: src/ros/rover/core/urdf/ros2_control.xacro (robot description, xacro)
@@ -1,89 +1,22 @@
 <?xml version="1.0" encoding="utf-8"?>
 <robot xmlns:xacro="http://www.ros.org/wiki/xacro">
-    <ros2_control name="GazeboSystem" type="system">
+    <ros2_control name="BLCMDHardware" type="actuator">
         <hardware>
-            <plugin>gazebo_ros2_control/GazeboSystem</plugin>
+            <plugin>rover_hardware/BLCMDHardware</plugin>
         </hardware>
-        <joint name='flw'>
+        <joint name="flp">
+            <command_interface name="position">
+                <param name="min">-${pi/2}</param>
+                <param name="max">{pi/2}</param>
+            </command_interface>
             <command_interface name="velocity">
-                <param name="min">-50</param>
-                <param name="max">50</param>
+                <param name="min">-${pi}</param>
+                <param name="max">${pi}</param>
             </command_interface>
             <state_interface name="velocity"/>
+            <state_interface name="position"/>
+            <param name="id">5</param>
         </joint>
-        <joint name='frw'>
-            <command_interface name="velocity">
-                <param name="min">-50</param>
-                <param name="max">50</param>
-            </command_interface>
-            <state_interface name="velocity"/>
-        </joint>
-         <joint name='blw'>
-            <command_interface name="velocity">
-                <param name="min">-50</param>
-                <param name="max">50</param>
-            </command_interface>
-            <state_interface name="velocity"/>
-        </joint>
-        <joint name='brw'>
-            <command_interface name="velocity">
-                <param name="min">-50</param>
-                <param name="max">50</param>
-            </command_interface>
-            <state_interface name="velocity"/>
-        </joint>
-        <joint name="flp">
-        <command_interface name="position">
-          <param name="min">-${pi}</param>
-          <param name="max">${pi}</param>
-        </command_interface>
-        <command_interface name="velocity">
-          <param name="min">-${pi}</param>
-          <param name="max">${pi}</param>
-        </command_interface>
-        <state_interface name="velocity"/>
-        <state_interface name="position"/>
-        </joint>
-        <joint name="frp">
-        <command_interface name="position">
-          <param name="min">-${pi}</param>
-          <param name="max">${pi}</param>
-        </command_interface>
-        <command_interface name="velocity">
-          <param name="min">-${pi}</param>
-          <param name="max">${pi}</param>
-        </command_interface>
-        <state_interface name="velocity"/>
-        <state_interface name="position"/>
-        </joint>
-        <joint name="blp">
-        <command_interface name="position">
-          <param name="min">-${pi}</param>
-          <param name="max">${pi}</param>
-        </command_interface>
-        <command_interface name="velocity">
-          <param name="min">-${pi}</param>
-          <param name="max">${pi}</param>
-        </command_interface>
-        <state_interface name="velocity"/>
-        <state_interface name="position"/>
-        </joint>
-        <joint name="brp">
-        <command_interface name="position">
-          <param name="min">-${pi}</param>
-          <param name="max">${pi}</param>
-        </command_interface>
-        <command_interface name="velocity">
-          <param name="min">-${pi}</param>
-          <param name="max">${pi}</param>
-        </command_interface>
-        <state_interface name="velocity"/>
-        <state_interface name="position"/>
-        </joint>
+        <param name="candevice">can0</param>
     </ros2_control>
-    <gazebo>
-        <plugin filename="libgazebo_ros2_control.so" name="gazebo_ros2_control">
-            <parameters>$(find core)/params/controllers.yaml</parameters>
-        </plugin>
-    </gazebo>
 </robot>

File: src/ros/rover/core/urdf/rover.urdf.xacro (robot description, xacro)
@@ -6,4 +6,5 @@
   name="rover"
   xmlns:xacro="http://www.ros.org/wiki/xacro">
+  <xacro:arg name="gazebo" default="false"/>
   <!-- Manually added links-->
   <link name="base_link"></link>
@@ -611,4 +612,10 @@
       xyz="1 0 0" />
   </joint>
-  <xacro:include filename="ros2_control.xacro" />
+  <!-- gazebo -->
+  <xacro:if value="$(arg gazebo)">
+  <xacro:include filename="$(find core)/urdf/gazebo_ros2_control.xacro" />
+  </xacro:if>
+  <xacro:unless value="$(arg gazebo)">
+  <xacro:include filename="$(find core)/urdf/ros2_control.xacro" />
+  </xacro:unless>
 </robot>

Commit message: modified ros2_control urdf and controllers yaml for debugging

File: src/ros/rover/core/urdf/ros2_control.xacro (robot description, xacro)
@@ -7,12 +7,12 @@
             <param name="canid">5</param>
         </hardware>
-        <joint name="flp">
-            <command_interface name="position">
+        <joint name="flw">
+            <command_interface name="velocity">
                 <param name="min">-${pi/2}</param>
                 <param name="max">${pi/2}</param>
             </command_interface>
-            <command_interface name="velocity">
-                <param name="min">-${pi}</param>
-                <param name="max">${pi}</param>
+            <command_interface name="effort">
+                <param name="min">-1</param>
+                <param name="max">1</param>
             </command_interface>
             <state_interface name="velocity">
@@ -20,9 +20,4 @@
                 <param name="max">${pi}</param>
             </state_interface>
-            <state_interface name="position">
-                <param name="min">-${pi/2}</param>
-                <param name="max">${pi/2}</param>
-            </state_interface>
-            <param name="resolver_reduction">${4./3.}</param>
         </joint>
     </ros2_control>

Commit message: Added pivot to ros2_control urdf

File: src/ros/rover/core/urdf/ros2_control.xacro (robot description, xacro)
@@ -5,7 +5,32 @@
             <plugin>blcmd_hardware/BLCMDHardware</plugin>
             <param name="candevice">can0</param>
-            <param name="canid">3</param>
+            <param name="canid">1</param>
         </hardware>
         <joint name="flw">
+            <command_interface name="velocity">
+                <param name="min">-5.0</param>
+                <param name="max">5.0</param>
+            </command_interface>
+            <command_interface name="effort">
+                <param name="min">-1</param>
+                <param name="max">1</param>
+            </command_interface>
+            <state_interface name="velocity">
+                <param name="min">-5</param>
+                <param name="max">5</param>
+            </state_interface>
+        </joint>
+    </ros2_control>
+        <ros2_control name="BLCMDHardware" type="actuator">
+        <hardware>
+            <plugin>blcmd_hardware/BLCMDHardware</plugin>
+            <param name="candevice">can0</param>
+            <param name="canid">5</param>
+        </hardware>
+        <joint name="flp">
+            <command_interface name="position">
+                <param name="min">-5.0</param>
+                <param name="max">5.0</param>
+            </command_interface>
             <command_interface name="velocity">
                 <param name="min">-5.0</param>

Commit message: blcmd_hardware: added mock param for off rover testing

File: src/ros/rover/core/urdf/ros2_control.xacro (robot description, xacro)
@@ -2,4 +2,24 @@
 <robot xmlns:xacro="http://www.ros.org/wiki/xacro">
     <ros2_control name="FrontLeftWheel" type="actuator">
+        <hardware>
+            <plugin>blcmd_hardware/BLCMDHardware</plugin>
+            <param name="candevice">can0</param>
+            <param name="canid">1</param>
+            <param name="resolver_reduction">1</param>
+            <param name="clock_rate">100000000</param>
+            <param name="revolution_pulses">8192</param>
+            <param name="mock">true</param>
+        </hardware>
+        <joint name="flw">
+            <command_interface name="velocity">
+            </command_interface>
+            <command_interface name="effort">
+                <param name="max">1</param>
+            </command_interface>
+            <state_interface name="velocity">
+            </state_interface>
+        </joint>
+    </ros2_control>
+    <ros2_control name="BackLeftWheel" type="actuator">
         <hardware>
             <plugin>blcmd_hardware/BLCMDHardware</plugin>
@@ -9,6 +29,47 @@
             <param name="clock_rate">100000000</param>
             <param name="revolution_pulses">8192</param>
+            <param name="mock">true</param>
         </hardware>
-        <joint name="flw">
+        <joint name="blw">
+            <command_interface name="velocity">
+            </command_interface>
+            <command_interface name="effort">
+                <param name="max">1</param>
+            </command_interface>
+            <state_interface name="velocity">
+            </state_interface>
+        </joint>
+    </ros2_control>
+    <ros2_control name="BackRightWheel" type="actuator">
+        <hardware>
+            <plugin>blcmd_hardware/BLCMDHardware</plugin>
+            <param name="candevice">can0</param>
+            <param name="canid">3</param>
+            <param name="resolver_reduction">1</param>
+            <param name="clock_rate">100000000</param>
+            <param name="revolution_pulses">8192</param>
+            <param name="mock">true</param>
+        </hardware>
+        <joint name="brw">
+            <command_interface name="velocity">
+            </command_interface>
+            <command_interface name="effort">
+                <param name="max">1</param>
+            </command_interface>
+            <state_interface name="velocity">
+            </state_interface>
+        </joint>
+    </ros2_control>
+    <ros2_control name="FronRightWheel" type="actuator">
+        <hardware>
+            <plugin>blcmd_hardware/BLCMDHardware</plugin>
+            <param name="candevice">can0</param>
+            <param name="canid">4</param>
+            <param name="resolver_reduction">1</param>
+            <param name="clock_rate">100000000</param>
+            <param name="revolution_pulses">8192</param>
+            <param name="mock">true</param>
+        </hardware>
+        <joint name="frw">
             <command_interface name="velocity">
             </command_interface>
@@ -28,4 +89,5 @@
             <param name="clock_rate">100000000</param>
             <param name="revolution_pulses">8192</param>
+            <param name="mock">true</param>
         </hardware>
         <joint name="flp">
@@ -45,3 +107,81 @@
         </joint>
     </ros2_control>
+    <ros2_control name="BackLeftPivot" type="actuator">
+        <hardware>
+            <plugin>blcmd_hardware/BLCMDHardware</plugin>
+            <param name="candevice">can0</param>
+            <param name="canid">6</param>
+            <param name="resolver_reduction">1</param>
+            <param name="clock_rate">100000000</param>
+            <param name="revolution_pulses">8192</param>
+            <param name="mock">true</param>
+        </hardware>
+        <joint name="blp">
+            <command_interface name="position">
+                <param name="max">5.0</param>
+            </command_interface>
+            <command_interface name="velocity">
+            </command_interface>
+            <command_interface name="effort">
+                <param name="max">1</param>
+            </command_interface>
+            <state_interface name="velocity">
+            </state_interface>
+            <state_interface name="position">
+                <param name="max">5.0</param>
+            </state_interface>
+        </joint>
+    </ros2_control>
+        <ros2_control name="BackRightPivot" type="actuator">
+        <hardware>
+            <plugin>blcmd_hardware/BLCMDHardware</plugin>
+            <param name="candevice">can0</param>
+            <param name="canid">7</param>
+            <param name="resolver_reduction">1</param>
+            <param name="clock_rate">100000000</param>
+            <param name="revolution_pulses">8192</param>
+            <param name="mock">true</param>
+        </hardware>
+        <joint name="brp">
+            <command_interface name="position">
+                <param name="max">5.0</param>
+            </command_interface>
+            <command_interface name="velocity">
+            </command_interface>
+            <command_interface name="effort">
+                <param name="max">1</param>
+            </command_interface>
+            <state_interface name="velocity">
+            </state_interface>
+            <state_interface name="position">
+                <param name="max">5.0</param>
+            </state_interface>
+        </joint>
+    </ros2_control>
+    <ros2_control name="FrontRightPivot" type="actuator">
+        <hardware>
+            <plugin>blcmd_hardware/BLCMDHardware</plugin>
+            <param name="candevice">can0</param>
+            <param name="canid">8</param>
+            <param name="resolver_reduction">1</param>
+            <param name="clock_rate">100000000</param>
+            <param name="revolution_pulses">8192</param>
+            <param name="mock">true</param>
+        </hardware>
+        <joint name="frp">
+            <command_interface name="position">
+                <param name="max">5.0</param>
+            </command_interface>
+            <command_interface name="velocity">
+            </command_interface>
+            <command_interface name="effort">
+                <param name="max">1</param>
+            </command_interface>
+            <state_interface name="velocity">
+            </state_interface>
+            <state_interface name="position">
+                <param name="max">5.0</param>
+            </state_interface>
+        </joint>
+    </ros2_control>
 </robot>
