Commit message: pivot_drive_controller: added support for mock_components/GenericSystem

File: src/ros/rover/core/urdf/ros2_control.xacro (robot description, xacro)
@@ -1,187 +1,274 @@
 <?xml version="1.0" encoding="utf-8"?>
 <robot xmlns:xacro="http://www.ros.org/wiki/xacro">
-    <ros2_control name="FrontLeftWheel" type="actuator">
-        <hardware>
-            <plugin>blcmd_hardware/BLCMDHardware</plugin>
-            <param name="candevice">can0</param>
-            <param name="canid">1</param>
-            <param name="resolver_reduction">1</param>
-            <param name="clock_rate">100000000</param>
-            <param name="revolution_pulses">8192</param>
-            <param name="mock">true</param>
-        </hardware>
-        <joint name="flw">
-            <command_interface name="velocity">
-            </command_interface>
-            <command_interface name="effort">
-                <param name="max">1</param>
-            </command_interface>
-            <state_interface name="velocity">
-            </state_interface>
-        </joint>
-    </ros2_control>
-    <ros2_control name="BackLeftWheel" type="actuator">
-        <hardware>
-            <plugin>blcmd_hardware/BLCMDHardware</plugin>
-            <param name="candevice">can0</param>
-            <param name="canid">2</param>
-            <param name="resolver_reduction">1</param>
-            <param name="clock_rate">100000000</param>
-            <param name="revolution_pulses">8192</param>
-            <param name="mock">true</param>
-        </hardware>
-        <joint name="blw">
-            <command_interface name="velocity">
-            </command_interface>
-            <command_interface name="effort">
-                <param name="max">1</param>
-            </command_interface>
-            <state_interface name="velocity">
-            </state_interface>
-        </joint>
-    </ros2_control>
-    <ros2_control name="BackRightWheel" type="actuator">
-        <hardware>
-            <plugin>blcmd_hardware/BLCMDHardware</plugin>
-            <param name="candevice">can0</param>
-            <param name="canid">3</param>
-            <param name="resolver_reduction">1</param>
-            <param name="clock_rate">100000000</param>
-            <param name="revolution_pulses">8192</param>
-            <param name="mock">true</param>
-        </hardware>
-        <joint name="brw">
-            <command_interface name="velocity">
-            </command_interface>
-            <command_interface name="effort">
-                <param name="max">1</param>
-            </command_interface>
-            <state_interface name="velocity">
-            </state_interface>
-        </joint>
-    </ros2_control>
-    <ros2_control name="FronRightWheel" type="actuator">
-        <hardware>
-            <plugin>blcmd_hardware/BLCMDHardware</plugin>
-            <param name="candevice">can0</param>
-            <param name="canid">4</param>
-            <param name="resolver_reduction">1</param>
-            <param name="clock_rate">100000000</param>
-            <param name="revolution_pulses">8192</param>
-            <param name="mock">true</param>
-        </hardware>
-        <joint name="frw">
-            <command_interface name="velocity">
-            </command_interface>
-            <command_interface name="effort">
-                <param name="max">1</param>
-            </command_interface>
-            <state_interface name="velocity">
-            </state_interface>
-        </joint>
-    </ros2_control>
-    <ros2_control name="FrontLeftPivot" type="actuator">
-        <hardware>
-            <plugin>blcmd_hardware/BLCMDHardware</plugin>
-            <param name="candevice">can0</param>
-            <param name="canid">5</param>
-            <param name="resolver_reduction">1</param>
-            <param name="clock_rate">100000000</param>
-            <param name="revolution_pulses">8192</param>
-            <param name="mock">true</param>
-        </hardware>
-        <joint name="flp">
-            <command_interface name="position">
-                <param name="max">5.0</param>
-            </command_interface>
-            <command_interface name="velocity">
-            </command_interface>
-            <command_interface name="effort">
-                <param name="max">1</param>
-            </command_interface>
-            <state_interface name="velocity">
-            </state_interface>
-            <state_interface name="position">
-                <param name="max">5.0</param>
-            </state_interface>
-        </joint>
-    </ros2_control>
-    <ros2_control name="BackLeftPivot" type="actuator">
-        <hardware>
-            <plugin>blcmd_hardware/BLCMDHardware</plugin>
-            <param name="candevice">can0</param>
-            <param name="canid">6</param>
-            <param name="resolver_reduction">1</param>
-            <param name="clock_rate">100000000</param>
-            <param name="revolution_pulses">8192</param>
-            <param name="mock">true</param>
-        </hardware>
-        <joint name="blp">
-            <command_interface name="position">
-                <param name="max">5.0</param>
-            </command_interface>
-            <command_interface name="velocity">
-            </command_interface>
-            <command_interface name="effort">
-                <param name="max">1</param>
-            </command_interface>
-            <state_interface name="velocity">
-            </state_interface>
-            <state_interface name="position">
-                <param name="max">5.0</param>
-            </state_interface>
-        </joint>
-    </ros2_control>
+    <xacro:macro name="rover_ros2_control" params="use_mock_hardware">
+        <ros2_control name="FrontLeftWheel" type="actuator">
+        <!-- <ros2_control name="FrontLeftWheel" type="system"> -->
+            <xacro:unless value="${use_mock_hardware}">
+                <hardware>
+                    <plugin>blcmd_hardware/BLCMDHardware</plugin>
+                    <param name="candevice">can0</param>
+                    <param name="canid">1</param>
+                    <param name="resolver_reduction">1</param>
+                    <param name="clock_rate">100000000</param>
+                    <param name="revolution_pulses">8192</param>
+                    <param name="mock">true</param>
+                </hardware>
+            </xacro:unless>
+            <xacro:if value="${use_mock_hardware}">
+                <hardware>
+                    <plugin>mock_components/GenericSystem</plugin>
+                    <param name="calculate_dynamics">true</param>
+                </hardware>
+            </xacro:if>
+            <joint name="flw">
+                <command_interface name="velocity">
+                </command_interface>
+                <command_interface name="effort">
+                    <param name="max">1</param>
+                </command_interface>
+                <state_interface name="velocity">
+                    <param name="initial_value">0.0</param>
+                </state_interface>
+            </joint>
+        </ros2_control>
+        <ros2_control name="BackLeftWheel" type="actuator">
+        <!-- <ros2_control name="BackLeftWheel" type="system"> -->
+            <xacro:unless value="${use_mock_hardware}">
+                <hardware>
+                    <plugin>blcmd_hardware/BLCMDHardware</plugin>
+                    <param name="candevice">can0</param>
+                    <param name="canid">2</param>
+                    <param name="resolver_reduction">1</param>
+                    <param name="clock_rate">100000000</param>
+                    <param name="revolution_pulses">8192</param>
+                    <param name="mock">true</param>
+                </hardware>
+            </xacro:unless>
+            <xacro:if value="${use_mock_hardware}">
+                <hardware>
+                    <plugin>mock_components/GenericSystem</plugin>
+                    <param name="calculate_dynamics">true</param>
+                </hardware>
+            </xacro:if>
+            <joint name="blw">
+                <command_interface name="velocity">
+                </command_interface>
+                <command_interface name="effort">
+                    <param name="max">1</param>
+                </command_interface>
+                <state_interface name="velocity">
+                    <param name="initial_value">0.0</param>
+                </state_interface>
+            </joint>
+        </ros2_control>
+        <ros2_control name="BackRightWheel" type="actuator">
+        <!-- <ros2_control name="BackRightWheel" type="system"> -->
+            <xacro:unless value="${use_mock_hardware}">
+                <hardware>
+                    <plugin>blcmd_hardware/BLCMDHardware</plugin>
+                    <param name="candevice">can0</param>
+                    <param name="canid">3</param>
+                    <param name="resolver_reduction">1</param>
+                    <param name="clock_rate">100000000</param>
+                    <param name="revolution_pulses">8192</param>
+                    <param name="mock">true</param    <param name="initial_value">0.0</param>
+>
+                </hardware>
+            </xacro:unless>
+            <xacro:if value="${use_mock_hardware}">
+                <hardware>
+                    <plugin>mock_components/GenericSystem</plugin>
+                    <param name="calculate_dynamics">true</param>
+                </hardware>
+            </xacro:if>
+            <joint name="brw">
+                <command_interface name="velocity">
+                </command_interface>
+                <command_interface name="effort">
+                    <param name="max">1</param>
+                </command_interface>
+                <state_interface name="velocity">
+                    <param name="initial_value">0.0</param>
+                </state_interface>
+            </joint>
+        </ros2_control>
+        <ros2_control name="FrontRightWheel" type="actuator">
+        <!-- <ros2_control name="FrontRightWheel" type="system"> -->
+            <xacro:unless value="${use_mock_hardware}">
+                <hardware>
+                    <plugin>blcmd_hardware/BLCMDHardware</plugin>
+                    <param name="candevice">can0</param>
+                    <param name="canid">4</param>
+                    <param name="resolver_reduction">1</param>
+                    <param name="clock_rate">100000000</param>
+                    <param name="revolution_pulses">8192</param>
+                    <param name="mock">true</param>
+                </hardware>
+            </xacro:unless>
+            <xacro:if value="${use_mock_hardware}">
+                <hardware>
+                    <plugin>mock_components/GenericSystem</plugin>
+                    <param name="calculate_dynamics">true</param>
+                </hardware>
+            </xacro:if>
+            <joint name="frw">
+                <command_interface name="velocity">
+                </command_interface>
+                <command_interface name="effort">
+                    <param name="max">1</param>
+                </command_interface>
+                <state_interface name="velocity">
+                    <param name="initial_value">0.0</param>
+                </state_interface>
+            </joint>
+        </ros2_control>
+        <ros2_control name="FrontLeftPivot" type="actuator">
+        <!-- <ros2_control name="FrontLeftPivot" type="system"> -->
+            <xacro:unless value="${use_mock_hardware}">
+                <hardware>
+                    <plugin>blcmd_hardware/BLCMDHardware</plugin>
+                    <param name="candevice">can0</param>
+                    <param name="canid">5</param>
+                    <param name="resolver_reduction">1</param>
+                    <param name="clock_rate">100000000</param>
+                    <param name="revolution_pulses">8192</param>
+                    <param name="mock">true</param>
+                </hardware>
+            </xacro:unless>
+            <xacro:if value="${use_mock_hardware}">
+                <hardware>
+                    <plugin>mock_components/GenericSystem</plugin>
+                    <param name="calculate_dynamics">true</param>
+                </hardware>
+            </xacro:if>
+            <joint name="flp">
+                <command_interface name="position">
+                    <param name="max">5.0</param>
+                </command_interface>
+                <command_interface name="velocity">
+                </command_interface>
+                <command_interface name="effort">
+                    <param name="max">1</param>
+                </command_interface>
+                <state_interface name="velocity">
+                    <param name="initial_value">0.0</param>
+                </state_interface>
+                <state_interface name="position">
+                    <param name="inital_value">0.0</param>
+                    <param name="max">5.0</param>    <param name="initial_value">0.0</param>
+                </state_interface>
+            </joint>
+        </ros2_control>
+        <!-- <ros2_control name="BackLeftPivot" type="system"> -->
+        <ros2_control name="BackLeftPivot" type="actuator">
+            <xacro:unless value="${use_mock_hardware}">
+                <hardware>
+                    <plugin>blcmd_hardware/BLCMDHardware</plugin>
+                    <param name="candevice">can0</param>
+                    <param name="canid">6</param>
+                    <param name="resolver_reduction">1</param>
+                    <param name="clock_rate">100000000</param>
+                    <param name="revolution_pulses">8192</param>
+                    <param name="mock">true</param>
+                </hardware>
+            </xacro:unless>
+            <xacro:if value="${use_mock_hardware}">
+                <hardware>
+                    <plugin>mock_components/GenericSystem</plugin>
+                    <param name="calculate_dynamics">true</param>
+                </hardware>
+            </xacro:if>
+            <joint name="blp">
+                <command_interface name="position">
+                    <param name="max">5.0</param>
+                </command_interface>
+                <command_interface name="velocity">
+                </command_interface>
+                <command_interface name="effort">
+                    <param name="max">1</param>
+                </command_interface>
+                <state_interface name="velocity">
+                    <param name="initial_value">0.0</param>
+                </state_interface>
+                <state_interface name="position">
+                    <param name="initial_value">0.0</param>
+                    <param name="max">5.0</param>
+                </state_interface>
+            </joint>
+        </ros2_control>
         <ros2_control name="BackRightPivot" type="actuator">
-        <hardware>
-            <plugin>blcmd_hardware/BLCMDHardware</plugin>
-            <param name="candevice">can0</param>
-            <param name="canid">7</param>
-            <param name="resolver_reduction">1</param>
-            <param name="clock_rate">100000000</param>
-            <param name="revolution_pulses">8192</param>
-            <param name="mock">true</param>
-        </hardware>
-        <joint name="brp">
-            <command_interface name="position">
-                <param name="max">5.0</param>
-            </command_interface>
-            <command_interface name="velocity">
-            </command_interface>
-            <command_interface name="effort">
-                <param name="max">1</param>
-            </command_interface>
-            <state_interface name="velocity">
-            </state_interface>
-            <state_interface name="position">
-                <param name="max">5.0</param>
-            </state_interface>
-        </joint>
-    </ros2_control>
-    <ros2_control name="FrontRightPivot" type="actuator">
-        <hardware>
-            <plugin>blcmd_hardware/BLCMDHardware</plugin>
-            <param name="candevice">can0</param>
-            <param name="canid">8</param>
-            <param name="resolver_reduction">1</param>
-            <param name="clock_rate">100000000</param>
-            <param name="revolution_pulses">8192</param>
-            <param name="mock">true</param>
-        </hardware>
-        <joint name="frp">
-            <command_interface name="position">
-                <param name="max">5.0</param>
-            </command_interface>
-            <command_interface name="velocity">
-            </command_interface>
-            <command_interface name="effort">
-                <param name="max">1</param>
-            </command_interface>
-            <state_interface name="velocity">
-            </state_interface>
-            <state_interface name="position">
-                <param name="max">5.0</param>
-            </state_interface>
-        </joint>
-    </ros2_control>
+        <!-- <ros2_control name="BackRightPivot" type="system"> -->
+            <xacro:unless value="${use_mock_hardware}">
+                <hardware>
+                    <plugin>blcmd_hardware/BLCMDHardware</plugin>
+                    <param name="candevice">can0</param>
+                    <param name="canid">7</param>
+                    <param name="resolver_reduction">1</param>
+                    <param name="clock_rate">100000000</param>
+                    <param name="revolution_pulses">8192</param>
+                    <param name="mock">true</param>
+                </hardware>
+            </xacro:unless>
+            <xacro:if value="${use_mock_hardware}">
+                <hardware>
+                    <plugin>mock_components/GenericSystem</plugin>
+                    <param name="calculate_dynamics">true</param>
+                </hardware>
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
File: src/ros/rover/core/urdf/rover.urdf.xacro (robot description, xacro)
@@ -7,4 +7,5 @@
   xmlns:xacro="http://www.ros.org/wiki/xacro">
   <xacro:arg name="gazebo" default="false"/>
+  <xacro:arg name="use_mock_hardware" default="false"/>
   <!-- Manually added links-->
   <link name="base_link"></link>
@@ -614,8 +615,9 @@
   <!-- gazebo -->
   <xacro:if value="$(arg gazebo)">
-  <xacro:include filename="$(find core)/urdf/gazebo_ros2_control.xacro" />
+    <xacro:include filename="$(find core)/urdf/gazebo_ros2_control.xacro" />
   </xacro:if>
   <xacro:unless value="$(arg gazebo)">
-  <xacro:include filename="$(find core)/urdf/ros2_control.xacro" />
+    <xacro:include filename="$(find core)/urdf/ros2_control.xacro" />
+    <xacro:rover_ros2_control use_mock_hardware="$(arg use_mock_hardware)"/>
   </xacro:unless>
 </robot>
