Commit message: param, launch, urdf changes

File: src/ros/rover/core/urdf/ros2_control.xacro (robot description, xacro)
@@ -233,4 +233,43 @@
                     <param name="clock_rate">100000000</param>
                     <param name="revolution_pulses">8192</param>
+                    <param name="min_interval">233</param>
+                    <param name="gear_ratio">36.0</param>
+	            <param name="mock">true</param>
+                </hardware>
+            </xacro:unless>
+            <xacro:if value="${use_mock_hardware}">
+                <hardware>
+                    <plugin>mock_components/GenericSystem</plugin>
+                    <param name="calculate_dynamics">true</param>
+                </hardware>
+            </xacro:if>
+            <joint name="brp">
+                <command_interface name="position">
+                    <param name="max">1.57079632679</param>
+                </command_interface>
+                <command_interface name="velocity">
+                    <param name="max">1.0</param>
+                </command_interface>
+                <command_interface name="effort">
+                    <param name="max">1</param>
+                </command_interface>
+                <state_interface name="velocity">
+                    <param name="initial_value">0.0</param>
+                </state_interface>
+                <state_interface name="position">
+                    <param name="initial_value">0.0</param>
+                    <param name="max">1.57079632679</param>
+                </state_interface>
+            </joint>
+        </ros2_control>
+        <ros2_control name="FrontRightPivot" type="system">
+            <xacro:unless value="${use_mock_hardware}">
+                <hardware>
+                    <plugin>blcmd_hardware/BLCMDHardware</plugin>
+                    <param name="candevice">can0</param>
+                    <param name="canid">8</param>
+                    <param name="resolver_reduction">1.33333333333</param>
+                    <param name="clock_rate">100000000</param>
+                    <param name="revolution_pulses">8192</param>
                     <param name="reversed">true</param>
                     <param name="min_interval">233</param>
@@ -245,44 +284,4 @@
                 </hardware>
             </xacro:if>
-            <joint name="brp">
-                <command_interface name="position">
-                    <param name="max">1.57079632679</param>
-                </command_interface>
-                <command_interface name="velocity">
-                    <param name="max">1.0</param>
-                </command_interface>
-                <command_interface name="effort">
-                    <param name="max">1</param>
-                </command_interface>
-                <state_interface name="velocity">
-                    <param name="initial_value">0.0</param>
-                </state_interface>
-                <state_interface name="position">
-                    <param name="initial_value">0.0</param>
-                    <param name="max">1.57079632679</param>
-                </state_interface>
-            </joint>
-        </ros2_control>
-        <ros2_control name="FrontRightPivot" type="system">
-            <xacro:unless value="${use_mock_hardware}">
-                <hardware>
-                    <plugin>blcmd_hardware/BLCMDHardware</plugin>
-                    <param name="candevice">can0</param>
-                    <param name="canid">8</param>
-                    <param name="resolver_reduction">1.33333333333</param>
-                    <param name="clock_rate">100000000</param>
-                    <param name="revolution_pulses">8192</param>
-                    <param name="reversed">true</param>
-                    <param name="min_interval">233</param>
-                    <param name="gear_ratio">36.0</param>
-	            <param name="mock">true</param>
-                </hardware>
-            </xacro:unless>
-            <xacro:if value="${use_mock_hardware}">
-                <hardware>
-                    <plugin>mock_components/GenericSystem</plugin>
-                    <param name="calculate_dynamics">true</param>
-                </hardware>
-            </xacro:if>
             <joint name="frp">
                 <command_interface name="position">
