Commit message: Changing Filename for meshes

File: src/ros/rover/rover_description/urdf/arm_rover.urdf.xacro (robot description, xacro)
@@ -27,19 +27,19 @@
       <geometry>
         <mesh
-          filename="package://URDF_PART_FILES/meshes/base_link.STL" />
-      </geometry>
-      <material
-        name="">
-        <color
-          rgba="0.792156862745098 0.819607843137255 0.933333333333333 1" />
-      </material>
-    </visual>
-    <collision>
-      <origin
-        xyz="0 0 0"
-        rpy="0 0 0" />
-      <geometry>
-        <mesh
-          filename="package://URDF_PART_FILES/meshes/base_link.STL" />
+          filename="file:///$(find rover_description)/meshes/base_link.STL" />
+      </geometry>
+      <material
+        name="">
+        <color
+          rgba="0.792156862745098 0.819607843137255 0.933333333333333 1" />
+      </material>
+    </visual>
+    <collision>
+      <origin
+        xyz="0 0 0"
+        rpy="0 0 0" />
+      <geometry>
+        <mesh
+          filename="file:///$(find rover_description)/meshes/base_link.STL" />
       </geometry>
     </collision>
@@ -67,19 +67,19 @@
       <geometry>
         <mesh
-          filename="package://URDF_PART_FILES/meshes/link1.STL" />
-      </geometry>
-      <material
-        name="">
-        <color
-          rgba="0.792156862745098 0.819607843137255 0.933333333333333 1" />
-      </material>
-    </visual>
-    <collision>
-      <origin
-        xyz="0 0 0"
-        rpy="0 0 0" />
-      <geometry>
-        <mesh
-          filename="package://URDF_PART_FILES/meshes/link1.STL" />
+          filename="file:///$(find rover_description)/meshes/link1.STL" />
+      </geometry>
+      <material
+        name="">
+        <color
+          rgba="0.792156862745098 0.819607843137255 0.933333333333333 1" />
+      </material>
+    </visual>
+    <collision>
+      <origin
+        xyz="0 0 0"
+        rpy="0 0 0" />
+      <geometry>
+        <mesh
+          filename="file:///$(find rover_description)/meshes/link1.STL" />
       </geometry>
     </collision>
@@ -125,19 +125,19 @@
       <geometry>
         <mesh
-          filename="package://URDF_PART_FILES/meshes/link2.STL" />
-      </geometry>
-      <material
-        name="">
-        <color
-          rgba="0.792156862745098 0.819607843137255 0.933333333333333 1" />
-      </material>
-    </visual>
-    <collision>
-      <origin
-        xyz="0 0 0"
-        rpy="0 0 0" />
-      <geometry>
-        <mesh
-          filename="package://URDF_PART_FILES/meshes/link2.STL" />
+          filename="file:///$(find rover_description)/meshes/link2.STL" />
+      </geometry>
+      <material
+        name="">
+        <color
+          rgba="0.792156862745098 0.819607843137255 0.933333333333333 1" />
+      </material>
+    </visual>
+    <collision>
+      <origin
+        xyz="0 0 0"
+        rpy="0 0 0" />
+      <geometry>
+        <mesh
+          filename="file:///$(find rover_description)/meshes/link2.STL" />
       </geometry>
     </collision>
@@ -183,19 +183,19 @@
       <geometry>
         <mesh
-          filename="package://URDF_PART_FILES/meshes/link3.STL" />
-      </geometry>
-      <material
-        name="">
-        <color
-          rgba="0.792156862745098 0.819607843137255 0.933333333333333 1" />
-      </material>
-    </visual>
-    <collision>
-      <origin
-        xyz="0 0 0"
-        rpy="0 0 0" />
-      <geometry>
-        <mesh
-          filename="package://URDF_PART_FILES/meshes/link3.STL" />
+          filename="file:///$(find rover_description)/meshes/link3.STL" />
+      </geometry>
+      <material
+        name="">
+        <color
+          rgba="0.792156862745098 0.819607843137255 0.933333333333333 1" />
+      </material>
+    </visual>
+    <collision>
+      <origin
+        xyz="0 0 0"
+        rpy="0 0 0" />
+      <geometry>
+        <mesh
+          filename="file:///$(find rover_description)/meshes/link3.STL" />
       </geometry>
     </collision>
@@ -241,19 +241,19 @@
       <geometry>
         <mesh
-          filename="package://URDF_PART_FILES/meshes/link4.STL" />
-      </geometry>
-      <material
-        name="">
-        <color
-          rgba="0.792156862745098 0.819607843137255 0.933333333333333 1" />
-      </material>
-    </visual>
-    <collision>
-      <origin
-        xyz="0 0 0"
-        rpy="0 0 0" />
-      <geometry>
-        <mesh
-          filename="package://URDF_PART_FILES/meshes/link4.STL" />
+          filename="file:///$(find rover_description)/meshes/link4.STL" />
+      </geometry>
+      <material
+        name="">
+        <color
+          rgba="0.792156862745098 0.819607843137255 0.933333333333333 1" />
+      </material>
+    </visual>
+    <collision>
+      <origin
+        xyz="0 0 0"
+        rpy="0 0 0" />
+      <geometry>
+        <mesh
+          filename="file:///$(find rover_description)/meshes/link4.STL" />
       </geometry>
     </collision>
@@ -294,19 +294,19 @@
       <geometry>
         <mesh
-          filename="package://URDF_PART_FILES/meshes/link5.STL" />
-      </geometry>
-      <material
-        name="">
-        <color
-          rgba="0.792156862745098 0.819607843137255 0.933333333333333 1" />
-      </material>
-    </visual>
-    <collision>
-      <origin
-        xyz="0 0 0"
-        rpy="0 0 0" />
-      <geometry>
-        <mesh
-          filename="package://URDF_PART_FILES/meshes/link5.STL" />
+          filename="file:///$(find rover_description)/meshes/link5.STL" />
+      </geometry>
+      <material
+        name="">
+        <color
+          rgba="0.792156862745098 0.819607843137255 0.933333333333333 1" />
+      </material>
+    </visual>
+    <collision>
+      <origin
+        xyz="0 0 0"
+        rpy="0 0 0" />
+      <geometry>
+        <mesh
+          filename="file:///$(find rover_description)/meshes/link5.STL" />
       </geometry>
     </collision>
@@ -352,19 +352,19 @@
       <geometry>
         <mesh
-          filename="package://URDF_PART_FILES/meshes/link6.STL" />
-      </geometry>
-      <material
-        name="">
-        <color
-          rgba="0.792156862745098 0.819607843137255 0.933333333333333 1" />
-      </material>
-    </visual>
-    <collision>
-      <origin
-        xyz="0 0 0"
-        rpy="0 0 0" />
-      <geometry>
-        <mesh
-          filename="package://URDF_PART_FILES/meshes/link6.STL" />
+          filename="file:///$(find rover_description)/meshes/link6.STL" />
+      </geometry>
+      <material
+        name="">
+        <color
+          rgba="0.792156862745098 0.819607843137255 0.933333333333333 1" />
+      </material>
+    </visual>
+    <collision>
+      <origin
+        xyz="0 0 0"
+        rpy="0 0 0" />
+      <geometry>
+        <mesh
+          filename="file:///$(find rover_description)/meshes/link6.STL" />
       </geometry>
     </collision>
@@ -410,5 +410,5 @@
       <geometry>
         <mesh
-          filename="package://URDF_PART_FILES/meshes/EE.STL" />
+          filename="file:///$(find rover_description)/meshes/EE.STL" />
       </geometry>
       <material
@@ -424,5 +424,5 @@
       <geometry>
         <mesh
-          filename="package://URDF_PART_FILES/meshes/EE.STL" />
+          filename="file:///$(find rover_description)/meshes/EE.STL" />
       </geometry>
     </collision>

Commit message: Change Zero Position

File: src/ros/rover/rover_description/urdf/arm_rover.urdf.xacro (robot description, xacro)
@@ -4,97 +4,97 @@
      For more information, please see http://wiki.ros.org/sw_urdf_exporter -->
 <robot
-  name="URDF_PART_FILES">
-  <link
-    name="base_link">
-    <inertial>
-      <origin
-        xyz="0.124895291114619 0.105803300474521 0.151689368311352"
-        rpy="0 0 0" />
-      <mass
-        value="0.964885521720054" />
-      <inertia
-        ixx="0.00737801555834588"
-        ixy="3.46523316685227E-08"
-        ixz="4.42994703749863E-08"
-        iyy="0.0112664844620674"
-        iyz="-0.000899960613165917"
-        izz="0.00586330404662385" />
-    </inertial>
-    <visual>
-      <origin
-        xyz="0 0 0"
-        rpy="0 0 0" />
-      <geometry>
-        <mesh
-          filename="file:///$(find rover_description)/meshes/base_link.STL" />
-      </geometry>
-      <material
-        name="">
-        <color
-          rgba="0.792156862745098 0.819607843137255 0.933333333333333 1" />
-      </material>
-    </visual>
-    <collision>
-      <origin
-        xyz="0 0 0"
-        rpy="0 0 0" />
-      <geometry>
-        <mesh
-          filename="file:///$(find rover_description)/meshes/base_link.STL" />
-      </geometry>
-    </collision>
-  </link>
-  <link
-    name="link1">
-    <inertial>
-      <origin
-        xyz="0.114459650115267 0.000894475466029554 4.63193089098174E-05"
-        rpy="0 0 0" />
-      <mass
-        value="1.06782992821244" />
-      <inertia
-        ixx="0.00110450364652873"
-        ixy="-1.13558642402736E-06"
-        ixz="0.000123600017443695"
-        iyy="0.0010668360523279"
-        iyz="-7.98361132115831E-07"
-        izz="0.00136059075592228" />
-    </inertial>
-    <visual>
-      <origin
-        xyz="0 0 0"
-        rpy="0 0 0" />
-      <geometry>
-        <mesh
-          filename="file:///$(find rover_description)/meshes/link1.STL" />
-      </geometry>
-      <material
-        name="">
-        <color
-          rgba="0.792156862745098 0.819607843137255 0.933333333333333 1" />
-      </material>
-    </visual>
-    <collision>
-      <origin
-        xyz="0 0 0"
-        rpy="0 0 0" />
-      <geometry>
-        <mesh
-          filename="file:///$(find rover_description)/meshes/link1.STL" />
-      </geometry>
-    </collision>
-  </link>
-  <joint
-    name="base-rotation"
-    type="revolute">
-    <origin
-      xyz="0.1249 -0.106 0.15434"
-      rpy="2.6199 -1.5571 0.6857" />
-    <parent
-      link="base_link" />
-    <child
-      link="link1" />
-    <axis
-      xyz="0.99991 0.0068196 -0.011865" />
+  name="URDF_PART_ASSEMBLY">
+  <link
+    name="ArmBase">
+    <inertial>
+      <origin
+        xyz="0.0463984559338307 -0.000244629347594962 0.105803300473719"
+        rpy="0 0 0" />
+      <mass
+        value="0.964885521729071" />
+      <inertia
+        ixx="0.00586330404665839"
+        ixy="4.42994692639774E-08"
+        ixz="-0.00089996061315548"
+        iyy="0.00737801555838317"
+        iyz="3.46523353363795E-08"
+        izz="0.0112664844620711" />
+    </inertial>
+    <visual>
+      <origin
+        xyz="0 0 0"
+        rpy="0 0 0" />
+      <geometry>
+        <mesh
+          filename="package://URDF_PART_ASSEMBLY/meshes/ArmBase.STL" />
+      </geometry>
+      <material
+        name="">
+        <color
+          rgba="0.792156862745098 0.819607843137255 0.933333333333333 1" />
+      </material>
+    </visual>
+    <collision>
+      <origin
+        xyz="0 0 0"
+        rpy="0 0 0" />
+      <geometry>
+        <mesh
+          filename="package://URDF_PART_ASSEMBLY/meshes/ArmBase.STL" />
+      </geometry>
+    </collision>
+  </link>
+  <link
+    name="BaseToJ1">
+    <inertial>
+      <origin
+        xyz="-0.00115949735646111 0.0892985869596572 -0.000828732075412772"
+        rpy="0 0 0" />
+      <mass
+        value="1.06782865454781" />
+      <inertia
+        ixx="0.00136349514209711"
+        ixy="-0.000120523153646633"
+        ixz="-4.27584675271316E-07"
+        iyy="0.00110158912271039"
+        iyz="8.73000906376952E-07"
+        izz="0.00106684454111778" />
+    </inertial>
+    <visual>
+      <origin
+        xyz="0 0 0"
+        rpy="0 0 0" />
+      <geometry>
+        <mesh
+          filename="package://URDF_PART_ASSEMBLY/meshes/BaseToJ1.STL" />
+      </geometry>
+      <material
+        name="">
+        <color
+          rgba="0.792156862745098 0.819607843137255 0.933333333333333 1" />
+      </material>
+    </visual>
+    <collision>
+      <origin
+        xyz="0 0 0"
+        rpy="0 0 0" />
+      <geometry>
+        <mesh
+          filename="package://URDF_PART_ASSEMBLY/meshes/BaseToJ1.STL" />
+      </geometry>
+    </collision>
+  </link>
+  <joint
+    name="J1"
+    type="revolute">
+    <origin
+      xyz="0 0 0.1795"
+      rpy="1.5708 0 -1.5708" />
+    <parent
+      link="ArmBase" />
+    <child
+      link="BaseToJ1" />
+    <axis
+      xyz="0 1 0" />
     <limit
       lower="0"
@@ -104,55 +104,55 @@
   </joint>
   <link
-    name="link2">
-    <inertial>
-      <origin
-        xyz="-0.0727312955042903 -0.261084601636969 -0.152093536327788"
-        rpy="0 0 0" />
-      <mass
-        value="0.692669362097279" />
-      <inertia
-        ixx="0.00581162431890537"
-        ixy="3.66152054222498E-06"
-        ixz="-7.38995480405447E-06"
-        iyy="0.00189230548123107"
-        iyz="-0.00194817270298663"
-        izz="0.00406780326105112" />
-    </inertial>
-    <visual>
-      <origin
-        xyz="0 0 0"
-        rpy="0 0 0" />
-      <geometry>
-        <mesh
-          filename="file:///$(find rover_description)/meshes/link2.STL" />
-      </geometry>
-      <material
-        name="">
-        <color
-          rgba="0.792156862745098 0.819607843137255 0.933333333333333 1" />
-      </material>
-    </visual>
-    <collision>
-      <origin
-        xyz="0 0 0"
-        rpy="0 0 0" />
-      <geometry>
-        <mesh
-          filename="file:///$(find rover_description)/meshes/link2.STL" />
-      </geometry>
-    </collision>
-  </link>
-  <joint
-    name="shoulder"
-    type="revolute">
-    <origin
-      xyz="0.096952 0.00025571 -0.043073"
-      rpy="1.3139 -1.5629 -1.7961" />
-    <parent
-      link="link1" />
-    <child
-      link="link2" />
-    <axis
-      xyz="0.99991 0.0068196 -0.011865" />
+    name="J2ToLink1">
+    <inertial>
+      <origin
+        xyz="0.302150544196856 -0.00272064453324986 0.0215545407301324"
+        rpy="0 0 0" />
+      <mass
+        value="0.692670468382813" />
+      <inertia
+        ixx="0.000749127415490433"
+        ixy="3.9226287616403E-05"
+        ixz="1.68457558241152E-07"
+        iyy="0.00521089609335111"
+        iyz="-1.840147885579E-06"
+        izz="0.00581175230962762" />
+    </inertial>
+    <visual>
+      <origin
+        xyz="0 0 0"
+        rpy="0 0 0" />
+      <geometry>
+        <mesh
+          filename="package://URDF_PART_ASSEMBLY/meshes/J2ToLink1.STL" />
+      </geometry>
+      <material
+        name="">
+        <color
+          rgba="0.792156862745098 0.819607843137255 0.933333333333333 1" />
+      </material>
+    </visual>
+    <collision>
+      <origin
+        xyz="0 0 0"
+        rpy="0 0 0" />
+      <geometry>
+        <mesh
+          filename="package://URDF_PART_ASSEMBLY/meshes/J2ToLink1.STL" />
+      </geometry>
+    </collision>
+  </link>
+  <joint
+    name="J2"
+    type="revolute">
+    <origin
+      xyz="0.0933 0.0723 -0.00028711"
+      rpy="1.5708 0 1.5708" />
+    <parent
+      link="BaseToJ1" />
+    <child
+      link="J2ToLink1" />
+    <axis
+      xyz="0 0 -1" />
     <limit
       lower="-1.75"
@@ -162,55 +162,55 @@
   </joint>
   <link
-    name="link3">
-    <inertial>
-      <origin
-        xyz="0.0366028999656508 -0.0895330260674386 0.118561290612098"
-        rpy="0 0 0" />
-      <mass
-        value="1.15373119624722" />
-      <inertia
-        ixx="0.00391492060968911"
-        ixy="-6.46459234827351E-05"
-        ixz="-0.00017879907270972"
-        iyy="0.00149074655925531"
-        iyz="0.000919585901244272"
-        izz="0.00339029817500588" />
-    </inertial>
-    <visual>
-      <origin
-        xyz="0 0 0"
-        rpy="0 0 0" />
-      <geometry>
-        <mesh
-          filename="file:///$(find rover_description)/meshes/link3.STL" />
-      </geometry>
-      <material
-        name="">
-        <color
-          rgba="0.792156862745098 0.819607843137255 0.933333333333333 1" />
-      </material>
-    </visual>
-    <collision>
-      <origin
-        xyz="0 0 0"
-        rpy="0 0 0" />
-      <geometry>
-        <mesh
-          filename="file:///$(find rover_description)/meshes/link3.STL" />
-      </geometry>
-    </collision>
-  </link>
-  <joint
-    name="elbow"
-    type="revolute">
-    <origin
-      xyz="-6.0514E-05 -0.41827 -0.24551"
-      rpy="-2.764 0.020381 0.017534" />
-    <parent
-      link="link2" />
-    <child
-      link="link3" />
-    <axis
-      xyz="0.99991 0.0068196 -0.011865" />
+    name="J3ToLink2">
+    <inertial>
+      <origin
+        xyz="0.129966189328165 0.0732399519417659 -0.0854948314562504"
+        rpy="0 0 0" />
+      <mass
+        value="1.1537312044344" />
+      <inertia
+        ixx="0.00112066300003786"
+        ixy="7.23793330716904E-05"
+        ixz="-1.74454352298505E-05"
+        iyy="0.00375619318284082"
+        iyz="0.00018874261573622"
+        izz="0.00391910919823574" />
+    </inertial>
+    <visual>
+      <origin
+        xyz="0 0 0"
+        rpy="0 0 0" />
+      <geometry>
+        <mesh
+          filename="package://URDF_PART_ASSEMBLY/meshes/J3ToLink2.STL" />
+      </geometry>
+      <material
+        name="">
+        <color
+          rgba="0.792156862745098 0.819607843137255 0.933333333333333 1" />
+      </material>
+    </visual>
+    <collision>
+      <origin
+        xyz="0 0 0"
+        rpy="0 0 0" />
+      <geometry>
+        <mesh
+          filename="package://URDF_PART_ASSEMBLY/meshes/J3ToLink2.STL" />
+      </geometry>
+    </collision>
+  </link>
+  <joint
+    name="J3"
+    type="revolute">
+    <origin
+      xyz="0.48498 -0.0042617 -1.3115E-05"
+      rpy="0 0 0" />
+    <parent
+      link="J2ToLink1" />
+    <child
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