Commit message: Change filename path

File: src/ros/rover/rover_description/urdf/arm_rover.urdf.xacro (robot description, xacro)
@@ -27,19 +27,19 @@
       <geometry>
         <mesh
-          filename="package://URDF_PART_ASSEMBLY/meshes/ArmBase.STL" />
-      </geometry>
-      <material
-        name="">
-        <color
-          rgba="0.792156862745098 0.819607843137255 0.933333333333333 1" />
-      </material>
-    </visual>
-    <collision>
-      <origin
-        xyz="0 0 0"
-        rpy="0 0 0" />
-      <geometry>
-        <mesh
-          filename="package://URDF_PART_ASSEMBLY/meshes/ArmBase.STL" />
+          filename="file:///$(find rover_description)/meshes/ArmBase.STL" />
+      </geometry>
+      <material
+        name="">
+        <color
+          rgba="0.792156862745098 0.819607843137255 0.933333333333333 1" />
+      </material>
+    </visual>
+    <collision>
+      <origin
+        xyz="0 0 0"
+        rpy="0 0 0" />
+      <geometry>
+        <mesh
+          filename="file:///$(find rover_description)/meshes/ArmBase.STL" />
       </geometry>
     </collision>
@@ -67,19 +67,19 @@
       <geometry>
         <mesh
-          filename="package://URDF_PART_ASSEMBLY/meshes/BaseToJ1.STL" />
-      </geometry>
-      <material
-        name="">
-        <color
-          rgba="0.792156862745098 0.819607843137255 0.933333333333333 1" />
-      </material>
-    </visual>
-    <collision>
-      <origin
-        xyz="0 0 0"
-        rpy="0 0 0" />
-      <geometry>
-        <mesh
-          filename="package://URDF_PART_ASSEMBLY/meshes/BaseToJ1.STL" />
+          filename="file:///$(find rover_description)/meshes/BaseToJ1.STL" />
+      </geometry>
+      <material
+        name="">
+        <color
+          rgba="0.792156862745098 0.819607843137255 0.933333333333333 1" />
+      </material>
+    </visual>
+    <collision>
+      <origin
+        xyz="0 0 0"
+        rpy="0 0 0" />
+      <geometry>
+        <mesh
+          filename="file:///$(find rover_description)/meshes/BaseToJ1.STL" />
       </geometry>
     </collision>
@@ -125,19 +125,19 @@
       <geometry>
         <mesh
-          filename="package://URDF_PART_ASSEMBLY/meshes/J2ToLink1.STL" />
-      </geometry>
-      <material
-        name="">
-        <color
-          rgba="0.792156862745098 0.819607843137255 0.933333333333333 1" />
-      </material>
-    </visual>
-    <collision>
-      <origin
-        xyz="0 0 0"
-        rpy="0 0 0" />
-      <geometry>
-        <mesh
-          filename="package://URDF_PART_ASSEMBLY/meshes/J2ToLink1.STL" />
+          filename="file:///$(find rover_description)/meshes/J2ToLink1.STL" />
+      </geometry>
+      <material
+        name="">
+        <color
+          rgba="0.792156862745098 0.819607843137255 0.933333333333333 1" />
+      </material>
+    </visual>
+    <collision>
+      <origin
+        xyz="0 0 0"
+        rpy="0 0 0" />
+      <geometry>
+        <mesh
+          filename="file:///$(find rover_description)/meshes/J2ToLink1.STL" />
       </geometry>
     </collision>
@@ -183,19 +183,19 @@
       <geometry>
         <mesh
-          filename="package://URDF_PART_ASSEMBLY/meshes/J3ToLink2.STL" />
-      </geometry>
-      <material
-        name="">
-        <color
-          rgba="0.792156862745098 0.819607843137255 0.933333333333333 1" />
-      </material>
-    </visual>
-    <collision>
-      <origin
-        xyz="0 0 0"
-        rpy="0 0 0" />
-      <geometry>
-        <mesh
-          filename="package://URDF_PART_ASSEMBLY/meshes/J3ToLink2.STL" />
+          filename="file:///$(find rover_description)/meshes/J3ToLink2.STL" />
+      </geometry>
+      <material
+        name="">
+        <color
+          rgba="0.792156862745098 0.819607843137255 0.933333333333333 1" />
+      </material>
+    </visual>
+    <collision>
+      <origin
+        xyz="0 0 0"
+        rpy="0 0 0" />
+      <geometry>
+        <mesh
+          filename="file:///$(find rover_description)/meshes/J3ToLink2.STL" />
       </geometry>
     </collision>
@@ -241,19 +241,19 @@
       <geometry>
         <mesh
-          filename="package://URDF_PART_ASSEMBLY/meshes/Link2toFixedJ4.STL" />
-      </geometry>
-      <material
-        name="">
-        <color
-          rgba="0.792156862745098 0.819607843137255 0.933333333333333 1" />
-      </material>
-    </visual>
-    <collision>
-      <origin
-        xyz="0 0 0"
-        rpy="0 0 0" />
-      <geometry>
-        <mesh
-          filename="package://URDF_PART_ASSEMBLY/meshes/Link2toFixedJ4.STL" />
+          filename="file:///$(find rover_description)/meshes/Link2toFixedJ4.STL" />
+      </geometry>
+      <material
+        name="">
+        <color
+          rgba="0.792156862745098 0.819607843137255 0.933333333333333 1" />
+      </material>
+    </visual>
+    <collision>
+      <origin
+        xyz="0 0 0"
+        rpy="0 0 0" />
+      <geometry>
+        <mesh
+          filename="file:///$(find rover_description)/meshes/Link2toFixedJ4.STL" />
       </geometry>
     </collision>
@@ -294,19 +294,19 @@
       <geometry>
         <mesh
-          filename="package://URDF_PART_ASSEMBLY/meshes/J4ToJ5.STL" />
-      </geometry>
-      <material
-        name="">
-        <color
-          rgba="0.792156862745098 0.819607843137255 0.933333333333333 1" />
-      </material>
-    </visual>
-    <collision>
-      <origin
-        xyz="0 0 0"
-        rpy="0 0 0" />
-      <geometry>
-        <mesh
-          filename="package://URDF_PART_ASSEMBLY/meshes/J4ToJ5.STL" />
+          filename="file:///$(find rover_description)/meshes/J4ToJ5.STL" />
+      </geometry>
+      <material
+        name="">
+        <color
+          rgba="0.792156862745098 0.819607843137255 0.933333333333333 1" />
+      </material>
+    </visual>
+    <collision>
+      <origin
+        xyz="0 0 0"
+        rpy="0 0 0" />
+      <geometry>
+        <mesh
+          filename="file:///$(find rover_description)/meshes/J4ToJ5.STL" />
       </geometry>
     </collision>
@@ -352,19 +352,19 @@
       <geometry>
         <mesh
-          filename="package://URDF_PART_ASSEMBLY/meshes/J5ToJ6.STL" />
-      </geometry>
-      <material
-        name="">
-        <color
-          rgba="0.792156862745098 0.819607843137255 0.933333333333333 1" />
-      </material>
-    </visual>
-    <collision>
-      <origin
-        xyz="0 0 0"
-        rpy="0 0 0" />
-      <geometry>
-        <mesh
-          filename="package://URDF_PART_ASSEMBLY/meshes/J5ToJ6.STL" />
+          filename="file:///$(find rover_description)/meshes/J5ToJ6.STL" />
+      </geometry>
+      <material
+        name="">
+        <color
+          rgba="0.792156862745098 0.819607843137255 0.933333333333333 1" />
+      </material>
+    </visual>
+    <collision>
+      <origin
+        xyz="0 0 0"
+        rpy="0 0 0" />
+      <geometry>
+        <mesh
+          filename="file:///$(find rover_description)/meshes/J5ToJ6.STL" />
       </geometry>
     </collision>
@@ -410,19 +410,19 @@
       <geometry>
         <mesh
-          filename="package://URDF_PART_ASSEMBLY/meshes/J6ToEE.STL" />
-      </geometry>
-      <material
-        name="">
-        <color
-          rgba="0.792156862745098 0.819607843137255 0.933333333333333 1" />
-      </material>
-    </visual>
-    <collision>
-      <origin
-        xyz="0 0 0"
-        rpy="0 0 0" />
-      <geometry>
-        <mesh
-          filename="package://URDF_PART_ASSEMBLY/meshes/J6ToEE.STL" />
+          filename="file:///$(find rover_description)/meshes/J6ToEE.STL" />
+      </geometry>
+      <material
+        name="">
+        <color
+          rgba="0.792156862745098 0.819607843137255 0.933333333333333 1" />
+      </material>
+    </visual>
+    <collision>
+      <origin
+        xyz="0 0 0"
+        rpy="0 0 0" />
+      <geometry>
+        <mesh
+          filename="file:///$(find rover_description)/meshes/J6ToEE.STL" />
       </geometry>
     </collision>

Commit message: Modified URDF Orientation

File: src/ros/rover/rover_description/urdf/arm_rover.urdf.xacro (robot description, xacro)
@@ -4,10 +4,10 @@
      For more information, please see http://wiki.ros.org/sw_urdf_exporter -->
 <robot
-  name="URDF_PART_ASSEMBLY">
+  name="URDF_PART_ASSEMBLY_URDFONLY">
   <link
     name="ArmBase">
     <inertial>
       <origin
-        xyz="0.0463984559338307 -0.000244629347594962 0.105803300473719"
+        xyz="0.0463984559338307 -0.000244629347594955 0.105803300473719"
         rpy="0 0 0" />
       <mass
@@ -15,8 +15,8 @@
       <inertia
         ixx="0.00586330404665839"
-        ixy="4.42994692639774E-08"
-        ixz="-0.00089996061315548"
+        ixy="4.42994692638961E-08"
+        ixz="-0.000899960613155479"
         iyy="0.00737801555838317"
-        iyz="3.46523353363795E-08"
+        iyz="3.46523353363265E-08"
         izz="0.0112664844620711" />
     </inertial>
@@ -49,5 +49,5 @@
     <inertial>
       <origin
-        xyz="-0.00115949735646111 0.0892985869596572 -0.000828732075412772"
+        xyz="-0.0011594973564611 0.0892985869596572 -0.000828732075412786"
         rpy="0 0 0" />
       <mass
@@ -58,5 +58,5 @@
         ixz="-4.27584675271316E-07"
         iyy="0.00110158912271039"
-        iyz="8.73000906376952E-07"
+        iyz="8.73000906376955E-07"
         izz="0.00106684454111778" />
     </inertial>
@@ -86,9 +86,9 @@
   </link>
   <joint
-    name="base-rotation"
+    name="J1"
     type="revolute">
     <origin
       xyz="0 0 0.1795"
-      rpy="1.5708 0 -1.5708" />
+      rpy="1.5707963267949 0 -1.57079632679489" />
     <parent
       link="ArmBase" />
@@ -114,5 +114,5 @@
         ixx="0.000749127415490433"
         ixy="3.9226287616403E-05"
-        ixz="1.68457558241152E-07"
+        ixz="1.68457558241151E-07"
         iyy="0.00521089609335111"
         iyz="-1.840147885579E-06"
@@ -144,9 +144,9 @@
   </link>
   <joint
-    name="shoulder"
-    type="revolute">
-    <origin
-      xyz="0.0933 0.0723 -0.00028711"
-      rpy="1.5708 0 1.5708" />
+    name="J2"
+    type="revolute">
+    <origin
+      xyz="0.0932995582406649 0.0723000000000009 -0.000287109904390681"
+      rpy="1.5707963267949 0 1.5707963267949" />
     <parent
       link="BaseToJ1" />
@@ -154,5 +154,5 @@
       link="J2ToLink1" />
     <axis
-      xyz="0 0 -1" />
+      xyz="0 0.00307727657437369 -0.999995265173233" />
     <limit
       lower="-1.75"
@@ -165,15 +165,15 @@
     <inertial>
       <origin
-        xyz="0.129966189328165 0.0732399519417659 -0.0854948314562504"
-        rpy="0 0 0" />
-      <mass
-        value="1.1537312044344" />
-      <inertia
-        ixx="0.00112066300003786"
-        ixy="7.23793330716904E-05"
-        ixz="-1.74454352298505E-05"
-        iyy="0.00375619318284082"
-        iyz="0.00018874261573622"
-        izz="0.00391910919823574" />
+        xyz="0.129966189327722 0.0732399519418239 -0.0854948314565011"
+        rpy="0 0 0" />
+      <mass
+        value="1.15373120443012" />
+      <inertia
+        ixx="0.00112066300003723"
+        ixy="7.23793330717775E-05"
+        ixz="-1.74454352295001E-05"
+        iyy="0.00375619318284003"
+        iyz="0.00018874261573637"
+        izz="0.00391910919823546" />
     </inertial>
     <visual>
@@ -202,5 +202,5 @@
   </link>
   <joint
-    name="elbow"
+    name="J3"
     type="revolute">
     <origin
@@ -212,5 +212,5 @@
       link="J3ToLink2" />
     <axis
-      xyz="0 0 -1" />
+      xyz="0 0.0030773 -1" />
     <limit
       lower="-2.85"
@@ -223,5 +223,5 @@
     <inertial>
       <origin
-        xyz="-0.000854379754759105 -0.00771635785912597 -0.0386037875911855"
+        xyz="-0.000854379754758439 -0.00771635785912593 -0.0386037875911855"
         rpy="0 0 0" />
       <mass
@@ -229,6 +229,6 @@
       <inertia
         ixx="0.000107515397522057"
-        ixy="-1.35212786806063E-07"
-        ixz="2.57896496508744E-08"
+        ixy="-1.35212786806066E-07"
+        ixz="2.57896496508754E-08"
         iyy="9.97191040148142E-05"
         iyz="1.40048478553512E-06"
@@ -276,5 +276,5 @@
     <inertial>
       <origin
-        xyz="-0.000364137980536139 0.0341611309238566 0.0243774183852719"
+        xyz="-0.000364137980536805 0.0341611309238566 0.0243774183852719"
         rpy="0 0 0" />
       <mass
@@ -282,6 +282,6 @@
       <inertia
         ixx="0.000132808935473041"
-        ixy="-1.6412565053747E-07"
-        ixz="-8.70461792617816E-08"
+        ixy="-1.64125650537469E-07"
+        ixz="-8.70461792617826E-08"
         iyy="0.000109691860796545"
         iyz="-1.48854544793139E-06"
@@ -313,5 +313,5 @@
   </link>
   <joint
-    name="j4"
+    name="J4"
     type="revolute">
     <origin
@@ -323,5 +323,5 @@
       link="J4ToJ5" />
     <axis
-      xyz="0 0 -1" />
+      xyz="0 0.0030773 -1" />
     <limit
       lower="-2.85"
@@ -334,5 +334,5 @@
     <inertial>
       <origin
-        xyz="0.000187662498820879 -0.0176175749877335 0.0215384550975011"
+        xyz="0.000960068820124615 0.0034018297209792 0.0213979775114195"
         rpy="0 0 0" />
       <mass
@@ -340,9 +340,9 @@
       <inertia
         ixx="0.000112193318899533"
-        ixy="-2.61131401507365E-07"
-        ixz="-5.05759999511541E-09"
+        ixy="-2.61131401507366E-07"
+        ixz="-5.05759999511561E-09"
         iyy="0.000121789710790359"
         iyz="-1.61568500189792E-07"
-        izz="9.87854347259817E-05" />
+        izz="9.87854347259818E-05" />
     </inertial>
     <visual>
@@ -371,8 +371,8 @@
   </link>
   <joint
-    name="j5"
-    type="revolute">
-    <origin
-      xyz="8.5143E-05 0.081342 0.02135"
+    name="J5"
+    type="revolute">
+    <origin
+      xyz="0.00022562 0.10236 0.020578"
       rpy="0 -1.5708 0" />
     <parent
@@ -381,5 +381,5 @@
       link="J5ToJ6" />
     <axis
-      xyz="0 -1 0" />
+      xyz="0.0030772 -0.99997 0.0065737" />
     <limit
       lower="-1.88"
@@ -392,15 +392,15 @@
     <inertial>
       <origin
-        xyz="0.0313403405257765 -0.0154054918446249 0.0972054188783789"
-        rpy="0 0 0" />
-      <mass
-        value="0.55463240302887" />
-      <inertia
-        ixx="0.000376073601133984"
-        ixy="-1.35551673721987E-05"
-        ixz="-9.98929456115085E-07"
-        iyy="0.000644904140085136"
-        iyz="1.10813236344385E-05"
-        izz="0.000454272721609693" />
+        xyz="0.0313403405158062 -0.0154054918426727 0.0972054188871159"
+        rpy="0 0 0" />
+      <mass
+        value="0.55463240309873" />
+      <inertia
+        ixx="0.000376073601172609"
+        ixy="-1.35551673726115E-05"
+        ixz="-9.98929458571701E-07"
+        iyy="0.000644904140123714"
+        iyz="1.10813236363224E-05"
+        izz="0.000454272721612088" />
     </inertial>
     <visual>
@@ -429,8 +429,8 @@
   </link>
   <joint
-    name="j6"
-    type="revolute">
-    <origin
-      xyz="0.00018845 -0.020463 0.081623"
+    name="J6"
+    type="revolute">
+    <origin
+      xyz="0.00096086 0.00055601 0.081482"
       rpy="0 0 0" />
     <parent
@@ -439,5 +439,5 @@
       link="J6ToEE" />
     <axis
-      xyz="0 0 1" />
+      xyz="0.0027468 0.0065821 0.99997" />
     <limit
       lower="0"
