Commit message: rover_description: changed references to meshes/urdf in core to rover_description

File: src/ros/rover/rover_description/urdf/depth_camera.xacro (robot description, xacro)
@@ -13,5 +13,5 @@
       <geometry>
         <mesh
-          filename="file:///$(find core)/meshes/d455.STL"
+          filename="file:///$(find rover_description)/meshes/d455.STL"
           scale="0.001 0.001 0.001" />
       </geometry>

File: src/ros/rover/rover_description/urdf/gazebo_ros2_control.xacro (robot description, xacro)
@@ -123,5 +123,5 @@
     <gazebo>
         <plugin filename="libgazebo_ros2_control.so" name="gazebo_ros2_control">
-            <parameters>$(find core)/params/controllers.yaml</parameters>
+            <parameters>$(find rover_description)/params/controllers.yaml</parameters>
         </plugin>
     </gazebo>

File: src/ros/rover/rover_description/urdf/rover.urdf (robot description, URDF)
Before this commit: robot rover, 12 links, 11 joints
Links:
- link back_left_pivot: geometry collision mesh filename=file:///$(find rover_description)/meshes/back_left_pivot.STL; visual mesh filename=file:///$(find rover_description)/meshes/back_left_pivot.STL
- link back_left_wheel: geometry collision mesh filename=file:///$(find rover_description)/meshes/wheel_collision.stl; visual mesh filename=file:///$(find rover_description)/meshes/back_left_wheel.STL
- link back_right_pivot: geometry collision mesh filename=file:///$(find rover_description)/meshes/back_right_pivot.S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; visual mesh filename=file:///$(find rover_description)/meshes/back_right_pivot.S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
- link back_right_wheel: geometry collision mesh filename=file:///$(find rover_description)/meshes/wheel_collision.stl; visual mesh filename=file:///$(find rover_description)/meshes/back_right_wheel.S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
- link chassis: geometry collision mesh filename=file:///$(find rover_description)/meshes/chassis.STL; visual mesh filename=file:///$(find rover_description)/meshes/chassis.STL
- link front_left_pivot: geometry collision mesh filename=file:///$(find rover_description)/meshes/front_left_pivot.S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; visual mesh filename=file:///$(find rover_description)/meshes/front_left_pivot.S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
- link front_left_wheel: geometry collision mesh filename=file:///$(find rover_description)/meshes/wheel_collision.stl; visual mesh filename=file:///$(find rover_description)/meshes/front_left_wheel.S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
- link front_right_pivot: geometry collision mesh filename=file:///$(find rover_description)/meshes/front_right_pivot.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; visual mesh filename=file:///$(find rover_description)/meshes/front_right_pivot.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
- link front_right_wheel: geometry collision mesh filename=file:///$(find rover_description)/meshes/wheel_collision.stl; visual mesh filename=file:///$(find rover_description)/meshes/front_right_wheel.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
- link left_leg: geometry collision mesh filename=file:///$(find rover_description)/meshes/left_leg.STL; visual mesh filename=file:///$(find rover_description)/meshes/left_leg.STL
- link right_leg: geometry collision mesh filename=file:///$(find rover_description)/meshes/right_leg.STL; visual mesh filename=file:///$(find rover_description)/meshes/right_leg.STL

File: src/ros/rover/rover_description/urdf/simple_rover.xacro (robot description, xacro)
@@ -30,5 +30,5 @@
       <geometry>
         <mesh
-          filename="file:///$(find core)/meshes/chassis.STL" />
+          filename="file:///$(find rover_description)/meshes/chassis.STL" />
       </geometry>
       <material
@@ -78,5 +78,5 @@
       <geometry>
         <mesh
-          filename="file:///$(find core)/meshes/left_leg.STL" />
+          filename="file:///$(find rover_description)/meshes/left_leg.STL" />
         <!--cylinder
           radius="0.05"
@@ -95,5 +95,5 @@
       <geometry>
         <!--mesh
-          filename="file:///$(find core)/meshes/left_leg.STL" /-->
+          filename="file:///$(find rover_description)/meshes/left_leg.STL" /-->
         <cylinder
           radius="0.03"
@@ -137,5 +137,5 @@
       <geometry>
         <mesh
-          filename="file:///$(find core)/meshes/front_left_pivot.STL" />
+          filename="file:///$(find rover_description)/meshes/front_left_pivot.STL" />
       </geometry>
       <material
@@ -151,5 +151,5 @@
       <geometry>
         <mesh
-          filename="file:///$(find core)/meshes/front_left_pivot.STL" />
+          filename="file:///$(find rover_description)/meshes/front_left_pivot.STL" />
       </geometry>
     </collision>
@@ -196,5 +196,5 @@
       <geometry>
         <mesh
-          filename="file:///$(find core)/meshes/front_left_wheel.STL" />
+          filename="file:///$(find rover_description)/meshes/front_left_wheel.STL" />
       </geometry>
       <material
@@ -210,5 +210,5 @@
       <geometry>
         <mesh
-          filename="file:///$(find core)/meshes/wheel_collision.stl" />
+          filename="file:///$(find rover_description)/meshes/wheel_collision.stl" />
       </geometry>
     </collision>
@@ -249,5 +249,5 @@
       <geometry>
         <mesh
-          filename="file:///$(find core)/meshes/back_left_pivot.STL" />
+          filename="file:///$(find rover_description)/meshes/back_left_pivot.STL" />
       </geometry>
       <material
@@ -263,5 +263,5 @@
       <geometry>
         <mesh
-          filename="file:///$(find core)/meshes/back_left_pivot.STL" />
+          filename="file:///$(find rover_description)/meshes/back_left_pivot.STL" />
       </geometry>
     </collision>
@@ -308,5 +308,5 @@
       <geometry>
         <mesh
-          filename="file:///$(find core)/meshes/back_left_wheel.STL" />
+          filename="file:///$(find rover_description)/meshes/back_left_wheel.STL" />
       </geometry>
       <material
@@ -322,5 +322,5 @@
       <geometry>
         <mesh
-          filename="file:///$(find core)/meshes/wheel_collision.stl" />
+          filename="file:///$(find rover_description)/meshes/wheel_collision.stl" />
       </geometry>
     </collision>
@@ -361,5 +361,5 @@
       <geometry>
         <mesh
-          filename="file:///$(find core)/meshes/right_leg.STL" />
+          filename="file:///$(find rover_description)/meshes/right_leg.STL" />
       </geometry>
       <material
@@ -375,5 +375,5 @@
       <geometry>
         <mesh
-          filename="file:///$(find core)/meshes/right_leg.STL" />
+          filename="file:///$(find rover_description)/meshes/right_leg.STL" />
       </geometry>
     </collision>
@@ -414,5 +414,5 @@
       <geometry>
         <mesh
-          filename="file:///$(find core)/meshes/front_right_pivot.STL" />
+          filename="file:///$(find rover_description)/meshes/front_right_pivot.STL" />
       </geometry>
       <material
@@ -428,5 +428,5 @@
       <geometry>
         <mesh
-          filename="file:///$(find core)/meshes/front_right_pivot.STL" />
+          filename="file:///$(find rover_description)/meshes/front_right_pivot.STL" />
       </geometry>
     </collision>
@@ -473,5 +473,5 @@
       <geometry>
         <mesh
-          filename="file:///$(find core)/meshes/front_right_wheel.STL" />
+          filename="file:///$(find rover_description)/meshes/front_right_wheel.STL" />
       </geometry>
       <material
@@ -487,5 +487,5 @@
       <geometry>
         <mesh
-          filename="file:///$(find core)/meshes/wheel_collision.stl" />
+          filename="file:///$(find rover_description)/meshes/wheel_collision.stl" />
       </geometry>
     </collision>
@@ -526,5 +526,5 @@
       <geometry>
         <mesh
-          filename="file:///$(find core)/meshes/back_right_pivot.STL" />
+          filename="file:///$(find rover_description)/meshes/back_right_pivot.STL" />
       </geometry>
       <material
@@ -540,5 +540,5 @@
       <geometry>
         <mesh
-          filename="file:///$(find core)/meshes/back_right_pivot.STL" />
+          filename="file:///$(find rover_description)/meshes/back_right_pivot.STL" />
       </geometry>
     </collision>
@@ -585,5 +585,5 @@
       <geometry>
         <mesh
-          filename="file:///$(find core)/meshes/back_right_wheel.STL" />
+          filename="file:///$(find rover_description)/meshes/back_right_wheel.STL" />
       </geometry>
       <material
@@ -599,5 +599,5 @@
       <geometry>
         <mesh
-          filename="file:///$(find core)/meshes/wheel_collision.stl" />
+          filename="file:///$(find rover_description)/meshes/wheel_collision.stl" />
       </geometry>
     </collision>

Commit message: rover_description: update gazebo depth camera to match oak

File: src/ros/rover/rover_description/urdf/depth_camera.xacro (robot description, xacro)
@@ -3,4 +3,5 @@
 which is how it gets added to the gazebo sim. Author/s: Victor Bartlinski-->
 <robot xmlns:xacro="http://www.ros.org/wiki/xacro" >
+  <link name='camera_link'></link>
   <joint name="camera_joint" type="fixed">
     <origin xyz="0.49 0 0.48" rpy="0 0 0" />
@@ -8,30 +9,18 @@
     <child link="camera_link" />
   </joint>
-  <link name='camera_link'>
-    <visual>
-      <origin xyz="0 0 0" rpy="${pi/2} 0 ${pi/2}" />
-      <geometry>
-        <mesh
-          filename="file:///$(find rover_description)/meshes/d455.STL"
-          scale="0.001 0.001 0.001" />
-      </geometry>
-    </visual>
-  </link>
-  <joint name="camera_frame_joint" type="fixed">
-    <origin xyz="0 0 0" rpy="${-pi/2} 0 ${-pi/2}" />
-    <parent link="camera_link" />
-    <child link="camera_link_frame" />
-  </joint>
-  <link name="camera_link_frame"></link>
-  <gazebo reference="camera_link">
-    <sensor type="depth" name="camera">
+  <xacro:include filename="$(find depthai_descriptions)/urdf/include/depthai_macro.urdf.xacro"/>
+  <xacro:depthai_camera camera_name = "oak" parent = "camera_link" camera_model = "OAK-D-LR"
+   base_frame = "oak-d_frame" cam_pos_x = "0.0" cam_pos_y = "0.0" cam_pos_z = "0.0"
+   cam_roll = "0.0" cam_pitch = "0.0" cam_yaw = "0.0"/>
+  <gazebo reference="oak_rgb_camera_frame">
+    <sensor type="depth" name="oak">
       <pose>0 0 0 0 0 0</pose>
       <visualize>true</visualize>
-      <update_rate>10</update_rate>
+      <update_rate>5</update_rate>
       <camera>
-        <horizontal_fov>${radians(87)}</horizontal_fov>
+        <horizontal_fov>${radians(82)}</horizontal_fov>
         <image>
-          <width>1280</width>
-          <height>720</height>
+          <width>600</width>
+          <height>400</height>
           <format>B8G8R8</format>
         </image>
@@ -42,7 +31,19 @@
       </camera>
       <plugin name="camera_controller" filename="libgazebo_ros_camera.so">
-        <frame_name>camera_link_frame</frame_name>
-        <min_depth>0.6</min_depth>
-        <max_depth>6.0</max_depth>
+        <frame_name>oak_rgb_camera_frame</frame_name>
+            <ros>
+              <remapping>/oak/image_raw:=/oak/rgb/image_raw</remapping>
+              <remapping>/oak/image_raw/compressed:=/oak/rgb/image_raw/compressed</remapping>
+              <remapping>/oak/image_raw/compressedDepth:=/oak/rgb/image_raw/compressedDepth</remapping>
+              <remapping>/oak/image_raw/theora:=/oak/rgb/image_raw/theora</remapping>
+              <remapping>/oak/camera_info:=/oak/rgb/camera_info</remapping>
+              <remapping>/oak/depth/image_raw:=/oak/stereo/image_raw</remapping>
+              <remapping>/oak/depth/image_raw/compressed:=/oak/stereo/image_raw/compressed</remapping>
+              <remapping>/oak/depth/image_raw/compressedDepth:=/oak/stereo/image_raw/compressedDepth</remapping>
+              <remapping>/oak/depth/image_raw/theora:=/oak/depth/image_raw/theora</remapping>
+              <remapping>/oak/depth/camera_info:=/oak/stereo/camera_info</remapping>
+            </ros>
+        <min_depth>0.3</min_depth>
+        <max_depth>12.0</max_depth>
       </plugin>
     </sensor>

Commit message: rover_description: add imu to depth cameras, fix depth_camera plugin frame

File: src/ros/rover/rover_description/urdf/depth_camera.xacro (robot description, xacro)
@@ -31,5 +31,5 @@
       </camera>
       <plugin name="camera_controller" filename="libgazebo_ros_camera.so">
-        <frame_name>oak_rgb_camera_frame</frame_name>
+        <frame_name>oak_rgb_camera_optical_frame</frame_name>
             <ros>
               <remapping>/oak/image_raw:=/oak/rgb/image_raw</remapping>
@@ -49,3 +49,71 @@
     </sensor>
   </gazebo>
+  <gazebo reference="oak_imu_frame">
+    <sensor name="imu_sensor" type="imu">
+    <plugin filename="libgazebo_ros_imu_sensor.so" name="imu_plugin">
+    <frame_name>oak_imu_frame</frame_name>
+        <ros>
+          <remapping>~/out:=/oak/imu/data</remapping>
+        </ros>
+        <initial_orientation_as_reference>false</initial_orientation_as_reference>
+      </plugin>
+      <always_on>true</always_on>
+      <update_rate>100</update_rate>
+      <visualize>true</visualize>
+      <imu>
+        <angular_velocity>
+          <x>
+            <noise type="gaussian">
+              <mean>0.0</mean>
+              <stddev>2e-4</stddev>
+              <bias_mean>0.0000075</bias_mean>
+              <bias_stddev>0.0000008</bias_stddev>
+            </noise>
+          </x>
+          <y>
+            <noise type="gaussian">
+              <mean>0.0</mean>
+              <stddev>2e-4</stddev>
+              <bias_mean>0.0000075</bias_mean>
+              <bias_stddev>0.0000008</bias_stddev>
+            </noise>
+          </y>
+          <z>
+            <noise type="gaussian">
+              <mean>0.0</mean>
+              <stddev>2e-4</stddev>
+              <bias_mean>0.0000075</bias_mean>
+              <bias_stddev>0.0000008</bias_stddev>
+            </noise>
+          </z>
+        </angular_velocity>
+        <linear_acceleration>
+          <x>
+            <noise type="gaussian">
+              <mean>0.0</mean>
+              <stddev>1.7e-2</stddev>
+              <bias_mean>0.1</bias_mean>
+              <bias_stddev>0.001</bias_stddev>
+            </noise>
+          </x>
+          <y>
+            <noise type="gaussian">
+              <mean>0.0</mean>
+              <stddev>1.7e-2</stddev>
+              <bias_mean>0.1</bias_mean>
+              <bias_stddev>0.001</bias_stddev>
+            </noise>
+          </y>
+          <z>
+            <noise type="gaussian">
+              <mean>0.0</mean>
+              <stddev>1.7e-2</stddev>
+              <bias_mean>0.1</bias_mean>
+              <bias_stddev>0.001</bias_stddev>
+            </noise>
+          </z>
+        </linear_acceleration>
+      </imu>
+    </sensor>
+  </gazebo>
 </robot>

File: src/ros/rover/rover_description/urdf/imu.xacro (robot description, xacro)
@@ -3,21 +3,4 @@
 which is how it gets added to the gazebo sim. Author/s: Max Tory -->
 <robot xmlns:xacro="http://www.ros.org/wiki/xacro" >
-  <link name="imu_link">
-    <visual>
-      <geometry>
-        <box size="0.065 0.08 0.04"/>
-      </geometry>
-    </visual>
-    <collision>
-      <geometry>
-        <box size="0.1 0.1 0.1"/>
-      </geometry>
-    </collision>
-  </link>
-  <joint name="imu_joint" type="fixed">
-    <parent link="base_link"/>
-    <child link="imu_link"/>
-    <origin xyz="0.04 0.26 0.445"/>
-  </joint>
   <gazebo reference="imu_link">
     <sensor name="imu_sensor" type="imu">

File: src/ros/rover/rover_description/urdf/rover.urdf.xacro (robot description, xacro)
@@ -622,5 +622,4 @@
   <xacro:include filename="depth_camera.xacro" />
   <xacro:include filename="p3d.xacro" />
-  <xacro:include filename="imu.xacro" />
   <xacro:include filename="gps.xacro" />
 </robot>

Commit message: parameters the same as navigation2_tutorial

File: src/ros/rover/rover_description/urdf/depth_camera.xacro (robot description, xacro)
@@ -49,8 +49,8 @@
     </sensor>
   </gazebo>
-  <gazebo reference="oak_imu_frame">
+  <gazebo reference="base_link">
     <sensor name="imu_sensor" type="imu">
     <plugin filename="libgazebo_ros_imu_sensor.so" name="imu_plugin">
-    <frame_name>oak_imu_frame</frame_name>
+    <frame_name>base_link</frame_name>
         <ros>
           <remapping>~/out:=/oak/imu/data</remapping>
@@ -59,5 +59,5 @@
       </plugin>
       <always_on>true</always_on>
-      <update_rate>100</update_rate>
+      <update_rate>200</update_rate>
       <visualize>true</visualize>
       <imu>

File: src/ros/rover/rover_description/urdf/gps.xacro (robot description, xacro)
@@ -3,9 +3,25 @@
 which is how it gets added to the gazebo sim. Author/s: Dylan Gonzalez-->
 <robot xmlns:xacro="http://www.ros.org/wiki/xacro" >
-  <link name="gps" />
+  <link name="gps">
+    <!--
+    <inertial>
+      <pose>-0.052 0 0.111 0 0 0</pose>
+      <inertia>
+        <mass>0.001</mass>
+        <ixx>0.001</ixx>
+        <ixy>0.000</ixy>
+        <ixz>0.000</ixz>
+        <iyy>0.001</iyy>
+        <iyz>0.000</iyz>
+        <izz>0.001</izz>
+      </inertia>
+      <mass>0.125</mass>
+    </inertial>
+    -->
+  </link>
   <joint name="gps_joint" type="fixed">
     <parent link="base_link"/>
     <child link="gps"/>
-    <origin xyz="0.04 -0.26 0.614"/> <!-- copied from imu.xacro -->
+    <origin xyz="0.04 -0.26 0.614" rpy="0 0 0"/> <!-- copied from imu.xacro -->
   </joint>
   <gazebo reference="gps">
@@ -17,5 +33,5 @@
       </plugin>
       <always_on>true</always_on>
-      <update_rate>5</update_rate>
+      <update_rate>1</update_rate>
       <pose>0 0 0 0 0 0</pose>
       <gps>
