Commit message: reformatted gazebo_ros2_control xacro file

File: src/ros/rover/rover_description/urdf/gazebo_ros2_control.xacro (robot description, xacro)
@@ -1,128 +1,128 @@
 <?xml version="1.0" encoding="utf-8"?>
 <robot xmlns:xacro="http://www.ros.org/wiki/xacro">
-    <ros2_control name="GazeboSimSystem" type="system">
-        <hardware>
-            <plugin>gz_ros2_control/GazeboSimSystem</plugin>
-        </hardware>
-        <joint name='flw'>
-            <command_interface name="velocity">
-                <param name="min">-50</param>
-                <param name="max">50</param>
-            </command_interface>
-            <state_interface name="velocity">
-              <param name="initial_value">0.0</param>
-            </state_interface>
-            <state_interface name="position">
-              <param name="initial_value">0.0</param>
-            </state_interface>
-        </joint>
-        <joint name='frw'>
-            <command_interface name="velocity">
-                <param name="min">-50</param>
-                <param name="max">50</param>
-            </command_interface>
-            <state_interface name="velocity">
-              <param name="initial_value">0.0</param>
-            </state_interface>
-            <state_interface name="velocity">
-              <param name="initial_value">0.0</param>
-            </state_interface>
-            <state_interface name="position">
-              <param name="initial_value">0.0</param>
-            </state_interface>
-        </joint>
-        <joint name='blw'>
-            <command_interface name="velocity">
-                <param name="min">-50</param>
-                <param name="max">50</param>
-            </command_interface>
-            <state_interface name="velocity">
-              <param name="initial_value">0.0</param>
-            </state_interface>
-            <state_interface name="position">
-              <param name="initial_value">0.0</param>
-            </state_interface>
-        </joint>
-        <joint name='brw'>
-            <command_interface name="velocity">
-                <param name="min">-50</param>
-                <param name="max">50</param>
-            </command_interface>
-            <state_interface name="velocity">
-              <param name="initial_value">0.0</param>
-            </state_interface>
-            <state_interface name="position">
-              <param name="initial_value">0.0</param>
-            </state_interface>
-        </joint>
-        <joint name="flp">
-            <command_interface name="position">
-                <param name="min">-${pi}</param>
-                <param name="max">${pi}</param>
-            </command_interface>
-            <command_interface name="velocity">
-                <param name="min">-${pi}</param>
-                <param name="max">${pi}</param>
-            </command_interface>
-            <state_interface name="velocity">
-              <param name="initial_value">0.0</param>
-            </state_interface>
-            <state_interface name="position">
-              <param name="initial_value">0.0</param>
-            </state_interface>
-        </joint>
-        <joint name="frp">
-            <command_interface name="position">
-                <param name="min">-${pi}</param>
-                <param name="max">${pi}</param>
-            </command_interface>
-            <command_interface name="velocity">
-                <param name="min">-${pi}</param>
-                <param name="max">${pi}</param>
-            </command_interface>
-            <state_interface name="velocity">
-              <param name="initial_value">0.0</param>
-            </state_interface>
-            <state_interface name="position">
-              <param name="initial_value">0.0</param>
-            </state_interface>
-        </joint>
-        <joint name="blp">
-            <command_interface name="position">
-                <param name="min">-${pi}</param>
-                <param name="max">${pi}</param>
-            </command_interface>
-            <command_interface name="velocity">
-                <param name="min">-${pi}</param>
-                <param name="max">${pi}</param>
-            </command_interface>
-            <state_interface name="velocity">
-              <param name="initial_value">0.0</param>
-            </state_interface>
-            <state_interface name="position">
-              <param name="initial_value">0.0</param>
-            </state_interface>
-        </joint>
-        <joint name="brp">
-            <command_interface name="position">
-                <param name="min">-${pi}</param>
-                <param name="max">${pi}</param>
-            </command_interface>
-            <command_interface name="velocity">
-                <param name="min">-${pi}</param>
-                <param name="max">${pi}</param>
-            </command_interface>
-            <state_interface name="velocity">
-              <param name="initial_value">0.0</param>
-            </state_interface>
-            <state_interface name="position">
-              <param name="initial_value">0.0</param>
-            </state_interface>
-        </joint>
-    </ros2_control>
-    <gazebo>
-        <plugin filename="libgz_ros2_control-system" name="gz_ros2_control::GazeboSimROS2ControlPlugin">
-            <parameters>$(find auto_bringup)/params/controllers.yaml</parameters>
-        </plugin>
-    </gazebo>
+  <ros2_control name="GazeboSimSystem" type="system">
+    <hardware>
+      <plugin>gz_ros2_control/GazeboSimSystem</plugin>
+    </hardware>
+    <joint name='flw'>
+      <command_interface name="velocity">
+        <param name="min">-50</param>
+        <param name="max">50</param>
+      </command_interface>
+      <state_interface name="velocity">
+        <param name="initial_value">0.0</param>
+      </state_interface>
+      <state_interface name="position">
+        <param name="initial_value">0.0</param>
+      </state_interface>
+    </joint>
+    <joint name='frw'>
+      <command_interface name="velocity">
+        <param name="min">-50</param>
+        <param name="max">50</param>
+      </command_interface>
+      <state_interface name="velocity">
+        <param name="initial_value">0.0</param>
+      </state_interface>
+      <state_interface name="velocity">
+        <param name="initial_value">0.0</param>
+      </state_interface>
+      <state_interface name="position">
+        <param name="initial_value">0.0</param>
+      </state_interface>
+    </joint>
+    <joint name='blw'>
+      <command_interface name="velocity">
+        <param name="min">-50</param>
+        <param name="max">50</param>
+      </command_interface>
+      <state_interface name="velocity">
+        <param name="initial_value">0.0</param>
+      </state_interface>
+      <state_interface name="position">
+        <param name="initial_value">0.0</param>
+      </state_interface>
+    </joint>
+    <joint name='brw'>
+      <command_interface name="velocity">
+        <param name="min">-50</param>
+        <param name="max">50</param>
+      </command_interface>
+      <state_interface name="velocity">
+        <param name="initial_value">0.0</param>
+      </state_interface>
+      <state_interface name="position">
+        <param name="initial_value">0.0</param>
+      </state_interface>
+    </joint>
+    <joint name="flp">
+      <command_interface name="position">
+        <param name="min">-${pi}</param>
+        <param name="max">${pi}</param>
+      </command_interface>
+      <command_interface name="velocity">
+        <param name="min">-${pi}</param>
+        <param name="max">${pi}</param>
+      </command_interface>
+      <state_interface name="velocity">
+        <param name="initial_value">0.0</param>
+      </state_interface>
+      <state_interface name="position">
+        <param name="initial_value">0.0</param>
+      </state_interface>
+    </joint>
+    <joint name="frp">
+      <command_interface name="position">
+        <param name="min">-${pi}</param>
+        <param name="max">${pi}</param>
+      </command_interface>
+      <command_interface name="velocity">
+        <param name="min">-${pi}</param>
+        <param name="max">${pi}</param>
+      </command_interface>
+      <state_interface name="velocity">
+        <param name="initial_value">0.0</param>
+      </state_interface>
+      <state_interface name="position">
+        <param name="initial_value">0.0</param>
+      </state_interface>
+    </joint>
+    <joint name="blp">
+      <command_interface name="position">
+        <param name="min">-${pi}</param>
+        <param name="max">${pi}</param>
+      </command_interface>
+      <command_interface name="velocity">
+        <param name="min">-${pi}</param>
+        <param name="max">${pi}</param>
+      </command_interface>
+      <state_interface name="velocity">
+        <param name="initial_value">0.0</param>
+      </state_interface>
+      <state_interface name="position">
+        <param name="initial_value">0.0</param>
+      </state_interface>
+    </joint>
+    <joint name="brp">
+      <command_interface name="position">
+        <param name="min">-${pi}</param>
+        <param name="max">${pi}</param>
+      </command_interface>
+      <command_interface name="velocity">
+        <param name="min">-${pi}</param>
+        <param name="max">${pi}</param>
+      </command_interface>
+      <state_interface name="velocity">
+        <param name="initial_value">0.0</param>
+      </state_interface>
+      <state_interface name="position">
+        <param name="initial_value">0.0</param>
+      </state_interface>
+    </joint>
+  </ros2_control>
+  <gazebo>
+      <plugin filename="libgz_ros2_control-system" name="gz_ros2_control::GazeboSimROS2ControlPlugin">
+          <parameters>$(find auto_bringup)/params/controllers.yaml</parameters>
+      </plugin>
+  </gazebo>
 </robot>
