Commit message: fixed pivot drive controller integration with gazebo

File: src/ros/rover/rover_description/urdf/gz_ros2_control.xacro (robot description, xacro)
@@ -22,7 +22,4 @@
         <param name="max">50</param>
       </command_interface>
-      <state_interface name="velocity">
-        <param name="initial_value">0.0</param>
-      </state_interface>
       <state_interface name="velocity">
         <param name="initial_value">0.0</param>
@@ -122,7 +119,7 @@
   </ros2_control>
   <gazebo>
-      <plugin filename="libgz_ros2_control-system" name="gz_ros2_control::GazeboSimROS2ControlPlugin">
-          <parameters>$(find auto_bringup)/params/controllers.yaml</parameters>
-      </plugin>
+    <plugin filename="gz_ros2_control-system" name="gz_ros2_control::GazeboSimROS2ControlPlugin">
+        <parameters>$(find auto_bringup)/params/controllers.yaml</parameters>
+    </plugin>
   </gazebo>
 </robot>

File: src/ros/rover/rover_description/urdf/rover.urdf.xacro (robot description, xacro)
@@ -40,7 +40,4 @@
     </inertial>
     <visual>
-      <origin
-        xyz="0 0 0"
-        rpy="0 0 0" />
       <geometry>
         <mesh
@@ -53,13 +50,4 @@
       </material>
     </visual>
-    <collision>
-      <origin
-        xyz="0 0 0"
-        rpy="0 0 0" />
-      <geometry>
-        <mesh
-          filename="file://$(find rover_description)/meshes/chassis.STL" />
-      </geometry>
-    </collision>
   </link>
   <!-- Positions the chassis mesh in space relative to the wheel base -->
@@ -97,7 +85,4 @@
     </inertial>
     <visual>
-      <origin
-        xyz="0 0 0"
-        rpy="0 0 0" />
       <geometry>
         <mesh
@@ -110,13 +95,4 @@
       </material>
     </visual>
-    <collision>
-      <origin
-        xyz="0 0 0"
-        rpy="0 0 0" />
-      <geometry>
-        <mesh
-          filename="file://$(find rover_description)/meshes/left_leg.STL" />
-      </geometry>
-    </collision>
   </link>
   <joint
@@ -150,7 +126,4 @@
     </inertial>
     <visual>
-      <origin
-        xyz="0 0 0"
-        rpy="0 0 0" />
       <geometry>
         <mesh
@@ -163,13 +136,4 @@
       </material>
     </visual>
-    <collision>
-      <origin
-        xyz="0 0 0"
-        rpy="0 0 0" />
-      <geometry>
-        <mesh
-          filename="file://$(find rover_description)/meshes/front_left_pivot.STL" />
-      </geometry>
-    </collision>
   </link>
   <joint
@@ -188,7 +152,6 @@
       lower="-3.141592654"
       upper="3.141592654"
-      effort="1"
+      effort="20"
       velocity="1" />
-    <dynamics damping="10.0" friction="10.0"/>
   </joint>
   <link
@@ -209,7 +172,4 @@
     </inertial>
     <visual>
-      <origin
-        xyz="0 0 0"
-        rpy="0 0 0" />
       <geometry>
         <mesh
@@ -223,7 +183,4 @@
     </visual>
     <collision>
-      <origin
-        xyz="0 0 0"
-        rpy="0 0 0" />
       <geometry>
         <mesh
@@ -262,7 +219,4 @@
     </inertial>
     <visual>
-      <origin
-        xyz="0 0 0"
-        rpy="0 0 0" />
       <geometry>
         <mesh
@@ -275,20 +229,7 @@
       </material>
     </visual>
-    <collision>
-      <origin
-        xyz="0 0 0"
-        rpy="0 0 0" />
-      <geometry>
-        <mesh
-          filename="file://$(find rover_description)/meshes/back_left_pivot.STL" />
-      </geometry>
-    </collision>
-  </link>
-  <joint
-    name="blp"
-    type="revolute">
-    <origin
-      xyz="-0.0093548 0.20893 0.87956"
-      rpy="0.10777 0.18 1.5292" />
+  </link>
+  <joint name="blp" type="revolute">
+    <origin xyz="-0.0093548 0.20893 0.87956" rpy="0.10777 0.18 1.5292" />
     <parent
       link="left_leg" />
@@ -297,10 +238,8 @@
     <axis
       xyz="0 1 0" />
-    <limit
-      lower="-3.141592654"
+    <limit lower="-3.141592654"
       upper="3.141592654"
-      effort="1"
+      effort="20"
       velocity="1" />
-    <dynamics damping="10.0" friction="10.0"/>
   </joint>
   <link
@@ -321,7 +260,4 @@
     </inertial>
     <visual>
-      <origin
-        xyz="0 0 0"
-        rpy="0 0 0" />
       <geometry>
         <mesh
@@ -335,7 +271,4 @@
     </visual>
     <collision>
-      <origin
-        xyz="0 0 0"
-        rpy="0 0 0" />
       <geometry>
         <mesh
@@ -374,7 +307,4 @@
     </inertial>
     <visual>
-      <origin
-        xyz="0 0 0"
-        rpy="0 0 0" />
       <geometry>
         <mesh
@@ -387,13 +317,4 @@
       </material>
     </visual>
-    <collision>
-      <origin
-        xyz="0 0 0"
-        rpy="0 0 0" />
-      <geometry>
-        <mesh
-          filename="file://$(find rover_description)/meshes/right_leg.STL" />
-      </geometry>
-    </collision>
   </link>
   <joint
@@ -427,7 +348,4 @@
     </inertial>
     <visual>
-      <origin
-        xyz="0 0 0"
-        rpy="0 0 0" />
       <geometry>
         <mesh
@@ -440,13 +358,4 @@
       </material>
     </visual>
-    <collision>
-      <origin
-        xyz="0 0 0"
-        rpy="0 0 0" />
-      <geometry>
-        <mesh
-          filename="file://$(find rover_description)/meshes/front_right_pivot.STL" />
-      </geometry>
-    </collision>
   </link>
   <joint
@@ -465,7 +374,6 @@
       lower="-3.141592654"
       upper="3.141592654"
-      effort="1"
+      effort="20"
       velocity="1" />
-    <dynamics damping="10.0" friction="10.0"/>
   </joint>
   <link
@@ -486,7 +394,4 @@
     </inertial>
     <visual>
-      <origin
-        xyz="0 0 0"
-        rpy="0 0 0" />
       <geometry>
         <mesh
@@ -500,7 +405,4 @@
     </visual>
     <collision>
-      <origin
-        xyz="0 0 0"
-        rpy="0 0 0" />
       <geometry>
         <mesh
@@ -539,7 +441,4 @@
     </inertial>
     <visual>
-      <origin
-        xyz="0 0 0"
-        rpy="0 0 0" />
       <geometry>
         <mesh
@@ -552,13 +451,4 @@
       </material>
     </visual>
-    <collision>
-      <origin
-        xyz="0 0 0"
-        rpy="0 0 0" />
-      <geometry>
-        <mesh
-          filename="file://$(find rover_description)/meshes/back_right_pivot.STL" />
-      </geometry>
-    </collision>
   </link>
   <joint
@@ -577,7 +467,6 @@
       lower="-3.141592654"
       upper="3.141592654"
-      effort="1"
+      effort="20"
       velocity="1" />
-    <dynamics damping="10.0" friction="10.0"/>
   </joint>
   <link
@@ -598,7 +487,4 @@
     </inertial>
     <visual>
-      <origin
-        xyz="0 0 0"
-        rpy="0 0 0" />
       <geometry>
         <mesh
@@ -612,7 +498,4 @@
     </visual>
     <collision>
-      <origin
-        xyz="0 0 0"
-        rpy="0 0 0" />
       <geometry>
         <mesh
@@ -635,5 +518,5 @@
   </joint>
   <xacro:if value="$(arg gazebo)">
-    <xacro:include filename="$(find rover_description)/urdf/gazebo_ros2_control.xacro" />
+    <xacro:include filename="$(find rover_description)/urdf/gz_ros2_control.xacro" />
   </xacro:if>
   <xacro:if value="$(arg arm)">
