Commit message: fieldtest updates

File: src/ros/rover/rover_description/urdf/gps.xacro (robot description, xacro)
@@ -3,4 +3,5 @@
 which is how it gets added to the gazebo sim. Author/s: Dylan Gonzalez-->
 <robot xmlns:xacro="http://www.ros.org/wiki/xacro" >
+<<<<<<< Updated upstream
   <link name="gps_link" />
   <joint name="gps_joint" type="fixed">
@@ -10,4 +11,13 @@
   </joint>
   <gazebo reference="gps_link">
+=======
+  <link name="gps" />
+  <joint name="gps_joint" type="fixed">
+    <parent link="base_link"/>
+    <child link="gps"/>
+    <origin xyz="0.04 -0.26 0.614"/> <!-- copied from imu.xacro -->
+  </joint>
+  <gazebo reference="gps">
+>>>>>>> Stashed changes
     <sensor name="skytraq_gps" type="gps">
       <plugin filename="libgazebo_ros_gps_sensor.so" name="gps_plugin">

Commit message: fieldtest updates

File: src/ros/rover/rover_description/urdf/gps.xacro (robot description, xacro)
@@ -3,13 +3,4 @@
 which is how it gets added to the gazebo sim. Author/s: Dylan Gonzalez-->
 <robot xmlns:xacro="http://www.ros.org/wiki/xacro" >
-<<<<<<< Updated upstream
-  <link name="gps_link" />
-  <joint name="gps_joint" type="fixed">
-    <parent link="base_link"/>
-    <child link="gps_link"/>
-    <origin xyz="0.04 -0.26 0.614"/> <!-- copied from imu.xacro -->
-  </joint>
-  <gazebo reference="gps_link">
-=======
   <link name="gps" />
   <joint name="gps_joint" type="fixed">
@@ -19,5 +10,4 @@
   </joint>
   <gazebo reference="gps">
->>>>>>> Stashed changes
     <sensor name="skytraq_gps" type="gps">
       <plugin filename="libgazebo_ros_gps_sensor.so" name="gps_plugin">

Commit message: Merge branch 'master' into feat/battery-gui

File: src/ros/rover/rover_description/urdf/gps.xacro (robot description, xacro)
@@ -23,16 +23,15 @@
     <parent link="base_link"/>
     <child link="gps"/>
-    <origin xyz="0.04 -0.26 0.614" rpy="0 0 0"/> <!-- copied from imu.xacro -->
+    <origin xyz="0.04 -0.26 0.614" rpy="0 0 0"/>
   </joint>
   <gazebo reference="gps">
     <sensor name="skytraq_gps" type="gps">
-      <plugin filename="libgazebo_ros_gps_sensor.so" name="gps_plugin">
-        <ros>
-          <remapping>~/out:=/fix</remapping>
-        </ros>
+      <topic>gps</topic>
+      <plugin
+        filename="gz-sim-navsat-system"
+        name="gz::sim::systems::NavSat">
       </plugin>
       <always_on>true</always_on>
       <update_rate>1</update_rate>
-      <pose>0 0 0 0 0 0</pose>
       <gps>
         <position_sensing>

File: src/ros/rover/rover_description/urdf/p3d.xacro (robot description, xacro)
@@ -4,12 +4,8 @@
 <robot xmlns:xacro="http://www.ros.org/wiki/xacro" >
   <gazebo>
-    <plugin name="gazebo_ros_p3d" filename="libgazebo_ros_p3d.so">
-      <ros>
-        <remapping>odom:=odom/gazebo</remapping>
-      </ros>
+    <plugin name="gz::sim::systems::PosePublisher" filename="gz-sim-pose-publisher-system">
       <body_name>base_link</body_name>
       <frame_name>odom</frame_name>
-      <update_rate>30</update_rate>
-      <!-- <gaussian_noise>0.05</gaussian_noise> -->
+      <update_frequency>30</update_frequency>
     </plugin>
   </gazebo>
