Commit message: Squashed commit of the following:
commit acbfda0be7e85d624c2e02d3c67386ac57eea039
Author: Dylan Gonzalez <dylcg10@gmail.com>
Date:   Tue May 14 01:36:41 2024 +1000

    add mast

commit adad26c5e381e0c2762d60865cd5981ec58c1f14
Author: novarover <novaroverteam-projectmanager@monash.edu>
Date:   Tue May 14 01:16:42 2024 +1000

    add joint state publisher aggregator node

commit 7141ef67feec09287dbfd900a5d5f2dfbb349b57
Author: Dylan Gonzalez <dylcg10@gmail.com>
Date:   Mon May 13 23:06:23 2024 +1000

    set wrist_cycloidal joint names

commit 7a4ae9f1c3b49025b15fb24f0ebf33862c2ca118
Author: Dylan Gonzalez <dylcg10@gmail.com>
Date:   Mon May 13 23:06:15 2024 +1000

    stop using arm namespace

commit 337997bc6741074e118e547cb0b28e56c627a9b1
Author: Dylan Gonzalez <dylcg10@gmail.com>
Date:   Mon May 13 22:35:07 2024 +1000

    fix file prefix url

commit 9370e6da92bc95566cd0e49f5798b83ea5db46ef
Author: Dylan Gonzalez <dylcg10@gmail.com>
Date:   Mon May 13 22:14:56 2024 +1000

    fix launch files

commit 44e3b64e232ee65683d8515cb7e6589bad17a9fc
Author: Dylan Gonzalez <dylcg10@gmail.com>
Date:   Mon May 13 22:14:44 2024 +1000

    fix transform arm_link -> chassis

commit 5bd62d526e1850eceab5955788211fe37ee01193
Author: Dylan Gonzalez <dylcg10@gmail.com>
Date:   Mon May 13 22:14:30 2024 +1000

    update joints to match urdf changes

commit f2dd98ccb7d603a5f11da63f0f06959ba4aad199
Author: Dylan Gonzalez <dylcg10@gmail.com>
Date:   Mon May 13 20:44:21 2024 +1000

    fix urdf joints

commit b07ba742bc3225702e9e3ccef066c9417b80ec4a
Author: Dylan Gonzalez <dylcg10@gmail.com>
Date:   Mon May 13 20:43:25 2024 +1000

    fix launch file bugs

commit 543913b2639cadc420e8cd6fde33919c6c7f61ba
Author: Dylan Gonzalez <dylcg10@gmail.com>
Date:   Mon May 13 15:39:35 2024 +1000

    configure launch files

commit 5009a18a0fe21e3c174974c850b927f58e127519
Author: Dylan Gonzalez <dylcg10@gmail.com>
Date:   Mon May 13 12:13:44 2024 +1000

    add chassis to arm link

commit a9057aef0d35fbb2fad541ad696a7761244cf8d9
Author: Dylan Gonzalez <dylcg10@gmail.com>
Date:   Mon May 13 12:14:02 2024 +1000

    rename arm base link

commit 79544845e6b51498f3c3708f8a7bddfa4cda95fc
Author: Dylan Gonzalez <dylcg10@gmail.com>
Date:   Sun May 12 14:24:06 2024 +1000

    configure launch files - launch urdf from arm launch

commit 5da8cd4946ed90bfd2c554d5feefd34885e523dd
Author: Dylan Gonzalez <dylcg10@gmail.com>
Date:   Sun May 12 14:23:52 2024 +1000

    re-name joints in resolver_publisher

commit 15cc96a4afdaf8481a86c1c11dd22140de1e0186
Author: novarover <novaroverteam-projectmanager@monash.edu>
Date:   Fri May 10 17:30:30 2024 +1000

    rename joints and links - untested

File: src/ros/rover/rover_description/urdf/arm.urdf.xacro (robot description, xacro)
@@ -4,7 +4,9 @@
      For more information, please see http://wiki.ros.org/sw_urdf_exporter -->
 <robot
-  name="URDF_PART_ASSEMBLY_URDFONLY">
-  <link
-    name="ArmBase">
+  name="URDF_PART_ASSEMBLY_URDFONLY"
+  xmlns:xacro="http://www.ros.org/wiki/xacro">
+	<xacro:arg name="prefix" default="arm" />
+  <link
+    name="$(arg prefix)_link">
     <inertial>
       <origin
@@ -27,24 +29,24 @@
       <geometry>
         <mesh
-          filename="file:///$(find rover_description)/meshes/ArmBase.STL" />
-      </geometry>
-      <material
-        name="">
-        <color
-          rgba="0.792156862745098 0.819607843137255 0.933333333333333 1" />
-      </material>
-    </visual>
-    <collision>
-      <origin
-        xyz="0 0 0"
-        rpy="0 0 0" />
-      <geometry>
-        <mesh
-          filename="file:///$(find rover_description)/meshes/ArmBase.STL" />
-      </geometry>
-    </collision>
-  </link>
-  <link
-    name="BaseToJ1">
+          filename="file://$(find rover_description)/meshes/ArmBase.STL" />
+      </geometry>
+      <material
+        name="">
+        <color
+          rgba="0.792156862745098 0.819607843137255 0.933333333333333 1" />
+      </material>
+    </visual>
+    <collision>
+      <origin
+        xyz="0 0 0"
+        rpy="0 0 0" />
+      <geometry>
+        <mesh
+          filename="file://$(find rover_description)/meshes/ArmBase.STL" />
+      </geometry>
+    </collision>
+  </link>
+  <link
+    name="$(arg prefix)_base_to_j1">
     <inertial>
       <origin
@@ -67,24 +69,24 @@
       <geometry>
         <mesh
-          filename="file:///$(find rover_description)/meshes/BaseToJ1.STL" />
-      </geometry>
-      <material
-        name="">
-        <color
-          rgba="0.792156862745098 0.819607843137255 0.933333333333333 1" />
-      </material>
-    </visual>
-    <collision>
-      <origin
-        xyz="0 0 0"
-        rpy="0 0 0" />
-      <geometry>
-        <mesh
-          filename="file:///$(find rover_description)/meshes/BaseToJ1.STL" />
-      </geometry>
-    </collision>
-  </link>
-  <joint
-    name="base-rotation"
+          filename="file://$(find rover_description)/meshes/BaseToJ1.STL" />
+      </geometry>
+      <material
+        name="">
+        <color
+          rgba="0.792156862745098 0.819607843137255 0.933333333333333 1" />
+      </material>
+    </visual>
+    <collision>
+      <origin
+        xyz="0 0 0"
+        rpy="0 0 0" />
+      <geometry>
+        <mesh
+          filename="file://$(find rover_description)/meshes/BaseToJ1.STL" />
+      </geometry>
+    </collision>
+  </link>
+  <joint
+    name="$(arg prefix)_j1"
     type="revolute">
     <origin
@@ -92,7 +94,7 @@
       rpy="1.5707963267949 0 -1.57079632679489" />
     <parent
-      link="ArmBase" />
-    <child
-      link="BaseToJ1" />
+      link="$(arg prefix)_link" />
+    <child
+      link="$(arg prefix)_base_to_j1" />
     <axis
       xyz="0 1 0" />
@@ -104,5 +106,5 @@
   </joint>
   <link
-    name="J2ToLink1">
+    name="$(arg prefix)_j2_to_j3">
     <inertial>
       <origin
@@ -125,24 +127,24 @@
       <geometry>
         <mesh
-          filename="file:///$(find rover_description)/meshes/J2ToLink1.STL" />
-      </geometry>
-      <material
-        name="">
-        <color
-          rgba="0.792156862745098 0.819607843137255 0.933333333333333 1" />
-      </material>
-    </visual>
-    <collision>
-      <origin
-        xyz="0 0 0"
-        rpy="0 0 0" />
-      <geometry>
-        <mesh
-          filename="file:///$(find rover_description)/meshes/J2ToLink1.STL" />
-      </geometry>
-    </collision>
-  </link>
-  <joint
-    name="shoulder"
+          filename="file://$(find rover_description)/meshes/J2ToLink1.STL" />
+      </geometry>
+      <material
+        name="">
+        <color
+          rgba="0.792156862745098 0.819607843137255 0.933333333333333 1" />
+      </material>
+    </visual>
+    <collision>
+      <origin
+        xyz="0 0 0"
+        rpy="0 0 0" />
+      <geometry>
+        <mesh
+          filename="file://$(find rover_description)/meshes/J2ToLink1.STL" />
+      </geometry>
+    </collision>
+  </link>
+  <joint
+    name="$(arg prefix)_j2"
     type="revolute">
     <origin
@@ -150,7 +152,7 @@
       rpy="1.5707963267949 0 1.5707963267949" />
     <parent
-      link="BaseToJ1" />
-    <child
-      link="J2ToLink1" />
+      link="$(arg prefix)_base_to_j1" />
+    <child
+      link="$(arg prefix)_j2_to_j3" />
     <axis
       xyz="0 0 1" />
@@ -162,5 +164,5 @@
   </joint>
   <link
-    name="J3ToLink2">
+    name="$(arg prefix)_j3_to_j4">
     <inertial>
       <origin
@@ -183,24 +185,24 @@
       <geometry>
         <mesh
-          filename="file:///$(find rover_description)/meshes/J3ToLink2.STL" />
-      </geometry>
-      <material
-        name="">
-        <color
-          rgba="0.792156862745098 0.819607843137255 0.933333333333333 1" />
-      </material>
-    </visual>
-    <collision>
-      <origin
-        xyz="0 0 0"
-        rpy="0 0 0" />
-      <geometry>
-        <mesh
-          filename="file:///$(find rover_description)/meshes/J3ToLink2.STL" />
-      </geometry>
-    </collision>
-  </link>
-  <joint
-    name="elbow"
+          filename="file://$(find rover_description)/meshes/J3ToLink2.STL" />
+      </geometry>
+      <material
+        name="">
+        <color
+          rgba="0.792156862745098 0.819607843137255 0.933333333333333 1" />
+      </material>
+    </visual>
+    <collision>
+      <origin
+        xyz="0 0 0"
+        rpy="0 0 0" />
+      <geometry>
+        <mesh
+          filename="file://$(find rover_description)/meshes/J3ToLink2.STL" />
+      </geometry>
+    </collision>
+  </link>
+  <joint
+    name="$(arg prefix)_j3"
     type="revolute">
     <origin
@@ -208,7 +210,7 @@
       rpy="0 0 0" />
     <parent
-      link="J2ToLink1" />
-    <child
-      link="J3ToLink2" />
+      link="$(arg prefix)_j2_to_j3" />
+    <child
+      link="$(arg prefix)_j3_to_j4" />
     <axis
       xyz="0 0 1" />
@@ -220,5 +222,5 @@
   </joint>
   <link
-    name="Link2toFixedJ4">
+    name="$(arg prefix)_j4_to_j4_base">
     <inertial>
       <origin
@@ -241,24 +243,24 @@
       <geometry>
         <mesh
-          filename="file:///$(find rover_description)/meshes/Link2toFixedJ4.STL" />
-      </geometry>
-      <material
-        name="">
-        <color
-          rgba="0.792156862745098 0.819607843137255 0.933333333333333 1" />
-      </material>
-    </visual>
-    <collision>
-      <origin
-        xyz="0 0 0"
-        rpy="0 0 0" />
-      <geometry>
-        <mesh
-          filename="file:///$(find rover_description)/meshes/Link2toFixedJ4.STL" />
-      </geometry>
-    </collision>
-  </link>
-  <joint
-    name="J4_Fixed"
+          filename="file://$(find rover_description)/meshes/Link2toFixedJ4.STL" />
+      </geometry>
+      <material
+        name="">
+        <color
+          rgba="0.792156862745098 0.819607843137255 0.933333333333333 1" />
+      </material>
+    </visual>
+    <collision>
+      <origin
+        xyz="0 0 0"
+        rpy="0 0 0" />
+      <geometry>
+        <mesh
+          filename="file://$(find rover_description)/meshes/Link2toFixedJ4.STL" />
+      </geometry>
+    </collision>
+  </link>
+  <joint
+    name="$(arg prefix)_j4_base"
     type="fixed">
     <origin
@@ -266,12 +268,12 @@
       rpy="0 0 0" />
     <parent
-      link="J3ToLink2" />
-    <child
-      link="Link2toFixedJ4" />
+      link="$(arg prefix)_j3_to_j4" />
+    <child
+      link="$(arg prefix)_j4_to_j4_base" />
     <axis
       xyz="0 0 0" />
   </joint>
   <link
-    name="J4ToJ5">
+    name="$(arg prefix)_j4_to_j5">
     <inertial>
       <origin
@@ -294,24 +296,24 @@
       <geometry>
         <mesh
-          filename="file:///$(find rover_description)/meshes/J4ToJ5.STL" />
-      </geometry>
-      <material
-        name="">
-        <color
-          rgba="0.792156862745098 0.819607843137255 0.933333333333333 1" />
-      </material>
-    </visual>
-    <collision>
-      <origin
-        xyz="0 0 0"
-        rpy="0 0 0" />
-      <geometry>
-        <mesh
-          filename="file:///$(find rover_description)/meshes/J4ToJ5.STL" />
-      </geometry>
-    </collision>
-  </link>
-  <joint
-    name="j4"
+          filename="file://$(find rover_description)/meshes/J4ToJ5.STL" />
+      </geometry>
+      <material
+        name="">
+        <color
+          rgba="0.792156862745098 0.819607843137255 0.933333333333333 1" />
+      </material>
+    </visual>
+    <collision>
+      <origin
+        xyz="0 0 0"
+        rpy="0 0 0" />
+      <geometry>
+        <mesh
+          filename="file://$(find rover_description)/meshes/J4ToJ5.STL" />
+      </geometry>
+    </collision>
+  </link>
+  <joint
+    name="$(arg prefix)_j4"
     type="revolute">
     <origin
@@ -319,7 +321,7 @@
       rpy="0 0 0" />
     <parent
-      link="Link2toFixedJ4" />
-    <child
-      link="J4ToJ5" />
+      link="$(arg prefix)_j4_to_j4_base" />
+    <child
+      link="$(arg prefix)_j4_to_j5" />
     <axis
       xyz="0 0 1" />
@@ -331,5 +333,5 @@
   </joint>
   <link
-    name="J5ToJ6">
+    name="$(arg prefix)_j5_to_j6">
     <inertial>
       <origin
@@ -352,24 +354,24 @@
       <geometry>
         <mesh
-          filename="file:///$(find rover_description)/meshes/J5ToJ6.STL" />
-      </geometry>
-      <material
-        name="">
-        <color
-          rgba="0.792156862745098 0.819607843137255 0.933333333333333 1" />
-      </material>
-    </visual>
-    <collision>
-      <origin
-        xyz="0 0 0"
-        rpy="0 0 0" />
-      <geometry>
-        <mesh
-          filename="file:///$(find rover_description)/meshes/J5ToJ6.STL" />
-      </geometry>
-    </collision>
-  </link>
-  <joint
-    name="j5"
+          filename="file://$(find rover_description)/meshes/J5ToJ6.STL" />
+      </geometry>
+      <material
+        name="">
+        <color
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
File: src/ros/rover/rover_description/urdf/rover.urdf.xacro (robot description, xacro)
@@ -8,6 +8,19 @@
   <xacro:arg name="gazebo" default="false"/>
   <xacro:arg name="use_mock_hardware" default="false"/>
+  <xacro:arg name="arm" default="false"/>
+  <xacro:arg name="depth_camera" default="true"/>
   <!-- Manually added links-->
-  <link name="base_link"></link>
+  <link name="base_link" />
+  <link name="mast_link" >
+    <visual>
+      <origin xyz="0.23 -0.35 0.475" rpy="0 0 0" />
+      <geometry>
+        <cylinder radius="0.01" length="1" />
+      </geometry>
+      <material name="Green">
+        <color rgba="0 1 0 1.0"/>
+      </material>
+    </visual>
+  </link>
   <link
     name="chassis">
@@ -32,5 +45,5 @@
       <geometry>
         <mesh
-          filename="file:///$(find rover_description)/meshes/chassis.STL" />
+          filename="file://$(find rover_description)/meshes/chassis.STL" />
       </geometry>
       <material
@@ -46,5 +59,5 @@
       <geometry>
         <mesh
-          filename="file:///$(find rover_description)/meshes/chassis.STL" />
+          filename="file://$(find rover_description)/meshes/chassis.STL" />
       </geometry>
     </collision>
@@ -57,4 +70,12 @@
         xyz="0. -0. 0.38"
         rpy="0. 0. ${-pi/2}"
+    />
+  </joint>
+  <joint name="mast_to_chassis" type="fixed">
+    <parent link="chassis" />
+    <child link="mast_link" />
+    <origin
+        xyz="0 0 0"
+        rpy="0 0 0"
     />
   </joint>
@@ -81,5 +102,5 @@
       <geometry>
         <mesh
-          filename="file:///$(find rover_description)/meshes/left_leg.STL" />
+          filename="file://$(find rover_description)/meshes/left_leg.STL" />
       </geometry>
       <material
@@ -95,5 +116,5 @@
       <geometry>
         <mesh
-          filename="file:///$(find rover_description)/meshes/left_leg.STL" />
+          filename="file://$(find rover_description)/meshes/left_leg.STL" />
       </geometry>
     </collision>
@@ -134,5 +155,5 @@
       <geometry>
         <mesh
-          filename="file:///$(find rover_description)/meshes/front_left_pivot.STL" />
+          filename="file://$(find rover_description)/meshes/front_left_pivot.STL" />
       </geometry>
       <material
@@ -148,5 +169,5 @@
       <geometry>
         <mesh
-          filename="file:///$(find rover_description)/meshes/front_left_pivot.STL" />
+          filename="file://$(find rover_description)/meshes/front_left_pivot.STL" />
       </geometry>
     </collision>
@@ -193,5 +214,5 @@
       <geometry>
         <mesh
-          filename="file:///$(find rover_description)/meshes/front_left_wheel.STL" />
+          filename="file://$(find rover_description)/meshes/front_left_wheel.STL" />
       </geometry>
       <material
@@ -207,5 +228,5 @@
       <geometry>
         <mesh
-          filename="file:///$(find rover_description)/meshes/wheel_collision.stl" />
+          filename="file://$(find rover_description)/meshes/wheel_collision.stl" />
       </geometry>
     </collision>
@@ -246,5 +267,5 @@
       <geometry>
         <mesh
-          filename="file:///$(find rover_description)/meshes/back_left_pivot.STL" />
+          filename="file://$(find rover_description)/meshes/back_left_pivot.STL" />
       </geometry>
       <material
@@ -260,5 +281,5 @@
       <geometry>
         <mesh
-          filename="file:///$(find rover_description)/meshes/back_left_pivot.STL" />
+          filename="file://$(find rover_description)/meshes/back_left_pivot.STL" />
       </geometry>
     </collision>
@@ -305,5 +326,5 @@
       <geometry>
         <mesh
-          filename="file:///$(find rover_description)/meshes/back_left_wheel.STL" />
+          filename="file://$(find rover_description)/meshes/back_left_wheel.STL" />
       </geometry>
       <material
@@ -319,5 +340,5 @@
       <geometry>
         <mesh
-          filename="file:///$(find rover_description)/meshes/wheel_collision.stl" />
+          filename="file://$(find rover_description)/meshes/wheel_collision.stl" />
       </geometry>
     </collision>
@@ -358,5 +379,5 @@
       <geometry>
         <mesh
-          filename="file:///$(find rover_description)/meshes/right_leg.STL" />
+          filename="file://$(find rover_description)/meshes/right_leg.STL" />
       </geometry>
       <material
@@ -372,5 +393,5 @@
       <geometry>
         <mesh
-          filename="file:///$(find rover_description)/meshes/right_leg.STL" />
+          filename="file://$(find rover_description)/meshes/right_leg.STL" />
       </geometry>
     </collision>
@@ -411,5 +432,5 @@
       <geometry>
         <mesh
-          filename="file:///$(find rover_description)/meshes/front_right_pivot.STL" />
+          filename="file://$(find rover_description)/meshes/front_right_pivot.STL" />
       </geometry>
       <material
@@ -425,5 +446,5 @@
       <geometry>
         <mesh
-          filename="file:///$(find rover_description)/meshes/front_right_pivot.STL" />
+          filename="file://$(find rover_description)/meshes/front_right_pivot.STL" />
       </geometry>
     </collision>
@@ -470,5 +491,5 @@
       <geometry>
         <mesh
-          filename="file:///$(find rover_description)/meshes/front_right_wheel.STL" />
+          filename="file://$(find rover_description)/meshes/front_right_wheel.STL" />
       </geometry>
       <material
@@ -484,5 +505,5 @@
       <geometry>
         <mesh
-          filename="file:///$(find rover_description)/meshes/wheel_collision.stl" />
+          filename="file://$(find rover_description)/meshes/wheel_collision.stl" />
       </geometry>
     </collision>
@@ -523,5 +544,5 @@
       <geometry>
         <mesh
-          filename="file:///$(find rover_description)/meshes/back_right_pivot.STL" />
+          filename="file://$(find rover_description)/meshes/back_right_pivot.STL" />
       </geometry>
       <material
@@ -537,5 +558,5 @@
       <geometry>
         <mesh
-          filename="file:///$(find rover_description)/meshes/back_right_pivot.STL" />
+          filename="file://$(find rover_description)/meshes/back_right_pivot.STL" />
       </geometry>
     </collision>
@@ -582,5 +603,5 @@
       <geometry>
         <mesh
-          filename="file:///$(find rover_description)/meshes/back_right_wheel.STL" />
+          filename="file://$(find rover_description)/meshes/back_right_wheel.STL" />
       </geometry>
       <material
@@ -596,5 +617,5 @@
       <geometry>
         <mesh
-          filename="file:///$(find rover_description)/meshes/wheel_collision.stl" />
+          filename="file://$(find rover_description)/meshes/wheel_collision.stl" />
       </geometry>
     </collision>
@@ -615,4 +636,18 @@
   <xacro:if value="$(arg gazebo)">
     <xacro:include filename="$(find rover_description)/urdf/gazebo_ros2_control.xacro" />
+  </xacro:if>
+  <xacro:if value="$(arg arm)">
+    <xacro:include filename="$(find rover_description)/urdf/arm.urdf.xacro" />
+    <joint
+      name="chassis_to_arm_base"
+      type="fixed">
+      <origin
+        xyz="0 0.15 -0.06"
+        rpy="0 0 1.57"/>
+      <parent
+        link="chassis" />
+      <child
+        link="arm_link" /> <!-- should use a prefix arg instead of hardcoding 'arm' -->
+    </joint>
   </xacro:if>
   <xacro:unless value="$(arg gazebo)">
@@ -620,5 +655,7 @@
     <xacro:rover_ros2_control use_mock_hardware="$(arg use_mock_hardware)"/>
   </xacro:unless>
-  <xacro:include filename="depth_camera.xacro" />
+  <xacro:if value="$(arg depth_camera)">
+    <xacro:include filename="depth_camera.xacro" />
+  </xacro:if>
   <xacro:include filename="p3d.xacro" />
   <xacro:include filename="gps.xacro" />
