Commit message: cleaned up gz plugins, added names, mapped p3d to ROS

File: src/ros/rover/rover_description/urdf/auto_camera.xacro (robot description, xacro)
@@ -15,4 +15,5 @@
   <gazebo reference="oak_rgb_camera_frame">
     <sensor type="depth" name="oak">
+      <topic>oak/depth_image</topic>
       <pose>0 0 0 0 0 0</pose>
       <visualize>true</visualize>
@@ -32,15 +33,4 @@
       <plugin name="gz::sim::systems::Sensors" filename="gz-sim-sensors-system">
         <frame_name>oak_rgb_camera_optical_frame</frame_name>
-            <ros>
-              <remapping>/oak/image_raw:=/oak/rgb/image_rect</remapping>
-              <remapping>/oak/image_raw/compressed:=/oak/rgb/image_raw/compressed</remapping>
-              <remapping>/oak/image_raw/compressedDepth:=/oak/rgb/image_raw/compressedDepth</remapping>
-              <remapping>/oak/image_raw/theora:=/oak/rgb/image_raw/theora</remapping>
-              <remapping>/oak/camera_info:=/oak/rgb/camera_info</remapping>
-              <remapping>/oak/depth/image_raw/compressed:=/oak/stereo/image_raw/compressed</remapping>
-              <remapping>/oak/depth/image_raw/compressedDepth:=/oak/stereo/image_raw/compressedDepth</remapping>
-              <remapping>/oak/depth/image_raw/theora:=/oak/depth/image_raw/theora</remapping>
-              <remapping>/oak/depth/camera_info:=/oak/stereo/camera_info</remapping>
-            </ros>
         <min_depth>0.3</min_depth>
         <max_depth>12.0</max_depth>
@@ -50,9 +40,7 @@
   <gazebo reference="oak_imu_frame">
     <sensor name="imu_sensor" type="imu">
-    <plugin filename="gz-sim-imu-system" name="gz::sim::systems::Imu">
-    <frame_name>oak_imu_frame</frame_name>
-        <ros>
-          <remapping>~/out:=/oak/imu/transformed</remapping>
-        </ros>
+      <topic>oak/imu</topic>
+      <plugin filename="gz-sim-imu-system" name="gz::sim::systems::Imu">
+      <frame_name>oak_imu_frame</frame_name>
         <initial_orientation_as_reference>false</initial_orientation_as_reference>
       </plugin>

File: src/ros/rover/rover_description/urdf/gps.xacro (robot description, xacro)
@@ -23,16 +23,15 @@
     <parent link="base_link"/>
     <child link="gps"/>
-    <origin xyz="0.04 -0.26 0.614" rpy="0 0 0"/> <!-- copied from imu.xacro -->
+    <origin xyz="0.04 -0.26 0.614" rpy="0 0 0"/>
   </joint>
   <gazebo reference="gps">
     <sensor name="skytraq_gps" type="gps">
-      <plugin filename="gz-sim-navsat-system" name="gz::sim::systems::NavSat">
-        <ros>
-          <remapping>~/out:=/fix</remapping>
-        </ros>
+      <topic>gps</topic>
+      <plugin
+        filename="gz-sim-navsat-system"
+        name="gz::sim::systems::NavSat">
       </plugin>
       <always_on>true</always_on>
       <update_rate>1</update_rate>
-      <pose>0 0 0 0 0 0</pose>
       <gps>
         <position_sensing>

File: src/ros/rover/rover_description/urdf/p3d.xacro (robot description, xacro)
@@ -5,11 +5,7 @@
   <gazebo>
     <plugin name="gz::sim::systems::PosePublisher" filename="gz-sim-pose-publisher-system">
-      <ros>
-        <remapping>odom:=odom/gazebo</remapping>
-      </ros>
       <body_name>base_link</body_name>
       <frame_name>odom</frame_name>
-      <update_rate>30</update_rate>
-      <!-- <gaussian_noise>0.05</gaussian_noise> -->
+      <update_frequency>30</update_frequency>
     </plugin>
   </gazebo>

File: src/ros/rover/rover_description/urdf/rover.urdf.xacro (robot description, xacro)
@@ -549,5 +549,5 @@
         name="">
         <color
-          rgba="0.533333333 0.545098039 0.552941176 1" /> />
+          rgba="0.533333333 0.545098039 0.552941176 1" />
       </material>
     </visual>
@@ -656,7 +656,7 @@
   </xacro:unless>
   <xacro:if value="$(arg auto_camera)">
-    <xacro:include filename="auto_camera.xacro" />
+    <xacro:include filename="auto_camera.xacro"/>
   </xacro:if>
-  <xacro:include filename="p3d.xacro" />
-  <xacro:include filename="gps.xacro" />
+  <xacro:include filename="p3d.xacro"/>
+  <xacro:include filename="gps.xacro"/>
 </robot>

Commit message: Fixed location of auto camera

File: src/ros/rover/rover_description/urdf/auto_camera.xacro (robot description, xacro)
@@ -6,5 +6,5 @@
 <!-- Need to be fixed, OR ADD AUTO CAMERA MOUNT to URDF-->
   <joint name="camera_joint" type="fixed">
-    <origin xyz="0 -0.26 0.2" rpy="0 0 -1.57" />
+    <origin xyz="0.26 0 0.2" rpy="0 0 0" />
     <parent link="chassis" />
     <child link="camera_link" />
