Commit message: CKC and ball joints simulation implemented

File: src/ros/rover/rover_description/urdf/ckc.xacro (robot description, xacro)
@@ -1,5 +1,5 @@
 <?xml version="1.0" encoding="utf-8"?>
 <!-- Configure Closed Kinetic Chains for Rover -->
-<robot xmlns:xacro="http://www.ros.org/wiki/xacro" >
+<robot xmlns:xacro="http://www.ros.org/wiki/xacro">
     <xacro:macro name="call_ckc" params="robot_name">
         <gazebo>

File: src/ros/rover/rover_description/urdf/rover.urdf.xacro (robot description, xacro)
@@ -14,5 +14,5 @@
     <xacro:arg name="auto_camera" default="true"/>
     <xacro:arg name="robot_name" default="rover"/>
-    <xacro:arg name="use_diff_ball" default="false"/>
+    <xacro:arg name="use_diff_ball" default="true"/>
     <!-- Robot properties-->
     <gazebo>
@@ -391,5 +391,5 @@
         <child link="rightleg" />
         <axis xyz="0 0 1"/>
-        <limit effort="20" velocity="20" />
+        <limit effort="20" velocity="20" lower="-3.141592654" upper="3.141592654"/>
         <joint_properties friction="0.0"/>
     </joint>
@@ -714,5 +714,5 @@
         <child link="leftleg" />
         <axis xyz="0 0 1"/>
-        <limit effort="20" velocity="20" />
+        <limit effort="20" velocity="20" lower="-3.141592654" upper="3.141592654"/>
         <joint_properties friction="0.0"/>
     </joint>
@@ -827,5 +827,5 @@
         <child link="diffend" />
         <axis xyz="0 0 1"/>
-        <limit effort="1" velocity="20" lower="0" upper="0"/>
+        <limit effort="1" velocity="20" lower="-3.141592654" upper="3.141592654"/>
         <joint_properties friction="0.0"/>
     </joint>
@@ -836,5 +836,5 @@
         <child link="difflinkbottom" />
         <axis xyz="0 0 1"/>
-        <limit effort="1" velocity="20" lower="0" upper="0"/>
+        <limit effort="1" velocity="20" lower="-3.141592654" upper="3.141592654"/>
         <joint_properties friction="0.0"/>
     </joint>
@@ -844,5 +844,5 @@
         <child link="difflinkbody" />
         <axis xyz="0 0 1"/>
-        <limit effort="1" velocity="20" lower="0" upper="0"/>
+        <limit effort="1" velocity="20" lower="-3.141592654" upper="3.141592654"/>
         <joint_properties friction="0.0"/>
     </joint>
@@ -853,5 +853,5 @@
         <child link="difflinktop" />
         <axis xyz="0 0 1"/>
-        <limit effort="1" velocity="20" lower="0" upper="0"/>
+        <limit effort="1" velocity="20" lower="-3.141592654" upper="3.141592654"/>
         <joint_properties friction="0.0"/>
     </joint>
@@ -927,5 +927,5 @@
         <child link="diffend_2" />
         <axis xyz="0 0 1"/>
-        <limit effort="1" velocity="20" lower="0" upper="0"/>
+        <limit effort="1" velocity="20" lower="-3.141592654" upper="3.141592654"/>
         <joint_properties friction="0.0"/>
     </joint>
@@ -936,5 +936,5 @@
         <child link="difflinkbottom_2" />
         <axis xyz="0 0 1"/>
-        <limit effort="1" velocity="20" lower="0" upper="0"/>
+        <limit effort="1" velocity="20" lower="-3.141592654" upper="3.141592654"/>
         <joint_properties friction="0.0"/>
     </joint>
@@ -944,5 +944,5 @@
         <child link="difflinkbody_2" />
         <axis xyz="0 0 1"/>
-        <limit effort="1" velocity="20" lower="0" upper="0"/>
+        <limit effort="1" velocity="20" lower="-3.141592654" upper="3.141592654"/>
         <joint_properties friction="0.0"/>
     </joint>
@@ -953,5 +953,5 @@
         <child link="difflinktop_2" />
         <axis xyz="0 0 1"/>
-        <limit effort="1" velocity="20" lower="0" upper="0"/>
+        <limit effort="1" velocity="20" lower="-3.141592654" upper="3.141592654"/>
         <joint_properties friction="0.0"/>
     </joint>
@@ -962,5 +962,5 @@
         <child link="diffbar" />
         <axis xyz="0 0 1"/>
-        <limit effort="1" velocity="20" lower="0" upper="0"/>
+        <limit effort="1" velocity="20" lower="-3.141592654" upper="3.141592654"/>
         <joint_properties friction="0.0"/>
     </joint>
@@ -981,5 +981,5 @@
             <child link="difflinktop" />
             <axis xyz="0 0 1"/>
-            <limit effort="1" velocity="20" lower="0" upper="0"/>
+            <limit effort="1" velocity="20" lower="-3.141592654" upper="3.141592654"/>
             <joint_properties friction="0.0"/>
         </joint>
@@ -989,5 +989,5 @@
             <child link="difflinktop_2" />
             <axis xyz="0 0 1"/>
-            <limit effort="1" velocity="20" lower="0" upper="0"/>
+            <limit effort="1" velocity="20" lower="-3.141592654" upper="3.141592654"/>
             <joint_properties friction="0.0"/>
         </joint>
@@ -997,5 +997,5 @@
             <child link="diffend" />
             <axis xyz="0 0 1"/>
-            <limit effort="1" velocity="20" lower="0" upper="0"/>
+            <limit effort="1" velocity="20" lower="-3.141592654" upper="3.141592654"/>
             <joint_properties friction="0.0"/>
         </joint>
@@ -1005,5 +1005,5 @@
             <child link="diffend_2" />
             <axis xyz="0 0 1"/>
-            <limit effort="1" velocity="20" lower="0" upper="0"/>
+            <limit effort="1" velocity="20" lower="-3.141592654" upper="3.141592654"/>
             <joint_properties friction="0.0"/>
         </joint>
@@ -1013,5 +1013,5 @@
     <xacro:call_ckc robot_name="$(arg robot_name)"/>
     <xacro:if value="$(arg use_diff_ball)">
-        <xacro:include filename="joints.xacro"/>
+        <xacro:include filename="sim_ball_joints.xacro"/>
     </xacro:if>
     <xacro:if value="$(arg auto_camera)">

File: src/ros/rover/rover_description/urdf/sim_ball_joints.xacro (robot description, xacro)
@@ -21,8 +21,7 @@
         <parent link="diffbar"/>
         <child link="tr_difflink_1"/>
-        <origin xyz="-0.38912669878348526975 0.0080507423534933592046 7.771561172376095783e-16"
-            rpy="1.5453959963367629449 0.84953874853766309094 -1.271352236581491546" />
+        <origin xyz="-0.38912669878348532526 0.0080507423534932481823 7.2164496600635175128e-16" rpy="1.8972013954619286746 0.81245706006717677283 -1.1914339028340867888" />
         <axis xyz="1 0 0"/>
-        <limit effort="20.0" velocity="20.0" lower="-0.2618" upper="0.2618"/> <!-- +/- 15 degrees -->
+        <limit effort="20.0" velocity="20.0" lower="-3.141592654" upper="3.141592654"/>
         <dynamics damping="0.01" friction="0.0"/>
     </joint>
@@ -31,6 +30,4 @@
         <parent link="tr_difflink_1"/>
         <child link="tr_difflink_2"/>
-        <origin xyz="-0.38912669878348526975 0.0080507423534933592046 7.771561172376095783e-16"
-            rpy="1.5453959963367629449 0.84953874853766309094 -1.271352236581491546" />
         <axis xyz="0 1 0"/>
         <limit effort="20.0" velocity="20.0" lower="-0.2618" upper="0.2618"/> <!-- +/- 15 degrees -->
@@ -41,6 +38,4 @@
         <parent link="tr_difflink_2"/>
         <child link="difflinktop_2"/>
-        <origin xyz="-0.38912669878348526975 0.0080507423534933592046 7.771561172376095783e-16"
-            rpy="1.5453959963367629449 0.84953874853766309094 -1.271352236581491546" />
         <axis xyz="0 0 1"/>
         <limit effort="20.0" velocity="20.0" lower="-0.2618" upper="0.2618"/> <!-- +/- 15 degrees -->
@@ -66,8 +61,7 @@
         <parent link="difflinkbottom_2"/>
         <child link="br_difflink_1"/>
-        <origin xyz="-2.7755575615628913511e-17 0 0.030366069404429957279"
-            rpy="-1.8211554193643901822 0.38630147202971765186 1.6973296137818383311" />
+        <origin xyz="-2.2204460492503130808e-16 -2.2204460492503130808e-16 0.030366069404429846257" rpy="1.3580572734639122512 0.40045540725920980574 1.5193397039318303765" />
         <axis xyz="1 0 0"/>
-        <limit effort="20.0" velocity="20.0" lower="-0.2618" upper="0.2618"/> <!-- +/- 15 degrees -->
+        <limit effort="20.0" velocity="20.0" lower="-3.141592654" upper="3.141592654"/>
         <dynamics damping="0.01" friction="0.0"/>
     </joint>
@@ -76,6 +70,4 @@
         <parent link="br_difflink_1"/>
         <child link="br_difflink_2"/>
-        <origin xyz="-2.7755575615628913511e-17 0 0.030366069404429957279"
-            rpy="-1.8211554193643901822 0.38630147202971765186 1.6973296137818383311" />
         <axis xyz="0 1 0"/>
         <limit effort="20.0" velocity="20.0" lower="-0.2618" upper="0.2618"/> <!-- +/- 15 degrees -->
@@ -86,6 +78,4 @@
         <parent link="br_difflink_2"/>
         <child link="diffend_2"/>
-        <origin xyz="-2.7755575615628913511e-17 0 0.030366069404429957279"
-            rpy="-1.8211554193643901822 0.38630147202971765186 1.6973296137818383311" />
         <axis xyz="0 0 1"/>
         <limit effort="20.0" velocity="20.0" lower="-0.2618" upper="0.2618"/> <!-- +/- 15 degrees -->
@@ -111,8 +101,7 @@
         <parent link="difflinkbottom"/>
         <child link="bl_difflink_1"/>
-        <origin xyz="1.6653345369377348106e-16 -1.1102230246251565404e-16 0.03036606940442982544"
-            rpy="1.8137134713184706047 0.40491568475361000568 2.0095824661262473576" />
+        <origin xyz="2.7755575615628913511e-16 4.4408920985006261617e-16 0.03036606940442951319" rpy="-1.3819198339232898753 0.4052315082576601335 1.6592791076415036589" />
         <axis xyz="1 0 0"/>
-        <limit effort="20.0" velocity="20.0" lower="-0.2618" upper="0.2618"/> <!-- +/- 15 degrees -->
+        <limit effort="20.0" velocity="20.0" lower="-3.141592654" upper="3.141592654"/>
         <dynamics damping="0.01" friction="0.0"/>
     </joint>
@@ -121,6 +110,4 @@
         <parent link="bl_difflink_1"/>
         <child link="bl_difflink_2"/>
-        <origin xyz="1.6653345369377348106e-16 -1.1102230246251565404e-16 0.03036606940442982544"
-            rpy="1.8137134713184706047 0.40491568475361000568 2.0095824661262473576" />
         <axis xyz="0 1 0"/>
         <limit effort="20.0" velocity="20.0" lower="-0.2618" upper="0.2618"/> <!-- +/- 15 degrees -->
@@ -131,6 +118,4 @@
         <parent link="bl_difflink_2"/>
         <child link="diffend"/>
-        <origin xyz="1.6653345369377348106e-16 -1.1102230246251565404e-16 0.03036606940442982544"
-            rpy="1.8137134713184706047 0.40491568475361000568 2.0095824661262473576" />
         <axis xyz="0 0 1"/>
         <limit effort="20.0" velocity="20.0" lower="-0.2618" upper="0.2618"/> <!-- +/- 15 degrees -->
@@ -156,8 +141,7 @@
         <parent link="diffbar"/>
         <child link="tl_difflink_1"/>
-        <origin xyz="0.36851088408476390113 0.12523629853057588468 1.6653345369377348106e-16"
-            rpy="1.4197870096866769263 0.82783261508436067899 -1.5853143941314711274" />
+        <origin xyz="0.36851088408476384561 0.12523629853057594019 5.5511151231257827021e-17" rpy="-1.5857491383211548275 0.08564555364187358133 -1.4824560922687248787" />
         <axis xyz="1 0 0"/>
-        <limit effort="20.0" velocity="20.0" lower="-0.2618" upper="0.2618"/> <!-- +/- 15 degrees -->
+        <limit effort="20.0" velocity="20.0" lower="-3.141592654" upper="3.141592654"/>
         <dynamics damping="0.01" friction="0.0"/>
     </joint>
@@ -166,6 +150,4 @@
         <parent link="tl_difflink_1"/>
         <child link="tl_difflink_2"/>
-        <origin xyz="0.36851088408476390113 0.12523629853057588468 1.6653345369377348106e-16"
-            rpy="1.4197870096866769263 0.82783261508436067899 -1.5853143941314711274" />
         <axis xyz="0 1 0"/>
         <limit effort="20.0" velocity="20.0" lower="-0.2618" upper="0.2618"/> <!-- +/- 15 degrees -->
@@ -176,6 +158,4 @@
         <parent link="tl_difflink_2"/>
         <child link="difflinktop"/>
-        <origin xyz="0.36851088408476390113 0.12523629853057588468 1.6653345369377348106e-16"
-            rpy="1.4197870096866769263 0.82783261508436067899 -1.5853143941314711274" />
         <axis xyz="0 0 1"/>
         <limit effort="20.0" velocity="20.0" lower="-0.2618" upper="0.2618"/> <!-- +/- 15 degrees -->

Commit message: Small fixes to gz_bridge, and urdf

File: src/ros/rover/rover_description/urdf/ckc.xacro (robot description, xacro)
@@ -8,5 +8,5 @@
                 <child_model>${robot_name}</child_model>
                 <child_link>diffend_2</child_link>
-                <attach_topic>close_loop_left</attach_topic>
+                <output_topic>close_loop_left</output_topic>
             </plugin>
             <plugin filename="libgz-sim-detachable-joint-system.so" name="gz::sim::systems::DetachableJoint">
@@ -14,5 +14,5 @@
                 <child_model>${robot_name}</child_model>
                 <child_link>diffend</child_link>
-                <attach_topic>close_loop_right</attach_topic>
+                <output_topic>close_loop_right</output_topic>
             </plugin>
         </gazebo>

File: src/ros/rover/rover_description/urdf/rover.urdf.xacro (robot description, xacro)
@@ -970,5 +970,4 @@
     <!-- Generated ball differential bar joints (Generated as revolute) -->
     <xacro:unless value="$(arg use_diff_ball)">
-        <!-- Note: these aren't defined in controllers.yaml so the TF will break-->
         <joint name="tl_difflink" type="revolute">
             <origin xyz="0.36851088408476384561 0.12523629853057594019 5.5511151231257827021e-17" rpy="-1.5857491383211548275 0.08564555364187358133 -1.4824560922687248787" />

File: src/ros/rover/rover_description/urdf/sim_ball_joints.xacro (robot description, xacro)
@@ -6,5 +6,5 @@
     <link name="tr_difflink_1">
         <inertial>
-        <mass value="0.1"/>
+        <mass value="0.001"/>
         <inertia ixx="0.01" iyy="0.01" izz="0.01" ixy="0.0" ixz="0.0" iyz="0.0"/>
         </inertial>
@@ -13,5 +13,5 @@
     <link name="tr_difflink_2">
         <inertial>
-        <mass value="0.1"/>
+        <mass value="0.001"/>
         <inertia ixx="0.01" iyy="0.01" izz="0.01" ixy="0.0" ixz="0.0" iyz="0.0"/>
         </inertial>
@@ -46,5 +46,5 @@
     <link name="br_difflink_1">
         <inertial>
-        <mass value="0.1"/>
+        <mass value="0.0001"/>
         <inertia ixx="0.01" iyy="0.01" izz="0.01" ixy="0.0" ixz="0.0" iyz="0.0"/>
         </inertial>
@@ -53,5 +53,5 @@
     <link name="br_difflink_2">
         <inertial>
-        <mass value="0.1"/>
+        <mass value="0.0001"/>
         <inertia ixx="0.01" iyy="0.01" izz="0.01" ixy="0.0" ixz="0.0" iyz="0.0"/>
         </inertial>
@@ -86,5 +86,5 @@
     <link name="bl_difflink_1">
         <inertial>
-        <mass value="0.1"/>
+        <mass value="0.0001"/>
         <inertia ixx="0.01" iyy="0.01" izz="0.01" ixy="0.0" ixz="0.0" iyz="0.0"/>
         </inertial>
@@ -93,5 +93,5 @@
     <link name="bl_difflink_2">
         <inertial>
-        <mass value="0.1"/>
+        <mass value="0.0001"/>
         <inertia ixx="0.01" iyy="0.01" izz="0.01" ixy="0.0" ixz="0.0" iyz="0.0"/>
         </inertial>
@@ -126,5 +126,5 @@
     <link name="tl_difflink_1">
         <inertial>
-        <mass value="0.1"/>
+        <mass value="0.0001"/>
         <inertia ixx="0.01" iyy="0.01" izz="0.01" ixy="0.0" ixz="0.0" iyz="0.0"/>
         </inertial>
@@ -133,5 +133,5 @@
     <link name="tl_difflink_2">
         <inertial>
-        <mass value="0.1"/>
+        <mass value="0.0001"/>
         <inertia ixx="0.01" iyy="0.01" izz="0.01" ixy="0.0" ixz="0.0" iyz="0.0"/>
         </inertial>
