Commit message: fix: redefine base_link joint so that rviz grid spawns contacting wheels

File: src/ros/rover/rover_description/urdf/rover.urdf.xacro (robot description, xacro)
@@ -18,5 +18,5 @@
         <parent link="base_link"/>
         <child link="chassis" />
-        <origin rpy="0.0 0 0" xyz="0 0 0"/>
+        <origin rpy="0.0 0 0" xyz="0 0 0.45"/>
     </joint>
     <link name="chassis">

Commit message: More accurate cylinderical joints

File: src/ros/rover/rover_description/urdf/rover.urdf.xacro (robot description, xacro)
@@ -824,5 +824,4 @@
         <joint_properties friction="0.0"/>
     </joint>
-    -->
     <joint name="bl_difflinkeye" type="revolute">
         <origin xyz="-1.1102230246251565404e-16 1.1102230246251565404e-16 -0.059500000000000233258" rpy="3.1415926535897868987 5.0960784183182330152e-15 -2.3408550063658504214" />
@@ -841,5 +840,4 @@
         <joint_properties friction="0.0"/>
     </joint>
-    <!--
     <joint name="tl_difflink" type="revolute">
         <origin xyz="0.36851088408476384561 0.12523629853057594019 5.5511151231257827021e-17" rpy="-1.5857491383211548275 0.08564555364187358133 -1.4824560922687248787" />
@@ -924,5 +922,4 @@
         <joint_properties friction="0.0"/>
     </joint>
-    -->
     <joint name="br_difflinkeye" type="revolute">
         <origin xyz="1.6653345369377348106e-16 -1.1102230246251565404e-16 -0.059499795362094654028" rpy="-3.1415926535897402694 1.3056345544300866556e-14 -1.2925601884114563678" />
@@ -941,5 +938,4 @@
         <joint_properties friction="0.0"/>
     </joint>
-    <!--
     <joint name="tr_difflink" type="revolute">
         <origin xyz="-0.38912669878348532526 0.0080507423534932481823 7.2164496600635175128e-16" rpy="1.8972013954619286746 0.81245706006717677283 -1.1914339028340867888" />
@@ -950,5 +946,4 @@
         <joint_properties friction="0.0"/>
     </joint>
-    -->
     <joint name="diffbar_joint" type="revolute">
         <origin xyz="0.018499995185548932103 1.3346709641398613044e-05 0.019800000000001038991" rpy="3.141592653589793116 -6.9464785874916311517e-17 0.15327080924390459882" />
@@ -958,5 +953,5 @@
         <limit effort="1" velocity="20" lower="-3.141592654" upper="3.141592654"/>
         <joint_properties friction="0.0"/>
-    </joint>
+    </joint> -->
     <joint name="diffmount_join" type="fixed">
         <origin xyz="-0.44600000000001260858 -0.018500000000000033779 0.04651879619332278254" rpy="-1.5707963267949107689 -2.2204460492504235214e-16 1.57079632679489678" />
@@ -1002,4 +997,45 @@
             <joint_properties friction="0.0"/>
         </joint>
+        <!-- Generated cylindrical joints (Generated as revolute) -->
+        <joint name="br_difflinkeye" type="revolute">
+            <origin xyz="1.6653345369377348106e-16 -1.1102230246251565404e-16 -0.059499795362094654028" rpy="-3.1415926535897402694 1.3056345544300866556e-14 -1.2925601884114563678" />
+            <parent link="difflinkbody_2" />
+            <child link="difflinkbottom_2" />
+            <axis xyz="0 0 1"/>
+            <limit effort="1" velocity="20" lower="-3.141592654" upper="3.141592654"/>
+            <joint_properties friction="0.0"/>
+        </joint>
+        <joint name="tr_difflinkeye" type="revolute">
+            <origin xyz="0.030163508761794161073 0.011735637514349694932 2.7755575615628913511e-16" rpy="1.5707963267949009989 -0.18611770882550127126 -1.1997499986779625036" />
+            <parent link="difflinktop_2" />
+            <child link="difflinkbody_2" />
+            <axis xyz="0 0 1"/>
+            <limit effort="1" velocity="20" lower="-3.141592654" upper="3.141592654"/>
+            <joint_properties friction="0.0"/>
+        </joint>
+        <joint name="bl_difflinkeye" type="revolute">
+            <origin xyz="-1.1102230246251565404e-16 1.1102230246251565404e-16 -0.059500000000000233258" rpy="3.1415926535897868987 5.0960784183182330152e-15 -2.3408550063658504214" />
+            <parent link="difflinkbody" />
+            <child link="difflinkbottom" />
+            <axis xyz="0 0 1"/>
+            <limit effort="1" velocity="20" lower="-3.141592654" upper="3.141592654"/>
+            <joint_properties friction="0.0"/>
+        </joint>
+        <joint name="tl_difflinkeye" type="revolute">
+            <origin xyz="0.030163508747499123697 0.011735637508787977179 -0.004749999999999865441" rpy="-1.5707963267949025532 0.57279739609381175036 1.9418426549118157354" />
+            <parent link="difflinktop" />
+            <child link="difflinkbody" />
+            <axis xyz="0 0 1"/>
+            <limit effort="1" velocity="20" lower="-3.141592654" upper="3.141592654"/>
+            <joint_properties friction="0.0"/>
+        </joint>
+        <joint name="diffbar_joint" type="revolute">
+            <origin xyz="0.018499995185548932103 1.3346709641398613044e-05 0.019800000000001038991" rpy="3.141592653589793116 -6.9464785874916311517e-17 0.15327080924390459882" />
+            <parent link="diffmount" />
+            <child link="diffbar" />
+            <axis xyz="0 0 1"/>
+            <limit effort="1" velocity="20" lower="-3.141592654" upper="3.141592654"/>
+            <joint_properties friction="0.0"/>
+        </joint>
     </xacro:unless>
     <!-- Include additional xacro files-->
@@ -1007,5 +1043,5 @@
     <xacro:call_ckc robot_name="$(arg robot_name)"/>
     <xacro:if value="$(arg use_diff_ball)">
-        <xacro:include filename="sim_ball_joints.xacro"/>
+        <xacro:include filename="joints.xacro"/>
     </xacro:if>
     <xacro:if value="$(arg auto_camera)">
