Commit message: Preparing rover for simulated ball joints

File: src/ros/rover/rover_description/urdf/joints.xacro (robot description, xacro)
@@ -24,5 +24,5 @@
             rpy="1.5453959963367629449 0.84953874853766309094 -1.271352236581491546" />
         <axis xyz="1 0 0"/>
-        <limit effort="1.0" velocity="20.0" lower="-0.2618" upper="0.2618"/> <!-- +/- 15 degrees -->
+        <limit effort="20.0" velocity="20.0" lower="-0.2618" upper="0.2618"/> <!-- +/- 15 degrees -->
         <dynamics damping="0.01" friction="0.0"/>
     </joint>
@@ -34,5 +34,5 @@
             rpy="1.5453959963367629449 0.84953874853766309094 -1.271352236581491546" />
         <axis xyz="0 1 0"/>
-        <limit effort="1.0" velocity="20.0" lower="-0.2618" upper="0.2618"/> <!-- +/- 15 degrees -->
+        <limit effort="20.0" velocity="20.0" lower="-0.2618" upper="0.2618"/> <!-- +/- 15 degrees -->
         <dynamics damping="0.01" friction="0.0"/>
     </joint>
@@ -44,5 +44,5 @@
             rpy="1.5453959963367629449 0.84953874853766309094 -1.271352236581491546" />
         <axis xyz="0 0 1"/>
-        <limit effort="1.0" velocity="20.0" lower="-0.2618" upper="0.2618"/> <!-- +/- 15 degrees -->
+        <limit effort="20.0" velocity="20.0" lower="-0.2618" upper="0.2618"/> <!-- +/- 15 degrees -->
         <dynamics damping="0.01" friction="0.0"/>
     </joint>
@@ -69,5 +69,5 @@
             rpy="-1.8211554193643901822 0.38630147202971765186 1.6973296137818383311" />
         <axis xyz="1 0 0"/>
-        <limit effort="1.0" velocity="20.0" lower="-0.2618" upper="0.2618"/> <!-- +/- 15 degrees -->
+        <limit effort="20.0" velocity="20.0" lower="-0.2618" upper="0.2618"/> <!-- +/- 15 degrees -->
         <dynamics damping="0.01" friction="0.0"/>
     </joint>
@@ -79,5 +79,5 @@
             rpy="-1.8211554193643901822 0.38630147202971765186 1.6973296137818383311" />
         <axis xyz="0 1 0"/>
-        <limit effort="1.0" velocity="20.0" lower="-0.2618" upper="0.2618"/> <!-- +/- 15 degrees -->
+        <limit effort="20.0" velocity="20.0" lower="-0.2618" upper="0.2618"/> <!-- +/- 15 degrees -->
         <dynamics damping="0.01" friction="0.0"/>
     </joint>
@@ -89,5 +89,5 @@
             rpy="-1.8211554193643901822 0.38630147202971765186 1.6973296137818383311" />
         <axis xyz="0 0 1"/>
-        <limit effort="1.0" velocity="20.0" lower="-0.2618" upper="0.2618"/> <!-- +/- 15 degrees -->
+        <limit effort="20.0" velocity="20.0" lower="-0.2618" upper="0.2618"/> <!-- +/- 15 degrees -->
         <dynamics damping="0.01" friction="0.0"/>
     </joint>
@@ -114,5 +114,5 @@
             rpy="1.8137134713184706047 0.40491568475361000568 2.0095824661262473576" />
         <axis xyz="1 0 0"/>
-        <limit effort="1.0" velocity="20.0" lower="-0.2618" upper="0.2618"/> <!-- +/- 15 degrees -->
+        <limit effort="20.0" velocity="20.0" lower="-0.2618" upper="0.2618"/> <!-- +/- 15 degrees -->
         <dynamics damping="0.01" friction="0.0"/>
     </joint>
@@ -124,5 +124,5 @@
             rpy="1.8137134713184706047 0.40491568475361000568 2.0095824661262473576" />
         <axis xyz="0 1 0"/>
-        <limit effort="1.0" velocity="20.0" lower="-0.2618" upper="0.2618"/> <!-- +/- 15 degrees -->
+        <limit effort="20.0" velocity="20.0" lower="-0.2618" upper="0.2618"/> <!-- +/- 15 degrees -->
         <dynamics damping="0.01" friction="0.0"/>
     </joint>
@@ -134,5 +134,5 @@
             rpy="1.8137134713184706047 0.40491568475361000568 2.0095824661262473576" />
         <axis xyz="0 0 1"/>
-        <limit effort="1.0" velocity="20.0" lower="-0.2618" upper="0.2618"/> <!-- +/- 15 degrees -->
+        <limit effort="20.0" velocity="20.0" lower="-0.2618" upper="0.2618"/> <!-- +/- 15 degrees -->
         <dynamics damping="0.01" friction="0.0"/>
     </joint>
@@ -159,5 +159,5 @@
             rpy="1.4197870096866769263 0.82783261508436067899 -1.5853143941314711274" />
         <axis xyz="1 0 0"/>
-        <limit effort="1.0" velocity="20.0" lower="-0.2618" upper="0.2618"/> <!-- +/- 15 degrees -->
+        <limit effort="20.0" velocity="20.0" lower="-0.2618" upper="0.2618"/> <!-- +/- 15 degrees -->
         <dynamics damping="0.01" friction="0.0"/>
     </joint>
@@ -169,5 +169,5 @@
             rpy="1.4197870096866769263 0.82783261508436067899 -1.5853143941314711274" />
         <axis xyz="0 1 0"/>
-        <limit effort="1.0" velocity="20.0" lower="-0.2618" upper="0.2618"/> <!-- +/- 15 degrees -->
+        <limit effort="20.0" velocity="20.0" lower="-0.2618" upper="0.2618"/> <!-- +/- 15 degrees -->
         <dynamics damping="0.01" friction="0.0"/>
     </joint>
@@ -179,5 +179,5 @@
             rpy="1.4197870096866769263 0.82783261508436067899 -1.5853143941314711274" />
         <axis xyz="0 0 1"/>
-        <limit effort="1.0" velocity="20.0" lower="-0.2618" upper="0.2618"/> <!-- +/- 15 degrees -->
+        <limit effort="20.0" velocity="20.0" lower="-0.2618" upper="0.2618"/> <!-- +/- 15 degrees -->
         <dynamics damping="0.01" friction="0.0"/>
     </joint>

File: src/ros/rover/rover_description/urdf/rover.urdf.xacro (robot description, xacro)
@@ -14,4 +14,5 @@
     <xacro:arg name="auto_camera" default="true"/>
     <xacro:arg name="robot_name" default="rover"/>
+    <xacro:arg name="use_diff_ball" default="false"/>
     <!-- Robot properties-->
     <gazebo>
@@ -820,4 +821,5 @@
         </inertial>
     </link>
+    <!--
     <joint name="bl_difflink" type="revolute">
         <origin xyz="2.7755575615628913511e-16 4.4408920985006261617e-16 0.03036606940442951319" rpy="-1.3819198339232898753 0.4052315082576601335 1.6592791076415036589" />
@@ -828,4 +830,5 @@
         <joint_properties friction="0.0"/>
     </joint>
+    -->
     <joint name="bl_difflinkeye" type="revolute">
         <origin xyz="-1.1102230246251565404e-16 1.1102230246251565404e-16 -0.059500000000000233258" rpy="3.1415926535897868987 5.0960784183182330152e-15 -2.3408550063658504214" />
@@ -844,4 +847,5 @@
         <joint_properties friction="0.0"/>
     </joint>
+    <!--
     <joint name="tl_difflink" type="revolute">
         <origin xyz="0.36851088408476384561 0.12523629853057594019 5.5511151231257827021e-17" rpy="-1.5857491383211548275 0.08564555364187358133 -1.4824560922687248787" />
@@ -852,4 +856,5 @@
         <joint_properties friction="0.0"/>
     </joint>
+    -->
     <link name="difflinktop_2">
         <visual>
@@ -916,4 +921,5 @@
         </inertial>
     </link>
+    <!--
     <joint name="br_difflink" type="revolute">
         <origin xyz="-2.2204460492503130808e-16 -2.2204460492503130808e-16 0.030366069404429846257" rpy="1.3580572734639122512 0.40045540725920980574 1.5193397039318303765" />
@@ -924,4 +930,5 @@
         <joint_properties friction="0.0"/>
     </joint>
+    -->
     <joint name="br_difflinkeye" type="revolute">
         <origin xyz="1.6653345369377348106e-16 -1.1102230246251565404e-16 -0.059499795362094654028" rpy="-3.1415926535897402694 1.3056345544300866556e-14 -1.2925601884114563678" />
@@ -940,4 +947,5 @@
         <joint_properties friction="0.0"/>
     </joint>
+    <!--
     <joint name="tr_difflink" type="revolute">
         <origin xyz="-0.38912669878348532526 0.0080507423534932481823 7.2164496600635175128e-16" rpy="1.8972013954619286746 0.81245706006717677283 -1.1914339028340867888" />
@@ -948,4 +956,5 @@
         <joint_properties friction="0.0"/>
     </joint>
+    -->
     <joint name="diffbar_joint" type="revolute">
         <origin xyz="0.018499995185548932103 1.3346709641398613044e-05 0.019800000000001038991" rpy="3.141592653589793116 -6.9464785874916311517e-17 0.15327080924390459882" />
@@ -965,8 +974,45 @@
     </joint>
     <!-- End of Generated URDF -->
+    <!-- Generated ball differential bar joints (Generated as revolute) -->
+    <xacro:unless value="$(arg use_diff_ball)">
+        <joint name="tl_difflink" type="revolute">
+            <origin xyz="0.36851088408476384561 0.12523629853057594019 5.5511151231257827021e-17" rpy="-1.5857491383211548275 0.08564555364187358133 -1.4824560922687248787" />
+            <parent link="diffbar" />
+            <child link="difflinktop" />
+            <axis xyz="0 0 1"/>
+            <limit effort="1" velocity="20" lower="0" upper="0"/>
+            <joint_properties friction="0.0"/>
+        </joint>
+        <joint name="tr_difflink" type="revolute">
+            <origin xyz="-0.38912669878348532526 0.0080507423534932481823 7.2164496600635175128e-16" rpy="1.8972013954619286746 0.81245706006717677283 -1.1914339028340867888" />
+            <parent link="diffbar" />
+            <child link="difflinktop_2" />
+            <axis xyz="0 0 1"/>
+            <limit effort="1" velocity="20" lower="0" upper="0"/>
+            <joint_properties friction="0.0"/>
+        </joint>
+        <joint name="bl_difflink" type="revolute">
+            <origin xyz="2.7755575615628913511e-16 4.4408920985006261617e-16 0.03036606940442951319" rpy="-1.3819198339232898753 0.4052315082576601335 1.6592791076415036589" />
+            <parent link="difflinkbottom" />
+            <child link="diffend" />
+            <axis xyz="0 0 1"/>
+            <limit effort="1" velocity="20" lower="0" upper="0"/>
+            <joint_properties friction="0.0"/>
+        </joint>
+        <joint name="br_difflink" type="revolute">
+            <origin xyz="-2.2204460492503130808e-16 -2.2204460492503130808e-16 0.030366069404429846257" rpy="1.3580572734639122512 0.40045540725920980574 1.5193397039318303765" />
+            <parent link="difflinkbottom_2" />
+            <child link="diffend_2" />
+            <axis xyz="0 0 1"/>
+            <limit effort="1" velocity="20" lower="0" upper="0"/>
+            <joint_properties friction="0.0"/>
+        </joint>
+    </xacro:unless>
     <!-- Include additional xacro files-->
     <xacro:include filename="ckc.xacro"/>
     <xacro:call_ckc robot_name="$(arg robot_name)"/>
-    <!--<xacro:include filename="joints.xacro"/>-->
+    <xacro:if value="$(arg use_diff_ball)">
+        <xacro:include filename="joints.xacro"/>
+    </xacro:if>
     <xacro:if value="$(arg auto_camera)">
         <xacro:include filename="$(find rover_description)/urdf/auto_camera.xacro"/>

Commit message: Added diffend collision and correct joints for diffential bar (cylindrical and planar)

File: src/ros/rover/rover_description/urdf/joints.xacro (robot description, xacro)
@@ -7,5 +7,5 @@
         <inertial>
         <mass value="0.00001"/>
-        <inertia ixx="0.0001" iyy="0.0001" izz="0.0001" ixy="0.0" ixz="0.0" iyz="0.0"/>
+        <inertia ixx="0.01" iyy="0.01" izz="0.01" ixy="0.0" ixz="0.0" iyz="0.0"/>
         </inertial>
     </link>
@@ -14,5 +14,5 @@
         <inertial>
         <mass value="0.00001"/>
-        <inertia ixx="0.0001" iyy="0.0001" izz="0.0001" ixy="0.0" ixz="0.0" iyz="0.0"/>
+        <inertia ixx="0.01" iyy="0.01" izz="0.01" ixy="0.0" ixz="0.0" iyz="0.0"/>
         </inertial>
     </link>
@@ -48,5 +48,5 @@
         <inertial>
         <mass value="0.0001"/>
-        <inertia ixx="0.0001" iyy="0.0001" izz="0.0001" ixy="0.0" ixz="0.0" iyz="0.0"/>
+        <inertia ixx="0.01" iyy="0.01" izz="0.01" ixy="0.0" ixz="0.0" iyz="0.0"/>
         </inertial>
     </link>
@@ -55,5 +55,5 @@
         <inertial>
         <mass value="0.0001"/>
-        <inertia ixx="0.0001" iyy="0.0001" izz="0.0001" ixy="0.0" ixz="0.0" iyz="0.0"/>
+        <inertia ixx="0.01" iyy="0.01" izz="0.01" ixy="0.0" ixz="0.0" iyz="0.0"/>
         </inertial>
     </link>
@@ -88,5 +88,5 @@
         <inertial>
         <mass value="0.0001"/>
-        <inertia ixx="0.0001" iyy="0.0001" izz="0.0001" ixy="0.0" ixz="0.0" iyz="0.0"/>
+        <inertia ixx="0.01" iyy="0.01" izz="0.01" ixy="0.0" ixz="0.0" iyz="0.0"/>
         </inertial>
     </link>
@@ -95,5 +95,5 @@
         <inertial>
         <mass value="0.0001"/>
-        <inertia ixx="0.0001" iyy="0.0001" izz="0.0001" ixy="0.0" ixz="0.0" iyz="0.0"/>
+        <inertia ixx="0.01" iyy="0.01" izz="0.01" ixy="0.0" ixz="0.0" iyz="0.0"/>
         </inertial>
     </link>
@@ -128,5 +128,5 @@
         <inertial>
         <mass value="0.0001"/>
-        <inertia ixx="0.0001" iyy="0.0001" izz="0.0001" ixy="0.0" ixz="0.0" iyz="0.0"/>
+        <inertia ixx="0.01" iyy="0.01" izz="0.01" ixy="0.0" ixz="0.0" iyz="0.0"/>
         </inertial>
     </link>
@@ -135,5 +135,5 @@
         <inertial>
         <mass value="0.0001"/>
-        <inertia ixx="0.0001" iyy="0.0001" izz="0.0001" ixy="0.0" ixz="0.0" iyz="0.0"/>
+        <inertia ixx="0.01" iyy="0.01" izz="0.01" ixy="0.0" ixz="0.0" iyz="0.0"/>
         </inertial>
     </link>
@@ -176,5 +176,5 @@
         <inertial>
         <mass value="0.00001"/>
-        <inertia ixx="0.0001" iyy="0.0001" izz="0.0001" ixy="0.0" ixz="0.0" iyz="0.0"/>
+        <inertia ixx="0.01" iyy="0.01" izz="0.01" ixy="0.0" ixz="0.0" iyz="0.0"/>
         </inertial>
     </link>
@@ -183,5 +183,5 @@
         <child link="difflinkbottom_2" />
         <axis xyz="0 0 1"/>
-        <limit effort="1" velocity="2" lower="-0.002" upper="0.002"/>
+        <limit effort="1" velocity="2" lower="-0.01" upper="0.01"/>
         <joint_properties friction="0.0"/>
     </joint>
@@ -198,5 +198,5 @@
         <inertial>
         <mass value="0.00001"/>
-        <inertia ixx="0.0001" iyy="0.0001" izz="0.0001" ixy="0.0" ixz="0.0" iyz="0.0"/>
+        <inertia ixx="0.01" iyy="0.01" izz="0.01" ixy="0.0" ixz="0.0" iyz="0.0"/>
         </inertial>
     </link>
@@ -205,5 +205,5 @@
         <child link="difflinkbody_2" />
         <axis xyz="0 0 1"/>
-        <limit effort="1" velocity="2" lower="-0.002" upper="0.002"/>
+        <limit effort="1" velocity="2" lower="-0.01" upper="0.01"/>
         <joint_properties friction="0.0"/>
     </joint>
@@ -220,5 +220,5 @@
         <inertial>
         <mass value="0.00001"/>
-        <inertia ixx="0.0001" iyy="0.0001" izz="0.0001" ixy="0.0" ixz="0.0" iyz="0.0"/>
+        <inertia ixx="0.01" iyy="0.01" izz="0.01" ixy="0.0" ixz="0.0" iyz="0.0"/>
         </inertial>
     </link>
@@ -227,5 +227,5 @@
         <child link="difflinkbottom" />
         <axis xyz="0 0 1"/>
-        <limit effort="1" velocity="2" lower="-0.002" upper="0.002"/>
+        <limit effort="1" velocity="2" lower="-0.01" upper="0.01"/>
         <joint_properties friction="0.0"/>
     </joint>
@@ -242,5 +242,5 @@
         <inertial>
         <mass value="0.00001"/>
-        <inertia ixx="0.0001" iyy="0.0001" izz="0.0001" ixy="0.0" ixz="0.0" iyz="0.0"/>
+        <inertia ixx="0.01" iyy="0.01" izz="0.01" ixy="0.0" ixz="0.0" iyz="0.0"/>
         </inertial>
     </link>
@@ -249,28 +249,50 @@
         <child link="difflinkbody" />
         <axis xyz="0 0 1"/>
-        <limit effort="1" velocity="2" lower="-0.002" upper="0.002"/>
-        <joint_properties friction="0.0"/>
-    </joint>
-    <!-- Cylindrical joint for diffbar_joint-->
+        <limit effort="1" velocity="2" lower="-0.01" upper="0.01"/>
+        <joint_properties friction="0.0"/>
+    </joint>
+    <!-- Planar joint for diffbar_joint-->
     <joint name="diffbar_joint" type="revolute">
         <origin xyz="0.018499995185548932103 1.3346709641398613044e-05 0.019800000000001038991" rpy="3.141592653589793116 -6.9464785874916311517e-17 0.15327080924390459882" />
         <parent link="diffmount" />
-        <child link="diffbar_joint_slide" />
-        <axis xyz="0 0 1"/>
-        <limit effort="1" velocity="2" lower="-3.141592654" upper="3.141592654"/>
-        <joint_properties friction="0.0"/>
-    </joint>
-    <link name="diffbar_joint_slide">
-        <inertial>
-        <mass value="0.00001"/>
-        <inertia ixx="0.0001" iyy="0.0001" izz="0.0001" ixy="0.0" ixz="0.0" iyz="0.0"/>
+        <child link="diffbar_joint_slide_z" />
+        <axis xyz="0 0 1"/>
+        <limit effort="1" velocity="2" lower="-3.141592654" upper="3.141592654"/>
+    </joint>
+    <link name="diffbar_joint_slide_z">
+        <inertial>
+        <mass value="0.00001"/>
+        <inertia ixx="0.01" iyy="0.01" izz="0.01" ixy="0.0" ixz="0.0" iyz="0.0"/>
         </inertial>
     </link>
     <joint name="diffbar_joint_socket" type="prismatic">
-        <parent link="diffbar_joint_slide" />
+        <parent link="diffbar_joint_slide_z" />
+        <child link="diffbar_joint_slide_x" />
+        <axis xyz="0 0 1"/>
+        <limit effort="1" velocity="2" lower="-0.005" upper="0.015"/>
+    </joint>
+    <link name="diffbar_joint_slide_x">
+        <inertial>
+        <mass value="0.00001"/>
+        <inertia ixx="0.01" iyy="0.01" izz="0.01" ixy="0.0" ixz="0.0" iyz="0.0"/>
+        </inertial>
+    </link>
+    <joint name="diffbar_joint_bend_x" type="prismatic">
+        <parent link="diffbar_joint_slide_x" />
+        <child link="diffbar_joint_slide_y" />
+        <axis xyz="0 1 0"/>
+        <limit effort="1" velocity="2" lower="-0.002" upper="0.002"/>
+    </joint>
+    <link name="diffbar_joint_slide_y">
+        <inertial>
+        <mass value="0.00001"/>
+        <inertia ixx="0.01" iyy="0.01" izz="0.01" ixy="0.0" ixz="0.0" iyz="0.0"/>
+        </inertial>
+    </link>
+    <joint name="diffbar_joint_bend_y" type="prismatic">
+        <parent link="diffbar_joint_slide_y" />
         <child link="diffbar" />
-        <axis xyz="0 0 1"/>
-        <limit effort="1" velocity="2" lower="-0.005" upper="0.0025"/>
-        <joint_properties friction="0.0"/>
+        <axis xyz="1 0 0"/>
+        <limit effort="1" velocity="2" lower="-0.002" upper="0.002"/>
     </joint>
 </robot>

File: src/ros/rover/rover_description/urdf/rover.urdf.xacro (robot description, xacro)
@@ -814,4 +814,28 @@
             <inertia ixx="2.7300446323037492185e-06" ixy="-2.6448797816963012353e-23" ixz="9.2601573929015424771e-23" iyy="2.730044632303750489e-06" iyz="3.2150007718201620802e-25" izz="4.1163841102364620038e-07" />
         </inertial>
+        <collision>
+            <origin xyz="2.221228561399990431e-16 -2.4806533051080637723e-16 1.8908485888147197329e-16" rpy="1.1458335418325183448e-19 -3.1952971976532285507e-17 -3.340430445091672281e-18" />
+            <geometry>
+                <sphere radius="0.0080000000000000001665" />
+            </geometry>
+        </collision>
+        <collision>
+            <origin xyz="2.2225327483161193479e-16 -2.4806511958767798179e-16 0.010000000000000189293" rpy="1.1458335418325183448e-19 -3.1952971976532285507e-17 -3.340430445091672281e-18" />
+            <geometry>
+                <cylinder length="0.0080000000000000001665" radius="0.0064999999999999997016" />
+            </geometry>
+        </collision>
+        <collision>
+            <origin xyz="2.2191418623341841639e-16 -2.4806566798781180994e-16 -0.015999999999999812983" rpy="1.1458335418325183448e-19 -3.1952971976532285507e-17 -3.340430445091672281e-18" />
+            <geometry>
+                <cylinder length="0.020000000000000000416" radius="0.0070499999999999998432" />
+            </geometry>
+        </collision>
+        <collision>
+            <origin xyz="2.2173812099974102494e-16 -2.4806595273403515612e-16 -0.029499999999999811096" rpy="1.1458335418325183448e-19 -3.1952971976532285507e-17 -3.340430445091672281e-18" />
+            <geometry>
+                <cylinder length="0.00899999999999999932" radius="0.0040999999999999994782" />
+            </geometry>
+        </collision>
     </link>
     <!--
@@ -912,4 +936,28 @@
             <inertia ixx="2.7300446323037500655e-06" ixy="-1.6137459473690096736e-23" ixz="-1.2343453944887831449e-22" iyy="2.730044632303749642e-06" iyz="-1.2983835509205830424e-25" izz="4.1163841102364620038e-07" />
         </inertial>
+        <collision>
+            <origin xyz="3.3318508949653362996e-16 -2.5067009591092206444e-16 2.7235158572835871382e-16" rpy="1.6614075194504958245e-20 4.8183310687119230618e-17 -4.8954206465600695793e-18" />
+            <geometry>
+                <sphere radius="0.0080000000000000001665" />
+            </geometry>
+        </collision>
+        <collision>
+            <origin xyz="3.3338205967817805991e-16 -2.5067435196471117923e-16 0.01000000000000027256" rpy="1.6614075194504958245e-20 4.8183310687119230618e-17 -4.8954206465600695793e-18" />
+            <geometry>
+                <cylinder length="0.0080000000000000001665" radius="0.0064999999999999997016" />
+            </geometry>
+        </collision>
+        <collision>
+            <origin xyz="3.3286993720590253218e-16 -2.5066328622485951035e-16 -0.015999999999999729716" rpy="1.6614075194504958245e-20 4.8183310687119230618e-17 -4.8954206465600695793e-18" />
+            <geometry>
+                <cylinder length="0.020000000000000000416" radius="0.0070499999999999998432" />
+            </geometry>
+        </collision>
+        <collision>
+            <origin xyz="3.3260402746068251723e-16 -2.5065754055224425961e-16 -0.029499999999999727829" rpy="1.6614075194504958245e-20 4.8183310687119230618e-17 -4.8954206465600695793e-18" />
+            <geometry>
+                <cylinder length="0.00899999999999999932" radius="0.0040999999999999994782" />
+            </geometry>
+        </collision>
     </link>
     <!--
