Commit message: Attempted mimic joints, added toggle for ball joints and mimic joints

File: src/ros/rover/rover_description/urdf/dynamic_joints.xacro (robot description, xacro)
@@ -2,5 +2,5 @@
 <!-- Publish dynamic joint states for Rover -->
 <robot xmlns:xacro="http://www.ros.org/wiki/xacro">
-    <xacro:unless value="$(arg use_diff_ball)">
+    <xacro:unless value="$(arg use_true_joints)">
         <gazebo>
             <plugin filename="gz-sim-joint-state-publisher-system" name="gz::sim::systems::JointStatePublisher">
@@ -22,5 +22,5 @@
                 <joint_name>br_difflinkeye</joint_name>
                 <joint_name>tl_difflink</joint_name>
-                <joint_name>tf_difflink</joint_name>
+                <joint_name>tr_difflink</joint_name>
                 <joint_name>bl_difflink</joint_name>
                 <joint_name>br_difflink</joint_name>
@@ -28,5 +28,5 @@
         </gazebo>
     </xacro:unless>
-    <xacro:if value="$(arg use_diff_ball)">
+    <xacro:if value="$(arg use_true_joints)">
         <gazebo>
             <plugin filename="gz-sim-joint-state-publisher-system" name="gz::sim::systems::JointStatePublisher">

File: src/ros/rover/rover_description/urdf/joints.xacro (robot description, xacro)
@@ -1,4 +1,5 @@
 <?xml version="1.0" encoding="utf-8"?>
 <!-- Handle custom joints that are not supported by gazebo -->
+<!-- Works except it breaks detachable joint for closing ckc -->
 <robot xmlns:xacro="http://www.ros.org/wiki/xacro" >
     <!-- Ball joint for tr_difflink-->

File: src/ros/rover/rover_description/urdf/rover.urdf.xacro (robot description, xacro)
@@ -8,5 +8,6 @@
     <xacro:arg name="auto_camera" default="true"/>
     <xacro:arg name="robot_name" default="rover"/>
-    <xacro:arg name="use_diff_ball" default="true"/>
+    <xacro:arg name="use_true_joints" default="true"/>
+    <xacro:arg name="use_mimic" default="false"/>
     <!-- Robot properties-->
     <gazebo>
@@ -1012,5 +1013,5 @@
     <!-- End of Generated URDF -->
     <!-- Generated ball differential bar joints (Generated as revolute) -->
-    <xacro:unless value="$(arg use_diff_ball)">
+    <xacro:unless value="$(arg use_true_joints)">
         <joint name="tl_difflink" type="revolute">
             <origin xyz="0.36851088408476384561 0.12523629853057594019 5.5511151231257827021e-17" rpy="-1.5857491383211548275 0.08564555364187358133 -1.4824560922687248787" />
@@ -1018,5 +1019,5 @@
             <child link="difflinktop" />
             <axis xyz="0 0 1"/>
-            <limit effort="1" velocity="20" lower="-3.141592654" upper="3.141592654"/>
+            <limit effort="20" velocity="20" lower="${-2 * pi}" upper="${2 * pi}"/>
             <joint_properties friction="0.0"/>
         </joint>
@@ -1026,5 +1027,5 @@
             <child link="difflinktop_2" />
             <axis xyz="0 0 1"/>
-            <limit effort="1" velocity="20" lower="-3.141592654" upper="3.141592654"/>
+            <limit effort="20" velocity="20" lower="${-2 * pi}" upper="${2 * pi}"/>
             <joint_properties friction="0.0"/>
         </joint>
@@ -1034,5 +1035,5 @@
             <child link="diffend" />
             <axis xyz="0 0 1"/>
-            <limit effort="1" velocity="20" lower="-3.141592654" upper="3.141592654"/>
+            <limit effort="20" velocity="20" lower="${-2 * pi}" upper="${2 * pi}"/>
             <joint_properties friction="0.0"/>
         </joint>
@@ -1042,5 +1043,5 @@
             <child link="diffend_2" />
             <axis xyz="0 0 1"/>
-            <limit effort="1" velocity="20" lower="-3.141592654" upper="3.141592654"/>
+            <limit effort="20" velocity="20" lower="${-2 * pi}" upper="${2 * pi}"/>
             <joint_properties friction="0.0"/>
         </joint>
@@ -1051,5 +1052,5 @@
             <child link="difflinkbottom_2" />
             <axis xyz="0 0 1"/>
-            <limit effort="1" velocity="20" lower="-3.141592654" upper="3.141592654"/>
+            <limit effort="20" velocity="20" lower="${-2 * pi}" upper="${2 * pi}"/>
             <joint_properties friction="0.0"/>
         </joint>
@@ -1059,5 +1060,5 @@
             <child link="difflinkbody_2" />
             <axis xyz="0 0 1"/>
-            <limit effort="1" velocity="20" lower="-3.141592654" upper="3.141592654"/>
+            <limit effort="20" velocity="20" lower="${-2 * pi}" upper="${2 * pi}"/>
             <joint_properties friction="0.0"/>
         </joint>
@@ -1067,5 +1068,5 @@
             <child link="difflinkbottom" />
             <axis xyz="0 0 1"/>
-            <limit effort="1" velocity="20" lower="-3.141592654" upper="3.141592654"/>
+            <limit effort="20" velocity="20" lower="${-2 * pi}" upper="${2 * pi}"/>
             <joint_properties friction="0.0"/>
         </joint>
@@ -1075,5 +1076,5 @@
             <child link="difflinkbody" />
             <axis xyz="0 0 1"/>
-            <limit effort="1" velocity="20" lower="-3.141592654" upper="3.141592654"/>
+            <limit effort="20" velocity="20" lower="${-2 * pi}" upper="${2 * pi}"/>
             <joint_properties friction="0.0"/>
         </joint>
@@ -1083,12 +1084,17 @@
             <child link="diffbar" />
             <axis xyz="0 0 1"/>
-            <limit effort="1" velocity="20" lower="-3.141592654" upper="3.141592654"/>
+            <limit effort="20" velocity="20" lower="${-2 * pi}" upper="${2 * pi}"/>
             <joint_properties friction="0.0"/>
         </joint>
     </xacro:unless>
     <!-- Include additional xacro files-->
-    <xacro:include filename="ckc.xacro"/>
-    <xacro:call_ckc robot_name="$(arg robot_name)"/>
-    <xacro:if value="$(arg use_diff_ball)">
+    <xacro:if value="$(arg use_mimic)">
+        <xacro:include filename="mimic.xacro"/>
+    </xacro:if>
+    <xacro:unless value="$(arg use_mimic)">
+        <xacro:include filename="ckc.xacro"/>
+        <xacro:call_ckc robot_name="$(arg robot_name)"/>
+    </xacro:unless>
+    <xacro:if value="$(arg use_true_joints)">
         <xacro:include filename="joints.xacro"/>
     </xacro:if>
