Commit message: Model fully formed. No controllers yet

File: src/ros/rover/new_rover_description/urdf/ckc.xacro (robot description, xacro)
@@ -2,18 +2,20 @@
 <!-- Configure Closed Kinetic Chains for Rover -->
 <robot xmlns:xacro="http://www.ros.org/wiki/xacro" >
-    <gazebo>
-        <plugin filename="libgz-sim-detachable-joint-system.so" name="gz::sim::systems::DetachableJoint">
-            <parent_link>leftleg</parent_link>
-            <child_model>Rover7</child_model>
-            <child_link>diffend_2</child_link>
-            <attach_topic>close_loop_left</attach_topic>
-        </plugin>
-        <plugin filename="libgz-sim-detachable-joint-system.so" name="gz::sim::systems::DetachableJoint">
-            <parent_link>rightleg</parent_link>
-            <child_model>Rover7</child_model>
-            <child_link>diffend</child_link>
-            <attach_topic>close_loop_right</attach_topic>
-        </plugin>
-    </gazebo>
+    <xacro:macro name="call_ckc" params="robot_name">
+        <gazebo>
+            <plugin filename="libgz-sim-detachable-joint-system.so" name="gz::sim::systems::DetachableJoint">
+                <parent_link>leftleg</parent_link>
+                <child_model>${robot_name}</child_model>
+                <child_link>diffend_2</child_link>
+                <attach_topic>close_loop_left</attach_topic>
+            </plugin>
+            <plugin filename="libgz-sim-detachable-joint-system.so" name="gz::sim::systems::DetachableJoint">
+                <parent_link>rightleg</parent_link>
+                <child_model>${robot_name}</child_model>
+                <child_link>diffend</child_link>
+                <attach_topic>close_loop_right</attach_topic>
+            </plugin>
+        </gazebo>
+    </xacro:macro>
 </robot>
 <!-- Currently, the child_model must be named the rover's namespace which in the rover.urdf.xacro file is rover,

File: src/ros/rover/new_rover_description/urdf/rover.urdf.xacro (robot description, xacro)
@@ -12,4 +12,9 @@
     <xacro:arg name="arm" default="false"/>
     <xacro:arg name="auto_camera" default="true"/>
+    <xacro:arg name="robot_name" default="rover"/>
+    <!-- Robot properties-->
+    <gazebo>
+        <self_collide>false</self_collide>
+    </gazebo>
     <!-- Dummy base link to prevent issues-->
     <link name="base_link" />
@@ -958,6 +963,6 @@
         <joint_properties friction="0.0" />
     </joint>
-    <!-- Ball joints with pitch and yaw restricted to 15 deg -->
-    <!-- Redefined in joints.xacro since gazebo doesn't support it yet
+    <!-- Ball joints with pitch and yaw restricted to 15 deg
+        Redefined in joints.xacro since gazebo doesn't support it yet -->
          When gazebo does, make sure to change the type to ball and change the axis and limits properly
     <joint name="br_difflink" type="revolute">
@@ -996,8 +1001,9 @@
         <limit effort="1" velocity="20" />
         <joint_properties friction="0.0" />
-    </joint> -->
+    </joint>
     <!-- Include additional xacro files-->
     <xacro:include filename="ckc.xacro"/>
-    <xacro:include filename="joints.xacro"/>
+    <xacro:call_ckc robot_name="$(arg robot_name)"/>
+    <!--<xacro:include filename="joints.xacro"/>-->
     <xacro:if value="$(arg auto_camera)">
         <xacro:include filename="$(find new_rover_description)/urdf/auto_camera.xacro"/>
