Commit message: Added simplified collision

File: src/ros/rover/new_rover_description/urdf/auto_camera.xacro (robot description, xacro)
@@ -4,6 +4,7 @@
 <robot xmlns:xacro="http://www.ros.org/wiki/xacro" >
   <link name='camera_link'></link>
+<!-- Need to be fixed, OR ADD AUTO CAMERA MOUNT to URDF-->
   <joint name="camera_joint" type="fixed">
-    <origin xyz="0.49 0 0.48" rpy="0 0 0" />
+    <origin xyz="0 0 0" rpy="0 0 90" />
     <parent link="chassis" />
     <child link="camera_link" />

File: src/ros/rover/new_rover_description/urdf/ckc.xacro (robot description, xacro)
@@ -19,4 +19,3 @@
     </xacro:macro>
 </robot>
-<!-- Currently, the child_model must be named the rover's namespace which in the rover.urdf.xacro file is rover,
- but if running using our launch files, gets changed to Rover7 or Waratah, how do we prevent hard coding?-->
+<!-- diffend_2 is on the left leg, diffend is on the right leg, could be renamed? -->
