Commit message: Added simplified collision

File: src/ros/rover/new_rover_description/urdf/rover.urdf.xacro (robot description, xacro)
@@ -5,4 +5,5 @@
       - CKC is handled in ckc.xacro
       - joints.xacro handles ball joints and other non-vanilla joints
+      - ankles collision handles both ankle and ankle motor
 -->
 <robot name="rover"  xmlns:xacro="http://www.ros.org/wiki/xacro" >
@@ -23,967 +24,944 @@
         <parent link="base_link"/>
         <child link="chassis"/>
-        <origin xyz="0. -0. 0.38" rpy="0. 0. ${-pi/2}"/>
+        <origin rpy="0.0 0 0" xyz="0 0 0"/>
     </joint>
     <link name="chassis">
         <visual>
-            <origin xyz="-0.018984610583012817564 -0.11072106393638803112 0.061040732012669463025"
-                rpy="1.110223024625156146e-15 6.106226635438357028e-16 2.7755575615628895022e-17" />
+            <origin xyz="-0.018984610583012817564 -0.11072106393638803112 0.061040732012669463025" rpy="1.1102230246251559488e-15 6.106226635438357028e-16 2.7755575615628895022e-17" />
             <geometry>
                 <mesh filename="file://$(find new_rover_description)/meshes/chassis.stl" />
             </geometry>
             <material name="chassis_material">
-                <color
-                    rgba="0.67843137254901964006 0.17647058823529412908 0.40392156862745098866 1.0" />
-            </material>
-        </visual>
-        <inertial>
-            <origin xyz="-0.019045218507636810235 -0.087993046828656773517 0.087385944696220851924"
-                rpy="0 0 0" />
-            <mass value="7.6906345059940948161" />
-            <inertia ixx="0.44733237602571912506" ixy="-0.00012066720320086161587"
-                ixz="-0.00020251363375000226924" iyy="0.19488738906767785752"
-                iyz="0.0095851903407345208363" izz="0.56806231569085507971" />
+                <color rgba="0.866666666666666667 0.074509803921568627 0.325490196078431373 1.0"/>
+            </material>
+        </visual>
+        <!-- Shapes for chassis -->
+        <collision>
+            <origin xyz="-0.018984610583012928586 0.061778936063612260865 0.08454073201266965043" rpy="1.1102230246251559488e-15 6.106226635438357028e-16 2.7755575615628895022e-17" />
+            <geometry>
+                <box size="0.47999999999999998224 0.54500000000000003997 0.1749999999999999889" />
+            </geometry>
+        </collision>
+        <collision>
+            <origin xyz="-0.018984610583012675317 -0.33772106393638834376 0.094540732012669229101" rpy="1.1102230246251559488e-15 6.106226635438357028e-16 2.7755575615628895022e-17" />
+            <geometry>
+                <box size="0.34000000000000002442 0.26000000000000000888 0.19500000000000000666" />
+            </geometry>
+        </collision>
+        <inertial>
+            <origin xyz="-0.019045218507636789418 -0.087993046828656260039 0.087385944696220199668" rpy="0 0 0"/>
+            <mass value="7.6906345059941179088" />
+            <inertia ixx="0.44733237602571923608" ixy="-0.00012066720320078725315" ixz="-0.00020251363375000666026" iyy="0.19488738906767866244" iyz="0.0095851903407344826724" izz="0.56806231569085607891" />
         </inertial>
     </link>
     <link name="crossbar">
         <visual>
-            <origin
-                xyz="-2.7755575615628913511e-17 -5.5511151231257827021e-17 -0.14100000000000956213"
-                rpy="1.570796326794896558 1.570796326794896558 0" />
-            <geometry>
-                <mesh filename="file://$(find new_rover_description)/meshes/crossbar.stl" />
+            <origin xyz="-2.7755575615628913511e-17 -5.5511151231257827021e-17 -0.14100000000000956213" rpy="1.570796326794896558 1.570796326794896558 0" />
+            <geometry>
+                <mesh filename="file://$(find new_rover_description)/meshes/crossbar.stl"/>
             </geometry>
             <material name="crossbar_material">
-                <color
-                    rgba="0.91764705882352937127 0.91764705882352937127 0.91764705882352937127 1.0" />
-            </material>
-        </visual>
-        <inertial>
-            <origin xyz="-0.0010899117823054067008 4.0413800272093150103e-06 -0.1399993129761559485"
-                rpy="0 0 0" />
-            <mass value="0.61929085260862071216" />
-            <inertia ixx="0.022394047093070128251" ixy="-6.3774127350866009372e-09"
-                ixz="2.4803302241999911587e-10" iyy="0.022366401167997828486"
-                iyz="-1.5472398701492628437e-08" izz="0.00052067562621966299603" />
+                <color rgba="0.866666666666666667 0.074509803921568627 0.325490196078431373 1.0"/>
+            </material>
+        </visual>
+        <inertial>
+            <origin xyz="-0.0010899117823054075681 4.0413800272093209395e-06 -0.1399993129761559485" rpy="0 0 0"/>
+            <mass value="0.61929085260862060114" />
+            <inertia ixx="0.022394047093070107435" ixy="-6.3774127350865959741e-09" ixz="2.480330224169302758e-10" iyy="0.02236640116799780767" iyz="-1.5472398701492618511e-08" izz="0.00052067562621966310445" />
         </inertial>
     </link>
     <link name="rightleg">
         <visual>
-            <origin xyz="0.074734192136231336612 0.15002553566875342916 -0.27453363429541915997"
-                rpy="-1.5976312533649206227 -0.14736445394616992655 -5.841052856855955895e-18" />
-            <geometry>
-                <mesh filename="file://$(find new_rover_description)/meshes/rightleg.stl" />
+            <origin xyz="-2.7755575615628913511e-17 0 -0.0010000000000006115108" rpy="-3.4694469519539061598e-18 -3.7838655819744529992e-17 -5.216321704935387389e-18" />
+            <geometry>
+                <mesh filename="file://$(find new_rover_description)/meshes/rightleg.stl"/>
             </geometry>
             <material name="rightleg_material">
-                <color
-                    rgba="0.49803921568627451677 0.49803921568627451677 0.49803921568627451677 1.0" />
-            </material>
-        </visual>
-        <collision>
-            <origin xyz="0.074734192136231336612 0.15002553566875342916 -0.27453363429541915997"
-                rpy="-1.5976312533649206227 -0.14736445394616992655 -5.841052856855955895e-18" />
-            <geometry>
-                <mesh filename="file://$(find new_rover_description)/meshes/rightleg.stl" />
-            </geometry>
-        </collision>
-        <inertial>
-            <origin
-                xyz="0.0039717287152238600623 -0.0038738969203747086745 -0.053343764207219812601"
-                rpy="0 0 0" />
-            <mass value="3.3445666178870414598" />
-            <inertia ixx="0.0097840090697630006933" ixy="0.013186503315028193228"
-                ixz="0.0014151848627837386538" iyy="0.49540614693113899092"
-                iyz="0.00019502537856914164863" izz="0.49156963066925923878" />
+                <color rgba="0.866666666666666667 0.074509803921568627 0.325490196078431373 1.0"/>
+            </material>
+        </visual>
+        <!-- Shapes for rightleg -->
+        <collision>
+            <origin xyz="-2.7755575615628913511e-17 0 -0.0010000000000006115108" rpy="-3.4694469519539061598e-18 -3.7838655819744529992e-17 -5.216321704935387389e-18" />
+            <geometry>
+                <cylinder length="0.058000000000000002942" radius="0.042999999999999996558" />
+            </geometry>
+        </collision>
+        <collision>
+            <origin xyz="-0.085433336758075018036 0.0098574827027250004619 -0.0083467600000006175048" rpy="-0.12217294850606505441 1.308997029405494894 -0.23561907663390052603" />
+            <geometry>
+                <cylinder length="0.089999999999999996669" radius="0.02999999999999999889" />
+            </geometry>
+        </collision>
+        <collision>
+            <origin xyz="-0.31437167947314503813 0.038053876881360006179 -0.066033037700000615788" rpy="-0.12217302310744593274 1.3264501982056555729 -0.23561907663390055379" />
+            <geometry>
+                <cylinder length="0.39000000000000001332" radius="0.025000000000000001388" />
+            </geometry>
+        </collision>
+        <collision>
+            <origin xyz="-0.4536556182500000034 -0.0013318353999999964134 -0.10360017400000062771" rpy="2.2332973632360295351e-18 0.27925237217133341838 3.1066861154931633138" />
+            <geometry>
+                <box size="0.105999999999999997 0.06500000000000000222 0.076999999999999999001" />
+            </geometry>
+        </collision>
+        <collision>
+            <origin xyz="-0.44472929400000005273 -0.0099999999999999984734 -0.032885924000000628376" rpy="3.5918351426029592641e-18 0.26179929927377626475 3.141592653589793116" />
+            <geometry>
+                <cylinder length="0.051999999999999997613" radius="0.044999999999999998335" />
+            </geometry>
+        </collision>
+        <collision>
+            <origin xyz="0.085869139396912486095 0.004569547336145000048 -0.0084571750000006096909" rpy="0.069813040387381189444 1.3089970756114859274 -3.0194199283152816093" />
+            <geometry>
+                <cylinder length="0.089999999999999996669" radius="0.02999999999999999889" />
+            </geometry>
+        </collision>
+        <collision>
+            <origin xyz="0.31601584183032671582 0.019116378127553800698 -0.066387337800000598143" rpy="0.069812975010840438994 1.326450241590472201 -3.0194199283152811653" />
+            <geometry>
+                <cylinder length="0.39000000000000001332" radius="0.025000000000000001388" />
+            </geometry>
+        </collision>
+        <collision>
+            <origin xyz="0.46313595625000003597 -0.024684938350000001223 -0.10573799250000059935" rpy="-2.2332973632360295351e-18 0.27925237217133330736 -0.034906538096629968759" />
+            <geometry>
+                <box size="0.10699999999999999789 0.06500000000000000222 0.076999999999999999001" />
+            </geometry>
+        </collision>
+        <collision>
+            <origin xyz="0.4537292939999999497 -0.034000000000000002442 -0.035885924000000596346" rpy="-3.5918351426029592641e-18 0.26179929927377615373 -6.145956884708687905e-18" />
+            <geometry>
+                <cylinder length="0.051999999999999997613" radius="0.044999999999999998335" />
+            </geometry>
+        </collision>
+        <inertial>
+            <origin xyz="0.003971818209179544569 -0.0038738765067834368856 -0.053343546583699073815" rpy="0 0 0"/>
+            <mass value="3.3445649589086539066" />
+            <inertia ixx="0.0097839331373918841939" ixy="0.013186544376772954545" ixz="0.0014152217803643420829" iyy="0.49540599288668413225" iyz="0.00019501354500449987481" izz="0.491569558377862037" />
         </inertial>
     </link>
     <link name="fr_ankle">
         <visual>
-            <origin xyz="0.015614489500176853554 0.67994599685157042224 0.18062285001424138731"
-                rpy="-0.080461825812964266058 -0.08792239097089690758 -5.8568768164772501268e-17" />
-            <geometry>
-                <mesh filename="file://$(find new_rover_description)/meshes/ankle.stl" />
-            </geometry>
-            <material name="ankle_material">
-                <color
-                    rgba="0.64705882352941179736 0.64705882352941179736 0.64705882352941179736 1.0" />
-            </material>
-        </visual>
-        <collision>
-            <origin xyz="0.015614489500176853554 0.67994599685157042224 0.18062285001424138731"
-                rpy="-0.080461825812964266058 -0.08792239097089690758 -5.8568768164772501268e-17" />
-            <geometry>
-                <mesh filename="file://$(find new_rover_description)/meshes/ankle.stl" />
-            </geometry>
-        </collision>
-        <inertial>
-            <origin xyz="-0.044294303560196875147 -0.051143872404985656066 -0.07162417341397339654"
-                rpy="0 0 0" />
-            <mass value="0.40704209227750914879" />
-            <inertia ixx="0.0020666572037422062218" ixy="-0.00036892344710024777997"
-                ixz="-0.0005270304242319385872" iyy="0.0019576639497774187167"
-                iyz="-0.00060807735844362184249" izz="0.0011614748478770173072" />
+            <origin xyz="-0.12415341931613704807 2.2204460492503130808e-16 -0.12500000000000027756" rpy="-1.570796326794896558 -0.13351607992219355348 1.2815911973435683748e-17" />
+            <geometry>
+                <mesh filename="file://$(find new_rover_description)/meshes/fr_ankle.stl"/>
+            </geometry>
+            <material name="fr_ankle_material">
+                <color rgba="0.866666666666666667 0.074509803921568627 0.325490196078431373 1.0"/>
+            </material>
+        </visual>
+        <!-- Shapes for fr_ankle -->
+        <collision>
+            <origin xyz="-0.11601914642063092253 2.1996240131282945813e-16 -0.1030492935317774833" rpy="-1.570796326794896558 0.0061101698267938854559 2.7535978555462142625e-17" />
+            <geometry>
+                <box size="0.032000000000000000666 0.080000000000000001665 0.05999999999999999778" />
+            </geometry>
+        </collision>
+        <collision>
+            <origin xyz="-0.091894553662955694162 2.2695085610775315725e-16 -0.16352745890207484591" rpy="-1.570796326794896558 -0.79674066942340771025 -8.0334679081213468265e-17" />
+            <geometry>
+                <box size="0.020000000000000000416 0.080000000000000001665 0.05999999999999999778" />
+            </geometry>
+        </collision>
+        <collision>
+            <origin xyz="-0.063800853957741640587 2.3151083068364006152e-16 -0.19982021317550338613" rpy="-1.570796326794896558 -0.011343354647681720693 2.5706357119274463868e-17" />
+            <geometry>
+                <box size="0.025000000000000001388 0.030999999999999999778 0.05999999999999999778" />
+            </geometry>
+        </collision>
+        <collision>
+            <origin xyz="-0.067081786006729482441 2.1511999285781526099e-16 -0.044297919093382362443" rpy="-1.570796326794896558 0.80896192356999552242 1.3678059764689873618e-16" />
+            <geometry>
+                <box size="0.01200000000000000025 0.075999999999999998113 0.05999999999999999778" />
+            </geometry>
+        </collision>
+        <collision>
+            <origin xyz="-0.1077783872900700407 2.1669981272594380024e-16 -0.069810716156365762441" rpy="-1.570796326794886788 1.5594529721472150108 9.2675761695923834513e-15" />
+            <geometry>
+                <box size="0.01200000000000000025 0.02999999999999999889 0.05999999999999999778" />
+            </geometry>
+        </collision>
+        <collision>
+            <origin xyz="-0.00045306036165813912131 2.1339573766264431403e-16 -0.010753702302991177686" rpy="1.1176025369121745707e-16 0.0061101698267938854559 2.7535978555462142625e-17" />
+            <geometry>
+                <cylinder length="0.025999999999999998807" radius="0.037999999999999999056" />
+            </geometry>
+        </collision>
+        <collision>
+            <origin xyz="-0.028495306304552450727 2.1335735431760094025e-16 -0.017582487382379483054" rpy="1.1176025369121745707e-16 0.0061101698267938854559 2.7535978555462142625e-17" />
+            <geometry>
+                <box size="0.02999999999999999889 0.05999999999999999778 0.01200000000000000025" />
+            </geometry>
+        </collision>
+        <inertial>
+            <origin xyz="-0.067658474648355587666 -0.00014463856991169088515 -0.071624633432967391156" rpy="0 0 0"/>
+            <mass value="0.40704474660617540049" />
+            <inertia ixx="0.0016392589144157163148" ixy="-2.8493978195282914987e-06" ixz="-0.00080468641679309026171" iyy="0.0023850903898398135086" iyz="-1.4225306394300022135e-06" izz="0.0011614760148504986968" />
         </inertial>
     </link>
     <link name="fr_anklemotor">
         <visual>
-            <origin xyz="0.62946589948944542403 -0.30151197824312137019 0.41046026989988010358"
-                rpy="1.389724805628755222 0.85047616912755763519 -5.818813789397256689e-18" />
-            <geometry>
-                <mesh filename="file://$(find new_rover_description)/meshes/anklemotor.stl" />
-            </geometry>
-            <material name="anklemotor_material">
-                <color
-                    rgba="0.97254901960784312376 0.52941176470588235947 0.0039215686274509803377 1.0" />
-            </material>
-        </visual>
-        <collision>
-            <origin xyz="0.62946589948944542403 -0.30151197824312137019 0.41046026989988010358"
-                rpy="1.389724805628755222 0.85047616912755763519 -5.818813789397256689e-18" />
-            <geometry>
-                <mesh filename="file://$(find new_rover_description)/meshes/anklemotor.stl" />
-            </geometry>
-        </collision>
-        <inertial>
-            <origin xyz="-0.021959006082670595728 0.03562303636279906538 -0.023997480599055761447"
-                rpy="0 0 0" />
-            <mass value="0.67137253036121347094" />
-            <inertia ixx="0.00067218986057567616139" ixy="-3.5904904907073095582e-05"
-                ixz="7.9308197451476638579e-09" iyy="0.00100880238518442477"
-                iyz="6.7335639484740268811e-08" izz="0.001027383014246707315" />
+            <origin xyz="-0.052882847177904201974 -0.084794424783462968298 -0.024000000000003463008" rpy="4.616963723962202702e-16 -3.6197019301521464944e-15 2.7297295375811919005e-17" />
+            <geometry>
+                <mesh filename="file://$(find new_rover_description)/meshes/fr_anklemotor.stl"/>
+            </geometry>
+            <material name="fr_anklemotor_material">
+                <color rgba="0.866666666666666667 0.074509803921568627 0.325490196078431373 1.0"/>
+            </material>
+        </visual>
+        <inertial>
+            <origin xyz="-0.021958993625958610901 0.035623040808488035114 -0.023997480138994699284" rpy="0 0 0"/>
+            <mass value="0.6713726821856261795" />
+            <inertia ixx="0.00067219001428469400596" ixy="-3.5905106721074112476e-05" ixz="7.9146449531207723378e-09" iyy="0.0010088029360243399007" iyz="6.7337379884121410906e-08" izz="0.0010273836245733481039" />
         </inertial>
     </link>
     <link name="fr_wheel">
         <visual>
-            <origin xyz="-0.38259960033318879402 0.46918983337575870252 -0.51922643103692456279"
-                rpy="-1.5750276880577298577 0.71253568943758915921 1.4063130289565325269e-16" />
-            <geometry>
-                <mesh filename="file://$(find new_rover_description)/meshes/wheel.stl" />
-            </geometry>
-            <material name="wheel_material">
-                <color
-                    rgba="0.49803921568627451677 0.49803921568627451677 0.49803921568627451677 1.0" />
-            </material>
-        </visual>
-        <collision>
-            <origin xyz="-0.38259960033318879402 0.46918983337575870252 -0.51922643103692456279"
-                rpy="-1.5750276880577298577 0.71253568943758915921 1.4063130289565325269e-16" />
-            <geometry>
-                <mesh filename="file://$(find new_rover_description)/meshes/wheel.stl" />
-            </geometry>
-        </collision>
-        <inertial>
-            <origin
-                xyz="-4.4336846478920666215e-08 -5.0174766008659332783e-09 1.2572917233201474918e-05"
-                rpy="0 0 0" />
-            <mass value="1.8501383764095644668" />
-            <inertia ixx="0.020701697509521672924" ixy="2.9116893000832806047e-05"
-                ixz="2.3771624222687381634e-09" iyy="0.020861646227223414746"
-                iyz="4.0000680648983471388e-09" izz="0.032713950134905432632" />
+            <origin xyz="1.1102230246251565404e-16 2.7755575615628913511e-17 5.5511151231257827021e-17" rpy="-3.7684101850198562197e-18 9.8339211963253905402e-17 7.5358637265652170988e-17" />
+            <geometry>
+                <mesh filename="file://$(find new_rover_description)/meshes/fr_wheel.stl"/>
+            </geometry>
+            <material name="fr_wheel_material">
+                <color rgba="0.866666666666666667 0.074509803921568627 0.325490196078431373 1.0"/>
+            </material>
+        </visual>
+        <!-- Shapes for fr_wheel -->
+        <collision>
+            <origin xyz="1.1102230246251565404e-16 2.7755575615628913511e-17 5.5511151231257827021e-17" rpy="-3.7684101850198562197e-18 9.8339211963253905402e-17 7.5358637265652170988e-17" />
+            <geometry>
+                <cylinder length="0.16000000000000000333" radius="0.15700000000000000067" />
+            </geometry>
+        </collision>
+        <inertial>
+            <origin xyz="-1.3294988566060514049e-07 -1.1207731105235597487e-07 1.2648623649773514758e-05" rpy="0 0 0"/>
+            <mass value="1.8501412404055204153" />
+            <inertia ixx="0.020701719473910005359" ixy="2.9104723315617238169e-05" ixz="1.0888320723649892053e-08" iyy="0.020861663662014588022" iyz="1.4322179502267095375e-08" izz="0.032713974764007988649" />
         </inertial>
     </link>
     <joint name="frw" type="continuous">
-        <origin xyz="0.053292508052297793419 0.046508209944849943085 -0.02400000000000451772"
-            rpy="1.5707963267948876762 -1.0191759065537659978 -1.4372802468726955105" />
+        <origin xyz="0.053292508052297626886 0.046508209944849610018 -0.024000000000004129141" rpy="-1.5707963267944027308 -0.9386371689836430221 1.7043124067166892655" />
         <parent link="fr_anklemotor" />
         <child link="fr_wheel" />
-        <axis xyz="0 0 1" />
-        <limit effort="1" velocity="20" />
-        <joint_properties friction="0.0" />
+        <axis xyz="0 0 1"/>
+        <limit effort="1" velocity="20" />
+        <joint_properties friction="0.0"/>
     </joint>
     <joint name="fr_ankle_motor_join" type="fixed">
-        <origin xyz="-0.057783171745668049368 -0.02986169737344709918 -0.2020000000000001239"
-            rpy="-1.570796326794896558 -0.13351607992219322041 0.85490567283933871501" />
+        <origin xyz="-0.060453419316137235739 0.024000000000000021316 -0.20199999999999984635" rpy="-1.570796326794896336 -0.1335160799221936645 1.6816785893668983015e-15" />
         <parent link="fr_ankle" />
         <child link="fr_anklemotor" />
-        <axis xyz="0 0 1" />
-        <limit effort="1" velocity="20" />
-        <joint_properties friction="0.0" />
+        <axis xyz="0 0 1"/>
+        <limit effort="1" velocity="20" />
+        <joint_properties friction="0.0"/>
     </joint>
     <joint name="frp" type="revolute">
-        <origin xyz="-0.47013767878255990906 -0.026528595964174069011 -0.10561814293695770406"
-            rpy="1.570796326794901665 1.0073002592573416791 3.1148421188216253164" />
+        <origin xyz="-0.47013767878255952049 -0.026528595964175290256 -0.10561814293695775957" rpy="1.5707963267949240915 1.4738395407249911262 3.1148421188216217637" />
         <parent link="rightleg" />
         <child link="fr_ankle" />
-        <axis xyz="0 0 1" />
-        <limit effort="1" velocity="20" />
-        <joint_properties friction="0.0" />
+        <axis xyz="0 0 1"/>
+        <limit lower="-3.141592654" upper="3.141592654" effort="20" velocity="1" />
+        <joint_properties friction="0.0"/>
     </joint>
     <link name="br_ankle">
         <visual>
-            <origin xyz="0.015614489500176909065 0.67994599685157053326 0.18062285001424135955"
-                rpy="-0.080461825812964266058 -0.08792239097089690758 1.5540142649877242431e-16" />
-            <geometry>
-                <mesh filename="file://$(find new_rover_description)/meshes/ankle.stl" />
-            </geometry>
-            <material name="ankle_material">
-                <color
-                    rgba="0.64705882352941179736 0.64705882352941179736 0.64705882352941179736 1.0" />
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