Commit message: Updated URDF to zero wheels

File: src/ros/rover/new_rover_description/urdf/auto_camera.xacro (robot description, xacro)
@@ -6,5 +6,5 @@
 <!-- Need to be fixed, OR ADD AUTO CAMERA MOUNT to URDF-->
   <joint name="camera_joint" type="fixed">
-    <origin xyz="0 0 0" rpy="0 0 90" />
+    <origin xyz="0 0.3 0.2" rpy="0 0 -1.57" />
     <parent link="chassis" />
     <child link="camera_link" />
