Commit message: Updated URDF to zero wheels

File: src/ros/rover/new_rover_description/urdf/rover.urdf.xacro (robot description, xacro)
@@ -18,25 +18,24 @@
         <self_collide>false</self_collide>
     </gazebo>
-    <!-- Dummy base link to prevent issues-->
-    <link name="base_link" />
-    <!-- Positions the chassis mesh in space relative to the wheel base (Stolen from Waratah and may need to be configured)-->
-    <joint name="base_to_chassis" type="fixed">
+    <!-- Generated URDF -->
+    <link name="base_link"></link>
+    <joint name="base_link_to_base" type="fixed">
         <parent link="base_link"/>
-        <child link="chassis"/>
+        <child link="chassis" />
         <origin rpy="0.0 0 0" xyz="0 0 0"/>
     </joint>
     <link name="chassis">
         <visual>
-            <origin xyz="-0.018984610583012817564 -0.11072106393638803112 0.061040732012669463025" rpy="1.1102230246251559488e-15 6.106226635438357028e-16 2.7755575615628895022e-17" />
-            <geometry>
-                <mesh filename="file://$(find new_rover_description)/meshes/chassis.stl" />
+            <origin xyz="0 0 0" rpy="-1.7225464241988315416e-16 -5.3673954127953012992e-32 4.9303806576313237838e-32" />
+            <geometry>
+                <mesh filename="file://$(find new_rover_description)/meshes/chassis.stl"/>
             </geometry>
             <material name="chassis_material">
-                <color rgba="0.866666666666666667 0.074509803921568627 0.325490196078431373 1.0"/>
+                <color rgba="0.86666666666666669627 0.074509803921568626417 0.32549019607843138191 1.0"/>
             </material>
         </visual>
         <!-- Shapes for chassis -->
         <collision>
-            <origin xyz="-0.018984610583012928586 0.061778936063612260865 0.08454073201266965043" rpy="1.1102230246251559488e-15 6.106226635438357028e-16 2.7755575615628895022e-17" />
+            <origin xyz="1.2023483457100103294e-32 0.1725000000000000977 0.0234999999999999723" rpy="-1.7225464241988315416e-16 -5.3673954127953012992e-32 4.9303806576313237838e-32" />
             <geometry>
                 <box size="0.47999999999999998224 0.54500000000000003997 0.1749999999999999889" />
@@ -44,5 +43,5 @@
         </collision>
         <collision>
-            <origin xyz="-0.018984610583012675317 -0.33772106393638834376 0.094540732012669229101" rpy="1.1102230246251559488e-15 6.106226635438357028e-16 2.7755575615628895022e-17" />
+            <origin xyz="-1.2005115520421823681e-32 -0.22700000000000009059 0.03350000000000005751" rpy="-1.7225464241988315416e-16 -5.3673954127953012992e-32 4.9303806576313237838e-32" />
             <geometry>
                 <box size="0.34000000000000002442 0.26000000000000000888 0.19500000000000000666" />
@@ -50,38 +49,44 @@
         </collision>
         <inertial>
-            <origin xyz="-0.019045218507636789418 -0.087993046828656260039 0.087385944696220199668" rpy="0 0 0"/>
-            <mass value="7.6906345059941179088" />
-            <inertia ixx="0.44733237602571923608" ixy="-0.00012066720320078725315" ixz="-0.00020251363375000666026" iyy="0.19488738906767866244" iyz="0.0095851903407344826724" izz="0.56806231569085607891" />
+            <origin xyz="-6.0607924624012111654e-05 0.022728017107731372098 0.026345212683551427063" rpy="0 0 0"/>
+            <mass value="7.6906345059940930398" />
+            <inertia ixx="0.44733237602571801483" ixy="-0.00012066720320065656613" ixz="-0.00020251363374967481308" iyy="0.19488738906767796855" iyz="0.0095851903407342710361" izz="0.56806231569085485766" />
         </inertial>
     </link>
     <link name="crossbar">
         <visual>
-            <origin xyz="-2.7755575615628913511e-17 -5.5511151231257827021e-17 -0.14100000000000956213" rpy="1.570796326794896558 1.570796326794896558 0" />
+            <origin xyz="-2.7755575615624180345e-17 -5.0143501740629135245e-17 -0.14100000000000956213" rpy="1.570796326794896558 1.570796326794896558 0" />
             <geometry>
                 <mesh filename="file://$(find new_rover_description)/meshes/crossbar.stl"/>
             </geometry>
             <material name="crossbar_material">
-                <color rgba="0.866666666666666667 0.074509803921568627 0.325490196078431373 1.0"/>
-            </material>
-        </visual>
-        <inertial>
-            <origin xyz="-0.0010899117823054075681 4.0413800272093209395e-06 -0.1399993129761559485" rpy="0 0 0"/>
-            <mass value="0.61929085260862060114" />
-            <inertia ixx="0.022394047093070107435" ixy="-6.3774127350865959741e-09" ixz="2.480330224169302758e-10" iyy="0.02236640116799780767" iyz="-1.5472398701492618511e-08" izz="0.00052067562621966310445" />
+                <color rgba="0.86666666666666669627 0.074509803921568626417 0.32549019607843138191 1.0"/>
+            </material>
+        </visual>
+        <collision>
+            <origin xyz="-2.7755575615624180345e-17 -5.0143501740629135245e-17 -0.14100000000000956213" rpy="1.570796326794896558 1.570796326794896558 0" />
+            <geometry>
+                <mesh filename="file://$(find new_rover_description)/meshes/crossbar.stl"/>
+            </geometry>
+        </collision>
+        <inertial>
+            <origin xyz="-0.0010899117823054069176 4.0413800272146775758e-06 -0.13999931297615592074" rpy="0 0 0"/>
+            <mass value="0.61929085260862082318" />
+            <inertia ixx="0.022394047093070128251" ixy="-6.3774127350866646301e-09" ixz="2.4803302241675610258e-10" iyy="0.022366401167997828486" iyz="-1.5472398701493171067e-08" izz="0.00052067562621966299603" />
         </inertial>
     </link>
     <link name="rightleg">
         <visual>
-            <origin xyz="-2.7755575615628913511e-17 0 -0.0010000000000006115108" rpy="-3.4694469519539061598e-18 -3.7838655819744529992e-17 -5.216321704935387389e-18" />
+            <origin xyz="-7.9461177221469483058e-19 7.285838599104098493e-20 -0.001000000000000667022" rpy="-3.4694469519552373626e-18 -3.7838655819743790435e-17 -2.5742563695788228314e-18" />
             <geometry>
                 <mesh filename="file://$(find new_rover_description)/meshes/rightleg.stl"/>
             </geometry>
             <material name="rightleg_material">
-                <color rgba="0.866666666666666667 0.074509803921568627 0.325490196078431373 1.0"/>
+                <color rgba="0.86666666666666669627 0.074509803921568626417 0.32549019607843138191 1.0"/>
             </material>
         </visual>
         <!-- Shapes for rightleg -->
         <collision>
-            <origin xyz="-2.7755575615628913511e-17 0 -0.0010000000000006115108" rpy="-3.4694469519539061598e-18 -3.7838655819744529992e-17 -5.216321704935387389e-18" />
+            <origin xyz="-7.9461177221469483058e-19 7.285838599104098493e-20 -0.001000000000000667022" rpy="-3.4694469519552373626e-18 -3.7838655819743790435e-17 -2.5742563695788228314e-18" />
             <geometry>
                 <cylinder length="0.058000000000000002942" radius="0.042999999999999996558" />
@@ -89,5 +94,5 @@
         </collision>
         <collision>
-            <origin xyz="-0.085433336758075018036 0.0098574827027250004619 -0.0083467600000006175048" rpy="-0.12217294850606505441 1.308997029405494894 -0.23561907663390052603" />
+            <origin xyz="-0.08543333675807499028 0.0098574827027250004619 -0.008346760000000673016" rpy="-0.12217294850606505441 1.308997029405494894 -0.23561907663390052603" />
             <geometry>
                 <cylinder length="0.089999999999999996669" radius="0.02999999999999999889" />
@@ -95,5 +100,5 @@
         </collision>
         <collision>
-            <origin xyz="-0.31437167947314503813 0.038053876881360006179 -0.066033037700000615788" rpy="-0.12217302310744593274 1.3264501982056555729 -0.23561907663390055379" />
+            <origin xyz="-0.31437167947314498262 0.038053876881360006179 -0.0660330377000006713" rpy="-0.12217302310744593274 1.3264501982056555729 -0.23561907663390055379" />
             <geometry>
                 <cylinder length="0.39000000000000001332" radius="0.025000000000000001388" />
@@ -101,5 +106,5 @@
         </collision>
         <collision>
-            <origin xyz="-0.4536556182500000034 -0.0013318353999999964134 -0.10360017400000062771" rpy="2.2332973632360295351e-18 0.27925237217133341838 3.1066861154931633138" />
+            <origin xyz="-0.4536556182500000034 -0.0013318353999999977145 -0.10360017400000068322" rpy="2.2332973632374404714e-18 0.27925237217133341838 3.1066861154931633138" />
             <geometry>
                 <box size="0.105999999999999997 0.06500000000000000222 0.076999999999999999001" />
@@ -107,5 +112,5 @@
         </collision>
         <collision>
-            <origin xyz="-0.44472929400000005273 -0.0099999999999999984734 -0.032885924000000628376" rpy="3.5918351426029592641e-18 0.26179929927377626475 3.141592653589793116" />
+            <origin xyz="-0.44472929399999999722 -0.0099999999999999984734 -0.032885924000000683887" rpy="3.5918351426043374596e-18 0.26179929927377626475 3.141592653589793116" />
             <geometry>
                 <cylinder length="0.051999999999999997613" radius="0.044999999999999998335" />
@@ -113,5 +118,5 @@
         </collision>
         <collision>
-            <origin xyz="0.085869139396912486095 0.004569547336145000048 -0.0084571750000006096909" rpy="0.069813040387381189444 1.3089970756114859274 -3.0194199283152816093" />
+            <origin xyz="0.085869139396912513851 0.0045695473361450009153 -0.008457175000000665202" rpy="0.069813040387381189444 1.3089970756114859274 -3.0194199283152816093" />
             <geometry>
                 <cylinder length="0.089999999999999996669" radius="0.02999999999999999889" />
@@ -119,5 +124,5 @@
         </collision>
         <collision>
-            <origin xyz="0.31601584183032671582 0.019116378127553800698 -0.066387337800000598143" rpy="0.069812975010840438994 1.326450241590472201 -3.0194199283152811653" />
+            <origin xyz="0.31601584183032671582 0.019116378127553800698 -0.066387337800000653654" rpy="0.069812975010840438994 1.326450241590472201 -3.0194199283152811653" />
             <geometry>
                 <cylinder length="0.39000000000000001332" radius="0.025000000000000001388" />
@@ -125,5 +130,5 @@
         </collision>
         <collision>
-            <origin xyz="0.46313595625000003597 -0.024684938350000001223 -0.10573799250000059935" rpy="-2.2332973632360295351e-18 0.27925237217133330736 -0.034906538096629968759" />
+            <origin xyz="0.46313595625000003597 -0.024684938349999997753 -0.10573799250000065486" rpy="-2.2332973632374404714e-18 0.27925237217133330736 -0.03490653809662996182" />
             <geometry>
                 <box size="0.10699999999999999789 0.06500000000000000222 0.076999999999999999001" />
@@ -131,5 +136,5 @@
         </collision>
         <collision>
-            <origin xyz="0.4537292939999999497 -0.034000000000000002442 -0.035885924000000596346" rpy="-3.5918351426029592641e-18 0.26179929927377615373 -6.145956884708687905e-18" />
+            <origin xyz="0.45372929400000000522 -0.034000000000000002442 -0.035885924000000651857" rpy="-3.5918351426043374596e-18 0.26179929927377615373 -3.5038915493521025473e-18" />
             <geometry>
                 <cylinder length="0.051999999999999997613" radius="0.044999999999999998335" />
@@ -137,22 +142,22 @@
         </collision>
         <inertial>
-            <origin xyz="0.003971818209179544569 -0.0038738765067834368856 -0.053343546583699073815" rpy="0 0 0"/>
-            <mass value="3.3445649589086539066" />
-            <inertia ixx="0.0097839331373918841939" ixy="0.013186544376772954545" ixz="0.0014152217803643420829" iyy="0.49540599288668413225" iyz="0.00019501354500449987481" izz="0.491569558377862037" />
+            <origin xyz="0.003971818209179431812 -0.0038738765067834251762 -0.053343546583699143204" rpy="0 0 0"/>
+            <mass value="3.3445649589086552389" />
+            <inertia ixx="0.0097839331373918876633" ixy="0.013186544376772944137" ixz="0.0014152217803643362282" iyy="0.4954059928866839102" iyz="0.00019501354500450057954" izz="0.49156955837786181496" />
         </inertial>
     </link>
     <link name="fr_ankle">
         <visual>
-            <origin xyz="-0.12415341931613704807 2.2204460492503130808e-16 -0.12500000000000027756" rpy="-1.570796326794896558 -0.13351607992219355348 1.2815911973435683748e-17" />
+            <origin xyz="-0.12415341931613699256 2.2898349882893853646e-16 -0.1250000000000002498" rpy="-1.570796326794896558 -0.13351607992219352572 1.2181229582827242785e-16" />
             <geometry>
                 <mesh filename="file://$(find new_rover_description)/meshes/fr_ankle.stl"/>
             </geometry>
             <material name="fr_ankle_material">
-                <color rgba="0.866666666666666667 0.074509803921568627 0.325490196078431373 1.0"/>
+                <color rgba="0.86666666666666669627 0.074509803921568626417 0.32549019607843138191 1.0"/>
             </material>
         </visual>
         <!-- Shapes for fr_ankle -->
         <collision>
-            <origin xyz="-0.11601914642063092253 2.1996240131282945813e-16 -0.1030492935317774833" rpy="-1.570796326794896558 0.0061101698267938854559 2.7535978555462142625e-17" />
+            <origin xyz="-0.11601914642063086702 2.2769578193000160333e-16 -0.10304929353177745555" rpy="-1.570796326794896558 0.0061101698267938975989 1.3715254847787124342e-16" />
             <geometry>
                 <box size="0.032000000000000000666 0.080000000000000001665 0.05999999999999999778" />
@@ -160,5 +165,5 @@
         </collision>
         <collision>
-            <origin xyz="-0.091894553662955694162 2.2695085610775315725e-16 -0.16352745890207484591" rpy="-1.570796326794896558 -0.79674066942340771025 -8.0334679081213468265e-17" />
+            <origin xyz="-0.091894553662955638651 2.3759514146060475226e-16 -0.16352745890207481816" rpy="-1.570796326794896558 -0.79674066942340771025 2.4737082664321076987e-17" />
             <geometry>
                 <box size="0.020000000000000000416 0.080000000000000001665 0.05999999999999999778" />
@@ -166,5 +171,5 @@
         </collision>
         <collision>
-            <origin xyz="-0.063800853957741640587 2.3151083068364006152e-16 -0.19982021317550338613" rpy="-1.570796326794896558 -0.011343354647681720693 2.5706357119274463868e-17" />
+            <origin xyz="-0.063800853957741585076 2.4539417915154796666e-16 -0.19982021317550335837" rpy="-1.570796326794896558 -0.011343354647681706815 1.3524584140369868879e-16" />
             <geometry>
                 <box size="0.025000000000000001388 0.030999999999999999778 0.05999999999999999778" />
@@ -172,5 +177,5 @@
         </collision>
         <collision>
-            <origin xyz="-0.067081786006729482441 2.1511999285781526099e-16 -0.044297919093382362443" rpy="-1.570796326794896558 0.80896192356999552242 1.3678059764689873618e-16" />
+            <origin xyz="-0.06708178600672942693 2.2795692414257300287e-16 -0.044297919093382348565" rpy="-1.570796326794896558 0.80896192356999552242 2.5099986351094729997e-16" />
             <geometry>
                 <box size="0.01200000000000000025 0.075999999999999998113 0.05999999999999999778" />
@@ -178,5 +183,5 @@
         </collision>
         <collision>
-            <origin xyz="-0.1077783872900700407 2.1669981272594380024e-16 -0.069810716156365762441" rpy="-1.570796326794886788 1.5594529721472150108 9.2675761695923834513e-15" />
+            <origin xyz="-0.10777838729006998519 2.2518949717502131371e-16 -0.069810716156365748564" rpy="-1.570796326794886566 1.5594529721472150108 9.7664942524092150172e-15" />
             <geometry>
                 <box size="0.01200000000000000025 0.02999999999999999889 0.05999999999999999778" />
@@ -184,5 +189,5 @@
         </collision>
         <collision>
-            <origin xyz="-0.00045306036165813912131 2.1339573766264431403e-16 -0.010753702302991177686" rpy="1.1176025369121745707e-16 0.0061101698267938854559 2.7535978555462142625e-17" />
+            <origin xyz="-0.00045306036165808361016 2.3338633589782932004e-16 -0.010753702302991163808" rpy="1.13113734796077825e-16 0.0061101698267938975989 1.3715254847787124342e-16" />
             <geometry>
                 <cylinder length="0.025999999999999998807" radius="0.037999999999999999056" />
@@ -190,5 +195,5 @@
         </collision>
         <collision>
-            <origin xyz="-0.028495306304552450727 2.1335735431760094025e-16 -0.017582487382379483054" rpy="1.1176025369121745707e-16 0.0061101698267938854559 2.7535978555462142625e-17" />
+            <origin xyz="-0.028495306304552395216 2.3030497367880861351e-16 -0.017582487382379469176" rpy="1.13113734796077825e-16 0.0061101698267938975989 1.3715254847787124342e-16" />
             <geometry>
                 <box size="0.02999999999999999889 0.05999999999999999778 0.01200000000000000025" />
@@ -196,38 +201,44 @@
         </collision>
         <inertial>
-            <origin xyz="-0.067658474648355587666 -0.00014463856991169088515 -0.071624633432967391156" rpy="0 0 0"/>
-            <mass value="0.40704474660617540049" />
-            <inertia ixx="0.0016392589144157163148" ixy="-2.8493978195282914987e-06" ixz="-0.00080468641679309026171" iyy="0.0023850903898398135086" iyz="-1.4225306394300022135e-06" izz="0.0011614760148504986968" />
+            <origin xyz="-0.067658474648355559911 -0.0001446385699116739987 -0.071624633432967321767" rpy="0 0 0"/>
+            <mass value="0.40704474660617523396" />
+            <inertia ixx="0.0016392589144157154474" ixy="-2.8493978195281487737e-06" ixz="-0.00080468641679309058697" iyy="0.0023850903898398122076" iyz="-1.4225306394299920491e-06" izz="0.0011614760148504976126" />
         </inertial>
     </link>
     <link name="fr_anklemotor">
         <visual>
-            <origin xyz="-0.052882847177904201974 -0.084794424783462968298 -0.024000000000003463008" rpy="4.616963723962202702e-16 -3.6197019301521464944e-15 2.7297295375811919005e-17" />
+            <origin xyz="-0.052882847177904201974 -0.084794424783462968298 -0.024000000000003525458" rpy="4.6845761985724690052e-16 -3.6608319069462070423e-15 2.1539843060241694836e-17" />
             <geometry>
                 <mesh filename="file://$(find new_rover_description)/meshes/fr_anklemotor.stl"/>
             </geometry>
             <material name="fr_anklemotor_material">
-                <color rgba="0.866666666666666667 0.074509803921568627 0.325490196078431373 1.0"/>
-            </material>
-        </visual>
-        <inertial>
-            <origin xyz="-0.021958993625958610901 0.035623040808488035114 -0.023997480138994699284" rpy="0 0 0"/>
+                <color rgba="0.86666666666666669627 0.074509803921568626417 0.32549019607843138191 1.0"/>
+            </material>
+        </visual>
+        <collision>
+            <origin xyz="-0.052882847177904201974 -0.084794424783462968298 -0.024000000000003525458" rpy="4.6845761985724690052e-16 -3.6608319069462070423e-15 2.1539843060241694836e-17" />
+            <geometry>
+                <mesh filename="file://$(find new_rover_description)/meshes/fr_anklemotor.stl"/>
+            </geometry>
+        </collision>
+        <inertial>
+            <origin xyz="-0.02195899362595862131 0.035623040808488035114 -0.023997480138994768673" rpy="0 0 0"/>
             <mass value="0.6713726821856261795" />
-            <inertia ixx="0.00067219001428469400596" ixy="-3.5905106721074112476e-05" ixz="7.9146449531207723378e-09" iyy="0.0010088029360243399007" iyz="6.7337379884121410906e-08" izz="0.0010273836245733481039" />
+            <inertia ixx="0.00067219001428469400596" ixy="-3.5905106721074085371e-05" ixz="7.9146449531927569034e-09" iyy="0.001008802936024339467" iyz="6.7337379884120219766e-08" izz="0.0010273836245733476702" />
         </inertial>
     </link>
     <link name="fr_wheel">
         <visual>
-            <origin xyz="1.1102230246251565404e-16 2.7755575615628913511e-17 5.5511151231257827021e-17" rpy="-3.7684101850198562197e-18 9.8339211963253905402e-17 7.5358637265652170988e-17" />
+            <origin xyz="0 -1.0408340855860842566e-16 -1.1102230246251565404e-16" rpy="-1.985058964698083451e-17 1.1378066708760287058e-16 4.352542615723205238e-17" />
             <geometry>
                 <mesh filename="file://$(find new_rover_description)/meshes/fr_wheel.stl"/>
             </geometry>
             <material name="fr_wheel_material">
-                <color rgba="0.866666666666666667 0.074509803921568627 0.325490196078431373 1.0"/>
+                <color rgba="0.86666666666666669627 0.074509803921568626417 0.32549019607843138191 1.0"/>
             </material>
         </visual>
         <!-- Shapes for fr_wheel -->
         <collision>
-            <origin xyz="1.1102230246251565404e-16 2.7755575615628913511e-17 5.5511151231257827021e-17" rpy="-3.7684101850198562197e-18 9.8339211963253905402e-17 7.5358637265652170988e-17" />
+            <origin xyz="0 -1.0408340855860842566e-16 -1.1102230246251565404e-16" rpy="-1.985058964698083451e-17 1.1378066708760287058e-16 4.352542615723205238e-17" />
             <geometry>
                 <cylinder length="0.16000000000000000333" radius="0.15700000000000000067" />
@@ -235,11 +246,11 @@
         </collision>
         <inertial>
-            <origin xyz="-1.3294988566060514049e-07 -1.1207731105235597487e-07 1.2648623649773514758e-05" rpy="0 0 0"/>
-            <mass value="1.8501412404055204153" />
-            <inertia ixx="0.020701719473910005359" ixy="2.9104723315617238169e-05" ixz="1.0888320723649892053e-08" iyy="0.020861663662014588022" iyz="1.4322179502267095375e-08" izz="0.032713974764007988649" />
+            <origin xyz="-1.3294988575974222074e-07 -1.1207731119699009317e-07 1.2648623649608361968e-05" rpy="0 0 0"/>
+            <mass value="1.8501412404055221916" />
+            <inertia ixx="0.020701719473909988012" ixy="2.9104723315617173795e-05" ixz="1.0888320723220448003e-08" iyy="0.020861663662014574144" iyz="1.4322179505643800491e-08" izz="0.032713974764007967833" />
         </inertial>
     </link>
     <joint name="frw" type="continuous">
-        <origin xyz="0.053292508052297626886 0.046508209944849610018 -0.024000000000004129141" rpy="-1.5707963267944027308 -0.9386371689836430221 1.7043124067166892655" />
+        <origin xyz="0.053292508052297460353 0.046508209944849887574 -0.024000000000004365064" rpy="1.5707963267948921171 0.28883585951286211424 -1.4372802468727061687" />
         <parent link="fr_anklemotor" />
         <child link="fr_wheel" />
@@ -249,5 +260,5 @@
     </joint>
     <joint name="fr_ankle_motor_join" type="fixed">
-        <origin xyz="-0.060453419316137235739 0.024000000000000021316 -0.20199999999999984635" rpy="-1.570796326794896336 -0.1335160799221936645 1.6816785893668983015e-15" />
+        <origin xyz="-0.060453419316137124717 0.023999999999999910294 -0.20200000000000017941" rpy="-1.570796326794896558 -0.13351607992219347021 -1.0877595247438724004e-14" />
         <parent link="fr_ankle" />
         <child link="fr_anklemotor" />
@@ -257,24 +268,24 @@
     </joint>
     <joint name="frp" type="revolute">
-        <origin xyz="-0.47013767878255952049 -0.026528595964175290256 -0.10561814293695775957" rpy="1.5707963267949240915 1.4738395407249911262 3.1148421188216217637" />
+        <origin xyz="-0.47013767878255974253 -0.026528595964174089827 -0.10561814293695781508" rpy="1.5707963267949005548 0.78539816339749224383 3.1148421188216199873" />
         <parent link="rightleg" />
         <child link="fr_ankle" />
         <axis xyz="0 0 1"/>
-        <limit lower="-3.141592654" upper="3.141592654" effort="20" velocity="1" />
+        <limit lower="-3.141592654" upper="3.141592654" effort="20" velocity="20" />
         <joint_properties friction="0.0"/>
     </joint>
     <link name="br_ankle">
         <visual>
-            <origin xyz="-0.12415341931613707582 2.2204460492503130808e-16 -0.12500000000000027756" rpy="-1.570796326794896558 -0.13351607992219352572 8.9072605256713899112e-17" />
+            <origin xyz="-0.12415341931613710358 2.8449465006019636348e-16 -0.12500000000000027756" rpy="-1.570796326794896558 -0.13351607992219349796 4.5136769332523039787e-17" />
             <geometry>
                 <mesh filename="file://$(find new_rover_description)/meshes/br_ankle.stl"/>
             </geometry>
             <material name="br_ankle_material">
-                <color rgba="0.866666666666666667 0.074509803921568627 0.325490196078431373 1.0"/>
+                <color rgba="0.86666666666666669627 0.074509803921568626417 0.32549019607843138191 1.0"/>
             </material>
         </visual>
         <!-- Shapes for br_ankle -->
         <collision>
-            <origin xyz="-0.11601914642063095029 2.2054127170802484242e-16 -0.1030492935317774833" rpy="-1.570796326794896558 0.0061101698267938854559 1.0407154370150894309e-16" />
+            <origin xyz="-0.11601914642063097804 2.8279533064878078663e-16 -0.1030492935317774833" rpy="-1.570796326794896558 0.0061101698267939123441 5.9049099273200022083e-17" />
             <geometry>
                 <box size="0.032000000000000000666 0.080000000000000001665 0.05999999999999999778" />
@@ -282,5 +293,5 @@
         </collision>
         <collision>
-            <origin xyz="-0.09189455366295570804 2.2949592715125738859e-16 -0.16352745890207484591" rpy="-1.570796326794896558 -0.79674066942340771025 -5.8427250197757135313e-18" />
+            <origin xyz="-0.091894553662955735795 2.901969999439457232e-16 -0.16352745890207484591" rpy="-1.570796326794896558 -0.79674066942340759923 -4.2902353975772878232e-17" />
             <geometry>
                 <box size="0.020000000000000000416 0.080000000000000001665 0.05999999999999999778" />
@@ -288,5 +299,5 @@
         </collision>
         <collision>
-            <origin xyz="-0.063800853957741654465 2.3627780206583784495e-16 -0.19982021317550338613" rpy="-1.570796326794896558 -0.011343354647681718958 1.0220726006218328079e-16" />
+            <origin xyz="-0.063800853957741682221 2.9543452362823638508e-16 -0.19982021317550338613" rpy="-1.570796326794896558 -0.011343354647681691202 5.731987495584140101e-17" />
             <geometry>
                 <box size="0.025000000000000001388 0.030999999999999999778 0.05999999999999999778" />
@@ -294,5 +305,5 @@
         </collision>
         <collision>
-            <origin xyz="-0.067081786006729510197 2.1932704316674944891e-16 -0.044297919093382362443" rpy="-1.570796326794896558 0.80896192356999552242 2.1538580359611101293e-16" />
+            <origin xyz="-0.067081786006729537952 2.7983475309870370178e-16 -0.044297919093382376321" rpy="-1.570796326794896558 0.80896192356999552242 1.6229912036341811687e-16" />
             <geometry>
                 <box size="0.01200000000000000025 0.075999999999999998113 0.05999999999999999778" />
@@ -300,5 +311,5 @@
         </collision>
         <collision>
-            <origin xyz="-0.10777838729007006846 2.1784328554040162551e-16 -0.069810716156365762441" rpy="-1.570796326794886566 1.5594529721472150108 9.5191644225623612698e-15" />
+            <origin xyz="-0.10777838729007009622 2.799839143349007714e-16 -0.069810716156365762441" rpy="-1.570796326794886566 1.5594529721472150108 8.7920590409391449246e-15" />
             <geometry>
                 <box size="0.01200000000000000025 0.02999999999999999889 0.05999999999999999778" />
@@ -306,5 +317,5 @@
         </collision>
         <collision>
-            <origin xyz="-0.00045306036165813912131 2.2263483093216927108e-16 -0.010753702302991177686" rpy="1.1404439476390272962e-16 0.0061101698267938854559 1.0407154370150894309e-16" />
+            <origin xyz="-0.00045306036165816687689 2.8040546740891948302e-16 -0.010753702302991177686" rpy="1.1329300829137536362e-16 0.0061101698267939123441 5.9049099273200022083e-17" />
             <geometry>
                 <cylinder length="0.025999999999999998807" radius="0.037999999999999999056" />
@@ -312,5 +323,5 @@
         </collision>
         <collision>
-            <origin xyz="-0.028495306304552464605 2.2046412005707661052e-16 -0.017582487382379483054" rpy="1.1404439476390272962e-16 0.0061101698267938854559 1.0407154370150894309e-16" />
+            <origin xyz="-0.028495306304552478482 2.7944312014866511832e-16 -0.017582487382379483054" rpy="1.1329300829137536362e-16 0.0061101698267939123441 5.9049099273200022083e-17" />
             <geometry>
                 <box size="0.02999999999999999889 0.05999999999999999778 0.01200000000000000025" />
@@ -318,38 +329,44 @@
         </collision>
         <inertial>
-            <origin xyz="-0.067658474648355601544 -0.00014463856991168400046 -0.0716246334329673634" rpy="0 0 0"/>
-            <mass value="0.40704474660617528947" />
-            <inertia ixx="0.0016392589144157163148" ixy="-2.8493978195280716937e-06" ixz="-0.00080468641679309080381" iyy="0.0023850903898398139423" iyz="-1.422530639429918569e-06" izz="0.00116147601485049848" />
+            <origin xyz="-0.0676584746483556293 -0.00014463856991162512828 -0.0716246334329673634" rpy="0 0 0"/>
+            <mass value="0.40704474660617523396" />
+            <inertia ixx="0.001639258914415717399" ixy="-2.8493978195283287682e-06" ixz="-0.00080468641679309047855" iyy="0.0023850903898398139423" iyz="-1.422530639429990355e-06" izz="0.0011614760148504982631" />
         </inertial>
     </link>
     <link name="br_anklemotor">
         <visual>
-            <origin xyz="-0.05288284717790422973 -0.084794424783462982176 -0.02400000000000357403" rpy="4.5639387072788777526e-16 -3.6295598010595551636e-15 -1.3158340023943098711e-17" />
+            <origin xyz="-0.052882847177904201974 -0.084794424783462996054 -0.024000000000003515049" rpy="4.5456107424398069396e-16 -3.6175975286945226714e-15 2.6973788537147245028e-17" />
             <geometry>
                 <mesh filename="file://$(find new_rover_description)/meshes/br_anklemotor.stl"/>
             </geometry>
             <material name="br_anklemotor_material">
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