Commit message: Model fully formed. No controllers yet

File: src/ros/rover/new_rover_description/urdf/rover.urdf.xacro (robot description, xacro)
@@ -1026,7 +1026,43 @@
         <parent link="difflinktop_2" />
         <child link="difflinkbody_2" />
+<<<<<<< HEAD
         <axis xyz="0 0 1"/>
         <limit effort="1" velocity="20" lower="0" upper="0"/>
         <joint_properties friction="0.0"/>
+=======
+        <axis xyz="0 0 1" />
+        <limit effort="1" velocity="20" lower="0" upper="0" />
+        <joint_properties friction="0.0" />
+    </joint>
+    <joint name="diffbar_joint" type="revolute">
+        <origin xyz="0.018499995185549067411 1.3346709641412490832e-05 0.019799999999998652012"
+            rpy="-3.1415926535897917837 1.7332256379891775137e-17 0.17052131402235523594" />
+        <parent link="diffmount" />
+        <child link="diffbar" />
+        <axis xyz="0 0 1" />
+        <limit effort="1" velocity="20" lower="0" upper="0" />
+        <joint_properties friction="0.0" />
+    </joint>
+    <joint name="diffmount_join" type="fixed">
+        <origin xyz="-0.037484610583013076857 0.33527893606361253154 0.10755952820599778974"
+            rpy="-1.5707963267948956698 6.2866740546731004924e-16 3.4368525624018690139e-16" />
+        <parent link="chassis" />
+        <child link="diffmount" />
+        <axis xyz="0 0 1" />
+        <limit effort="1" velocity="20" />
+        <joint_properties friction="0.0" />
+    </joint>
+    <!-- Ball joints with pitch and yaw restricted to 15 deg
+        Redefined in joints.xacro since gazebo doesn't support it yet -->
+         When gazebo does, make sure to change the type to ball and change the axis and limits properly
+    <joint name="br_difflink" type="revolute">
+        <origin xyz="-2.7755575615628913511e-17 0 0.030366069404429957279"
+            rpy="-1.8211554193643901822 0.38630147202971765186 1.6973296137818383311" />
+        <parent link="difflinkbottom_2" />
+        <child link="diffend_2" />
+        <axis xyz="0 0 1" />
+        <limit effort="1" velocity="20" />
+        <joint_properties friction="0.0" />
+>>>>>>> ab25130 (Model fully formed. No controllers yet)
     </joint>
     <joint name="tr_difflink" type="revolute">
@@ -1052,7 +1088,12 @@
         <axis xyz="0 0 1"/>
         <limit effort="1" velocity="20" />
+<<<<<<< HEAD
         <joint_properties friction="0.0"/>
     </joint>
     <!-- End of Generated URDF -->
+=======
+        <joint_properties friction="0.0" />
+    </joint>
+>>>>>>> ab25130 (Model fully formed. No controllers yet)
     <!-- Include additional xacro files-->
     <xacro:include filename="ckc.xacro"/>

Commit message: Remove Chassis and Crossbar collision

File: src/ros/rover/new_rover_description/urdf/rover.urdf.xacro (robot description, xacro)
@@ -37,11 +37,4 @@
             </material>
         </visual>
-        <collision>
-            <origin xyz="-0.018984610583012817564 -0.11072106393638803112 0.061040732012669463025"
-                rpy="1.110223024625156146e-15 6.106226635438357028e-16 2.7755575615628895022e-17" />
-            <geometry>
-                <mesh filename="file://$(find new_rover_description)/meshes/chassis.stl" />
-            </geometry>
-        </collision>
         <inertial>
             <origin xyz="-0.019045218507636810235 -0.087993046828656773517 0.087385944696220851924"
@@ -66,12 +59,4 @@
             </material>
         </visual>
-        <collision>
-            <origin
-                xyz="-2.7755575615628913511e-17 -5.5511151231257827021e-17 -0.14100000000000956213"
-                rpy="1.570796326794896558 1.570796326794896558 0" />
-            <geometry>
-                <mesh filename="file://$(find new_rover_description)/meshes/crossbar.stl" />
-            </geometry>
-        </collision>
         <inertial>
             <origin xyz="-0.0010899117823054067008 4.0413800272093150103e-06 -0.1399993129761559485"

Commit message: Fixed git rebase error

File: src/ros/rover/new_rover_description/urdf/rover.urdf.xacro (robot description, xacro)
@@ -1026,43 +1026,7 @@
         <parent link="difflinktop_2" />
         <child link="difflinkbody_2" />
-<<<<<<< HEAD
         <axis xyz="0 0 1"/>
         <limit effort="1" velocity="20" lower="0" upper="0"/>
         <joint_properties friction="0.0"/>
-=======
-        <axis xyz="0 0 1" />
-        <limit effort="1" velocity="20" lower="0" upper="0" />
-        <joint_properties friction="0.0" />
-    </joint>
-    <joint name="diffbar_joint" type="revolute">
-        <origin xyz="0.018499995185549067411 1.3346709641412490832e-05 0.019799999999998652012"
-            rpy="-3.1415926535897917837 1.7332256379891775137e-17 0.17052131402235523594" />
-        <parent link="diffmount" />
-        <child link="diffbar" />
-        <axis xyz="0 0 1" />
-        <limit effort="1" velocity="20" lower="0" upper="0" />
-        <joint_properties friction="0.0" />
-    </joint>
-    <joint name="diffmount_join" type="fixed">
-        <origin xyz="-0.037484610583013076857 0.33527893606361253154 0.10755952820599778974"
-            rpy="-1.5707963267948956698 6.2866740546731004924e-16 3.4368525624018690139e-16" />
-        <parent link="chassis" />
-        <child link="diffmount" />
-        <axis xyz="0 0 1" />
-        <limit effort="1" velocity="20" />
-        <joint_properties friction="0.0" />
-    </joint>
-    <!-- Ball joints with pitch and yaw restricted to 15 deg
-        Redefined in joints.xacro since gazebo doesn't support it yet -->
-         When gazebo does, make sure to change the type to ball and change the axis and limits properly
-    <joint name="br_difflink" type="revolute">
-        <origin xyz="-2.7755575615628913511e-17 0 0.030366069404429957279"
-            rpy="-1.8211554193643901822 0.38630147202971765186 1.6973296137818383311" />
-        <parent link="difflinkbottom_2" />
-        <child link="diffend_2" />
-        <axis xyz="0 0 1" />
-        <limit effort="1" velocity="20" />
-        <joint_properties friction="0.0" />
->>>>>>> ab25130 (Model fully formed. No controllers yet)
     </joint>
     <joint name="tr_difflink" type="revolute">
@@ -1088,12 +1052,7 @@
         <axis xyz="0 0 1"/>
         <limit effort="1" velocity="20" />
-<<<<<<< HEAD
         <joint_properties friction="0.0"/>
     </joint>
     <!-- End of Generated URDF -->
-=======
-        <joint_properties friction="0.0" />
-    </joint>
->>>>>>> ab25130 (Model fully formed. No controllers yet)
     <!-- Include additional xacro files-->
     <xacro:include filename="ckc.xacro"/>

Commit message: Fixed limits. MILESTONE parallel wheels but legs are rotating in opposite directions.

File: src/ros/rover/new_rover_description/urdf/rover.urdf.xacro (robot description, xacro)
@@ -256,5 +256,5 @@
         <child link="fr_wheel" />
         <axis xyz="0 0 1"/>
-        <limit effort="1" velocity="20" />
+        <limit effort="20" velocity="20" />
         <joint_properties friction="0.0"/>
     </joint>
@@ -384,5 +384,5 @@
         <child link="br_wheel" />
         <axis xyz="0 0 1"/>
-        <limit effort="1" velocity="20" />
+        <limit effort="20" velocity="20" />
         <joint_properties friction="0.0"/>
     </joint>
@@ -591,5 +591,5 @@
         <child link="fl_wheel" />
         <axis xyz="0 0 1"/>
-        <limit effort="1" velocity="20" />
+        <limit effort="20" velocity="20" />
         <joint_properties friction="0.0"/>
     </joint>
@@ -719,5 +719,5 @@
         <child link="bl_wheel" />
         <axis xyz="0 0 1"/>
-        <limit effort="1" velocity="20" />
+        <limit effort="20" velocity="20" />
         <joint_properties friction="0.0"/>
     </joint>
