Commit message: Updated rover params for controller, updated urdf with correct axis for rotation

File: src/ros/rover/new_rover_description/urdf/rover.urdf.xacro (robot description, xacro)
@@ -49,7 +49,7 @@
         </collision>
         <inertial>
-            <origin xyz="-6.0607924624012111654e-05 0.022728017107731372098 0.026345212683551427063" rpy="0 0 0"/>
-            <mass value="7.6906345059940930398" />
-            <inertia ixx="0.44733237602571801483" ixy="-0.00012066720320065656613" ixz="-0.00020251363374967481308" iyy="0.19488738906767796855" iyz="0.0095851903407342710361" izz="0.56806231569085485766" />
+            <origin xyz="-6.060792462398293984e-05 0.022728017107731847413 0.026345212683551218896" rpy="0 0 0"/>
+            <mass value="7.6906345059941259024" />
+            <inertia ixx="0.44733237602571868097" ixy="-0.00012066720320063805338" ixz="-0.00020251363374965811637" iyy="0.1948873890676779963" iyz="0.0095851903407340489915" izz="0.56806231569085563482" />
         </inertial>
     </link>
@@ -71,7 +71,7 @@
         </collision>
         <inertial>
-            <origin xyz="-0.0010899117823054069176 4.0413800272146775758e-06 -0.13999931297615592074" rpy="0 0 0"/>
-            <mass value="0.61929085260862082318" />
-            <inertia ixx="0.022394047093070128251" ixy="-6.3774127350866646301e-09" ixz="2.4803302241675610258e-10" iyy="0.022366401167997828486" iyz="-1.5472398701493171067e-08" izz="0.00052067562621966299603" />
+            <origin xyz="-0.0010899117823054075681 4.041380027214682658e-06 -0.1399993129761559485" rpy="0 0 0"/>
+            <mass value="0.61929085260862060114" />
+            <inertia ixx="0.022394047093070124782" ixy="-6.3774127350866712475e-09" ixz="2.4803302240859229522e-10" iyy="0.022366401167997825017" iyz="-1.5472398701493753402e-08" izz="0.00052067562621966288761" />
         </inertial>
     </link>
@@ -142,7 +142,7 @@
         </collision>
         <inertial>
-            <origin xyz="0.003971818209179431812 -0.0038738765067834251762 -0.053343546583699143204" rpy="0 0 0"/>
-            <mass value="3.3445649589086552389" />
-            <inertia ixx="0.0097839331373918876633" ixy="0.013186544376772944137" ixz="0.0014152217803643362282" iyy="0.4954059928866839102" iyz="0.00019501354500450057954" izz="0.49156955837786181496" />
+            <origin xyz="0.0039718182091793233918 -0.003873876506783426911 -0.053343546583699136265" rpy="0 0 0"/>
+            <mass value="3.344564958908655683" />
+            <inertia ixx="0.0097839331373918859286" ixy="0.013186544376772938933" ixz="0.0014152217803643308072" iyy="0.49540599288668402123" iyz="0.0001950135450044998206" izz="0.49156955837786198149" />
         </inertial>
     </link>
@@ -201,7 +201,7 @@
         </collision>
         <inertial>
-            <origin xyz="-0.067658474648355559911 -0.0001446385699116739987 -0.071624633432967321767" rpy="0 0 0"/>
-            <mass value="0.40704474660617523396" />
-            <inertia ixx="0.0016392589144157154474" ixy="-2.8493978195281487737e-06" ixz="-0.00080468641679309058697" iyy="0.0023850903898398122076" iyz="-1.4225306394299920491e-06" izz="0.0011614760148504976126" />
+            <origin xyz="-0.067658474648355532155 -0.00014463856991167397159 -0.0716246334329673634" rpy="0 0 0"/>
+            <mass value="0.40704474660617540049" />
+            <inertia ixx="0.0016392589144157169653" ixy="-2.8493978195280827051e-06" ixz="-0.00080468641679309037013" iyy="0.002385090389839814376" iyz="-1.4225306394299746849e-06" izz="0.0011614760148504982631" />
         </inertial>
     </link>
@@ -223,7 +223,7 @@
         </collision>
         <inertial>
-            <origin xyz="-0.02195899362595862131 0.035623040808488035114 -0.023997480138994768673" rpy="0 0 0"/>
-            <mass value="0.6713726821856261795" />
-            <inertia ixx="0.00067219001428469400596" ixy="-3.5905106721074085371e-05" ixz="7.9146449531927569034e-09" iyy="0.001008802936024339467" iyz="6.7337379884120219766e-08" izz="0.0010273836245733476702" />
+            <origin xyz="-0.021958993625958544982 0.035623040808488048992 -0.023997480138994761734" rpy="0 0 0"/>
+            <mass value="0.67137268218562695665" />
+            <inertia ixx="0.00067219001428469411438" ixy="-3.590510672107426833e-05" ixz="7.9146449530338902493e-09" iyy="0.0010088029360243425028" iyz="6.7337379884079747473e-08" izz="0.0010273836245733511396" />
         </inertial>
     </link>
@@ -246,7 +246,7 @@
         </collision>
         <inertial>
-            <origin xyz="-1.3294988575974222074e-07 -1.1207731119699009317e-07 1.2648623649608361968e-05" rpy="0 0 0"/>
-            <mass value="1.8501412404055221916" />
-            <inertia ixx="0.020701719473909988012" ixy="2.9104723315617173795e-05" ixz="1.0888320723220448003e-08" iyy="0.020861663662014574144" iyz="1.4322179505643800491e-08" izz="0.032713974764007967833" />
+            <origin xyz="-1.3294988576507908417e-07 -1.1207731120965171372e-07 1.2648623649607755492e-05" rpy="0 0 0"/>
+            <mass value="1.8501412404055219696" />
+            <inertia ixx="0.020701719473909981073" ixy="2.9104723315617180571e-05" ixz="1.0888320723437134582e-08" iyy="0.020861663662014574144" iyz="1.4322179505752822895e-08" izz="0.032713974764007960894" />
         </inertial>
     </link>
@@ -329,7 +329,7 @@
         </collision>
         <inertial>
-            <origin xyz="-0.0676584746483556293 -0.00014463856991162512828 -0.0716246334329673634" rpy="0 0 0"/>
-            <mass value="0.40704474660617523396" />
-            <inertia ixx="0.001639258914415717399" ixy="-2.8493978195283287682e-06" ixz="-0.00080468641679309047855" iyy="0.0023850903898398139423" iyz="-1.422530639429990355e-06" izz="0.0011614760148504982631" />
+            <origin xyz="-0.0676584746483556293 -0.00014463856991162531802 -0.0716246334329673634" rpy="0 0 0"/>
+            <mass value="0.40704474660617540049" />
+            <inertia ixx="0.0016392589144157167485" ixy="-2.8493978195284693756e-06" ixz="-0.00080468641679309080381" iyy="0.0023850903898398135086" iyz="-1.4225306394299431329e-06" izz="0.0011614760148504986968" />
         </inertial>
     </link>
@@ -351,7 +351,7 @@
         </collision>
         <inertial>
-            <origin xyz="-0.021958993625958642126 0.035623040808488007358 -0.023997480138994758264" rpy="0 0 0"/>
-            <mass value="0.67137268218562562438" />
-            <inertia ixx="0.00067219001428469433122" ixy="-3.5905106721073936293e-05" ixz="7.914644953215370367e-09" iyy="0.0010088029360243388165" iyz="6.733737988409814397e-08" izz="0.0010273836245733474534" />
+            <origin xyz="-0.021958993625958579676 0.035623040808488035114 -0.023997480138994754795" rpy="0 0 0"/>
+            <mass value="0.67137268218562629052" />
+            <inertia ixx="0.0006721900142846942228" ixy="-3.5905106721074166686e-05" ixz="7.914644953067262024e-09" iyy="0.0010088029360243414186" iyz="6.7337379884058293717e-08" izz="0.0010273836245733500554" />
         </inertial>
     </link>
@@ -374,7 +374,7 @@
         </collision>
         <inertial>
-            <origin xyz="-1.329498858041898776e-07 -1.120773111240936304e-07 1.2648623649717603807e-05" rpy="0 0 0"/>
-            <mass value="1.8501412404055204153" />
-            <inertia ixx="0.02070171947390999842" ixy="2.9104723315617946289e-05" ixz="1.0888320728816993209e-08" iyy="0.020861663662014577614" iyz="1.4322179504212514988e-08" izz="0.032713974764007995588" />
+            <origin xyz="-1.3294988579020083731e-07 -1.1207731110083104841e-07 1.2648623649721515405e-05" rpy="0 0 0"/>
+            <mass value="1.8501412404055210814" />
+            <inertia ixx="0.020701719473909994951" ixy="2.9104723315619088089e-05" ixz="1.0888320728761805373e-08" iyy="0.020861663662014581083" iyz="1.4322179504180785994e-08" izz="0.032713974764007995588" />
         </inertial>
     </link>
@@ -477,7 +477,7 @@
         </collision>
         <inertial>
-            <origin xyz="0.0015090549949553736398 0.0038104460972311618092 -0.054086077114160538426" rpy="0 0 0"/>
-            <mass value="3.3446449370365769482" />
-            <inertia ixx="0.0098743756931083757206" ixy="-0.013941425601706266754" ixz="0.0002430603067200729178" iyy="0.50330609956377914127" iyz="-0.00018934670901982260274" izz="0.4994508758193977882" />
+            <origin xyz="0.0015090549950636225531 0.0038104460972356269874 -0.054086077114172882718" rpy="0 0 0"/>
+            <mass value="3.3446449370376427623" />
+            <inertia ixx="0.0098743756931102995289" ixy="-0.013941425601711875115" ixz="0.00024306030673493643512" iyy="0.50330609956391281212" iyz="-0.00018934670901919053998" izz="0.49945087581952996025" />
         </inertial>
     </link>
@@ -536,7 +536,7 @@
         </collision>
         <inertial>
-            <origin xyz="0.067658474648355504399 0.00014463856991165835908 -0.071624633432967307889" rpy="0 0 0"/>
-            <mass value="0.40704474660617528947" />
-            <inertia ixx="0.0016392589144157158811" ixy="-2.8493978195287586374e-06" ixz="0.00080468641679309026171" iyy="0.0023850903898398139423" iyz="1.4225306394298158662e-06" izz="0.0011614760148504986968" />
+            <origin xyz="0.067658474648355532155 0.00014463856991165860303 -0.071624633432967307889" rpy="0 0 0"/>
+            <mass value="0.40704474660617523396" />
+            <inertia ixx="0.0016392589144157156643" ixy="-2.8493978195287798132e-06" ixz="0.00080468641679309080381" iyy="0.0023850903898398126413" iyz="1.4225306394298241248e-06" izz="0.0011614760148504982631" />
         </inertial>
     </link>
@@ -558,12 +558,12 @@
         </collision>
         <inertial>
-            <origin xyz="0.021958993625958541512 -0.035623040808488035114 -0.023997480138994806836" rpy="0 0 0"/>
-            <mass value="0.67137268218562540234" />
-            <inertia ixx="0.00067219001428469411438" ixy="-3.5905106721074004055e-05" ixz="-7.9146449531200741973e-09" iyy="0.0010088029360243383828" iyz="-6.7337379884104761415e-08" izz="0.001027383624573347887" />
+            <origin xyz="0.021958993625958444368 -0.035623040808488048992 -0.023997480138994803367" rpy="0 0 0"/>
+            <mass value="0.67137268218562673461" />
+            <inertia ixx="0.00067219001428469411438" ixy="-3.5905106721074241225e-05" ixz="-7.914644952971332234e-09" iyy="0.0010088029360243420691" iyz="-6.7337379884061734788e-08" izz="0.0010273836245733513565" />
         </inertial>
     </link>
     <link name="fl_wheel">
         <visual>
-            <origin xyz="2.7755575615628913511e-17 -5.5511151231257827021e-17 0" rpy="4.989850109249110714e-17 9.2702961518020513559e-17 1.0763017799346475639e-16" />
+            <origin xyz="0 -1.1102230246251565404e-16 0" rpy="-5.32811638513845946e-17 1.0671623748771702756e-16 -1.6245626009394877393e-18" />
             <geometry>
                 <mesh filename="file://$(find new_rover_description)/meshes/fl_wheel.stl"/>
@@ -575,5 +575,5 @@
         <!-- Shapes for fl_wheel -->
         <collision>
-            <origin xyz="2.7755575615628913511e-17 -5.5511151231257827021e-17 0" rpy="4.989850109249110714e-17 9.2702961518020513559e-17 1.0763017799346475639e-16" />
+            <origin xyz="0 -1.1102230246251565404e-16 0" rpy="-5.32811638513845946e-17 1.0671623748771702756e-16 -1.6245626009394877393e-18" />
             <geometry>
                 <cylinder length="0.16000000000000000333" radius="0.15700000000000000067" />
@@ -581,11 +581,11 @@
         </collision>
         <inertial>
-            <origin xyz="-1.3294988573961809434e-07 -1.1207731114294712797e-07 1.2648623649716966838e-05" rpy="0 0 0"/>
+            <origin xyz="-1.3294988577583259096e-07 -1.1207731118863899682e-07 1.2648623649717768131e-05" rpy="0 0 0"/>
             <mass value="1.8501412404055213035" />
-            <inertia ixx="0.020701719473909977604" ixy="2.9104723315619240555e-05" ixz="1.0888320722002813326e-08" iyy="0.020861663662014577614" iyz="1.4322179506926620309e-08" izz="0.032713974764007953955" />
+            <inertia ixx="0.020701719473909988012" ixy="2.9104723315617888691e-05" ixz="1.0888320724736239932e-08" iyy="0.020861663662014584553" iyz="1.4322179502484274953e-08" izz="0.032713974764007953955" />
         </inertial>
     </link>
     <joint name="flw" type="continuous">
-        <origin xyz="-0.053292508052297682397 -0.046508209944849887574 -0.024000000000004427514" rpy="-1.5707963267948923392 -0.68040816644748991493 -1.4372802468727061687" />
+        <origin xyz="-0.053292508052297682397 -0.046508209944849887574 -0.024000000000004469147" rpy="1.5707963267948996666 -6.6254394877328790055e-14 -1.4372802468727043923" />
         <parent link="fl_anklemotor" />
         <child link="fl_wheel" />
@@ -664,7 +664,7 @@
         </collision>
         <inertial>
-            <origin xyz="0.067658474648355615422 0.00014463856991167256213 -0.071624633432967335644" rpy="0 0 0"/>
-            <mass value="0.40704474660617528947" />
-            <inertia ixx="0.0016392589144157158811" ixy="-2.8493978195285756783e-06" ixz="0.00080468641679309047855" iyy="0.0023850903898398130749" iyz="1.4225306394299012048e-06" izz="0.00116147601485049848" />
+            <origin xyz="0.067658474648355615422 0.00014463856991167505579 -0.0716246334329673634" rpy="0 0 0"/>
+            <mass value="0.40704474660617540049" />
+            <inertia ixx="0.0016392589144157158811" ixy="-2.8493978195285684785e-06" ixz="0.00080468641679309026171" iyy="0.0023850903898398135086" iyz="1.4225306394298772761e-06" izz="0.00116147601485049848" />
         </inertial>
     </link>
@@ -686,12 +686,12 @@
         </collision>
         <inertial>
-            <origin xyz="0.021958993625958603962 -0.035623040808488062869 -0.02399748013899478602" rpy="0 0 0"/>
-            <mass value="0.67137268218562562438" />
-            <inertia ixx="0.0006721900142846942228" ixy="-3.5905106721073990503e-05" ixz="-7.9146449531680225487e-09" iyy="0.0010088029360243385996" iyz="-6.7337379884133189958e-08" izz="0.0010273836245733470197" />
+            <origin xyz="0.021958993625958510287 -0.035623040808488062869 -0.02399748013899478255" rpy="0 0 0"/>
+            <mass value="0.67137268218562651256" />
+            <inertia ixx="0.00067219001428469400596" ixy="-3.5905106721074248001e-05" ixz="-7.9146449530227266198e-09" iyy="0.0010088029360243422859" iyz="-6.7337379884099480694e-08" izz="0.0010273836245733504891" />
         </inertial>
     </link>
     <link name="bl_wheel">
         <visual>
-            <origin xyz="0 5.5511151231257827021e-17 -1.1102230246251565404e-16" rpy="6.1631746718314039636e-17 1.0513636403582013988e-16 -9.8671009379435180601e-19" />
+            <origin xyz="5.5511151231257827021e-17 1.3877787807814456755e-17 0" rpy="1.571267953360436636e-17 1.0599853521721016491e-16 -5.3080271561233027682e-19" />
             <geometry>
                 <mesh filename="file://$(find new_rover_description)/meshes/bl_wheel.stl"/>
@@ -703,5 +703,5 @@
         <!-- Shapes for bl_wheel -->
         <collision>
-            <origin xyz="0 5.5511151231257827021e-17 -1.1102230246251565404e-16" rpy="6.1631746718314039636e-17 1.0513636403582013988e-16 -9.8671009379435180601e-19" />
+            <origin xyz="5.5511151231257827021e-17 1.3877787807814456755e-17 0" rpy="1.571267953360436636e-17 1.0599853521721016491e-16 -5.3080271561233027682e-19" />
             <geometry>
                 <cylinder length="0.16000000000000000333" radius="0.15700000000000000067" />
@@ -709,11 +709,11 @@
         </collision>
         <inertial>
-            <origin xyz="-1.3294988577383833129e-07 -1.1207731101024211878e-07 1.2648623649607884241e-05" rpy="0 0 0"/>
-            <mass value="1.8501412404055217475" />
-            <inertia ixx="0.020701719473909977604" ixy="2.910472331561667574e-05" ixz="1.0888320724793288925e-08" iyy="0.020861663662014581083" iyz="1.432217950346995826e-08" izz="0.032713974764007967833" />
+            <origin xyz="-1.3294988570786547613e-07 -1.1207731107355732866e-07 1.2648623649718386465e-05" rpy="0 0 0"/>
+            <mass value="1.8501412404055228578" />
+            <inertia ixx="0.020701719473910005359" ixy="2.9104723315618119084e-05" ixz="1.0888320724682670061e-08" iyy="0.020861663662014581083" iyz="1.4322179499909491663e-08" izz="0.032713974764007995588" />
         </inertial>
     </link>
     <joint name="blw" type="continuous">
-        <origin xyz="-0.053292508052297460353 -0.046508209944849943085 -0.024000000000004365064" rpy="-1.5707963267948918951 -9.5936419862544196574e-15 -1.4372802468727412517" />
+        <origin xyz="-0.053292508052297571375 -0.046508209944849943085 -0.024000000000004288736" rpy="1.5707963267949012209 7.9710534704695101609e-14 -1.4372802468727035041" />
         <parent link="bl_anklemotor" />
         <child link="bl_wheel" />
@@ -771,7 +771,7 @@
         </collision>
         <inertial>
-            <origin xyz="0.018499888960637339563 1.3272597548194587806e-05 -0.014774229179233584405" rpy="0 0 0"/>
-            <mass value="0.041267529904965544185" />
-            <inertia ixx="1.230119964094838682e-05" ixy="-1.6133742293471586687e-09" ixz="2.126163018675682121e-10" iyy="1.4223599828696047078e-05" iyz="1.4267112581668452433e-10" izz="4.6158516095823752166e-06" />
+            <origin xyz="0.018499888960637339563 1.3272597548194584418e-05 -0.014774229179233589609" rpy="0 0 0"/>
+            <mass value="0.041267529904965537246" />
+            <inertia ixx="1.2301199640948390208e-05" ixy="-1.6133742293471528785e-09" ixz="2.1261630186769510678e-10" iyy="1.4223599828696047078e-05" iyz="1.4267112581666524068e-10" izz="4.6158516095823760636e-06" />
         </inertial>
     </link>
@@ -793,7 +793,7 @@
         </collision>
         <inertial>
-            <origin xyz="-0.0046325031628368451911 0.029950435987357082457 5.5999979714990694712e-16" rpy="0 0 0"/>
+            <origin xyz="-0.0046325031628368477932 0.029950435987357047762 5.599926671769394372e-16" rpy="0 0 0"/>
             <mass value="0.41604445274443546676" />
-            <inertia ixx="0.00069051715503048516961" ixy="-0.0028951365691400419294" ixz="2.245872099445990809e-08" iyy="0.018960630107717146853" iyz="-1.0250324667922003086e-07" izz="0.019624856180076557383" />
+            <inertia ixx="0.00069051715503048386856" ixy="-0.0028951365691400423631" ixz="2.2458720994459689714e-08" iyy="0.018960630107717146853" iyz="-1.0250324667921997792e-07" izz="0.019624856180076553913" />
         </inertial>
     </link>
@@ -817,5 +817,5 @@
             <origin xyz="0.009179146420314058738 0.0035713065058396789575 -0.0047499999999999270237" rpy="0 0 0"/>
             <mass value="0.013606078196486367723" />
-            <inertia ixx="8.9873051197638599787e-07" ixy="-8.3553864179412247474e-07" ixz="-6.3814463543586609943e-21" iyy="2.7211919051775411284e-06" iyz="-1.3280968007678257561e-21" izz="3.4319611912568939363e-06" />
+            <inertia ixx="8.9873051197638568024e-07" ixy="-8.3553864179412183946e-07" ixz="-6.1167485583416921384e-21" iyy="2.7211919051775402814e-06" iyz="-1.2089827925601897709e-21" izz="3.4319611912568930893e-06" />
         </inertial>
     </link>
@@ -839,5 +839,5 @@
             <origin xyz="9.3891908137244683985e-17 8.8318431344311387754e-17 -0.028750000000000029005" rpy="0 0 0"/>
             <mass value="0.012008474024564124924" />
-            <inertia ixx="3.4513655264616822869e-06" ixy="-3.242635199973633313e-22" ixz="-2.2433643952463179971e-22" iyy="3.4513655264616822869e-06" iyz="1.5622476239461400526e-22" izz="2.8556151230413454125e-07" />
+            <inertia ixx="3.4513655264616822869e-06" ixy="-3.308809648977875527e-22" ixz="-2.2433643952463179971e-22" iyy="3.4513655264616822869e-06" iyz="1.5622476239461400526e-22" izz="2.8556151230413454125e-07" />
         </inertial>
     </link>
@@ -859,7 +859,7 @@
         </collision>
         <inertial>
-            <origin xyz="-4.336808689942017736e-17 8.8470897274817161815e-17 0.020516655251079467942" rpy="0 0 0"/>
+            <origin xyz="-4.2500725161431773813e-17 8.8470897274817161815e-17 0.020516655251079467942" rpy="0 0 0"/>
             <mass value="0.013606078196486367723" />
-            <inertia ixx="3.394313300366512233e-06" ixy="1.144683057326582978e-07" ixz="-3.7661707272435695869e-23" iyy="3.0839206315490952579e-06" iyz="4.160907714125237401e-22" izz="5.7364967649520563078e-07" />
+            <inertia ixx="3.394313300366511386e-06" ixy="1.1446830573265832427e-07" ixz="-1.435408256792232265e-22" iyy="3.0839206315490939874e-06" iyz="4.9528238804368667924e-22" izz="5.736496764952055249e-07" />
         </inertial>
     </link>
@@ -881,6 +881,6 @@
         </collision>
         <inertial>
-            <origin xyz="2.3613122599928090328e-16 -2.3979336119469146679e-16 -0.0082589798435497296936" rpy="0 0 0"/>
-            <mass value="0.017189483651432656275" />
+            <origin xyz="2.3613202218671822299e-16 -2.3979300951305169181e-16 -0.0082589798435497296936" rpy="0 0 0"/>
+            <mass value="0.017189483651432659744" />
             <inertia ixx="2.7300446323037500655e-06" ixy="4.3175643094029759655e-24" ixz="4.1243337953494242241e-24" iyy="2.730044632303748795e-06" iyz="1.0343161054676291692e-24" izz="4.116384110236460945e-07" />
         </inertial>
@@ -937,5 +937,5 @@
             <origin xyz="0.0091791464203140483297 0.0035713065058395748741 5.1391182975812916335e-17" rpy="0 0 0"/>
             <mass value="0.013606078196486367723" />
-            <inertia ixx="8.9873051197638620963e-07" ixy="-8.3553864179412258062e-07" ixz="-6.3637276556021325388e-21" iyy="2.7211919051775390109e-06" iyz="-1.4316281780738464051e-21" izz="3.4319611912568952069e-06" />
+            <inertia ixx="8.98730511976385892e-07" ixy="-8.3553864179412194534e-07" ixz="-6.1213625506974658401e-21" iyy="2.7211919051775381638e-06" iyz="-1.2901814787539084507e-21" izz="3.4319611912568939363e-06" />
         </inertial>
     </link>
@@ -959,5 +959,5 @@
             <origin xyz="-7.2641545556528797078e-17 3.2676837039176398481e-17 -0.028750000000000001249" rpy="0 0 0"/>
             <mass value="0.012008474024564124924" />
-            <inertia ixx="3.4513655264616827105e-06" ixy="1.2603457792596389042e-22" ixz="9.1559138304309485887e-23" iyy="3.4513655264616822869e-06" iyz="-2.1584708677119758702e-24" izz="2.8556151230413454125e-07" />
+            <inertia ixx="3.4513655264616827105e-06" ixy="1.1941713302553966902e-22" ixz="9.1559138304309485887e-23" iyy="3.4513655264616822869e-06" iyz="-2.1584708677119758702e-24" izz="2.8556151230413454125e-07" />
         </inertial>
     </link>
@@ -979,7 +979,7 @@
         </collision>
         <inertial>
-            <origin xyz="-7.1340502949546191758e-17 -1.3227266504323154095e-16 0.020516655251079578964" rpy="0 0 0"/>
+            <origin xyz="-7.047314121155778821e-17 -1.3227266504323154095e-16 0.020516655251079578964" rpy="0 0 0"/>
             <mass value="0.013606078196486367723" />
-            <inertia ixx="3.394313300366512233e-06" ixy="1.1446830573265833751e-07" ixz="-1.435408256792232265e-22" iyy="3.0839206315490948344e-06" iyz="3.6228032351341928638e-22" izz="5.736496764952055249e-07" />
+            <inertia ixx="3.394313300366511386e-06" ixy="1.1446830573265836398e-07" ixz="-2.4941994408601076888e-22" iyy="3.0839206315490935638e-06" iyz="4.2823705034373387676e-22" izz="5.736496764952055249e-07" />
         </inertial>
     </link>
@@ -1001,6 +1001,6 @@
         </collision>
         <inertial>
-            <origin xyz="1.4100694636232458442e-17 -2.3805923228539552531e-16 -0.008258979843549701938" rpy="0 0 0"/>
-            <mass value="0.017189483651432656275" />
+            <origin xyz="1.4101490823669815125e-17 -2.3805888060375575033e-16 -0.008258979843549701938" rpy="0 0 0"/>
+            <mass value="0.017189483651432659744" />
             <inertia ixx="2.7300446323037500655e-06" ixy="-3.8663918950212358023e-24" ixz="-4.8362005466282607768e-23" iyy="2.730044632303749642e-06" iyz="1.4619118715956014005e-24" izz="4.1163841102364620038e-07" />
         </inertial>
