Commit message: Parameters finalised. Rover wheels parallel

File: src/ros/rover/new_rover_description/urdf/rover.urdf.xacro (robot description, xacro)
@@ -49,7 +49,7 @@
         </collision>
         <inertial>
-            <origin xyz="-6.060792462398293984e-05 0.022728017107731847413 0.026345212683551218896" rpy="0 0 0"/>
-            <mass value="7.6906345059941259024" />
-            <inertia ixx="0.44733237602571868097" ixy="-0.00012066720320063805338" ixz="-0.00020251363374965811637" iyy="0.1948873890676779963" iyz="0.0095851903407340489915" izz="0.56806231569085563482" />
+            <origin xyz="-6.0607924624055432307e-05 0.022728017107731385976 0.026345212683551333388" rpy="0 0 0"/>
+            <mass value="7.6906345059940734998" />
+            <inertia ixx="0.44733237602571951363" ixy="-0.00012066720320065034552" ixz="-0.00020251363374966605815" iyy="0.19488738906767741343" iyz="0.0095851903407342259333" izz="0.56806231569085596789" />
         </inertial>
     </link>
@@ -71,7 +71,7 @@
         </collision>
         <inertial>
-            <origin xyz="-0.0010899117823054075681 4.041380027214682658e-06 -0.1399993129761559485" rpy="0 0 0"/>
+            <origin xyz="-0.0010899117823054075681 4.0413800272146792699e-06 -0.1399993129761559485" rpy="0 0 0"/>
             <mass value="0.61929085260862060114" />
-            <inertia ixx="0.022394047093070124782" ixy="-6.3774127350866712475e-09" ixz="2.4803302240859229522e-10" iyy="0.022366401167997825017" iyz="-1.5472398701493753402e-08" izz="0.00052067562621966288761" />
+            <inertia ixx="0.022394047093070124782" ixy="-6.377412735086659667e-09" ixz="2.480330224217088465e-10" iyy="0.022366401167997825017" iyz="-1.5472398701492062645e-08" izz="0.00052067562621966299603" />
         </inertial>
     </link>
@@ -142,12 +142,12 @@
         </collision>
         <inertial>
-            <origin xyz="0.0039718182091793233918 -0.003873876506783426911 -0.053343546583699136265" rpy="0 0 0"/>
-            <mass value="3.344564958908655683" />
-            <inertia ixx="0.0097839331373918859286" ixy="0.013186544376772938933" ixz="0.0014152217803643308072" iyy="0.49540599288668402123" iyz="0.0001950135450044998206" izz="0.49156955837786198149" />
+            <origin xyz="0.0039718182091793893113 -0.0038738765067834204057 -0.053343546583699136265" rpy="0 0 0"/>
+            <mass value="3.3445649589086552389" />
+            <inertia ixx="0.0097839331373918841939" ixy="0.013186544376772937198" ixz="0.0014152217803643295062" iyy="0.4954059928866839102" iyz="0.0001950135450045003627" izz="0.49156955837786181496" />
         </inertial>
     </link>
     <link name="fr_ankle">
         <visual>
-            <origin xyz="-0.12415341931613699256 2.2898349882893853646e-16 -0.1250000000000002498" rpy="-1.570796326794896558 -0.13351607992219352572 1.2181229582827242785e-16" />
+            <origin xyz="-0.12415341931613710358 2.498001805406602216e-16 -0.12500000000000027756" rpy="-1.570796326794896558 -0.13351607992219355348 -7.6813912419263841209e-17" />
             <geometry>
                 <mesh filename="file://$(find new_rover_description)/meshes/fr_ankle.stl"/>
@@ -159,5 +159,5 @@
         <!-- Shapes for fr_ankle -->
         <collision>
-            <origin xyz="-0.11601914642063086702 2.2769578193000160333e-16 -0.10304929353177745555" rpy="-1.570796326794896558 0.0061101698267938975989 1.3715254847787124342e-16" />
+            <origin xyz="-0.11601914642063097804 2.4694101913642000327e-16 -0.1030492935317774833" rpy="-1.570796326794896558 0.0061101698267938863232 -6.1771469324893414164e-17" />
             <geometry>
                 <box size="0.032000000000000000666 0.080000000000000001665 0.05999999999999999778" />
@@ -165,5 +165,5 @@
         </collision>
         <collision>
-            <origin xyz="-0.091894553662955638651 2.3759514146060475226e-16 -0.16352745890207481816" rpy="-1.570796326794896558 -0.79674066942340771025 2.4737082664321076987e-17" />
+            <origin xyz="-0.091894553662955749673 2.5191347026720868665e-16 -0.16352745890207484591" rpy="-1.570796326794896558 -0.79674066942340782127 -1.7200454605793530007e-16" />
             <geometry>
                 <box size="0.020000000000000000416 0.080000000000000001665 0.05999999999999999778" />
@@ -171,5 +171,5 @@
         </collision>
         <collision>
-            <origin xyz="-0.063800853957741585076 2.4539417915154796666e-16 -0.19982021317550335837" rpy="-1.570796326794896558 -0.011343354647681706815 1.3524584140369868879e-16" />
+            <origin xyz="-0.063800853957741709976 2.5404739191211583917e-16 -0.19982021317550338613" rpy="-1.570796326794896558 -0.011343354647681722427 -6.3641160347330659717e-17" />
             <geometry>
                 <box size="0.025000000000000001388 0.030999999999999999778 0.05999999999999999778" />
@@ -177,5 +177,5 @@
         </collision>
         <collision>
-            <origin xyz="-0.06708178600672942693 2.2795692414257300287e-16 -0.044297919093382348565" rpy="-1.570796326794896558 0.80896192356999552242 2.5099986351094729997e-16" />
+            <origin xyz="-0.06708178600672955183 2.3759257712076676596e-16 -0.044297919093382362443" rpy="-1.570796326794896558 0.80896192356999563344 4.986565927720294372e-17" />
             <geometry>
                 <box size="0.01200000000000000025 0.075999999999999998113 0.05999999999999999778" />
@@ -183,5 +183,5 @@
         </collision>
         <collision>
-            <origin xyz="-0.10777838729006998519 2.2518949717502131371e-16 -0.069810716156365748564" rpy="-1.570796326794886566 1.5594529721472150108 9.7664942524092150172e-15" />
+            <origin xyz="-0.10777838729007011009 2.4286604753035148434e-16 -0.069810716156365762441" rpy="-1.570796326794886788 1.5594529721472150108 9.3806300299374657517e-15" />
             <geometry>
                 <box size="0.01200000000000000025 0.02999999999999999889 0.05999999999999999778" />
@@ -189,5 +189,5 @@
         </collision>
         <collision>
-            <origin xyz="-0.00045306036165808361016 2.3338633589782932004e-16 -0.010753702302991163808" rpy="1.13113734796077825e-16 0.0061101698267938975989 1.3715254847787124342e-16" />
+            <origin xyz="-0.00045306036165819463246 2.298399379395962547e-16 -0.010753702302991177686" rpy="1.1224846204185424354e-16 0.0061101698267938863232 -6.1771469324893414164e-17" />
             <geometry>
                 <cylinder length="0.025999999999999998807" radius="0.037999999999999999056" />
@@ -195,5 +195,5 @@
         </collision>
         <collision>
-            <origin xyz="-0.028495306304552395216 2.3030497367880861351e-16 -0.017582487382379469176" rpy="1.13113734796077825e-16 0.0061101698267938975989 1.3715254847787124342e-16" />
+            <origin xyz="-0.028495306304552506238 2.3232200630689366419e-16 -0.017582487382379483054" rpy="1.1224846204185424354e-16 0.0061101698267938863232 -6.1771469324893414164e-17" />
             <geometry>
                 <box size="0.02999999999999999889 0.05999999999999999778 0.01200000000000000025" />
@@ -201,12 +201,12 @@
         </collision>
         <inertial>
-            <origin xyz="-0.067658474648355532155 -0.00014463856991167397159 -0.0716246334329673634" rpy="0 0 0"/>
+            <origin xyz="-0.067658474648355657055 -0.00014463856991166535219 -0.0716246334329673634" rpy="0 0 0"/>
             <mass value="0.40704474660617540049" />
-            <inertia ixx="0.0016392589144157169653" ixy="-2.8493978195280827051e-06" ixz="-0.00080468641679309037013" iyy="0.002385090389839814376" iyz="-1.4225306394299746849e-06" izz="0.0011614760148504982631" />
+            <inertia ixx="0.0016392589144157158811" ixy="-2.8493978195283016631e-06" ixz="-0.00080468641679309058697" iyy="0.0023850903898398135086" iyz="-1.4225306394298707116e-06" izz="0.00116147601485049848" />
         </inertial>
     </link>
     <link name="fr_anklemotor">
         <visual>
-            <origin xyz="-0.052882847177904201974 -0.084794424783462968298 -0.024000000000003525458" rpy="4.6845761985724690052e-16 -3.6608319069462070423e-15 2.1539843060241694836e-17" />
+            <origin xyz="-0.052882847177904201974 -0.084794424783463051565 -0.024000000000003601786" rpy="4.4687731154414894265e-16 -3.6583860602508457291e-15 2.2874474444740127584e-17" />
             <geometry>
                 <mesh filename="file://$(find new_rover_description)/meshes/fr_anklemotor.stl"/>
@@ -217,5 +217,5 @@
         </visual>
         <collision>
-            <origin xyz="-0.052882847177904201974 -0.084794424783462968298 -0.024000000000003525458" rpy="4.6845761985724690052e-16 -3.6608319069462070423e-15 2.1539843060241694836e-17" />
+            <origin xyz="-0.052882847177904201974 -0.084794424783463051565 -0.024000000000003601786" rpy="4.4687731154414894265e-16 -3.6583860602508457291e-15 2.2874474444740127584e-17" />
             <geometry>
                 <mesh filename="file://$(find new_rover_description)/meshes/fr_anklemotor.stl"/>
@@ -223,12 +223,12 @@
         </collision>
         <inertial>
-            <origin xyz="-0.021958993625958544982 0.035623040808488048992 -0.023997480138994761734" rpy="0 0 0"/>
-            <mass value="0.67137268218562695665" />
-            <inertia ixx="0.00067219001428469411438" ixy="-3.590510672107426833e-05" ixz="7.9146449530338902493e-09" iyy="0.0010088029360243425028" iyz="6.7337379884079747473e-08" izz="0.0010273836245733511396" />
+            <origin xyz="-0.021958993625958635187 0.035623040808487965725 -0.023997480138994841531" rpy="0 0 0"/>
+            <mass value="0.67137268218562584643" />
+            <inertia ixx="0.00067219001428469389754" ixy="-3.5905106721073943069e-05" ixz="7.914644953418578865e-09" iyy="0.0010088029360243383828" iyz="6.7337379884156059847e-08" izz="0.001027383624573347887" />
         </inertial>
     </link>
     <link name="fr_wheel">
         <visual>
-            <origin xyz="0 -1.0408340855860842566e-16 -1.1102230246251565404e-16" rpy="-1.985058964698083451e-17 1.1378066708760287058e-16 4.352542615723205238e-17" />
+            <origin xyz="0 1.7347234759768070944e-18 0" rpy="-2.1979634337389811138e-17 5.4832000926005038323e-17 3.4959276618369156618e-17" />
             <geometry>
                 <mesh filename="file://$(find new_rover_description)/meshes/fr_wheel.stl"/>
@@ -240,5 +240,5 @@
         <!-- Shapes for fr_wheel -->
         <collision>
-            <origin xyz="0 -1.0408340855860842566e-16 -1.1102230246251565404e-16" rpy="-1.985058964698083451e-17 1.1378066708760287058e-16 4.352542615723205238e-17" />
+            <origin xyz="0 1.7347234759768070944e-18 0" rpy="-2.1979634337389811138e-17 5.4832000926005038323e-17 3.4959276618369156618e-17" />
             <geometry>
                 <cylinder length="0.16000000000000000333" radius="0.15700000000000000067" />
@@ -246,11 +246,11 @@
         </collision>
         <inertial>
-            <origin xyz="-1.3294988576507908417e-07 -1.1207731120965171372e-07 1.2648623649607755492e-05" rpy="0 0 0"/>
-            <mass value="1.8501412404055219696" />
-            <inertia ixx="0.020701719473909981073" ixy="2.9104723315617180571e-05" ixz="1.0888320723437134582e-08" iyy="0.020861663662014574144" iyz="1.4322179505752822895e-08" izz="0.032713974764007960894" />
+            <origin xyz="-1.3294988577306983418e-07 -1.1207731109163011331e-07 1.2648623649714051351e-05" rpy="0 0 0"/>
+            <mass value="1.8501412404055235239" />
+            <inertia ixx="0.020701719473909988012" ixy="2.9104723315619284601e-05" ixz="1.0888320726562165034e-08" iyy="0.020861663662014584553" iyz="1.4322179502165461347e-08" izz="0.032713974764007967833" />
         </inertial>
     </link>
     <joint name="frw" type="continuous">
-        <origin xyz="0.053292508052297460353 0.046508209944849887574 -0.024000000000004365064" rpy="1.5707963267948921171 0.28883585951286211424 -1.4372802468727061687" />
+        <origin xyz="0.053292508052297571375 0.046508209944849832063 -0.024000000000004462208" rpy="1.5707963267948921171 0.28883585951287249483 -1.4372802468727092773" />
         <parent link="fr_anklemotor" />
         <child link="fr_wheel" />
@@ -260,5 +260,5 @@
     </joint>
     <joint name="fr_ankle_motor_join" type="fixed">
-        <origin xyz="-0.060453419316137124717 0.023999999999999910294 -0.20200000000000017941" rpy="-1.570796326794896558 -0.13351607992219347021 -1.0877595247438724004e-14" />
+        <origin xyz="-0.060453419316137124717 0.023999999999999993561 -0.20200000000000020717" rpy="-1.570796326794896558 -0.13351607992219358123 -3.5655310271105493798e-14" />
         <parent link="fr_ankle" />
         <child link="fr_anklemotor" />
@@ -268,5 +268,5 @@
     </joint>
     <joint name="frp" type="revolute">
-        <origin xyz="-0.47013767878255974253 -0.026528595964174089827 -0.10561814293695781508" rpy="1.5707963267949005548 0.78539816339749224383 3.1148421188216199873" />
+        <origin xyz="-0.47013767878255985355 -0.026528595964174034316 -0.1056181429369579261" rpy="1.5707963267949009989 0.86524872200545932532 3.11484211882162354" />
         <parent link="rightleg" />
         <child link="fr_ankle" />
@@ -277,5 +277,5 @@
     <link name="br_ankle">
         <visual>
-            <origin xyz="-0.12415341931613710358 2.8449465006019636348e-16 -0.12500000000000027756" rpy="-1.570796326794896558 -0.13351607992219349796 4.5136769332523039787e-17" />
+            <origin xyz="-0.12415341931613704807 2.6367796834847467835e-16 -0.12500000000000027756" rpy="-1.570796326794896558 -0.13351607992219355348 2.8933441911753607959e-17" />
             <geometry>
                 <mesh filename="file://$(find new_rover_description)/meshes/br_ankle.stl"/>
@@ -287,5 +287,5 @@
         <!-- Shapes for br_ankle -->
         <collision>
-            <origin xyz="-0.11601914642063097804 2.8279533064878078663e-16 -0.1030492935317774833" rpy="-1.570796326794896558 0.0061101698267939123441 5.9049099273200022083e-17" />
+            <origin xyz="-0.11601914642063092253 2.6183924338317619713e-16 -0.1030492935317774833" rpy="-1.570796326794896558 0.0061101698267938854559 4.289696008220557727e-17" />
             <geometry>
                 <box size="0.032000000000000000666 0.080000000000000001665 0.05999999999999999778" />
@@ -293,5 +293,5 @@
         </collision>
         <collision>
-            <origin xyz="-0.091894553662955735795 2.901969999439457232e-16 -0.16352745890207484591" rpy="-1.570796326794896558 -0.79674066942340759923 -4.2902353975772878232e-17" />
+            <origin xyz="-0.091894553662955694162 2.6887324082196188064e-16 -0.16352745890207484591" rpy="-1.570796326794896558 -0.79674066942340771025 -5.9429607503262674962e-17" />
             <geometry>
                 <box size="0.020000000000000000416 0.080000000000000001665 0.05999999999999999778" />
@@ -299,5 +299,5 @@
         </collision>
         <collision>
-            <origin xyz="-0.063800853957741682221 2.9543452362823638508e-16 -0.19982021317550338613" rpy="-1.570796326794896558 -0.011343354647681691202 5.731987495584140101e-17" />
+            <origin xyz="-0.063800853957741640587 2.7367015811300166119e-16 -0.19982021317550338613" rpy="-1.570796326794896558 -0.011343354647681720693 4.1161373355957363927e-17" />
             <geometry>
                 <box size="0.025000000000000001388 0.030999999999999999778 0.05999999999999999778" />
@@ -305,5 +305,5 @@
         </collision>
         <collision>
-            <origin xyz="-0.067081786006729537952 2.7983475309870370178e-16 -0.044297919093382376321" rpy="-1.570796326794896558 0.80896192356999552242 1.6229912036341811687e-16" />
+            <origin xyz="-0.067081786006729482441 2.5806669757403521094e-16 -0.044297919093382362443" rpy="-1.570796326794896558 0.80896192356999552242 1.4652687338504176792e-16" />
             <geometry>
                 <box size="0.01200000000000000025 0.075999999999999998113 0.05999999999999999778" />
@@ -311,5 +311,5 @@
         </collision>
         <collision>
-            <origin xyz="-0.10777838729007009622 2.799839143349007714e-16 -0.069810716156365762441" rpy="-1.570796326794886566 1.5594529721472150108 8.7920590409391449246e-15" />
+            <origin xyz="-0.1077783872900700407 2.5888258661389069449e-16 -0.069810716156365762441" rpy="-1.5707963267948874542 1.5594529721472150108 8.808038638231368023e-15" />
             <geometry>
                 <box size="0.01200000000000000025 0.02999999999999999889 0.05999999999999999778" />
@@ -317,5 +317,5 @@
         </collision>
         <collision>
-            <origin xyz="-0.00045306036165816687689 2.8040546740891948302e-16 -0.010753702302991177686" rpy="1.1329300829137536362e-16 0.0061101698267939123441 5.9049099273200022083e-17" />
+            <origin xyz="-0.00045306036165812524352 2.5754883940531762658e-16 -0.010753702302991177686" rpy="1.0517633863451059952e-16 0.0061101698267938854559 4.289696008220557727e-17" />
             <geometry>
                 <cylinder length="0.025999999999999998807" radius="0.037999999999999999056" />
@@ -323,5 +323,5 @@
         </collision>
         <collision>
-            <origin xyz="-0.028495306304552478482 2.7944312014866511832e-16 -0.017582487382379483054" rpy="1.1329300829137536362e-16 0.0061101698267939123441 5.9049099273200022083e-17" />
+            <origin xyz="-0.028495306304552450727 2.5704198611026095152e-16 -0.017582487382379483054" rpy="1.0517633863451059952e-16 0.0061101698267938854559 4.289696008220557727e-17" />
             <geometry>
                 <box size="0.02999999999999999889 0.05999999999999999778 0.01200000000000000025" />
@@ -329,12 +329,12 @@
         </collision>
         <inertial>
-            <origin xyz="-0.0676584746483556293 -0.00014463856991162531802 -0.0716246334329673634" rpy="0 0 0"/>
-            <mass value="0.40704474660617540049" />
-            <inertia ixx="0.0016392589144157167485" ixy="-2.8493978195284693756e-06" ixz="-0.00080468641679309080381" iyy="0.0023850903898398135086" iyz="-1.4225306394299431329e-06" izz="0.0011614760148504986968" />
+            <origin xyz="-0.067658474648355559911 -0.00014463856991164654128 -0.0716246334329673634" rpy="0 0 0"/>
+            <mass value="0.40704474660617528947" />
+            <inertia ixx="0.0016392589144157156643" ixy="-2.8493978195285714431e-06" ixz="-0.00080468641679309015329" iyy="0.0023850903898398135086" iyz="-1.4225306394299465211e-06" izz="0.0011614760148504982631" />
         </inertial>
     </link>
     <link name="br_anklemotor">
         <visual>
-            <origin xyz="-0.052882847177904201974 -0.084794424783462996054 -0.024000000000003515049" rpy="4.5456107424398069396e-16 -3.6175975286945226714e-15 2.6973788537147245028e-17" />
+            <origin xyz="-0.052882847177904201974 -0.084794424783463023809 -0.02400000000000357403" rpy="4.515177172886114136e-16 -3.5943511837517746456e-15 2.1213417495586426316e-17" />
             <geometry>
                 <mesh filename="file://$(find new_rover_description)/meshes/br_anklemotor.stl"/>
@@ -345,5 +345,5 @@
         </visual>
         <collision>
-            <origin xyz="-0.052882847177904201974 -0.084794424783462996054 -0.024000000000003515049" rpy="4.5456107424398069396e-16 -3.6175975286945226714e-15 2.6973788537147245028e-17" />
+            <origin xyz="-0.052882847177904201974 -0.084794424783463023809 -0.02400000000000357403" rpy="4.515177172886114136e-16 -3.5943511837517746456e-15 2.1213417495586426316e-17" />
             <geometry>
                 <mesh filename="file://$(find new_rover_description)/meshes/br_anklemotor.stl"/>
@@ -351,12 +351,12 @@
         </collision>
         <inertial>
-            <origin xyz="-0.021958993625958579676 0.035623040808488035114 -0.023997480138994754795" rpy="0 0 0"/>
-            <mass value="0.67137268218562629052" />
-            <inertia ixx="0.0006721900142846942228" ixy="-3.5905106721074166686e-05" ixz="7.914644953067262024e-09" iyy="0.0010088029360243414186" iyz="6.7337379884058293717e-08" izz="0.0010273836245733500554" />
+            <origin xyz="-0.021958993625958652535 0.03562304080848799348 -0.023997480138994817245" rpy="0 0 0"/>
+            <mass value="0.67137268218562540234" />
+            <inertia ixx="0.00067219001428469411438" ixy="-3.5905106721073970174e-05" ixz="7.9146449531624854017e-09" iyy="0.0010088029360243388165" iyz="6.7337379884114131717e-08" izz="0.0010273836245733470197" />
         </inertial>
     </link>
     <link name="br_wheel">
         <visual>
-            <origin xyz="-2.7755575615628913511e-17 -2.7755575615628913511e-17 0" rpy="3.7777461231176036507e-17 1.4728947712454568872e-16 4.9611706014273251116e-17" />
+            <origin xyz="-2.7755575615628913511e-17 2.7755575615628913511e-17 0" rpy="-2.4576217954427888305e-17 1.4101281192975104818e-16 4.8942876908257451025e-18" />
             <geometry>
                 <mesh filename="file://$(find new_rover_description)/meshes/br_wheel.stl"/>
@@ -368,5 +368,5 @@
         <!-- Shapes for br_wheel -->
         <collision>
-            <origin xyz="-2.7755575615628913511e-17 -2.7755575615628913511e-17 0" rpy="3.7777461231176036507e-17 1.4728947712454568872e-16 4.9611706014273251116e-17" />
+            <origin xyz="-2.7755575615628913511e-17 2.7755575615628913511e-17 0" rpy="-2.4576217954427888305e-17 1.4101281192975104818e-16 4.8942876908257451025e-18" />
             <geometry>
                 <cylinder length="0.16000000000000000333" radius="0.15700000000000000067" />
@@ -374,11 +374,11 @@
         </collision>
         <inertial>
-            <origin xyz="-1.3294988579020083731e-07 -1.1207731110083104841e-07 1.2648623649721515405e-05" rpy="0 0 0"/>
-            <mass value="1.8501412404055210814" />
-            <inertia ixx="0.020701719473909994951" ixy="2.9104723315619088089e-05" ixz="1.0888320728761805373e-08" iyy="0.020861663662014581083" iyz="1.4322179504180785994e-08" izz="0.032713974764007995588" />
+            <origin xyz="-1.3294988579468931784e-07 -1.1207731105968185696e-07 1.2648623649719740024e-05" rpy="0 0 0"/>
+            <mass value="1.8501412404055208594" />
+            <inertia ixx="0.020701719473909988012" ixy="2.9104723315617475339e-05" ixz="1.088832072359006208e-08" iyy="0.020861663662014577614" iyz="1.4322179504244014025e-08" izz="0.032713974764007967833" />
         </inertial>
     </link>
     <joint name="brw" type="continuous">
-        <origin xyz="0.053292508052299680799 0.046508209944850331663 -0.024000000000004354656" rpy="1.5707963267948881203 -0.97072198262952236192 -1.4372802468726910696" />
+        <origin xyz="0.053292508052299569776 0.046508209944850276152 -0.024000000000004600986" rpy="1.5707963267948887864 -0.97072198262967801519 -1.4372802468726915137" />
         <parent link="br_anklemotor" />
         <child link="br_wheel" />
@@ -388,5 +388,5 @@
     </joint>
     <joint name="br_ankle_motor_join" type="fixed">
-        <origin xyz="-0.060453419316137235739 0.023999999999999913763 -0.20200000000000020717" rpy="-1.570796326794896558 -0.13351607992219374776 9.6061137978268971728e-16" />
+        <origin xyz="-0.060453419316137235739 0.023999999999999951927 -0.20200000000000017941" rpy="-1.570796326794896558 -0.13351607992219344245 -2.7584080234938445875e-15" />
         <parent link="br_ankle" />
         <child link="br_anklemotor" />
@@ -396,5 +396,5 @@
     </joint>
     <joint name="brp" type="revolute">
-        <origin xyz="0.47757721986905654621 -0.051886525235696062675 -0.1080377003968426286" rpy="-1.570796326794901665 0.78539816339744172868 -0.026750534768215941672" />
+        <origin xyz="0.4775772198690564907 -0.05188652523569609043 -0.1080377003968426286" rpy="-1.5707963267948985564 0.86524793678182976286 -0.026750534768215854936" />
         <parent link="rightleg" />
         <child link="br_ankle" />
@@ -477,12 +477,12 @@
         </collision>
         <inertial>
-            <origin xyz="0.0015090549950636225531 0.0038104460972356269874 -0.054086077114172882718" rpy="0 0 0"/>
-            <mass value="3.3446449370376427623" />
-            <inertia ixx="0.0098743756931102995289" ixy="-0.013941425601711875115" ixz="0.00024306030673493643512" iyy="0.50330609956391281212" iyz="-0.00018934670901919053998" izz="0.49945087581952996025" />
+            <origin xyz="0.0015090549949552927583 0.003810446097231147064 -0.054086077114160552304" rpy="0 0 0"/>
+            <mass value="3.3446449370365796128" />
+            <inertia ixx="0.0098743756931083757206" ixy="-0.013941425601706268489" ixz="0.00024306030672006825573" iyy="0.50330609956377958536" iyz="-0.00018934670901982211485" izz="0.49945087581939817678" />
         </inertial>
     </link>
     <link name="fl_ankle">
         <visual>
-            <origin xyz="0.12415341931613699256 -2.5673907444456744997e-16 -0.12500000000000022204" rpy="-1.57079632679489678 0.13351607992219349796 -7.4321158163832004697e-17" />
+            <origin xyz="0.12415341931613710358 -2.2204460492503130808e-16 -0.1250000000000002498" rpy="-1.57079632679489678 0.13351607992219352572 -3.311491634449110225e-17" />
             <geometry>
                 <mesh filename="file://$(find new_rover_description)/meshes/fl_ankle.stl"/>
@@ -494,5 +494,5 @@
         <!-- Shapes for fl_ankle -->
         <collision>
-            <origin xyz="0.11601914642063086702 -2.5378889907506002558e-16 -0.10304929353177742779" rpy="-1.57079632679489678 0.0061101698267938975989 3.141592653589793116" />
+            <origin xyz="0.11601914642063097804 -2.1935154896097820824e-16 -0.10304929353177745555" rpy="-1.57079632679489678 0.0061101698267939140788 3.141592653589793116" />
             <geometry>
                 <box size="0.032000000000000000666 0.080000000000000001665 0.05999999999999999778" />
@@ -500,5 +500,5 @@
         </collision>
         <collision>
-            <origin xyz="0.091894553662955624773 -2.5916146300540073653e-16 -0.1635274589020747904" rpy="-1.57079632679489678 -0.79674066942340759923 3.141592653589793116" />
+            <origin xyz="0.091894553662955749673 -2.2595666849132184554e-16 -0.16352745890207481816" rpy="-1.57079632679489678 -0.79674066942340771025 3.141592653589793116" />
             <geometry>
                 <box size="0.020000000000000000416 0.080000000000000001665 0.05999999999999999778" />
@@ -506,5 +506,5 @@
         </collision>
         <collision>
-            <origin xyz="0.063800853957741571199 -2.6157919229030686768e-16 -0.19982021317550330286" rpy="-1.57079632679489678 -0.01134335464768170508 3.141592653589793116" />
+            <origin xyz="0.063800853957741709976 -2.2968198460293791177e-16 -0.19982021317550335837" rpy="-1.57079632679489678 -0.011343354647681694672 3.141592653589793116" />
             <geometry>
                 <box size="0.025000000000000001388 0.030999999999999999778 0.05999999999999999778" />
@@ -512,5 +512,5 @@
         </collision>
         <collision>
-            <origin xyz="0.06708178600672942693 -2.4428404318959647598e-16 -0.04429791909338232081" rpy="-1.57079632679489678 0.80896192356999552242 -3.141592653589793116" />
+            <origin xyz="0.06708178600672955183 -2.1166793586556722328e-16 -0.044297919093382348565" rpy="-1.57079632679489678 0.80896192356999563344 -3.141592653589793116" />
             <geometry>
                 <box size="0.01200000000000000025 0.075999999999999998113 0.05999999999999999778" />
@@ -518,5 +518,5 @@
         </collision>
         <collision>
-            <origin xyz="0.10777838729006998519 -2.4956302771801039225e-16 -0.069810716156365720808" rpy="-1.57079632679490655 1.5594529721472150108 -3.141592653589783346" />
+            <origin xyz="0.10777838729007011009 -2.1534499261437189196e-16 -0.069810716156365734686" rpy="-1.57079632679490655 1.5594529721472150108 -3.1415926535897829019" />
             <geometry>
                 <box size="0.01200000000000000025 0.02999999999999999889 0.05999999999999999778" />
@@ -524,5 +524,5 @@
         </collision>
         <collision>
-            <origin xyz="0.00045306036165805585458 -2.3656626417547686098e-16 -0.010753702302991136053" rpy="-1.1242822262008714609e-16 0.0061101698267938975989 3.141592653589793116" />
+            <origin xyz="0.00045306036165819463246 -2.066036274581091018e-16 -0.010753702302991149931" rpy="-1.1162719770636109546e-16 0.0061101698267939140788 3.141592653589793116" />
             <geometry>
                 <cylinder length="0.025999999999999998807" radius="0.037999999999999999056" />
@@ -530,5 +530,5 @@
         </collision>
         <collision>
-            <origin xyz="0.028495306304552381338 -2.3899476924491850661e-16 -0.017582487382379441421" rpy="-1.1242822262008714609e-16 0.0061101698267938975989 3.141592653589793116" />
+            <origin xyz="0.028495306304552506238 -2.0788807782892385009e-16 -0.017582487382379455298" rpy="-1.1162719770636109546e-16 0.0061101698267939140788 3.141592653589793116" />
             <geometry>
                 <box size="0.02999999999999999889 0.05999999999999999778 0.01200000000000000025" />
@@ -536,12 +536,12 @@
         </collision>
         <inertial>
-            <origin xyz="0.067658474648355532155 0.00014463856991165860303 -0.071624633432967307889" rpy="0 0 0"/>
-            <mass value="0.40704474660617523396" />
-            <inertia ixx="0.0016392589144157156643" ixy="-2.8493978195287798132e-06" ixz="0.00080468641679309080381" iyy="0.0023850903898398126413" iyz="1.4225306394298241248e-06" izz="0.0011614760148504982631" />
+            <origin xyz="0.0676584746483556293 0.00014463856991168868964 -0.071624633432967335644" rpy="0 0 0"/>
+            <mass value="0.40704474660617545601" />
+            <inertia ixx="0.0016392589144157152306" ixy="-2.8493978195286015128e-06" ixz="0.00080468641679309026171" iyy="0.0023850903898398135086" iyz="1.4225306394297637737e-06" izz="0.0011614760148504982631" />
         </inertial>
     </link>
     <link name="fl_anklemotor">
         <visual>
-            <origin xyz="0.052882847177904090952 0.084794424783462968298 -0.024000000000003567091" rpy="3.1415926535897926719 3.6350210430096300376e-15 5.6926304281998261602e-18" />
+            <origin xyz="0.052882847177904090952 0.084794424783463023809 -0.024000000000003546274" rpy="3.1415926535897926719 3.5630644103241003019e-15 -4.5251936750014645249e-18" />
             <geometry>
                 <mesh filename="file://$(find new_rover_description)/meshes/fl_anklemotor.stl"/>
@@ -552,5 +552,5 @@
         </visual>
         <collision>
-            <origin xyz="0.052882847177904090952 0.084794424783462968298 -0.024000000000003567091" rpy="3.1415926535897926719 3.6350210430096300376e-15 5.6926304281998261602e-18" />
+            <origin xyz="0.052882847177904090952 0.084794424783463023809 -0.024000000000003546274" rpy="3.1415926535897926719 3.5630644103241003019e-15 -4.5251936750014645249e-18" />
             <geometry>
                 <mesh filename="file://$(find new_rover_description)/meshes/fl_anklemotor.stl"/>
@@ -558,12 +558,12 @@
         </collision>
         <inertial>
-            <origin xyz="0.021958993625958444368 -0.035623040808488048992 -0.023997480138994803367" rpy="0 0 0"/>
-            <mass value="0.67137268218562673461" />
-            <inertia ixx="0.00067219001428469411438" ixy="-3.5905106721074241225e-05" ixz="-7.914644952971332234e-09" iyy="0.0010088029360243420691" iyz="-6.7337379884061734788e-08" izz="0.0010273836245733513565" />
+            <origin xyz="0.021958993625958531104 -0.035623040808487951847 -0.02399748013899478255" rpy="0 0 0"/>
+            <mass value="0.67137268218562573541" />
+            <inertia ixx="0.00067219001428469400596" ixy="-3.5905106721073929517e-05" ixz="-7.9146449532461067442e-09" iyy="0.0010088029360243383828" iyz="-6.7337379884146530727e-08" izz="0.001027383624573346586" />
         </inertial>
     </link>
     <link name="fl_wheel">
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