Commit message: Rotated the rover and implemented correct zero positions

File: src/ros/rover/new_rover_description/urdf/rover.urdf.xacro (robot description, xacro)
@@ -27,5 +27,5 @@
     <link name="chassis">
         <visual>
-            <origin xyz="0 0 0" rpy="-1.7225464241988315416e-16 -5.3673954127953012992e-32 4.9303806576313237838e-32" />
+            <origin xyz="0 0 0" rpy="-1.4216575903928091376e-14 -2.4289199034476236505e-16 1.57079632679489678" />
             <geometry>
                 <mesh filename="file://$(find new_rover_description)/meshes/chassis.stl"/>
@@ -37,5 +37,5 @@
         <!-- Shapes for chassis -->
         <collision>
-            <origin xyz="1.2023483457100103294e-32 0.1725000000000000977 0.0234999999999999723" rpy="-1.7225464241988315416e-16 -5.3673954127953012992e-32 4.9303806576313237838e-32" />
+            <origin xyz="-0.17250000000000492717 -3.1536932067734256925e-17 0.023499999999998209821" rpy="-1.4216575903928091376e-14 -2.4289199034476236505e-16 1.57079632679489678" />
             <geometry>
                 <box size="0.47999999999999998224 0.54500000000000003997 0.1749999999999999889" />
@@ -43,5 +43,5 @@
         </collision>
         <collision>
-            <origin xyz="-1.2005115520421823681e-32 -0.22700000000000009059 0.03350000000000005751" rpy="-1.7225464241988315416e-16 -5.3673954127953012992e-32 4.9303806576313237838e-32" />
+            <origin xyz="0.22700000000000641887 2.5852545899575362104e-17 0.033500000000004179213" rpy="-1.4216575903928091376e-14 -2.4289199034476236505e-16 1.57079632679489678" />
             <geometry>
                 <box size="0.34000000000000002442 0.26000000000000000888 0.19500000000000000666" />
@@ -49,12 +49,12 @@
         </collision>
         <inertial>
-            <origin xyz="-6.0607924624055432307e-05 0.022728017107731385976 0.026345212683551333388" rpy="0 0 0"/>
-            <mass value="7.6906345059940734998" />
-            <inertia ixx="0.44733237602571951363" ixy="-0.00012066720320065034552" ixz="-0.00020251363374966605815" iyy="0.19488738906767741343" iyz="0.0095851903407342259333" izz="0.56806231569085596789" />
+            <origin xyz="-0.022728017107732267216 -6.0607924624050736357e-05 0.02634521268355138196" rpy="0 0 0"/>
+            <mass value="7.6906345059940406372" />
+            <inertia ixx="0.19488738906768895975" ixy="0.00012066720320064144151" ixz="-0.0095851903407318372191" iyy="0.44733237602571790381" iyz="-0.00020251363374969993947" izz="0.56806231569088649902" />
         </inertial>
     </link>
     <link name="crossbar">
         <visual>
-            <origin xyz="-2.7755575615624180345e-17 -5.0143501740629135245e-17 -0.14100000000000956213" rpy="1.570796326794896558 1.570796326794896558 0" />
+            <origin xyz="-2.7755575615624322094e-17 -5.0143501740629135245e-17 -0.14100000000000956213" rpy="1.570796326794896558 1.570796326794896558 0" />
             <geometry>
                 <mesh filename="file://$(find new_rover_description)/meshes/crossbar.stl"/>
@@ -64,19 +64,13 @@
             </material>
         </visual>
-        <collision>
-            <origin xyz="-2.7755575615624180345e-17 -5.0143501740629135245e-17 -0.14100000000000956213" rpy="1.570796326794896558 1.570796326794896558 0" />
-            <geometry>
-                <mesh filename="file://$(find new_rover_description)/meshes/crossbar.stl"/>
-            </geometry>
-        </collision>
-        <inertial>
-            <origin xyz="-0.0010899117823054075681 4.0413800272146792699e-06 -0.1399993129761559485" rpy="0 0 0"/>
+        <inertial>
+            <origin xyz="-0.0010899117823054075681 4.0413800272146868932e-06 -0.1399993129761559485" rpy="0 0 0"/>
             <mass value="0.61929085260862060114" />
-            <inertia ixx="0.022394047093070124782" ixy="-6.377412735086659667e-09" ixz="2.480330224217088465e-10" iyy="0.022366401167997825017" iyz="-1.5472398701492062645e-08" izz="0.00052067562621966299603" />
+            <inertia ixx="0.022394047093070124782" ixy="-6.3774127350866025915e-09" ixz="2.4803302242181307125e-10" iyy="0.022366401167997825017" iyz="-1.5472398701492635054e-08" izz="0.00052067562621966299603" />
         </inertial>
     </link>
     <link name="rightleg">
         <visual>
-            <origin xyz="-7.9461177221469483058e-19 7.285838599104098493e-20 -0.001000000000000667022" rpy="-3.4694469519552373626e-18 -3.7838655819743790435e-17 -2.5742563695788228314e-18" />
+            <origin xyz="-7.9461177221464860826e-19 7.2858385991028658978e-20 -0.001000000000000667022" rpy="-3.4694469519535448553e-18 -3.7838655819744067769e-17 -1.939189151781589847e-18" />
             <geometry>
                 <mesh filename="file://$(find new_rover_description)/meshes/rightleg.stl"/>
@@ -88,5 +82,5 @@
         <!-- Shapes for rightleg -->
         <collision>
-            <origin xyz="-7.9461177221469483058e-19 7.285838599104098493e-20 -0.001000000000000667022" rpy="-3.4694469519552373626e-18 -3.7838655819743790435e-17 -2.5742563695788228314e-18" />
+            <origin xyz="-7.9461177221464860826e-19 7.2858385991028658978e-20 -0.001000000000000667022" rpy="-3.4694469519535448553e-18 -3.7838655819744067769e-17 -1.939189151781589847e-18" />
             <geometry>
                 <cylinder length="0.058000000000000002942" radius="0.042999999999999996558" />
@@ -94,5 +88,5 @@
         </collision>
         <collision>
-            <origin xyz="-0.08543333675807499028 0.0098574827027250004619 -0.008346760000000673016" rpy="-0.12217294850606505441 1.308997029405494894 -0.23561907663390052603" />
+            <origin xyz="-0.085433336758075004158 0.0098574827027250004619 -0.008346760000000673016" rpy="-0.12217294850606505441 1.308997029405494894 -0.23561907663390049827" />
             <geometry>
                 <cylinder length="0.089999999999999996669" radius="0.02999999999999999889" />
@@ -100,5 +94,5 @@
         </collision>
         <collision>
-            <origin xyz="-0.31437167947314498262 0.038053876881360006179 -0.0660330377000006713" rpy="-0.12217302310744593274 1.3264501982056555729 -0.23561907663390055379" />
+            <origin xyz="-0.31437167947314503813 0.038053876881360006179 -0.0660330377000006713" rpy="-0.12217302310744593274 1.3264501982056553508 -0.23561907663390049827" />
             <geometry>
                 <cylinder length="0.39000000000000001332" radius="0.025000000000000001388" />
@@ -106,5 +100,5 @@
         </collision>
         <collision>
-            <origin xyz="-0.4536556182500000034 -0.0013318353999999977145 -0.10360017400000068322" rpy="2.2332973632374404714e-18 0.27925237217133341838 3.1066861154931633138" />
+            <origin xyz="-0.45365561825000011442 -0.0013318353999999979313 -0.10360017400000068322" rpy="2.2332973632356705417e-18 0.27925237217133336287 3.1066861154931633138" />
             <geometry>
                 <box size="0.105999999999999997 0.06500000000000000222 0.076999999999999999001" />
@@ -112,5 +106,5 @@
         </collision>
         <collision>
-            <origin xyz="-0.44472929399999999722 -0.0099999999999999984734 -0.032885924000000683887" rpy="3.5918351426043374596e-18 0.26179929927377626475 3.141592653589793116" />
+            <origin xyz="-0.44472929400000010824 -0.010000000000000000208 -0.032885924000000683887" rpy="3.5918351426025856337e-18 0.26179929927377615373 3.141592653589793116" />
             <geometry>
                 <cylinder length="0.051999999999999997613" radius="0.044999999999999998335" />
@@ -118,5 +112,5 @@
         </collision>
         <collision>
-            <origin xyz="0.085869139396912513851 0.0045695473361450009153 -0.008457175000000665202" rpy="0.069813040387381189444 1.3089970756114859274 -3.0194199283152816093" />
+            <origin xyz="0.085869139396912527729 0.0045695473361450009153 -0.008457175000000665202" rpy="0.069813040387381189444 1.3089970756114859274 -3.0194199283152816093" />
             <geometry>
                 <cylinder length="0.089999999999999996669" radius="0.02999999999999999889" />
@@ -124,5 +118,5 @@
         </collision>
         <collision>
-            <origin xyz="0.31601584183032671582 0.019116378127553800698 -0.066387337800000653654" rpy="0.069812975010840438994 1.326450241590472201 -3.0194199283152811653" />
+            <origin xyz="0.31601584183032677133 0.019116378127553800698 -0.066387337800000653654" rpy="0.069812975010840438994 1.326450241590471979 -3.0194199283152816093" />
             <geometry>
                 <cylinder length="0.39000000000000001332" radius="0.025000000000000001388" />
@@ -130,5 +124,5 @@
         </collision>
         <collision>
-            <origin xyz="0.46313595625000003597 -0.024684938349999997753 -0.10573799250000065486" rpy="-2.2332973632374404714e-18 0.27925237217133330736 -0.03490653809662996182" />
+            <origin xyz="0.46313595625000014699 -0.024684938349999997753 -0.10573799250000065486" rpy="-2.2332973632356705417e-18 0.27925237217133325185 -0.034906538096629954882" />
             <geometry>
                 <box size="0.10699999999999999789 0.06500000000000000222 0.076999999999999999001" />
@@ -136,5 +130,5 @@
         </collision>
         <collision>
-            <origin xyz="0.45372929400000000522 -0.034000000000000002442 -0.035885924000000651857" rpy="-3.5918351426043374596e-18 0.26179929927377615373 -3.5038915493521025473e-18" />
+            <origin xyz="0.45372929400000011624 -0.034000000000000002442 -0.035885924000000651857" rpy="-3.5918351426025856337e-18 0.26179929927377609822 -2.8688243315548591629e-18" />
             <geometry>
                 <cylinder length="0.051999999999999997613" radius="0.044999999999999998335" />
@@ -142,12 +136,12 @@
         </collision>
         <inertial>
-            <origin xyz="0.0039718182091793893113 -0.0038738765067834204057 -0.053343546583699136265" rpy="0 0 0"/>
+            <origin xyz="0.0039718182091794838537 -0.0038738765067834169363 -0.053343546583699136265" rpy="0 0 0"/>
             <mass value="3.3445649589086552389" />
-            <inertia ixx="0.0097839331373918841939" ixy="0.013186544376772937198" ixz="0.0014152217803643295062" iyy="0.4954059928866839102" iyz="0.0001950135450045003627" izz="0.49156955837786181496" />
+            <inertia ixx="0.0097839331373918911328" ixy="0.013186544376772938933" ixz="0.0014152217803643357946" iyy="0.49540599288668396571" iyz="0.00019501354500450093191" izz="0.49156955837786192598" />
         </inertial>
     </link>
     <link name="fr_ankle">
         <visual>
-            <origin xyz="-0.12415341931613710358 2.498001805406602216e-16 -0.12500000000000027756" rpy="-1.570796326794896558 -0.13351607992219355348 -7.6813912419263841209e-17" />
+            <origin xyz="0.12415341931613700643 -2.2204460492503130808e-16 -0.1250000000000002498" rpy="-1.57079632679489678 0.13351607992219349796 -1.5575592168678192124e-17" />
             <geometry>
                 <mesh filename="file://$(find new_rover_description)/meshes/fr_ankle.stl"/>
@@ -159,5 +153,5 @@
         <!-- Shapes for fr_ankle -->
         <collision>
-            <origin xyz="-0.11601914642063097804 2.4694101913642000327e-16 -0.1030492935317774833" rpy="-1.570796326794896558 0.0061101698267938863232 -6.1771469324893414164e-17" />
+            <origin xyz="0.1160191464206308809 -2.1951768438536825843e-16 -0.10304929353177745555" rpy="-1.57079632679489678 0.0061101698267938975989 -3.141592653589793116" />
             <geometry>
                 <box size="0.032000000000000000666 0.080000000000000001665 0.05999999999999999778" />
@@ -165,5 +159,5 @@
         </collision>
         <collision>
-            <origin xyz="-0.091894553662955749673 2.5191347026720868665e-16 -0.16352745890207484591" rpy="-1.570796326794896558 -0.79674066942340782127 -1.7200454605793530007e-16" />
+            <origin xyz="0.091894553662955652529 -2.2647424860939617769e-16 -0.16352745890207481816" rpy="-1.57079632679489678 -0.79674066942340771025 3.141592653589793116" />
             <geometry>
                 <box size="0.020000000000000000416 0.080000000000000001665 0.05999999999999999778" />
@@ -171,5 +165,5 @@
         </collision>
         <collision>
-            <origin xyz="-0.063800853957741709976 2.5404739191211583917e-16 -0.19982021317550338613" rpy="-1.570796326794896558 -0.011343354647681722427 -6.3641160347330659717e-17" />
+            <origin xyz="0.063800853957741585076 -2.3064723410920053192e-16 -0.19982021317550335837" rpy="-1.57079632679489678 -0.01134335464768170508 3.141592653589793116" />
             <geometry>
                 <box size="0.025000000000000001388 0.030999999999999999778 0.05999999999999999778" />
@@ -177,5 +171,5 @@
         </collision>
         <collision>
-            <origin xyz="-0.06708178600672955183 2.3759257712076676596e-16 -0.044297919093382362443" rpy="-1.570796326794896558 0.80896192356999563344 4.986565927720294372e-17" />
+            <origin xyz="0.067081786006729454686 -2.1275110104758894607e-16 -0.044297919093382348565" rpy="-1.57079632679489678 0.80896192356999552242 -3.141592653589793116" />
             <geometry>
                 <box size="0.01200000000000000025 0.075999999999999998113 0.05999999999999999778" />
@@ -183,5 +177,5 @@
         </collision>
         <collision>
-            <origin xyz="-0.10777838729007011009 2.4286604753035148434e-16 -0.069810716156365762441" rpy="-1.570796326794886788 1.5594529721472150108 9.3806300299374657517e-15" />
+            <origin xyz="0.10777838729006999907 -2.1569181411638127462e-16 -0.069810716156365748564" rpy="-1.570796326794906328 1.5594529721472150108 -3.1415926535897829019" />
             <geometry>
                 <box size="0.01200000000000000025 0.02999999999999999889 0.05999999999999999778" />
@@ -189,5 +183,5 @@
         </collision>
         <collision>
-            <origin xyz="-0.00045306036165819463246 2.298399379395962547e-16 -0.010753702302991177686" rpy="1.1224846204185424354e-16 0.0061101698267938863232 -6.1771469324893414164e-17" />
+            <origin xyz="0.00045306036165806973237 -2.0888308521874781661e-16 -0.010753702302991163808" rpy="-1.0904930851879991199e-16 0.0061101698267938975989 -3.141592653589793116" />
             <geometry>
                 <cylinder length="0.025999999999999998807" radius="0.037999999999999999056" />
@@ -195,5 +189,5 @@
         </collision>
         <collision>
-            <origin xyz="-0.028495306304552506238 2.3232200630689366419e-16 -0.017582487382379483054" rpy="1.1224846204185424354e-16 0.0061101698267938863232 -6.1771469324893414164e-17" />
+            <origin xyz="0.028495306304552395216 -2.0967224842280919382e-16 -0.017582487382379469176" rpy="-1.0904930851879991199e-16 0.0061101698267938975989 -3.141592653589793116" />
             <geometry>
                 <box size="0.02999999999999999889 0.05999999999999999778 0.01200000000000000025" />
@@ -201,12 +195,12 @@
         </collision>
         <inertial>
-            <origin xyz="-0.067658474648355657055 -0.00014463856991166535219 -0.0716246334329673634" rpy="0 0 0"/>
+            <origin xyz="0.067658474648355559911 0.00014463856991169001778 -0.0716246334329673634" rpy="0 0 0"/>
             <mass value="0.40704474660617540049" />
-            <inertia ixx="0.0016392589144157158811" ixy="-2.8493978195283016631e-06" ixz="-0.00080468641679309058697" iyy="0.0023850903898398135086" iyz="-1.4225306394298707116e-06" izz="0.00116147601485049848" />
+            <inertia ixx="0.001639258914415716098" ixy="-2.8493978195280856697e-06" ixz="0.00080468641679309047855" iyy="0.0023850903898398126413" iyz="1.4225306394299708733e-06" izz="0.0011614760148504976126" />
         </inertial>
     </link>
     <link name="fr_anklemotor">
         <visual>
-            <origin xyz="-0.052882847177904201974 -0.084794424783463051565 -0.024000000000003601786" rpy="4.4687731154414894265e-16 -3.6583860602508457291e-15 2.2874474444740127584e-17" />
+            <origin xyz="0.052882847177904160341 0.084794424783463023809 -0.02400000000000357403" rpy="3.1415926535897926719 3.6092105290609542102e-15 2.6435513327198779569e-17" />
             <geometry>
                 <mesh filename="file://$(find new_rover_description)/meshes/fr_anklemotor.stl"/>
@@ -216,19 +210,13 @@
             </material>
         </visual>
-        <collision>
-            <origin xyz="-0.052882847177904201974 -0.084794424783463051565 -0.024000000000003601786" rpy="4.4687731154414894265e-16 -3.6583860602508457291e-15 2.2874474444740127584e-17" />
-            <geometry>
-                <mesh filename="file://$(find new_rover_description)/meshes/fr_anklemotor.stl"/>
-            </geometry>
-        </collision>
-        <inertial>
-            <origin xyz="-0.021958993625958635187 0.035623040808487965725 -0.023997480138994841531" rpy="0 0 0"/>
-            <mass value="0.67137268218562584643" />
-            <inertia ixx="0.00067219001428469389754" ixy="-3.5905106721073943069e-05" ixz="7.914644953418578865e-09" iyy="0.0010088029360243383828" iyz="6.7337379884156059847e-08" izz="0.001027383624573347887" />
+        <inertial>
+            <origin xyz="0.021958993625958534573 -0.035623040808487965725 -0.023997480138994813775" rpy="0 0 0"/>
+            <mass value="0.67137268218562651256" />
+            <inertia ixx="0.00067219001428469400596" ixy="-3.5905106721074180238e-05" ixz="-7.9146449530728703085e-09" iyy="0.0010088029360243412017" iyz="-6.7337379884094067624e-08" izz="0.0010273836245733504891" />
         </inertial>
     </link>
     <link name="fr_wheel">
         <visual>
-            <origin xyz="0 1.7347234759768070944e-18 0" rpy="-2.1979634337389811138e-17 5.4832000926005038323e-17 3.4959276618369156618e-17" />
+            <origin xyz="0 -1.3877787807814456755e-17 1.2143064331837649661e-17" rpy="-1.2522724101700229322e-17 1.2946497167643599861e-16 -6.0959126447348472264e-18" />
             <geometry>
                 <mesh filename="file://$(find new_rover_description)/meshes/fr_wheel.stl"/>
@@ -240,5 +228,5 @@
         <!-- Shapes for fr_wheel -->
         <collision>
-            <origin xyz="0 1.7347234759768070944e-18 0" rpy="-2.1979634337389811138e-17 5.4832000926005038323e-17 3.4959276618369156618e-17" />
+            <origin xyz="0 -1.3877787807814456755e-17 1.2143064331837649661e-17" rpy="-1.2522724101700229322e-17 1.2946497167643599861e-16 -6.0959126447348472264e-18" />
             <geometry>
                 <cylinder length="0.16000000000000000333" radius="0.15700000000000000067" />
@@ -246,11 +234,11 @@
         </collision>
         <inertial>
-            <origin xyz="-1.3294988577306983418e-07 -1.1207731109163011331e-07 1.2648623649714051351e-05" rpy="0 0 0"/>
-            <mass value="1.8501412404055235239" />
-            <inertia ixx="0.020701719473909988012" ixy="2.9104723315619284601e-05" ixz="1.0888320726562165034e-08" iyy="0.020861663662014584553" iyz="1.4322179502165461347e-08" izz="0.032713974764007967833" />
+            <origin xyz="-1.3294988576060987365e-07 -1.1207731108261813274e-07 1.2648623649732672523e-05" rpy="0 0 0"/>
+            <mass value="1.850141240405538845" />
+            <inertia ixx="0.020701719473909967195" ixy="2.9104723315617021329e-05" ixz="1.0888320727146682287e-08" iyy="0.020861663662014605369" iyz="1.4322179502038958962e-08" izz="0.032713974764007974771" />
         </inertial>
     </link>
     <joint name="frw" type="continuous">
-        <origin xyz="0.053292508052297571375 0.046508209944849832063 -0.024000000000004462208" rpy="1.5707963267948921171 0.28883585951287249483 -1.4372802468727092773" />
+        <origin xyz="-0.053292508052299646104 -0.04650820994485016513 -0.024000000000004573231" rpy="-1.5707963267948781283 -1.3226789075248936989 -1.4372802468725507374" />
         <parent link="fr_anklemotor" />
         <child link="fr_wheel" />
@@ -259,14 +247,14 @@
         <joint_properties friction="0.0"/>
     </joint>
-    <joint name="fr_ankle_motor_join" type="fixed">
-        <origin xyz="-0.060453419316137124717 0.023999999999999993561 -0.20200000000000020717" rpy="-1.570796326794896558 -0.13351607992219358123 -3.5655310271105493798e-14" />
+    <joint name="fl_ankle_motor_join" type="fixed">
+        <origin xyz="0.060453419316137110839 -0.023999999999999799272 -0.20200000000000017941" rpy="1.570796326794896558 0.13351607992219349796 4.5491461274967382195e-14" />
         <parent link="fr_ankle" />
         <child link="fr_anklemotor" />
         <axis xyz="0 0 1"/>
-        <limit effort="1" velocity="20" />
+        <limit effort="20" velocity="20" />
         <joint_properties friction="0.0"/>
     </joint>
     <joint name="frp" type="revolute">
-        <origin xyz="-0.47013767878255985355 -0.026528595964174034316 -0.1056181429369579261" rpy="1.5707963267949009989 0.86524872200545932532 3.11484211882162354" />
+        <origin xyz="-0.470137678782559576 -0.026528595964174079419 -0.10561814293695809264" rpy="1.5707963267949007768 -0.86524793679314937478 3.1148421188216208755" />
         <parent link="rightleg" />
         <child link="fr_ankle" />
@@ -277,5 +265,5 @@
     <link name="br_ankle">
         <visual>
-            <origin xyz="-0.12415341931613704807 2.6367796834847467835e-16 -0.12500000000000027756" rpy="-1.570796326794896558 -0.13351607992219355348 2.8933441911753607959e-17" />
+            <origin xyz="0.12415341931613711746 -1.1102230246251565404e-16 -0.1250000000000002498" rpy="-1.57079632679489678 0.13351607992219349796 -7.1937670166723611946e-17" />
             <geometry>
                 <mesh filename="file://$(find new_rover_description)/meshes/br_ankle.stl"/>
@@ -287,5 +275,5 @@
         <!-- Shapes for br_ankle -->
         <collision>
-            <origin xyz="-0.11601914642063092253 2.6183924338317619713e-16 -0.1030492935317774833" rpy="-1.570796326794896558 0.0061101698267938854559 4.289696008220557727e-17" />
+            <origin xyz="0.11601914642063099192 -1.080805915287935907e-16 -0.10304929353177745555" rpy="-1.57079632679489678 0.0061101698267938975989 3.141592653589793116" />
             <geometry>
                 <box size="0.032000000000000000666 0.080000000000000001665 0.05999999999999999778" />
@@ -293,5 +281,5 @@
         </collision>
         <collision>
-            <origin xyz="-0.091894553662955694162 2.6887324082196188064e-16 -0.16352745890207484591" rpy="-1.570796326794896558 -0.79674066942340771025 -5.9429607503262674962e-17" />
+            <origin xyz="0.091894553662955763551 -1.1354402577905127896e-16 -0.16352745890207481816" rpy="-1.57079632679489678 -0.79674066942340759923 3.141592653589793116" />
             <geometry>
                 <box size="0.020000000000000000416 0.080000000000000001665 0.05999999999999999778" />
@@ -299,5 +287,5 @@
         </collision>
         <collision>
-            <origin xyz="-0.063800853957741640587 2.7367015811300166119e-16 -0.19982021317550338613" rpy="-1.570796326794896558 -0.011343354647681720693 4.1161373355957363927e-17" />
+            <origin xyz="0.063800853957741709976 -1.1604969888808644052e-16 -0.19982021317550335837" rpy="-1.57079632679489678 -0.01134335464768170508 3.141592653589793116" />
             <geometry>
                 <box size="0.025000000000000001388 0.030999999999999999778 0.05999999999999999778" />
@@ -305,5 +293,5 @@
         </collision>
         <collision>
-            <origin xyz="-0.067081786006729482441 2.5806669757403521094e-16 -0.044297919093382362443" rpy="-1.570796326794896558 0.80896192356999552242 1.4652687338504176792e-16" />
+            <origin xyz="0.06708178600672955183 -9.8665051223184460813e-17 -0.044297919093382348565" rpy="-1.57079632679489678 0.80896192356999552242 -3.141592653589793116" />
             <geometry>
                 <box size="0.01200000000000000025 0.075999999999999998113 0.05999999999999999778" />
@@ -311,5 +299,5 @@
         </collision>
         <collision>
-            <origin xyz="-0.1077783872900700407 2.5888258661389069449e-16 -0.069810716156365762441" rpy="-1.5707963267948874542 1.5594529721472150108 8.808038638231368023e-15" />
+            <origin xyz="0.10777838729007011009 -1.0385753439843163474e-16 -0.069810716156365748564" rpy="-1.570796326794906328 1.5594529721472150108 -3.141592653589783346" />
             <geometry>
                 <box size="0.01200000000000000025 0.02999999999999999889 0.05999999999999999778" />
@@ -317,5 +305,5 @@
         </collision>
         <collision>
-            <origin xyz="-0.00045306036165812524352 2.5754883940531762658e-16 -0.010753702302991177686" rpy="1.0517633863451059952e-16 0.0061101698267938854559 4.289696008220557727e-17" />
+            <origin xyz="0.00045306036165818075467 -9.1093200482247960024e-17 -0.010753702302991163808" rpy="-1.1004571489386627502e-16 0.0061101698267938975989 3.141592653589793116" />
             <geometry>
                 <cylinder length="0.025999999999999998807" radius="0.037999999999999999056" />
@@ -323,5 +311,5 @@
         </collision>
         <collision>
-            <origin xyz="-0.028495306304552450727 2.5704198611026095152e-16 -0.017582487382379483054" rpy="1.0517633863451059952e-16 0.0061101698267938854559 4.289696008220557727e-17" />
+            <origin xyz="0.028495306304552506238 -9.3456470928104384066e-17 -0.017582487382379469176" rpy="-1.1004571489386627502e-16 0.0061101698267938975989 3.141592653589793116" />
             <geometry>
                 <box size="0.02999999999999999889 0.05999999999999999778 0.01200000000000000025" />
@@ -329,12 +317,12 @@
         </collision>
         <inertial>
-            <origin xyz="-0.067658474648355559911 -0.00014463856991164654128 -0.0716246334329673634" rpy="0 0 0"/>
-            <mass value="0.40704474660617528947" />
-            <inertia ixx="0.0016392589144157156643" ixy="-2.8493978195285714431e-06" ixz="-0.00080468641679309015329" iyy="0.0023850903898398135086" iyz="-1.4225306394299465211e-06" izz="0.0011614760148504982631" />
+            <origin xyz="0.067658474648355643177 0.00014463856991180293744 -0.071624633432967349522" rpy="0 0 0"/>
+            <mass value="0.40704474660617551152" />
+            <inertia ixx="0.0016392589144157163148" ixy="-2.8493978195282402532e-06" ixz="0.00080468641679309047855" iyy="0.002385090389839814376" iyz="1.4225306394298810878e-06" izz="0.00116147601485049848" />
         </inertial>
     </link>
     <link name="br_anklemotor">
         <visual>
-            <origin xyz="-0.052882847177904201974 -0.084794424783463023809 -0.02400000000000357403" rpy="4.515177172886114136e-16 -3.5943511837517746456e-15 2.1213417495586426316e-17" />
+            <origin xyz="0.052882847177904201974 0.084794424783463023809 -0.02400000000000357403" rpy="3.1415926535897926719 3.7053285121669173598e-15 1.3904604908716712116e-17" />
             <geometry>
                 <mesh filename="file://$(find new_rover_description)/meshes/br_anklemotor.stl"/>
@@ -344,19 +332,13 @@
             </material>
         </visual>
-        <collision>
-            <origin xyz="-0.052882847177904201974 -0.084794424783463023809 -0.02400000000000357403" rpy="4.515177172886114136e-16 -3.5943511837517746456e-15 2.1213417495586426316e-17" />
-            <geometry>
-                <mesh filename="file://$(find new_rover_description)/meshes/br_anklemotor.stl"/>
-            </geometry>
-        </collision>
-        <inertial>
-            <origin xyz="-0.021958993625958652535 0.03562304080848799348 -0.023997480138994817245" rpy="0 0 0"/>
-            <mass value="0.67137268218562540234" />
-            <inertia ixx="0.00067219001428469411438" ixy="-3.5905106721073970174e-05" ixz="7.9146449531624854017e-09" iyy="0.0010088029360243388165" iyz="6.7337379884114131717e-08" izz="0.0010273836245733470197" />
+        <inertial>
+            <origin xyz="0.021958993625958565798 -0.03562304080848799348 -0.023997480138994806836" rpy="0 0 0"/>
+            <mass value="0.67137268218562695665" />
+            <inertia ixx="0.00067219001428469400596" ixy="-3.5905106721074254777e-05" ixz="-7.9146449529637320985e-09" iyy="0.0010088029360243416354" iyz="-6.7337379884056983462e-08" izz="0.0010273836245733500554" />
         </inertial>
     </link>
     <link name="br_wheel">
         <visual>
-            <origin xyz="-2.7755575615628913511e-17 2.7755575615628913511e-17 0" rpy="-2.4576217954427888305e-17 1.4101281192975104818e-16 4.8942876908257451025e-18" />
+            <origin xyz="-5.5511151231257827021e-17 0 1.7916440900322960772e-17" rpy="-2.6934967810890594315e-17 1.2251598845994900865e-16 -2.9380925782674715695e-17" />
             <geometry>
                 <mesh filename="file://$(find new_rover_description)/meshes/br_wheel.stl"/>
@@ -368,5 +350,5 @@
         <!-- Shapes for br_wheel -->
         <collision>
-            <origin xyz="-2.7755575615628913511e-17 2.7755575615628913511e-17 0" rpy="-2.4576217954427888305e-17 1.4101281192975104818e-16 4.8942876908257451025e-18" />
+            <origin xyz="-5.5511151231257827021e-17 0 1.7916440900322960772e-17" rpy="-2.6934967810890594315e-17 1.2251598845994900865e-16 -2.9380925782674715695e-17" />
             <geometry>
                 <cylinder length="0.16000000000000000333" radius="0.15700000000000000067" />
@@ -374,11 +356,11 @@
         </collision>
         <inertial>
-            <origin xyz="-1.3294988579468931784e-07 -1.1207731105968185696e-07 1.2648623649719740024e-05" rpy="0 0 0"/>
-            <mass value="1.8501412404055208594" />
-            <inertia ixx="0.020701719473909988012" ixy="2.9104723315617475339e-05" ixz="1.088832072359006208e-08" iyy="0.020861663662014577614" iyz="1.4322179504244014025e-08" izz="0.032713974764007967833" />
+            <origin xyz="-1.3294988581389118417e-07 -1.1207731107610705665e-07 1.2648623649735715065e-05" rpy="0 0 0"/>
+            <mass value="1.8501412404055219696" />
+            <inertia ixx="0.02070171947390999842" ixy="2.910472331561540519e-05" ixz="1.0888320726009092224e-08" iyy="0.020861663662014581083" iyz="1.4322179499440228792e-08" izz="0.032713974764007995588" />
         </inertial>
     </link>
     <joint name="brw" type="continuous">
-        <origin xyz="0.053292508052299569776 0.046508209944850276152 -0.024000000000004600986" rpy="1.5707963267948887864 -0.97072198262967801519 -1.4372802468726915137" />
+        <origin xyz="-0.053292508052297592192 -0.046508209944849887574 -0.024000000000004573231" rpy="-1.5707963267948856778 -1.1473962864655451455 -1.4372802468727257086" />
         <parent link="br_anklemotor" />
         <child link="br_wheel" />
@@ -387,14 +369,14 @@
         <joint_properties friction="0.0"/>
     </joint>
-    <joint name="br_ankle_motor_join" type="fixed">
-        <origin xyz="-0.060453419316137235739 0.023999999999999951927 -0.20200000000000017941" rpy="-1.570796326794896558 -0.13351607992219344245 -2.7584080234938445875e-15" />
+    <joint name="bl_ankle_motor_join" type="fixed">
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