Commit message: Fixed anti-parallel wheel issue :happy_cry:

File: src/ros/rover/new_rover_description/urdf/rover.urdf.xacro (robot description, xacro)
@@ -259,5 +259,5 @@
         <parent link="rightleg" />
         <child link="fr_ankle" />
-        <axis xyz="0 0 1"/>
+        <axis xyz="0 0 -1"/>
         <limit lower="-3.141592654" upper="3.141592654" effort="20" velocity="20" />
         <joint_properties friction="0.0"/>
@@ -381,5 +381,5 @@
         <parent link="rightleg" />
         <child link="br_ankle" />
-        <axis xyz="0 0 1"/>
+        <axis xyz="0 0 -1"/>
         <limit lower="-3.141592654" upper="3.141592654" effort="20" velocity="20" />
         <joint_properties friction="0.0"/>
@@ -582,5 +582,5 @@
         <parent link="leftleg" />
         <child link="fl_ankle" />
-        <axis xyz="0 0 1"/>
+        <axis xyz="0 0 -1"/>
         <limit lower="-3.141592654" upper="3.141592654" effort="20" velocity="20" />
         <joint_properties friction="0.0"/>
@@ -704,5 +704,5 @@
         <parent link="leftleg" />
         <child link="bl_ankle" />
-        <axis xyz="0 0 1"/>
+        <axis xyz="0 0 -1"/>
         <limit lower="-3.141592654" upper="3.141592654" effort="20" velocity="20" />
         <joint_properties friction="0.0"/>
