Commit message: added oak camera angle as a launch param to gazebo.launch.py and urdf.launch.py

File: src/ros/rover/rover_description/waratah/urdf/auto_camera.xacro (robot description, xacro)
@@ -3,120 +3,122 @@
 which is how it gets added to the gazebo sim. Author/s: Victor Bartlinski-->
 <robot xmlns:xacro="http://www.ros.org/wiki/xacro" >
-  <link name='camera_link'></link>
-  <joint name="camera_joint" type="fixed">
-    <origin xyz="0.49 0 0.48" rpy="0 0 0" />
-    <parent link="base_link" />
-    <child link="camera_link" />
-  </joint>
-  <xacro:include filename="$(find depthai_descriptions)/urdf/include/depthai_macro.urdf.xacro"/>
-  <xacro:depthai_camera camera_name = "oak" parent = "camera_link" camera_model = "OAK-D-LR"
-   base_frame = "oak-d_frame" cam_pos_x = "0.0" cam_pos_y = "0.0" cam_pos_z = "0.0"
-   cam_roll = "0.0" cam_pitch = "0.0" cam_yaw = "0.0"/>
-  <gazebo reference="oak_rgb_camera_frame">
-    <sensor name="oak/stereo" type="depth_camera">
-      <topic>oak/depth</topic>
-      <gz_frame_id>camera_link</gz_frame_id> <!-- Sets the frame_id so that rviz2 correctly transforms it -->
-      <visualize>true</visualize>
-      <update_rate>30</update_rate>
-      <always_on>1</always_on>
-      <camera>
-        <horizontal_fov>${radians(82)}</horizontal_fov>
-        <image>
-          <width>600</width>
-          <height>400</height>
-        </image>
-        <clip>
-          <near>0.4</near>
-          <far>100.0</far>
-        </clip>
-      </camera>
-      <plugin name="gz::sim::systems::Sensors" filename="gz-sim-sensors-system">
-        <frame_name>oak_rgb_camera_optical_frame</frame_name>
-      </plugin>
-    </sensor>
-    <sensor name="oak/rgb" type="camera">
-      <topic>oak/rgb</topic>
-      <visualize>true</visualize>
-      <update_rate>30</update_rate>
-      <always_on>1</always_on>
-      <camera>
-        <horizontal_fov>${radians(82)}</horizontal_fov>
-        <image>
-          <width>600</width>
-          <height>400</height>
-        </image>
-        <clip>
-          <near>0.4</near>
-          <far>100.0</far>
-        </clip>
-      </camera>
-      <!-- <plugin name="gz::sim::systems::Sensors" filename="gz-sim-sensors-system"></plugin> -->
-    </sensor>
-  </gazebo>
-  <gazebo reference="oak_imu_frame">
-    <sensor name="imu_sensor" type="imu">
-      <topic>oak/imu</topic>
-      <plugin filename="gz-sim-imu-system" name="gz::sim::systems::Imu">
-        <frame_name>oak_imu_frame</frame_name>
-        <initial_orientation_as_reference>false</initial_orientation_as_reference>
-      </plugin>
-      <always_on>true</always_on>
-      <update_rate>200</update_rate>
-      <visualize>true</visualize>
-      <imu>
-        <angular_velocity>
-          <x>
-            <noise type="gaussian">
-              <mean>0.0</mean>
-              <stddev>2e-4</stddev>
-              <bias_mean>0.0000075</bias_mean>
-              <bias_stddev>0.0000008</bias_stddev>
-            </noise>
-          </x>
-          <y>
-            <noise type="gaussian">
-              <mean>0.0</mean>
-              <stddev>2e-4</stddev>
-              <bias_mean>0.0000075</bias_mean>
-              <bias_stddev>0.0000008</bias_stddev>
-            </noise>
-          </y>
-          <z>
-            <noise type="gaussian">
-              <mean>0.0</mean>
-              <stddev>2e-4</stddev>
-              <bias_mean>0.0000075</bias_mean>
-              <bias_stddev>0.0000008</bias_stddev>
-            </noise>
-          </z>
-        </angular_velocity>
-        <linear_acceleration>
-          <x>
-            <noise type="gaussian">
-              <mean>0.0</mean>
-              <stddev>1.7e-2</stddev>
-              <bias_mean>0.1</bias_mean>
-              <bias_stddev>0.001</bias_stddev>
-            </noise>
-          </x>
-          <y>
-            <noise type="gaussian">
-              <mean>0.0</mean>
-              <stddev>1.7e-2</stddev>
-              <bias_mean>0.1</bias_mean>
-              <bias_stddev>0.001</bias_stddev>
-            </noise>
-          </y>
-          <z>
-            <noise type="gaussian">
-              <mean>0.0</mean>
-              <stddev>1.7e-2</stddev>
-              <bias_mean>0.1</bias_mean>
-              <bias_stddev>0.001</bias_stddev>
-            </noise>
-          </z>
-        </linear_acceleration>
-      </imu>
-    </sensor>
-  </gazebo>
+  <xacro:macro name="auto_cam" params="angle">
+    <link name='camera_link'></link>
+    <joint name="camera_joint" type="fixed">
+      <origin xyz="0.49 0 0.48" rpy="0 ${angle} 0" />
+      <parent link="base_link" />
+      <child link="camera_link" />
+    </joint>
+    <xacro:include filename="$(find depthai_descriptions)/urdf/include/depthai_macro.urdf.xacro"/>
+    <xacro:depthai_camera camera_name = "oak" parent = "camera_link" camera_model = "OAK-D-LR"
+    base_frame = "oak-d_frame" cam_pos_x = "0.0" cam_pos_y = "0.0" cam_pos_z = "0.0"
+    cam_roll = "0.0" cam_pitch = "0.0" cam_yaw = "0.0"/>
+    <gazebo reference="oak_rgb_camera_frame">
+      <sensor name="oak/stereo" type="depth_camera">
+        <topic>oak/depth</topic>
+        <gz_frame_id>camera_link</gz_frame_id> <!-- Sets the frame_id so that rviz2 correctly transforms it -->
+        <visualize>true</visualize>
+        <update_rate>30</update_rate>
+        <always_on>1</always_on>
+        <camera>
+          <horizontal_fov>${radians(82)}</horizontal_fov>
+          <image>
+            <width>600</width>
+            <height>400</height>
+          </image>
+          <clip>
+            <near>0.4</near>
+            <far>100.0</far>
+          </clip>
+        </camera>
+        <plugin name="gz::sim::systems::Sensors" filename="gz-sim-sensors-system">
+          <frame_name>oak_rgb_camera_optical_frame</frame_name>
+        </plugin>
+      </sensor>
+      <sensor name="oak/rgb" type="camera">
+        <topic>oak/rgb</topic>
+        <visualize>true</visualize>
+        <update_rate>30</update_rate>
+        <always_on>1</always_on>
+        <camera>
+          <horizontal_fov>${radians(82)}</horizontal_fov>
+          <image>
+            <width>600</width>
+            <height>400</height>
+          </image>
+          <clip>
+            <near>0.4</near>
+            <far>100.0</far>
+          </clip>
+        </camera>
+        <!-- <plugin name="gz::sim::systems::Sensors" filename="gz-sim-sensors-system"></plugin> -->
+      </sensor>
+    </gazebo>
+    <gazebo reference="oak_imu_frame">
+      <sensor name="imu_sensor" type="imu">
+        <topic>oak/imu</topic>
+        <plugin filename="gz-sim-imu-system" name="gz::sim::systems::Imu">
+          <frame_name>oak_imu_frame</frame_name>
+          <initial_orientation_as_reference>false</initial_orientation_as_reference>
+        </plugin>
+        <always_on>true</always_on>
+        <update_rate>200</update_rate>
+        <visualize>true</visualize>
+        <imu>
+          <angular_velocity>
+            <x>
+              <noise type="gaussian">
+                <mean>0.0</mean>
+                <stddev>2e-4</stddev>
+                <bias_mean>0.0000075</bias_mean>
+                <bias_stddev>0.0000008</bias_stddev>
+              </noise>
+            </x>
+            <y>
+              <noise type="gaussian">
+                <mean>0.0</mean>
+                <stddev>2e-4</stddev>
+                <bias_mean>0.0000075</bias_mean>
+                <bias_stddev>0.0000008</bias_stddev>
+              </noise>
+            </y>
+            <z>
+              <noise type="gaussian">
+                <mean>0.0</mean>
+                <stddev>2e-4</stddev>
+                <bias_mean>0.0000075</bias_mean>
+                <bias_stddev>0.0000008</bias_stddev>
+              </noise>
+            </z>
+          </angular_velocity>
+          <linear_acceleration>
+            <x>
+              <noise type="gaussian">
+                <mean>0.0</mean>
+                <stddev>1.7e-2</stddev>
+                <bias_mean>0.1</bias_mean>
+                <bias_stddev>0.001</bias_stddev>
+              </noise>
+            </x>
+            <y>
+              <noise type="gaussian">
+                <mean>0.0</mean>
+                <stddev>1.7e-2</stddev>
+                <bias_mean>0.1</bias_mean>
+                <bias_stddev>0.001</bias_stddev>
+              </noise>
+            </y>
+            <z>
+              <noise type="gaussian">
+                <mean>0.0</mean>
+                <stddev>1.7e-2</stddev>
+                <bias_mean>0.1</bias_mean>
+                <bias_stddev>0.001</bias_stddev>
+              </noise>
+            </z>
+          </linear_acceleration>
+        </imu>
+      </sensor>
+    </gazebo>
+  </xacro:macro>
 </robot>

File: src/ros/rover/rover_description/waratah/urdf/rover.urdf.xacro (robot description, xacro)
@@ -10,4 +10,5 @@
   <xacro:arg name="auto_camera" default="true"/>
   <xacro:arg name="robot_name" default="rover"/>
+  <xacro:arg name="angle" default="0"/>
   <!-- Manually added links-->
   <link name="base_link" />
@@ -526,4 +527,5 @@
   <xacro:if value="$(arg auto_camera)">
     <xacro:include filename="$(find rover_description)/waratah/urdf/auto_camera.xacro"/>
+    <xacro:auto_cam angle="$(arg angle)"></xacro:auto_cam>
   </xacro:if>
   <xacro:include filename="$(find rover_description)/waratah/urdf/p3d.xacro"/>
