Commit message: renamed rightleg/leftleg to right_leg/left_leg

File: src/ros/rover/rover_description/base/urdf/ckc.xacro (robot description, xacro)
@@ -4,5 +4,5 @@
     <gazebo>
         <plugin filename="libgz-sim-detachable-joint-system.so" name="gz::sim::systems::DetachableJoint">
-            <parent_link>leftleg</parent_link>
+            <parent_link>left_leg</parent_link>
             <child_model>$(arg robot_name)</child_model>
             <child_link>diffend</child_link>
@@ -10,5 +10,5 @@
         </plugin>
         <plugin filename="libgz-sim-detachable-joint-system.so" name="gz::sim::systems::DetachableJoint">
-            <parent_link>rightleg</parent_link>
+            <parent_link>right_leg</parent_link>
             <child_model>$(arg robot_name)</child_model>
             <child_link>diffend_2</child_link>

File: src/ros/rover/rover_description/base/urdf/rover.urdf.xacro (robot description, xacro)
@@ -48,15 +48,15 @@
         </inertial>
     </link>
-    <link name="rightleg">
+    <link name="right_leg">
         <visual>
             <origin xyz="-7.9461177221464552678e-19 -7.285838599104098493e-20 -0.02099999999999946354" rpy="3.141592653589793116 3.7838655819744073932e-17 2.5353252380137503331e-18" />
             <geometry>
-                <mesh filename="file://$(find rover_description)/base/meshes/rightleg.stl"/>
-            </geometry>
-            <material name="rightleg_material">
-                <color rgba="0.86666666666666669627 0.074509803921568626417 0.32549019607843138191 1.0"/>
-            </material>
-        </visual>
-        <!-- Shapes for rightleg -->
+                <mesh filename="file://$(find rover_description)/base/meshes/right_leg.stl"/>
+            </geometry>
+            <material name="right_leg_material">
+                <color rgba="0.86666666666666669627 0.074509803921568626417 0.32549019607843138191 1.0"/>
+            </material>
+        </visual>
+        <!-- Shapes for right_leg -->
         <collision>
             <origin xyz="-7.9461177221464552678e-19 -7.285838599104098493e-20 -0.02099999999999946354" rpy="3.141592653589793116 3.7838655819744073932e-17 2.5353252380137503331e-18" />
@@ -211,5 +211,5 @@
     <joint name="frp" type="revolute">
         <origin xyz="-0.47013767878255968702 0.026528595964174069011 0.083618142936957629008" rpy="-1.5707963267948923392 0.8652479366072932665 -3.11484211882162354" />
-        <parent link="rightleg" />
+        <parent link="right_leg" />
         <child link="fr_ankle" />
         <axis xyz="0 0 -1"/>
@@ -309,5 +309,5 @@
     <joint name="brp" type="revolute">
         <origin xyz="0.47757721986905643519 0.051886525235696055736 0.086037700396842498041" rpy="1.5707963267948947816 0.86524793660728771538 0.02675053476816627307" />
-        <parent link="rightleg" />
+        <parent link="right_leg" />
         <child link="br_ankle" />
         <axis xyz="0 0 -1"/>
@@ -318,20 +318,20 @@
         <origin xyz="-4.511276110173610435e-17 -0.32285000000001146114 -2.4144264060824868906e-16" rpy="-1.5707963267948972241 -0.04120766744252004482 -3.141592653589793116" />
         <parent link="chassis" />
-        <child link="rightleg" />
+        <child link="right_leg" />
         <axis xyz="0 0 1"/>
         <limit effort="20" velocity="20" />
         <joint_properties friction="0.0"/>
     </joint>
-    <link name="leftleg">
+    <link name="left_leg">
         <visual>
             <origin xyz="-1.307880673257705575e-20 8.6736173798839122125e-19 -0.021000000000000518252" rpy="3.141592653589793116 6.2280032059899110289e-19 6.6901195618365661673e-19" />
             <geometry>
-                <mesh filename="file://$(find rover_description)/base/meshes/leftleg.stl"/>
-            </geometry>
-            <material name="leftleg_material">
-                <color rgba="0.86666666666666669627 0.074509803921568626417 0.32549019607843138191 1.0"/>
-            </material>
-        </visual>
-        <!-- Shapes for leftleg -->
+                <mesh filename="file://$(find rover_description)/base/meshes/left_leg.stl"/>
+            </geometry>
+            <material name="left_leg_material">
+                <color rgba="0.86666666666666669627 0.074509803921568626417 0.32549019607843138191 1.0"/>
+            </material>
+        </visual>
+        <!-- Shapes for left_leg -->
         <collision>
             <origin xyz="-1.307880673257705575e-20 8.6736173798839122125e-19 -0.021000000000000518252" rpy="3.141592653589793116 6.2280032059899110289e-19 6.6901195618365661673e-19" />
@@ -486,5 +486,5 @@
     <joint name="flp" type="revolute">
         <origin xyz="-0.47964586704902811842 -0.025616433642942935955 0.086267061908379294444" rpy="-1.570796326794896558 -0.865247936793150485 -0.028123902821395457829" />
-        <parent link="leftleg" />
+        <parent link="left_leg" />
         <child link="fl_ankle" />
         <axis xyz="0 0 -1"/>
@@ -584,5 +584,5 @@
     <joint name="blp" type="revolute">
         <origin xyz="0.47750427808995571377 -0.052542330732558047146 0.086042547141643943576" rpy="1.5707963267948954478 -0.86524793660727672417 3.1134687507683778129" />
-        <parent link="leftleg" />
+        <parent link="left_leg" />
         <child link="bl_ankle" />
         <axis xyz="0 0 -1"/>
@@ -593,5 +593,5 @@
         <origin xyz="-3.4940027607927698323e-17 0.32284999999999253184 1.4340253524620971087e-16" rpy="1.5707963267948961139 -0.042581035495765612309 -3.141592653589793116" />
         <parent link="chassis" />
-        <child link="leftleg" />
+        <child link="left_leg" />
         <axis xyz="0 0 1"/>
         <limit effort="20" velocity="20" />

Commit message: PR cleanups

File: src/ros/rover/rover_description/base/urdf/ckc.xacro (robot description, xacro)
@@ -1,10 +1,12 @@
 <?xml version="1.0" encoding="utf-8"?>
-<!-- Configure Closed Kinetic Chains for Rover -->
-<robot xmlns:xacro="http://www.ros.org/wiki/xacro">
+<!-- Handle custom joints that are not supported by gazebo -->
+<!-- Works except it breaks detachable joint for closing ckc -->
+<robot xmlns:xacro="http://www.ros.org/wiki/xacro" >
+    <!-- Plugin to allow Closed Kinetic Chains for Rover -->
     <gazebo>
         <plugin filename="libgz-sim-detachable-joint-system.so" name="gz::sim::systems::DetachableJoint">
             <parent_link>left_leg</parent_link>
             <child_model>$(arg robot_name)</child_model>
-            <child_link>diffend</child_link>
+            <child_link>left_diffend_dummy</child_link>
             <output_topic>close_loop_left</output_topic>
         </plugin>
@@ -12,8 +14,135 @@
             <parent_link>right_leg</parent_link>
             <child_model>$(arg robot_name)</child_model>
-            <child_link>diffend_2</child_link>
+            <child_link>right_diffend_dummy</child_link>
             <output_topic>close_loop_right</output_topic>
         </plugin>
     </gazebo>
+    <!-- Ball joint for top left on diff bar-->
+    <link name="tl_ball">
+        <inertial>
+        <mass value="0.00001"/>
+        <inertia ixx="0.01" iyy="0.01" izz="0.01" ixy="0.0" ixz="0.0" iyz="0.0"/>
+        </inertial>
+    </link>
+    <link name="tl_ball_dummy">
+        <inertial>
+        <mass value="0.00001"/>
+        <inertia ixx="0.01" iyy="0.01" izz="0.01" ixy="0.0" ixz="0.0" iyz="0.0"/>
+        </inertial>
+    </link>
+    <joint name="tl_ball_roll" type="revolute">
+        <parent link="diffbar"/>
+        <child link="tl_ball"/>
+        <origin xyz="0.38332334967290787597 -0.067590248755372686618 -0.010000000000001729727" rpy="-1.1995263624187955109 -0.95290201305807298304 -1.8975045742137988114" />
+        <axis xyz="1 0 0"/>
+        <limit effort="20" velocity="20" lower="-0.26179938779914940783" upper="0.26179938779914940783"/>
+    </joint>
+    <joint name="tl_ball_pitch" type="revolute">
+        <parent link="tl_ball"/>
+        <child link="tl_ball_dummy"/>
+        <axis xyz="0 1 0"/>
+        <limit effort="20" velocity="20" lower="-0.26179938779914940783" upper="0.26179938779914940783"/>
+    </joint>
+    <joint name="tl_ball_yaw" type="continuous">
+        <parent link="tl_ball_dummy"/>
+        <child link="left_difflink"/>
+        <axis xyz="0 0 1"/>
+        <limit effort="20" velocity="20" />
+    </joint>
+    <!-- Ball joint for bottom left on diff bar-->
+    <link name="bl_ball">
+        <inertial>
+        <mass value="0.00001"/>
+        <inertia ixx="0.01" iyy="0.01" izz="0.01" ixy="0.0" ixz="0.0" iyz="0.0"/>
+        </inertial>
+    </link>
+    <link name="bl_ball_dummy">
+        <inertial>
+        <mass value="0.00001"/>
+        <inertia ixx="0.01" iyy="0.01" izz="0.01" ixy="0.0" ixz="0.0" iyz="0.0"/>
+        </inertial>
+    </link>
+    <joint name="bl_ball_roll" type="revolute">
+        <parent link="left_difflink"/>
+        <child link="bl_ball"/>
+        <origin xyz="-2.8310687127941491781e-15 -0.11550000000000194833 3.5527136788005009294e-15" rpy="3.1415926535897913396 0.20093653079504641967 3.1415926535897602534" />
+        <axis xyz="1 0 0"/>
+        <limit effort="20" velocity="20" lower="-0.26179938779914940783" upper="0.26179938779914940783"/>
+    </joint>
+    <joint name="bl_ball_pitch" type="revolute">
+        <parent link="bl_ball"/>
+        <child link="bl_ball_dummy"/>
+        <axis xyz="0 1 0"/>
+        <limit effort="20" velocity="20" lower="-0.26179938779914940783" upper="0.26179938779914940783"/>
+    </joint>
+    <joint name="bl_ball_yaw" type="continuous">
+        <parent link="bl_ball_dummy"/>
+        <child link="left_diffend_dummy"/>
+        <axis xyz="0 0 1"/>
+        <limit effort="20" velocity="20" />
+    </joint>
+        <!-- Ball joint for top right on diff bar-->
+    <link name="tr_ball">
+        <inertial>
+        <mass value="0.00001"/>
+        <inertia ixx="0.01" iyy="0.01" izz="0.01" ixy="0.0" ixz="0.0" iyz="0.0"/>
+        </inertial>
+    </link>
+    <link name="tr_ball_dummy">
+        <inertial>
+        <mass value="0.00001"/>
+        <inertia ixx="0.01" iyy="0.01" izz="0.01" ixy="0.0" ixz="0.0" iyz="0.0"/>
+        </inertial>
+    </link>
+    <joint name="tr_ball_roll" type="revolute">
+        <parent link="diffbar"/>
+        <child link="tr_ball"/>
+        <origin xyz="-0.38332334962930325606 -0.067590249002697472269 -0.010000000000000064393" rpy="-1.940682273124183288 -0.95328403917359394448 -1.2457859294461617328" />
+        <axis xyz="1 0 0"/>
+        <limit effort="20" velocity="20" lower="-0.26179938779914940783" upper="0.26179938779914940783"/>
+    </joint>
+    <joint name="tr_ball_pitch" type="revolute">
+        <parent link="tr_ball"/>
+        <child link="tr_ball_dummy"/>
+        <axis xyz="0 1 0"/>
+        <limit effort="20" velocity="20" lower="-0.26179938779914940783" upper="0.26179938779914940783"/>
+    </joint>
+    <joint name="tr_ball_yaw" type="continuous">
+        <parent link="tr_ball_dummy"/>
+        <child link="right_difflink"/>
+        <axis xyz="0 0 1"/>
+        <limit effort="20" velocity="20" />
+    </joint>
+    <!-- Ball joint for bottom right on diff bar-->
+    <link name="br_ball">
+        <inertial>
+        <mass value="0.00001"/>
+        <inertia ixx="0.01" iyy="0.01" izz="0.01" ixy="0.0" ixz="0.0" iyz="0.0"/>
+        </inertial>
+    </link>
+    <link name="br_ball_dummy">
+        <inertial>
+        <mass value="0.00001"/>
+        <inertia ixx="0.01" iyy="0.01" izz="0.01" ixy="0.0" ixz="0.0" iyz="0.0"/>
+        </inertial>
+    </link>
+    <joint name="br_ball_roll" type="revolute">
+        <parent link="right_difflink"/>
+        <child link="br_ball"/>
+        <origin xyz="1.3711254354120683274e-14 -0.11549999999999875644 -6.0507154842071031453e-15" rpy="-4.0861161763381464503e-15 -0.42892757732778930002 -3.1415926535897278349" />
+        <axis xyz="1 0 0"/>
+        <limit effort="20" velocity="20" lower="-0.26179938779914940783" upper="0.26179938779914940783"/>
+    </joint>
+    <joint name="br_ball_pitch" type="revolute">
+        <parent link="br_ball"/>
+        <child link="br_ball_dummy"/>
+        <axis xyz="0 1 0"/>
+        <limit effort="20" velocity="20" lower="-0.26179938779914940783" upper="0.26179938779914940783"/>
+    </joint>
+    <joint name="br_ball_yaw" type="continuous">
+        <parent link="br_ball_dummy"/>
+        <child link="right_diffend_dummy"/>
+        <axis xyz="0 0 1"/>
+        <limit effort="20" velocity="20" />
+    </joint>
 </robot>
-<!-- diffend is on the left leg, diffend_2 is on the right leg, this is temp. -->
