Commit message: fix: diffbar position for real this time. Also added some comments

File: src/ros/rover/rover_description/base/urdf/ckc.xacro (robot description, xacro)
@@ -1,7 +1,11 @@
 <?xml version="1.0" encoding="utf-8"?>
 <!-- Handle custom joints that are not supported by gazebo -->
-<!-- Works except it breaks detachable joint for closing ckc -->
+<!-- To create ball joints, the origin from the generated revolute joints have been copied to the first axis of the ball joint (roll)
+     The generated revolute joints were then deleted. -->
 <robot xmlns:xacro="http://www.ros.org/wiki/xacro" >
-    <!-- Plugin to allow Closed Kinetic Chains for Rover -->
+    <!-- Plugin to allow Closed Kinetic Chains for Rover
+         Defines a fixed joint between a dummy link with the inertia of the "diffend" (part of leg attached to the difflink) and the leg on each side
+         See Onshape for more details.
+    -->
     <gazebo>
         <plugin filename="libgz-sim-detachable-joint-system.so" name="gz::sim::systems::DetachableJoint">
@@ -34,5 +38,5 @@
         <parent link="diffbar"/>
         <child link="tl_ball"/>
-        <origin xyz="0.38332334967290787597 -0.067590248755372686618 -0.010000000000001729727" rpy="-1.1995263624187955109 -0.95290201305807298304 -1.8975045742137988114" />
+        <origin xyz="0.38332334967291109562 -0.067590248755372728251 -0.010000000000001008083" rpy="-1.2881840847457926014 -1.0674573312881561193 -1.7779955883383502524" />
         <axis xyz="1 0 0"/>
         <limit effort="20" velocity="20" lower="-0.26179938779914940783" upper="0.26179938779914940783"/>
@@ -66,5 +70,5 @@
         <parent link="left_difflink"/>
         <child link="bl_ball"/>
-        <origin xyz="-2.8310687127941491781e-15 -0.11550000000000194833 3.5527136788005009294e-15" rpy="3.1415926535897913396 0.20093653079504641967 3.1415926535897602534" />
+        <origin xyz="-2.720046410331633524e-15 -0.11550000000000196221 3.6082248300317587564e-15" rpy="-3.1415926535897891192 0.2009365307950475299 3.1415926535897802374" />
         <axis xyz="1 0 0"/>
         <limit effort="20" velocity="20" lower="-0.26179938779914940783" upper="0.26179938779914940783"/>
@@ -98,5 +102,5 @@
         <parent link="diffbar"/>
         <child link="tr_ball"/>
-        <origin xyz="-0.38332334962930325606 -0.067590249002697472269 -0.010000000000000064393" rpy="-1.940682273124183288 -0.95328403917359394448 -1.2457859294461617328" />
+        <origin xyz="-0.3833233496293029785 -0.067590249002697777581 -0.0099999999999998423483" rpy="-1.9920835247378900768 -1.038397915447168085 -1.2040941380156902074" />
         <axis xyz="1 0 0"/>
         <limit effort="20" velocity="20" lower="-0.26179938779914940783" upper="0.26179938779914940783"/>
@@ -130,5 +134,5 @@
         <parent link="right_difflink"/>
         <child link="br_ball"/>
-        <origin xyz="1.3711254354120683274e-14 -0.11549999999999875644 -6.0507154842071031453e-15" rpy="-4.0861161763381464503e-15 -0.42892757732778930002 -3.1415926535897278349" />
+        <origin xyz="1.3655743202889425447e-14 -0.11549999999999870093 -5.9952043329758453183e-15" rpy="-3.6772342970642588874e-15 -0.42892757732776881641 -3.141592653589728279" />
         <axis xyz="1 0 0"/>
         <limit effort="20" velocity="20" lower="-0.26179938779914940783" upper="0.26179938779914940783"/>

File: src/ros/rover/rover_description/base/urdf/joint_states.xacro (robot description, xacro)
@@ -15,6 +15,5 @@
             <joint_name>chassis_to_right_leg</joint_name>
             <joint_name>chassis_to_left_leg</joint_name>
-            <joint_name>chassis_to_diffbar_axle_dummy</joint_name>
-            <joint_name>diffbar_axle_dummy_to_diffbar</joint_name>
+            <joint_name>chassis_to_diffbar</joint_name>
             <joint_name>tl_ball_roll</joint_name>
             <joint_name>tl_ball_pitch</joint_name>
