Commit message: fix: diffbar position for real this time. Also added some comments

File: src/ros/rover/rover_description/base/urdf/rover.urdf.xacro (robot description, xacro)
@@ -1,4 +1,8 @@
 <?xml version="1.0" encoding="utf-8"?>
 <!-- Generated using onshape-to-robot and modified to include CKCs and ball joints by Anthony Lew -->
+<!-- Collisions added using openscad (see .scad files)-->
+<!-- Note: Rover pivots' z axis has been inverted to correct for pivot_drive_controller's zero angle.
+           Therefore if exported from onshape, don't forget to add a negative sign to the z of the axis tag on each pivot
+     Note 2: Exporting from onshape has _continuous at the end of continuous joint names these have been removed post-export -->
 <robot name="rover"  xmlns:xacro="http://www.ros.org/wiki/xacro" >
     <!-- Loading args -->
@@ -14,584 +18,4 @@
     <!-- Generated URDF -->
     <link name="base_link"></link>
-    <link name="chassis">
-        <visual>
-            <origin xyz="1.2353683969592321892e-17 1.3877787807815553765e-17 -1.2992673251725723918e-16" rpy="-4.03091968774772598e-16 -5.9777162559529608526e-16 1.57079632679489678" />
-            <geometry>
-                <mesh filename="file://$(find rover_description)/base/meshes/chassis.stl"/>
-            </geometry>
-            <material name="chassis_material">
-                <color rgba="0.86666666666666669627 0.074509803921568626417 0.32549019607843138191 1.0"/>
-            </material>
-        </visual>
-        <!-- Shapes for chassis -->
-        <collision>
-            <origin xyz="-0.17250000000000031974 9.3018238151966802719e-18 0.023499999999999854339" rpy="-4.03091968774772598e-16 -5.9777162559529608526e-16 1.57079632679489678" />
-            <geometry>
-                <box size="0.47999999999999998224 0.54500000000000003997 0.1749999999999999889" />
-            </geometry>
-        </collision>
-        <collision>
-            <origin xyz="0.22700000000000039591 2.8459855857991392753e-18 0.033500000000000043632" rpy="-4.03091968774772598e-16 -5.9777162559529608526e-16 1.57079632679489678" />
-            <geometry>
-                <box size="0.34000000000000002442 0.26000000000000000888 0.19500000000000000666" />
-            </geometry>
-        </collision>
-        <inertial>
-            <origin xyz="-0.022980723180786914728 -0.00012909338240177744466 0.024515364506931040106" rpy="0 0 0"/>
-            <mass value="8.3419541100883467521" />
-            <inertia ixx="0.2173768709359497342" ixy="0.00013546851964914256188" ixz="-0.0088627259627339118053" iyy="0.45541406320296684562" iyz="-0.00021657327861197947678" izz="0.59726536058024304321" />
-        </inertial>
-    </link>
-    <link name="left_leg">
-        <visual>
-            <origin xyz="-1.307880673257705575e-20 8.6736173798839122125e-19 -0.021000000000000518252" rpy="3.141592653589793116 6.2280032059899110289e-19 6.6901195618365661673e-19" />
-            <geometry>
-                <mesh filename="file://$(find rover_description)/base/meshes/left_leg.stl"/>
-            </geometry>
-            <material name="left_leg_material">
-                <color rgba="0.86666666666666669627 0.074509803921568626417 0.32549019607843138191 1.0"/>
-            </material>
-        </visual>
-        <!-- Shapes for left_leg -->
-        <collision>
-            <origin xyz="-1.307880673257705575e-20 8.6736173798839122125e-19 -0.021000000000000518252" rpy="3.141592653589793116 6.2280032059899110289e-19 6.6901195618365661673e-19" />
-            <geometry>
-                <cylinder length="0.058000000000000002942" radius="0.042999999999999996558" />
-            </geometry>
-        </collision>
-        <collision>
-            <origin xyz="-0.085373995000000008071 0.010358865000000001821 -0.013653240000000515728" rpy="3.0194197050837283669 -1.3089970275211204598 6.6901195618327056408e-19" />
-            <geometry>
-                <cylinder length="0.089999999999999996669" radius="0.02999999999999999889" />
-            </geometry>
-        </collision>
-        <collision>
-            <origin xyz="-0.31456908199999999987 0.036386049000000003639 0.044033037699999472148" rpy="3.0194196304823472943 -1.3264501964363342168 6.6901195618324186772e-19" />
-            <geometry>
-                <cylinder length="0.39000000000000001332" radius="0.025000000000000001388" />
-            </geometry>
-        </collision>
-        <collision>
-            <origin xyz="-0.46338715075000003196 0.0056285796000000000786 0.083600173999999485841" rpy="-3.141592653589793116 -0.27925237217133336287 3.1066861154931633138" />
-            <geometry>
-                <box size="0.105999999999999997 0.06500000000000000222 0.076999999999999999001" />
-            </geometry>
-        </collision>
-        <collision>
-            <origin xyz="-0.45372929400000000522 -0.0080000000000000001665 0.01388592399999948046" rpy="-3.141592653589793116 -0.26179929927377620924 -3.141592653589793116" />
-            <geometry>
-                <cylinder length="0.051999999999999997613" radius="0.044999999999999998335" />
-            </geometry>
-        </collision>
-        <collision>
-            <origin xyz="0.085785990000000020284 0.0059293025000000014815 -0.013542825000000516603" rpy="-3.071779613202412218 -1.3089970275211204598 -3.141592653589793116" />
-            <geometry>
-                <cylinder length="0.089999999999999996669" radius="0.02999999999999999889" />
-            </geometry>
-        </collision>
-        <collision>
-            <origin xyz="0.31599007519999999793 0.019538657500000000677 0.044387337799999482257" rpy="-3.0717796785789528435 -1.3264501964363342168 -3.141592653589793116" />
-            <geometry>
-                <cylinder length="0.39000000000000001332" radius="0.025000000000000001388" />
-            </geometry>
-        </collision>
-        <collision>
-            <origin xyz="0.46386748875000005654 -0.019645353349999998549 0.083737992499999483464" rpy="3.141592653589793116 -0.27925237217133336287 -0.03490653809662996182" />
-            <geometry>
-                <box size="0.10699999999999999789 0.06500000000000000222 0.076999999999999999001" />
-            </geometry>
-        </collision>
-        <collision>
-            <origin xyz="0.45372929400000000522 -0.034000000000000002442 0.01388592399999948046" rpy="3.141592653589793116 -0.26179929927377620924 6.6901195618362888334e-19" />
-            <geometry>
-                <cylinder length="0.051999999999999997613" radius="0.044999999999999998335" />
-            </geometry>
-        </collision>
-        <inertial>
-            <origin xyz="0.0041039510716027695 -0.0038139455320622536391 0.032209303220248945709" rpy="0 0 0"/>
-            <mass value="3.3615479324277939277" />
-            <inertia ixx="0.009886946037537942128" ixy="0.013947531498206865511" ixz="-0.00045516790513678542958" iyy="0.50779944212378647084" iyz="-0.00018907601015774903527" izz="0.50393207699993247672" />
-        </inertial>
-    </link>
-    <link name="fl_ankle">
-        <visual>
-            <origin xyz="-0.12415341931613703419 2.2204460492503130808e-16 -0.12500000000000027756" rpy="-1.570796326794896558 -0.13351607992219352572 -9.2297733002794394222e-17" />
-            <geometry>
-                <mesh filename="file://$(find rover_description)/base/meshes/fl_ankle.stl"/>
-            </geometry>
-            <material name="fl_ankle_material">
-                <color rgba="0.86666666666666669627 0.074509803921568626417 0.32549019607843138191 1.0"/>
-            </material>
-        </visual>
-        <!-- Shapes for fl_ankle -->
-        <collision>
-            <origin xyz="-0.11601914642063090866 2.19292275781973355e-16 -0.1030492935317774833" rpy="-1.570796326794896558 0.0061101698267939132114 -7.8822470542670411585e-17" />
-            <geometry>
-                <box size="0.032000000000000000666 0.080000000000000001665 0.05999999999999999778" />
-            </geometry>
-        </collision>
-        <collision>
-            <origin xyz="-0.091894553662955680284 2.2318007294450709291e-16 -0.16352745890207484591" rpy="-1.570796326794896558 -0.79674066942340771025 -1.7757103362153874007e-16" />
-            <geometry>
-                <box size="0.020000000000000000416 0.080000000000000001665 0.05999999999999999778" />
-            </geometry>
-        </collision>
-        <collision>
-            <origin xyz="-0.06380085395774162671 2.2443184893324340788e-16 -0.19982021317550338613" rpy="-1.570796326794896558 -0.011343354647681692937 -8.0497369831876207913e-17" />
-            <geometry>
-                <box size="0.025000000000000001388 0.030999999999999999778 0.05999999999999999778" />
-            </geometry>
-        </collision>
-        <collision>
-            <origin xyz="-0.067081786006729482441 2.0976841911263922843e-16 -0.044297919093382376321" rpy="-1.570796326794896558 0.80896192356999563344 2.1183864782663456072e-17" />
-            <geometry>
-                <box size="0.01200000000000000025 0.075999999999999998113 0.05999999999999999778" />
-            </geometry>
-        </collision>
-        <collision>
-            <origin xyz="-0.10777838729007002683 2.15448303306492849e-16 -0.069810716156365762441" rpy="-1.570796326794886566 1.5594529721472147887 8.3798326600223183008e-15" />
-            <geometry>
-                <box size="0.01200000000000000025 0.02999999999999999889 0.05999999999999999778" />
-            </geometry>
-        </collision>
-        <collision>
-            <origin xyz="-0.00045306036165812524352 2.0125859836172068672e-16 -0.010753702302991177686" rpy="1.1392031010790054614e-16 0.0061101698267939132114 -7.8822470542670411585e-17" />
-            <geometry>
-                <cylinder length="0.025999999999999998807" radius="0.037999999999999999056" />
-            </geometry>
-        </collision>
-        <collision>
-            <origin xyz="-0.028495306304552436849 2.0414069199384847611e-16 -0.017582487382379483054" rpy="1.1392031010790054614e-16 0.0061101698267939132114 -7.8822470542670411585e-17" />
-            <geometry>
-                <box size="0.02999999999999999889 0.05999999999999999778 0.01200000000000000025" />
-            </geometry>
-        </collision>
-        <inertial>
-            <origin xyz="-0.073764311118006867241 -5.3026499041559700556e-05 -0.1765990951707425427" rpy="0 0 0"/>
-            <mass value="1.0788921168880700741" />
-            <inertia ixx="0.0095121735844276439353" ixy="-2.4669708784030105233e-06" ixz="-0.0012337645500674794541" iyy="0.010640921973106964166" iyz="4.8002683989303085102e-06" izz="0.0021986116105612192595" />
-        </inertial>
-    </link>
-    <link name="fl_wheel">
-        <visual>
-            <origin xyz="-1.1102230246251565404e-16 2.7755575615628913511e-17 1.9678269430611905477e-17" rpy="7.6465249148938200431e-18 1.8025269388467532324e-16 -6.7707851923284363593e-17" />
-            <geometry>
-                <mesh filename="file://$(find rover_description)/base/meshes/fl_wheel.stl"/>
-            </geometry>
-            <material name="fl_wheel_material">
-                <color rgba="0.86666666666666669627 0.074509803921568626417 0.32549019607843138191 1.0"/>
-            </material>
-        </visual>
-        <!-- Shapes for fl_wheel -->
-        <collision>
-            <origin xyz="-1.1102230246251565404e-16 2.7755575615628913511e-17 1.9678269430611905477e-17" rpy="7.6465249148938200431e-18 1.8025269388467532324e-16 -6.7707851923284363593e-17" />
-            <geometry>
-                <cylinder length="0.16000000000000000333" radius="0.15700000000000000067" />
-            </geometry>
-        </collision>
-        <inertial>
-            <origin xyz="-1.3294988587091283338e-07 -1.120773110686008889e-07 1.2648623649737114364e-05" rpy="0 0 0"/>
-            <mass value="1.8501412404055226357" />
-            <inertia ixx="0.020701719473909981073" ixy="2.9104723315616116698e-05" ixz="1.0888320725737932493e-08" iyy="0.020861663662014581083" iyz="1.4322179501904065656e-08" izz="0.032713974764007960894" />
-        </inertial>
-    </link>
-    <link name="bl_ankle">
-        <visual>
-            <origin xyz="-0.12415341931613702031 2.2204460492503130808e-16 -0.12500000000000027756" rpy="-1.570796326794896558 -0.13351607992219355348 -6.6381828885871895555e-17" />
-            <geometry>
-                <mesh filename="file://$(find rover_description)/base/meshes/bl_ankle.stl"/>
-            </geometry>
-            <material name="bl_ankle_material">
-                <color rgba="0.86666666666666669627 0.074509803921568626417 0.32549019607843138191 1.0"/>
-            </material>
-        </visual>
-        <!-- Shapes for bl_ankle -->
-        <collision>
-            <origin xyz="-0.11601914642063089478 2.1922540380547800281e-16 -0.10304929353177746942" rpy="-1.570796326794896558 0.006110169826793900201 -5.1037120378405970166e-17" />
-            <geometry>
-                <box size="0.032000000000000000666 0.080000000000000001665 0.05999999999999999778" />
-            </geometry>
-        </collision>
-        <collision>
-            <origin xyz="-0.091894553662955666407 2.2458667857737462654e-16 -0.16352745890207487367" rpy="-1.570796326794896558 -0.79674066942340771025 -1.6348523932676255028e-16" />
-            <geometry>
-                <box size="0.020000000000000000416 0.080000000000000001665 0.05999999999999999778" />
-            </geometry>
-        </collision>
-        <collision>
-            <origin xyz="-0.063800853957741612832 2.2709991838731532888e-16 -0.19982021317550338613" rpy="-1.570796326794896558 -0.011343354647681706815 -5.2944381290635227026e-17" />
-            <geometry>
-                <box size="0.025000000000000001388 0.030999999999999999778 0.05999999999999999778" />
-            </geometry>
-        </collision>
-        <collision>
-            <origin xyz="-0.067081786006729454686 2.1027516663082543176e-16 -0.044297919093382362443" rpy="-1.570796326794896558 0.80896192356999563344 6.2843263696355972548e-17" />
-            <geometry>
-                <box size="0.01200000000000000025 0.075999999999999998113 0.05999999999999999778" />
-            </geometry>
-        </collision>
-        <collision>
-            <origin xyz="-0.10777838729007001295 2.151672370229256027e-16 -0.069810716156365748564" rpy="-1.5707963267948870101 1.5594529721472150108 9.5811016025438767714e-15" />
-            <geometry>
-                <box size="0.01200000000000000025 0.02999999999999999889 0.05999999999999999778" />
-            </geometry>
-        </collision>
-        <collision>
-            <origin xyz="-0.00045306036165811136573 2.0316466325611159672e-16 -0.010753702302991163808" rpy="1.0958381951900984966e-16 0.006110169826793900201 -5.1037120378405970166e-17" />
-            <geometry>
-                <cylinder length="0.025999999999999998807" radius="0.037999999999999999056" />
-            </geometry>
-        </collision>
-        <collision>
-            <origin xyz="-0.028495306304552422971 2.0536078413716914081e-16 -0.017582487382379469176" rpy="1.0958381951900984966e-16 0.006110169826793900201 -5.1037120378405970166e-17" />
-            <geometry>
-                <box size="0.02999999999999999889 0.05999999999999999778 0.01200000000000000025" />
-            </geometry>
-        </collision>
-        <inertial>
-            <origin xyz="-0.073764311118006825607 -5.3026499041556129465e-05 -0.17659909517074257046" rpy="0 0 0"/>
-            <mass value="1.0788921168880702961" />
-            <inertia ixx="0.0095121735844276474048" ixy="-2.4669708784009319045e-06" ixz="-0.0012337645500674777194" iyy="0.010640921973106972839" iyz="4.8002683989302153366e-06" izz="0.0021986116105612214279" />
-        </inertial>
-    </link>
-    <link name="bl_wheel">
-        <visual>
-            <origin xyz="0 0 5.4426949058772322587e-17" rpy="2.0912147866144306179e-17 8.2022383815773806625e-17 2.4684305037247577125e-17" />
-            <geometry>
-                <mesh filename="file://$(find rover_description)/base/meshes/bl_wheel.stl"/>
-            </geometry>
-            <material name="bl_wheel_material">
-                <color rgba="0.86666666666666669627 0.074509803921568626417 0.32549019607843138191 1.0"/>
-            </material>
-        </visual>
-        <!-- Shapes for bl_wheel -->
-        <collision>
-            <origin xyz="0 0 5.4426949058772322587e-17" rpy="2.0912147866144306179e-17 8.2022383815773806625e-17 2.4684305037247577125e-17" />
-            <geometry>
-                <cylinder length="0.16000000000000000333" radius="0.15700000000000000067" />
-            </geometry>
-        </collision>
-        <inertial>
-            <origin xyz="-1.3294988576900886706e-07 -1.1207731110400924837e-07 1.264862364977300315e-05" rpy="0 0 0"/>
-            <mass value="1.8501412404055224137" />
-            <inertia ixx="0.020701719473909988012" ixy="2.9104723315619704729e-05" ixz="1.0888320722569594173e-08" iyy="0.020861663662014577614" iyz="1.4322179499876510317e-08" izz="0.032713974764007967833" />
-        </inertial>
-    </link>
-    <link name="right_leg">
-        <visual>
-            <origin xyz="-7.9461177221464552678e-19 -7.285838599104098493e-20 -0.02099999999999946354" rpy="3.141592653589793116 3.7838655819744073932e-17 2.5353252380137503331e-18" />
-            <geometry>
-                <mesh filename="file://$(find rover_description)/base/meshes/right_leg.stl"/>
-            </geometry>
-            <material name="right_leg_material">
-                <color rgba="0.86666666666666669627 0.074509803921568626417 0.32549019607843138191 1.0"/>
-            </material>
-        </visual>
-        <!-- Shapes for right_leg -->
-        <collision>
-            <origin xyz="-7.9461177221464552678e-19 -7.285838599104098493e-20 -0.02099999999999946354" rpy="3.141592653589793116 3.7838655819744073932e-17 2.5353252380137503331e-18" />
-            <geometry>
-                <cylinder length="0.058000000000000002942" radius="0.042999999999999996558" />
-            </geometry>
-        </collision>
-        <collision>
-            <origin xyz="-0.08543333675807499028 -0.0098574827027249987271 -0.013653239999999457546" rpy="3.0194197050837283669 -1.308997029405494894 0.23561907663390049827" />
-            <geometry>
-                <cylinder length="0.089999999999999996669" radius="0.02999999999999999889" />
-            </geometry>
-        </collision>
-        <collision>
-            <origin xyz="-0.31437167947314498262 -0.038053876881360006179 0.044033037700000540737" rpy="3.0194196304823472943 -1.3264501982056555729 0.23561907663390052603" />
-            <geometry>
-                <cylinder length="0.39000000000000001332" radius="0.025000000000000001388" />
-            </geometry>
-        </collision>
-        <collision>
-            <origin xyz="-0.4536556182500000034 0.0013318353999999974976 0.081600174000000552654" rpy="-3.141592653589793116 -0.27925237217133341838 -3.1066861154931633138" />
-            <geometry>
-                <box size="0.105999999999999997 0.06500000000000000222 0.076999999999999999001" />
-            </geometry>
-        </collision>
-        <collision>
-            <origin xyz="-0.44472929399999999722 0.0099999999999999984734 0.010885924000000553324" rpy="-3.141592653589793116 -0.26179929927377626475 -3.141592653589793116" />
-            <geometry>
-                <cylinder length="0.051999999999999997613" radius="0.044999999999999998335" />
-            </geometry>
-        </collision>
-        <collision>
-            <origin xyz="0.085869139396912513851 -0.004569547336145000048 -0.01354282499999946536" rpy="-3.071779613202412218 -1.3089970756114859274 3.0194199283152816093" />
-            <geometry>
-                <cylinder length="0.089999999999999996669" radius="0.02999999999999999889" />
-            </geometry>
-        </collision>
-        <collision>
-            <origin xyz="0.31601584183032671582 -0.019116378127553797228 0.044387337800000523091" rpy="-3.0717796785789528435 -1.326450241590472201 3.0194199283152816093" />
-            <geometry>
-                <cylinder length="0.39000000000000001332" radius="0.025000000000000001388" />
-            </geometry>
-        </collision>
-        <collision>
-            <origin xyz="0.46313595625000003597 0.024684938349999997753 0.083737992500000524299" rpy="3.141592653589793116 -0.27925237217133330736 0.03490653809662996182" />
-            <geometry>
-                <box size="0.10699999999999999789 0.06500000000000000222 0.076999999999999999001" />
-            </geometry>
-        </collision>
-        <collision>
-            <origin xyz="0.45372929400000000522 0.034000000000000002442 0.013885924000000521294" rpy="3.141592653589793116 -0.26179929927377615373 3.4649604177870138712e-18" />
-            <geometry>
-                <cylinder length="0.051999999999999997613" radius="0.044999999999999998335" />
-            </geometry>
-        </collision>
-        <inertial>
-            <origin xyz="0.0065545825522057010737 0.0038734960638154166367 0.031470479082600665011" rpy="0 0 0"/>
-            <mass value="3.3614658220654676235" />
-            <inertia ixx="0.0097971101985132036383" ixy="-0.013185915364469004765" ixz="-0.0016327606378981796183" iyy="0.49985708628931829756" iyz="0.0001950608943907389801" izz="0.49600788361886782862" />
-        </inertial>
-    </link>
-    <link name="fr_ankle">
-        <visual>
-            <origin xyz="0.12415341931613703419 -2.2204460492503130808e-16 -0.12500000000000027756" rpy="-1.57079632679489678 0.13351607992219352572 -1.4831077253695265766e-16" />
-            <geometry>
-                <mesh filename="file://$(find rover_description)/base/meshes/fr_ankle.stl"/>
-            </geometry>
-            <material name="fr_ankle_material">
-                <color rgba="0.86666666666666669627 0.074509803921568626417 0.32549019607843138191 1.0"/>
-            </material>
-        </visual>
-        <!-- Shapes for fr_ankle -->
-        <collision>
-            <origin xyz="0.11601914642063090866 -2.182962099663631774e-16 -0.1030492935317774833" rpy="-1.57079632679489678 0.0061101698267938845885 3.141592653589793116" />
-            <geometry>
-                <box size="0.032000000000000000666 0.080000000000000001665 0.05999999999999999778" />
-            </geometry>
-        </collision>
-        <collision>
-            <origin xyz="0.091894553662955680284 -2.2248367844818289892e-16 -0.16352745890207484591" rpy="-1.57079632679489678 -0.79674066942340759923 3.141592653589793116" />
-            <geometry>
-                <box size="0.020000000000000000416 0.080000000000000001665 0.05999999999999999778" />
-            </geometry>
-        </collision>
-        <collision>
-            <origin xyz="0.063800853957741612832 -2.2319996635520368764e-16 -0.19982021317550338613" rpy="-1.57079632679489678 -0.011343354647681718958 3.141592653589793116" />
-            <geometry>
-                <box size="0.025000000000000001388 0.030999999999999999778 0.05999999999999999778" />
-            </geometry>
-        </collision>
-        <collision>
-            <origin xyz="0.067081786006729454686 -2.0467926758057256531e-16 -0.044297919093382362443" rpy="-1.57079632679489678 0.8089619235699954114 3.141592653589793116" />
-            <geometry>
-                <box size="0.01200000000000000025 0.075999999999999998113 0.05999999999999999778" />
-            </geometry>
-        </collision>
-        <collision>
-            <origin xyz="0.10777838729007002683 -2.1315810577579124768e-16 -0.069810716156365762441" rpy="-1.57079632679490655 1.5594529721472150108 -3.1415926535897824579" />
-            <geometry>
-                <box size="0.01200000000000000025 0.02999999999999999889 0.05999999999999999778" />
-            </geometry>
-        </collision>
-        <collision>
-            <origin xyz="0.00045306036165809748795 -1.9180010690625083433e-16 -0.010753702302991177686" rpy="-1.1172631868889083112e-16 0.0061101698267938845885 3.141592653589793116" />
-            <geometry>
-                <cylinder length="0.025999999999999998807" radius="0.037999999999999999056" />
-            </geometry>
-        </collision>
-        <collision>
-            <origin xyz="0.028495306304552409093 -1.9633227666158057138e-16 -0.017582487382379483054" rpy="-1.1172631868889083112e-16 0.0061101698267938845885 3.141592653589793116" />
-            <geometry>
-                <box size="0.02999999999999999889 0.05999999999999999778 0.01200000000000000025" />
-            </geometry>
-        </collision>
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