Commit message: Reorganised joints to follow left/forward/back/right convention

File: src/ros/rover/rover_description/base/urdf/gz_ros2_control.xacro (robot description, xacro)
@@ -17,5 +17,5 @@
       </state_interface>
     </joint>
-    <joint name='frw'>
+    <joint name='blw'>
       <command_interface name="velocity">
         <param name="min">-50</param>
@@ -29,5 +29,5 @@
       </state_interface>
     </joint>
-    <joint name='blw'>
+    <joint name='frw'>
       <command_interface name="velocity">
         <param name="min">-50</param>
@@ -69,5 +69,5 @@
       </state_interface>
     </joint>
-    <joint name="frp">
+    <joint name="blp">
       <command_interface name="position">
         <param name="min">-${pi}</param>
@@ -85,5 +85,5 @@
       </state_interface>
     </joint>
-    <joint name="blp">
+    <joint name="frp">
       <command_interface name="position">
         <param name="min">-${pi}</param>
@@ -120,5 +120,5 @@
   <gazebo>
     <plugin filename="gz_ros2_control-system" name="gz_ros2_control::GazeboSimROS2ControlPlugin">
-        <parameters>$(find auto_bringup)/params/controllers.yaml</parameters>
+      <parameters>$(find auto_bringup)/params/controllers.yaml</parameters>
     </plugin>
   </gazebo>

File: src/ros/rover/rover_description/base/urdf/joint_states.xacro (robot description, xacro)
@@ -5,14 +5,14 @@
         <plugin filename="gz-sim-joint-state-publisher-system" name="gz::sim::systems::JointStatePublisher">
             <topic>joint_states</topic>
+            <joint_name>chassis_to_left_leg</joint_name>
+            <joint_name>flp</joint_name>
+            <joint_name>flw</joint_name>
             <joint_name>blp</joint_name>
+            <joint_name>blw</joint_name>
+            <joint_name>chassis_to_right_leg</joint_name>
+            <joint_name>frp</joint_name>
+            <joint_name>frw</joint_name>
             <joint_name>brp</joint_name>
-            <joint_name>flp</joint_name>
-            <joint_name>frp</joint_name>
-            <joint_name>blw</joint_name>
             <joint_name>brw</joint_name>
-            <joint_name>flw</joint_name>
-            <joint_name>frw</joint_name>
-            <joint_name>chassis_to_right_leg</joint_name>
-            <joint_name>chassis_to_left_leg</joint_name>
             <joint_name>chassis_to_diffbar</joint_name>
             <joint_name>tl_ball_roll</joint_name>
