Commit message: Reorganised joints to follow left/forward/back/right convention

File: src/ros/rover/rover_description/base/urdf/rover.urdf.xacro (robot description, xacro)
@@ -18,4 +18,590 @@
     <!-- Generated URDF -->
     <link name="base_link"></link>
+    <link name="chassis">
+        <visual>
+            <origin xyz="1.2353683969592321892e-17 1.3877787807815553765e-17 -1.2992673251725723918e-16" rpy="-4.03091968774772598e-16 -5.9777162559529608526e-16 1.57079632679489678" />
+            <geometry>
+                <mesh filename="file://$(find rover_description)/base/meshes/chassis.stl"/>
+            </geometry>
+            <material name="chassis_material">
+                <color rgba="0.86666666666666669627 0.074509803921568626417 0.32549019607843138191 1.0"/>
+            </material>
+        </visual>
+        <!-- Shapes for chassis -->
+        <collision>
+            <origin xyz="-0.17250000000000031974 9.3018238151966802719e-18 0.023499999999999854339" rpy="-4.03091968774772598e-16 -5.9777162559529608526e-16 1.57079632679489678" />
+            <geometry>
+                <box size="0.47999999999999998224 0.54500000000000003997 0.1749999999999999889" />
+            </geometry>
+        </collision>
+        <collision>
+            <origin xyz="0.22700000000000039591 2.8459855857991392753e-18 0.033500000000000043632" rpy="-4.03091968774772598e-16 -5.9777162559529608526e-16 1.57079632679489678" />
+            <geometry>
+                <box size="0.34000000000000002442 0.26000000000000000888 0.19500000000000000666" />
+            </geometry>
+        </collision>
+        <inertial>
+            <origin xyz="-0.022980723180787008403 -0.00012909338240173079686 0.024515364506931026228" rpy="0 0 0"/>
+            <mass value="8.3419541100883876084" />
+            <inertia ixx="0.21737687093594976195" ixy="0.00013546851964915839124" ixz="-0.0088627259627339308873" iyy="0.45541406320296751176" iyz="-0.00021657327861196811977" izz="0.59726536058024382037" />
+        </inertial>
+    </link>
+    <link name="left_leg">
+        <visual>
+            <origin xyz="-1.3078806732583218725e-20 8.6736173798840354721e-19 -0.021000000000000518252" rpy="-3.141592653589793116 6.2280032059897877693e-19 -4.1232880706353110482e-18" />
+            <geometry>
+                <mesh filename="file://$(find rover_description)/base/meshes/left_leg.stl"/>
+            </geometry>
+            <material name="left_leg_material">
+                <color rgba="0.86666666666666669627 0.074509803921568626417 0.32549019607843138191 1.0"/>
+            </material>
+        </visual>
+        <!-- Shapes for left_leg -->
+        <collision>
+            <origin xyz="-1.3078806732583218725e-20 8.6736173798840354721e-19 -0.021000000000000518252" rpy="-3.141592653589793116 6.2280032059897877693e-19 -4.1232880706353110482e-18" />
+            <geometry>
+                <cylinder length="0.058000000000000002942" radius="0.042999999999999996558" />
+            </geometry>
+        </collision>
+        <collision>
+            <origin xyz="-0.085373995000000008071 0.010358865000000005291 -0.013653240000000515728" rpy="3.0194197050837283669 -1.3089970275211204598 -4.1232880706353857743e-18" />
+            <geometry>
+                <cylinder length="0.089999999999999996669" radius="0.02999999999999999889" />
+            </geometry>
+        </collision>
+        <collision>
+            <origin xyz="-0.31456908199999999987 0.036386049000000010578 0.044033037699999472148" rpy="3.0194196304823472943 -1.3264501964363342168 -4.1232880706353919373e-18" />
+            <geometry>
+                <cylinder length="0.39000000000000001332" radius="0.025000000000000001388" />
+            </geometry>
+        </collision>
+        <collision>
+            <origin xyz="-0.46338715075000003196 0.005628579600000003548 0.083600173999999485841" rpy="-3.141592653589793116 -0.27925237217133336287 3.1066861154931633138" />
+            <geometry>
+                <box size="0.105999999999999997 0.06500000000000000222 0.076999999999999999001" />
+            </geometry>
+        </collision>
+        <collision>
+            <origin xyz="-0.45372929400000000522 -0.0080000000000000001665 0.01388592399999948046" rpy="3.141592653589793116 -0.26179929927377620924 3.141592653589793116" />
+            <geometry>
+                <cylinder length="0.051999999999999997613" radius="0.044999999999999998335" />
+            </geometry>
+        </collision>
+        <collision>
+            <origin xyz="0.085785990000000020284 0.0059293025000000023489 -0.013542825000000516603" rpy="-3.071779613202412218 -1.3089970275211204598 3.141592653589793116" />
+            <geometry>
+                <cylinder length="0.089999999999999996669" radius="0.02999999999999999889" />
+            </geometry>
+        </collision>
+        <collision>
+            <origin xyz="0.31599007519999999793 0.019538657500000004147 0.044387337799999482257" rpy="-3.0717796785789528435 -1.3264501964363342168 3.141592653589793116" />
+            <geometry>
+                <cylinder length="0.39000000000000001332" radius="0.025000000000000001388" />
+            </geometry>
+        </collision>
+        <collision>
+            <origin xyz="0.46386748875000005654 -0.019645353350000005488 0.083737992499999483464" rpy="3.141592653589793116 -0.27925237217133336287 -0.034906538096629975698" />
+            <geometry>
+                <box size="0.10699999999999999789 0.06500000000000000222 0.076999999999999999001" />
+            </geometry>
+        </collision>
+        <collision>
+            <origin xyz="0.45372929400000000522 -0.034000000000000009381 0.01388592399999948046" rpy="-3.141592653589793116 -0.26179929927377620924 -4.1232880706353164408e-18" />
+            <geometry>
+                <cylinder length="0.051999999999999997613" radius="0.044999999999999998335" />
+            </geometry>
+        </collision>
+        <inertial>
+            <origin xyz="0.0041039510717090109046 -0.0038139455320666411885 0.032209303220261088774" rpy="0 0 0"/>
+            <mass value="3.3615479324288504159" />
+            <inertia ixx="0.0098869460375398468543" ixy="0.01394753149821242183" ixz="-0.00045516790515138128449" iyy="0.50779944212391792124" iyz="-0.00018907601015712540218" izz="0.50393207700006215077" />
+        </inertial>
+    </link>
+    <link name="fl_ankle">
+        <visual>
+            <origin xyz="-0.12415341931613717297 2.2204460492503130808e-16 -0.1250000000000002498" rpy="-1.570796326794896558 -0.13351607992219349796 -5.9804098682663148249e-17" />
+            <geometry>
+                <mesh filename="file://$(find rover_description)/base/meshes/fl_ankle.stl"/>
+            </geometry>
+            <material name="fl_ankle_material">
+                <color rgba="0.86666666666666669627 0.074509803921568626417 0.32549019607843138191 1.0"/>
+            </material>
+        </visual>
+        <!-- Shapes for fl_ankle -->
+        <collision>
+            <origin xyz="-0.11601914642063104743 2.1917184460597340255e-16 -0.10304929353177745555" rpy="-1.570796326794896558 0.0061101698267938967316 -4.3738590858638602357e-17" />
+            <geometry>
+                <box size="0.032000000000000000666 0.080000000000000001665 0.05999999999999999778" />
+            </geometry>
+        </collision>
+        <collision>
+            <origin xyz="-0.091894553662955805184 2.2501886937905229218e-16 -0.16352745890207481816" rpy="-1.570796326794896558 -0.79674066942340759923 -1.6146882560911951828e-16" />
+            <geometry>
+                <box size="0.020000000000000000416 0.080000000000000001665 0.05999999999999999778" />
+            </geometry>
+        </collision>
+        <collision>
+            <origin xyz="-0.063800853957741737732 2.2792256036812134626e-16 -0.19982021317550335837" rpy="-1.570796326794896558 -0.01134335464768170508 -4.5735443069481638918e-17" />
+            <geometry>
+                <box size="0.025000000000000001388 0.030999999999999999778 0.05999999999999999778" />
+            </geometry>
+        </collision>
+        <collision>
+            <origin xyz="-0.067081786006729593463 2.1027567432387604672e-16 -0.044297919093382348565" rpy="-1.570796326794896558 0.8089619235699954114 7.549118795832927374e-17" />
+            <geometry>
+                <box size="0.01200000000000000025 0.075999999999999998113 0.05999999999999999778" />
+            </geometry>
+        </collision>
+        <collision>
+            <origin xyz="-0.10777838729007016561 2.1500295217861853941e-16 -0.069810716156365748564" rpy="-1.570796326794886788 1.5594529721472150108 1.0040858320181206805e-14" />
+            <geometry>
+                <box size="0.01200000000000000025 0.02999999999999999889 0.05999999999999999778" />
+            </geometry>
+        </collision>
+        <collision>
+            <origin xyz="-0.00045306036165823626582 2.0347719150069473786e-16 -0.010753702302991163808" rpy="1.1151930949963332936e-16 0.0061101698267938967316 -4.3738590858638602357e-17" />
+            <geometry>
+                <cylinder length="0.025999999999999998807" radius="0.037999999999999999056" />
+            </geometry>
+        </collision>
+        <collision>
+            <origin xyz="-0.028495306304552547871 2.0550457667705022165e-16 -0.017582487382379469176" rpy="1.1151930949963332936e-16 0.0061101698267938967316 -4.3738590858638602357e-17" />
+            <geometry>
+                <box size="0.02999999999999999889 0.05999999999999999778 0.01200000000000000025" />
+            </geometry>
+        </collision>
+        <inertial>
+            <origin xyz="-0.073764311118006964385 -5.3026499041438283466e-05 -0.17659909517074259822" rpy="0 0 0"/>
+            <mass value="1.078892116888069852" />
+            <inertia ixx="0.0095121735844276578131" ixy="-2.4669708784088618269e-06" ixz="-0.0012337645500674738162" iyy="0.010640921973106971105" iyz="4.8002683989353873197e-06" izz="0.0021986116105612218616" />
+        </inertial>
+    </link>
+    <link name="fl_wheel">
+        <visual>
+            <origin xyz="5.5511151231257827021e-17 0 5.963111948670274387e-18" rpy="7.279848939407052303e-17 1.0638440422271473935e-16 -6.3914183266779029169e-20" />
+            <geometry>
+                <mesh filename="file://$(find rover_description)/base/meshes/fl_wheel.stl"/>
+            </geometry>
+            <material name="fl_wheel_material">
+                <color rgba="0.86666666666666669627 0.074509803921568626417 0.32549019607843138191 1.0"/>
+            </material>
+        </visual>
+        <!-- Shapes for fl_wheel -->
+        <collision>
+            <origin xyz="5.5511151231257827021e-17 0 5.963111948670274387e-18" rpy="7.279848939407052303e-17 1.0638440422271473935e-16 -6.3914183266779029169e-20" />
+            <geometry>
+                <cylinder length="0.16000000000000000333" radius="0.15700000000000000067" />
+            </geometry>
+        </collision>
+        <inertial>
+            <origin xyz="-1.3294988570490371955e-07 -1.1207731107302232147e-07 1.264862364972365501e-05" rpy="0 0 0"/>
+            <mass value="1.8501412404055228578" />
+            <inertia ixx="0.02070171947391000189" ixy="2.910472331561674689e-05" ixz="1.0888320724661912791e-08" iyy="0.020861663662014588022" iyz="1.4322179500244521317e-08" izz="0.03271397476400798171" />
+        </inertial>
+    </link>
+    <link name="bl_ankle">
+        <visual>
+            <origin xyz="-0.12415341931613714521 2.2204460492503130808e-16 -0.1250000000000002498" rpy="-1.570796326794896558 -0.13351607992219349796 -7.1088909477657821376e-17" />
+            <geometry>
+                <mesh filename="file://$(find rover_description)/base/meshes/bl_ankle.stl"/>
+            </geometry>
+            <material name="bl_ankle_material">
+                <color rgba="0.86666666666666669627 0.074509803921568626417 0.32549019607843138191 1.0"/>
+            </material>
+        </visual>
+        <!-- Shapes for bl_ankle -->
+        <collision>
+            <origin xyz="-0.11601914642063101968 2.1928653432828202268e-16 -0.10304929353177745555" rpy="-1.570796326794896558 0.0061101698267938975989 -5.6413530748343955555e-17" />
+            <geometry>
+                <box size="0.032000000000000000666 0.080000000000000001665 0.05999999999999999778" />
+            </geometry>
+        </collision>
+        <collision>
+            <origin xyz="-0.091894553662955791307 2.2423054222269956331e-16 -0.16352745890207481816" rpy="-1.570796326794896558 -0.79674066942340759923 -1.6395670969913067589e-16" />
+            <geometry>
+                <box size="0.020000000000000000416 0.080000000000000001665 0.05999999999999999778" />
+            </geometry>
+        </collision>
+        <collision>
+            <origin xyz="-0.063800853957741737732 2.2642056960643821642e-16 -0.19982021317550335837" rpy="-1.570796326794896558 -0.01134335464768170508 -5.8237597735928808813e-17" />
+            <geometry>
+                <box size="0.025000000000000001388 0.030999999999999999778 0.05999999999999999778" />
+            </geometry>
+        </collision>
+        <collision>
+            <origin xyz="-0.067081786006729579586 2.1035465020333938258e-16 -0.044297919093382348565" rpy="-1.570796326794896558 0.80896192356999552242 5.2499438522054276927e-17" />
+            <geometry>
+                <box size="0.01200000000000000025 0.075999999999999998113 0.05999999999999999778" />
+            </geometry>
+        </collision>
+        <collision>
+            <origin xyz="-0.10777838729007013785 2.1534273165818391301e-16 -0.069810716156365748564" rpy="-1.5707963267948870101 1.5594529721472150108 9.1555753228293068482e-15" />
+            <geometry>
+                <box size="0.01200000000000000025 0.02999999999999999889 0.05999999999999999778" />
+            </geometry>
+        </collision>
+        <collision>
+            <origin xyz="-0.00045306036165820851025 2.0304775058502743355e-16 -0.010753702302991163808" rpy="1.1008132477927107497e-16 0.0061101698267938975989 -5.6413530748343955555e-17" />
+            <geometry>
+                <cylinder length="0.025999999999999998807" radius="0.037999999999999999056" />
+            </geometry>
+        </collision>
+        <collision>
+            <origin xyz="-0.028495306304552533994 2.0536127236143874224e-16 -0.017582487382379469176" rpy="1.1008132477927107497e-16 0.0061101698267938975989 -5.6413530748343955555e-17" />
+            <geometry>
+                <box size="0.02999999999999999889 0.05999999999999999778 0.01200000000000000025" />
+            </geometry>
+        </collision>
+        <inertial>
+            <origin xyz="-0.073764311118006936629 -5.3026499041441197259e-05 -0.1765990951707425427" rpy="0 0 0"/>
+            <mass value="1.0788921168880714063" />
+            <inertia ixx="0.009512173584427652609" ixy="-2.4669708784086771737e-06" ixz="-0.0012337645500674753341" iyy="0.010640921973106972839" iyz="4.8002683989354982811e-06" izz="0.0021986116105612205605" />
+        </inertial>
+    </link>
+    <link name="bl_wheel">
+        <visual>
+            <origin xyz="0 1.1102230246251565404e-16 1.7780915628762272718e-17" rpy="4.6040217445536182725e-17 1.0513492286565858337e-16 2.3412503191653332746e-19" />
+            <geometry>
+                <mesh filename="file://$(find rover_description)/base/meshes/bl_wheel.stl"/>
+            </geometry>
+            <material name="bl_wheel_material">
+                <color rgba="0.86666666666666669627 0.074509803921568626417 0.32549019607843138191 1.0"/>
+            </material>
+        </visual>
+        <!-- Shapes for bl_wheel -->
+        <collision>
+            <origin xyz="0 1.1102230246251565404e-16 1.7780915628762272718e-17" rpy="4.6040217445536182725e-17 1.0513492286565858337e-16 2.3412503191653332746e-19" />
+            <geometry>
+                <cylinder length="0.16000000000000000333" radius="0.15700000000000000067" />
+            </geometry>
+        </collision>
+        <inertial>
+            <origin xyz="-1.3294988576672050168e-07 -1.1207731096237849715e-07 1.2648623649735338983e-05" rpy="0 0 0"/>
+            <mass value="1.8501412404055201932" />
+            <inertia ixx="0.020701719473909970665" ixy="2.9104723315617170407e-05" ixz="1.0888320724778338462e-08" iyy="0.020861663662014581083" iyz="1.4322179503676726944e-08" izz="0.032713974764007967833" />
+        </inertial>
+    </link>
+    <link name="right_leg">
+        <visual>
+            <origin xyz="-7.9461177221465168975e-19 -7.2858385990954703269e-20 -0.020999999999999519051" rpy="3.141592653589793116 3.7838655819744092421e-17 -5.8406613147999892266e-19" />
+            <geometry>
+                <mesh filename="file://$(find rover_description)/base/meshes/right_leg.stl"/>
+            </geometry>
+            <material name="right_leg_material">
+                <color rgba="0.86666666666666669627 0.074509803921568626417 0.32549019607843138191 1.0"/>
+            </material>
+        </visual>
+        <!-- Shapes for right_leg -->
+        <collision>
+            <origin xyz="-7.9461177221465168975e-19 -7.2858385990954703269e-20 -0.020999999999999519051" rpy="3.141592653589793116 3.7838655819744092421e-17 -5.8406613147999892266e-19" />
+            <geometry>
+                <cylinder length="0.058000000000000002942" radius="0.042999999999999996558" />
+            </geometry>
+        </collision>
+        <collision>
+            <origin xyz="-0.08543333675807499028 -0.0098574827027249987271 -0.013653239999999513057" rpy="3.0194197050837283669 -1.308997029405494894 0.23561907663390049827" />
+            <geometry>
+                <cylinder length="0.089999999999999996669" radius="0.02999999999999999889" />
+            </geometry>
+        </collision>
+        <collision>
+            <origin xyz="-0.31437167947314498262 -0.03805387688135999924 0.044033037700000485226" rpy="3.0194196304823472943 -1.3264501982056555729 0.23561907663390052603" />
+            <geometry>
+                <cylinder length="0.39000000000000001332" radius="0.025000000000000001388" />
+            </geometry>
+        </collision>
+        <collision>
+            <origin xyz="-0.4536556182500000034 0.0013318353999999990155 0.081600174000000497143" rpy="-3.141592653589793116 -0.27925237217133341838 -3.1066861154931633138" />
+            <geometry>
+                <box size="0.105999999999999997 0.06500000000000000222 0.076999999999999999001" />
+            </geometry>
+        </collision>
+        <collision>
+            <origin xyz="-0.44472929399999999722 0.010000000000000000208 0.010885924000000497813" rpy="-3.141592653589793116 -0.26179929927377626475 3.141592653589793116" />
+            <geometry>
+                <cylinder length="0.051999999999999997613" radius="0.044999999999999998335" />
+            </geometry>
+        </collision>
+        <collision>
+            <origin xyz="0.085869139396912513851 -0.004569547336145000048 -0.013542824999999520871" rpy="-3.071779613202412218 -1.3089970756114859274 3.0194199283152816093" />
+            <geometry>
+                <cylinder length="0.089999999999999996669" radius="0.02999999999999999889" />
+            </geometry>
+        </collision>
+        <collision>
+            <origin xyz="0.31601584183032671582 -0.019116378127553797228 0.04438733780000046758" rpy="-3.0717796785789528435 -1.326450241590472201 3.0194199283152816093" />
+            <geometry>
+                <cylinder length="0.39000000000000001332" radius="0.025000000000000001388" />
+            </geometry>
+        </collision>
+        <collision>
+            <origin xyz="0.46313595625000003597 0.024684938349999994284 0.083737992500000468787" rpy="3.141592653589793116 -0.27925237217133330736 0.034906538096629954882" />
+            <geometry>
+                <box size="0.10699999999999999789 0.06500000000000000222 0.076999999999999999001" />
+            </geometry>
+        </collision>
+        <collision>
+            <origin xyz="0.45372929400000000522 0.033999999999999995504 0.013885924000000465783" rpy="3.141592653589793116 -0.26179929927377615373 3.4556904829327689326e-19" />
+            <geometry>
+                <cylinder length="0.051999999999999997613" radius="0.044999999999999998335" />
+            </geometry>
+        </collision>
+        <inertial>
+            <origin xyz="0.0065545825522055648979 0.0038734960638154075294 0.031470479082600609499" rpy="0 0 0"/>
+            <mass value="3.3614658220654680676" />
+            <inertia ixx="0.009797110198513205373" ixy="-0.013185915364468982214" ixz="-0.0016327606378981614037" iyy="0.49985708628931824204" iyz="0.00019506089439073800431" izz="0.49600788361886777311" />
+        </inertial>
+    </link>
+    <link name="fr_ankle">
+        <visual>
+            <origin xyz="0.12415341931613695092 -2.2204460492503130808e-16 -0.12500000000000027756" rpy="-1.57079632679489678 0.13351607992219352572 9.9507186100571649487e-18" />
+            <geometry>
+                <mesh filename="file://$(find rover_description)/base/meshes/fr_ankle.stl"/>
+            </geometry>
+            <material name="fr_ankle_material">
+                <color rgba="0.86666666666666669627 0.074509803921568626417 0.32549019607843138191 1.0"/>
+            </material>
+        </visual>
+        <!-- Shapes for fr_ankle -->
+        <collision>
+            <origin xyz="0.11601914642063082539 -2.1992446762904779943e-16 -0.1030492935317774833" rpy="-1.57079632679489678 0.0061101698267938854559 -3.141592653589793116" />
+            <geometry>
+                <box size="0.032000000000000000666 0.080000000000000001665 0.05999999999999999778" />
+            </geometry>
+        </collision>
+        <collision>
+            <origin xyz="0.091894553662955597018 -2.2688848533221555828e-16 -0.16352745890207484591" rpy="-1.57079632679489678 -0.79674066942340771025 3.141592653589793116" />
+            <geometry>
+                <box size="0.020000000000000000416 0.080000000000000001665 0.05999999999999999778" />
+            </geometry>
+        </collision>
+        <collision>
+            <origin xyz="0.063800853957741543443 -2.3139606365514587764e-16 -0.19982021317550338613" rpy="-1.57079632679489678 -0.011343354647681718958 -3.141592653589793116" />
+            <geometry>
+                <box size="0.025000000000000001388 0.030999999999999999778 0.05999999999999999778" />
+            </geometry>
+        </collision>
+        <collision>
+            <origin xyz="0.067081786006729385297 -2.1490525250526497332e-16 -0.044297919093382362443" rpy="-1.57079632679489678 0.80896192356999552242 -3.141592653589793116" />
+            <geometry>
+                <box size="0.01200000000000000025 0.075999999999999998113 0.05999999999999999778" />
+            </geometry>
+        </collision>
+        <collision>
+            <origin xyz="0.10777838729006994356 -2.1661573431850512129e-16 -0.069810716156365762441" rpy="-1.570796326794906328 1.5594529721472150108 -3.1415926535897837901" />
+            <geometry>
+                <box size="0.01200000000000000025 0.02999999999999999889 0.05999999999999999778" />
+            </geometry>
+        </collision>
+        <collision>
+            <origin xyz="0.00045306036165801422122 -2.129728451494317697e-16 -0.010753702302991177686" rpy="-1.1068855744643065578e-16 0.0061101698267938854559 -3.141592653589793116" />
+            <geometry>
+                <cylinder length="0.025999999999999998807" radius="0.037999999999999999056" />
+            </geometry>
+        </collision>
+        <collision>
+            <origin xyz="0.028495306304552339705 -2.1301695578387221224e-16 -0.017582487382379483054" rpy="-1.1068855744643065578e-16 0.0061101698267938854559 -3.141592653589793116" />
+            <geometry>
+                <box size="0.02999999999999999889 0.05999999999999999778 0.01200000000000000025" />
+            </geometry>
+        </collision>
+        <inertial>
+            <origin xyz="0.073764311118006756218 5.3026499041436704596e-05 -0.17659909517074259822" rpy="0 0 0"/>
+            <mass value="1.078892116888069852" />
+            <inertia ixx="0.0095121735844276543437" ixy="-2.4669708784060717004e-06" ixz="0.0012337645500674742499" iyy="0.010640921973106974574" iyz="-4.8002683989354288244e-06" izz="0.0021986116105612205605" />
+        </inertial>
+    </link>
+    <link name="fr_wheel">
+        <visual>
+            <origin xyz="5.5511151231257827021e-17 -1.1102230246251565404e-16 -3.0791341698588325926e-17" rpy="-3.6194812825998444115e-17 1.0511409763610977507e-16 -2.2325341479697011877e-19" />
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