Commit message: removing complex difflink collision meshes

File: src/ros/rover/rover_description/base/urdf/rover.urdf.xacro (robot description, xacro)
@@ -556,10 +556,4 @@
             </material>
         </visual>
-        <collision>
-            <origin xyz="-2.7755575615628913511e-15 -0.057750000000000162315 3.3306690738754696213e-16" rpy="1.5707963267948350516 -1.5127867282353739675 -3.1415926535897926719" />
-            <geometry>
-                <mesh filename="file://$(find rover_description)/base/meshes/left_difflink.stl"/>
-            </geometry>
-        </collision>
         <inertial>
             <origin xyz="-1.8798676496980571235e-15 -0.057750000000001855405 1.1529028097132935777e-15" rpy="0 0 0"/>
@@ -585,10 +579,4 @@
             </material>
         </visual>
-        <collision>
-            <origin xyz="6.2172489379008766264e-15 -0.057749999999999454547 -2.4424906541753443889e-15" rpy="1.5707963267948286123 1.512786629442331332 3.141592653589793116" />
-            <geometry>
-                <mesh filename="file://$(find rover_description)/base/meshes/right_difflink.stl"/>
-            </geometry>
-        </collision>
         <inertial>
             <origin xyz="6.539347896424171253e-15 -0.057749999999999142297 -2.7764723681069561858e-15" rpy="0 0 0"/>
