Commit message: add auger/drill controllers

File: src/ros/rover/rover_description/base/urdf/ros2_control.xacro (robot description, xacro)
@@ -307,5 +307,5 @@
             </joint>
         </ros2_control>
-        <ros2_control name="Auger" type="system">
+	<ros2_control name="Auger" type="system">
             <xacro:unless value="${use_mock_hardware}">
                 <hardware>
@@ -313,14 +313,44 @@
 		    <!-- What's the canid? Is it useful? -->
 		    <!-- <param name="canid">8</param> -->
-		    <param name="auger_max_vel">24575</param>
-		    <param name="drill_max_vel">24575</param>
-                </hardware>
-            </xacro:unless>
-            <xacro:if value="${use_mock_hardware}">
-                <hardware>
-                    <plugin>mock_components/GenericSystem</plugin>
-                    <param name="calculate_dynamics">true</param>
-                </hardware>
-            </xacro:if>
+                </hardware>
+	    </xacro:unless>
+            <xacro:if value="${use_mock_hardware}">
+                <hardware>
+                    <plugin>mock_components/GenericSystem</plugin>
+                    <param name="calculate_dynamics">true</param>
+                </hardware>
+            </xacro:if>
+	    <joint name="auger">
+		<command_interface name="direction">
+		    <param name="min">-1</param>
+	      	    <param name="max">1</param>
+                </command_interface>
+                <command_interface name="velocity">
+		    <!-- 24575 = 32767 (max velocity) * 3/4 -->
+		    <param name="max">24575</param>
+                </command_interface>
+		<state_interface name="direction">
+                    <param name="initial_value">1</param>
+                </state_interface>
+		<state_interface name="velocity">
+                    <param name="initial_value">0.0</param>
+                </state_interface>
+            </joint>
+	    <joint name="drill">
+		<command_interface name="direction">
+		    <param name="min">-1</param>
+	      	    <param name="max">1</param>
+                </command_interface>
+                <command_interface name="velocity">
+		    <!-- 24575 = 32767 (max velocity) * 3/4 -->
+		    <param name="max">24575</param>
+                </command_interface>
+		<state_interface name="direction">
+                    <param name="initial_value">1</param>
+                </state_interface>
+		<state_interface name="velocity">
+                    <param name="initial_value">0.0</param>
+                </state_interface>
+            </joint>
         </ros2_control>
     </xacro:macro>

Commit message: created .xacro for scraper. scraper_hardware interface may be abandoned currently, realigning to QCMD hardware interface

File: src/ros/rover/rover_description/base/urdf/ros2_control.xacro (robot description, xacro)
@@ -307,4 +307,39 @@
             </joint>
         </ros2_control>
+        <ros2_control name="Scraper" type="system">
+            <xacro>
+                <hardware>
+                    <plugin>scraper_hardware/ScraperHardware</plugin>
+                    <param name="candevice">can1</param>
+                    <param name="canid">1</param>
+                    <param name="resolver_reduction">1.33333333333</param>
+                    <param name="clock_rate">100000000</param>
+                    <param name="revolution_pulses">8192</param>
+                    <param name="min_interval">122</param>
+                    <param name="gear_ratio">36.0</param>
+                    <param name="mock">true</param>
+                    <param name="reversed">true</param>
+                    <param name="integrate_velocity">true</param>
+                </hardware>
+            </xacro>
+            <joint name="arm">
+		        <command_interface name="velocity">
+                    <param name="max_scaling">1</param>
+                </command_interface>
+            </joint>
+            <joint name="bucket">
+                <command_interface name="velocity">
+                    <param name="max_scaling">0.6</param>
+                </command_interface>
+                <state_interface name="position">
+                    <param name="initial_value">0</param>
+                </state_interface>
+            </joint>
+            <joint name="scoop">
+		        <command_interface name="velocity">
+                    <param name="max_scaling">1</param>
+                </command_interface>
+            </joint>
+        </ros2_control>
     </xacro:macro>
 </robot>

Commit message: Revert "add auger/drill controllers"
This reverts commit 253f54f6a5235aa6eae5fcba91d565acfdc20c00.

File: src/ros/rover/rover_description/base/urdf/ros2_control.xacro (robot description, xacro)
@@ -307,5 +307,5 @@
             </joint>
         </ros2_control>
-	<ros2_control name="Auger" type="system">
+        <ros2_control name="Auger" type="system">
             <xacro:unless value="${use_mock_hardware}">
                 <hardware>
@@ -313,44 +313,14 @@
 		    <!-- What's the canid? Is it useful? -->
 		    <!-- <param name="canid">8</param> -->
-                </hardware>
-	    </xacro:unless>
-            <xacro:if value="${use_mock_hardware}">
-                <hardware>
-                    <plugin>mock_components/GenericSystem</plugin>
-                    <param name="calculate_dynamics">true</param>
-                </hardware>
-            </xacro:if>
-	    <joint name="auger">
-		<command_interface name="direction">
-		    <param name="min">-1</param>
-	      	    <param name="max">1</param>
-                </command_interface>
-                <command_interface name="velocity">
-		    <!-- 24575 = 32767 (max velocity) * 3/4 -->
-		    <param name="max">24575</param>
-                </command_interface>
-		<state_interface name="direction">
-                    <param name="initial_value">1</param>
-                </state_interface>
-		<state_interface name="velocity">
-                    <param name="initial_value">0.0</param>
-                </state_interface>
-            </joint>
-	    <joint name="drill">
-		<command_interface name="direction">
-		    <param name="min">-1</param>
-	      	    <param name="max">1</param>
-                </command_interface>
-                <command_interface name="velocity">
-		    <!-- 24575 = 32767 (max velocity) * 3/4 -->
-		    <param name="max">24575</param>
-                </command_interface>
-		<state_interface name="direction">
-                    <param name="initial_value">1</param>
-                </state_interface>
-		<state_interface name="velocity">
-                    <param name="initial_value">0.0</param>
-                </state_interface>
-            </joint>
+		    <param name="auger_max_vel">24575</param>
+		    <param name="drill_max_vel">24575</param>
+                </hardware>
+            </xacro:unless>
+            <xacro:if value="${use_mock_hardware}">
+                <hardware>
+                    <plugin>mock_components/GenericSystem</plugin>
+                    <param name="calculate_dynamics">true</param>
+                </hardware>
+            </xacro:if>
         </ros2_control>
     </xacro:macro>

Commit message: Created .xacro template for joints on QCMD and removed scraper hardware interface

File: src/ros/rover/rover_description/base/urdf/ros2_control.xacro (robot description, xacro)
@@ -307,39 +307,4 @@
             </joint>
         </ros2_control>
-        <ros2_control name="Scraper" type="system">
-            <xacro>
-                <hardware>
-                    <plugin>scraper_hardware/ScraperHardware</plugin>
-                    <param name="candevice">can1</param>
-                    <param name="canid">1</param>
-                    <param name="resolver_reduction">1.33333333333</param>
-                    <param name="clock_rate">100000000</param>
-                    <param name="revolution_pulses">8192</param>
-                    <param name="min_interval">122</param>
-                    <param name="gear_ratio">36.0</param>
-                    <param name="mock">true</param>
-                    <param name="reversed">true</param>
-                    <param name="integrate_velocity">true</param>
-                </hardware>
-            </xacro>
-            <joint name="arm">
-		        <command_interface name="velocity">
-                    <param name="max_scaling">1</param>
-                </command_interface>
-            </joint>
-            <joint name="bucket">
-                <command_interface name="velocity">
-                    <param name="max_scaling">0.6</param>
-                </command_interface>
-                <state_interface name="position">
-                    <param name="initial_value">0</param>
-                </state_interface>
-            </joint>
-            <joint name="scoop">
-		        <command_interface name="velocity">
-                    <param name="max_scaling">1</param>
-                </command_interface>
-            </joint>
-        </ros2_control>
     </xacro:macro>
 </robot>
