Commit message: renamed base to rover7 in rover_description, and corrected filepaths for arm.urdf.xacro

File: src/ros/rover/rover_description/arm/urdf/arm.urdf.xacro (robot description, xacro)
@@ -29,19 +29,19 @@
       <geometry>
         <mesh
-          filename="file://$(find rover_description)/meshes/arm_base.stl" />
-      </geometry>
-      <material
-        name="">
-        <color
-          rgba="0.792156862745098 0.819607843137255 0.933333333333333 1" />
-      </material>
-    </visual>
-    <collision>
-      <origin
-        xyz="0 0 0"
-        rpy="0 0 0" />
-      <geometry>
-        <mesh
-          filename="file://$(find rover_description)/meshes/arm_base.stl" />
+          filename="file://$(find rover_description)/arm/meshes/arm_base.stl" />
+      </geometry>
+      <material
+        name="">
+        <color
+          rgba="0.792156862745098 0.819607843137255 0.933333333333333 1" />
+      </material>
+    </visual>
+    <collision>
+      <origin
+        xyz="0 0 0"
+        rpy="0 0 0" />
+      <geometry>
+        <mesh
+          filename="file://$(find rover_description)/arm/meshes/arm_base.stl" />
       </geometry>
     </collision>
@@ -69,19 +69,19 @@
       <geometry>
         <mesh
-          filename="file://$(find rover_description)/meshes/base_to_j1.stl" />
-      </geometry>
-      <material
-        name="">
-        <color
-          rgba="0.792156862745098 0.819607843137255 0.933333333333333 1" />
-      </material>
-    </visual>
-    <collision>
-      <origin
-        xyz="0 0 0"
-        rpy="0 0 0" />
-      <geometry>
-        <mesh
-          filename="file://$(find rover_description)/meshes/base_to_j1.stl" />
+          filename="file://$(find rover_description)/arm/meshes/base_to_j1.stl" />
+      </geometry>
+      <material
+        name="">
+        <color
+          rgba="0.792156862745098 0.819607843137255 0.933333333333333 1" />
+      </material>
+    </visual>
+    <collision>
+      <origin
+        xyz="0 0 0"
+        rpy="0 0 0" />
+      <geometry>
+        <mesh
+          filename="file://$(find rover_description)/arm/meshes/base_to_j1.stl" />
       </geometry>
     </collision>
@@ -127,19 +127,19 @@
       <geometry>
         <mesh
-          filename="file://$(find rover_description)/meshes/j2_to_link1.stl" />
-      </geometry>
-      <material
-        name="">
-        <color
-          rgba="0.792156862745098 0.819607843137255 0.933333333333333 1" />
-      </material>
-    </visual>
-    <collision>
-      <origin
-        xyz="0 0 0"
-        rpy="0 0 0" />
-      <geometry>
-        <mesh
-          filename="file://$(find rover_description)/meshes/j2_to_link1.stl" />
+          filename="file://$(find rover_description)/arm/meshes/j2_to_link1.stl" />
+      </geometry>
+      <material
+        name="">
+        <color
+          rgba="0.792156862745098 0.819607843137255 0.933333333333333 1" />
+      </material>
+    </visual>
+    <collision>
+      <origin
+        xyz="0 0 0"
+        rpy="0 0 0" />
+      <geometry>
+        <mesh
+          filename="file://$(find rover_description)/arm/meshes/j2_to_link1.stl" />
       </geometry>
     </collision>
@@ -185,19 +185,19 @@
       <geometry>
         <mesh
-          filename="file://$(find rover_description)/meshes/j3_to_link2.stl" />
-      </geometry>
-      <material
-        name="">
-        <color
-          rgba="0.792156862745098 0.819607843137255 0.933333333333333 1" />
-      </material>
-    </visual>
-    <collision>
-      <origin
-        xyz="0 0 0"
-        rpy="0 0 0" />
-      <geometry>
-        <mesh
-          filename="file://$(find rover_description)/meshes/j3_to_link2.stl" />
+          filename="file://$(find rover_description)/arm/meshes/j3_to_link2.stl" />
+      </geometry>
+      <material
+        name="">
+        <color
+          rgba="0.792156862745098 0.819607843137255 0.933333333333333 1" />
+      </material>
+    </visual>
+    <collision>
+      <origin
+        xyz="0 0 0"
+        rpy="0 0 0" />
+      <geometry>
+        <mesh
+          filename="file://$(find rover_description)/arm/meshes/j3_to_link2.stl" />
       </geometry>
     </collision>
@@ -243,19 +243,19 @@
       <geometry>
         <mesh
-          filename="file://$(find rover_description)/meshes/link2_to_fixed_j4.stl" />
-      </geometry>
-      <material
-        name="">
-        <color
-          rgba="0.792156862745098 0.819607843137255 0.933333333333333 1" />
-      </material>
-    </visual>
-    <collision>
-      <origin
-        xyz="0 0 0"
-        rpy="0 0 0" />
-      <geometry>
-        <mesh
-          filename="file://$(find rover_description)/meshes/link2_to_fixed_j4.stl" />
+          filename="file://$(find rover_description)/arm/meshes/link2_to_fixed_j4.stl" />
+      </geometry>
+      <material
+        name="">
+        <color
+          rgba="0.792156862745098 0.819607843137255 0.933333333333333 1" />
+      </material>
+    </visual>
+    <collision>
+      <origin
+        xyz="0 0 0"
+        rpy="0 0 0" />
+      <geometry>
+        <mesh
+          filename="file://$(find rover_description)/arm/meshes/link2_to_fixed_j4.stl" />
       </geometry>
     </collision>
@@ -296,19 +296,19 @@
       <geometry>
         <mesh
-          filename="file://$(find rover_description)/meshes/j4_to_j5.stl" />
-      </geometry>
-      <material
-        name="">
-        <color
-          rgba="0.792156862745098 0.819607843137255 0.933333333333333 1" />
-      </material>
-    </visual>
-    <collision>
-      <origin
-        xyz="0 0 0"
-        rpy="0 0 0" />
-      <geometry>
-        <mesh
-          filename="file://$(find rover_description)/meshes/j4_to_j5.stl" />
+          filename="file://$(find rover_description)/arm/meshes/j4_to_j5.stl" />
+      </geometry>
+      <material
+        name="">
+        <color
+          rgba="0.792156862745098 0.819607843137255 0.933333333333333 1" />
+      </material>
+    </visual>
+    <collision>
+      <origin
+        xyz="0 0 0"
+        rpy="0 0 0" />
+      <geometry>
+        <mesh
+          filename="file://$(find rover_description)/arm/meshes/j4_to_j5.stl" />
       </geometry>
     </collision>
@@ -354,19 +354,19 @@
       <geometry>
         <mesh
-          filename="file://$(find rover_description)/meshes/j5_to_j6.stl" />
-      </geometry>
-      <material
-        name="">
-        <color
-          rgba="0.792156862745098 0.819607843137255 0.933333333333333 1" />
-      </material>
-    </visual>
-    <collision>
-      <origin
-        xyz="0 0 0"
-        rpy="0 0 0" />
-      <geometry>
-        <mesh
-          filename="file://$(find rover_description)/meshes/j5_to_j6.stl" />
+          filename="file://$(find rover_description)/arm/meshes/j5_to_j6.stl" />
+      </geometry>
+      <material
+        name="">
+        <color
+          rgba="0.792156862745098 0.819607843137255 0.933333333333333 1" />
+      </material>
+    </visual>
+    <collision>
+      <origin
+        xyz="0 0 0"
+        rpy="0 0 0" />
+      <geometry>
+        <mesh
+          filename="file://$(find rover_description)/arm/meshes/j5_to_j6.stl" />
       </geometry>
     </collision>
@@ -412,19 +412,19 @@
       <geometry>
         <mesh
-          filename="file://$(find rover_description)/meshes/j6_to_ee.stl" />
-      </geometry>
-      <material
-        name="">
-        <color
-          rgba="0.792156862745098 0.819607843137255 0.933333333333333 1" />
-      </material>
-    </visual>
-    <collision>
-      <origin
-        xyz="0 0 0"
-        rpy="0 0 0" />
-      <geometry>
-        <mesh
-          filename="file://$(find rover_description)/meshes/j6_to_ee.stl" />
+          filename="file://$(find rover_description)/arm/meshes/j6_to_ee.stl" />
+      </geometry>
+      <material
+        name="">
+        <color
+          rgba="0.792156862745098 0.819607843137255 0.933333333333333 1" />
+      </material>
+    </visual>
+    <collision>
+      <origin
+        xyz="0 0 0"
+        rpy="0 0 0" />
+      <geometry>
+        <mesh
+          filename="file://$(find rover_description)/arm/meshes/j6_to_ee.stl" />
       </geometry>
     </collision>

File: src/ros/rover/rover_description/rover7/urdf/rover.urdf.xacro (robot description, xacro)
@@ -22,5 +22,5 @@
             <origin xyz="1.2353683969592321892e-17 1.3877787807815553765e-17 -1.2992673251725723918e-16" rpy="-4.03091968774772598e-16 -5.9777162559529608526e-16 1.57079632679489678" />
             <geometry>
-                <mesh filename="file://$(find rover_description)/base/meshes/chassis.stl"/>
+                <mesh filename="file://$(find rover_description)/rover7/meshes/chassis.stl"/>
             </geometry>
             <material name="chassis_material">
@@ -51,5 +51,5 @@
             <origin xyz="-1.3078806732583218725e-20 8.6736173798840354721e-19 -0.021000000000000518252" rpy="-3.141592653589793116 6.2280032059897877693e-19 -4.1232880706353110482e-18" />
             <geometry>
-                <mesh filename="file://$(find rover_description)/base/meshes/left_leg.stl"/>
+                <mesh filename="file://$(find rover_description)/rover7/meshes/left_leg.stl"/>
             </geometry>
             <material name="left_leg_material">
@@ -122,5 +122,5 @@
             <origin xyz="-0.12415341931613717297 2.2204460492503130808e-16 -0.1250000000000002498" rpy="-1.570796326794896558 -0.13351607992219349796 -5.9804098682663148249e-17" />
             <geometry>
-                <mesh filename="file://$(find rover_description)/base/meshes/fl_ankle.stl"/>
+                <mesh filename="file://$(find rover_description)/rover7/meshes/fl_ankle.stl"/>
             </geometry>
             <material name="fl_ankle_material">
@@ -181,5 +181,5 @@
             <origin xyz="5.5511151231257827021e-17 0 5.963111948670274387e-18" rpy="7.279848939407052303e-17 1.0638440422271473935e-16 -6.3914183266779029169e-20" />
             <geometry>
-                <mesh filename="file://$(find rover_description)/base/meshes/fl_wheel.stl"/>
+                <mesh filename="file://$(find rover_description)/rover7/meshes/fl_wheel.stl"/>
             </geometry>
             <material name="fl_wheel_material">
@@ -204,5 +204,5 @@
             <origin xyz="-0.12415341931613714521 2.2204460492503130808e-16 -0.1250000000000002498" rpy="-1.570796326794896558 -0.13351607992219349796 -7.1088909477657821376e-17" />
             <geometry>
-                <mesh filename="file://$(find rover_description)/base/meshes/bl_ankle.stl"/>
+                <mesh filename="file://$(find rover_description)/rover7/meshes/bl_ankle.stl"/>
             </geometry>
             <material name="bl_ankle_material">
@@ -263,5 +263,5 @@
             <origin xyz="0 1.1102230246251565404e-16 1.7780915628762272718e-17" rpy="4.6040217445536182725e-17 1.0513492286565858337e-16 2.3412503191653332746e-19" />
             <geometry>
-                <mesh filename="file://$(find rover_description)/base/meshes/bl_wheel.stl"/>
+                <mesh filename="file://$(find rover_description)/rover7/meshes/bl_wheel.stl"/>
             </geometry>
             <material name="bl_wheel_material">
@@ -286,5 +286,5 @@
             <origin xyz="-7.9461177221465168975e-19 -7.2858385990954703269e-20 -0.020999999999999519051" rpy="3.141592653589793116 3.7838655819744092421e-17 -5.8406613147999892266e-19" />
             <geometry>
-                <mesh filename="file://$(find rover_description)/base/meshes/right_leg.stl"/>
+                <mesh filename="file://$(find rover_description)/rover7/meshes/right_leg.stl"/>
             </geometry>
             <material name="right_leg_material">
@@ -357,5 +357,5 @@
             <origin xyz="0.12415341931613695092 -2.2204460492503130808e-16 -0.12500000000000027756" rpy="-1.57079632679489678 0.13351607992219352572 9.9507186100571649487e-18" />
             <geometry>
-                <mesh filename="file://$(find rover_description)/base/meshes/fr_ankle.stl"/>
+                <mesh filename="file://$(find rover_description)/rover7/meshes/fr_ankle.stl"/>
             </geometry>
             <material name="fr_ankle_material">
@@ -416,5 +416,5 @@
             <origin xyz="5.5511151231257827021e-17 -1.1102230246251565404e-16 -3.0791341698588325926e-17" rpy="-3.6194812825998444115e-17 1.0511409763610977507e-16 -2.2325341479697011877e-19" />
             <geometry>
-                <mesh filename="file://$(find rover_description)/base/meshes/fr_wheel.stl"/>
+                <mesh filename="file://$(find rover_description)/rover7/meshes/fr_wheel.stl"/>
             </geometry>
             <material name="fr_wheel_material">
@@ -439,5 +439,5 @@
             <origin xyz="0.12415341931613720072 -2.2204460492503130808e-16 -0.12500000000000027756" rpy="-1.57079632679489678 0.13351607992219349796 -6.7670245197813334123e-17" />
             <geometry>
-                <mesh filename="file://$(find rover_description)/base/meshes/br_ankle.stl"/>
+                <mesh filename="file://$(find rover_description)/rover7/meshes/br_ankle.stl"/>
             </geometry>
             <material name="br_ankle_material">
@@ -498,5 +498,5 @@
             <origin xyz="5.5511151231257827021e-17 0 5.8763757748714340323e-17" rpy="1.4537948349788456791e-16 1.0501738044156386319e-16 -7.6074648532850333807e-21" />
             <geometry>
-                <mesh filename="file://$(find rover_description)/base/meshes/br_wheel.stl"/>
+                <mesh filename="file://$(find rover_description)/rover7/meshes/br_wheel.stl"/>
             </geometry>
             <material name="br_wheel_material">
@@ -521,5 +521,5 @@
             <origin xyz="4.9770590769729886024e-14 -0.00015426611885745872277 -0.010000000000000730527" rpy="1.570796326794896558 -3.0512890594788867116e-34 0" />
             <geometry>
-                <mesh filename="file://$(find rover_description)/base/meshes/diffbar.stl"/>
+                <mesh filename="file://$(find rover_description)/rover7/meshes/diffbar.stl"/>
             </geometry>
             <material name="diffbar_material">
@@ -550,5 +550,5 @@
             <origin xyz="-2.7755575615628913511e-15 -0.057750000000000162315 3.3306690738754696213e-16" rpy="1.5707963267948350516 -1.5127867282353739675 -3.1415926535897926719" />
             <geometry>
-                <mesh filename="file://$(find rover_description)/base/meshes/left_difflink.stl"/>
+                <mesh filename="file://$(find rover_description)/rover7/meshes/left_difflink.stl"/>
             </geometry>
             <material name="left_difflink_material">
@@ -573,5 +573,5 @@
             <origin xyz="6.2172489379008766264e-15 -0.057749999999999454547 -2.4424906541753443889e-15" rpy="1.5707963267948286123 1.512786629442331332 3.141592653589793116" />
             <geometry>
-                <mesh filename="file://$(find rover_description)/base/meshes/right_difflink.stl"/>
+                <mesh filename="file://$(find rover_description)/rover7/meshes/right_difflink.stl"/>
             </geometry>
             <material name="right_difflink_material">
@@ -687,7 +687,7 @@
     <!-- End of Generated URDF -->
     <!-- Include additional xacro files-->
-    <xacro:include filename="$(find rover_description)/base/urdf/ckc.xacro"/>
+    <xacro:include filename="$(find rover_description)/rover7/urdf/ckc.xacro"/>
     <xacro:if value="$(arg auto_camera)">
-        <xacro:include filename="$(find rover_description)/base/urdf/auto_camera.xacro"/>
+        <xacro:include filename="$(find rover_description)/rover7/urdf/auto_camera.xacro"/>
     </xacro:if>
     <xacro:if value="$(arg arm)">
@@ -701,13 +701,13 @@
     </xacro:if>
     <xacro:unless value="$(arg gazebo)">
-        <xacro:include filename="$(find rover_description)/base/urdf/ros2_control.xacro" />
+        <xacro:include filename="$(find rover_description)/rover7/urdf/ros2_control.xacro" />
         <xacro:rover_ros2_control use_mock_hardware="$(arg use_mock_hardware)"/>
     </xacro:unless>
     <xacro:if value="$(arg gazebo)">
-        <xacro:include filename="$(find rover_description)/base/urdf/gz_ros2_control.xacro" />
+        <xacro:include filename="$(find rover_description)/rover7/urdf/gz_ros2_control.xacro" />
     </xacro:if>
-    <xacro:include filename="$(find rover_description)/base/urdf/p3d.xacro"/>
-    <xacro:include filename="$(find rover_description)/base/urdf/odom.xacro"/>
-    <xacro:include filename="$(find rover_description)/base/urdf/gps.xacro"/>
-    <xacro:include filename="$(find rover_description)/base/urdf/joint_states.xacro"/>
+    <xacro:include filename="$(find rover_description)/rover7/urdf/p3d.xacro"/>
+    <xacro:include filename="$(find rover_description)/rover7/urdf/odom.xacro"/>
+    <xacro:include filename="$(find rover_description)/rover7/urdf/gps.xacro"/>
+    <xacro:include filename="$(find rover_description)/rover7/urdf/joint_states.xacro"/>
 </robot>
