Commit message: Merged master and relevant arm-urdf files

File: src/ros/rover/rover_description/arm/urdf/arm.urdf.xacro (robot description, xacro)
@@ -29,19 +29,19 @@
       <geometry>
         <mesh
-          filename="file://$(find rover_description)/arm/meshes/arm_base.stl" />
-      </geometry>
-      <material
-        name="">
-        <color
-          rgba="0.792156862745098 0.819607843137255 0.933333333333333 1" />
-      </material>
-    </visual>
-    <collision>
-      <origin
-        xyz="0 0 0"
-        rpy="0 0 0" />
-      <geometry>
-        <mesh
-          filename="file://$(find rover_description)/arm/meshes/arm_base.stl" />
+          filename="file://$(find rover_description)/meshes/arm_base.stl" />
+      </geometry>
+      <material
+        name="">
+        <color
+          rgba="0.792156862745098 0.819607843137255 0.933333333333333 1" />
+      </material>
+    </visual>
+    <collision>
+      <origin
+        xyz="0 0 0"
+        rpy="0 0 0" />
+      <geometry>
+        <mesh
+          filename="file://$(find rover_description)/meshes/arm_base.stl" />
       </geometry>
     </collision>
@@ -69,19 +69,19 @@
       <geometry>
         <mesh
-          filename="file://$(find rover_description)/arm/meshes/base_to_j1.stl" />
-      </geometry>
-      <material
-        name="">
-        <color
-          rgba="0.792156862745098 0.819607843137255 0.933333333333333 1" />
-      </material>
-    </visual>
-    <collision>
-      <origin
-        xyz="0 0 0"
-        rpy="0 0 0" />
-      <geometry>
-        <mesh
-          filename="file://$(find rover_description)/arm/meshes/base_to_j1.stl" />
+          filename="file://$(find rover_description)/meshes/base_to_j1.stl" />
+      </geometry>
+      <material
+        name="">
+        <color
+          rgba="0.792156862745098 0.819607843137255 0.933333333333333 1" />
+      </material>
+    </visual>
+    <collision>
+      <origin
+        xyz="0 0 0"
+        rpy="0 0 0" />
+      <geometry>
+        <mesh
+          filename="file://$(find rover_description)/meshes/base_to_j1.stl" />
       </geometry>
     </collision>
@@ -127,19 +127,19 @@
       <geometry>
         <mesh
-          filename="file://$(find rover_description)/arm/meshes/j2_to_link1.stl" />
-      </geometry>
-      <material
-        name="">
-        <color
-          rgba="0.792156862745098 0.819607843137255 0.933333333333333 1" />
-      </material>
-    </visual>
-    <collision>
-      <origin
-        xyz="0 0 0"
-        rpy="0 0 0" />
-      <geometry>
-        <mesh
-          filename="file://$(find rover_description)/arm/meshes/j2_to_link1.stl" />
+          filename="file://$(find rover_description)/meshes/j2_to_link1.stl" />
+      </geometry>
+      <material
+        name="">
+        <color
+          rgba="0.792156862745098 0.819607843137255 0.933333333333333 1" />
+      </material>
+    </visual>
+    <collision>
+      <origin
+        xyz="0 0 0"
+        rpy="0 0 0" />
+      <geometry>
+        <mesh
+          filename="file://$(find rover_description)/meshes/j2_to_link1.stl" />
       </geometry>
     </collision>
@@ -185,19 +185,19 @@
       <geometry>
         <mesh
-          filename="file://$(find rover_description)/arm/meshes/j3_to_link2.stl" />
-      </geometry>
-      <material
-        name="">
-        <color
-          rgba="0.792156862745098 0.819607843137255 0.933333333333333 1" />
-      </material>
-    </visual>
-    <collision>
-      <origin
-        xyz="0 0 0"
-        rpy="0 0 0" />
-      <geometry>
-        <mesh
-          filename="file://$(find rover_description)/arm/meshes/j3_to_link2.stl" />
+          filename="file://$(find rover_description)/meshes/j3_to_link2.stl" />
+      </geometry>
+      <material
+        name="">
+        <color
+          rgba="0.792156862745098 0.819607843137255 0.933333333333333 1" />
+      </material>
+    </visual>
+    <collision>
+      <origin
+        xyz="0 0 0"
+        rpy="0 0 0" />
+      <geometry>
+        <mesh
+          filename="file://$(find rover_description)/meshes/j3_to_link2.stl" />
       </geometry>
     </collision>
@@ -243,19 +243,19 @@
       <geometry>
         <mesh
-          filename="file://$(find rover_description)/arm/meshes/link2_to_fixed_j4.stl" />
-      </geometry>
-      <material
-        name="">
-        <color
-          rgba="0.792156862745098 0.819607843137255 0.933333333333333 1" />
-      </material>
-    </visual>
-    <collision>
-      <origin
-        xyz="0 0 0"
-        rpy="0 0 0" />
-      <geometry>
-        <mesh
-          filename="file://$(find rover_description)/arm/meshes/link2_to_fixed_j4.stl" />
+          filename="file://$(find rover_description)/meshes/link2_to_fixed_j4.stl" />
+      </geometry>
+      <material
+        name="">
+        <color
+          rgba="0.792156862745098 0.819607843137255 0.933333333333333 1" />
+      </material>
+    </visual>
+    <collision>
+      <origin
+        xyz="0 0 0"
+        rpy="0 0 0" />
+      <geometry>
+        <mesh
+          filename="file://$(find rover_description)/meshes/link2_to_fixed_j4.stl" />
       </geometry>
     </collision>
@@ -296,19 +296,19 @@
       <geometry>
         <mesh
-          filename="file://$(find rover_description)/arm/meshes/j4_to_j5.stl" />
-      </geometry>
-      <material
-        name="">
-        <color
-          rgba="0.792156862745098 0.819607843137255 0.933333333333333 1" />
-      </material>
-    </visual>
-    <collision>
-      <origin
-        xyz="0 0 0"
-        rpy="0 0 0" />
-      <geometry>
-        <mesh
-          filename="file://$(find rover_description)/arm/meshes/j4_to_j5.stl" />
+          filename="file://$(find rover_description)/meshes/j4_to_j5.stl" />
+      </geometry>
+      <material
+        name="">
+        <color
+          rgba="0.792156862745098 0.819607843137255 0.933333333333333 1" />
+      </material>
+    </visual>
+    <collision>
+      <origin
+        xyz="0 0 0"
+        rpy="0 0 0" />
+      <geometry>
+        <mesh
+          filename="file://$(find rover_description)/meshes/j4_to_j5.stl" />
       </geometry>
     </collision>
@@ -354,19 +354,19 @@
       <geometry>
         <mesh
-          filename="file://$(find rover_description)/arm/meshes/j5_to_j6.stl" />
-      </geometry>
-      <material
-        name="">
-        <color
-          rgba="0.792156862745098 0.819607843137255 0.933333333333333 1" />
-      </material>
-    </visual>
-    <collision>
-      <origin
-        xyz="0 0 0"
-        rpy="0 0 0" />
-      <geometry>
-        <mesh
-          filename="file://$(find rover_description)/arm/meshes/j5_to_j6.stl" />
+          filename="file://$(find rover_description)/meshes/j5_to_j6.stl" />
+      </geometry>
+      <material
+        name="">
+        <color
+          rgba="0.792156862745098 0.819607843137255 0.933333333333333 1" />
+      </material>
+    </visual>
+    <collision>
+      <origin
+        xyz="0 0 0"
+        rpy="0 0 0" />
+      <geometry>
+        <mesh
+          filename="file://$(find rover_description)/meshes/j5_to_j6.stl" />
       </geometry>
     </collision>
@@ -412,19 +412,19 @@
       <geometry>
         <mesh
-          filename="file://$(find rover_description)/arm/meshes/j6_to_ee.stl" />
-      </geometry>
-      <material
-        name="">
-        <color
-          rgba="0.792156862745098 0.819607843137255 0.933333333333333 1" />
-      </material>
-    </visual>
-    <collision>
-      <origin
-        xyz="0 0 0"
-        rpy="0 0 0" />
-      <geometry>
-        <mesh
-          filename="file://$(find rover_description)/arm/meshes/j6_to_ee.stl" />
+          filename="file://$(find rover_description)/meshes/j6_to_ee.stl" />
+      </geometry>
+      <material
+        name="">
+        <color
+          rgba="0.792156862745098 0.819607843137255 0.933333333333333 1" />
+      </material>
+    </visual>
+    <collision>
+      <origin
+        xyz="0 0 0"
+        rpy="0 0 0" />
+      <geometry>
+        <mesh
+          filename="file://$(find rover_description)/meshes/j6_to_ee.stl" />
       </geometry>
     </collision>
@@ -448,3 +448,6 @@
       velocity="0" />
   </joint>
+  <!-- gazebo bridge joints -->
+  <xacro:include filename="$(find rover_description)/arm/urdf/arm_joints.xacro"/>
+  <xacro:include filename="$(find rover_description)/arm/urdf/arm_odom.xacro"/>
 </robot>

File: src/ros/rover/rover_description/rover7/urdf/rover.urdf.xacro (robot description, xacro)
@@ -692,12 +692,18 @@
     </xacro:if>
     <xacro:if value="$(arg arm)">
-        <!-- Needs to be updated for new arm-->
-        <xacro:include filename="$(find rover_description)/arm/urdf/arm.urdf.xacro" />
-        <joint name="chassis_to_arm_base" type="fixed">
-            <origin xyz="0 0.15 -0.06" rpy="0 0 1.57"/>
+        <xacro:include filename="$(find rover_description)/arm/urdf/newarm.urdf.xacro" />
+        <joint name="J1_gbp_chassis" type="revolute">
+            <origin xyz="0.22899999999999565148 1.1102230246251564172e-16 0.11707476398169122667" rpy="-3.141592653589793116 -1.3309679851047901909e-16 0" />
             <parent link="chassis" />
-            <child link="arm_link" />
+            <child link="gearbox" />
+            <axis xyz="0 0 1"/>
+            <limit effort="20" velocity="20" lower="-3.141592653589793116" upper="3.141592653589793116"/>
+            <joint_properties friction="0.3"/>
         </joint>
+        <xacro:include filename="$(find rover_description)/arm/urdf/dynamic_joints_with_arm.xacro"/>
     </xacro:if>
+    <xacro:unless value="$(arg arm)">
+        <xacro:include filename="$(find rover_description)/rover7/urdf/joint_states.xacro"/>
+    </xacro:unless>
     <xacro:unless value="$(arg gazebo)">
         <xacro:include filename="$(find rover_description)/rover7/urdf/ros2_control.xacro" />
@@ -710,4 +716,3 @@
     <xacro:include filename="$(find rover_description)/rover7/urdf/odom.xacro"/>
     <xacro:include filename="$(find rover_description)/rover7/urdf/gps.xacro"/>
-    <xacro:include filename="$(find rover_description)/rover7/urdf/joint_states.xacro"/>
 </robot>
