Commit message: fixes to ros2 control arm done at workshop

File: src/ros/rover/rover_description/arm/urdf/newarm_joints.xacro (robot description, xacro)
@@ -5,13 +5,13 @@
           <plugin filename="gz-sim-joint-state-publisher-system" name="gz::sim::systems::JointStatePublisher">
                <topic>arm_joints</topic>
-               <joint_name>J1_gbp_chassis</joint_name>
-               <joint_name>J2_l1a_bp</joint_name>
-               <joint_name>J3_l2b_bp</joint_name>
+               <joint_name>j1</joint_name>
+               <joint_name>j2</joint_name>
+               <joint_name>j3</joint_name>
                <joint_name>l1b_bp</joint_name>
                <joint_name>l1b_tp</joint_name>
                <joint_name>l1a_tp</joint_name>
-               <joint_name>wrist_pitch</joint_name>
-               <joint_name>wrist_yaw</joint_name>
-               <joint_name>wrist_roll</joint_name>
+               <joint_name>j4</joint_name>
+               <joint_name>j5</joint_name>
+               <joint_name>j6</joint_name>
                <joint_name>rf_slide</joint_name>
                <joint_name>lf_slide</joint_name>

File: src/ros/rover/rover_description/rover7/urdf/rover.urdf.xacro (robot description, xacro)
@@ -693,5 +693,5 @@
     <xacro:if value="$(arg arm)">
         <xacro:include filename="$(find rover_description)/arm/urdf/newarm.urdf.xacro" />
-        <joint name="J1_gbp_chassis" type="revolute">
+        <joint name="j1" type="revolute">
             <origin xyz="0.22899999999999565148 1.1102230246251564172e-16 0.11707476398169122667" rpy="-3.141592653589793116 -1.3309679851047901909e-16 0" />
             <parent link="chassis" />
