Commit message: fix merge conflicts

File: src/ros/rover/rover_description/arm/urdf/newarm.gz_ros2_control.xacro (robot description, xacro)
@@ -1,5 +1,5 @@
 <?xml version="1.0" encoding="utf-8"?>
 <robot xmlns:xacro="http://www.ros.org/wiki/xacro">
-  <ros2_control name="GazeboSimSystem" type="system">
+  <ros2_control name="GazeboSimSystemArm" type="system">
     <hardware>
       <plugin>gz_ros2_control/GazeboSimSystem</plugin>
@@ -138,8 +138,8 @@
       </joint>
   </ros2_control>
-  <!-- <gazebo>
+  <gazebo>
     <plugin filename="gz_ros2_control-system" name="gz_ros2_control::GazeboSimROS2ControlPlugin">
       <parameters>$(find auto_bringup)/params/controllers.yaml</parameters>
     </plugin>
-  </gazebo> -->
+  </gazebo>
 </robot>

File: src/ros/rover/rover_description/arm/urdf/newarm.ros2_control.xacro (robot description, xacro)
@@ -4,10 +4,10 @@
   <!-- Initial definition based on https://github.com/xArm-Developer/xarm_ros2/blob/master/xarm_description/urdf/xarm6/xarm6.ros2_control.xacro -->
   <xacro:macro name="newarm_ros2_control" params="use_mock_hardware">
-    <ros2_control name="J1" type="system">
+    <ros2_control name="arm" type="system">
 	  <xacro:unless value="${use_mock_hardware}">
         <hardware>
 		  <plugin>blcmd_hardware/BLCMDHardware</plugin>
 		  <param name="candevice">can1</param>
-      <param name="canid">4</param>
+      	  <param name="canid">4</param>
 		  <param name="resolver_reduction">1.33333333333</param>
 		  <param name="clock_rate">100000000</param>
@@ -26,7 +26,4 @@
         </hardware>
 	  </xacro:if>
-<<<<<<< Updated upstream
-	  <joint name="J1_gbp_chassis">
-=======
 	  <!--
 	  <hardware>
@@ -47,9 +44,5 @@
       </joint>
 	  <joint name="j2">
->>>>>>> Stashed changes
 		<command_interface name="velocity">
-		  <param name="max">1</param>
-		</command_interface>
-		<command_interface name="effort">
 		  <param name="max">1</param>
 		</command_interface>
@@ -61,36 +54,6 @@
 		</state_interface>
       </joint>
-<<<<<<< Updated upstream
-    </ros2_control>
-    <ros2_control name="J2" type="system">
-	  <xacro:unless value="${use_mock_hardware}">
-        <hardware>
-		  <plugin>blcmd_hardware/BLCMDHardware</plugin>
-		  <param name="candevice">can1</param>
-      <param name="canid">8</param>
-		  <param name="resolver_reduction">1.33333333333</param>
-		  <param name="clock_rate">100000000</param>
-		  <param name="revolution_pulses">8192</param>
-		  <param name="min_interval">122</param>
-		  <param name="gear_ratio">36.0</param>
-		  <param name="mock">true</param>
-		  <param name="reversed">true</param>
-		  <param name="integrate_velocity">true</param>
-        </hardware>
-      </xacro:unless>
-      <xacro:if value="${use_mock_hardware}">
-        <hardware>
-          <plugin>mock_components/GenericSystem</plugin>
-          <param name="calculate_dynamics">true</param>
-        </hardware>
-	  </xacro:if>
-	  <joint name="J2_l1a_bp">
-=======
 	  <joint name="j3">
->>>>>>> Stashed changes
 		<command_interface name="velocity">
-		  <param name="max">1</param>
-		</command_interface>
-		<command_interface name="effort">
 		  <param name="max">1</param>
 		</command_interface>
@@ -102,71 +65,6 @@
 		</state_interface>
       </joint>
-<<<<<<< Updated upstream
-    </ros2_control>
-    <ros2_control name="J3" type="system">
-	  <xacro:unless value="${use_mock_hardware}">
-        <hardware>
-		  <plugin>blcmd_hardware/BLCMDHardware</plugin>
-		  <param name="candevice">can1</param>
-      <param name="canid">12</param> <!-- XXX -->
-		  <param name="resolver_reduction">1.33333333333</param>
-		  <param name="clock_rate">100000000</param>
-		  <param name="revolution_pulses">8192</param>
-		  <param name="min_interval">122</param>
-		  <param name="gear_ratio">36.0</param>
-		  <param name="mock">true</param>
-		  <param name="reversed">true</param>
-		  <param name="integrate_velocity">true</param>
-        </hardware>
-      </xacro:unless>
-      <xacro:if value="${use_mock_hardware}">
-        <hardware>
-          <plugin>mock_components/GenericSystem</plugin>
-          <param name="calculate_dynamics">true</param>
-        </hardware>
-	  </xacro:if>
-	  <joint name="J3_l2b_bp">
-		<command_interface name="velocity">
-		  <param name="max">1</param>
-		</command_interface>
-		<command_interface name="effort">
-		  <param name="max">1</param>
-		</command_interface>
-		<state_interface name="velocity">
-		  <param name="initial_value">0.0</param>
-		</state_interface>
-		<state_interface name="position">
-		  <param name="initial_value">0.0</param>
-		</state_interface>
-      </joint>
-    </ros2_control>
-    <ros2_control name="J4" type="system">
-	  <xacro:unless value="${use_mock_hardware}">
-        <hardware>
-		  <plugin>blcmd_hardware/BLCMDHardware</plugin>
-		  <param name="candevice">can1</param>
-      <param name="canid">16</param> <!-- XXX -->
-		  <param name="resolver_reduction">1.33333333333</param>
-		  <param name="clock_rate">100000000</param>
-		  <param name="revolution_pulses">8192</param>
-		  <param name="min_interval">122</param>
-		  <param name="gear_ratio">36.0</param>
-		  <param name="mock">true</param>
-		  <param name="reversed">true</param>
-		  <param name="integrate_velocity">true</param>
-        </hardware>
-      </xacro:unless>
-      <xacro:if value="${use_mock_hardware}">
-        <hardware>
-          <plugin>mock_components/GenericSystem</plugin>
-          <param name="calculate_dynamics">true</param>
-        </hardware>
-	  </xacro:if>
-=======
 	  <!-- <joint name="l1b_bp">
 		<command_interface name="velocity">
-		  <param name="max">1</param>
-		</command_interface>
-		<command_interface name="effort">
 		  <param name="max">1</param>
 		</command_interface>
@@ -182,7 +80,4 @@
 		  <param name="max">1</param>
 		</command_interface>
-		<command_interface name="effort">
-		  <param name="max">1</param>
-		</command_interface>
 		<state_interface name="velocity">
 		  <param name="initial_value">0.0</param>
@@ -196,7 +91,4 @@
 		  <param name="max">1</param>
 		</command_interface>
-		<command_interface name="effort">
-		  <param name="max">1</param>
-		</command_interface>
 		<state_interface name="velocity">
 		  <param name="initial_value">0.0</param>
@@ -206,10 +98,6 @@
 		</state_interface>
       </joint> -->
->>>>>>> Stashed changes
 	  <joint name="j4">
 		<command_interface name="velocity">
-		  <param name="max">1</param>
-		</command_interface>
-		<command_interface name="effort">
 		  <param name="max">1</param>
 		</command_interface>
@@ -221,36 +109,6 @@
 		</state_interface>
       </joint>
-<<<<<<< Updated upstream
-    </ros2_control>
-    <ros2_control name="J5" type="system">
-	  <xacro:unless value="${use_mock_hardware}">
-        <hardware>
-		  <plugin>blcmd_hardware/BLCMDHardware</plugin>
-		  <param name="candevice">can1</param>
-      <param name="canid">20</param> <!-- XXX -->
-		  <param name="resolver_reduction">1.33333333333</param>
-		  <param name="clock_rate">100000000</param>
-		  <param name="revolution_pulses">8192</param>
-		  <param name="min_interval">122</param>
-		  <param name="gear_ratio">36.0</param>
-		  <param name="mock">true</param>
-		  <param name="reversed">true</param>
-		  <param name="integrate_velocity">true</param>
-        </hardware>
-      </xacro:unless>
-      <xacro:if value="${use_mock_hardware}">
-        <hardware>
-          <plugin>mock_components/GenericSystem</plugin>
-          <param name="calculate_dynamics">true</param>
-        </hardware>
-	  </xacro:if>
-	  <joint name="wrist_yaw">
-=======
 	  <joint name="j5">
->>>>>>> Stashed changes
 		<command_interface name="velocity">
-		  <param name="max">1</param>
-		</command_interface>
-		<command_interface name="effort">
 		  <param name="max">1</param>
 		</command_interface>
@@ -262,36 +120,6 @@
 		</state_interface>
       </joint>
-<<<<<<< Updated upstream
-    </ros2_control>
-    <ros2_control name="J6" type="system">
-	  <xacro:unless value="${use_mock_hardware}">
-        <hardware>
-		  <plugin>blcmd_hardware/BLCMDHardware</plugin>
-		  <param name="candevice">can1</param>
-      <param name="canid">24</param> <!-- XXX  not too sure about this, might need to be hexadecimal-->
-		  <param name="resolver_reduction">1.33333333333</param>
-		  <param name="clock_rate">100000000</param>
-		  <param name="revolution_pulses">8192</param>
-		  <param name="min_interval">122</param>
-		  <param name="gear_ratio">36.0</param>
-		  <param name="mock">true</param>
-		  <param name="reversed">true</param>
-		  <param name="integrate_velocity">true</param>
-        </hardware>
-      </xacro:unless>
-      <xacro:if value="${use_mock_hardware}">
-        <hardware>
-          <plugin>mock_components/GenericSystem</plugin>
-          <param name="calculate_dynamics">true</param>
-        </hardware>
-	  </xacro:if>
-	  <joint name="wrist_roll">
-=======
 	  <joint name="j6">
->>>>>>> Stashed changes
 		<command_interface name="velocity">
-		  <param name="max">1</param>
-		</command_interface>
-		<command_interface name="effort">
 		  <param name="max">1</param>
 		</command_interface>
@@ -309,7 +137,4 @@
 		  <param name="max">1</param>
 		</command_interface>
-		<command_interface name="effort">
-		  <param name="max">1</param>
-		</command_interface>
 		<state_interface name="velocity">
 		  <param name="initial_value">0.0</param>
@@ -321,7 +146,4 @@
 	  <joint name="lf_slide">
 		<command_interface name="velocity">
-		  <param name="max">1</param>
-		</command_interface>
-		<command_interface name="effort">
 		  <param name="max">1</param>
 		</command_interface>
@@ -337,7 +159,4 @@
 		  <param name="max">1</param>
 		</command_interface>
-		<command_interface name="effort">
-		  <param name="max">1</param>
-		</command_interface>
 		<state_interface name="velocity">
 		  <param name="initial_value">0.0</param>

File: src/ros/rover/rover_description/arm/urdf/newarm.urdf.xacro (robot description, xacro)
@@ -565,7 +565,4 @@
     </gazebo>
     <!--xacro:include filename="arm_odom.xacro"/ -->
-<<<<<<< Updated upstream
-    <xacro:if value="$(arg gazebo)">
-=======
     <!-- <xacro:if value="$(arg gazebo)">
         <xacro:include filename="$(find rover_description)/arm/urdf/newarm.ros2_control.xacro" />
@@ -584,5 +581,4 @@
         <xacro:include filename="$(find rover_description)/arm/urdf/newarm.gz_ros2_control.xacro" />
         <!-- hahah gazebo end -->
->>>>>>> Stashed changes
     </xacro:if>
     <!-- XXX: ask why this isn't enabled for not gazebo -->

Commit message: fixes: bunch of changes to fix up arm-master including commenting out the IK controller

File: src/ros/rover/rover_description/arm/urdf/newarm.gz_ros2_control.xacro (robot description, xacro)
@@ -5,5 +5,5 @@
       <plugin>gz_ros2_control/GazeboSimSystem</plugin>
     </hardware>
-    <joint name="j1">
+    <joint name="J1">
 		<command_interface name="velocity">
 		  <param name="max">1</param>
@@ -16,5 +16,5 @@
 		</state_interface>
       </joint>
-	  <joint name="j2">
+	  <joint name="J2">
 		<command_interface name="velocity">
 		  <param name="max">1</param>
@@ -27,5 +27,5 @@
 		</state_interface>
       </joint>
-	  <joint name="j3">
+	  <joint name="J3">
 		<command_interface name="velocity">
 		  <param name="max">1</param>
@@ -71,5 +71,5 @@
 		</state_interface>
       </joint> -->
-	  <joint name="j4">
+	  <joint name="J4">
 		<command_interface name="velocity">
 		  <param name="max">1</param>
@@ -82,5 +82,5 @@
 		</state_interface>
       </joint>
-	  <joint name="j5">
+	  <joint name="J5">
 		<command_interface name="velocity">
 		  <param name="max">1</param>
@@ -93,5 +93,5 @@
 		</state_interface>
       </joint>
-	  <joint name="j6">
+	  <joint name="J6">
 		<command_interface name="velocity">
 		  <param name="max">1</param>

File: src/ros/rover/rover_description/arm/urdf/newarm.urdf.xacro (robot description, xacro)
@@ -560,5 +560,5 @@
     <!-- End of Generated URDF -->
     <!-- Close ckc -->
-    <xacro:include filename="newarm_ckc.xacro"/>
+    <!-- <xacro:include filename="newarm_ckc.xacro"/> -->
     <!-- gazebo parameters-->
     <gazebo>

Commit message: fix: removed capitalisation from joint j's

File: src/ros/rover/rover_description/arm/urdf/newarm.gz_ros2_control.xacro (robot description, xacro)
@@ -5,5 +5,5 @@
       <plugin>gz_ros2_control/GazeboSimSystem</plugin>
     </hardware>
-    <joint name="J1">
+    <joint name="j1">
 		<command_interface name="velocity">
 		  <param name="max">1</param>
@@ -16,5 +16,5 @@
 		</state_interface>
       </joint>
-	  <joint name="J2">
+	  <joint name="j2">
 		<command_interface name="velocity">
 		  <param name="max">1</param>
@@ -27,5 +27,5 @@
 		</state_interface>
       </joint>
-	  <joint name="J3">
+	  <joint name="j3">
 		<command_interface name="velocity">
 		  <param name="max">1</param>
@@ -71,5 +71,5 @@
 		</state_interface>
       </joint> -->
-	  <joint name="J4">
+	  <joint name="j4">
 		<command_interface name="velocity">
 		  <param name="max">1</param>
@@ -82,5 +82,5 @@
 		</state_interface>
       </joint>
-	  <joint name="J5">
+	  <joint name="j5">
 		<command_interface name="velocity">
 		  <param name="max">1</param>
@@ -93,5 +93,5 @@
 		</state_interface>
       </joint>
-	  <joint name="J6">
+	  <joint name="j6">
 		<command_interface name="velocity">
 		  <param name="max">1</param>
