Commit message: MVP nova ik controller (#225)
Co-authored-by: arbabf <arbab.fahm@gmail.com>
Co-authored-by: Monash Nova Rover <novaroverteam@monash.edu>
Co-authored-by: RohitPilakkat <rohit.pilakkat@gmail.com>

File: src/ros/rover/rover_description/arm/urdf/newarm.gz_ros2_control.xacro (robot description, xacro)
@@ -8,4 +8,6 @@
 		<command_interface name="velocity">
 		  <param name="max">1</param>
+		</command_interface>
+		<command_interface name="position">
 		</command_interface>
 		<state_interface name="velocity">
@@ -20,4 +22,6 @@
 		  <param name="max">1</param>
 		</command_interface>
+		<command_interface name="position">
+		</command_interface>
 		<state_interface name="velocity">
 		  <param name="initial_value">0.0</param>
@@ -30,4 +34,6 @@
 		<command_interface name="velocity">
 		  <param name="max">1</param>
+		</command_interface>
+		<command_interface name="position">
 		</command_interface>
 		<state_interface name="velocity">
@@ -75,4 +81,6 @@
 		  <param name="max">1</param>
 		</command_interface>
+		<command_interface name="position">
+		</command_interface>
 		<state_interface name="velocity">
 		  <param name="initial_value">0.0</param>
@@ -85,4 +93,6 @@
 		<command_interface name="velocity">
 		  <param name="max">1</param>
+		</command_interface>
+		<command_interface name="position">
 		</command_interface>
 		<state_interface name="velocity">
@@ -97,4 +107,6 @@
 		  <param name="max">1</param>
 		</command_interface>
+		<command_interface name="position">
+		</command_interface>
 		<state_interface name="velocity">
 		  <param name="initial_value">0.0</param>
@@ -107,4 +119,6 @@
 		<command_interface name="velocity">
 		  <param name="max">1</param>
+		</command_interface>
+		<command_interface name="position">
 		</command_interface>
 		<state_interface name="velocity">
@@ -119,4 +133,6 @@
 		  <param name="max">1</param>
 		</command_interface>
+		<command_interface name="position">
+		</command_interface>
 		<state_interface name="velocity">
 		  <param name="initial_value">0.0</param>
@@ -129,4 +145,6 @@
 		<command_interface name="velocity">
 		  <param name="max">1</param>
+		</command_interface>
+		<command_interface name="position">
 		</command_interface>
 		<state_interface name="velocity">

File: src/ros/rover/rover_description/arm/urdf/newarm.ros2_control.xacro (robot description, xacro)
@@ -1,30 +1,30 @@
 <?xml version="1.0" encoding="utf-8"?>
 <robot xmlns:xacro="http://www.ros.org/wiki/xacro">
-  <!-- Test trying to make a ros2_control URDF for the new arm -->
-  <!-- Initial definition based on https://github.com/xArm-Developer/xarm_ros2/blob/master/xarm_description/urdf/xarm6/xarm6.ros2_control.xacro -->
-  <xacro:macro name="newarm_ros2_control" params="use_mock_hardware">
-    <ros2_control name="arm_J1" type="system">
-	  <xacro:unless value="${use_mock_hardware}">
-        <hardware>
-		  <plugin>blcmd_hardware/BLCMDHardware</plugin>
-		  <param name="candevice">can1</param>
-      	  <param name="canid">4F1</param>
-		  <param name="resolver_reduction">1.33333333333</param>
-		  <param name="clock_rate">100000000</param>
-		  <param name="revolution_pulses">8192</param>
-		  <param name="min_interval">122</param>
-		  <param name="gear_ratio">36.0</param>
-		  <param name="mock">true</param>
-		  <param name="reversed">true</param>
-		  <param name="integrate_velocity">true</param>
-        </hardware>
-      </xacro:unless>
-      <xacro:if value="${use_mock_hardware}">
-        <hardware>
-          <plugin>mock_components/GenericSystem</plugin>
-          <param name="calculate_dynamics">true</param>
-        </hardware>
-	  </xacro:if>
-	  <!--
+	<!-- Test trying to make a ros2_control URDF for the new arm -->
+	<!-- Initial definition based on https://github.com/xArm-Developer/xarm_ros2/blob/master/xarm_description/urdf/xarm6/xarm6.ros2_control.xacro -->
+	<xacro:macro name="newarm_ros2_control" params="use_mock_hardware">
+		<ros2_control name="arm_J1" type="system">
+			<xacro:unless value="${use_mock_hardware}">
+				<hardware>
+					<plugin>blcmd_hardware/BLCMDHardware</plugin>
+					<param name="candevice">can1</param>
+					<param name="canid">4F1</param>
+					<param name="resolver_reduction">1.33333333333</param>
+					<param name="clock_rate">100000000</param>
+					<param name="revolution_pulses">8192</param>
+					<param name="min_interval">122</param>
+					<param name="gear_ratio">36.0</param>
+					<param name="mock">true</param>
+					<param name="reversed">true</param>
+					<param name="integrate_velocity">true</param>
+				</hardware>
+			</xacro:unless>
+			<xacro:if value="${use_mock_hardware}">
+				<hardware>
+					<plugin>mock_components/GenericSystem</plugin>
+					<param name="calculate_dynamics">true</param>
+				</hardware>
+			</xacro:if>
+			<!--
 	  <hardware>
         TODO: Figure out and add the Hardware interface
@@ -32,187 +32,163 @@
 	  </hardware>
 	  -->
-	  <joint name="J1">
-		<command_interface name="velocity">
-		  <param name="max">1</param>
-		</command_interface>
-		<state_interface name="velocity">
-		  <param name="initial_value">0.0</param>
-		</state_interface>
-		<state_interface name="position">
-		  <param name="initial_value">0.0</param>
-		</state_interface>
-      </joint>
-	</ros2_control>
-	<ros2_control name="arm_J2" type="system">
-	  <xacro:unless value="${use_mock_hardware}">
-        <hardware>
-		  <plugin>blcmd_hardware/BLCMDHardware</plugin>
-		  <param name="candevice">can1</param>
-      	  <param name="canid">4F1</param>
-		  <param name="resolver_reduction">1.33333333333</param>
-		  <param name="clock_rate">100000000</param>
-		  <param name="revolution_pulses">8192</param>
-		  <param name="min_interval">122</param>
-		  <param name="gear_ratio">36.0</param>
-		  <param name="mock">true</param>
-		  <param name="reversed">true</param>
-		  <param name="integrate_velocity">true</param>
-        </hardware>
-      </xacro:unless>
-      <xacro:if value="${use_mock_hardware}">
-        <hardware>
-          <plugin>mock_components/GenericSystem</plugin>
-          <param name="calculate_dynamics">true</param>
-        </hardware>
-	  </xacro:if>
-	  <joint name="J2">
-		<command_interface name="velocity">
-		  <param name="max">1</param>
-		</command_interface>
-		<state_interface name="velocity">
-		  <param name="initial_value">0.0</param>
-		</state_interface>
-		<state_interface name="position">
-		  <param name="initial_value">0.0</param>
-		</state_interface>
-      </joint>
-	</ros2_control>
-	<ros2_control name="arm_J3" type="system">
-	  <xacro:unless value="${use_mock_hardware}">
-        <hardware>
-		  <plugin>blcmd_hardware/BLCMDHardware</plugin>
-		  <param name="candevice">can1</param>
-      	  <param name="canid">4F1</param>
-		  <param name="resolver_reduction">1.33333333333</param>
-		  <param name="clock_rate">100000000</param>
-		  <param name="revolution_pulses">8192</param>
-		  <param name="min_interval">122</param>
-		  <param name="gear_ratio">36.0</param>
-		  <param name="mock">true</param>
-		  <param name="reversed">true</param>
-		  <param name="integrate_velocity">true</param>
-        </hardware>
-      </xacro:unless>
-      <xacro:if value="${use_mock_hardware}">
-        <hardware>
-          <plugin>mock_components/GenericSystem</plugin>
-          <param name="calculate_dynamics">true</param>
-        </hardware>
-	  </xacro:if>
-	  <joint name="J3">
-		<command_interface name="velocity">
-		  <param name="max">1</param>
-		</command_interface>
-		<state_interface name="velocity">
-		  <param name="initial_value">0.0</param>
-		</state_interface>
-		<state_interface name="position">
-		  <param name="initial_value">0.0</param>
-		</state_interface>
-      </joint>
-	</ros2_control>
-	<ros2_control name="arm_J4" type="system">
-	  <xacro:unless value="${use_mock_hardware}">
-        <hardware>
-		  <plugin>blcmd_hardware/BLCMDHardware</plugin>
-		  <param name="candevice">can1</param>
-      	  <param name="canid">4F1</param>
-		  <param name="resolver_reduction">1.33333333333</param>
-		  <param name="clock_rate">100000000</param>
-		  <param name="revolution_pulses">8192</param>
-		  <param name="min_interval">122</param>
-		  <param name="gear_ratio">36.0</param>
-		  <param name="mock">true</param>
-		  <param name="reversed">true</param>
-		  <param name="integrate_velocity">true</param>
-        </hardware>
-      </xacro:unless>
-      <xacro:if value="${use_mock_hardware}">
-        <hardware>
-          <plugin>mock_components/GenericSystem</plugin>
-          <param name="calculate_dynamics">true</param>
-        </hardware>
-	  </xacro:if>
-	  <joint name="J4">
-		<command_interface name="velocity">
-		  <param name="max">1</param>
-		</command_interface>
-		<state_interface name="velocity">
-		  <param name="initial_value">0.0</param>
-		</state_interface>
-		<state_interface name="position">
-		  <param name="initial_value">0.0</param>
-		</state_interface>
-      </joint>
-	</ros2_control>
-	<ros2_control name="arm_J6" type="system">
-	  <xacro:unless value="${use_mock_hardware}">
-        <hardware>
-		  <plugin>blcmd_hardware/BLCMDHardware</plugin>
-		  <param name="candevice">can1</param>
-      	  <param name="canid">4F1</param>
-		  <param name="resolver_reduction">1.33333333333</param>
-		  <param name="clock_rate">100000000</param>
-		  <param name="revolution_pulses">8192</param>
-		  <param name="min_interval">122</param>
-		  <param name="gear_ratio">36.0</param>
-		  <param name="mock">true</param>
-		  <param name="reversed">true</param>
-		  <param name="integrate_velocity">true</param>
-        </hardware>
-      </xacro:unless>
-      <xacro:if value="${use_mock_hardware}">
-        <hardware>
-          <plugin>mock_components/GenericSystem</plugin>
-          <param name="calculate_dynamics">true</param>
-        </hardware>
-	  </xacro:if>
-	  <joint name="J6">
-		<command_interface name="velocity">
-		  <param name="max">1</param>
-		</command_interface>
-		<state_interface name="velocity">
-		  <param name="initial_value">0.0</param>
-		</state_interface>
-		<state_interface name="position">
-		  <param name="initial_value">0.0</param>
-		</state_interface>
-      </joint>
-	</ros2_control>
-	<ros2_control name="arm_J6" type="system">
-	  <xacro:unless value="${use_mock_hardware}">
-        <hardware>
-		  <plugin>blcmd_hardware/BLCMDHardware</plugin>
-		  <param name="candevice">can0</param>
-      	  <param name="canid">5</param>
-		  <param name="resolver_reduction">1.33333333333</param>
-		  <param name="clock_rate">100000000</param>
-		  <param name="revolution_pulses">8192</param>
-		  <param name="min_interval">122</param>
-		  <param name="gear_ratio">36.0</param>
-		  <param name="mock">true</param>
-		  <param name="reversed">true</param>
-		  <param name="integrate_velocity">true</param>
-        </hardware>
-      </xacro:unless>
-      <xacro:if value="${use_mock_hardware}">
-        <hardware>
-          <plugin>mock_components/GenericSystem</plugin>
-          <param name="calculate_dynamics">true</param>
-        </hardware>
-	  </xacro:if>
-	  <joint name="J6">
-		<command_interface name="velocity">
-		  <param name="max">1</param>
-		</command_interface>
-		<state_interface name="velocity">
-		  <param name="initial_value">0.0</param>
-		</state_interface>
-		<state_interface name="position">
-		  <param name="initial_value">0.0</param>
-		</state_interface>
-      </joint>
-    </ros2_control>
-        <!--
+			<joint name="J1">
+				<command_interface name="velocity">
+					<param name="max">1</param>
+				</command_interface>
+				<command_interface name="position">
+				</command_interface>
+			</joint>
+		</ros2_control>
+		<ros2_control name="arm_J2" type="system">
+			<xacro:unless value="${use_mock_hardware}">
+				<hardware>
+					<plugin>blcmd_hardware/BLCMDHardware</plugin>
+					<param name="candevice">can1</param>
+					<param name="canid">4F2</param>
+					<param name="resolver_reduction">1.33333333333</param>
+					<param name="clock_rate">100000000</param>
+					<param name="revolution_pulses">8192</param>
+					<param name="min_interval">122</param>
+					<param name="gear_ratio">36.0</param>
+					<param name="mock">true</param>
+					<param name="reversed">true</param>
+					<param name="integrate_velocity">true</param>
+				</hardware>
+			</xacro:unless>
+			<xacro:if value="${use_mock_hardware}">
+				<hardware>
+					<plugin>mock_components/GenericSystem</plugin>
+					<param name="calculate_dynamics">true</param>
+				</hardware>
+			</xacro:if>
+			<joint name="J2">
+				<command_interface name="velocity">
+					<param name="max">1</param>
+				</command_interface>
+				<command_interface name="position">
+				</command_interface>
+			</joint>
+		</ros2_control>
+		<ros2_control name="arm_J3" type="system">
+			<xacro:unless value="${use_mock_hardware}">
+				<hardware>
+					<plugin>blcmd_hardware/BLCMDHardware</plugin>
+					<param name="candevice">can1</param>
+					<param name="canid">4F3</param>
+					<param name="resolver_reduction">1.33333333333</param>
+					<param name="clock_rate">100000000</param>
+					<param name="revolution_pulses">8192</param>
+					<param name="min_interval">122</param>
+					<param name="gear_ratio">36.0</param>
+					<param name="mock">true</param>
+					<param name="reversed">true</param>
+					<param name="integrate_velocity">true</param>
+				</hardware>
+			</xacro:unless>
+			<xacro:if value="${use_mock_hardware}">
+				<hardware>
+					<plugin>mock_components/GenericSystem</plugin>
+					<param name="calculate_dynamics">true</param>
+				</hardware>
+			</xacro:if>
+			<joint name="J3">
+				<command_interface name="velocity">
+					<param name="max">1</param>
+				</command_interface>
+				<command_interface name="position">
+				</command_interface>
+			</joint>
+		</ros2_control>
+		<ros2_control name="arm_J4" type="system">
+			<xacro:unless value="${use_mock_hardware}">
+				<hardware>
+					<plugin>blcmd_hardware/BLCMDHardware</plugin>
+					<param name="candevice">can1</param>
+					<param name="canid">4F4</param>
+					<param name="resolver_reduction">1.33333333333</param>
+					<param name="clock_rate">100000000</param>
+					<param name="revolution_pulses">8192</param>
+					<param name="min_interval">122</param>
+					<param name="gear_ratio">36.0</param>
+					<param name="mock">true</param>
+					<param name="reversed">true</param>
+					<param name="integrate_velocity">true</param>
+				</hardware>
+			</xacro:unless>
+			<xacro:if value="${use_mock_hardware}">
+				<hardware>
+					<plugin>mock_components/GenericSystem</plugin>
+					<param name="calculate_dynamics">true</param>
+				</hardware>
+			</xacro:if>
+			<joint name="J4">
+				<command_interface name="velocity">
+					<param name="max">1</param>
+				</command_interface>
+				<command_interface name="position">
+				</command_interface>
+			</joint>
+		</ros2_control>
+		<ros2_control name="arm_J5" type="system">
+			<xacro:unless value="${use_mock_hardware}">
+				<hardware>
+					<plugin>blcmd_hardware/BLCMDHardware</plugin>
+					<param name="candevice">can1</param>
+					<param name="canid">4F5</param>
+					<param name="resolver_reduction">1.33333333333</param>
+					<param name="clock_rate">100000000</param>
+					<param name="revolution_pulses">8192</param>
+					<param name="min_interval">122</param>
+					<param name="gear_ratio">36.0</param>
+					<param name="mock">true</param>
+					<param name="reversed">true</param>
+					<param name="integrate_velocity">true</param>
+				</hardware>
+			</xacro:unless>
+			<xacro:if value="${use_mock_hardware}">
+				<hardware>
+					<plugin>mock_components/GenericSystem</plugin>
+					<param name="calculate_dynamics">true</param>
+				</hardware>
+			</xacro:if>
+			<joint name="J5">
+				<command_interface name="velocity">
+					<param name="max">1</param>
+				</command_interface>
+				<command_interface name="position">
+				</command_interface>
+			</joint>
+		</ros2_control>
+		<ros2_control name="arm_J6" type="system">
+			<xacro:unless value="${use_mock_hardware}">
+				<hardware>
+					<plugin>blcmd_hardware/BLCMDHardware</plugin>
+					<param name="candevice">can1</param>
+					<param name="canid">4F6</param>
+					<param name="resolver_reduction">1.33333333333</param>
+					<param name="clock_rate">100000000</param>
+					<param name="revolution_pulses">8192</param>
+					<param name="min_interval">122</param>
+					<param name="gear_ratio">36.0</param>
+					<param name="mock">true</param>
+					<param name="reversed">true</param>
+					<param name="integrate_velocity">true</param>
+				</hardware>
+			</xacro:unless>
+			<xacro:if value="${use_mock_hardware}">
+				<hardware>
+					<plugin>mock_components/GenericSystem</plugin>
+					<param name="calculate_dynamics">true</param>
+				</hardware>
+			</xacro:if>
+			<joint name="J6">
+				<command_interface name="velocity">
+					<param name="max">1</param>
+				</command_interface>
+				<command_interface name="position">
+				</command_interface>
+			</joint>
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