Commit message: feat: add ros2_control definitions to new arm

File: src/ros/rover/rover_description/arm/urdf/newarm.ros2_control.xacro (robot description, xacro)
@@ -5,8 +5,199 @@
   <xacro:macro name="newarm_ros2_control" params="use_mock_hardware">
     <ros2_control name="arm" type="system">
-      <hardware>
-        <!-- TODO: Figure out and add the Hardware interface -->
-        <plugin>${ros2_control_plugin}</plugin>
-      </hardware>
+	  <xacro:unless value="${use_mock_hardware}">
+        <hardware>
+		  <plugin>blcmd_hardware/BLCMDHardware</plugin>
+		  <param name="candevice">can0</param>
+		  <param name="canid">1</param>
+		  <param name="resolver_reduction">1.33333333333</param>
+		  <param name="clock_rate">100000000</param>
+		  <param name="revolution_pulses">8192</param>
+		  <param name="min_interval">122</param>
+		  <param name="gear_ratio">36.0</param>
+		  <param name="mock">true</param>
+		  <param name="reversed">true</param>
+		  <param name="integrate_velocity">true</param>
+        </hardware>
+      </xacro:unless>
+      <xacro:if value="${use_mock_hardware}">
+        <hardware>
+          <plugin>mock_components/GenericSystem</plugin>
+          <param name="calculate_dynamics">true</param>
+        </hardware>
+	  </xacro:if>
+	  <!--
+	  <hardware>
+        TODO: Figure out and add the Hardware interface
+	  <plugin>${ros2_control_plugin}</plugin>
+	  </hardware>
+	  -->
+	  <joint name="J1_gbp_chassis">
+		<command_interface name="velocity">
+		  <param name="max">1</param>
+		</command_interface>
+		<command_interface name="effort">
+		  <param name="max">1</param>
+		</command_interface>
+		<state_interface name="velocity">
+		  <param name="initial_value">0.0</param>
+		</state_interface>
+		<state_interface name="position">
+		  <param name="initial_value">0.0</param>
+		</state_interface>
+      </joint>
+	  <joint name="J2_l1a_bp">
+		<command_interface name="velocity">
+		  <param name="max">1</param>
+		</command_interface>
+		<command_interface name="effort">
+		  <param name="max">1</param>
+		</command_interface>
+		<state_interface name="velocity">
+		  <param name="initial_value">0.0</param>
+		</state_interface>
+		<state_interface name="position">
+		  <param name="initial_value">0.0</param>
+		</state_interface>
+      </joint>
+	  <joint name="J2_l2b_bp">
+		<command_interface name="velocity">
+		  <param name="max">1</param>
+		</command_interface>
+		<command_interface name="effort">
+		  <param name="max">1</param>
+		</command_interface>
+		<state_interface name="velocity">
+		  <param name="initial_value">0.0</param>
+		</state_interface>
+		<state_interface name="position">
+		  <param name="initial_value">0.0</param>
+		</state_interface>
+      </joint>
+	  <joint name="l1b_bp">
+		<command_interface name="velocity">
+		  <param name="max">1</param>
+		</command_interface>
+		<command_interface name="effort">
+		  <param name="max">1</param>
+		</command_interface>
+		<state_interface name="velocity">
+		  <param name="initial_value">0.0</param>
+		</state_interface>
+		<state_interface name="position">
+		  <param name="initial_value">0.0</param>
+		</state_interface>
+      </joint>
+	  <joint name="l1b_tp">
+		<command_interface name="velocity">
+		  <param name="max">1</param>
+		</command_interface>
+		<command_interface name="effort">
+		  <param name="max">1</param>
+		</command_interface>
+		<state_interface name="velocity">
+		  <param name="initial_value">0.0</param>
+		</state_interface>
+		<state_interface name="position">
+		  <param name="initial_value">0.0</param>
+		</state_interface>
+      </joint>
+	  <joint name="l1a_tp">
+		<command_interface name="velocity">
+		  <param name="max">1</param>
+		</command_interface>
+		<command_interface name="effort">
+		  <param name="max">1</param>
+		</command_interface>
+		<state_interface name="velocity">
+		  <param name="initial_value">0.0</param>
+		</state_interface>
+		<state_interface name="position">
+		  <param name="initial_value">0.0</param>
+		</state_interface>
+      </joint>
+	  <joint name="wrist_pitch">
+		<command_interface name="velocity">
+		  <param name="max">1</param>
+		</command_interface>
+		<command_interface name="effort">
+		  <param name="max">1</param>
+		</command_interface>
+		<state_interface name="velocity">
+		  <param name="initial_value">0.0</param>
+		</state_interface>
+		<state_interface name="position">
+		  <param name="initial_value">0.0</param>
+		</state_interface>
+      </joint>
+	  <joint name="wrist_yaw">
+		<command_interface name="velocity">
+		  <param name="max">1</param>
+		</command_interface>
+		<command_interface name="effort">
+		  <param name="max">1</param>
+		</command_interface>
+		<state_interface name="velocity">
+		  <param name="initial_value">0.0</param>
+		</state_interface>
+		<state_interface name="position">
+		  <param name="initial_value">0.0</param>
+		</state_interface>
+      </joint>
+	  <joint name="wrist_roll">
+		<command_interface name="velocity">
+		  <param name="max">1</param>
+		</command_interface>
+		<command_interface name="effort">
+		  <param name="max">1</param>
+		</command_interface>
+		<state_interface name="velocity">
+		  <param name="initial_value">0.0</param>
+		</state_interface>
+		<state_interface name="position">
+		  <param name="initial_value">0.0</param>
+		</state_interface>
+      </joint>
+	  <joint name="rf_slide">
+		<command_interface name="velocity">
+		  <param name="max">1</param>
+		</command_interface>
+		<command_interface name="effort">
+		  <param name="max">1</param>
+		</command_interface>
+		<state_interface name="velocity">
+		  <param name="initial_value">0.0</param>
+		</state_interface>
+		<state_interface name="position">
+		  <param name="initial_value">0.0</param>
+		</state_interface>
+      </joint>
+	  <joint name="lf_slide">
+		<command_interface name="velocity">
+		  <param name="max">1</param>
+		</command_interface>
+		<command_interface name="effort">
+		  <param name="max">1</param>
+		</command_interface>
+		<state_interface name="velocity">
+		  <param name="initial_value">0.0</param>
+		</state_interface>
+		<state_interface name="position">
+		  <param name="initial_value">0.0</param>
+		</state_interface>
+      </joint>
+	  <joint name="actuator_head">
+		<command_interface name="velocity">
+		  <param name="max">1</param>
+		</command_interface>
+		<command_interface name="effort">
+		  <param name="max">1</param>
+		</command_interface>
+		<state_interface name="velocity">
+		  <param name="initial_value">0.0</param>
+		</state_interface>
+		<state_interface name="position">
+		  <param name="initial_value">0.0</param>
+		</state_interface>
+      </joint>
     </ros2_control>
   </xacro:macro>

Commit message: refactor: changed new arm joint names to be more consistent

File: src/ros/rover/rover_description/arm/urdf/newarm.ros2_control.xacro (robot description, xacro)
@@ -32,75 +32,75 @@
 	  </hardware>
 	  -->
-	  <joint name="J1_gbp_chassis">
-		<command_interface name="velocity">
-		  <param name="max">1</param>
-		</command_interface>
-		<command_interface name="effort">
-		  <param name="max">1</param>
-		</command_interface>
-		<state_interface name="velocity">
-		  <param name="initial_value">0.0</param>
-		</state_interface>
-		<state_interface name="position">
-		  <param name="initial_value">0.0</param>
-		</state_interface>
-      </joint>
-	  <joint name="J2_l1a_bp">
-		<command_interface name="velocity">
-		  <param name="max">1</param>
-		</command_interface>
-		<command_interface name="effort">
-		  <param name="max">1</param>
-		</command_interface>
-		<state_interface name="velocity">
-		  <param name="initial_value">0.0</param>
-		</state_interface>
-		<state_interface name="position">
-		  <param name="initial_value">0.0</param>
-		</state_interface>
-      </joint>
-	  <joint name="J2_l2b_bp">
-		<command_interface name="velocity">
-		  <param name="max">1</param>
-		</command_interface>
-		<command_interface name="effort">
-		  <param name="max">1</param>
-		</command_interface>
-		<state_interface name="velocity">
-		  <param name="initial_value">0.0</param>
-		</state_interface>
-		<state_interface name="position">
-		  <param name="initial_value">0.0</param>
-		</state_interface>
-      </joint>
-	  <joint name="l1b_bp">
-		<command_interface name="velocity">
-		  <param name="max">1</param>
-		</command_interface>
-		<command_interface name="effort">
-		  <param name="max">1</param>
-		</command_interface>
-		<state_interface name="velocity">
-		  <param name="initial_value">0.0</param>
-		</state_interface>
-		<state_interface name="position">
-		  <param name="initial_value">0.0</param>
-		</state_interface>
-      </joint>
-	  <joint name="l1b_tp">
-		<command_interface name="velocity">
-		  <param name="max">1</param>
-		</command_interface>
-		<command_interface name="effort">
-		  <param name="max">1</param>
-		</command_interface>
-		<state_interface name="velocity">
-		  <param name="initial_value">0.0</param>
-		</state_interface>
-		<state_interface name="position">
-		  <param name="initial_value">0.0</param>
-		</state_interface>
-      </joint>
-	  <joint name="l1a_tp">
+	  <joint name="J1">
+		<command_interface name="velocity">
+		  <param name="max">1</param>
+		</command_interface>
+		<command_interface name="effort">
+		  <param name="max">1</param>
+		</command_interface>
+		<state_interface name="velocity">
+		  <param name="initial_value">0.0</param>
+		</state_interface>
+		<state_interface name="position">
+		  <param name="initial_value">0.0</param>
+		</state_interface>
+      </joint>
+	  <joint name="J2">
+		<command_interface name="velocity">
+		  <param name="max">1</param>
+		</command_interface>
+		<command_interface name="effort">
+		  <param name="max">1</param>
+		</command_interface>
+		<state_interface name="velocity">
+		  <param name="initial_value">0.0</param>
+		</state_interface>
+		<state_interface name="position">
+		  <param name="initial_value">0.0</param>
+		</state_interface>
+      </joint>
+	  <joint name="J3">
+		<command_interface name="velocity">
+		  <param name="max">1</param>
+		</command_interface>
+		<command_interface name="effort">
+		  <param name="max">1</param>
+		</command_interface>
+		<state_interface name="velocity">
+		  <param name="initial_value">0.0</param>
+		</state_interface>
+		<state_interface name="position">
+		  <param name="initial_value">0.0</param>
+		</state_interface>
+      </joint>
+	  <joint name="J4">
+		<command_interface name="velocity">
+		  <param name="max">1</param>
+		</command_interface>
+		<command_interface name="effort">
+		  <param name="max">1</param>
+		</command_interface>
+		<state_interface name="velocity">
+		  <param name="initial_value">0.0</param>
+		</state_interface>
+		<state_interface name="position">
+		  <param name="initial_value">0.0</param>
+		</state_interface>
+      </joint>
+	  <joint name="J5">
+		<command_interface name="velocity">
+		  <param name="max">1</param>
+		</command_interface>
+		<command_interface name="effort">
+		  <param name="max">1</param>
+		</command_interface>
+		<state_interface name="velocity">
+		  <param name="initial_value">0.0</param>
+		</state_interface>
+		<state_interface name="position">
+		  <param name="initial_value">0.0</param>
+		</state_interface>
+      </joint>
+	  <joint name="J6">
 		<command_interface name="velocity">
 		  <param name="max">1</param>

File: src/ros/rover/rover_description/arm/urdf/newarm_joints.xacro (robot description, xacro)
@@ -5,10 +5,10 @@
           <plugin filename="gz-sim-joint-state-publisher-system" name="gz::sim::systems::JointStatePublisher">
                <topic>arm_joints</topic>
-               <joint_name>J1_gbp_chassis</joint_name>
-               <joint_name>J2_l1a_bp</joint_name>
-               <joint_name>J3_l2b_bp</joint_name>
-               <joint_name>l1b_bp</joint_name>
-               <joint_name>l1b_tp</joint_name>
-               <joint_name>l1a_tp</joint_name>
+               <joint_name>J1</joint_name>
+               <joint_name>J2</joint_name>
+               <joint_name>J3</joint_name>
+               <joint_name>J4</joint_name>
+               <joint_name>J5</joint_name>
+               <joint_name>J6</joint_name>
                <joint_name>wrist_pitch</joint_name>
                <joint_name>wrist_yaw</joint_name>

Commit message: temp

File: src/ros/rover/rover_description/arm/urdf/newarm.ros2_control.xacro (robot description, xacro)
@@ -8,5 +8,5 @@
         <hardware>
 		  <plugin>blcmd_hardware/BLCMDHardware</plugin>
-		  <param name="candevice">can0</param>
+		  <param name="candevice">can1</param>
 		  <param name="canid">1</param>
 		  <param name="resolver_reduction">1.33333333333</param>
@@ -46,4 +46,5 @@
 		</state_interface>
       </joint>
+      <!--
 	  <joint name="J2_l1a_bp">
 		<command_interface name="velocity">
@@ -158,5 +159,7 @@
 		</state_interface>
       </joint>
-	  <joint name="rf_slide">
+      -->
+        <!--
+    <joint name="rf_slide">
 		<command_interface name="velocity">
 		  <param name="max">1</param>
@@ -200,4 +203,5 @@
 		</state_interface>
       </joint>
+    -->
     </ros2_control>
   </xacro:macro>
