Commit message: arm ros2 control
- make sure we call the macro defined in newarm.ros2_control.xacro
- have one joint per bclmd

still broken tho! Not sure why this doesn't occur for the drive stuff.

$ ros2 launch auto_bringup control.launch.py arm:=true model:="/home/nova/nova/src/ros/rover/rover_description/rover7/urdf/rover.urdf.xacro
[ros2_control_node-6] [INFO] [1738244473.583731451] [controller_manager]: Activating controllers: [ nova_arm_controller ]
[ros2_control_node-6] [FATAL] [1738244473.583812278] [J1]: Requested start interface J1_gbp_chassis/effort when control mode was not undefined
[ros2_control_node-6] [ERROR] [1738244473.583843616] [controller_manager.resource_manager]: Component 'J1' did not accept command interfaces combination:
[ros2_control_node-6] Start interfaces:
[ros2_control_node-6] [
[ros2_control_node-6]   J1_gbp_chassis/velocity
[ros2_control_node-6]   J2_l1a_bp/velocity
[ros2_control_node-6]   J3_l2b_bp/velocity
[ros2_control_node-6]   wrist_pitch/velocity
[ros2_control_node-6]   wrist_yaw/velocity
[ros2_control_node-6]   wrist_roll/velocity
[ros2_control_node-6]   J1_gbp_chassis/effort
[ros2_control_node-6]   J2_l1a_bp/effort
[ros2_control_node-6]   J3_l2b_bp/effort
[ros2_control_node-6]   wrist_pitch/effort
[ros2_control_node-6]   wrist_yaw/effort
[ros2_control_node-6]   wrist_roll/effort
[ros2_control_node-6] ]
[ros2_control_node-6] Stop interfaces:
[ros2_control_node-6] [
[ros2_control_node-6] ]
[ros2_control_node-6]
[ros2_control_node-6] [FATAL] [1738244473.583874147] [J2]: Requested start interface J2_l1a_bp/effort when control mode was not undefined
[ros2_control_node-6] [ERROR] [1738244473.583884031] [controller_manager.resource_manager]: Component 'J2' did not accept command interfaces combination:
[ros2_control_node-6] Start interfaces:
[ros2_control_node-6] [
[ros2_control_node-6]   J1_gbp_chassis/velocity
[ros2_control_node-6]   J2_l1a_bp/velocity
[ros2_control_node-6]   J3_l2b_bp/velocity
[ros2_control_node-6]   wrist_pitch/velocity
[ros2_control_node-6]   wrist_yaw/velocity
[ros2_control_node-6]   wrist_roll/velocity
[ros2_control_node-6]   J1_gbp_chassis/effort
[ros2_control_node-6]   J2_l1a_bp/effort
[ros2_control_node-6]   J3_l2b_bp/effort
[ros2_control_node-6]   wrist_pitch/effort
[ros2_control_node-6]   wrist_yaw/effort
[ros2_control_node-6]   wrist_roll/effort
[ros2_control_node-6] ]
[ros2_control_node-6] Stop interfaces:
[ros2_control_node-6] [
[ros2_control_node-6] ]
[ros2_control_node-6]
[ros2_control_node-6] [FATAL] [1738244473.583899978] [J3]: Requested start interface J3_l2b_bp/effort when control mode was not undefined
[ros2_control_node-6] [ERROR] [1738244473.583908568] [controller_manager.resource_manager]: Component 'J3' did not accept command interfaces combination:
[ros2_control_node-6] Start interfaces:
[ros2_control_node-6] [
[ros2_control_node-6]   J1_gbp_chassis/velocity
[ros2_control_node-6]   J2_l1a_bp/velocity
[ros2_control_node-6]   J3_l2b_bp/velocity
[ros2_control_node-6]   wrist_pitch/velocity
[ros2_control_node-6]   wrist_yaw/velocity
[ros2_control_node-6]   wrist_roll/velocity
[ros2_control_node-6]   J1_gbp_chassis/effort
[ros2_control_node-6]   J2_l1a_bp/effort
[ros2_control_node-6]   J3_l2b_bp/effort
[ros2_control_node-6]   wrist_pitch/effort
[ros2_control_node-6]   wrist_yaw/effort
[ros2_control_node-6]   wrist_roll/effort
[ros2_control_node-6] ]
[ros2_control_node-6] Stop interfaces:
[ros2_control_node-6] [
[ros2_control_node-6] ]
[ros2_control_node-6]
[ros2_control_node-6] [FATAL] [1738244473.583923049] [J4]: Requested start interface wrist_pitch/effort when control mode was not undefined
[ros2_control_node-6] [ERROR] [1738244473.583931352] [controller_manager.resource_manager]: Component 'J4' did not accept command interfaces combination:
[ros2_control_node-6] Start interfaces:
[ros2_control_node-6] [
[ros2_control_node-6]   J1_gbp_chassis/velocity
[ros2_control_node-6]   J2_l1a_bp/velocity
[ros2_control_node-6]   J3_l2b_bp/velocity
[ros2_control_node-6]   wrist_pitch/velocity
[ros2_control_node-6]   wrist_yaw/velocity
[ros2_control_node-6]   wrist_roll/velocity
[ros2_control_node-6]   J1_gbp_chassis/effort
[ros2_control_node-6]   J2_l1a_bp/effort
[ros2_control_node-6]   J3_l2b_bp/effort
[ros2_control_node-6]   wrist_pitch/effort
[ros2_control_node-6]   wrist_yaw/effort
[ros2_control_node-6]   wrist_roll/effort
[ros2_control_node-6] ]
[ros2_control_node-6] Stop interfaces:
[ros2_control_node-6] [
[ros2_control_node-6] ]
[ros2_control_node-6]
[ros2_control_node-6] [FATAL] [1738244473.583945877] [J5]: Requested start interface wrist_yaw/effort when control mode was not undefined
[ros2_control_node-6] [ERROR] [1738244473.583960271] [controller_manager.resource_manager]: Component 'J5' did not accept command interfaces combination:
[ros2_control_node-6] Start interfaces:
[ros2_control_node-6] [
[ros2_control_node-6]   J1_gbp_chassis/velocity
[ros2_control_node-6]   J2_l1a_bp/velocity
[ros2_control_node-6]   J3_l2b_bp/velocity
[ros2_control_node-6]   wrist_pitch/velocity
[ros2_control_node-6]   wrist_yaw/velocity
[ros2_control_node-6]   wrist_roll/velocity
[ros2_control_node-6]   J1_gbp_chassis/effort
[ros2_control_node-6]   J2_l1a_bp/effort
[ros2_control_node-6]   J3_l2b_bp/effort
[ros2_control_node-6]   wrist_pitch/effort
[ros2_control_node-6]   wrist_yaw/effort
[ros2_control_node-6]   wrist_roll/effort
[ros2_control_node-6] ]
[ros2_control_node-6] Stop interfaces:
[ros2_control_node-6] [
[ros2_control_node-6] ]
[ros2_control_node-6]
[ros2_control_node-6] [FATAL] [1738244473.583975923] [J6]: Requested start interface wrist_roll/effort when control mode was not undefined
[ros2_control_node-6] [ERROR] [1738244473.583984210] [controller_manager.resource_manager]: Component 'J6' did not accept command interfaces combination:
[ros2_control_node-6] Start interfaces:
[ros2_control_node-6] [
[ros2_control_node-6]   J1_gbp_chassis/velocity
[ros2_control_node-6]   J2_l1a_bp/velocity
[ros2_control_node-6]   J3_l2b_bp/velocity
[ros2_control_node-6]   wrist_pitch/velocity
[ros2_control_node-6]   wrist_yaw/velocity
[ros2_control_node-6]   wrist_roll/velocity
[ros2_control_node-6]   J1_gbp_chassis/effort
[ros2_control_node-6]   J2_l1a_bp/effort
[ros2_control_node-6]   J3_l2b_bp/effort
[ros2_control_node-6]   wrist_pitch/effort
[ros2_control_node-6]   wrist_yaw/effort
[ros2_control_node-6]   wrist_roll/effort
[ros2_control_node-6] ]
[ros2_control_node-6] Stop interfaces:
[ros2_control_node-6] [
[ros2_control_node-6] ]
[ros2_control_node-6]
[ros2_control_node-6] [ERROR] [1738244473.584001602] [controller_manager]: Could not switch controllers since prepare command mode switch was rejected.
[spawner-1] [ERROR] [1738244473.586613481] [spawner_nova_arm_controller]: Failed to activate controller
[INFO] [spawner-2]: process has finished cleanly [pid 998172]
[INFO] [spawner-4]: process has finished cleanly [pid 998174]
[ERROR] [spawner-1]: process has died [pid 998171, exit code 1, cmd '/nix/store/wzm385px7cdlqrjj3bv8ap2ykqxv7fmn-ros-jazzy-nova-workspace/lib/controller_manager/spawner nova_arm_controller --switch-timeout 10 --ros-args'].

File: src/ros/rover/rover_description/arm/urdf/newarm.ros2_control.xacro (robot description, xacro)
@@ -4,32 +4,26 @@
   <!-- Initial definition based on https://github.com/xArm-Developer/xarm_ros2/blob/master/xarm_description/urdf/xarm6/xarm6.ros2_control.xacro -->
   <xacro:macro name="newarm_ros2_control" params="use_mock_hardware">
-    <ros2_control name="arm" type="system">
-	  <xacro:unless value="${use_mock_hardware}">
-        <hardware>
-		  <plugin>blcmd_hardware/BLCMDHardware</plugin>
-		  <param name="candevice">can1</param>
-		  <param name="canid">1</param>
-		  <param name="resolver_reduction">1.33333333333</param>
-		  <param name="clock_rate">100000000</param>
-		  <param name="revolution_pulses">8192</param>
-		  <param name="min_interval">122</param>
-		  <param name="gear_ratio">36.0</param>
-		  <param name="mock">true</param>
-		  <param name="reversed">true</param>
-		  <param name="integrate_velocity">true</param>
-        </hardware>
-      </xacro:unless>
-      <xacro:if value="${use_mock_hardware}">
-        <hardware>
-          <plugin>mock_components/GenericSystem</plugin>
-          <param name="calculate_dynamics">true</param>
-        </hardware>
-	  </xacro:if>
-	  <!--
-	  <hardware>
-        TODO: Figure out and add the Hardware interface
-	  <plugin>${ros2_control_plugin}</plugin>
-	  </hardware>
-	  -->
+    <ros2_control name="J1" type="system">
+	  <xacro:unless value="${use_mock_hardware}">
+        <hardware>
+		  <plugin>blcmd_hardware/BLCMDHardware</plugin>
+		  <param name="candevice">can1</param>
+      <param name="canid">4</param>
+		  <param name="resolver_reduction">1.33333333333</param>
+		  <param name="clock_rate">100000000</param>
+		  <param name="revolution_pulses">8192</param>
+		  <param name="min_interval">122</param>
+		  <param name="gear_ratio">36.0</param>
+		  <param name="mock">true</param>
+		  <param name="reversed">true</param>
+		  <param name="integrate_velocity">true</param>
+        </hardware>
+      </xacro:unless>
+      <xacro:if value="${use_mock_hardware}">
+        <hardware>
+          <plugin>mock_components/GenericSystem</plugin>
+          <param name="calculate_dynamics">true</param>
+        </hardware>
+	  </xacro:if>
 	  <joint name="J1_gbp_chassis">
 		<command_interface name="velocity">
@@ -46,5 +40,27 @@
 		</state_interface>
       </joint>
-      <!--
+    </ros2_control>
+    <ros2_control name="J2" type="system">
+	  <xacro:unless value="${use_mock_hardware}">
+        <hardware>
+		  <plugin>blcmd_hardware/BLCMDHardware</plugin>
+		  <param name="candevice">can1</param>
+      <param name="canid">8</param>
+		  <param name="resolver_reduction">1.33333333333</param>
+		  <param name="clock_rate">100000000</param>
+		  <param name="revolution_pulses">8192</param>
+		  <param name="min_interval">122</param>
+		  <param name="gear_ratio">36.0</param>
+		  <param name="mock">true</param>
+		  <param name="reversed">true</param>
+		  <param name="integrate_velocity">true</param>
+        </hardware>
+      </xacro:unless>
+      <xacro:if value="${use_mock_hardware}">
+        <hardware>
+          <plugin>mock_components/GenericSystem</plugin>
+          <param name="calculate_dynamics">true</param>
+        </hardware>
+	  </xacro:if>
 	  <joint name="J2_l1a_bp">
 		<command_interface name="velocity">
@@ -61,60 +77,64 @@
 		</state_interface>
       </joint>
-	  <joint name="J2_l2b_bp">
-		<command_interface name="velocity">
-		  <param name="max">1</param>
-		</command_interface>
-		<command_interface name="effort">
-		  <param name="max">1</param>
-		</command_interface>
-		<state_interface name="velocity">
-		  <param name="initial_value">0.0</param>
-		</state_interface>
-		<state_interface name="position">
-		  <param name="initial_value">0.0</param>
-		</state_interface>
-      </joint>
-	  <joint name="l1b_bp">
-		<command_interface name="velocity">
-		  <param name="max">1</param>
-		</command_interface>
-		<command_interface name="effort">
-		  <param name="max">1</param>
-		</command_interface>
-		<state_interface name="velocity">
-		  <param name="initial_value">0.0</param>
-		</state_interface>
-		<state_interface name="position">
-		  <param name="initial_value">0.0</param>
-		</state_interface>
-      </joint>
-	  <joint name="l1b_tp">
-		<command_interface name="velocity">
-		  <param name="max">1</param>
-		</command_interface>
-		<command_interface name="effort">
-		  <param name="max">1</param>
-		</command_interface>
-		<state_interface name="velocity">
-		  <param name="initial_value">0.0</param>
-		</state_interface>
-		<state_interface name="position">
-		  <param name="initial_value">0.0</param>
-		</state_interface>
-      </joint>
-	  <joint name="l1a_tp">
-		<command_interface name="velocity">
-		  <param name="max">1</param>
-		</command_interface>
-		<command_interface name="effort">
-		  <param name="max">1</param>
-		</command_interface>
-		<state_interface name="velocity">
-		  <param name="initial_value">0.0</param>
-		</state_interface>
-		<state_interface name="position">
-		  <param name="initial_value">0.0</param>
-		</state_interface>
-      </joint>
+    </ros2_control>
+    <ros2_control name="J3" type="system">
+	  <xacro:unless value="${use_mock_hardware}">
+        <hardware>
+		  <plugin>blcmd_hardware/BLCMDHardware</plugin>
+		  <param name="candevice">can1</param>
+      <param name="canid">12</param> <!-- XXX -->
+		  <param name="resolver_reduction">1.33333333333</param>
+		  <param name="clock_rate">100000000</param>
+		  <param name="revolution_pulses">8192</param>
+		  <param name="min_interval">122</param>
+		  <param name="gear_ratio">36.0</param>
+		  <param name="mock">true</param>
+		  <param name="reversed">true</param>
+		  <param name="integrate_velocity">true</param>
+        </hardware>
+      </xacro:unless>
+      <xacro:if value="${use_mock_hardware}">
+        <hardware>
+          <plugin>mock_components/GenericSystem</plugin>
+          <param name="calculate_dynamics">true</param>
+        </hardware>
+	  </xacro:if>
+	  <joint name="J3_l2b_bp">
+		<command_interface name="velocity">
+		  <param name="max">1</param>
+		</command_interface>
+		<command_interface name="effort">
+		  <param name="max">1</param>
+		</command_interface>
+		<state_interface name="velocity">
+		  <param name="initial_value">0.0</param>
+		</state_interface>
+		<state_interface name="position">
+		  <param name="initial_value">0.0</param>
+		</state_interface>
+      </joint>
+    </ros2_control>
+    <ros2_control name="J4" type="system">
+	  <xacro:unless value="${use_mock_hardware}">
+        <hardware>
+		  <plugin>blcmd_hardware/BLCMDHardware</plugin>
+		  <param name="candevice">can1</param>
+      <param name="canid">16</param> <!-- XXX -->
+		  <param name="resolver_reduction">1.33333333333</param>
+		  <param name="clock_rate">100000000</param>
+		  <param name="revolution_pulses">8192</param>
+		  <param name="min_interval">122</param>
+		  <param name="gear_ratio">36.0</param>
+		  <param name="mock">true</param>
+		  <param name="reversed">true</param>
+		  <param name="integrate_velocity">true</param>
+        </hardware>
+      </xacro:unless>
+      <xacro:if value="${use_mock_hardware}">
+        <hardware>
+          <plugin>mock_components/GenericSystem</plugin>
+          <param name="calculate_dynamics">true</param>
+        </hardware>
+	  </xacro:if>
 	  <joint name="wrist_pitch">
 		<command_interface name="velocity">
@@ -131,4 +151,27 @@
 		</state_interface>
       </joint>
+    </ros2_control>
+    <ros2_control name="J5" type="system">
+	  <xacro:unless value="${use_mock_hardware}">
+        <hardware>
+		  <plugin>blcmd_hardware/BLCMDHardware</plugin>
+		  <param name="candevice">can1</param>
+      <param name="canid">20</param> <!-- XXX -->
+		  <param name="resolver_reduction">1.33333333333</param>
+		  <param name="clock_rate">100000000</param>
+		  <param name="revolution_pulses">8192</param>
+		  <param name="min_interval">122</param>
+		  <param name="gear_ratio">36.0</param>
+		  <param name="mock">true</param>
+		  <param name="reversed">true</param>
+		  <param name="integrate_velocity">true</param>
+        </hardware>
+      </xacro:unless>
+      <xacro:if value="${use_mock_hardware}">
+        <hardware>
+          <plugin>mock_components/GenericSystem</plugin>
+          <param name="calculate_dynamics">true</param>
+        </hardware>
+	  </xacro:if>
 	  <joint name="wrist_yaw">
 		<command_interface name="velocity">
@@ -145,4 +188,27 @@
 		</state_interface>
       </joint>
+    </ros2_control>
+    <ros2_control name="J6" type="system">
+	  <xacro:unless value="${use_mock_hardware}">
+        <hardware>
+		  <plugin>blcmd_hardware/BLCMDHardware</plugin>
+		  <param name="candevice">can1</param>
+      <param name="canid">24</param> <!-- XXX  not too sure about this, might need to be hexadecimal-->
+		  <param name="resolver_reduction">1.33333333333</param>
+		  <param name="clock_rate">100000000</param>
+		  <param name="revolution_pulses">8192</param>
+		  <param name="min_interval">122</param>
+		  <param name="gear_ratio">36.0</param>
+		  <param name="mock">true</param>
+		  <param name="reversed">true</param>
+		  <param name="integrate_velocity">true</param>
+        </hardware>
+      </xacro:unless>
+      <xacro:if value="${use_mock_hardware}">
+        <hardware>
+          <plugin>mock_components/GenericSystem</plugin>
+          <param name="calculate_dynamics">true</param>
+        </hardware>
+	  </xacro:if>
 	  <joint name="wrist_roll">
 		<command_interface name="velocity">
@@ -159,5 +225,5 @@
 		</state_interface>
       </joint>
-      -->
+    </ros2_control>
         <!--
     <joint name="rf_slide">
@@ -204,5 +270,4 @@
       </joint>
     -->
-    </ros2_control>
   </xacro:macro>
 </robot>

File: src/ros/rover/rover_description/arm/urdf/newarm.urdf.xacro (robot description, xacro)
@@ -569,4 +569,5 @@
     <!-- XXX: ask why this isn't enabled for not gazebo -->
         <xacro:include filename="$(find rover_description)/arm/urdf/newarm.ros2_control.xacro" />
+        <xacro:newarm_ros2_control use_mock_hardware="$(arg use_mock_hardware)" />
     <!-- Standalone arm definition -->
     <xacro:unless value="$(arg arm)">
