Commit message: fixes to ros2 control arm done at workshop

File: src/ros/rover/rover_description/arm/urdf/newarm.ros2_control.xacro (robot description, xacro)
@@ -26,18 +26,40 @@
         </hardware>
 	  </xacro:if>
+<<<<<<< Updated upstream
 	  <joint name="J1_gbp_chassis">
-		<command_interface name="velocity">
-		  <param name="max">1</param>
-		</command_interface>
-		<command_interface name="effort">
-		  <param name="max">1</param>
-		</command_interface>
-		<state_interface name="velocity">
-		  <param name="initial_value">0.0</param>
-		</state_interface>
-		<state_interface name="position">
-		  <param name="initial_value">0.0</param>
-		</state_interface>
-      </joint>
+=======
+	  <!--
+	  <hardware>
+        TODO: Figure out and add the Hardware interface
+	  <plugin>${ros2_control_plugin}</plugin>
+	  </hardware>
+	  -->
+	  <joint name="j1">
+		<command_interface name="velocity">
+		  <param name="max">1</param>
+		</command_interface>
+		<state_interface name="velocity">
+		  <param name="initial_value">0.0</param>
+		</state_interface>
+		<state_interface name="position">
+		  <param name="initial_value">0.0</param>
+		</state_interface>
+      </joint>
+	  <joint name="j2">
+>>>>>>> Stashed changes
+		<command_interface name="velocity">
+		  <param name="max">1</param>
+		</command_interface>
+		<command_interface name="effort">
+		  <param name="max">1</param>
+		</command_interface>
+		<state_interface name="velocity">
+		  <param name="initial_value">0.0</param>
+		</state_interface>
+		<state_interface name="position">
+		  <param name="initial_value">0.0</param>
+		</state_interface>
+      </joint>
+<<<<<<< Updated upstream
     </ros2_control>
     <ros2_control name="J2" type="system">
@@ -64,17 +86,21 @@
 	  </xacro:if>
 	  <joint name="J2_l1a_bp">
-		<command_interface name="velocity">
-		  <param name="max">1</param>
-		</command_interface>
-		<command_interface name="effort">
-		  <param name="max">1</param>
-		</command_interface>
-		<state_interface name="velocity">
-		  <param name="initial_value">0.0</param>
-		</state_interface>
-		<state_interface name="position">
-		  <param name="initial_value">0.0</param>
-		</state_interface>
-      </joint>
+=======
+	  <joint name="j3">
+>>>>>>> Stashed changes
+		<command_interface name="velocity">
+		  <param name="max">1</param>
+		</command_interface>
+		<command_interface name="effort">
+		  <param name="max">1</param>
+		</command_interface>
+		<state_interface name="velocity">
+		  <param name="initial_value">0.0</param>
+		</state_interface>
+		<state_interface name="position">
+		  <param name="initial_value">0.0</param>
+		</state_interface>
+      </joint>
+<<<<<<< Updated upstream
     </ros2_control>
     <ros2_control name="J3" type="system">
@@ -137,18 +163,63 @@
         </hardware>
 	  </xacro:if>
-	  <joint name="wrist_pitch">
-		<command_interface name="velocity">
-		  <param name="max">1</param>
-		</command_interface>
-		<command_interface name="effort">
-		  <param name="max">1</param>
-		</command_interface>
-		<state_interface name="velocity">
-		  <param name="initial_value">0.0</param>
-		</state_interface>
-		<state_interface name="position">
-		  <param name="initial_value">0.0</param>
-		</state_interface>
-      </joint>
+=======
+	  <!-- <joint name="l1b_bp">
+		<command_interface name="velocity">
+		  <param name="max">1</param>
+		</command_interface>
+		<command_interface name="effort">
+		  <param name="max">1</param>
+		</command_interface>
+		<state_interface name="velocity">
+		  <param name="initial_value">0.0</param>
+		</state_interface>
+		<state_interface name="position">
+		  <param name="initial_value">0.0</param>
+		</state_interface>
+      </joint>
+	  <joint name="l1b_tp">
+		<command_interface name="velocity">
+		  <param name="max">1</param>
+		</command_interface>
+		<command_interface name="effort">
+		  <param name="max">1</param>
+		</command_interface>
+		<state_interface name="velocity">
+		  <param name="initial_value">0.0</param>
+		</state_interface>
+		<state_interface name="position">
+		  <param name="initial_value">0.0</param>
+		</state_interface>
+      </joint>
+	  <joint name="l1a_tp">
+		<command_interface name="velocity">
+		  <param name="max">1</param>
+		</command_interface>
+		<command_interface name="effort">
+		  <param name="max">1</param>
+		</command_interface>
+		<state_interface name="velocity">
+		  <param name="initial_value">0.0</param>
+		</state_interface>
+		<state_interface name="position">
+		  <param name="initial_value">0.0</param>
+		</state_interface>
+      </joint> -->
+>>>>>>> Stashed changes
+	  <joint name="j4">
+		<command_interface name="velocity">
+		  <param name="max">1</param>
+		</command_interface>
+		<command_interface name="effort">
+		  <param name="max">1</param>
+		</command_interface>
+		<state_interface name="velocity">
+		  <param name="initial_value">0.0</param>
+		</state_interface>
+		<state_interface name="position">
+		  <param name="initial_value">0.0</param>
+		</state_interface>
+      </joint>
+<<<<<<< Updated upstream
     </ros2_control>
     <ros2_control name="J5" type="system">
@@ -175,17 +246,21 @@
 	  </xacro:if>
 	  <joint name="wrist_yaw">
-		<command_interface name="velocity">
-		  <param name="max">1</param>
-		</command_interface>
-		<command_interface name="effort">
-		  <param name="max">1</param>
-		</command_interface>
-		<state_interface name="velocity">
-		  <param name="initial_value">0.0</param>
-		</state_interface>
-		<state_interface name="position">
-		  <param name="initial_value">0.0</param>
-		</state_interface>
-      </joint>
+=======
+	  <joint name="j5">
+>>>>>>> Stashed changes
+		<command_interface name="velocity">
+		  <param name="max">1</param>
+		</command_interface>
+		<command_interface name="effort">
+		  <param name="max">1</param>
+		</command_interface>
+		<state_interface name="velocity">
+		  <param name="initial_value">0.0</param>
+		</state_interface>
+		<state_interface name="position">
+		  <param name="initial_value">0.0</param>
+		</state_interface>
+      </joint>
+<<<<<<< Updated upstream
     </ros2_control>
     <ros2_control name="J6" type="system">
@@ -212,4 +287,7 @@
 	  </xacro:if>
 	  <joint name="wrist_roll">
+=======
+	  <joint name="j6">
+>>>>>>> Stashed changes
 		<command_interface name="velocity">
 		  <param name="max">1</param>

File: src/ros/rover/rover_description/arm/urdf/newarm.urdf.xacro (robot description, xacro)
@@ -195,5 +195,5 @@
         <joint_properties friction="0.5" damping="0.5"/>
     </joint>
-    <joint name="J2_l1a_bp" type="revolute">
+    <joint name="j2" type="revolute">
         <origin xyz="-1.6653345369377348106e-16 -2.3967136596913301438e-07 -0.16497726032863463397" rpy="1.5707963267948961139 6.0217020942552186975e-15 5.3207089380869679575e-16" />
         <parent link="gearbox" />
@@ -310,5 +310,5 @@
         <joint_properties friction="0.5" damping="0.5"/>
     </joint>
-    <joint name="J3_l2b_bp" type="revolute">
+    <joint name="j3" type="revolute">
         <origin xyz="2.7755575615628913511e-17 -2.3967136592029097706e-07 -0.1649772603286343009" rpy="1.570796326794896558 7.3420626327675113628e-16 -1.8112369360797040431e-15" />
         <parent link="gearbox" />
@@ -526,5 +526,5 @@
         <joint_properties friction="0.0"/>
     </joint>
-    <joint name="wrist_roll" type="revolute">
+    <joint name="j6" type="revolute">
         <origin xyz="-0.00046582360769774496488 -0.086000000000003740119 0.00713417639229629863" rpy="-1.5707963267948990005 7.5034665064024681681e-09 1.0332187252429466388e-16" />
         <parent link="wrist_z" />
@@ -534,5 +534,5 @@
         <joint_properties friction="0.0"/>
     </joint>
-    <joint name="wrist_yaw" type="revolute">
+    <joint name="j5" type="revolute">
         <origin xyz="-1.4432899320127035026e-15 -0.010372222222245208734 -0.056404154590515238887" rpy="-1.5707963267948328312 1.5707963267948086283 0" />
         <parent link="wrist_y" />
@@ -542,5 +542,5 @@
         <joint_properties friction="0.0"/>
     </joint>
-    <joint name="wrist_pitch" type="revolute">
+    <joint name="j4" type="revolute">
         <origin xyz="4.4408920985006261617e-16 0.056950000000000632061 -0.19825000000000037037" rpy="-1.5707963267948878983 1.5707963267948819031 0" />
         <parent link="wrist_base" />
@@ -565,9 +565,29 @@
     </gazebo>
     <!--xacro:include filename="arm_odom.xacro"/ -->
+<<<<<<< Updated upstream
     <xacro:if value="$(arg gazebo)">
+=======
+    <!-- <xacro:if value="$(arg gazebo)">
+        <xacro:include filename="$(find rover_description)/arm/urdf/newarm.ros2_control.xacro" />
+    </xacro:if> -->
+    <!-- gz start -->
+    <xacro:unless value="$(arg gazebo)">
+        <!-- not gazebo start -->
+        <xacro:include filename="$(find rover_description)/arm/urdf/newarm.ros2_control.xacro" />
+        <!-- not gazebo middle -->
+        <xacro:newarm_ros2_control use_mock_hardware="$(arg use_mock_hardware)"/>
+        <!-- not gazebo end -->
+    </xacro:unless>
+    <!-- gz middle -->
+    <xacro:if value="$(arg gazebo)">
+        <!-- heehee gazebo start -->
+        <xacro:include filename="$(find rover_description)/arm/urdf/newarm.gz_ros2_control.xacro" />
+        <!-- hahah gazebo end -->
+>>>>>>> Stashed changes
     </xacro:if>
     <!-- XXX: ask why this isn't enabled for not gazebo -->
         <xacro:include filename="$(find rover_description)/arm/urdf/newarm.ros2_control.xacro" />
         <xacro:newarm_ros2_control use_mock_hardware="$(arg use_mock_hardware)" />
+    <!-- gz end -->
     <!-- Standalone arm definition -->
     <xacro:unless value="$(arg arm)">
@@ -601,5 +621,5 @@
             </inertial>
         </link>
-        <joint name="J1_gbp_chassis" type="revolute">
+        <joint name="j1" type="revolute">
             <origin xyz="0.22899999999999565148 1.1102230246251564172e-16 0.11707476398169122667" rpy="-3.141592653589793116 -1.3309679851047901909e-16 0" />
             <parent link="chassis" />

File: src/ros/rover/rover_description/waratah_arm/urdf/dynamic_joints_with_arm.xacro (robot description, xacro)
@@ -29,13 +29,13 @@
                 <joint_name>br_ball_yaw</joint_name>
                 <!-- Arm joints -->
-                <joint_name>J1_gbp_chassis</joint_name>
-                <joint_name>J2_l1a_bp</joint_name>
-                <joint_name>J3_l2b_bp</joint_name>
+                <joint_name>j1</joint_name>
+                <joint_name>j2</joint_name>
+                <joint_name>j3</joint_name>
                 <joint_name>l1b_bp</joint_name>
                 <joint_name>l1b_tp</joint_name>
                 <joint_name>l1a_tp</joint_name>
-                <joint_name>wrist_pitch</joint_name>
-                <joint_name>wrist_yaw</joint_name>
-                <joint_name>wrist_roll</joint_name>
+                <joint_name>j4</joint_name>
+                <joint_name>j5</joint_name>
+                <joint_name>j6</joint_name>
                 <joint_name>rf_slide</joint_name>
                 <joint_name>lf_slide</joint_name>
