Commit message: refactor: adjusted joint naming

File: src/ros/rover/rover_description/arm/urdf/newarm.ros2_control.xacro (robot description, xacro)
@@ -4,5 +4,5 @@
   <!-- Initial definition based on https://github.com/xArm-Developer/xarm_ros2/blob/master/xarm_description/urdf/xarm6/xarm6.ros2_control.xacro -->
   <xacro:macro name="newarm_ros2_control" params="use_mock_hardware">
-    <ros2_control name="arm_j1" type="system">
+    <ros2_control name="arm_J1" type="system">
 	  <xacro:unless value="${use_mock_hardware}">
         <hardware>
@@ -32,186 +32,153 @@
 	  </hardware>
 	  -->
-	  <joint name="j1">
-		<command_interface name="velocity">
-		  <param name="max">1</param>
-		</command_interface>
-		<state_interface name="velocity">
-		  <param name="initial_value">0.0</param>
-		</state_interface>
-		<state_interface name="position">
-		  <param name="initial_value">0.0</param>
-		</state_interface>
-      </joint>
-	</ros2_control>
-	<ros2_control name="arm_j2" type="system">
-	  <xacro:unless value="${use_mock_hardware}">
-        <hardware>
-		  <plugin>blcmd_hardware/BLCMDHardware</plugin>
-		  <param name="candevice">can1</param>
-      	  <param name="canid">4F1</param>
-		  <param name="resolver_reduction">1.33333333333</param>
-		  <param name="clock_rate">100000000</param>
-		  <param name="revolution_pulses">8192</param>
-		  <param name="min_interval">122</param>
-		  <param name="gear_ratio">36.0</param>
-		  <param name="mock">true</param>
-		  <param name="reversed">true</param>
-		  <param name="integrate_velocity">true</param>
-        </hardware>
-      </xacro:unless>
-      <xacro:if value="${use_mock_hardware}">
-        <hardware>
-          <plugin>mock_components/GenericSystem</plugin>
-          <param name="calculate_dynamics">true</param>
-        </hardware>
-	  </xacro:if>
-	  <joint name="j2">
-		<command_interface name="velocity">
-		  <param name="max">1</param>
-		</command_interface>
-		<state_interface name="velocity">
-		  <param name="initial_value">0.0</param>
-		</state_interface>
-		<state_interface name="position">
-		  <param name="initial_value">0.0</param>
-		</state_interface>
-      </joint>
-	</ros2_control>
-	<ros2_control name="arm_j3" type="system">
-	  <xacro:unless value="${use_mock_hardware}">
-        <hardware>
-		  <plugin>blcmd_hardware/BLCMDHardware</plugin>
-		  <param name="candevice">can1</param>
-      	  <param name="canid">4F1</param>
-		  <param name="resolver_reduction">1.33333333333</param>
-		  <param name="clock_rate">100000000</param>
-		  <param name="revolution_pulses">8192</param>
-		  <param name="min_interval">122</param>
-		  <param name="gear_ratio">36.0</param>
-		  <param name="mock">true</param>
-		  <param name="reversed">true</param>
-		  <param name="integrate_velocity">true</param>
-        </hardware>
-      </xacro:unless>
-      <xacro:if value="${use_mock_hardware}">
-        <hardware>
-          <plugin>mock_components/GenericSystem</plugin>
-          <param name="calculate_dynamics">true</param>
-        </hardware>
-	  </xacro:if>
-	  <joint name="j3">
-		<command_interface name="velocity">
-		  <param name="max">1</param>
-		</command_interface>
-		<state_interface name="velocity">
-		  <param name="initial_value">0.0</param>
-		</state_interface>
-		<state_interface name="position">
-		  <param name="initial_value">0.0</param>
-		</state_interface>
-      </joint>
-	</ros2_control>
-	  <!-- <joint name="l1b_bp">
-		<command_interface name="velocity">
-		  <param name="max">1</param>
-		</command_interface>
-		<state_interface name="velocity">
-		  <param name="initial_value">0.0</param>
-		</state_interface>
-		<state_interface name="position">
-		  <param name="initial_value">0.0</param>
-		</state_interface>
-      </joint>
-	  <joint name="l1b_tp">
-		<command_interface name="velocity">
-		  <param name="max">1</param>
-		</command_interface>
-		<state_interface name="velocity">
-		  <param name="initial_value">0.0</param>
-		</state_interface>
-		<state_interface name="position">
-		  <param name="initial_value">0.0</param>
-		</state_interface>
-      </joint>
-	  <joint name="l1a_tp">
-		<command_interface name="velocity">
-		  <param name="max">1</param>
-		</command_interface>
-		<state_interface name="velocity">
-		  <param name="initial_value">0.0</param>
-		</state_interface>
-		<state_interface name="position">
-		  <param name="initial_value">0.0</param>
-		</state_interface>
-      </joint> -->
-	<ros2_control name="arm_j4" type="system">
-	  <xacro:unless value="${use_mock_hardware}">
-        <hardware>
-		  <plugin>blcmd_hardware/BLCMDHardware</plugin>
-		  <param name="candevice">can1</param>
-      	  <param name="canid">4F1</param>
-		  <param name="resolver_reduction">1.33333333333</param>
-		  <param name="clock_rate">100000000</param>
-		  <param name="revolution_pulses">8192</param>
-		  <param name="min_interval">122</param>
-		  <param name="gear_ratio">36.0</param>
-		  <param name="mock">true</param>
-		  <param name="reversed">true</param>
-		  <param name="integrate_velocity">true</param>
-        </hardware>
-      </xacro:unless>
-      <xacro:if value="${use_mock_hardware}">
-        <hardware>
-          <plugin>mock_components/GenericSystem</plugin>
-          <param name="calculate_dynamics">true</param>
-        </hardware>
-	  </xacro:if>
-	  <joint name="j4">
-		<command_interface name="velocity">
-		  <param name="max">1</param>
-		</command_interface>
-		<state_interface name="velocity">
-		  <param name="initial_value">0.0</param>
-		</state_interface>
-		<state_interface name="position">
-		  <param name="initial_value">0.0</param>
-		</state_interface>
-      </joint>
-	</ros2_control>
-	<ros2_control name="arm_j5" type="system">
-	  <xacro:unless value="${use_mock_hardware}">
-        <hardware>
-		  <plugin>blcmd_hardware/BLCMDHardware</plugin>
-		  <param name="candevice">can1</param>
-      	  <param name="canid">4F1</param>
-		  <param name="resolver_reduction">1.33333333333</param>
-		  <param name="clock_rate">100000000</param>
-		  <param name="revolution_pulses">8192</param>
-		  <param name="min_interval">122</param>
-		  <param name="gear_ratio">36.0</param>
-		  <param name="mock">true</param>
-		  <param name="reversed">true</param>
-		  <param name="integrate_velocity">true</param>
-        </hardware>
-      </xacro:unless>
-      <xacro:if value="${use_mock_hardware}">
-        <hardware>
-          <plugin>mock_components/GenericSystem</plugin>
-          <param name="calculate_dynamics">true</param>
-        </hardware>
-	  </xacro:if>
-	  <joint name="j5">
-		<command_interface name="velocity">
-		  <param name="max">1</param>
-		</command_interface>
-		<state_interface name="velocity">
-		  <param name="initial_value">0.0</param>
-		</state_interface>
-		<state_interface name="position">
-		  <param name="initial_value">0.0</param>
-		</state_interface>
-      </joint>
-	</ros2_control>
-	<ros2_control name="arm_j6" type="system">
+	  <joint name="J1">
+		<command_interface name="velocity">
+		  <param name="max">1</param>
+		</command_interface>
+		<state_interface name="velocity">
+		  <param name="initial_value">0.0</param>
+		</state_interface>
+		<state_interface name="position">
+		  <param name="initial_value">0.0</param>
+		</state_interface>
+      </joint>
+	</ros2_control>
+	<ros2_control name="arm_J2" type="system">
+	  <xacro:unless value="${use_mock_hardware}">
+        <hardware>
+		  <plugin>blcmd_hardware/BLCMDHardware</plugin>
+		  <param name="candevice">can1</param>
+      	  <param name="canid">4F1</param>
+		  <param name="resolver_reduction">1.33333333333</param>
+		  <param name="clock_rate">100000000</param>
+		  <param name="revolution_pulses">8192</param>
+		  <param name="min_interval">122</param>
+		  <param name="gear_ratio">36.0</param>
+		  <param name="mock">true</param>
+		  <param name="reversed">true</param>
+		  <param name="integrate_velocity">true</param>
+        </hardware>
+      </xacro:unless>
+      <xacro:if value="${use_mock_hardware}">
+        <hardware>
+          <plugin>mock_components/GenericSystem</plugin>
+          <param name="calculate_dynamics">true</param>
+        </hardware>
+	  </xacro:if>
+	  <joint name="J2">
+		<command_interface name="velocity">
+		  <param name="max">1</param>
+		</command_interface>
+		<state_interface name="velocity">
+		  <param name="initial_value">0.0</param>
+		</state_interface>
+		<state_interface name="position">
+		  <param name="initial_value">0.0</param>
+		</state_interface>
+      </joint>
+	</ros2_control>
+	<ros2_control name="arm_J3" type="system">
+	  <xacro:unless value="${use_mock_hardware}">
+        <hardware>
+		  <plugin>blcmd_hardware/BLCMDHardware</plugin>
+		  <param name="candevice">can1</param>
+      	  <param name="canid">4F1</param>
+		  <param name="resolver_reduction">1.33333333333</param>
+		  <param name="clock_rate">100000000</param>
+		  <param name="revolution_pulses">8192</param>
+		  <param name="min_interval">122</param>
+		  <param name="gear_ratio">36.0</param>
+		  <param name="mock">true</param>
+		  <param name="reversed">true</param>
+		  <param name="integrate_velocity">true</param>
+        </hardware>
+      </xacro:unless>
+      <xacro:if value="${use_mock_hardware}">
+        <hardware>
+          <plugin>mock_components/GenericSystem</plugin>
+          <param name="calculate_dynamics">true</param>
+        </hardware>
+	  </xacro:if>
+	  <joint name="J3">
+		<command_interface name="velocity">
+		  <param name="max">1</param>
+		</command_interface>
+		<state_interface name="velocity">
+		  <param name="initial_value">0.0</param>
+		</state_interface>
+		<state_interface name="position">
+		  <param name="initial_value">0.0</param>
+		</state_interface>
+      </joint>
+	</ros2_control>
+	<ros2_control name="arm_J4" type="system">
+	  <xacro:unless value="${use_mock_hardware}">
+        <hardware>
+		  <plugin>blcmd_hardware/BLCMDHardware</plugin>
+		  <param name="candevice">can1</param>
+      	  <param name="canid">4F1</param>
+		  <param name="resolver_reduction">1.33333333333</param>
+		  <param name="clock_rate">100000000</param>
+		  <param name="revolution_pulses">8192</param>
+		  <param name="min_interval">122</param>
+		  <param name="gear_ratio">36.0</param>
+		  <param name="mock">true</param>
+		  <param name="reversed">true</param>
+		  <param name="integrate_velocity">true</param>
+        </hardware>
+      </xacro:unless>
+      <xacro:if value="${use_mock_hardware}">
+        <hardware>
+          <plugin>mock_components/GenericSystem</plugin>
+          <param name="calculate_dynamics">true</param>
+        </hardware>
+	  </xacro:if>
+	  <joint name="J4">
+		<command_interface name="velocity">
+		  <param name="max">1</param>
+		</command_interface>
+		<state_interface name="velocity">
+		  <param name="initial_value">0.0</param>
+		</state_interface>
+		<state_interface name="position">
+		  <param name="initial_value">0.0</param>
+		</state_interface>
+      </joint>
+	</ros2_control>
+	<ros2_control name="arm_J6" type="system">
+	  <xacro:unless value="${use_mock_hardware}">
+        <hardware>
+		  <plugin>blcmd_hardware/BLCMDHardware</plugin>
+		  <param name="candevice">can1</param>
+      	  <param name="canid">4F1</param>
+		  <param name="resolver_reduction">1.33333333333</param>
+		  <param name="clock_rate">100000000</param>
+		  <param name="revolution_pulses">8192</param>
+		  <param name="min_interval">122</param>
+		  <param name="gear_ratio">36.0</param>
+		  <param name="mock">true</param>
+		  <param name="reversed">true</param>
+		  <param name="integrate_velocity">true</param>
+        </hardware>
+      </xacro:unless>
+      <xacro:if value="${use_mock_hardware}">
+        <hardware>
+          <plugin>mock_components/GenericSystem</plugin>
+          <param name="calculate_dynamics">true</param>
+        </hardware>
+	  </xacro:if>
+	  <joint name="J6">
+		<command_interface name="velocity">
+		  <param name="max">1</param>
+		</command_interface>
+		<state_interface name="velocity">
+		  <param name="initial_value">0.0</param>
+		</state_interface>
+		<state_interface name="position">
+		  <param name="initial_value">0.0</param>
+		</state_interface>
+      </joint>
+	</ros2_control>
+	<ros2_control name="arm_J6" type="system">
 	  <xacro:unless value="${use_mock_hardware}">
         <hardware>
@@ -235,5 +202,5 @@
         </hardware>
 	  </xacro:if>
-	  <joint name="j6">
+	  <joint name="J6">
 		<command_interface name="velocity">
 		  <param name="max">1</param>

File: src/ros/rover/rover_description/arm/urdf/newarm.urdf.xacro (robot description, xacro)
@@ -195,5 +195,5 @@
         <joint_properties friction="0.5" damping="0.5"/>
     </joint>
-    <joint name="j2" type="revolute">
+    <joint name="J2" type="revolute">
         <origin xyz="-1.6653345369377348106e-16 -2.3967136596913301438e-07 -0.16497726032863463397" rpy="1.5707963267948961139 6.0217020942552186975e-15 5.3207089380869679575e-16" />
         <parent link="gearbox" />
@@ -310,5 +310,5 @@
         <joint_properties friction="0.5" damping="0.5"/>
     </joint>
-    <joint name="j3" type="revolute">
+    <joint name="J3" type="revolute">
         <origin xyz="2.7755575615628913511e-17 -2.3967136592029097706e-07 -0.1649772603286343009" rpy="1.570796326794896558 7.3420626327675113628e-16 -1.8112369360797040431e-15" />
         <parent link="gearbox" />
@@ -526,5 +526,5 @@
         <joint_properties friction="0.0"/>
     </joint>
-    <joint name="j6" type="revolute">
+    <joint name="J6" type="revolute">
         <origin xyz="-0.00046582360769774496488 -0.086000000000003740119 0.00713417639229629863" rpy="-1.5707963267948990005 7.5034665064024681681e-09 1.0332187252429466388e-16" />
         <parent link="wrist_z" />
@@ -534,5 +534,5 @@
         <joint_properties friction="0.0"/>
     </joint>
-    <joint name="j5" type="revolute">
+    <joint name="J5" type="revolute">
         <origin xyz="-1.4432899320127035026e-15 -0.010372222222245208734 -0.056404154590515238887" rpy="-1.5707963267948328312 1.5707963267948086283 0" />
         <parent link="wrist_y" />
@@ -542,5 +542,5 @@
         <joint_properties friction="0.0"/>
     </joint>
-    <joint name="j4" type="revolute">
+    <joint name="J4" type="revolute">
         <origin xyz="4.4408920985006261617e-16 0.056950000000000632061 -0.19825000000000037037" rpy="-1.5707963267948878983 1.5707963267948819031 0" />
         <parent link="wrist_base" />
@@ -614,5 +614,5 @@
             </inertial>
         </link>
-        <joint name="j1" type="revolute">
+        <joint name="J1" type="revolute">
             <origin xyz="0.22899999999999565148 1.1102230246251564172e-16 0.11707476398169122667" rpy="-3.141592653589793116 -1.3309679851047901909e-16 0" />
             <parent link="chassis" />

File: src/ros/rover/rover_description/waratah_arm/urdf/dynamic_joints_with_arm.xacro (robot description, xacro)
@@ -29,13 +29,13 @@
                 <joint_name>br_ball_yaw</joint_name>
                 <!-- Arm joints -->
-                <joint_name>j1</joint_name>
-                <joint_name>j2</joint_name>
-                <joint_name>j3</joint_name>
+                <joint_name>J1</joint_name>
+                <joint_name>J2</joint_name>
+                <joint_name>J3</joint_name>
                 <joint_name>l1b_bp</joint_name>
                 <joint_name>l1b_tp</joint_name>
                 <joint_name>l1a_tp</joint_name>
-                <joint_name>j4</joint_name>
-                <joint_name>j5</joint_name>
-                <joint_name>j6</joint_name>
+                <joint_name>J4</joint_name>
+                <joint_name>J5</joint_name>
+                <joint_name>J6</joint_name>
                 <joint_name>rf_slide</joint_name>
                 <joint_name>lf_slide</joint_name>
