Commit message: feat: arm can now be actuated in gazebo sim using manually published messages

File: src/ros/rover/rover_description/arm/urdf/newarm.urdf.xacro (robot description, xacro)
@@ -579,5 +579,5 @@
     <xacro:if value="$(arg gazebo)">
         <!-- heehee gazebo start -->
-        <xacro:include filename="$(find rover_description)/arm/urdf/newarm.gz_ros2_control.xacro" />
+        <!-- <xacro:include filename="$(find rover_description)/arm/urdf/newarm.gz_ros2_control.xacro" /> -->
         <!-- hahah gazebo end -->
     </xacro:if>

File: src/ros/rover/rover_description/banksia/urdf/gz_ros2_control.xacro (robot description, xacro)
@@ -117,4 +117,136 @@
       </state_interface>
     </joint>
+        <joint name="J1">
+		<command_interface name="velocity">
+		  <param name="max">1</param>
+		</command_interface>
+		<state_interface name="velocity">
+		  <param name="initial_value">0.0</param>
+		</state_interface>
+		<state_interface name="position">
+		  <param name="initial_value">0.0</param>
+		</state_interface>
+      </joint>
+	  <joint name="J2">
+		<command_interface name="velocity">
+		  <param name="max">1</param>
+		</command_interface>
+		<state_interface name="velocity">
+		  <param name="initial_value">0.0</param>
+		</state_interface>
+		<state_interface name="position">
+		  <param name="initial_value">0.0</param>
+		</state_interface>
+      </joint>
+	  <joint name="J3">
+		<command_interface name="velocity">
+		  <param name="max">1</param>
+		</command_interface>
+		<state_interface name="velocity">
+		  <param name="initial_value">0.0</param>
+		</state_interface>
+		<state_interface name="position">
+		  <param name="initial_value">0.0</param>
+		</state_interface>
+      </joint>
+	  <!-- <joint name="l1b_bp">
+		<command_interface name="velocity">
+		  <param name="max">1</param>
+		</command_interface>
+		<state_interface name="velocity">
+		  <param name="initial_value">0.0</param>
+		</state_interface>
+		<state_interface name="position">
+		  <param name="initial_value">0.0</param>
+		</state_interface>
+      </joint>
+	  <joint name="l1b_tp">
+		<command_interface name="velocity">
+		  <param name="max">1</param>
+		</command_interface>
+		<state_interface name="velocity">
+		  <param name="initial_value">0.0</param>
+		</state_interface>
+		<state_interface name="position">
+		  <param name="initial_value">0.0</param>
+		</state_interface>
+      </joint>
+	  <joint name="l1a_tp">
+		<command_interface name="velocity">
+		  <param name="max">1</param>
+		</command_interface>
+		<state_interface name="velocity">
+		  <param name="initial_value">0.0</param>
+		</state_interface>
+		<state_interface name="position">
+		  <param name="initial_value">0.0</param>
+		</state_interface>
+      </joint> -->
+	  <joint name="J4">
+		<command_interface name="velocity">
+		  <param name="max">1</param>
+		</command_interface>
+		<state_interface name="velocity">
+		  <param name="initial_value">0.0</param>
+		</state_interface>
+		<state_interface name="position">
+		  <param name="initial_value">0.0</param>
+		</state_interface>
+      </joint>
+	  <joint name="J5">
+		<command_interface name="velocity">
+		  <param name="max">1</param>
+		</command_interface>
+		<state_interface name="velocity">
+		  <param name="initial_value">0.0</param>
+		</state_interface>
+		<state_interface name="position">
+		  <param name="initial_value">0.0</param>
+		</state_interface>
+      </joint>
+	  <joint name="J6">
+		<command_interface name="velocity">
+		  <param name="max">1</param>
+		</command_interface>
+		<state_interface name="velocity">
+		  <param name="initial_value">0.0</param>
+		</state_interface>
+		<state_interface name="position">
+		  <param name="initial_value">0.0</param>
+		</state_interface>
+      </joint>
+	  <joint name="rf_slide">
+		<command_interface name="velocity">
+		  <param name="max">1</param>
+		</command_interface>
+		<state_interface name="velocity">
+		  <param name="initial_value">0.0</param>
+		</state_interface>
+		<state_interface name="position">
+		  <param name="initial_value">0.0</param>
+		</state_interface>
+      </joint>
+	  <joint name="lf_slide">
+		<command_interface name="velocity">
+		  <param name="max">1</param>
+		</command_interface>
+		<state_interface name="velocity">
+		  <param name="initial_value">0.0</param>
+		</state_interface>
+		<state_interface name="position">
+		  <param name="initial_value">0.0</param>
+		</state_interface>
+      </joint>
+	  <joint name="actuator_head">
+		<command_interface name="velocity">
+		  <param name="max">1</param>
+		</command_interface>
+		<state_interface name="velocity">
+		  <param name="initial_value">0.0</param>
+		</state_interface>
+		<state_interface name="position">
+		  <param name="initial_value">0.0</param>
+		</state_interface>
+      </joint>
   </ros2_control>
   <gazebo>

Commit message: in progress testing

File: src/ros/rover/rover_description/arm/urdf/newarm.urdf.xacro (robot description, xacro)
@@ -195,4 +195,6 @@
         <limit effort="20" velocity="20" lower="-1.3788101090755202627" upper="3.141592653589793116"/>
         <joint_properties friction="0.5" damping="0.5"/>
+        <!-- Elbow -->
+        <mimic joint="J3" multiplier="1"/>
     </joint>
     <joint name="J2" type="revolute">
@@ -310,4 +312,5 @@
         <limit effort="20" velocity="20" lower="-1.570796326794896558" upper="3.141592653589793116"/>
         <joint_properties friction="0.5" damping="0.5"/>
+        <mimic joint="J2" multiplier="-1"/>
     </joint>
     <joint name="J3" type="revolute">
@@ -623,5 +626,23 @@
             <joint_properties damping="20.0" friction="0.1"/>
         </joint>
+        <!-- Origin of arm for IK. Should align with J1, but not -->
+        <link name="arm_kinematics_origin"/>
+        <joint name="arm_kinematics_origin_joint" type="fixed">
+            <origin xyz="0.0 0.0 0.0" rpy="0.0 0.0 0.0" />
+            <parent link="chassis" />
+            <child link="arm_kinematics_origin" />
+        </joint>
+        <!-- Origin of arm for IK -->
         <xacro:include filename="newarm_joints.xacro"/>
     </xacro:unless>
+    <xacro:if value="$(arg arm)">
+        <!-- Origin of arm for IK. Should align with J1, but not -->
+        <link name="arm_kinematics_origin"/>
+        <joint name="arm_kinematics_origin_joint" type="fixed">
+            <origin xyz="0.22899999999999565148 1.1102230246251564172e-16 0.28205202431" rpy="0.0 0.0 0.0" />
+            <parent link="chassis" />
+            <child link="arm_kinematics_origin" />
+        </joint>
+        <!-- Origin of arm for IK -->
+    </xacro:if>
 </robot>

File: src/ros/rover/rover_description/banksia_arm/urdf/arm_joints.xacro (robot description, xacro)
@@ -5,4 +5,5 @@
           <plugin filename="gz-sim-joint-state-publisher-system" name="gz::sim::systems::JointStatePublisher">
                <topic>arm_joints</topic>
+               <joint_name>arm_kinematics_origin_joint</joint_name>
                <joint_name>J1</joint_name>
                <joint_name>J2</joint_name>

Commit message: feat: INITIAL ROTATION AFTER MODE SWITCHING!!!!!!!!!!!

File: src/ros/rover/rover_description/arm/urdf/newarm.urdf.xacro (robot description, xacro)
@@ -646,3 +646,14 @@
         <!-- Origin of arm for IK -->
     </xacro:if>
+    <link name="endeffector_kinematics"/>
+    <joint name="endeffector_kinematics_joint" type="fixed">
+        <!-- before rotating to match IK function expected 0: 1.5707963 0.0 1.5707963 -->
+        <origin xyz="0.0138 0.0 -0.012512" rpy="1.5707963 0.0 1.5707963" />
+        <parent link="endeffector" />
+        <child link="endeffector_kinematics" />
+    </joint>
+<!--    z at 1.2321-->
+<!--    1.0232 0.012512 1.2183-->
+<!--    up 0.0138-->
+<!--    forward 0.012512-->
 </robot>
