Commit message: fix: uncapitalized yet more j's

File: src/ros/rover/rover_description/rover7/urdf/gz_ros2_control.xacro (robot description, xacro)
@@ -117,27 +117,27 @@
       </state_interface>
     </joint>
-        <joint name="J1">
-		<command_interface name="velocity">
-		  <param name="max">1</param>
-		</command_interface>
-		<state_interface name="velocity">
-		  <param name="initial_value">0.0</param>
-		</state_interface>
-		<state_interface name="position">
-		  <param name="initial_value">0.0</param>
-		</state_interface>
-      </joint>
-	  <joint name="J2">
-		<command_interface name="velocity">
-		  <param name="max">1</param>
-		</command_interface>
-		<state_interface name="velocity">
-		  <param name="initial_value">0.0</param>
-		</state_interface>
-		<state_interface name="position">
-		  <param name="initial_value">0.0</param>
-		</state_interface>
-      </joint>
-	  <joint name="J3">
+        <joint name="j1">
+		<command_interface name="velocity">
+		  <param name="max">1</param>
+		</command_interface>
+		<state_interface name="velocity">
+		  <param name="initial_value">0.0</param>
+		</state_interface>
+		<state_interface name="position">
+		  <param name="initial_value">0.0</param>
+		</state_interface>
+      </joint>
+	  <joint name="j2">
+		<command_interface name="velocity">
+		  <param name="max">1</param>
+		</command_interface>
+		<state_interface name="velocity">
+		  <param name="initial_value">0.0</param>
+		</state_interface>
+		<state_interface name="position">
+		  <param name="initial_value">0.0</param>
+		</state_interface>
+      </joint>
+	  <joint name="j3">
 		<command_interface name="velocity">
 		  <param name="max">1</param>
@@ -183,27 +183,27 @@
 		</state_interface>
       </joint> -->
-	  <joint name="J4">
-		<command_interface name="velocity">
-		  <param name="max">1</param>
-		</command_interface>
-		<state_interface name="velocity">
-		  <param name="initial_value">0.0</param>
-		</state_interface>
-		<state_interface name="position">
-		  <param name="initial_value">0.0</param>
-		</state_interface>
-      </joint>
-	  <joint name="J5">
-		<command_interface name="velocity">
-		  <param name="max">1</param>
-		</command_interface>
-		<state_interface name="velocity">
-		  <param name="initial_value">0.0</param>
-		</state_interface>
-		<state_interface name="position">
-		  <param name="initial_value">0.0</param>
-		</state_interface>
-      </joint>
-	  <joint name="J6">
+	  <joint name="j4">
+		<command_interface name="velocity">
+		  <param name="max">1</param>
+		</command_interface>
+		<state_interface name="velocity">
+		  <param name="initial_value">0.0</param>
+		</state_interface>
+		<state_interface name="position">
+		  <param name="initial_value">0.0</param>
+		</state_interface>
+      </joint>
+	  <joint name="j5">
+		<command_interface name="velocity">
+		  <param name="max">1</param>
+		</command_interface>
+		<state_interface name="velocity">
+		  <param name="initial_value">0.0</param>
+		</state_interface>
+		<state_interface name="position">
+		  <param name="initial_value">0.0</param>
+		</state_interface>
+      </joint>
+	  <joint name="j6">
 		<command_interface name="velocity">
 		  <param name="max">1</param>
