Commit message: feat  : convert gazebo cams into RGBD Cam

File: src/ros/rover/rover_description/rover7/urdf/auto_camera.xacro (robot description, xacro)
@@ -1,7 +1,7 @@
-<?xml version="1.0" encoding="utf-8"?>
-<!--This is a file for the depth camera plugin for the rover in gazebo. This file is referenced at the bottom of rover.urdf.xacro,
+<?xml version="1.0" encoding="utf-8" ?>
+<!--This is a file for the depth camera plugin for the rover in gazebo. This file is referenced at the bottom of rover.urdf.3,
 which is how it gets added to the gazebo sim. Author/s: Victor Bartlinski-->
-<robot xmlns:xacro="http://www.ros.org/wiki/xacro" >
-  <link name='camera_link'></link>
+<robot xmlns:xacro="http://www.ros.org/wiki/xacro">
+  <link name='camera_link' />
 <!-- Need to be fixed, OR ADD AUTO CAMERA MOUNT to URDF-->
   <joint name="camera_joint" type="fixed">
@@ -10,16 +10,36 @@
     <child link="camera_link" />
   </joint>
-  <xacro:include filename="$(find depthai_descriptions)/urdf/include/depthai_macro.urdf.xacro"/>
-  <xacro:depthai_camera camera_name = "oak" parent = "camera_link" camera_model = "OAK-D-LR"
-   base_frame = "oak-d_frame" cam_pos_x = "0.0" cam_pos_y = "0.0" cam_pos_z = "0.0"
-   cam_roll = "0.0" cam_pitch = "0.0" cam_yaw = "0.0"/>
-  <gazebo reference="oak_rgb_camera_frame">
-    <sensor name="oak/stereo" type="depth_camera">
-      <topic>oak/depth</topic>
-      <gz_frame_id>camera_link</gz_frame_id> <!-- Sets the frame_id so that rviz2 correctly transforms it -->
+  <xacro:include
+        filename="$(find depthai_descriptions)/urdf/include/depthai_macro.urdf.xacro"
+    />
+  <xacro:depthai_camera
+        camera_name="oak"
+        parent="camera_link"
+        camera_model="OAK-D-LR"
+        base_frame="oak-d_frame"
+        cam_pos_x="0.0"
+        cam_pos_y="0.0"
+        cam_pos_z="0.0"
+        cam_roll="0.0"
+        cam_pitch="0.0"
+        cam_yaw="0.0"
+    />
+  <link name='camera_link_optical' />
+  <joint name="camera_optical_joint" type="fixed">
+    <origin xyz="0.0 0 0.0" rpy="${-pi/2} 0 ${-pi/2}" />
+    <parent link="camera_link" />
+    <child link="camera_link_optical" />
+  </joint>
+  <!-- Depth Camera for Gazebo-->
+  <gazebo reference="camera_link">
+    <sensor name="oak" type="rgbd_camera">
+      <gz_frame_id>camera_link_optical</gz_frame_id>
+      <!-- Link that corresponds to the Depth Point Clouds -->
+      <optical_frame_id>camera_link</optical_frame_id>
+      <topic>oak</topic>
       <visualize>true</visualize>
       <update_rate>30</update_rate>
       <always_on>1</always_on>
-      <camera>
+      <camera name="oak">
         <horizontal_fov>${radians(82)}</horizontal_fov>
         <image>
@@ -33,26 +53,9 @@
       </camera>
       <plugin name="gz::sim::systems::Sensors" filename="gz-sim-sensors-system">
-        <frame_name>oak_rgb_camera_optical_frame</frame_name>
+        <frame_name>camera_link_optical</frame_name>
       </plugin>
     </sensor>
-    <sensor name="oak/rgb" type="camera">
-      <topic>oak/rgb</topic>
-      <visualize>true</visualize>
-      <update_rate>30</update_rate>
-      <always_on>1</always_on>
-      <camera>
-        <horizontal_fov>${radians(82)}</horizontal_fov>
-        <image>
-          <width>600</width>
-          <height>400</height>
-        </image>
-        <clip>
-          <near>0.4</near>
-          <far>100.0</far>
-        </clip>
-      </camera>
-      <!-- <plugin name="gz::sim::systems::Sensors" filename="gz-sim-sensors-system"></plugin> -->
-    </sensor>
   </gazebo>
+  <!-- IMU for Gazebo-->
   <gazebo reference="oak_imu_frame">
     <sensor name="imu_sensor" type="imu">
@@ -60,5 +63,6 @@
       <plugin filename="gz-sim-imu-system" name="gz::sim::systems::Imu">
         <frame_name>oak_imu_frame</frame_name>
-        <initial_orientation_as_reference>false</initial_orientation_as_reference>
+        <initial_orientation_as_reference
+                >false</initial_orientation_as_reference>
       </plugin>
       <always_on>true</always_on>

Commit message: more cleanups

File: src/ros/rover/rover_description/rover7/urdf/auto_camera.xacro (robot description, xacro)
@@ -1,33 +1,31 @@
 <?xml version="1.0" encoding="utf-8" ?>
-<!--This is a file for the depth camera plugin for the rover in gazebo. This file is referenced at the bottom of rover.urdf.3,
-which is how it gets added to the gazebo sim. Author/s: Victor Bartlinski-->
+<!--This is a file for the depth camera plugin for the rover in gazebo. This file is referenced at the bottom of rover.urdf.xacro,
+which is how it gets added to the gazebo sim. Edited by: Victor Bartlinski, Kabi Velmurugan Sujatha -->
 <robot xmlns:xacro="http://www.ros.org/wiki/xacro">
-  <link name='camera_link' />
+  <link name="camera_link"/>
 <!-- Need to be fixed, OR ADD AUTO CAMERA MOUNT to URDF-->
   <joint name="camera_joint" type="fixed">
-    <origin xyz="0.26 0 0.2" rpy="0 0 0" />
-    <parent link="chassis" />
-    <child link="camera_link" />
+    <origin xyz="0.26 0 0.2" rpy="0 0 0"/>
+    <parent link="chassis"/>
+    <child link="camera_link"/>
   </joint>
-  <xacro:include
-        filename="$(find depthai_descriptions)/urdf/include/depthai_macro.urdf.xacro"
-    />
+  <xacro:include filename="$(find depthai_descriptions)/urdf/include/depthai_macro.urdf.xacro"/>
   <xacro:depthai_camera
-        camera_name="oak"
-        parent="camera_link"
-        camera_model="OAK-D-LR"
-        base_frame="oak-d_frame"
-        cam_pos_x="0.0"
-        cam_pos_y="0.0"
-        cam_pos_z="0.0"
-        cam_roll="0.0"
-        cam_pitch="0.0"
-        cam_yaw="0.0"
-    />
-  <link name='camera_link_optical' />
+    camera_name="oak"
+    parent="camera_link"
+    camera_model="OAK-D-LR"
+    base_frame="oak-d_frame"
+    cam_pos_x="0.0"
+    cam_pos_y="0.0"
+    cam_pos_z="0.0"
+    cam_roll="0.0"
+    cam_pitch="0.0"
+    cam_yaw="0.0"
+  />
+  <link name="camera_link_optical"/>
   <joint name="camera_optical_joint" type="fixed">
-    <origin xyz="0.0 0 0.0" rpy="${-pi/2} 0 ${-pi/2}" />
-    <parent link="camera_link" />
-    <child link="camera_link_optical" />
+    <origin xyz="0.0 0 0.0" rpy="${-pi/2} 0 ${-pi/2}"/>
+    <parent link="camera_link"/>
+    <child link="camera_link_optical"/>
   </joint>
   <!-- Depth Camera for Gazebo-->
@@ -63,6 +61,5 @@
       <plugin filename="gz-sim-imu-system" name="gz::sim::systems::Imu">
         <frame_name>oak_imu_frame</frame_name>
-        <initial_orientation_as_reference
-                >false</initial_orientation_as_reference>
+        <initial_orientation_as_reference>false</initial_orientation_as_reference>
       </plugin>
       <always_on>true</always_on>
