Commit message: fix

File: src/ros/rover/rover_description/rover7/urdf/auto_camera.xacro (robot description, xacro)
@@ -3,122 +3,124 @@
 which is how it gets added to the gazebo sim. Edited by: Victor Bartlinski, Kabi Velmurugan Sujatha -->
 <robot xmlns:xacro="http://www.ros.org/wiki/xacro">
-  <link name="camera_link"/>
-<!-- Need to be fixed, OR ADD AUTO CAMERA MOUNT to URDF-->
-  <joint name="camera_joint" type="fixed">
-    <origin xyz="0.26 0 0.2" rpy="0 0 0"/>
-    <parent link="chassis"/>
-    <child link="camera_link"/>
-  </joint>
-  <xacro:include filename="$(find depthai_descriptions)/urdf/include/depthai_macro.urdf.xacro"/>
-  <xacro:depthai_camera
-    camera_name="oak"
-    parent="camera_link"
-    camera_model="OAK-D-LR"
-    base_frame="oak-d_frame"
-    cam_pos_x="0.0"
-    cam_pos_y="0.0"
-    cam_pos_z="0.0"
-    cam_roll="0.0"
-    cam_pitch="0.0"
-    cam_yaw="0.0"
-  />
-  <link name="camera_link_optical"/>
-  <joint name="camera_optical_joint" type="fixed">
-    <origin xyz="0.0 0 0.0" rpy="${-pi/2} 0 ${-pi/2}"/>
-    <parent link="camera_link"/>
-    <child link="camera_link_optical"/>
-  </joint>
-  <!-- Depth Camera for Gazebo-->
-  <gazebo reference="camera_link">
-    <sensor name="oak" type="rgbd_camera">
-      <gz_frame_id>camera_link_optical</gz_frame_id>
-      <!-- Link that corresponds to the Depth Point Clouds -->
-      <optical_frame_id>camera_link</optical_frame_id>
-      <topic>oak</topic>
-      <visualize>true</visualize>
-      <update_rate>30</update_rate>
-      <always_on>1</always_on>
-      <camera name="oak">
-        <horizontal_fov>${radians(82)}</horizontal_fov>
-        <image>
-          <width>1280</width>
-          <height>900</height>
-        </image>
-        <clip>
-          <near>0.4</near>
-          <far>10.0</far>
-        </clip>
-      </camera>
-      <plugin name="gz::sim::systems::Sensors" filename="gz-sim-sensors-system">
-        <frame_name>camera_link_optical</frame_name>
-      </plugin>
-    </sensor>
-  </gazebo>
-  <!-- IMU for Gazebo-->
-  <gazebo reference="oak_imu_frame">
-    <sensor name="imu_sensor" type="imu">
-      <topic>oak/imu</topic>
-      <plugin filename="gz-sim-imu-system" name="gz::sim::systems::Imu">
-        <frame_name>oak_imu_frame</frame_name>
-        <initial_orientation_as_reference>false</initial_orientation_as_reference>
-      </plugin>
-      <always_on>true</always_on>
-      <update_rate>200</update_rate>
-      <visualize>true</visualize>
-      <imu>
-        <angular_velocity>
-          <x>
-            <noise type="gaussian">
-              <mean>0.0</mean>
-              <stddev>2e-4</stddev>
-              <bias_mean>0.0000075</bias_mean>
-              <bias_stddev>0.0000008</bias_stddev>
-            </noise>
-          </x>
-          <y>
-            <noise type="gaussian">
-              <mean>0.0</mean>
-              <stddev>2e-4</stddev>
-              <bias_mean>0.0000075</bias_mean>
-              <bias_stddev>0.0000008</bias_stddev>
-            </noise>
-          </y>
-          <z>
-            <noise type="gaussian">
-              <mean>0.0</mean>
-              <stddev>2e-4</stddev>
-              <bias_mean>0.0000075</bias_mean>
-              <bias_stddev>0.0000008</bias_stddev>
-            </noise>
-          </z>
-        </angular_velocity>
-        <linear_acceleration>
-          <x>
-            <noise type="gaussian">
-              <mean>0.0</mean>
-              <stddev>1.7e-2</stddev>
-              <bias_mean>0.1</bias_mean>
-              <bias_stddev>0.001</bias_stddev>
-            </noise>
-          </x>
-          <y>
-            <noise type="gaussian">
-              <mean>0.0</mean>
-              <stddev>1.7e-2</stddev>
-              <bias_mean>0.1</bias_mean>
-              <bias_stddev>0.001</bias_stddev>
-            </noise>
-          </y>
-          <z>
-            <noise type="gaussian">
-              <mean>0.0</mean>
-              <stddev>1.7e-2</stddev>
-              <bias_mean>0.1</bias_mean>
-              <bias_stddev>0.001</bias_stddev>
-            </noise>
-          </z>
-        </linear_acceleration>
-      </imu>
-    </sensor>
-  </gazebo>
+  <xacro:macro name="auto_cam" params="angle">
+    <link name="camera_link"/>
+  <!-- Need to be fixed, OR ADD AUTO CAMERA MOUNT to URDF-->
+    <joint name="camera_joint" type="fixed">
+      <origin xyz="0.26 0 0.2" rpy="0 ${angle} 0"/>
+      <parent link="chassis"/>
+      <child link="camera_link"/>
+    </joint>
+    <xacro:include filename="$(find depthai_descriptions)/urdf/include/depthai_macro.urdf.xacro"/>
+    <xacro:depthai_camera
+      camera_name="oak"
+      parent="camera_link"
+      camera_model="OAK-D-LR"
+      base_frame="oak-d_frame"
+      cam_pos_x="0.0"
+      cam_pos_y="0.0"
+      cam_pos_z="0.0"
+      cam_roll="0.0"
+      cam_pitch="0.0"
+      cam_yaw="0.0"
+    />
+    <link name="camera_link_optical"/>
+    <joint name="camera_optical_joint" type="fixed">
+      <origin xyz="0.0 0 0.0" rpy="${-pi/2} 0 ${-pi/2}"/>
+      <parent link="camera_link"/>
+      <child link="camera_link_optical"/>
+    </joint>
+    <!-- Depth Camera for Gazebo-->
+    <gazebo reference="camera_link">
+      <sensor name="oak" type="rgbd_camera">
+        <gz_frame_id>camera_link_optical</gz_frame_id>
+        <!-- Link that corresponds to the Depth Point Clouds -->
+        <optical_frame_id>camera_link</optical_frame_id>
+        <topic>oak</topic>
+        <visualize>true</visualize>
+        <update_rate>30</update_rate>
+        <always_on>1</always_on>
+        <camera name="oak">
+          <horizontal_fov>${radians(82)}</horizontal_fov>
+          <image>
+            <width>1280</width>
+            <height>900</height>
+          </image>
+          <clip>
+            <near>0.4</near>
+            <far>10.0</far>
+          </clip>
+        </camera>
+        <plugin name="gz::sim::systems::Sensors" filename="gz-sim-sensors-system">
+          <frame_name>camera_link_optical</frame_name>
+        </plugin>
+      </sensor>
+    </gazebo>
+    <!-- IMU for Gazebo-->
+    <gazebo reference="oak_imu_frame">
+      <sensor name="imu_sensor" type="imu">
+        <topic>oak/imu</topic>
+        <plugin filename="gz-sim-imu-system" name="gz::sim::systems::Imu">
+          <frame_name>oak_imu_frame</frame_name>
+          <initial_orientation_as_reference>false</initial_orientation_as_reference>
+        </plugin>
+        <always_on>true</always_on>
+        <update_rate>200</update_rate>
+        <visualize>true</visualize>
+        <imu>
+          <angular_velocity>
+            <x>
+              <noise type="gaussian">
+                <mean>0.0</mean>
+                <stddev>2e-4</stddev>
+                <bias_mean>0.0000075</bias_mean>
+                <bias_stddev>0.0000008</bias_stddev>
+              </noise>
+            </x>
+            <y>
+              <noise type="gaussian">
+                <mean>0.0</mean>
+                <stddev>2e-4</stddev>
+                <bias_mean>0.0000075</bias_mean>
+                <bias_stddev>0.0000008</bias_stddev>
+              </noise>
+            </y>
+            <z>
+              <noise type="gaussian">
+                <mean>0.0</mean>
+                <stddev>2e-4</stddev>
+                <bias_mean>0.0000075</bias_mean>
+                <bias_stddev>0.0000008</bias_stddev>
+              </noise>
+            </z>
+          </angular_velocity>
+          <linear_acceleration>
+            <x>
+              <noise type="gaussian">
+                <mean>0.0</mean>
+                <stddev>1.7e-2</stddev>
+                <bias_mean>0.1</bias_mean>
+                <bias_stddev>0.001</bias_stddev>
+              </noise>
+            </x>
+            <y>
+              <noise type="gaussian">
+                <mean>0.0</mean>
+                <stddev>1.7e-2</stddev>
+                <bias_mean>0.1</bias_mean>
+                <bias_stddev>0.001</bias_stddev>
+              </noise>
+            </y>
+            <z>
+              <noise type="gaussian">
+                <mean>0.0</mean>
+                <stddev>1.7e-2</stddev>
+                <bias_mean>0.1</bias_mean>
+                <bias_stddev>0.001</bias_stddev>
+              </noise>
+            </z>
+          </linear_acceleration>
+        </imu>
+      </sensor>
+    </gazebo>
+  </xacro:macro>
 </robot>

File: src/ros/rover/rover_description/waratah/urdf/auto_camera.xacro (robot description, xacro)
@@ -3,122 +3,120 @@
 which is how it gets added to the gazebo sim. Author/s: Victor Bartlinski-->
 <robot xmlns:xacro="http://www.ros.org/wiki/xacro" >
-  <xacro:macro name="auto_cam" params="angle">
-    <link name='camera_link'></link>
-    <joint name="camera_joint" type="fixed">
-      <origin xyz="0.49 0 0.48" rpy="0 ${angle} 0" />
-      <parent link="base_link" />
-      <child link="camera_link" />
-    </joint>
-    <xacro:include filename="$(find depthai_descriptions)/urdf/include/depthai_macro.urdf.xacro"/>
-    <xacro:depthai_camera camera_name = "oak" parent = "camera_link" camera_model = "OAK-D-LR"
-    base_frame = "oak-d_frame" cam_pos_x = "0.0" cam_pos_y = "0.0" cam_pos_z = "0.0"
-    cam_roll = "0.0" cam_pitch = "0.0" cam_yaw = "0.0"/>
-    <gazebo reference="oak_rgb_camera_frame">
-      <sensor name="oak/stereo" type="depth_camera">
-        <topic>oak/depth</topic>
-        <gz_frame_id>camera_link</gz_frame_id> <!-- Sets the frame_id so that rviz2 correctly transforms it -->
-        <visualize>true</visualize>
-        <update_rate>30</update_rate>
-        <always_on>1</always_on>
-        <camera>
-          <horizontal_fov>${radians(82)}</horizontal_fov>
-          <image>
-            <width>600</width>
-            <height>400</height>
-          </image>
-          <clip>
-            <near>0.4</near>
-            <far>100.0</far>
-          </clip>
-        </camera>
-        <plugin name="gz::sim::systems::Sensors" filename="gz-sim-sensors-system">
-          <frame_name>oak_rgb_camera_optical_frame</frame_name>
-        </plugin>
-      </sensor>
-      <sensor name="oak/rgb" type="camera">
-        <topic>oak/rgb</topic>
-        <visualize>true</visualize>
-        <update_rate>30</update_rate>
-        <always_on>1</always_on>
-        <camera>
-          <horizontal_fov>${radians(82)}</horizontal_fov>
-          <image>
-            <width>600</width>
-            <height>400</height>
-          </image>
-          <clip>
-            <near>0.4</near>
-            <far>100.0</far>
-          </clip>
-        </camera>
-        <!-- <plugin name="gz::sim::systems::Sensors" filename="gz-sim-sensors-system"></plugin> -->
-      </sensor>
-    </gazebo>
-    <gazebo reference="oak_imu_frame">
-      <sensor name="imu_sensor" type="imu">
-        <topic>oak/imu</topic>
-        <plugin filename="gz-sim-imu-system" name="gz::sim::systems::Imu">
-          <frame_name>oak_imu_frame</frame_name>
-          <initial_orientation_as_reference>false</initial_orientation_as_reference>
-        </plugin>
-        <always_on>true</always_on>
-        <update_rate>200</update_rate>
-        <visualize>true</visualize>
-        <imu>
-          <angular_velocity>
-            <x>
-              <noise type="gaussian">
-                <mean>0.0</mean>
-                <stddev>2e-4</stddev>
-                <bias_mean>0.0000075</bias_mean>
-                <bias_stddev>0.0000008</bias_stddev>
-              </noise>
-            </x>
-            <y>
-              <noise type="gaussian">
-                <mean>0.0</mean>
-                <stddev>2e-4</stddev>
-                <bias_mean>0.0000075</bias_mean>
-                <bias_stddev>0.0000008</bias_stddev>
-              </noise>
-            </y>
-            <z>
-              <noise type="gaussian">
-                <mean>0.0</mean>
-                <stddev>2e-4</stddev>
-                <bias_mean>0.0000075</bias_mean>
-                <bias_stddev>0.0000008</bias_stddev>
-              </noise>
-            </z>
-          </angular_velocity>
-          <linear_acceleration>
-            <x>
-              <noise type="gaussian">
-                <mean>0.0</mean>
-                <stddev>1.7e-2</stddev>
-                <bias_mean>0.1</bias_mean>
-                <bias_stddev>0.001</bias_stddev>
-              </noise>
-            </x>
-            <y>
-              <noise type="gaussian">
-                <mean>0.0</mean>
-                <stddev>1.7e-2</stddev>
-                <bias_mean>0.1</bias_mean>
-                <bias_stddev>0.001</bias_stddev>
-              </noise>
-            </y>
-            <z>
-              <noise type="gaussian">
-                <mean>0.0</mean>
-                <stddev>1.7e-2</stddev>
-                <bias_mean>0.1</bias_mean>
-                <bias_stddev>0.001</bias_stddev>
-              </noise>
-            </z>
-          </linear_acceleration>
-        </imu>
-      </sensor>
-    </gazebo>
-  </xacro:macro>
+  <link name='camera_link'></link>
+  <joint name="camera_joint" type="fixed">
+    <origin xyz="0.49 0 0.48" rpy="0 0 0" />
+    <parent link="base_link" />
+    <child link="camera_link" />
+  </joint>
+  <xacro:include filename="$(find depthai_descriptions)/urdf/include/depthai_macro.urdf.xacro"/>
+  <xacro:depthai_camera camera_name = "oak" parent = "camera_link" camera_model = "OAK-D-LR"
+   base_frame = "oak-d_frame" cam_pos_x = "0.0" cam_pos_y = "0.0" cam_pos_z = "0.0"
+   cam_roll = "0.0" cam_pitch = "0.0" cam_yaw = "0.0"/>
+  <gazebo reference="oak_rgb_camera_frame">
+    <sensor name="oak/stereo" type="depth_camera">
+      <topic>oak/depth</topic>
+      <gz_frame_id>camera_link</gz_frame_id> <!-- Sets the frame_id so that rviz2 correctly transforms it -->
+      <visualize>true</visualize>
+      <update_rate>30</update_rate>
+      <always_on>1</always_on>
+      <camera>
+        <horizontal_fov>${radians(82)}</horizontal_fov>
+        <image>
+          <width>600</width>
+          <height>400</height>
+        </image>
+        <clip>
+          <near>0.4</near>
+          <far>100.0</far>
+        </clip>
+      </camera>
+      <plugin name="gz::sim::systems::Sensors" filename="gz-sim-sensors-system">
+        <frame_name>oak_rgb_camera_optical_frame</frame_name>
+      </plugin>
+    </sensor>
+    <sensor name="oak/rgb" type="camera">
+      <topic>oak/rgb</topic>
+      <visualize>true</visualize>
+      <update_rate>30</update_rate>
+      <always_on>1</always_on>
+      <camera>
+        <horizontal_fov>${radians(82)}</horizontal_fov>
+        <image>
+          <width>600</width>
+          <height>400</height>
+        </image>
+        <clip>
+          <near>0.4</near>
+          <far>100.0</far>
+        </clip>
+      </camera>
+      <!-- <plugin name="gz::sim::systems::Sensors" filename="gz-sim-sensors-system"></plugin> -->
+    </sensor>
+  </gazebo>
+  <gazebo reference="oak_imu_frame">
+    <sensor name="imu_sensor" type="imu">
+      <topic>oak/imu</topic>
+      <plugin filename="gz-sim-imu-system" name="gz::sim::systems::Imu">
+        <frame_name>oak_imu_frame</frame_name>
+        <initial_orientation_as_reference>false</initial_orientation_as_reference>
+      </plugin>
+      <always_on>true</always_on>
+      <update_rate>200</update_rate>
+      <visualize>true</visualize>
+      <imu>
+        <angular_velocity>
+          <x>
+            <noise type="gaussian">
+              <mean>0.0</mean>
+              <stddev>2e-4</stddev>
+              <bias_mean>0.0000075</bias_mean>
+              <bias_stddev>0.0000008</bias_stddev>
+            </noise>
+          </x>
+          <y>
+            <noise type="gaussian">
+              <mean>0.0</mean>
+              <stddev>2e-4</stddev>
+              <bias_mean>0.0000075</bias_mean>
+              <bias_stddev>0.0000008</bias_stddev>
+            </noise>
+          </y>
+          <z>
+            <noise type="gaussian">
+              <mean>0.0</mean>
+              <stddev>2e-4</stddev>
+              <bias_mean>0.0000075</bias_mean>
+              <bias_stddev>0.0000008</bias_stddev>
+            </noise>
+          </z>
+        </angular_velocity>
+        <linear_acceleration>
+          <x>
+            <noise type="gaussian">
+              <mean>0.0</mean>
+              <stddev>1.7e-2</stddev>
+              <bias_mean>0.1</bias_mean>
+              <bias_stddev>0.001</bias_stddev>
+            </noise>
+          </x>
+          <y>
+            <noise type="gaussian">
+              <mean>0.0</mean>
+              <stddev>1.7e-2</stddev>
+              <bias_mean>0.1</bias_mean>
+              <bias_stddev>0.001</bias_stddev>
+            </noise>
+          </y>
+          <z>
+            <noise type="gaussian">
+              <mean>0.0</mean>
+              <stddev>1.7e-2</stddev>
+              <bias_mean>0.1</bias_mean>
+              <bias_stddev>0.001</bias_stddev>
+            </noise>
+          </z>
+        </linear_acceleration>
+      </imu>
+    </sensor>
+  </gazebo>
 </robot>

Commit message: feat : add bootie_camera_link

File: src/ros/rover/rover_description/rover7/urdf/auto_camera.xacro (robot description, xacro)
@@ -3,29 +3,38 @@
 which is how it gets added to the gazebo sim. Edited by: Victor Bartlinski, Kabi Velmurugan Sujatha -->
 <robot xmlns:xacro="http://www.ros.org/wiki/xacro">
-  <link name="camera_link"/>
+  <link name="camera_link" />
 <!-- Need to be fixed, OR ADD AUTO CAMERA MOUNT to URDF-->
   <joint name="camera_joint" type="fixed">
-    <origin xyz="0.26 0 0.2" rpy="0 0 0"/>
-    <parent link="chassis"/>
-    <child link="camera_link"/>
+    <origin xyz="0.795 0 0.535" rpy="0 0 0" />
+    <parent link="chassis" />
+    <child link="camera_link" />
   </joint>
-  <xacro:include filename="$(find depthai_descriptions)/urdf/include/depthai_macro.urdf.xacro"/>
+  <link name="bootie_camera_link" />
+<!-- Need to be fixed, OR ADD AUTO CAMERA MOUNT to URDF-->
+  <joint name="bootie_camera_joint" type="fixed">
+    <origin xyz="-0.330 0 0.115" rpy="0 0 0" />
+    <parent link="chassis" />
+    <child link="bootie_camera_link" />
+  </joint>
+  <xacro:include
+        filename="$(find depthai_descriptions)/urdf/include/depthai_macro.urdf.xacro"
+    />
   <xacro:depthai_camera
-    camera_name="oak"
-    parent="camera_link"
-    camera_model="OAK-D-LR"
-    base_frame="oak-d_frame"
-    cam_pos_x="0.0"
-    cam_pos_y="0.0"
-    cam_pos_z="0.0"
-    cam_roll="0.0"
-    cam_pitch="0.0"
-    cam_yaw="0.0"
-  />
-  <link name="camera_link_optical"/>
+        camera_name="oak"
+        parent="camera_link"
+        camera_model="OAK-D-LR"
+        base_frame="oak-d_frame"
+        cam_pos_x="0.0"
+        cam_pos_y="0.0"
+        cam_pos_z="0.0"
+        cam_roll="0.0"
+        cam_pitch="0.0"
+        cam_yaw="0.0"
+    />
+  <link name="camera_link_optical" />
   <joint name="camera_optical_joint" type="fixed">
-    <origin xyz="0.0 0 0.0" rpy="${-pi/2} 0 ${-pi/2}"/>
-    <parent link="camera_link"/>
-    <child link="camera_link_optical"/>
+    <origin xyz="0.0 0 0.0" rpy="${-pi/2} 0 ${-pi/2}" />
+    <parent link="camera_link" />
+    <child link="camera_link_optical" />
   </joint>
   <!-- Depth Camera for Gazebo-->
@@ -61,5 +70,6 @@
       <plugin filename="gz-sim-imu-system" name="gz::sim::systems::Imu">
         <frame_name>oak_imu_frame</frame_name>
-        <initial_orientation_as_reference>false</initial_orientation_as_reference>
+        <initial_orientation_as_reference
+                >false</initial_orientation_as_reference>
       </plugin>
       <always_on>true</always_on>

Commit message: fix: hardcode cam angles

File: src/ros/rover/rover_description/rover7/urdf/auto_camera.xacro (robot description, xacro)
@@ -6,5 +6,5 @@
 <!-- Need to be fixed, OR ADD AUTO CAMERA MOUNT to URDF-->
   <joint name="camera_joint" type="fixed">
-    <origin xyz="0.795 0 0.535" rpy="0 0 0" />
+    <origin xyz="0.795 0 0.535" rpy="0 0.5236 0" />
     <parent link="chassis" />
     <child link="camera_link" />
@@ -13,5 +13,5 @@
 <!-- Need to be fixed, OR ADD AUTO CAMERA MOUNT to URDF-->
   <joint name="bootie_camera_joint" type="fixed">
-    <origin xyz="-0.330 0 0.115" rpy="0 0 0" />
+    <origin xyz="-0.330 0 0.115" rpy="0 0.5236 0" />
     <parent link="chassis" />
     <child link="bootie_camera_link" />

Commit message: fix : add d455 description

File: src/ros/rover/rover_description/rover7/urdf/auto_camera.xacro (robot description, xacro)
@@ -9,11 +9,4 @@
     <parent link="chassis" />
     <child link="camera_link" />
-  </joint>
-  <link name="bootie_camera_link" />
-<!-- Need to be fixed, OR ADD AUTO CAMERA MOUNT to URDF-->
-  <joint name="bootie_camera_joint" type="fixed">
-    <origin xyz="-0.330 0 0.115" rpy="0 0.5236 0" />
-    <parent link="chassis" />
-    <child link="bootie_camera_link" />
   </joint>
   <xacro:include
@@ -38,4 +31,20 @@
     <child link="camera_link_optical" />
   </joint>
+  <link name='bootie_camera_link' />
+    <joint name="bootie_camera_joint" type="fixed">
+      <origin xyz="-0.437 0 0.280" rpy="0 0.523599 0" />
+      <parent link="chassis" />
+      <child link="bootie_camera_link" />
+    </joint>
+    <xacro:include
+        filename="$(find realsense2_description)/urdf/_d455.urdf.xacro"
+    />
+    <xacro:sensor_d455
+        name="bootie"
+        parent="bootie_camera_link"
+        use_nominal_extrinsics="true"
+    >
+      <origin xyz="0 0 0" rpy="0 0 0" />
+    </xacro:sensor_d455>
   <!-- Depth Camera for Gazebo-->
   <gazebo reference="camera_link">

Commit message: fix : rotate cam to face bootie

File: src/ros/rover/rover_description/rover7/urdf/auto_camera.xacro (robot description, xacro)
@@ -33,5 +33,5 @@
   <link name='bootie_camera_link' />
     <joint name="bootie_camera_joint" type="fixed">
-      <origin xyz="-0.437 0 0.280" rpy="0 0.523599 0" />
+      <origin xyz="-0.437 0 0.280" rpy="0 0.523599 3.14" />
       <parent link="chassis" />
       <child link="bootie_camera_link" />
