Commit message: feat : camera.launch is a piece of crap

File: src/ros/rover/rover_description/rover7/urdf/auto_camera.xacro (robot description, xacro)
@@ -3,124 +3,144 @@
 which is how it gets added to the gazebo sim. Edited by: Victor Bartlinski, Kabi Velmurugan Sujatha -->
 <robot xmlns:xacro="http://www.ros.org/wiki/xacro">
-  <xacro:macro name="auto_cam" params="angle">
-    <link name="camera_link"/>
-  <!-- Need to be fixed, OR ADD AUTO CAMERA MOUNT to URDF-->
-    <joint name="camera_joint" type="fixed">
-      <origin xyz="0.8 0 0.525" rpy="0 ${angle*(pi/180)} 0"/>
-      <parent link="chassis"/>
-      <child link="camera_link"/>
-    </joint>
-    <xacro:include filename="$(find depthai_descriptions)/urdf/include/depthai_macro.urdf.xacro"/>
+ <xacro:include
+        filename="$(find depthai_descriptions)/urdf/include/depthai_macro.urdf.xacro"
+    />
+  <link name="camera_link" />
+<!-- Need to be fixed, OR ADD AUTO CAMERA MOUNT to URDF-->
+  <joint name="camera_joint" type="fixed">
+    <origin xyz="0.26 0 0.2" rpy="0 0 0" />
+    <parent link="chassis" />
+    <child link="camera_link" />
+  </joint>
     <xacro:depthai_camera
-      camera_name="oak"
-      parent="camera_link"
-      camera_model="OAK-D-LR"
-      base_frame="oak-d_frame"
-      cam_pos_x="0.0"
-      cam_pos_y="0.0"
-      cam_pos_z="0.0"
-      cam_roll="0.0"
-      cam_pitch="0.0"
-      cam_yaw="0.0"
+        camera_name="oak"
+        parent="camera_link"
+        camera_model="OAK-D-LR"
+        base_frame="oak-base-frame"
+        cam_pos_x="0.0"
+        cam_pos_y="0.0"
+        cam_pos_z="0.0"
+        cam_roll="0.0"
+        cam_pitch="0.0"
+        cam_yaw="0.0"
     />
-    <link name="camera_link_optical"/>
-    <joint name="camera_optical_joint" type="fixed">
-      <origin xyz="0.0 0 0.0" rpy="${-pi/2} 0 ${-pi/2}"/>
-      <parent link="camera_link"/>
-      <child link="camera_link_optical"/>
-    </joint>
-    <!-- Depth Camera for Gazebo-->
-    <gazebo reference="camera_link">
-      <sensor name="oak" type="rgbd_camera">
-        <gz_frame_id>camera_link_optical</gz_frame_id>
-        <!-- Link that corresponds to the Depth Point Clouds -->
-        <optical_frame_id>camera_link</optical_frame_id>
-        <topic>oak</topic>
-        <visualize>true</visualize>
-        <update_rate>30</update_rate>
-        <always_on>1</always_on>
-        <camera name="oak">
-          <horizontal_fov>${radians(82)}</horizontal_fov>
-          <image>
-            <width>1280</width>
-            <height>900</height>
-          </image>
-          <clip>
-            <near>0.4</near>
-            <far>10.0</far>
-          </clip>
-        </camera>
-        <plugin name="gz::sim::systems::Sensors" filename="gz-sim-sensors-system">
-          <frame_name>camera_link_optical</frame_name>
-        </plugin>
-      </sensor>
-    </gazebo>
-    <!-- IMU for Gazebo-->
-    <gazebo reference="oak_imu_frame">
-      <sensor name="imu_sensor" type="imu">
-        <topic>oak/imu</topic>
-        <plugin filename="gz-sim-imu-system" name="gz::sim::systems::Imu">
-          <frame_name>oak_imu_frame</frame_name>
-          <initial_orientation_as_reference>false</initial_orientation_as_reference>
-        </plugin>
-        <always_on>true</always_on>
-        <update_rate>200</update_rate>
-        <visualize>true</visualize>
-        <imu>
-          <angular_velocity>
-            <x>
-              <noise type="gaussian">
-                <mean>0.0</mean>
-                <stddev>2e-4</stddev>
-                <bias_mean>0.0000075</bias_mean>
-                <bias_stddev>0.0000008</bias_stddev>
-              </noise>
-            </x>
-            <y>
-              <noise type="gaussian">
-                <mean>0.0</mean>
-                <stddev>2e-4</stddev>
-                <bias_mean>0.0000075</bias_mean>
-                <bias_stddev>0.0000008</bias_stddev>
-              </noise>
-            </y>
-            <z>
-              <noise type="gaussian">
-                <mean>0.0</mean>
-                <stddev>2e-4</stddev>
-                <bias_mean>0.0000075</bias_mean>
-                <bias_stddev>0.0000008</bias_stddev>
-              </noise>
-            </z>
-          </angular_velocity>
-          <linear_acceleration>
-            <x>
-              <noise type="gaussian">
-                <mean>0.0</mean>
-                <stddev>1.7e-2</stddev>
-                <bias_mean>0.1</bias_mean>
-                <bias_stddev>0.001</bias_stddev>
-              </noise>
-            </x>
-            <y>
-              <noise type="gaussian">
-                <mean>0.0</mean>
-                <stddev>1.7e-2</stddev>
-                <bias_mean>0.1</bias_mean>
-                <bias_stddev>0.001</bias_stddev>
-              </noise>
-            </y>
-            <z>
-              <noise type="gaussian">
-                <mean>0.0</mean>
-                <stddev>1.7e-2</stddev>
-                <bias_mean>0.1</bias_mean>
-                <bias_stddev>0.001</bias_stddev>
-              </noise>
-            </z>
-          </linear_acceleration>
-        </imu>
-      </sensor>
-    </gazebo>
-  </xacro:macro>
+  <link name="bootie_link" />
+<!-- Need to be fixed, OR ADD AUTO CAMERA MOUNT to URDF-->
+  <joint name="bootie_joint" type="fixed">
+    <origin xyz="0.20 0 0.19" rpy="0 0 3.14" />
+    <parent link="chassis" />
+    <child link="bootie_link" />
+  </joint>
+  <xacro:depthai_camera
+        camera_name="bootie"
+        parent="bootie_link"
+        camera_model="OAK-D-LR"
+        base_frame="bootie-base-frame"
+        cam_pos_x="0.0"
+        cam_pos_y="0.0"
+        cam_pos_z="0.0"
+        cam_roll="0.0"
+        cam_pitch="0.0"
+        cam_yaw="0.0"
+    />
+  <link name="camera_link_optical" />
+  <joint name="camera_optical_joint" type="fixed">
+    <origin xyz="0.0 0 0.0" rpy="${-pi/2} 0 ${-pi/2}" />
+    <parent link="camera_link" />
+    <child link="camera_link_optical" />
+  </joint>
+  <!-- Depth Camera for Gazebo-->
+  <gazebo reference="camera_link">
+    <sensor name="oak" type="rgbd_camera">
+      <gz_frame_id>camera_link_optical</gz_frame_id>
+      <!-- Link that corresponds to the Depth Point Clouds -->
+      <optical_frame_id>camera_link</optical_frame_id>
+      <topic>oak</topic>
+      <visualize>true</visualize>
+      <update_rate>30</update_rate>
+      <always_on>1</always_on>
+      <camera name="oak">
+        <horizontal_fov>${radians(82)}</horizontal_fov>
+        <image>
+          <width>1280</width>
+          <height>900</height>
+        </image>
+        <clip>
+          <near>0.4</near>
+          <far>10.0</far>
+        </clip>
+      </camera>
+      <plugin name="gz::sim::systems::Sensors" filename="gz-sim-sensors-system">
+        <frame_name>camera_link_optical</frame_name>
+      </plugin>
+    </sensor>
+  </gazebo>
+  <!-- IMU for Gazebo-->
+  <gazebo reference="oak_imu_frame">
+    <sensor name="imu_sensor" type="imu">
+      <topic>oak/imu</topic>
+      <plugin filename="gz-sim-imu-system" name="gz::sim::systems::Imu">
+        <frame_name>oak_imu_frame</frame_name>
+        <initial_orientation_as_reference
+                >false</initial_orientation_as_reference>
+      </plugin>
+      <always_on>true</always_on>
+      <update_rate>200</update_rate>
+      <visualize>true</visualize>
+      <imu>
+        <angular_velocity>
+          <x>
+            <noise type="gaussian">
+              <mean>0.0</mean>
+              <stddev>2e-4</stddev>
+              <bias_mean>0.0000075</bias_mean>
+              <bias_stddev>0.0000008</bias_stddev>
+            </noise>
+          </x>
+          <y>
+            <noise type="gaussian">
+              <mean>0.0</mean>
+              <stddev>2e-4</stddev>
+              <bias_mean>0.0000075</bias_mean>
+              <bias_stddev>0.0000008</bias_stddev>
+            </noise>
+          </y>
+          <z>
+            <noise type="gaussian">
+              <mean>0.0</mean>
+              <stddev>2e-4</stddev>
+              <bias_mean>0.0000075</bias_mean>
+              <bias_stddev>0.0000008</bias_stddev>
+            </noise>
+          </z>
+        </angular_velocity>
+        <linear_acceleration>
+          <x>
+            <noise type="gaussian">
+              <mean>0.0</mean>
+              <stddev>1.7e-2</stddev>
+              <bias_mean>0.1</bias_mean>
+              <bias_stddev>0.001</bias_stddev>
+            </noise>
+          </x>
+          <y>
+            <noise type="gaussian">
+              <mean>0.0</mean>
+              <stddev>1.7e-2</stddev>
+              <bias_mean>0.1</bias_mean>
+              <bias_stddev>0.001</bias_stddev>
+            </noise>
+          </y>
+          <z>
+            <noise type="gaussian">
+              <mean>0.0</mean>
+              <stddev>1.7e-2</stddev>
+              <bias_mean>0.1</bias_mean>
+              <bias_stddev>0.001</bias_stddev>
+            </noise>
+          </z>
+        </linear_acceleration>
+      </imu>
+    </sensor>
+  </gazebo>
 </robot>

File: src/ros/rover/rover_description/rover7/urdf/rover.urdf.xacro (robot description, xacro)
@@ -601,5 +601,5 @@
         <origin xyz="-2.0093446532916618082e-17 -0.32285000000001151665 -3.7293141980345759136e-16" rpy="-1.5707963267948972241 -0.031249812601371270565 -3.141592653589793116" />
         <parent link="chassis" />
-        <child link="right_leg" />
+        <child link="left_leg" />
         <axis xyz="0 0 1"/>
         <limit effort="20" velocity="20" />
@@ -641,5 +641,5 @@
         <origin xyz="-5.9970170628790449612e-17 0.32284999999999242082 1.2597556125372093456e-17" rpy="1.5707963267948943376 -0.032623180654612699003 -3.1415926535897904515" />
         <parent link="chassis" />
-        <child link="left_leg" />
+        <child link="right_leg" />
         <axis xyz="0 0 1"/>
         <limit effort="20" velocity="20" />

Commit message: (kabi) feat : camera.launch is a piece of crap

File: src/ros/rover/rover_description/rover7/urdf/auto_camera.xacro (robot description, xacro)
@@ -5,27 +5,15 @@
   <xacro:macro name="auto_cam" params="angle">
     <link name="camera_link"/>
- <xacro:include
+    <!-- <xacro:include
         filename="$(find depthai_descriptions)/urdf/include/depthai_macro.urdf.xacro"
-    />
-    <xacro:include filename="$(find depthai_descriptions)/urdf/include/depthai_macro.urdf.xacro"/>
-    <xacro:depthai_camera
-      camera_name="oak"
-      parent="camera_link"
-      camera_model="OAK-D-LR"
-      base_frame="oak-d_frame"
-      cam_pos_x="0.0"
-      cam_pos_y="0.0"
-      cam_pos_z="0.0"
-      cam_roll="0.0"
-      cam_pitch="0.0"
-      cam_yaw="0.0"
-    />
-    <link name="camera_link_optical"/>
-    <joint name="camera_optical_joint" type="fixed">
-      <origin xyz="0.0 0 0.0" rpy="${-pi/2} 0 ${-pi/2}"/>
-      <parent link="camera_link"/>
-      <child link="camera_link_optical"/>
-    </joint>
-    <xacro:depthai_camera
+    /> -->
+  <link name="camera_link" />
+<!-- Need to be fixed, OR ADD AUTO CAMERA MOUNT to URDF-->
+  <joint name="camera_joint" type="fixed">
+    <origin xyz="0.26 0 0.2" rpy="0 0 0" />
+    <parent link="chassis" />
+    <child link="camera_link" />
+  </joint>
+    <!-- <xacro:depthai_camera
         camera_name="oak"
         parent="camera_link"
@@ -38,5 +26,5 @@
         cam_pitch="0.0"
         cam_yaw="0.0"
-    />
+    /> -->
   <link name="bootie_link" />
 <!-- Need to be fixed, OR ADD AUTO CAMERA MOUNT to URDF-->
@@ -46,5 +34,5 @@
     <child link="bootie_link" />
   </joint>
-  <xacro:depthai_camera
+  <!-- <xacro:depthai_camera
         camera_name="bootie"
         parent="bootie_link"
@@ -57,5 +45,5 @@
         cam_pitch="0.0"
         cam_yaw="0.0"
-    />
+    /> -->
   <link name="camera_link_optical" />
   <joint name="camera_optical_joint" type="fixed">

File: src/ros/rover/rover_description/rover7/urdf/rover.urdf.xacro (robot description, xacro)
@@ -1156,5 +1156,5 @@
         <parent link="chassis" />
         <child link="left_leg" />
-        <!-- <axis xyz="0 0 1" />
+        <axis xyz="0 0 1"/>
         <limit effort="20" velocity="20" />
         <joint_properties friction="0.0" /> -->
@@ -1221,5 +1221,5 @@
         <parent link="chassis" />
         <child link="right_leg" />
-        <axis xyz="0 0 1" />
+        <axis xyz="0 0 1"/>
         <limit effort="20" velocity="20" />
         <joint_properties friction="0.0" />

Commit message: feat : camera.launch is a piece of crap

File: src/ros/rover/rover_description/rover7/urdf/auto_camera.xacro (robot description, xacro)
@@ -3,29 +3,50 @@
 which is how it gets added to the gazebo sim. Edited by: Victor Bartlinski, Kabi Velmurugan Sujatha -->
 <robot xmlns:xacro="http://www.ros.org/wiki/xacro">
-  <link name="camera_link"/>
+    <!-- <xacro:include
+        filename="$(find depthai_descriptions)/urdf/include/depthai_macro.urdf.xacro"
+    /> -->
+  <link name="camera_link" />
 <!-- Need to be fixed, OR ADD AUTO CAMERA MOUNT to URDF-->
   <joint name="camera_joint" type="fixed">
-    <origin xyz="0.26 0 0.2" rpy="0 0 0"/>
-    <parent link="chassis"/>
-    <child link="camera_link"/>
+    <origin xyz="0.26 0 0.2" rpy="0 0 0" />
+    <parent link="chassis" />
+    <child link="camera_link" />
   </joint>
-  <xacro:include filename="$(find depthai_descriptions)/urdf/include/depthai_macro.urdf.xacro"/>
-  <xacro:depthai_camera
-    camera_name="oak"
-    parent="camera_link"
-    camera_model="OAK-D-LR"
-    base_frame="oak-d_frame"
-    cam_pos_x="0.0"
-    cam_pos_y="0.0"
-    cam_pos_z="0.0"
-    cam_roll="0.0"
-    cam_pitch="0.0"
-    cam_yaw="0.0"
-  />
-  <link name="camera_link_optical"/>
+    <!-- <xacro:depthai_camera
+        camera_name="oak"
+        parent="camera_link"
+        camera_model="OAK-D-LR"
+        base_frame="oak-base-frame"
+        cam_pos_x="0.0"
+        cam_pos_y="0.0"
+        cam_pos_z="0.0"
+        cam_roll="0.0"
+        cam_pitch="0.0"
+        cam_yaw="0.0"
+    /> -->
+  <link name="bootie_link" />
+<!-- Need to be fixed, OR ADD AUTO CAMERA MOUNT to URDF-->
+  <joint name="bootie_joint" type="fixed">
+    <origin xyz="0.20 0 0.19" rpy="0 0 3.14" />
+    <parent link="chassis" />
+    <child link="bootie_link" />
+  </joint>
+  <!-- <xacro:depthai_camera
+        camera_name="bootie"
+        parent="bootie_link"
+        camera_model="OAK-D-LR"
+        base_frame="bootie-base-frame"
+        cam_pos_x="0.0"
+        cam_pos_y="0.0"
+        cam_pos_z="0.0"
+        cam_roll="0.0"
+        cam_pitch="0.0"
+        cam_yaw="0.0"
+    /> -->
+  <link name="camera_link_optical" />
   <joint name="camera_optical_joint" type="fixed">
-    <origin xyz="0.0 0 0.0" rpy="${-pi/2} 0 ${-pi/2}"/>
-    <parent link="camera_link"/>
-    <child link="camera_link_optical"/>
+    <origin xyz="0.0 0 0.0" rpy="${-pi/2} 0 ${-pi/2}" />
+    <parent link="camera_link" />
+    <child link="camera_link_optical" />
   </joint>
   <!-- Depth Camera for Gazebo-->
@@ -61,5 +82,6 @@
       <plugin filename="gz-sim-imu-system" name="gz::sim::systems::Imu">
         <frame_name>oak_imu_frame</frame_name>
-        <initial_orientation_as_reference>false</initial_orientation_as_reference>
+        <initial_orientation_as_reference
+                >false</initial_orientation_as_reference>
       </plugin>
       <always_on>true</always_on>

File: src/ros/rover/rover_description/rover7/urdf/rover.urdf.xacro (robot description, xacro)
@@ -600,5 +600,5 @@
         <origin xyz="-2.0093446532916618082e-17 -0.32285000000001151665 -3.7293141980345759136e-16" rpy="-1.5707963267948972241 -0.031249812601371270565 -3.141592653589793116" />
         <parent link="chassis" />
-        <child link="right_leg" />
+        <child link="left_leg" />
         <axis xyz="0 0 1"/>
         <limit effort="20" velocity="20" />
@@ -640,5 +640,5 @@
         <origin xyz="-5.9970170628790449612e-17 0.32284999999999242082 1.2597556125372093456e-17" rpy="1.5707963267948943376 -0.032623180654612699003 -3.1415926535897904515" />
         <parent link="chassis" />
-        <child link="left_leg" />
+        <child link="right_leg" />
         <axis xyz="0 0 1"/>
         <limit effort="20" velocity="20" />
