Commit message: fixing auto drive with new wheel gearboxes WIP

File: src/ros/rover/rover_description/rover7/urdf/ros2_control.xacro (robot description, xacro)
@@ -12,6 +12,80 @@
                     <param name="revolution_pulses">8192</param>
                     <param name="min_interval">122</param>
-                    <param name="gear_ratio">36.0</param>
+                    <param name="gear_ratio">15.0</param>
                     <param name="mock">true</param>
+                    <param name="reversed">false</param>
+                    <param name="integrate_velocity">true</param>
+                </hardware>
+            </xacro:unless>
+            <xacro:if value="${use_mock_hardware}">
+                <hardware>
+                    <plugin>mock_components/GenericSystem</plugin>
+                    <param name="calculate_dynamics">true</param>
+                </hardware>
+            </xacro:if>
+            <joint name="flw">
+		        <command_interface name="velocity">
+                    <param name="max">1</param>
+                </command_interface>
+                <command_interface name="effort">
+                    <param name="max">1</param>
+                </command_interface>
+                <state_interface name="velocity">
+                    <param name="initial_value">0.0</param>
+                </state_interface>
+                <state_interface name="position">
+                    <param name="initial_value">0.0</param>
+                </state_interface>
+            </joint>
+        </ros2_control>
+        <ros2_control name="BackLeftWheel" type="system">
+            <xacro:unless value="${use_mock_hardware}">
+                <hardware>
+                    <plugin>blcmd_hardware/BLCMDHardware</plugin>
+                    <param name="candevice">can0</param>
+                    <param name="canid">2</param>
+                    <param name="resolver_reduction">1.33333333333</param>
+                    <param name="clock_rate">100000000</param>
+                    <param name="revolution_pulses">8192</param>
+                    <param name="min_interval">122</param>
+                    <param name="gear_ratio">15.0</param>
+                    <param name="mock">true</param>
+                    <param name="reversed">false</param>
+                    <param name="integrate_velocity">true</param>
+                </hardware>
+            </xacro:unless>
+            <xacro:if value="${use_mock_hardware}">
+                <hardware>
+                    <plugin>mock_components/GenericSystem</plugin>
+                    <param name="calculate_dynamics">true</param>
+                </hardware>
+            </xacro:if>
+            <joint name="blw">
+                <command_interface name="velocity">
+                    <param name="max">1</param>
+                </command_interface>
+                <command_interface name="effort">
+                    <param name="max">1</param>
+                </command_interface>
+                <state_interface name="velocity">
+                    <param name="initial_value">0.0</param>
+                </state_interface>
+                <state_interface name="position">
+                    <param name="initial_value">0.0</param>
+                </state_interface>
+            </joint>
+        </ros2_control>
+        <ros2_control name="BackRightWheel" type="system">
+            <xacro:unless value="${use_mock_hardware}">
+                <hardware>
+                    <plugin>blcmd_hardware/BLCMDHardware</plugin>
+                    <param name="candevice">can0</param>
+                    <param name="canid">3</param>
+                    <param name="resolver_reduction">1.33333333333</param>
+                    <param name="clock_rate">100000000</param>
+                    <param name="revolution_pulses">8192</param>
+                    <param name="min_interval">122</param>
+                    <param name="gear_ratio">15.0</param>
+	                <param name="mock">true</param>
                     <param name="reversed">true</param>
                     <param name="integrate_velocity">true</param>
@@ -24,31 +98,31 @@
                 </hardware>
             </xacro:if>
-            <joint name="flw">
-		        <command_interface name="velocity">
-                    <param name="max">1</param>
-                </command_interface>
-                <command_interface name="effort">
-                    <param name="max">1</param>
-                </command_interface>
-                <state_interface name="velocity">
-                    <param name="initial_value">0.0</param>
-                </state_interface>
-                <state_interface name="position">
-                    <param name="initial_value">0.0</param>
-                </state_interface>
-            </joint>
-        </ros2_control>
-        <ros2_control name="BackLeftWheel" type="system">
-            <xacro:unless value="${use_mock_hardware}">
-                <hardware>
-                    <plugin>blcmd_hardware/BLCMDHardware</plugin>
-                    <param name="candevice">can0</param>
-                    <param name="canid">2</param>
+            <joint name="brw">
+                <command_interface name="velocity">
+                    <param name="max">1</param>
+                </command_interface>
+                <command_interface name="effort">
+                    <param name="max">1</param>
+                </command_interface>
+                <state_interface name="velocity">
+                    <param name="initial_value">0.0</param>
+                </state_interface>
+                <state_interface name="position">
+                    <param name="initial_value">0.0</param>
+                </state_interface>
+            </joint>
+        </ros2_control>
+        <ros2_control name="FrontRightWheel" type="system">
+            <xacro:unless value="${use_mock_hardware}">
+                <hardware>
+                    <plugin>blcmd_hardware/BLCMDHardware</plugin>
+                    <param name="candevice">can0</param>
+                    <param name="canid">4</param>
                     <param name="resolver_reduction">1.33333333333</param>
                     <param name="clock_rate">100000000</param>
                     <param name="revolution_pulses">8192</param>
                     <param name="min_interval">122</param>
-                    <param name="gear_ratio">36.0</param>
-                    <param name="mock">true</param>
+                    <param name="gear_ratio">15.0</param>
+	                <param name="mock">true</param>
                     <param name="reversed">true</param>
                     <param name="integrate_velocity">true</param>
@@ -61,76 +135,4 @@
                 </hardware>
             </xacro:if>
-            <joint name="blw">
-                <command_interface name="velocity">
-                    <param name="max">1</param>
-                </command_interface>
-                <command_interface name="effort">
-                    <param name="max">1</param>
-                </command_interface>
-                <state_interface name="velocity">
-                    <param name="initial_value">0.0</param>
-                </state_interface>
-                <state_interface name="position">
-                    <param name="initial_value">0.0</param>
-                </state_interface>
-            </joint>
-        </ros2_control>
-        <ros2_control name="BackRightWheel" type="system">
-            <xacro:unless value="${use_mock_hardware}">
-                <hardware>
-                    <plugin>blcmd_hardware/BLCMDHardware</plugin>
-                    <param name="candevice">can0</param>
-                    <param name="canid">3</param>
-                    <param name="resolver_reduction">1.33333333333</param>
-                    <param name="clock_rate">100000000</param>
-                    <param name="revolution_pulses">8192</param>
-                    <param name="min_interval">122</param>
-                    <param name="gear_ratio">36.0</param>
-	                <param name="mock">true</param>
-                    <param name="integrate_velocity">true</param>
-                </hardware>
-            </xacro:unless>
-            <xacro:if value="${use_mock_hardware}">
-                <hardware>
-                    <plugin>mock_components/GenericSystem</plugin>
-                    <param name="calculate_dynamics">true</param>
-                </hardware>
-            </xacro:if>
-            <joint name="brw">
-                <command_interface name="velocity">
-                    <param name="max">1</param>
-                </command_interface>
-                <command_interface name="effort">
-                    <param name="max">1</param>
-                </command_interface>
-                <state_interface name="velocity">
-                    <param name="initial_value">0.0</param>
-                </state_interface>
-                <state_interface name="position">
-                    <param name="initial_value">0.0</param>
-                </state_interface>
-            </joint>
-        </ros2_control>
-        <ros2_control name="FrontRightWheel" type="system">
-            <xacro:unless value="${use_mock_hardware}">
-                <hardware>
-                    <plugin>blcmd_hardware/BLCMDHardware</plugin>
-                    <param name="candevice">can0</param>
-                    <param name="canid">4</param>
-                    <param name="resolver_reduction">1.33333333333</param>
-                    <param name="clock_rate">100000000</param>
-                    <param name="revolution_pulses">8192</param>
-                    <param name="min_interval">122</param>
-                    <param name="gear_ratio">36.0</param>
-	                <param name="mock">true</param>
-                    <param name="integrate_velocity">true</param>
-                </hardware>
-            </xacro:unless>
-            <xacro:if value="${use_mock_hardware}">
-                <hardware>
-                    <plugin>mock_components/GenericSystem</plugin>
-                    <param name="calculate_dynamics">true</param>
-                </hardware>
-            </xacro:if>
             <joint name="frw">
                 <command_interface name="velocity">
@@ -159,5 +161,5 @@
                     <param name="min_interval">233</param>
                     <param name="gear_ratio">36.0</param>
-	            <param name="mock">true</param>
+	                <param name="mock">true</param>
                 </hardware>
             </xacro:unless>
@@ -198,7 +200,7 @@
                     <param name="min_interval">233</param>
                     <param name="gear_ratio">36.0</param>
-		    <param name="revolution_pulses">8192</param>
-	            <param name="reversed">true</param>
-	            <param name="mock">true</param>
+                    <param name="revolution_pulses">8192</param>
+                    <param name="reversed">true</param>
+                    <param name="mock">true</param>
                 </hardware>
             </xacro:unless>
@@ -239,5 +241,5 @@
                     <param name="min_interval">233</param>
                     <param name="gear_ratio">36.0</param>
-	            <param name="mock">true</param>
+	                <param name="mock">true</param>
                 </hardware>
             </xacro:unless>
@@ -279,5 +281,5 @@
                     <param name="min_interval">233</param>
                     <param name="gear_ratio">36.0</param>
-	            <param name="mock">true</param>
+	                <param name="mock">true</param>
                 </hardware>
             </xacro:unless>

Commit message: fixed wheel odom and compsim errors

File: src/ros/rover/rover_description/rover7/urdf/ros2_control.xacro (robot description, xacro)
@@ -14,5 +14,5 @@
                     <param name="gear_ratio">15.0</param>
                     <param name="mock">true</param>
-                    <param name="reversed">false</param>
+                    <param name="reversed">true</param>
                     <param name="integrate_velocity">true</param>
                 </hardware>
@@ -51,4 +51,41 @@
                     <param name="gear_ratio">15.0</param>
                     <param name="mock">true</param>
+                    <param name="reversed">true</param>
+                    <param name="integrate_velocity">true</param>
+                </hardware>
+            </xacro:unless>
+            <xacro:if value="${use_mock_hardware}">
+                <hardware>
+                    <plugin>mock_components/GenericSystem</plugin>
+                    <param name="calculate_dynamics">true</param>
+                </hardware>
+            </xacro:if>
+            <joint name="blw">
+                <command_interface name="velocity">
+                    <param name="max">1</param>
+                </command_interface>
+                <command_interface name="effort">
+                    <param name="max">1</param>
+                </command_interface>
+                <state_interface name="velocity">
+                    <param name="initial_value">0.0</param>
+                </state_interface>
+                <state_interface name="position">
+                    <param name="initial_value">0.0</param>
+                </state_interface>
+            </joint>
+        </ros2_control>
+        <ros2_control name="BackRightWheel" type="system">
+            <xacro:unless value="${use_mock_hardware}">
+                <hardware>
+                    <plugin>blcmd_hardware/BLCMDHardware</plugin>
+                    <param name="candevice">can0</param>
+                    <param name="canid">3</param>
+                    <param name="resolver_reduction">1.33333333333</param>
+                    <param name="clock_rate">100000000</param>
+                    <param name="revolution_pulses">8192</param>
+                    <param name="min_interval">122</param>
+                    <param name="gear_ratio">15.0</param>
+	                <param name="mock">true</param>
                     <param name="reversed">false</param>
                     <param name="integrate_velocity">true</param>
@@ -61,25 +98,25 @@
                 </hardware>
             </xacro:if>
-            <joint name="blw">
-                <command_interface name="velocity">
-                    <param name="max">1</param>
-                </command_interface>
-                <command_interface name="effort">
-                    <param name="max">1</param>
-                </command_interface>
-                <state_interface name="velocity">
-                    <param name="initial_value">0.0</param>
-                </state_interface>
-                <state_interface name="position">
-                    <param name="initial_value">0.0</param>
-                </state_interface>
-            </joint>
-        </ros2_control>
-        <ros2_control name="BackRightWheel" type="system">
-            <xacro:unless value="${use_mock_hardware}">
-                <hardware>
-                    <plugin>blcmd_hardware/BLCMDHardware</plugin>
-                    <param name="candevice">can0</param>
-                    <param name="canid">3</param>
+            <joint name="brw">
+                <command_interface name="velocity">
+                    <param name="max">1</param>
+                </command_interface>
+                <command_interface name="effort">
+                    <param name="max">1</param>
+                </command_interface>
+                <state_interface name="velocity">
+                    <param name="initial_value">0.0</param>
+                </state_interface>
+                <state_interface name="position">
+                    <param name="initial_value">0.0</param>
+                </state_interface>
+            </joint>
+        </ros2_control>
+        <ros2_control name="FrontRightWheel" type="system">
+            <xacro:unless value="${use_mock_hardware}">
+                <hardware>
+                    <plugin>blcmd_hardware/BLCMDHardware</plugin>
+                    <param name="candevice">can0</param>
+                    <param name="canid">4</param>
                     <param name="resolver_reduction">1.33333333333</param>
                     <param name="clock_rate">100000000</param>
@@ -88,42 +125,5 @@
                     <param name="gear_ratio">15.0</param>
 	                <param name="mock">true</param>
-                    <param name="reversed">true</param>
-                    <param name="integrate_velocity">true</param>
-                </hardware>
-            </xacro:unless>
-            <xacro:if value="${use_mock_hardware}">
-                <hardware>
-                    <plugin>mock_components/GenericSystem</plugin>
-                    <param name="calculate_dynamics">true</param>
-                </hardware>
-            </xacro:if>
-            <joint name="brw">
-                <command_interface name="velocity">
-                    <param name="max">1</param>
-                </command_interface>
-                <command_interface name="effort">
-                    <param name="max">1</param>
-                </command_interface>
-                <state_interface name="velocity">
-                    <param name="initial_value">0.0</param>
-                </state_interface>
-                <state_interface name="position">
-                    <param name="initial_value">0.0</param>
-                </state_interface>
-            </joint>
-        </ros2_control>
-        <ros2_control name="FrontRightWheel" type="system">
-            <xacro:unless value="${use_mock_hardware}">
-                <hardware>
-                    <plugin>blcmd_hardware/BLCMDHardware</plugin>
-                    <param name="candevice">can0</param>
-                    <param name="canid">4</param>
-                    <param name="resolver_reduction">1.33333333333</param>
-                    <param name="clock_rate">100000000</param>
-                    <param name="revolution_pulses">8192</param>
-                    <param name="min_interval">122</param>
-                    <param name="gear_ratio">15.0</param>
-	                <param name="mock">true</param>
-                    <param name="reversed">true</param>
+                    <param name="reversed">false</param>
                     <param name="integrate_velocity">true</param>
                 </hardware>
