Commit message: (kabi) feat : ladies and gentlmen... The BigBootieCam

File: src/ros/rover/rover_description/rover7/urdf/rover.urdf.xacro (robot description, xacro)
@@ -1,3 +1,3 @@
-<?xml version="1.0" encoding="utf-8"?>
+<?xml version="1.0" encoding="utf-8" ?>
 <!-- Generated using onshape-to-robot and modified to include CKCs and ball joints by Anthony Lew -->
 <!-- Collisions added using openscad (see .scad files)-->
@@ -5,12 +5,11 @@
            Therefore if exported from onshape, don't forget to add a negative sign to the z of the axis tag on each pivot
      Note 2: Exporting from onshape has _continuous at the end of continuous joint names these have been removed post-export -->
-<robot name="rover"  xmlns:xacro="http://www.ros.org/wiki/xacro" >
+<robot name="rover" xmlns:xacro="http://www.ros.org/wiki/xacro">
     <!-- Loading args -->
-    <xacro:arg name="gazebo" default="false"/>
-    <xacro:arg name="use_mock_hardware" default="false"/>
-    <xacro:arg name="arm" default="false"/>
-    <xacro:arg name="auto_camera" default="true"/>
-    <xacro:arg name="robot_name" default="rover"/>
-    <xacro:arg name="angle" default="0"/>
+    <xacro:arg name="gazebo" default="false" />
+    <xacro:arg name="use_mock_hardware" default="false" />
+    <xacro:arg name="arm" default="false" />
+    <xacro:arg name="auto_camera" default="true" />
+    <xacro:arg name="robot_name" default="rover" />
     <!-- Robot properties-->
     <gazebo>
@@ -18,684 +17,1292 @@
     </gazebo>
     <!-- Generated URDF -->
-    <link name="base_link"></link>
+    <link name="base_link" />
     <link name="chassis">
         <visual>
-            <origin xyz="1.2353683969592321892e-17 1.3877787807815553765e-17 -1.2992673251725723918e-16" rpy="-4.03091968774772598e-16 -5.9777162559529608526e-16 1.57079632679489678" />
-            <geometry>
-                <mesh filename="file://$(find rover_description)/rover7/meshes/chassis.stl"/>
+            <origin
+                xyz="1.2353683969592321892e-17 1.3877787807815553765e-17 -1.2992673251725723918e-16"
+                rpy="-4.03091968774772598e-16 -5.9777162559529608526e-16 1.57079632679489678"
+            />
+            <geometry>
+                <mesh
+                    filename="file://$(find rover_description)/rover7/meshes/chassis.stl"
+                />
             </geometry>
             <material name="chassis_material">
-                <color rgba="0.86666666666666669627 0.074509803921568626417 0.32549019607843138191 1.0"/>
+                <color
+                    rgba="0.86666666666666669627 0.074509803921568626417 0.32549019607843138191 1.0"
+                />
             </material>
         </visual>
         <!-- Shapes for chassis -->
         <collision>
-            <origin xyz="-0.17250000000000031974 9.3018238151966802719e-18 0.023499999999999854339" rpy="-4.03091968774772598e-16 -5.9777162559529608526e-16 1.57079632679489678" />
-            <geometry>
-                <box size="0.47999999999999998224 0.54500000000000003997 0.1749999999999999889" />
-            </geometry>
-        </collision>
-        <collision>
-            <origin xyz="0.22700000000000039591 2.8459855857991392753e-18 0.033500000000000043632" rpy="-4.03091968774772598e-16 -5.9777162559529608526e-16 1.57079632679489678" />
-            <geometry>
-                <box size="0.34000000000000002442 0.26000000000000000888 0.19500000000000000666" />
-            </geometry>
-        </collision>
-        <inertial>
-            <origin xyz="-0.022980723180787008403 -0.00012909338240173079686 0.024515364506931026228" rpy="0 0 0"/>
+            <origin
+                xyz="-0.17250000000000031974 9.3018238151966802719e-18 0.023499999999999854339"
+                rpy="-4.03091968774772598e-16 -5.9777162559529608526e-16 1.57079632679489678"
+            />
+            <geometry>
+                <box
+                    size="0.47999999999999998224 0.54500000000000003997 0.1749999999999999889"
+                />
+            </geometry>
+        </collision>
+        <collision>
+            <origin
+                xyz="0.22700000000000039591 2.8459855857991392753e-18 0.033500000000000043632"
+                rpy="-4.03091968774772598e-16 -5.9777162559529608526e-16 1.57079632679489678"
+            />
+            <geometry>
+                <box
+                    size="0.34000000000000002442 0.26000000000000000888 0.19500000000000000666"
+                />
+            </geometry>
+        </collision>
+        <inertial>
+            <origin
+                xyz="-0.022980723180787008403 -0.00012909338240173079686 0.024515364506931026228"
+                rpy="0 0 0"
+            />
             <mass value="8.3419541100883876084" />
-            <inertia ixx="0.21737687093594976195" ixy="0.00013546851964915839124" ixz="-0.0088627259627339308873" iyy="0.45541406320296751176" iyz="-0.00021657327861196811977" izz="0.59726536058024382037" />
+            <inertia
+                ixx="0.21737687093594976195"
+                ixy="0.00013546851964915839124"
+                ixz="-0.0088627259627339308873"
+                iyy="0.45541406320296751176"
+                iyz="-0.00021657327861196811977"
+                izz="0.59726536058024382037"
+            />
         </inertial>
     </link>
     <link name="left_leg">
         <visual>
-            <origin xyz="-1.3078806732583218725e-20 8.6736173798840354721e-19 -0.021000000000000518252" rpy="-3.141592653589793116 6.2280032059897877693e-19 -4.1232880706353110482e-18" />
-            <geometry>
-                <mesh filename="file://$(find rover_description)/rover7/meshes/left_leg.stl"/>
+            <origin
+                xyz="-1.3078806732583218725e-20 8.6736173798840354721e-19 -0.021000000000000518252"
+                rpy="-3.141592653589793116 6.2280032059897877693e-19 -4.1232880706353110482e-18"
+            />
+            <geometry>
+                <mesh
+                    filename="file://$(find rover_description)/rover7/meshes/left_leg.stl"
+                />
             </geometry>
             <material name="left_leg_material">
-                <color rgba="0.86666666666666669627 0.074509803921568626417 0.32549019607843138191 1.0"/>
+                <color
+                    rgba="0.86666666666666669627 0.074509803921568626417 0.32549019607843138191 1.0"
+                />
             </material>
         </visual>
         <!-- Shapes for left_leg -->
         <collision>
-            <origin xyz="-1.3078806732583218725e-20 8.6736173798840354721e-19 -0.021000000000000518252" rpy="-3.141592653589793116 6.2280032059897877693e-19 -4.1232880706353110482e-18" />
-            <geometry>
-                <cylinder length="0.058000000000000002942" radius="0.042999999999999996558" />
-            </geometry>
-        </collision>
-        <collision>
-            <origin xyz="-0.085373995000000008071 0.010358865000000005291 -0.013653240000000515728" rpy="3.0194197050837283669 -1.3089970275211204598 -4.1232880706353857743e-18" />
-            <geometry>
-                <cylinder length="0.089999999999999996669" radius="0.02999999999999999889" />
-            </geometry>
-        </collision>
-        <collision>
-            <origin xyz="-0.31456908199999999987 0.036386049000000010578 0.044033037699999472148" rpy="3.0194196304823472943 -1.3264501964363342168 -4.1232880706353919373e-18" />
-            <geometry>
-                <cylinder length="0.39000000000000001332" radius="0.025000000000000001388" />
-            </geometry>
-        </collision>
-        <collision>
-            <origin xyz="-0.46338715075000003196 0.005628579600000003548 0.083600173999999485841" rpy="-3.141592653589793116 -0.27925237217133336287 3.1066861154931633138" />
-            <geometry>
-                <box size="0.105999999999999997 0.06500000000000000222 0.076999999999999999001" />
-            </geometry>
-        </collision>
-        <collision>
-            <origin xyz="-0.45372929400000000522 -0.0080000000000000001665 0.01388592399999948046" rpy="3.141592653589793116 -0.26179929927377620924 3.141592653589793116" />
-            <geometry>
-                <cylinder length="0.051999999999999997613" radius="0.044999999999999998335" />
-            </geometry>
-        </collision>
-        <collision>
-            <origin xyz="0.085785990000000020284 0.0059293025000000023489 -0.013542825000000516603" rpy="-3.071779613202412218 -1.3089970275211204598 3.141592653589793116" />
-            <geometry>
-                <cylinder length="0.089999999999999996669" radius="0.02999999999999999889" />
-            </geometry>
-        </collision>
-        <collision>
-            <origin xyz="0.31599007519999999793 0.019538657500000004147 0.044387337799999482257" rpy="-3.0717796785789528435 -1.3264501964363342168 3.141592653589793116" />
-            <geometry>
-                <cylinder length="0.39000000000000001332" radius="0.025000000000000001388" />
-            </geometry>
-        </collision>
-        <collision>
-            <origin xyz="0.46386748875000005654 -0.019645353350000005488 0.083737992499999483464" rpy="3.141592653589793116 -0.27925237217133336287 -0.034906538096629975698" />
-            <geometry>
-                <box size="0.10699999999999999789 0.06500000000000000222 0.076999999999999999001" />
-            </geometry>
-        </collision>
-        <collision>
-            <origin xyz="0.45372929400000000522 -0.034000000000000009381 0.01388592399999948046" rpy="-3.141592653589793116 -0.26179929927377620924 -4.1232880706353164408e-18" />
-            <geometry>
-                <cylinder length="0.051999999999999997613" radius="0.044999999999999998335" />
-            </geometry>
-        </collision>
-        <inertial>
-            <origin xyz="0.0041039510717090109046 -0.0038139455320666411885 0.032209303220261088774" rpy="0 0 0"/>
+            <origin
+                xyz="-1.3078806732583218725e-20 8.6736173798840354721e-19 -0.021000000000000518252"
+                rpy="-3.141592653589793116 6.2280032059897877693e-19 -4.1232880706353110482e-18"
+            />
+            <geometry>
+                <cylinder
+                    length="0.058000000000000002942"
+                    radius="0.042999999999999996558"
+                />
+            </geometry>
+        </collision>
+        <collision>
+            <origin
+                xyz="-0.085373995000000008071 0.010358865000000005291 -0.013653240000000515728"
+                rpy="3.0194197050837283669 -1.3089970275211204598 -4.1232880706353857743e-18"
+            />
+            <geometry>
+                <cylinder
+                    length="0.089999999999999996669"
+                    radius="0.02999999999999999889"
+                />
+            </geometry>
+        </collision>
+        <collision>
+            <origin
+                xyz="-0.31456908199999999987 0.036386049000000010578 0.044033037699999472148"
+                rpy="3.0194196304823472943 -1.3264501964363342168 -4.1232880706353919373e-18"
+            />
+            <geometry>
+                <cylinder
+                    length="0.39000000000000001332"
+                    radius="0.025000000000000001388"
+                />
+            </geometry>
+        </collision>
+        <collision>
+            <origin
+                xyz="-0.46338715075000003196 0.005628579600000003548 0.083600173999999485841"
+                rpy="-3.141592653589793116 -0.27925237217133336287 3.1066861154931633138"
+            />
+            <geometry>
+                <box
+                    size="0.105999999999999997 0.06500000000000000222 0.076999999999999999001"
+                />
+            </geometry>
+        </collision>
+        <collision>
+            <origin
+                xyz="-0.45372929400000000522 -0.0080000000000000001665 0.01388592399999948046"
+                rpy="3.141592653589793116 -0.26179929927377620924 3.141592653589793116"
+            />
+            <geometry>
+                <cylinder
+                    length="0.051999999999999997613"
+                    radius="0.044999999999999998335"
+                />
+            </geometry>
+        </collision>
+        <collision>
+            <origin
+                xyz="0.085785990000000020284 0.0059293025000000023489 -0.013542825000000516603"
+                rpy="-3.071779613202412218 -1.3089970275211204598 3.141592653589793116"
+            />
+            <geometry>
+                <cylinder
+                    length="0.089999999999999996669"
+                    radius="0.02999999999999999889"
+                />
+            </geometry>
+        </collision>
+        <collision>
+            <origin
+                xyz="0.31599007519999999793 0.019538657500000004147 0.044387337799999482257"
+                rpy="-3.0717796785789528435 -1.3264501964363342168 3.141592653589793116"
+            />
+            <geometry>
+                <cylinder
+                    length="0.39000000000000001332"
+                    radius="0.025000000000000001388"
+                />
+            </geometry>
+        </collision>
+        <collision>
+            <origin
+                xyz="0.46386748875000005654 -0.019645353350000005488 0.083737992499999483464"
+                rpy="3.141592653589793116 -0.27925237217133336287 -0.034906538096629975698"
+            />
+            <geometry>
+                <box
+                    size="0.10699999999999999789 0.06500000000000000222 0.076999999999999999001"
+                />
+            </geometry>
+        </collision>
+        <collision>
+            <origin
+                xyz="0.45372929400000000522 -0.034000000000000009381 0.01388592399999948046"
+                rpy="-3.141592653589793116 -0.26179929927377620924 -4.1232880706353164408e-18"
+            />
+            <geometry>
+                <cylinder
+                    length="0.051999999999999997613"
+                    radius="0.044999999999999998335"
+                />
+            </geometry>
+        </collision>
+        <inertial>
+            <origin
+                xyz="0.0041039510717090109046 -0.0038139455320666411885 0.032209303220261088774"
+                rpy="0 0 0"
+            />
             <mass value="3.3615479324288504159" />
-            <inertia ixx="0.0098869460375398468543" ixy="0.01394753149821242183" ixz="-0.00045516790515138128449" iyy="0.50779944212391792124" iyz="-0.00018907601015712540218" izz="0.50393207700006215077" />
+            <inertia
+                ixx="0.0098869460375398468543"
+                ixy="0.01394753149821242183"
+                ixz="-0.00045516790515138128449"
+                iyy="0.50779944212391792124"
+                iyz="-0.00018907601015712540218"
+                izz="0.50393207700006215077"
+            />
         </inertial>
     </link>
     <link name="fl_ankle">
         <visual>
-            <origin xyz="-0.12415341931613717297 2.2204460492503130808e-16 -0.1250000000000002498" rpy="-1.570796326794896558 -0.13351607992219349796 -5.9804098682663148249e-17" />
-            <geometry>
-                <mesh filename="file://$(find rover_description)/rover7/meshes/fl_ankle.stl"/>
+            <origin
+                xyz="-0.12415341931613717297 2.2204460492503130808e-16 -0.1250000000000002498"
+                rpy="-1.570796326794896558 -0.13351607992219349796 -5.9804098682663148249e-17"
+            />
+            <geometry>
+                <mesh
+                    filename="file://$(find rover_description)/rover7/meshes/fl_ankle.stl"
+                />
             </geometry>
             <material name="fl_ankle_material">
-                <color rgba="0.86666666666666669627 0.074509803921568626417 0.32549019607843138191 1.0"/>
+                <color
+                    rgba="0.86666666666666669627 0.074509803921568626417 0.32549019607843138191 1.0"
+                />
             </material>
         </visual>
         <!-- Shapes for fl_ankle -->
         <collision>
-            <origin xyz="-0.11601914642063104743 2.1917184460597340255e-16 -0.10304929353177745555" rpy="-1.570796326794896558 0.0061101698267938967316 -4.3738590858638602357e-17" />
-            <geometry>
-                <box size="0.032000000000000000666 0.080000000000000001665 0.05999999999999999778" />
-            </geometry>
-        </collision>
-        <collision>
-            <origin xyz="-0.091894553662955805184 2.2501886937905229218e-16 -0.16352745890207481816" rpy="-1.570796326794896558 -0.79674066942340759923 -1.6146882560911951828e-16" />
-            <geometry>
-                <box size="0.020000000000000000416 0.080000000000000001665 0.05999999999999999778" />
-            </geometry>
-        </collision>
-        <collision>
-            <origin xyz="-0.063800853957741737732 2.2792256036812134626e-16 -0.19982021317550335837" rpy="-1.570796326794896558 -0.01134335464768170508 -4.5735443069481638918e-17" />
-            <geometry>
-                <box size="0.025000000000000001388 0.030999999999999999778 0.05999999999999999778" />
-            </geometry>
-        </collision>
-        <collision>
-            <origin xyz="-0.067081786006729593463 2.1027567432387604672e-16 -0.044297919093382348565" rpy="-1.570796326794896558 0.8089619235699954114 7.549118795832927374e-17" />
-            <geometry>
-                <box size="0.01200000000000000025 0.075999999999999998113 0.05999999999999999778" />
-            </geometry>
-        </collision>
-        <collision>
-            <origin xyz="-0.10777838729007016561 2.1500295217861853941e-16 -0.069810716156365748564" rpy="-1.570796326794886788 1.5594529721472150108 1.0040858320181206805e-14" />
-            <geometry>
-                <box size="0.01200000000000000025 0.02999999999999999889 0.05999999999999999778" />
-            </geometry>
-        </collision>
-        <collision>
-            <origin xyz="-0.00045306036165823626582 2.0347719150069473786e-16 -0.010753702302991163808" rpy="1.1151930949963332936e-16 0.0061101698267938967316 -4.3738590858638602357e-17" />
-            <geometry>
-                <cylinder length="0.025999999999999998807" radius="0.037999999999999999056" />
-            </geometry>
-        </collision>
-        <collision>
-            <origin xyz="-0.028495306304552547871 2.0550457667705022165e-16 -0.017582487382379469176" rpy="1.1151930949963332936e-16 0.0061101698267938967316 -4.3738590858638602357e-17" />
-            <geometry>
-                <box size="0.02999999999999999889 0.05999999999999999778 0.01200000000000000025" />
-            </geometry>
-        </collision>
-        <inertial>
-            <origin xyz="-0.073764311118006964385 -5.3026499041438283466e-05 -0.17659909517074259822" rpy="0 0 0"/>
+            <origin
+                xyz="-0.11601914642063104743 2.1917184460597340255e-16 -0.10304929353177745555"
+                rpy="-1.570796326794896558 0.0061101698267938967316 -4.3738590858638602357e-17"
+            />
+            <geometry>
+                <box
+                    size="0.032000000000000000666 0.080000000000000001665 0.05999999999999999778"
+                />
+            </geometry>
+        </collision>
+        <collision>
+            <origin
+                xyz="-0.091894553662955805184 2.2501886937905229218e-16 -0.16352745890207481816"
+                rpy="-1.570796326794896558 -0.79674066942340759923 -1.6146882560911951828e-16"
+            />
+            <geometry>
+                <box
+                    size="0.020000000000000000416 0.080000000000000001665 0.05999999999999999778"
+                />
+            </geometry>
+        </collision>
+        <collision>
+            <origin
+                xyz="-0.063800853957741737732 2.2792256036812134626e-16 -0.19982021317550335837"
+                rpy="-1.570796326794896558 -0.01134335464768170508 -4.5735443069481638918e-17"
+            />
+            <geometry>
+                <box
+                    size="0.025000000000000001388 0.030999999999999999778 0.05999999999999999778"
+                />
+            </geometry>
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