Commit message: fixing TF tree (thanks Anthony ;-;)

File: src/ros/rover/rover_description/rover7/urdf/rover.urdf.xacro (robot description, xacro)
@@ -20,31 +20,24 @@
     <link name="base_link"></link>
     <link name="chassis">
-        <visual>
-            <origin xyz="1.2353683969592321892e-17 1.3877787807815553765e-17 -1.2992673251725723918e-16" rpy="-4.03091968774772598e-16 -5.9777162559529608526e-16 1.57079632679489678" />
-            <geometry>
-                <mesh filename="file://$(find rover_description)/rover7/meshes/chassis.stl"/>
+        <inertial>
+            <origin xyz="-2.0406452760e-04 1.4041380148e-01 1.6607310545e-02" rpy="0 0 0" />
+            <mass value="5.45693" />
+            <inertia ixx="2.0399116109e-01" ixy="-2.7566460856e-04" ixz="-2.0923415351e-04" iyy="1.6687723829e-01" iyz="-7.4614396417e-03" izz="3.2174651883e-01" />
+        </inertial>
+        <visual>
+            <origin xyz="0 0 0" rpy="3.26128e-16 -1.01395e-15 1.5708" />
+            <geometry>
+                <mesh filename="file://$(find rover_description)/rover7/meshes/chassis.stl" />
             </geometry>
             <material name="chassis_material">
-                <color rgba="0.86666666666666669627 0.074509803921568626417 0.32549019607843138191 1.0"/>
-            </material>
-        </visual>
-        <!-- Shapes for chassis -->
-        <collision>
-            <origin xyz="-0.17250000000000031974 9.3018238151966802719e-18 0.023499999999999854339" rpy="-4.03091968774772598e-16 -5.9777162559529608526e-16 1.57079632679489678" />
-            <geometry>
-                <box size="0.47999999999999998224 0.54500000000000003997 0.1749999999999999889" />
-            </geometry>
-        </collision>
-        <collision>
-            <origin xyz="0.22700000000000039591 2.8459855857991392753e-18 0.033500000000000043632" rpy="-4.03091968774772598e-16 -5.9777162559529608526e-16 1.57079632679489678" />
-            <geometry>
-                <box size="0.34000000000000002442 0.26000000000000000888 0.19500000000000000666" />
-            </geometry>
-        </collision>
-        <inertial>
-            <origin xyz="-0.022980723180787008403 -0.00012909338240173079686 0.024515364506931026228" rpy="0 0 0"/>
-            <mass value="8.3419541100883876084" />
-            <inertia ixx="0.21737687093594976195" ixy="0.00013546851964915839124" ixz="-0.0088627259627339308873" iyy="0.45541406320296751176" iyz="-0.00021657327861196811977" izz="0.59726536058024382037" />
-        </inertial>
+                <color rgba="0.866667 0.0745098 0.32549 1.0" />
+            </material>
+        </visual>
+        <collision>
+            <origin xyz="-0.1725 6.96421e-18 0.0235" rpy="3.26128e-16 -1.01395e-15 1.5708" />
+            <geometry>
+                <box size="0.48 0.545 0.175" />
+            </geometry>
+        </collision>
     </link>
     <link name="left_leg">
@@ -597,12 +590,4 @@
         <child link="chassis" />
         <origin rpy="0.0 0 0" xyz="0 0 0.45"/>
-    </joint>
-    <joint name="chassis_to_left_leg" type="continuous">
-        <origin xyz="-2.0093446532916618082e-17 -0.32285000000001151665 -3.7293141980345759136e-16" rpy="-1.5707963267948972241 -0.031249812601371270565 -3.141592653589793116" />
-        <parent link="chassis" />
-        <child link="right_leg" />
-        <axis xyz="0 0 1"/>
-        <limit effort="20" velocity="20" />
-        <joint_properties friction="0.0"/>
     </joint>
     <joint name="flp" type="revolute">
@@ -638,12 +623,4 @@
         <joint_properties friction="0.0"/>
     </joint>
-    <joint name="chassis_to_right_leg" type="continuous">
-        <origin xyz="-5.9970170628790449612e-17 0.32284999999999242082 1.2597556125372093456e-17" rpy="1.5707963267948943376 -0.032623180654612699003 -3.1415926535897904515" />
-        <parent link="chassis" />
-        <child link="left_leg" />
-        <axis xyz="0 0 1"/>
-        <limit effort="20" velocity="20" />
-        <joint_properties friction="0.0"/>
-    </joint>
     <joint name="frp" type="revolute">
         <origin xyz="-0.47013767878255985355 0.026528595964174051663 0.083618142936957573497" rpy="-1.5707963267948938935 0.8652479367931649179 -3.1148421188216208755" />
@@ -678,4 +655,25 @@
         <joint_properties friction="0.0"/>
     </joint>
+    <xacro:unless value="$(arg gazebo)">
+        <xacro:property name="gazebo" value="true"/>
+    </xacro:unless>
+    <xacro:property name="gazebo" value="false"/>
+    <joint name="chassis_to_right_leg" type="${'fixed' if gazebo == 'true' else 'continuous'}">
+        <origin xyz="-2.0093446532916618082e-17 -0.32285000000001151665 -3.7293141980345759136e-16" rpy="-1.5707963267948972241 -0.031249812601371270565 -3.141592653589793116" />
+        <parent link="chassis" />
+        <child link="right_leg" />
+        <axis xyz="0 0 1"/>
+        <limit effort="20" velocity="20" />
+        <joint_properties friction="0.0"/>
+    </joint>
+    <joint name="chassis_to_left_leg" type="${'fixed' if gazebo == 'true' else 'continuous'}">
+        <origin xyz="-5.9970170628790449612e-17 0.32284999999999242082 1.2597556125372093456e-17" rpy="1.5707963267948943376 -0.032623180654612699003 -3.1415926535897904515" />
+        <parent link="chassis" />
+        <child link="left_leg" />
+        <axis xyz="0 0 1"/>
+        <limit effort="20" velocity="20" />
+        <joint_properties friction="0.0"/>
+    </joint>
+    <!-- Diffbar won't show up irl lol-->
     <joint name="chassis_to_diffbar" type="continuous">
         <origin xyz="-0.47600000000002590239 -4.8144507783734281313e-09 0.046505449483682070877" rpy="-1.5707963267949112129 -2.1008432044742341424e-09 1.570796326794896558" />
@@ -690,5 +688,5 @@
     <xacro:include filename="$(find rover_description)/rover7/urdf/ckc.xacro"/>
     <xacro:if value="$(arg auto_camera)">
-        <xacro:include filename="$(find rover_description)/rover7/urdf/auto_camera.xacro"/>
+        <xacro:include filename="$(find rover_description)/rover7/auto/auto_camera.xacro"/>
         <xacro:auto_cam angle="$(arg angle)"></xacro:auto_cam>
     </xacro:if>

Commit message: fixing IRL TF tree

File: src/ros/rover/rover_description/rover7/urdf/rover.urdf.xacro (robot description, xacro)
@@ -591,4 +591,12 @@
         <origin rpy="0.0 0 0" xyz="0 0 0.45"/>
     </joint>
+    <joint name="chassis_to_left_leg" type="continuous">
+        <origin xyz="-5.9970170628790449612e-17 0.32284999999999242082 1.2597556125372093456e-17" rpy="1.5707963267948943376 -0.032623180654612699003 -3.1415926535897904515" />
+        <parent link="chassis" />
+        <child link="left_leg" />
+        <axis xyz="0 0 1"/>
+        <limit effort="20" velocity="20" lower="0" upper="0"/>
+        <joint_properties friction="0.0"/>
+    </joint>
     <joint name="flp" type="revolute">
         <origin xyz="-0.4796458670490280074 -0.025616433642942942894 0.086267061908379405466" rpy="-1.5707963267948972241 -0.86524793679315337158 -0.028123902821415372455" />
@@ -623,4 +631,12 @@
         <joint_properties friction="0.0"/>
     </joint>
+    <joint name="chassis_to_right_leg" type="continuous">
+        <origin xyz="-2.0093446532916618082e-17 -0.32285000000001151665 -3.7293141980345759136e-16" rpy="-1.5707963267948972241 -0.031249812601371270565 -3.141592653589793116" />
+        <parent link="chassis" />
+        <child link="right_leg" />
+        <axis xyz="0 0 1"/>
+        <limit effort="20" velocity="20" lower="0" upper="0"/>
+        <joint_properties friction="0.0"/>
+    </joint>
     <joint name="frp" type="revolute">
         <origin xyz="-0.47013767878255985355 0.026528595964174051663 0.083618142936957573497" rpy="-1.5707963267948938935 0.8652479367931649179 -3.1148421188216208755" />
@@ -651,24 +667,4 @@
         <parent link="br_ankle" />
         <child link="br_wheel" />
-        <axis xyz="0 0 1"/>
-        <limit effort="20" velocity="20" />
-        <joint_properties friction="0.0"/>
-    </joint>
-    <xacro:unless value="$(arg gazebo)">
-        <xacro:property name="gazebo" value="true"/>
-    </xacro:unless>
-    <xacro:property name="gazebo" value="false"/>
-    <joint name="chassis_to_right_leg" type="${'fixed' if gazebo == 'true' else 'continuous'}">
-        <origin xyz="-2.0093446532916618082e-17 -0.32285000000001151665 -3.7293141980345759136e-16" rpy="-1.5707963267948972241 -0.031249812601371270565 -3.141592653589793116" />
-        <parent link="chassis" />
-        <child link="right_leg" />
-        <axis xyz="0 0 1"/>
-        <limit effort="20" velocity="20" />
-        <joint_properties friction="0.0"/>
-    </joint>
-    <joint name="chassis_to_left_leg" type="${'fixed' if gazebo == 'true' else 'continuous'}">
-        <origin xyz="-5.9970170628790449612e-17 0.32284999999999242082 1.2597556125372093456e-17" rpy="1.5707963267948943376 -0.032623180654612699003 -3.1415926535897904515" />
-        <parent link="chassis" />
-        <child link="left_leg" />
         <axis xyz="0 0 1"/>
         <limit effort="20" velocity="20" />

Commit message: Actual fix to TF tree

File: src/ros/rover/rover_description/rover7/urdf/rover.urdf.xacro (robot description, xacro)
@@ -596,5 +596,5 @@
         <child link="left_leg" />
         <axis xyz="0 0 1"/>
-        <limit effort="20" velocity="20" lower="0" upper="0"/>
+        <limit effort="20" velocity="20" />
         <joint_properties friction="0.0"/>
     </joint>
@@ -636,5 +636,5 @@
         <child link="right_leg" />
         <axis xyz="0 0 1"/>
-        <limit effort="20" velocity="20" lower="0" upper="0"/>
+        <limit effort="20" velocity="20" />
         <joint_properties friction="0.0"/>
     </joint>
@@ -671,5 +671,5 @@
         <joint_properties friction="0.0"/>
     </joint>
-    <!-- Diffbar won't show up irl lol-->
+    <!-- Diffbar won't show up in irl TF tree unless u add its dynamic joints to controllers.yaml extra joints-->
     <joint name="chassis_to_diffbar" type="continuous">
         <origin xyz="-0.47600000000002590239 -4.8144507783734281313e-09 0.046505449483682070877" rpy="-1.5707963267949112129 -2.1008432044742341424e-09 1.570796326794896558" />

Commit message: Adding cube localisation into feat/bt (#314)
Co-authored-by: Monash Nova Rover <novaroverteam@monash.edu>

File: src/ros/rover/rover_description/rover7/urdf/rover.urdf.xacro (robot description, xacro)
@@ -20,31 +20,24 @@
     <link name="base_link"></link>
     <link name="chassis">
-        <visual>
-            <origin xyz="1.2353683969592321892e-17 1.3877787807815553765e-17 -1.2992673251725723918e-16" rpy="-4.03091968774772598e-16 -5.9777162559529608526e-16 1.57079632679489678" />
-            <geometry>
-                <mesh filename="file://$(find rover_description)/rover7/meshes/chassis.stl"/>
+        <inertial>
+            <origin xyz="-2.0406452760e-04 1.4041380148e-01 1.6607310545e-02" rpy="0 0 0" />
+            <mass value="5.45693" />
+            <inertia ixx="2.0399116109e-01" ixy="-2.7566460856e-04" ixz="-2.0923415351e-04" iyy="1.6687723829e-01" iyz="-7.4614396417e-03" izz="3.2174651883e-01" />
+        </inertial>
+        <visual>
+            <origin xyz="0 0 0" rpy="3.26128e-16 -1.01395e-15 1.5708" />
+            <geometry>
+                <mesh filename="file://$(find rover_description)/rover7/meshes/chassis.stl" />
             </geometry>
             <material name="chassis_material">
-                <color rgba="0.86666666666666669627 0.074509803921568626417 0.32549019607843138191 1.0"/>
-            </material>
-        </visual>
-        <!-- Shapes for chassis -->
-        <collision>
-            <origin xyz="-0.17250000000000031974 9.3018238151966802719e-18 0.023499999999999854339" rpy="-4.03091968774772598e-16 -5.9777162559529608526e-16 1.57079632679489678" />
-            <geometry>
-                <box size="0.47999999999999998224 0.54500000000000003997 0.1749999999999999889" />
-            </geometry>
-        </collision>
-        <collision>
-            <origin xyz="0.22700000000000039591 2.8459855857991392753e-18 0.033500000000000043632" rpy="-4.03091968774772598e-16 -5.9777162559529608526e-16 1.57079632679489678" />
-            <geometry>
-                <box size="0.34000000000000002442 0.26000000000000000888 0.19500000000000000666" />
-            </geometry>
-        </collision>
-        <inertial>
-            <origin xyz="-0.022980723180787008403 -0.00012909338240173079686 0.024515364506931026228" rpy="0 0 0"/>
-            <mass value="8.3419541100883876084" />
-            <inertia ixx="0.21737687093594976195" ixy="0.00013546851964915839124" ixz="-0.0088627259627339308873" iyy="0.45541406320296751176" iyz="-0.00021657327861196811977" izz="0.59726536058024382037" />
-        </inertial>
+                <color rgba="0.866667 0.0745098 0.32549 1.0" />
+            </material>
+        </visual>
+        <collision>
+            <origin xyz="-0.1725 6.96421e-18 0.0235" rpy="3.26128e-16 -1.01395e-15 1.5708" />
+            <geometry>
+                <box size="0.48 0.545 0.175" />
+            </geometry>
+        </collision>
     </link>
     <link name="left_leg">
@@ -599,9 +592,9 @@
     </joint>
     <joint name="chassis_to_left_leg" type="continuous">
-        <origin xyz="-2.0093446532916618082e-17 -0.32285000000001151665 -3.7293141980345759136e-16" rpy="-1.5707963267948972241 -0.031249812601371270565 -3.141592653589793116" />
+        <origin xyz="-5.9970170628790449612e-17 0.32284999999999242082 1.2597556125372093456e-17" rpy="1.5707963267948943376 -0.032623180654612699003 -3.1415926535897904515" />
         <parent link="chassis" />
-        <child link="right_leg" />
+        <child link="left_leg" />
         <axis xyz="0 0 1"/>
-        <limit effort="20" velocity="20" />
+        <limit effort="20" velocity="20" lower="0" upper="0"/>
         <joint_properties friction="0.0"/>
     </joint>
@@ -639,9 +632,9 @@
     </joint>
     <joint name="chassis_to_right_leg" type="continuous">
-        <origin xyz="-5.9970170628790449612e-17 0.32284999999999242082 1.2597556125372093456e-17" rpy="1.5707963267948943376 -0.032623180654612699003 -3.1415926535897904515" />
+        <origin xyz="-2.0093446532916618082e-17 -0.32285000000001151665 -3.7293141980345759136e-16" rpy="-1.5707963267948972241 -0.031249812601371270565 -3.141592653589793116" />
         <parent link="chassis" />
-        <child link="left_leg" />
+        <child link="right_leg" />
         <axis xyz="0 0 1"/>
-        <limit effort="20" velocity="20" />
+        <limit effort="20" velocity="20" lower="0" upper="0"/>
         <joint_properties friction="0.0"/>
     </joint>
@@ -678,4 +671,5 @@
         <joint_properties friction="0.0"/>
     </joint>
+    <!-- Diffbar won't show up irl lol-->
     <joint name="chassis_to_diffbar" type="continuous">
         <origin xyz="-0.47600000000002590239 -4.8144507783734281313e-09 0.046505449483682070877" rpy="-1.5707963267949112129 -2.1008432044742341424e-09 1.570796326794896558" />

Commit message: fix: temporary fixes to make arm show on Banksia (#217)

File: src/ros/rover/rover_description/rover7/urdf/rover.urdf.xacro (robot description, xacro)
@@ -697,5 +697,5 @@
         <xacro:include filename="$(find rover_description)/arm/urdf/arm.urdf.xacro" />
         <joint name="chassis_to_arm_base" type="fixed">
-            <origin xyz="0 0.15 -0.06" rpy="0 0 1.57"/>
+            <origin xyz="0.18 0 -0.03" rpy="0 0 0"/>
             <parent link="chassis" />
             <child link="arm_link" />

Commit message: Feat/urdf fixes (#301)
Co-authored-by: Terry Tian <97772315+tytia@users.noreply.github.com>
Co-authored-by: Anthony Lew <anthony@v01dbreaker.cc>

File: src/ros/rover/rover_description/rover7/urdf/rover.urdf.xacro (robot description, xacro)
@@ -5,5 +5,5 @@
            Therefore if exported from onshape, don't forget to add a negative sign to the z of the axis tag on each pivot
      Note 2: Exporting from onshape has _continuous at the end of continuous joint names these have been removed post-export -->
-<robot name="rover"  xmlns:xacro="http://www.ros.org/wiki/xacro" >
+<robot name="rover7"  xmlns:xacro="http://www.ros.org/wiki/xacro" >
     <!-- Loading args -->
     <xacro:arg name="gazebo" default="false"/>
@@ -11,5 +11,5 @@
     <xacro:arg name="arm" default="false"/>
     <xacro:arg name="auto_camera" default="true"/>
-    <xacro:arg name="robot_name" default="rover"/>
+    <xacro:arg name="robot_name" default="rover7"/>
     <xacro:arg name="angle" default="0"/>
     <!-- Robot properties-->
@@ -596,5 +596,5 @@
         <child link="left_leg" />
         <axis xyz="0 0 1"/>
-        <limit effort="20" velocity="20" lower="0" upper="0"/>
+        <limit effort="20" velocity="20" />
         <joint_properties friction="0.0"/>
     </joint>
@@ -636,5 +636,5 @@
         <child link="right_leg" />
         <axis xyz="0 0 1"/>
-        <limit effort="20" velocity="20" lower="0" upper="0"/>
+        <limit effort="20" velocity="20" />
         <joint_properties friction="0.0"/>
     </joint>
@@ -671,5 +671,5 @@
         <joint_properties friction="0.0"/>
     </joint>
-    <!-- Diffbar won't show up irl lol-->
+    <!-- Diffbar won't show up in irl TF tree unless u add its dynamic joints to controllers.yaml extra joints-->
     <joint name="chassis_to_diffbar" type="continuous">
         <origin xyz="-0.47600000000002590239 -4.8144507783734281313e-09 0.046505449483682070877" rpy="-1.5707963267949112129 -2.1008432044742341424e-09 1.570796326794896558" />
@@ -684,12 +684,12 @@
     <xacro:include filename="$(find rover_description)/rover7/urdf/ckc.xacro"/>
     <xacro:if value="$(arg auto_camera)">
-        <xacro:include filename="$(find rover_description)/rover7/urdf/auto_camera.xacro"/>
+        <xacro:include filename="$(find rover_description)/auto_mount/urdf/auto_camera.xacro"/>
         <xacro:auto_cam angle="$(arg angle)"></xacro:auto_cam>
     </xacro:if>
     <xacro:if value="$(arg arm)">
-        <!-- Needs to be updated for new arm-->
-        <xacro:include filename="$(find rover_description)/arm/urdf/arm.urdf.xacro" />
+        <!-- Currently attaches waratah's arm, add rover7 arm after ARCh-->
+        <xacro:include filename="$(find rover_description)/waratah_arm/urdf/arm.urdf.xacro" />
         <joint name="chassis_to_arm_base" type="fixed">
-            <origin xyz="0.18 0 -0.03" rpy="0 0 0"/>
+            <origin xyz="0.2 0 -0.06" rpy="0 0 0"/>
             <parent link="chassis" />
             <child link="arm_link" />

Commit message: fix: Move rover origin (base link) to back right wheel (br corner of br wheel)

File: src/ros/rover/rover_description/rover7/urdf/rover.urdf.xacro (robot description, xacro)
@@ -598,5 +598,5 @@
         <parent link="base_link"/>
         <child link="chassis" />
-        <origin rpy="0.0 0 0" xyz="0 0 0.45"/>
+        <origin rpy="0.0 0 0" xyz="0.637181 0.487444 0.434263"/>
     </joint>
     <joint name="chassis_to_left_leg" type="continuous">

Commit message: fix static layer

File: src/ros/rover/rover_description/rover7/urdf/rover.urdf.xacro (robot description, xacro)
@@ -598,5 +598,5 @@
         <parent link="base_link"/>
         <child link="chassis" />
-        <origin rpy="0.0 0 0" xyz="0.637181 0.487444 0.434263"/>
+        <origin rpy="0.0 0 0" xyz="0 0 0.434263"/>
     </joint>
     <joint name="chassis_to_left_leg" type="continuous">
