Commit message: Deleting feat/bt (#372)
Co-authored-by: Terry Tian <97772315+tytia@users.noreply.github.com>
Co-authored-by: Anthony Lew <anthony@v01dbreaker.cc>
Co-authored-by: Kabilan VS <kabiniki4849@gmail.com>
Co-authored-by: JoelAKruger <pinklemonday@gmail.com>
Co-authored-by: Tarik Thomas <5tarikthomas5118@gmail.com>
Co-authored-by: Chetan Edupalli <cedu0001@student.monash.edu>
Co-authored-by: novarover <53011489+novarover@users.noreply.github.com>
Co-authored-by: Monash Nova Rover <novaroverteam@monash.edu>

File: src/ros/rover/rover_description/rover7/urdf/rover.urdf.xacro (robot description, xacro)
@@ -5,5 +5,5 @@
            Therefore if exported from onshape, don't forget to add a negative sign to the z of the axis tag on each pivot
      Note 2: Exporting from onshape has _continuous at the end of continuous joint names these have been removed post-export -->
-<robot name="rover"  xmlns:xacro="http://www.ros.org/wiki/xacro" >
+<robot name="rover7"  xmlns:xacro="http://www.ros.org/wiki/xacro" >
     <!-- Loading args -->
     <xacro:arg name="gazebo" default="false"/>
@@ -11,40 +11,42 @@
     <xacro:arg name="arm" default="false"/>
     <xacro:arg name="auto_camera" default="true"/>
-    <xacro:arg name="robot_name" default="rover"/>
+    <xacro:arg name="robot_name" default="rover7"/>
     <xacro:arg name="angle" default="0"/>
+    <xacro:arg name="use_local_mesh" default="false"/>
     <!-- Robot properties-->
     <gazebo>
         <self_collide>false</self_collide>
     </gazebo>
+    <!-- Variables -->
+    <xacro:if value="$(arg use_local_mesh)">
+        <xacro:property name="mesh_path" value="file://home/nova/nova/src/ros/rover/rover_description" />
+    </xacro:if>
+    <xacro:unless value="$(arg use_local_mesh)">
+        <xacro:property name="mesh_path" value="file://$(find rover_description)" />
+    </xacro:unless>
+    <xacro:property name="angle" value="$(arg angle)" />
     <!-- Generated URDF -->
     <link name="base_link"></link>
     <link name="chassis">
-        <visual>
-            <origin xyz="1.2353683969592321892e-17 1.3877787807815553765e-17 -1.2992673251725723918e-16" rpy="-4.03091968774772598e-16 -5.9777162559529608526e-16 1.57079632679489678" />
-            <geometry>
-                <mesh filename="file://$(find rover_description)/rover7/meshes/chassis.stl"/>
+        <inertial>
+            <origin xyz="-2.0406452760e-04 1.4041380148e-01 1.6607310545e-02" rpy="0 0 0" />
+            <mass value="5.45693" />
+            <inertia ixx="2.0399116109e-01" ixy="-2.7566460856e-04" ixz="-2.0923415351e-04" iyy="1.6687723829e-01" iyz="-7.4614396417e-03" izz="3.2174651883e-01" />
+        </inertial>
+        <visual>
+            <origin xyz="0 0 0" rpy="3.26128e-16 -1.01395e-15 1.5708" />
+            <geometry>
+                <mesh filename="${mesh_path}/rover7/meshes/chassis.stl" />
             </geometry>
             <material name="chassis_material">
-                <color rgba="0.86666666666666669627 0.074509803921568626417 0.32549019607843138191 1.0"/>
-            </material>
-        </visual>
-        <!-- Shapes for chassis -->
-        <collision>
-            <origin xyz="-0.17250000000000031974 9.3018238151966802719e-18 0.023499999999999854339" rpy="-4.03091968774772598e-16 -5.9777162559529608526e-16 1.57079632679489678" />
-            <geometry>
-                <box size="0.47999999999999998224 0.54500000000000003997 0.1749999999999999889" />
-            </geometry>
-        </collision>
-        <collision>
-            <origin xyz="0.22700000000000039591 2.8459855857991392753e-18 0.033500000000000043632" rpy="-4.03091968774772598e-16 -5.9777162559529608526e-16 1.57079632679489678" />
-            <geometry>
-                <box size="0.34000000000000002442 0.26000000000000000888 0.19500000000000000666" />
-            </geometry>
-        </collision>
-        <inertial>
-            <origin xyz="-0.022980723180787008403 -0.00012909338240173079686 0.024515364506931026228" rpy="0 0 0"/>
-            <mass value="8.3419541100883876084" />
-            <inertia ixx="0.21737687093594976195" ixy="0.00013546851964915839124" ixz="-0.0088627259627339308873" iyy="0.45541406320296751176" iyz="-0.00021657327861196811977" izz="0.59726536058024382037" />
-        </inertial>
+                <color rgba="0.866667 0.0745098 0.32549 1.0" />
+            </material>
+        </visual>
+        <collision>
+            <origin xyz="-0.1725 6.96421e-18 0.0235" rpy="3.26128e-16 -1.01395e-15 1.5708" />
+            <geometry>
+                <box size="0.48 0.545 0.175" />
+            </geometry>
+        </collision>
     </link>
     <link name="left_leg">
@@ -52,5 +54,5 @@
             <origin xyz="-1.3078806732583218725e-20 8.6736173798840354721e-19 -0.021000000000000518252" rpy="-3.141592653589793116 6.2280032059897877693e-19 -4.1232880706353110482e-18" />
             <geometry>
-                <mesh filename="file://$(find rover_description)/rover7/meshes/left_leg.stl"/>
+                <mesh filename="${mesh_path}/rover7/meshes/left_leg.stl"/>
             </geometry>
             <material name="left_leg_material">
@@ -123,5 +125,5 @@
             <origin xyz="-0.12415341931613717297 2.2204460492503130808e-16 -0.1250000000000002498" rpy="-1.570796326794896558 -0.13351607992219349796 -5.9804098682663148249e-17" />
             <geometry>
-                <mesh filename="file://$(find rover_description)/rover7/meshes/fl_ankle.stl"/>
+                <mesh filename="${mesh_path}/rover7/meshes/fl_ankle.stl"/>
             </geometry>
             <material name="fl_ankle_material">
@@ -182,5 +184,5 @@
             <origin xyz="5.5511151231257827021e-17 0 5.963111948670274387e-18" rpy="7.279848939407052303e-17 1.0638440422271473935e-16 -6.3914183266779029169e-20" />
             <geometry>
-                <mesh filename="file://$(find rover_description)/rover7/meshes/fl_wheel.stl"/>
+                <mesh filename="${mesh_path}/rover7/meshes/fl_wheel.stl"/>
             </geometry>
             <material name="fl_wheel_material">
@@ -205,5 +207,5 @@
             <origin xyz="-0.12415341931613714521 2.2204460492503130808e-16 -0.1250000000000002498" rpy="-1.570796326794896558 -0.13351607992219349796 -7.1088909477657821376e-17" />
             <geometry>
-                <mesh filename="file://$(find rover_description)/rover7/meshes/bl_ankle.stl"/>
+                <mesh filename="${mesh_path}/rover7/meshes/bl_ankle.stl"/>
             </geometry>
             <material name="bl_ankle_material">
@@ -264,5 +266,5 @@
             <origin xyz="0 1.1102230246251565404e-16 1.7780915628762272718e-17" rpy="4.6040217445536182725e-17 1.0513492286565858337e-16 2.3412503191653332746e-19" />
             <geometry>
-                <mesh filename="file://$(find rover_description)/rover7/meshes/bl_wheel.stl"/>
+                <mesh filename="${mesh_path}/rover7/meshes/bl_wheel.stl"/>
             </geometry>
             <material name="bl_wheel_material">
@@ -287,5 +289,5 @@
             <origin xyz="-7.9461177221465168975e-19 -7.2858385990954703269e-20 -0.020999999999999519051" rpy="3.141592653589793116 3.7838655819744092421e-17 -5.8406613147999892266e-19" />
             <geometry>
-                <mesh filename="file://$(find rover_description)/rover7/meshes/right_leg.stl"/>
+                <mesh filename="${mesh_path}/rover7/meshes/right_leg.stl"/>
             </geometry>
             <material name="right_leg_material">
@@ -358,5 +360,5 @@
             <origin xyz="0.12415341931613695092 -2.2204460492503130808e-16 -0.12500000000000027756" rpy="-1.57079632679489678 0.13351607992219352572 9.9507186100571649487e-18" />
             <geometry>
-                <mesh filename="file://$(find rover_description)/rover7/meshes/fr_ankle.stl"/>
+                <mesh filename="${mesh_path}/rover7/meshes/fr_ankle.stl"/>
             </geometry>
             <material name="fr_ankle_material">
@@ -417,5 +419,5 @@
             <origin xyz="5.5511151231257827021e-17 -1.1102230246251565404e-16 -3.0791341698588325926e-17" rpy="-3.6194812825998444115e-17 1.0511409763610977507e-16 -2.2325341479697011877e-19" />
             <geometry>
-                <mesh filename="file://$(find rover_description)/rover7/meshes/fr_wheel.stl"/>
+                <mesh filename="${mesh_path}/rover7/meshes/fr_wheel.stl"/>
             </geometry>
             <material name="fr_wheel_material">
@@ -440,5 +442,5 @@
             <origin xyz="0.12415341931613720072 -2.2204460492503130808e-16 -0.12500000000000027756" rpy="-1.57079632679489678 0.13351607992219349796 -6.7670245197813334123e-17" />
             <geometry>
-                <mesh filename="file://$(find rover_description)/rover7/meshes/br_ankle.stl"/>
+                <mesh filename="${mesh_path}/rover7/meshes/br_ankle.stl"/>
             </geometry>
             <material name="br_ankle_material">
@@ -499,5 +501,5 @@
             <origin xyz="5.5511151231257827021e-17 0 5.8763757748714340323e-17" rpy="1.4537948349788456791e-16 1.0501738044156386319e-16 -7.6074648532850333807e-21" />
             <geometry>
-                <mesh filename="file://$(find rover_description)/rover7/meshes/br_wheel.stl"/>
+                <mesh filename="${mesh_path}/rover7/meshes/br_wheel.stl"/>
             </geometry>
             <material name="br_wheel_material">
@@ -522,5 +524,5 @@
             <origin xyz="4.9770590769729886024e-14 -0.00015426611885745872277 -0.010000000000000730527" rpy="1.570796326794896558 -3.0512890594788867116e-34 0" />
             <geometry>
-                <mesh filename="file://$(find rover_description)/rover7/meshes/diffbar.stl"/>
+                <mesh filename="${mesh_path}/rover7/meshes/diffbar.stl"/>
             </geometry>
             <material name="diffbar_material">
@@ -551,5 +553,5 @@
             <origin xyz="-2.7755575615628913511e-15 -0.057750000000000162315 3.3306690738754696213e-16" rpy="1.5707963267948350516 -1.5127867282353739675 -3.1415926535897926719" />
             <geometry>
-                <mesh filename="file://$(find rover_description)/rover7/meshes/left_difflink.stl"/>
+                <mesh filename="${mesh_path}/rover7/meshes/left_difflink.stl"/>
             </geometry>
             <material name="left_difflink_material">
@@ -574,5 +576,5 @@
             <origin xyz="6.2172489379008766264e-15 -0.057749999999999454547 -2.4424906541753443889e-15" rpy="1.5707963267948286123 1.512786629442331332 3.141592653589793116" />
             <geometry>
-                <mesh filename="file://$(find rover_description)/rover7/meshes/right_difflink.stl"/>
+                <mesh filename="${mesh_path}/rover7/meshes/right_difflink.stl"/>
             </geometry>
             <material name="right_difflink_material">
@@ -596,10 +598,10 @@
         <parent link="base_link"/>
         <child link="chassis" />
-        <origin rpy="0.0 0 0" xyz="0 0 0.45"/>
+        <origin rpy="0.0 0 0" xyz="0 0 0.434263"/>
     </joint>
     <joint name="chassis_to_left_leg" type="continuous">
-        <origin xyz="-2.0093446532916618082e-17 -0.32285000000001151665 -3.7293141980345759136e-16" rpy="-1.5707963267948972241 -0.031249812601371270565 -3.141592653589793116" />
+        <origin xyz="-5.9970170628790449612e-17 0.32284999999999242082 1.2597556125372093456e-17" rpy="1.5707963267948943376 -0.032623180654612699003 -3.1415926535897904515" />
         <parent link="chassis" />
-        <child link="right_leg" />
+        <child link="left_leg" />
         <axis xyz="0 0 1"/>
         <limit effort="20" velocity="20" />
@@ -639,7 +641,7 @@
     </joint>
     <joint name="chassis_to_right_leg" type="continuous">
-        <origin xyz="-5.9970170628790449612e-17 0.32284999999999242082 1.2597556125372093456e-17" rpy="1.5707963267948943376 -0.032623180654612699003 -3.1415926535897904515" />
+        <origin xyz="-2.0093446532916618082e-17 -0.32285000000001151665 -3.7293141980345759136e-16" rpy="-1.5707963267948972241 -0.031249812601371270565 -3.141592653589793116" />
         <parent link="chassis" />
-        <child link="left_leg" />
+        <child link="right_leg" />
         <axis xyz="0 0 1"/>
         <limit effort="20" velocity="20" />
@@ -678,4 +680,5 @@
         <joint_properties friction="0.0"/>
     </joint>
+    <!-- Diffbar won't show up in irl TF tree unless u add its dynamic joints to controllers.yaml extra joints-->
     <joint name="chassis_to_diffbar" type="continuous">
         <origin xyz="-0.47600000000002590239 -4.8144507783734281313e-09 0.046505449483682070877" rpy="-1.5707963267949112129 -2.1008432044742341424e-09 1.570796326794896558" />
@@ -690,12 +693,11 @@
     <xacro:include filename="$(find rover_description)/rover7/urdf/ckc.xacro"/>
     <xacro:if value="$(arg auto_camera)">
-        <xacro:include filename="$(find rover_description)/rover7/urdf/auto_camera.xacro"/>
-        <xacro:auto_cam angle="$(arg angle)"></xacro:auto_cam>
+        <xacro:include filename="$(find rover_description)/auto_mount/urdf/auto_camera.xacro"/>
     </xacro:if>
     <xacro:if value="$(arg arm)">
-        <!-- Needs to be updated for new arm-->
-        <xacro:include filename="$(find rover_description)/arm/urdf/arm.urdf.xacro" />
+        <!-- Currently attaches waratah's arm, add rover7 arm after ARCh-->
+        <xacro:include filename="$(find rover_description)/waratah_arm/urdf/arm.urdf.xacro" />
         <joint name="chassis_to_arm_base" type="fixed">
-            <origin xyz="0.18 0 -0.03" rpy="0 0 0"/>
+            <origin xyz="0.2 0 -0.06" rpy="0 0 0"/>
             <parent link="chassis" />
             <child link="arm_link" />

Commit message: feat: Arm URDF

File: src/ros/rover/rover_description/rover7/urdf/rover.urdf.xacro (robot description, xacro)
@@ -696,5 +696,5 @@
     </xacro:if>
     <xacro:if value="$(arg arm)">
-        <!-- Currently attaches waratah's arm, add rover7 arm after ARCh-->
+        <!-- Waratah's arm
         <xacro:include filename="$(find rover_description)/waratah_arm/urdf/arm.urdf.xacro" />
         <joint name="chassis_to_arm_base" type="fixed">
@@ -702,6 +702,17 @@
             <parent link="chassis" />
             <child link="arm_link" />
+        </joint> -->
+        <!-- Banksia's arm -->
+        <xacro:include filename="$(find rover_description)/banksia_arm/urdf/arm.urdf.xacro" />
+        <joint name="chassis_to_arm_base" type="fixed">
+            <origin xyz="0.22899999999999606781 1.1022818830789207535e-16 0.11707476398169149034" rpy="0 0 1.5708" />
+            <parent link="chassis" />
+            <child link="arm_link" />
         </joint>
+        <xacro:include filename="$(find rover_description)/banksia_arm/urdf/joint_states_with_arm.xacro"/>
     </xacro:if>
+     <xacro:unless value="$(arg arm)">
+        <xacro:include filename="$(find rover_description)/rover7/urdf/joint_states.xacro"/>
+    </xacro:unless>
     <xacro:unless value="$(arg gazebo)">
         <xacro:include filename="$(find rover_description)/rover7/urdf/ros2_control.xacro" />

Commit message: Banksia's ARM! - feat/urdf-arm (#381)

File: src/ros/rover/rover_description/rover7/urdf/rover.urdf.xacro (robot description, xacro)
@@ -696,5 +696,5 @@
     </xacro:if>
     <xacro:if value="$(arg arm)">
-        <!-- Currently attaches waratah's arm, add rover7 arm after ARCh-->
+        <!-- Waratah's arm
         <xacro:include filename="$(find rover_description)/waratah_arm/urdf/arm.urdf.xacro" />
         <joint name="chassis_to_arm_base" type="fixed">
@@ -702,6 +702,17 @@
             <parent link="chassis" />
             <child link="arm_link" />
+        </joint> -->
+        <!-- Banksia's arm -->
+        <xacro:include filename="$(find rover_description)/banksia_arm/urdf/arm.urdf.xacro" />
+        <joint name="chassis_to_arm_base" type="fixed">
+            <origin xyz="0.234 -0.001 0.116750" rpy="0 0 1.5708"/>
+            <parent link="chassis" />
+            <child link="arm_link" />
         </joint>
+        <xacro:include filename="$(find rover_description)/banksia_arm/urdf/joint_states_with_arm.xacro"/>
     </xacro:if>
+     <xacro:unless value="$(arg arm)">
+        <xacro:include filename="$(find rover_description)/rover7/urdf/joint_states.xacro"/>
+    </xacro:unless>
     <xacro:unless value="$(arg gazebo)">
         <xacro:include filename="$(find rover_description)/rover7/urdf/ros2_control.xacro" />
