Commit message: fix: auto camera in correct spot and building!

File: src/ros/rover/rover_description/rover7/auto/auto_camera.xacro (robot description, xacro)
@@ -4,11 +4,105 @@
 <robot xmlns:xacro="http://www.ros.org/wiki/xacro">
   <xacro:macro name="auto_cam" params="angle">
+    <!-- Auto Mount start -->
+    <link name="clam">
+      <inertial>
+          <origin xyz="4.3618339694e-03 1.2133827812e-02 1.8554431144e-01" rpy="0 0 0" />
+          <mass value="3.34292" />
+          <inertia ixx="1.8690375727e-01" ixy="7.0026990242e-04" ixz="-1.0729852069e-03" iyy="1.7044341425e-01" iyz="4.9400999576e-02" izz="7.5561973482e-02" />
+      </inertial>
+      <visual>
+          <origin xyz="0.138856 0.281 0.00511278" rpy="3.14159 -0.00348764 3.3577e-34" />
+          <geometry>
+              <mesh filename="file://$(find rover_description)/rover7/auto/meshes/clam.stl" />
+          </geometry>
+          <material name="clam_material">
+              <color rgba="0.866667 0.0745098 0.32549 1.0" />
+          </material>
+      </visual>
+      <collision>
+          <origin xyz="0.138821 0.291 0.0151127" rpy="3.14159 -0.00348764 3.3577e-34" />
+          <geometry>
+              <box size="0.3 0.02 0.06" />
+          </geometry>
+      </collision>
+      <collision>
+          <origin xyz="0.278786 0.171 0.0256009" rpy="3.14159 -0.00348764 3.3577e-34" />
+          <geometry>
+              <box size="0.02 0.25 0.04" />
+          </geometry>
+      </collision>
+      <collision>
+          <origin xyz="-0.00121269 0.171 0.0246244" rpy="3.14159 -0.00348764 3.3577e-34" />
+          <geometry>
+              <box size="0.02 0.25 0.04" />
+          </geometry>
+      </collision>
+      <collision>
+          <origin xyz="0.0655542 0.3285 -0.195144" rpy="3.14159 -0.00348764 3.3577e-34" />
+          <geometry>
+              <cylinder length="0.4" radius="0.013" />
+          </geometry>
+      </collision>
+      <collision>
+          <origin xyz="0.226553 0.3285 -0.194583" rpy="3.14159 -0.00348764 3.3577e-34" />
+          <geometry>
+              <cylinder length="0.4" radius="0.013" />
+          </geometry>
+      </collision>
+      <collision>
+          <origin xyz="0.147338 0.331 -0.41986" rpy="3.14159 -0.00348764 3.3577e-34" />
+          <geometry>
+              <box size="0.2 0.04 0.05" />
+          </geometry>
+      </collision>
+    </link>
+    <link name="cameraholder">
+      <inertial>
+          <origin xyz="5.4750170172e-03 -1.5107203475e-01 4.4981914564e-01" rpy="0 0 0" />
+          <mass value="0.118957" />
+          <inertia ixx="8.8360989011e-05" ixy="-1.7069131990e-08" ixz="-1.0337114105e-06" iyy="3.3398137741e-04" iyz="4.8900042893e-06" izz="3.8467123592e-04" />
+      </inertial>
+      <visual>
+          <origin xyz="-0.433382 -0.134345 0.0529562" rpy="8.05372e-18 -1.56731 -3.0463" />
+          <geometry>
+              <mesh filename="file://$(find rover_description)/rover7/auto/meshes/cameraholder.stl" />
+          </geometry>
+          <material name="cameraholder_material">
+              <color rgba="0.866667 0.0745098 0.32549 1.0" />
+          </material>
+      </visual>
+      <collision>
+          <origin xyz="0.00218838 0.0378801 0.0590256" rpy="-0.113446 -1.56731 -3.0463" />
+          <geometry>
+              <box size="0.143 0.086 0.05" />
+          </geometry>
+      </collision>
+    </link>
+    <joint name="oak_to_mount" type="fixed">
+      <origin xyz="0.004 0.12 0.039" rpy="1.5708 0 1.5708" />
+      <parent link="cameraholder" />
+      <child link="camera_link" />
+      <axis xyz="0 0 1" />
+    </joint>
+    <joint name="camera_angle" type="fixed">
+      <origin xyz="0.0859 0.3735 -0.439086" rpy="1.5708 ${-angle*(pi/180)+1.54884} 1.5708" />
+      <parent link="clam" />
+      <child link="cameraholder" />
+      <axis xyz="0 0 1" />
+    </joint>
+    <joint name="auto_mount_to_chassis" type="fixed">
+      <origin xyz="0.124 -0.141 0.04" rpy="3.14159 -1.01333e-15 1.5708" />
+      <parent link="chassis" />
+      <child link="clam" />
+      <axis xyz="0 0 1" />
+    </joint>
+    <!-- Auto Mount stop -->
     <link name="camera_link"/>
-  <!-- Need to be fixed, OR ADD AUTO CAMERA MOUNT to URDF-->
+  <!-- Add camera directly to chassis
     <joint name="camera_joint" type="fixed">
       <origin xyz="0.8 0 0.525" rpy="0 ${angle*(pi/180)} 0"/>
       <parent link="chassis"/>
       <child link="camera_link"/>
-    </joint>
+    </joint> -->
     <xacro:include filename="$(find depthai_descriptions)/urdf/include/depthai_macro.urdf.xacro"/>
     <xacro:depthai_camera

File: src/ros/rover/rover_description/rover7/urdf/rover.urdf.xacro (robot description, xacro)
@@ -683,6 +683,6 @@
     <xacro:include filename="$(find rover_description)/rover7/urdf/ckc.xacro"/>
     <xacro:if value="$(arg auto_camera)">
-        <xacro:include filename="$(find rover_description)/rover7/urdf/auto/auto_camera.xacro"/>
-        <xacro:include filename="$(find rover_description)/rover7/urdf/auto/auto_mount.xacro"/>
+        <xacro:include filename="$(find rover_description)/rover7/auto/auto_camera.xacro"/>
+        <!--xacro:include filename="$(find rover_description)/rover7/auto/auto_mount.xacro"/-->
         <xacro:auto_cam angle="$(arg angle)"></xacro:auto_cam>
     </xacro:if>

Commit message: feat: Added bootie mount (no scad) must fix oaks positions

File: src/ros/rover/rover_description/rover7/auto/auto_camera.xacro (robot description, xacro)
@@ -6,97 +6,120 @@
     <!-- Auto Mount start -->
     <link name="clam">
-      <inertial>
-          <origin xyz="4.3618339694e-03 1.2133827812e-02 1.8554431144e-01" rpy="0 0 0" />
-          <mass value="3.34292" />
-          <inertia ixx="1.8690375727e-01" ixy="7.0026990242e-04" ixz="-1.0729852069e-03" iyy="1.7044341425e-01" iyz="4.9400999576e-02" izz="7.5561973482e-02" />
-      </inertial>
-      <visual>
-          <origin xyz="0.138856 0.281 0.00511278" rpy="3.14159 -0.00348764 3.3577e-34" />
-          <geometry>
-              <mesh filename="file://$(find rover_description)/rover7/auto/meshes/clam.stl" />
-          </geometry>
-          <material name="clam_material">
-              <color rgba="0.866667 0.0745098 0.32549 1.0" />
-          </material>
-      </visual>
-      <collision>
-          <origin xyz="0.138821 0.291 0.0151127" rpy="3.14159 -0.00348764 3.3577e-34" />
-          <geometry>
-              <box size="0.3 0.02 0.06" />
-          </geometry>
-      </collision>
-      <collision>
-          <origin xyz="0.278786 0.171 0.0256009" rpy="3.14159 -0.00348764 3.3577e-34" />
-          <geometry>
-              <box size="0.02 0.25 0.04" />
-          </geometry>
-      </collision>
-      <collision>
-          <origin xyz="-0.00121269 0.171 0.0246244" rpy="3.14159 -0.00348764 3.3577e-34" />
-          <geometry>
-              <box size="0.02 0.25 0.04" />
-          </geometry>
-      </collision>
-      <collision>
-          <origin xyz="0.0655542 0.3285 -0.195144" rpy="3.14159 -0.00348764 3.3577e-34" />
-          <geometry>
-              <cylinder length="0.4" radius="0.013" />
-          </geometry>
-      </collision>
-      <collision>
-          <origin xyz="0.226553 0.3285 -0.194583" rpy="3.14159 -0.00348764 3.3577e-34" />
-          <geometry>
-              <cylinder length="0.4" radius="0.013" />
-          </geometry>
-      </collision>
-      <collision>
-          <origin xyz="0.147338 0.331 -0.41986" rpy="3.14159 -0.00348764 3.3577e-34" />
-          <geometry>
-              <box size="0.2 0.04 0.05" />
-          </geometry>
-      </collision>
-    </link>
-    <link name="cameraholder">
-      <inertial>
-          <origin xyz="5.4750170172e-03 -1.5107203475e-01 4.4981914564e-01" rpy="0 0 0" />
-          <mass value="0.118957" />
-          <inertia ixx="8.8360989011e-05" ixy="-1.7069131990e-08" ixz="-1.0337114105e-06" iyy="3.3398137741e-04" iyz="4.8900042893e-06" izz="3.8467123592e-04" />
-      </inertial>
-      <visual>
-          <origin xyz="-0.433382 -0.134345 0.0529562" rpy="8.05372e-18 -1.56731 -3.0463" />
-          <geometry>
-              <mesh filename="file://$(find rover_description)/rover7/auto/meshes/cameraholder.stl" />
-          </geometry>
-          <material name="cameraholder_material">
-              <color rgba="0.866667 0.0745098 0.32549 1.0" />
-          </material>
-      </visual>
-      <collision>
-          <origin xyz="0.00218838 0.0378801 0.0590256" rpy="-0.113446 -1.56731 -3.0463" />
-          <geometry>
-              <box size="0.143 0.086 0.05" />
-          </geometry>
-      </collision>
-    </link>
-    <joint name="oak_to_mount" type="fixed">
-      <origin xyz="0.004 0.12 0.039" rpy="1.5708 0 1.5708" />
-      <parent link="cameraholder" />
-      <child link="camera_link" />
-      <axis xyz="0 0 1" />
-    </joint>
-    <joint name="camera_angle" type="fixed">
-      <origin xyz="0.0859 0.3735 -0.439086" rpy="1.5708 ${-angle*(pi/180)+1.54884} 1.5708" />
-      <parent link="clam" />
-      <child link="cameraholder" />
-      <axis xyz="0 0 1" />
+        <inertial>
+            <origin xyz="3.7286529733e-03 5.0083863736e-02 6.6873566534e-02" rpy="0 0 0" />
+            <mass value="2.24247" />
+            <inertia ixx="8.0102667275e-02" ixy="5.4258492784e-04" ixz="-5.9405379924e-04" iyy="7.0962055048e-02" iyz="1.8867799978e-02" izz="6.1017587486e-02" />
+        </inertial>
+        <visual>
+            <origin xyz="0.138856 0.281 0.00511278" rpy="3.14159 -0.00348764 3.3577e-34" />
+            <geometry>
+                <mesh filename="file://$(find rover_description)/rover7/auto/meshes/clam.stl" />
+            </geometry>
+            <material name="clam_material">
+                <color rgba="0.866667 0.0745098 0.32549 1.0" />
+            </material>
+        </visual>
+        <collision>
+            <origin xyz="0.138856 0.281 0.00511278" rpy="3.14159 -0.00348764 3.3577e-34" />
+            <geometry>
+                <mesh filename="file://$(find rover_description)/rover7/auto/meshes/clam.stl" />
+            </geometry>
+        </collision>
+    </link>
+    <link name="mount">
+        <inertial>
+            <origin xyz="1.1693270418e-05 -7.2712111739e-04 -9.4424832751e-07" rpy="0 0 0" />
+            <mass value="0.675321" />
+            <inertia ixx="1.3346354813e-03" ixy="2.0144673110e-06" ixz="-7.4564560876e-12" iyy="1.8911012391e-03" iyz="8.5183270804e-12" izz="2.9426778309e-03" />
+        </inertial>
+        <visual>
+            <origin xyz="0.081 0.000713936 -0.025" rpy="4.93038e-32 6.86401e-31 -3.70732e-33" />
+            <geometry>
+                <mesh filename="file://$(find rover_description)/rover7/auto/meshes/mount.stl" />
+            </geometry>
+            <material name="mount_material">
+                <color rgba="0.866667 0.0745098 0.32549 1.0" />
+            </material>
+        </visual>
+        <collision>
+            <origin xyz="0.081 0.000713936 -0.025" rpy="4.93038e-32 6.86401e-31 -3.70732e-33" />
+            <geometry>
+                <mesh filename="file://$(find rover_description)/rover7/auto/meshes/mount.stl" />
+            </geometry>
+        </collision>
+    </link>
+    <link name="camera_holder_front">
+        <inertial>
+            <origin xyz="-3.7228035090e-17 1.6127855240e-02 2.0602657902e-19" rpy="0 0 0" />
+            <mass value="0.138174" />
+            <inertia ixx="1.0267174221e-04" ixy="4.3986965268e-19" ixz="-3.1642726501e-10" iyy="3.8739942592e-04" iyz="-9.5101774211e-22" izz="4.4725908804e-04" />
+        </inertial>
+        <visual>
+            <origin xyz="-0.075 5.55112e-17 0.06" rpy="-1.5708 -1.5708 0" />
+            <geometry>
+                <mesh filename="file://$(find rover_description)/rover7/auto/meshes/camera_holder.stl" />
+            </geometry>
+            <material name="camera_holder_front_material">
+                <color rgba="0.866667 0.0745098 0.32549 1.0" />
+            </material>
+        </visual>
+        <collision>
+            <origin xyz="-0.075 5.55112e-17 0.06" rpy="-1.5708 -1.5708 0" />
+            <geometry>
+                <mesh filename="file://$(find rover_description)/rover7/auto/meshes/camera_holder.stl" />
+            </geometry>
+        </collision>
+    </link>
+    <joint name="mount_to_front_holder" type="fixed">
+        <origin xyz="0.141 0.045 -0.0075" rpy="1.5708 -${(angle)*(pi/180)} -1.5708" />
+        <parent link="mount" />
+        <child link="camera_holder_front" />
+        <axis xyz="0 0 -1" />
+    </joint>
+    <link name="camera_holder_back">
+        <inertial>
+            <origin xyz="-3.7228035090e-17 1.6127855240e-02 2.0602657902e-19" rpy="0 0 0" />
+            <mass value="0.138174" />
+            <inertia ixx="1.0267174221e-04" ixy="4.3986965268e-19" ixz="-3.1642726501e-10" iyy="3.8739942592e-04" iyz="-9.5101774211e-22" izz="4.4725908804e-04" />
+        </inertial>
+        <visual>
+            <origin xyz="-0.075 0 0.06" rpy="1.5708 1.5708 0" />
+            <geometry>
+                <mesh filename="file://$(find rover_description)/rover7/auto/meshes/camera_holder.stl" />
+            </geometry>
+            <material name="camera_holder_back_material">
+                <color rgba="0.866667 0.0745098 0.32549 1.0" />
+            </material>
+        </visual>
+        <collision>
+            <origin xyz="-0.075 0 0.06" rpy="1.5708 1.5708 0" />
+            <geometry>
+                <mesh filename="file://$(find rover_description)/rover7/auto/meshes/camera_holder.stl" />
+            </geometry>
+        </collision>
+    </link>
+    <joint name="mount_to_back_holder" type="fixed">
+        <origin xyz="0.141 -0.045 -0.0075" rpy="-1.5708 ${-angle*(pi/180)} 1.5708" />
+        <parent link="mount" />
+        <child link="camera_holder_back" />
+        <axis xyz="0 0 1" />
+    </joint>
+    <joint name="clam_to_mount" type="fixed">
+        <origin xyz="0.2269 0.3285 -0.436186" rpy="3.14159 5.13507e-14 3.14159" />
+        <parent link="clam" />
+        <child link="mount" />
+        <axis xyz="0 0 1" />
+        <limit effort="10" velocity="10" />
     </joint>
     <joint name="auto_mount_to_chassis" type="fixed">
-      <origin xyz="0.124 -0.141 0.04" rpy="3.14159 -1.01333e-15 1.5708" />
-      <parent link="chassis" />
-      <child link="clam" />
-      <axis xyz="0 0 1" />
+        <origin xyz="0.124 -0.141 0.04" rpy="3.14159 -1.01333e-15 1.5708" />
+        <parent link="chassis" />
+        <child link="clam" />
+        <axis xyz="0 0 1" />
+        <limit effort="10" velocity="10" />
     </joint>
     <!-- Auto Mount stop -->
     <link name="camera_link"/>
+    <link name="bootie_link"/> <!-- KABI OR SOMEONE ADD BOOTIE CAM GAZEBO SENSORS!!! -->
   <!-- Add camera directly to chassis
     <joint name="camera_joint" type="fixed">
@@ -105,4 +128,16 @@
       <child link="camera_link"/>
     </joint> -->
+    <joint name="oak_to_mount" type="fixed">
+      <origin xyz="0.004 0.12 0.039" rpy="0 0 1.5708" />
+      <parent link="camera_holder_front" />
+      <child link="camera_link" />
+      <axis xyz="0 0 1" />
+    </joint>
+    <joint name="bootie_to_mount" type="fixed">
+      <origin xyz="0.004 0.12 0.039" rpy="1.5708 0 1.5708" />
+      <parent link="camera_holder_back" />
+      <child link="bootie_link" />
+      <axis xyz="0 0 1" />
+    </joint>
     <xacro:include filename="$(find depthai_descriptions)/urdf/include/depthai_macro.urdf.xacro"/>
     <xacro:depthai_camera
@@ -110,5 +145,18 @@
       parent="camera_link"
       camera_model="OAK-D-LR"
-      base_frame="oak-d_frame"
+      base_frame="oak_frame"
+      cam_pos_x="0.0"
+      cam_pos_y="0.0"
+      cam_pos_z="0.0"
+      cam_roll="0.0"
+      cam_pitch="0.0"
+      cam_yaw="0.0"
+    />
+    <xacro:include filename="$(find depthai_descriptions)/urdf/include/depthai_macro.urdf.xacro"/>
+    <xacro:depthai_camera
+      camera_name="bootie"
+      parent="bootie_link"
+      camera_model="OAK-D-LR"
+      base_frame="bootie_frame"
       cam_pos_x="0.0"
       cam_pos_y="0.0"

File: src/ros/rover/rover_description/rover7/urdf/rover.urdf.xacro (robot description, xacro)
@@ -685,5 +685,4 @@
     <xacro:if value="$(arg auto_camera)">
         <xacro:include filename="$(find rover_description)/rover7/auto/auto_camera.xacro"/>
-        <!--xacro:include filename="$(find rover_description)/rover7/auto/auto_mount.xacro"/-->
         <xacro:auto_cam angle="$(arg angle)"></xacro:auto_cam>
     </xacro:if>

Commit message: fix: correct camera orientations, feat: added imu and depth to gazebo bootie (untested)

File: src/ros/rover/rover_description/rover7/auto/auto_camera.xacro (robot description, xacro)
@@ -129,5 +129,5 @@
     </joint> -->
     <joint name="oak_to_mount" type="fixed">
-      <origin xyz="0.004 0.12 0.039" rpy="0 0 1.5708" />
+      <origin xyz="-0.120 0.004 0.039" rpy="1.5708 0 3.14159" />
       <parent link="camera_holder_front" />
       <child link="camera_link" />
@@ -135,5 +135,5 @@
     </joint>
     <joint name="bootie_to_mount" type="fixed">
-      <origin xyz="0.004 0.12 0.039" rpy="1.5708 0 1.5708" />
+      <origin xyz="-0.120 -0.004 0.081" rpy="-1.5708 0 3.14159" />
       <parent link="camera_holder_back" />
       <child link="bootie_link" />
@@ -172,5 +172,5 @@
       <child link="camera_link_optical"/>
     </joint>
-    <!-- Depth Camera for Gazebo-->
+    <!-- Front Oak Depth Camera for Gazebo-->
     <gazebo reference="camera_link">
       <sensor name="oak" type="rgbd_camera">
@@ -198,5 +198,31 @@
       </sensor>
     </gazebo>
-    <!-- IMU for Gazebo-->
+    <!-- Bootie Rear Depth Camera for Gazebo-->
+    <gazebo reference="bootie_link">
+      <sensor name="bootie" type="rgbd_camera">
+        <gz_frame_id>bootie_link_optical</gz_frame_id>
+        <!-- Link that corresponds to the Depth Point Clouds -->
+        <optical_frame_id>bootie_link</optical_frame_id>
+        <topic>bootie</topic>
+        <visualize>true</visualize>
+        <update_rate>30</update_rate>
+        <always_on>1</always_on>
+        <camera name="bootie">
+          <horizontal_fov>${radians(82)}</horizontal_fov>
+          <image>
+            <width>1280</width>
+            <height>900</height>
+          </image>
+          <clip>
+            <near>0.4</near>
+            <far>10.0</far>
+          </clip>
+        </camera>
+        <plugin name="gz::sim::systems::Sensors" filename="gz-sim-sensors-system">
+          <frame_name>bootie_link_optical</frame_name>
+        </plugin>
+      </sensor>
+    </gazebo>
+    <!-- Front IMU for Gazebo-->
     <gazebo reference="oak_imu_frame">
       <sensor name="imu_sensor" type="imu">
@@ -265,4 +291,71 @@
       </sensor>
     </gazebo>
+    <!-- Bootie for Gazebo-->
+    <gazebo reference="bootie_imu_frame">
+      <sensor name="bootie_imu_sensor" type="imu">
+        <topic>bootie/imu</topic>
+        <plugin filename="gz-sim-imu-system" name="gz::sim::systems::Imu">
+          <frame_name>bootie_imu_frame</frame_name>
+          <initial_orientation_as_reference>false</initial_orientation_as_reference>
+        </plugin>
+        <always_on>true</always_on>
+        <update_rate>200</update_rate>
+        <visualize>true</visualize>
+        <imu>
+          <angular_velocity>
+            <x>
+              <noise type="gaussian">
+                <mean>0.0</mean>
+                <stddev>2e-4</stddev>
+                <bias_mean>0.0000075</bias_mean>
+                <bias_stddev>0.0000008</bias_stddev>
+              </noise>
+            </x>
+            <y>
+              <noise type="gaussian">
+                <mean>0.0</mean>
+                <stddev>2e-4</stddev>
+                <bias_mean>0.0000075</bias_mean>
+                <bias_stddev>0.0000008</bias_stddev>
+              </noise>
+            </y>
+            <z>
+              <noise type="gaussian">
+                <mean>0.0</mean>
+                <stddev>2e-4</stddev>
+                <bias_mean>0.0000075</bias_mean>
+                <bias_stddev>0.0000008</bias_stddev>
+              </noise>
+            </z>
+          </angular_velocity>
+          <linear_acceleration>
+            <x>
+              <noise type="gaussian">
+                <mean>0.0</mean>
+                <stddev>1.7e-2</stddev>
+                <bias_mean>0.1</bias_mean>
+                <bias_stddev>0.001</bias_stddev>
+              </noise>
+            </x>
+            <y>
+              <noise type="gaussian">
+                <mean>0.0</mean>
+                <stddev>1.7e-2</stddev>
+                <bias_mean>0.1</bias_mean>
+                <bias_stddev>0.001</bias_stddev>
+              </noise>
+            </y>
+            <z>
+              <noise type="gaussian">
+                <mean>0.0</mean>
+                <stddev>1.7e-2</stddev>
+                <bias_mean>0.1</bias_mean>
+                <bias_stddev>0.001</bias_stddev>
+              </noise>
+            </z>
+          </linear_acceleration>
+        </imu>
+      </sensor>
+    </gazebo>
   </xacro:macro>
 </robot>
