Commit message: fix: IK for the new arm urdf files

File: src/ros/rover/rover_description/banksia_arm/urdf/arm.urdf.xacro (robot description, xacro)
@@ -416,4 +416,5 @@
     <axis xyz="0 0 1" />
     <limit effort="10" velocity="10" />
+    <mimic joint="J3" multiplier="1" offset="0"/>
   </joint>
   <joint name="J2" type="revolute">
@@ -534,5 +535,5 @@
   <link name="arm_kinematics_origin"/>
   <joint name="arm_kinematics_origin_joint" type="fixed">
-    <origin xyz="0.0 0.0 0.0" rpy="0.0 0.0 0.0" />
+    <origin xyz="0.0 0.0 0.196" rpy="0.0 0.0 -1.57079632679" />
     <parent link="armmount" />
     <child link="arm_kinematics_origin" />
@@ -542,5 +543,5 @@
   <joint name="endeffector_kinematics_joint" type="fixed">
     <!-- before rotating to match IK function expected 0: 1.5707963 0.0 1.5707963 -->
-    <origin xyz="0.0138 0.0 -0.012512" rpy="1.5707963 0.0 1.5707963" />
+    <origin xyz="0.0067503 -0.0012 0.2225" rpy="-1.57079632679 -1.57079632679 0.0" />
     <parent link="eebase" />
     <child link="endeffector_kinematics" />

Commit message: fix: Correct camera positions and frames for arm

File: src/ros/rover/rover_description/banksia_arm/urdf/arm.urdf.xacro (robot description, xacro)
@@ -231,5 +231,5 @@
   </link>
   <joint name="camera_ee_side" type="fixed">
-    <origin xyz="-0.000216235 0.178108 -0.0547417" rpy="3.14159 0.00174763 1.5708" />
+    <origin xyz="-0.000216235 0.178108 -0.0547417" rpy="0 0.00174763 3.14159" />
     <parent link="rightfinger" />
     <child link="arm_end_side" />
@@ -318,5 +318,5 @@
   </link>
   <joint name="camera_ee_finger" type="fixed">
-    <origin xyz="1.96205e-05 -0.0711415 -0.0299814" rpy="-3.14152 1.52166 -1.5708" />
+    <origin xyz="1.96205e-05 -0.0711415 -0.0299814" rpy="-3.14152 ${radians(180) + 1.52166} -1.5708" />
     <parent link="leftfinger" />
     <child link="arm_end_finger" />
@@ -354,5 +354,5 @@
   </link>
   <joint name="camera_ee_top" type="fixed">
-    <origin xyz="-6.33269e-14 0.10042 0.231753" rpy="3.14159 -1.56853 1.5708" />
+    <origin xyz="-6.33269e-14 0.10042 0.231753" rpy="1.5708 ${-1.56853 - radians(90)} 0" />
     <parent link="eebase" />
     <child link="arm_end_top" />
@@ -383,5 +383,5 @@
   </link>
   <joint name="camera_ee_periscope" type="fixed">
-    <origin xyz="-0.00015 -0.0378336 0.0594947" rpy="-3.14159 -1.5708 1.5708" />
+     <origin xyz="-0.00015 -0.0378336 0.0594947" rpy="-3.14159 -3.14159 0" />
     <parent link="eebase" />
     <child link="arm_end_periscope" />

File: src/ros/rover/rover_description/banksia_arm/urdf/arm_joints.xacro (robot description, xacro)
@@ -4,5 +4,5 @@
      <gazebo>
           <plugin filename="gz-sim-joint-state-publisher-system" name="gz::sim::systems::JointStatePublisher">
-               <topic>arm_joints</topic>
+               <topic>joint_states</topic>
                <joint_name>arm_kinematics_origin_joint</joint_name>
                <joint_name>J1</joint_name>

File: src/ros/rover/rover_description/banksia_arm/urdf/arm_sensors.xacro (robot description, xacro)
@@ -10,4 +10,5 @@
       <!-- Note: plugin only needs to be loaded once, auto_mount also loads this plugin, so arm and auto_mount cannot both exist -->
       <plugin name="gz::sim::systems::Sensors" filename="gz-sim-sensors-system"></plugin>
+      <pose> 0 0 0 0 ${radians(-90)} ${radians(90)}</pose> <!-- To compensate for gazebo frame to ros optical frame-->
       <gz_frame_id>arm_end_top</gz_frame_id>
       <optical_frame_id>arm_end_top</optical_frame_id>
@@ -26,6 +27,5 @@
         </image>
         <clip>
-          <!-- "Fixed focus from 0.3m to 1.5m" since clip prevents seeing past each value, this has been relaxed to 0.3m to 10m-->
-          <near>0.3</near>
+          <near>0.001</near>
           <far>10</far>
         </clip>
@@ -35,4 +35,5 @@
   <gazebo reference="arm_end_periscope">
     <sensor name="arm_end_periscope" type="camera">
+      <pose> 0 0 0 0 ${radians(-90)} ${radians(90)}</pose> <!-- To compensate for gazebo frame to ros optical frame-->
       <gz_frame_id>arm_end_periscope</gz_frame_id>
       <optical_frame_id>arm_end_periscope</optical_frame_id>
@@ -51,6 +52,5 @@
         </image>
         <clip>
-          <!-- "Fixed focus from 0.3m to 1.5m" since clip prevents seeing past each value, this has been relaxed to 0.3m to 10m-->
-          <near>0.3</near>
+          <near>0.05</near>
           <far>10</far>
         </clip>
@@ -60,4 +60,5 @@
   <gazebo reference="arm_end_side">
     <sensor name="arm_end_side" type="camera">
+      <pose> 0 0 0 ${radians(-90)} 0 ${radians(-90)}</pose> <!-- To compensate for gazebo frame to ros optical frame-->
       <gz_frame_id>arm_end_side</gz_frame_id>
       <optical_frame_id>arm_end_side</optical_frame_id>
@@ -76,6 +77,5 @@
         </image>
         <clip>
-          <!-- "Fixed focus from 0.3m to 1.5m" since clip prevents seeing past each value, this has been relaxed to 0.3m to 10m-->
-          <near>0.3</near>
+          <near>0.01</near>
           <far>10</far>
         </clip>
@@ -85,4 +85,5 @@
   <gazebo reference="arm_end_finger">
     <sensor name="arm_end_finger" type="camera">
+      <pose> 0 0 0 0 ${radians(-90)} ${radians(90)}</pose> <!-- To compensate for gazebo frame to ros optical frame-->
       <gz_frame_id>arm_end_finger</gz_frame_id>
       <optical_frame_id>arm_end_finger</optical_frame_id>
@@ -101,6 +102,5 @@
         </image>
         <clip>
-          <!-- "Fixed focus from 0.3m to 1.5m" since clip prevents seeing past each value, this has been relaxed to 0.3m to 10m-->
-          <near>0.3</near>
+          <near>0.01</near>
           <far>10</far>
         </clip>

Commit message: temp: Fix arm in zero position

File: src/ros/rover/rover_description/banksia_arm/urdf/arm.urdf.xacro (robot description, xacro)
@@ -389,10 +389,10 @@
     <limit effort="10" velocity="10" />
   </joint>
-  <joint name="J6" type="continuous">
+  <joint name="J6" type="revolute">
     <origin xyz="5.64652e-16 -0.1945 0.05075" rpy="1.5708 -1.48145e-14 2.12503e-17" />
     <parent link="j6" />
     <child link="eebase" />
     <axis xyz="0 0 1" />
-    <limit effort="10" velocity="10" />
+    <limit effort="10" velocity="10" lower="0" upper="0"/>
   </joint>
   <joint name="J5" type="revolute">
@@ -401,5 +401,5 @@
     <child link="j6" />
     <axis xyz="0 0 1" />
-    <limit effort="10" velocity="10" lower="-1.5708" upper="1.91986" />
+    <limit effort="10" velocity="10" lower="0" upper="0" />
   </joint>
   <joint name="J4" type="revolute">
@@ -408,12 +408,12 @@
     <child link="j5" />
     <axis xyz="0 0 1" />
-    <limit effort="10" velocity="10" lower="-1.5708" upper="1.5708" />
-  </joint>
-  <joint name="l1a_tp" type="continuous">
+    <limit effort="10" velocity="10" lower="0" upper="0" />
+  </joint>
+  <joint name="l1a_tp" type="revolute">
     <origin xyz="7.73032e-10 -0.5 0.0239" rpy="5.57224e-15 1.15529e-15 1.5708" />
     <parent link="l1" />
     <child link="l2" />
     <axis xyz="0 0 1" />
-    <limit effort="10" velocity="10" />
+    <limit effort="10" velocity="10" lower="0" upper="0"/>
     <mimic joint="J3" multiplier="1" offset="0"/>
   </joint>
@@ -423,5 +423,5 @@
     <child link="l1" />
     <axis xyz="0 0 1" />
-    <limit effort="10" velocity="10" lower="-3.141592653589793" upper="3.141592653589793" />
+    <limit effort="10" velocity="10" lower="0" upper="0" />
   </joint>
   <link name="l2prime">
@@ -491,17 +491,17 @@
     </collision>
   </link>
-  <joint name="l1b_tp" type="continuous">
+  <joint name="l1b_tp" type="revolute">
     <origin xyz="3.05311e-16 -0.5 5.77479e-16" rpy="-1.0988e-15 4.62615e-16 0.648016" />
     <parent link="l1prime" />
     <child link="l2cam" />
     <axis xyz="0 0 1" />
-    <limit effort="10" velocity="10" />
-  </joint>
-  <joint name="l1b_bp" type="continuous">
+    <limit effort="10" velocity="10" lower="0" upper="0"/>
+  </joint>
+  <joint name="l1b_bp" type="revolute">
     <origin xyz="0.0797283 -0.0603606 -0.006" rpy="-1.08371e-22 -4.6005e-22 -0.648016" />
     <parent link="l2prime" />
     <child link="l1prime" />
     <axis xyz="0 0 1" />
-    <limit effort="10" velocity="10" />
+    <limit effort="10" velocity="10" lower="0" upper="0"/>
   </joint>
   <joint name="J3" type="revolute">
@@ -510,12 +510,12 @@
     <child link="l2prime" />
     <axis xyz="0 0 1" />
-    <limit effort="10" velocity="10" lower="-3.141592653589793" upper="3.141592653589793" />
-  </joint>
-  <joint name="J1" type="continuous">
+    <limit effort="10" velocity="10" lower="0" upper="0" />
+  </joint>
+  <joint name="J1" type="revolute">
     <origin xyz="-2.45166e-16 -1.77636e-15 -0.062" rpy="3.14159 -0 -7.70285e-39" />
     <parent link="gearbox" />
     <child link="linkagedrive" />
     <axis xyz="0 0 1" />
-    <limit effort="10" velocity="10" />
+    <limit effort="10" velocity="10" lower="0" upper="0"/>
   </joint>
   <joint name="base_to_gearbox" type="fixed">

Commit message: fix: rename arm cameras to add _optical suffix to follow REP103

File: src/ros/rover/rover_description/banksia_arm/urdf/arm.urdf.xacro (robot description, xacro)
@@ -208,5 +208,5 @@
     </collision>
   </link>
-  <link name="arm_end_side">
+  <link name="arm_end_side_optical">
     <inertial>
       <origin xyz="5.0388580281e-20 -5.0000002375e-04 -2.0596424901e-20" rpy="0 0 0" />
@@ -233,5 +233,5 @@
     <origin xyz="-0.000216235 0.178108 -0.0547417" rpy="0 0.00174763 3.14159" />
     <parent link="rightfinger" />
-    <child link="arm_end_side" />
+    <child link="arm_end_side_optical" />
     <axis xyz="0 0 1" />
     <limit effort="10" velocity="10" />
@@ -295,5 +295,5 @@
     <limit effort="10" velocity="10" lower="-1.22125e-15" upper="0.055" />
   </joint>
-  <link name="arm_end_finger">
+  <link name="arm_end_finger_optical">
     <inertial>
       <origin xyz="5.0388580281e-20 -5.0000002375e-04 -2.0596424901e-20" rpy="0 0 0" />
@@ -320,5 +320,5 @@
     <origin xyz="1.96205e-05 -0.0711415 -0.0299814" rpy="-3.14152 ${radians(180) + 1.52166} -1.5708" />
     <parent link="leftfinger" />
-    <child link="arm_end_finger" />
+    <child link="arm_end_finger_optical" />
     <axis xyz="0 0 1" />
     <limit effort="10" velocity="10" />
@@ -331,5 +331,5 @@
     <limit effort="10" velocity="10" lower="0" upper="0.084" />
   </joint>
-  <link name="arm_end_top">
+  <link name="arm_end_top_optical">
     <inertial>
       <origin xyz="5.0388580281e-20 -5.0000002375e-04 -2.0596424901e-20" rpy="0 0 0" />
@@ -356,9 +356,9 @@
     <origin xyz="-6.33269e-14 0.10042 0.231753" rpy="1.5708 ${-1.56853 - radians(90)} 0" />
     <parent link="eebase" />
-    <child link="arm_end_top" />
+    <child link="arm_end_top_optical" />
     <axis xyz="0 0 1" />
     <limit effort="10" velocity="10" />
   </joint>
-  <link name="arm_end_periscope">
+  <link name="arm_end_periscope_optical">
     <inertial>
       <origin xyz="5.0388580281e-20 -5.0000002375e-04 -2.0596424901e-20" rpy="0 0 0" />
@@ -385,5 +385,5 @@
      <origin xyz="-0.00015 -0.0378336 0.0594947" rpy="-3.14159 -3.14159 0" />
     <parent link="eebase" />
-    <child link="arm_end_periscope" />
+    <child link="arm_end_periscope_optical" />
     <axis xyz="0 0 1" />
     <limit effort="10" velocity="10" />

File: src/ros/rover/rover_description/banksia_arm/urdf/arm_sensors.xacro (robot description, xacro)
@@ -6,5 +6,5 @@
   <!-- Based on Microsoft Lifecam HD-3000 specs -->
   <!-- https://dl2jx7zfbtwvr.cloudfront.net/specsheets/WEBC1010.pdf -->
-  <gazebo reference="arm_end_top">
+  <gazebo reference="arm_end_top_optical">
     <sensor name="arm_end_top" type="camera">
       <!-- Note: plugin only needs to be loaded once, auto_mount also loads this plugin, so arm and auto_mount cannot both exist -->
@@ -33,5 +33,5 @@
     </sensor>
   </gazebo>
-  <gazebo reference="arm_end_periscope">
+  <gazebo reference="arm_end_periscope_optical">
     <sensor name="arm_end_periscope" type="camera">
       <pose> 0 0 0 0 ${radians(-90)} ${radians(90)}</pose> <!-- To compensate for gazebo frame to ros optical frame-->
@@ -58,5 +58,5 @@
     </sensor>
   </gazebo>
-  <gazebo reference="arm_end_side">
+  <gazebo reference="arm_end_side_optical">
     <sensor name="arm_end_side" type="camera">
       <pose> 0 0 0 ${radians(-90)} 0 ${radians(-90)}</pose> <!-- To compensate for gazebo frame to ros optical frame-->
@@ -83,5 +83,5 @@
     </sensor>
   </gazebo>
-  <gazebo reference="arm_end_finger">
+  <gazebo reference="arm_end_finger_optical">
     <sensor name="arm_end_finger" type="camera">
       <pose> 0 0 0 0 ${radians(-90)} ${radians(90)}</pose> <!-- To compensate for gazebo frame to ros optical frame-->
@@ -109,5 +109,2 @@
   </gazebo>
 </robot>
-<!-- arm_end_top -->
-<!-- arm_end_periscope -->
-<!-- arm_end_finger -->
