Commit message: feat: MVP for collision checking

File: src/ros/rover/rover_description/banksia_arm/urdf/arm.urdf.xacro (robot description, xacro)
@@ -25,10 +25,10 @@
       </material>
     </visual>
-    <collision>
-      <origin xyz="-0.0671788 0.129712 -0.183721" rpy="-1.88173e-16 -1.99729e-09 -1.5708" />
-      <geometry>
-        <mesh filename="file://$(find rover_description)/banksia_arm/meshes/armmount.stl" />
-      </geometry>
-    </collision>
+<!--    <collision>-->
+<!--      <origin xyz="-0.0671788 0.129712 -0.183721" rpy="-1.88173e-16 -1.99729e-09 -1.5708" />-->
+<!--      <geometry>-->
+<!--        <mesh filename="file://$(find rover_description)/banksia_arm/meshes/armmount.stl" />-->
+<!--      </geometry>-->
+<!--    </collision>-->
   </link>
   <link name="gearbox">
@@ -49,7 +49,7 @@
     <collision>
       <origin xyz="-9.93063e-18 0 5.55112e-17" rpy="3.14159 -0 -7.70285e-39" />
-      <geometry>
-        <mesh filename="file://$(find rover_description)/banksia_arm/meshes/gearbox.stl" />
-      </geometry>
+<!--      <geometry>-->
+<!--        <mesh filename="file://$(find rover_description)/banksia_arm/meshes/gearbox.stl" />-->
+<!--      </geometry>-->
     </collision>
   </link>
@@ -71,7 +71,7 @@
     <collision>
       <origin xyz="-1.58901e-15 -1.36391e-16 -5.55112e-17" rpy="6.68673e-23 -1.0222e-22 2.39693e-07" />
-      <geometry>
-        <mesh filename="file://$(find rover_description)/banksia_arm/meshes/linkagedrive.stl" />
-      </geometry>
+<!--      <geometry>-->
+<!--        <mesh filename="file://$(find rover_description)/banksia_arm/meshes/linkagedrive.stl" />-->
+<!--      </geometry>-->
     </collision>
   </link>
@@ -91,10 +91,10 @@
       </material>
     </visual>
-    <collision>
-      <origin xyz="3.1979e-15 -6.85563e-15 0.0239" rpy="1.5708 1.5708 0" />
-      <geometry>
-        <mesh filename="file://$(find rover_description)/banksia_arm/meshes/l1.stl" />
-      </geometry>
-    </collision>
+<!--    <collision>-->
+<!--      <origin xyz="3.1979e-15 -6.85563e-15 0.0239" rpy="1.5708 1.5708 0" />-->
+<!--      <geometry>-->
+<!--        <mesh filename="file://$(find rover_description)/banksia_arm/meshes/l1.stl" />-->
+<!--      </geometry>-->
+<!--    </collision>-->
   </link>
   <link name="l2">
@@ -113,8 +113,50 @@
       </material>
     </visual>
-    <collision>
-      <origin xyz="0.398641 0.301803 6.48063e-16" rpy="2.49358 1.5708 0" />
-      <geometry>
-        <mesh filename="file://$(find rover_description)/banksia_arm/meshes/l2.stl" />
+<!--    <collision>-->
+<!--      <origin xyz="0.398641 0.301803 6.48063e-16" rpy="2.49358 1.5708 0" />-->
+<!--      <geometry>-->
+<!--        <mesh filename="file://$(find rover_description)/banksia_arm/meshes/l2.stl" />-->
+<!--      </geometry>-->
+<!--    </collision>-->
+    <collision>
+      <origin xyz="0 0.11 0" rpy="0 0 0" />
+      <geometry>
+        <box size="0.04 0.44 0.028"/>
+      </geometry>
+    </collision>
+    <collision>
+      <origin xyz="0 0.33 0.0065" rpy="0 0 0" />
+      <geometry>
+        <box size="0.026 0.013 0.123"/>
+      </geometry>
+    </collision>
+    <collision>
+      <origin xyz="0 0.379 0.065" rpy="0 0 0" />
+      <geometry>
+        <box size="0.026 0.11 0.01"/>
+      </geometry>
+    </collision>
+    <collision>
+      <origin xyz="0 0.379 -0.05" rpy="0 0 0" />
+      <geometry>
+        <box size="0.026 0.11 0.01"/>
+      </geometry>
+    </collision>
+    <collision>
+      <origin xyz="0 0.349 -0.072" rpy="0 0 0" />
+      <geometry>
+        <box size="0.041 0.185 0.03"/>
+      </geometry>
+    </collision>
+    <collision>
+      <origin xyz="0 0.3635 -0.072" rpy="0 0 0" />
+      <geometry>
+        <box size="0.07 0.02 0.03"/>
+      </geometry>
+    </collision>
+    <collision>
+      <origin xyz="0 0.275 -0.0025" rpy="0 0 0" />
+      <geometry>
+        <cylinder length="0.082" radius="0.045"/>
       </geometry>
     </collision>
@@ -135,10 +177,10 @@
       </material>
     </visual>
-    <collision>
-      <origin xyz="1.94289e-15 0.05075 -0.0795" rpy="1.5708 1.5708 0" />
-      <geometry>
-        <mesh filename="file://$(find rover_description)/banksia_arm/meshes/j5.stl" />
-      </geometry>
-    </collision>
+<!--    <collision>-->
+<!--      <origin xyz="1.94289e-15 0.05075 -0.0795" rpy="1.5708 1.5708 0" />-->
+<!--      <geometry>-->
+<!--        <mesh filename="file://$(find rover_description)/banksia_arm/meshes/j5.stl" />-->
+<!--      </geometry>-->
+<!--    </collision>-->
   </link>
   <link name="j6">
@@ -157,8 +199,32 @@
       </material>
     </visual>
-    <collision>
-      <origin xyz="5.80265e-16 -0.1945 0.05075" rpy="-1.5708 -1.48145e-14 -7.47144e-23" />
-      <geometry>
-        <mesh filename="file://$(find rover_description)/banksia_arm/meshes/j6.stl" />
+<!--    <collision>-->
+<!--      <origin xyz="5.80265e-16 -0.1945 0.05075" rpy="-1.5708 -1.48145e-14 -7.47144e-23" />-->
+<!--      <geometry>-->
+<!--        <mesh filename="file://$(find rover_description)/banksia_arm/meshes/j6.stl" />-->
+<!--      </geometry>-->
+<!--    </collision>-->
+    <collision>
+      <origin xyz="0 -0.09 0.1" rpy="0 0 0" />
+      <geometry>
+        <box size="0.06 0.2 0.01"/>
+      </geometry>
+    </collision>
+    <collision>
+      <origin xyz="0 -0.09 0" rpy="0 0 0" />
+      <geometry>
+        <box size="0.06 0.2 0.01"/>
+      </geometry>
+    </collision>
+    <collision>
+      <origin xyz="0 -0.145 0.05" rpy="0 0 0" />
+      <geometry>
+        <box size="0.06 0.09 0.1"/>
+      </geometry>
+    </collision>
+    <collision>
+      <origin xyz="0 -0.169 0.05" rpy="1.5708 0 0" />
+      <geometry>
+        <cylinder length="0.025" radius="0.045"/>
       </geometry>
     </collision>
@@ -179,8 +245,14 @@
       </material>
     </visual>
-    <collision>
-      <origin xyz="0.00775 0.013 0.0215" rpy="-6.15694e-07 4.61983e-15 3.14159" />
-      <geometry>
-        <mesh filename="file://$(find rover_description)/banksia_arm/meshes/eebase.stl" />
+<!--    <collision>-->
+<!--      <origin xyz="0.00775 0.013 0.0215" rpy="-6.15694e-07 4.61983e-15 3.14159" />-->
+<!--      <geometry>-->
+<!--        <mesh filename="file://$(find rover_description)/banksia_arm/meshes/eebase.stl" />-->
+<!--      </geometry>-->
+<!--    </collision>-->
+    <collision>
+      <origin xyz="0 0.02 0.0675" rpy="0 0 0" />
+      <geometry>
+        <box size="0.25 0.08 0.075"/>
       </geometry>
     </collision>
@@ -201,10 +273,10 @@
       </material>
     </visual>
-    <collision>
-      <origin xyz="-3.64856e-05 0.115305 0.0109" rpy="-3.14159 -6.60532e-30 2.57948e-23" />
-      <geometry>
-        <mesh filename="file://$(find rover_description)/banksia_arm/meshes/rightfinger.stl" />
-      </geometry>
-    </collision>
+<!--    <collision>-->
+<!--      <origin xyz="-3.64856e-05 0.115305 0.0109" rpy="-3.14159 -6.60532e-30 2.57948e-23" />-->
+<!--      <geometry>-->
+<!--        <mesh filename="file://$(find rover_description)/banksia_arm/meshes/rightfinger.stl" />-->
+<!--      </geometry>-->
+<!--    </collision>-->
   </link>
   <link name="arm_end_side">
@@ -223,10 +295,10 @@
       </material>
     </visual>
-    <collision>
-      <origin xyz="0 0 0" rpy="1.5708 1.86776e-19 -2.0576e-24" />
-      <geometry>
-        <mesh filename="file://$(find rover_description)/banksia_arm/meshes/arm_end_side.stl" />
-      </geometry>
-    </collision>
+<!--    <collision>-->
+<!--      <origin xyz="0 0 0" rpy="1.5708 1.86776e-19 -2.0576e-24" />-->
+<!--      <geometry>-->
+<!--        <mesh filename="file://$(find rover_description)/banksia_arm/meshes/arm_end_side.stl" />-->
+<!--      </geometry>-->
+<!--    </collision>-->
   </link>
   <joint name="camera_ee_side" type="fixed">
@@ -259,10 +331,10 @@
       </material>
     </visual>
-    <collision>
-      <origin xyz="-8.71485e-06 -0.115251 0.0109" rpy="-3.14159 4.996e-15 -5.80744e-23" />
-      <geometry>
-        <mesh filename="file://$(find rover_description)/banksia_arm/meshes/leftfinger.stl" />
-      </geometry>
-    </collision>
+<!--    <collision>-->
+<!--      <origin xyz="-8.71485e-06 -0.115251 0.0109" rpy="-3.14159 4.996e-15 -5.80744e-23" />-->
+<!--      <geometry>-->
+<!--        <mesh filename="file://$(find rover_description)/banksia_arm/meshes/leftfinger.stl" />-->
+<!--      </geometry>-->
+<!--    </collision>-->
   </link>
   <link name="actuator">
@@ -281,10 +353,10 @@
       </material>
     </visual>
-    <collision>
-      <origin xyz="-1.38778e-17 0 -0.058" rpy="3.11287e-20 2.12505e-23 1.99292e-27" />
-      <geometry>
-        <mesh filename="file://$(find rover_description)/banksia_arm/meshes/actuator.stl" />
-      </geometry>
-    </collision>
+<!--    <collision>-->
+<!--      <origin xyz="-1.38778e-17 0 -0.058" rpy="3.11287e-20 2.12505e-23 1.99292e-27" />-->
+<!--      <geometry>-->
+<!--        <mesh filename="file://$(find rover_description)/banksia_arm/meshes/actuator.stl" />-->
+<!--      </geometry>-->
+<!--    </collision>-->
   </link>
   <joint name="actuator_head" type="prismatic">
@@ -310,10 +382,10 @@
       </material>
     </visual>
-    <collision>
-      <origin xyz="2.77556e-17 0 -1.11022e-16" rpy="1.5708 -2.87448e-18 1.5822e-23" />
-      <geometry>
-        <mesh filename="file://$(find rover_description)/banksia_arm/meshes/arm_end_finger.stl" />
-      </geometry>
-    </collision>
+<!--    <collision>-->
+<!--      <origin xyz="2.77556e-17 0 -1.11022e-16" rpy="1.5708 -2.87448e-18 1.5822e-23" />-->
+<!--      <geometry>-->
+<!--        <mesh filename="file://$(find rover_description)/banksia_arm/meshes/arm_end_finger.stl" />-->
+<!--      </geometry>-->
+<!--    </collision>-->
   </link>
   <joint name="camera_ee_finger" type="fixed">
@@ -346,10 +418,10 @@
       </material>
     </visual>
-    <collision>
-      <origin xyz="1.11022e-16 0 0" rpy="1.5708 -2.5589e-20 3.89707e-23" />
-      <geometry>
-        <mesh filename="file://$(find rover_description)/banksia_arm/meshes/arm_end_top.stl" />
-      </geometry>
-    </collision>
+<!--    <collision>-->
+<!--      <origin xyz="1.11022e-16 0 0" rpy="1.5708 -2.5589e-20 3.89707e-23" />-->
+<!--      <geometry>-->
+<!--        <mesh filename="file://$(find rover_description)/banksia_arm/meshes/arm_end_top.stl" />-->
+<!--      </geometry>-->
+<!--    </collision>-->
   </link>
   <joint name="camera_ee_top" type="fixed">
@@ -375,10 +447,10 @@
       </material>
     </visual>
-    <collision>
-      <origin xyz="0 0 0" rpy="1.5708 -1.12386e-23 -2.15772e-29" />
-      <geometry>
-        <mesh filename="file://$(find rover_description)/banksia_arm/meshes/arm_end_periscope.stl" />
-      </geometry>
-    </collision>
+<!--    <collision>-->
+<!--      <origin xyz="0 0 0" rpy="1.5708 -1.12386e-23 -2.15772e-29" />-->
+<!--      <geometry>-->
+<!--        <mesh filename="file://$(find rover_description)/banksia_arm/meshes/arm_end_periscope.stl" />-->
+<!--      </geometry>-->
+<!--    </collision>-->
   </link>
   <joint name="camera_ee_periscope" type="fixed">
@@ -440,10 +512,10 @@
       </material>
     </visual>
-    <collision>
-      <origin xyz="2.77556e-17 0 -0.006" rpy="1.5708 1.5708 0" />
-      <geometry>
-        <mesh filename="file://$(find rover_description)/banksia_arm/meshes/l2prime.stl" />
-      </geometry>
-    </collision>
+<!--    <collision>-->
+<!--      <origin xyz="2.77556e-17 0 -0.006" rpy="1.5708 1.5708 0" />-->
+<!--      <geometry>-->
+<!--        <mesh filename="file://$(find rover_description)/banksia_arm/meshes/l2prime.stl" />-->
+<!--      </geometry>-->
+<!--    </collision>-->
   </link>
   <link name="l1prime">
@@ -464,7 +536,7 @@
     <collision>
       <origin xyz="-0.0797283 0.0603606 1.05415e-16" rpy="1.5708 1.5708 0" />
-      <geometry>
-        <mesh filename="file://$(find rover_description)/banksia_arm/meshes/l1prime.stl" />
-      </geometry>
+<!--      <geometry>-->
+<!--        <mesh filename="file://$(find rover_description)/banksia_arm/meshes/l1prime.stl" />-->
+<!--      </geometry>-->
     </collision>
   </link>
@@ -486,7 +558,7 @@
     <collision>
       <origin xyz="-0.0797283 0.560361 2.48639e-16" rpy="1.5708 1.5708 0" />
-      <geometry>
-        <mesh filename="file://$(find rover_description)/banksia_arm/meshes/l2cam.stl" />
-      </geometry>
+<!--      <geometry>-->
+<!--        <mesh filename="file://$(find rover_description)/banksia_arm/meshes/l2cam.stl" />-->
+<!--      </geometry>-->
     </collision>
   </link>

Commit message: feat: l1 collider

File: src/ros/rover/rover_description/banksia_arm/urdf/arm.urdf.xacro (robot description, xacro)
@@ -97,4 +97,10 @@
 <!--      </geometry>-->
 <!--    </collision>-->
+    <collision>
+      <origin xyz="0 -0.255 0.024" rpy="0 0 0" />
+      <geometry>
+        <box size="0.043 0.53 0.1125"/>
+      </geometry>
+    </collision>
   </link>
   <link name="l2">

Commit message: feat: simple colliders for armmount and linkagedrive

File: src/ros/rover/rover_description/banksia_arm/urdf/arm.urdf.xacro (robot description, xacro)
@@ -31,4 +31,10 @@
 <!--      </geometry>-->
 <!--    </collision>-->
+    <collision>
+      <origin xyz="0 0 -0.085" rpy="0 0 0" />
+      <geometry>
+        <box size="0.34 0.27 0.19"/>
+      </geometry>
+    </collision>
   </link>
   <link name="gearbox">
@@ -69,9 +75,21 @@
       </material>
     </visual>
-    <collision>
-      <origin xyz="-1.58901e-15 -1.36391e-16 -5.55112e-17" rpy="6.68673e-23 -1.0222e-22 2.39693e-07" />
+<!--    <collision>-->
+<!--      <origin xyz="-1.58901e-15 -1.36391e-16 -5.55112e-17" rpy="6.68673e-23 -1.0222e-22 2.39693e-07" />-->
 <!--      <geometry>-->
 <!--        <mesh filename="file://$(find rover_description)/banksia_arm/meshes/linkagedrive.stl" />-->
 <!--      </geometry>-->
+<!--    </collision>-->
+    <collision>
+      <origin xyz="0 0 0.065" rpy="0 0 0" />
+      <geometry>
+        <box size="0.17 0.13 0.13"/>
+      </geometry>
+    </collision>
+    <collision>
+      <origin xyz="0 0 0.13" rpy="0 1.5708 0" />
+      <geometry>
+        <cylinder length="0.33" radius="0.065"/>
+      </geometry>
     </collision>
   </link>

Commit message: Automatic Keyboard Localiser + GUI (#441)

File: src/ros/rover/rover_description/banksia_arm/urdf/arm.urdf.xacro (robot description, xacro)
@@ -208,5 +208,5 @@
     </collision>
   </link>
-  <link name="arm_end_side">
+  <link name="arm_end_side_optical">
     <inertial>
       <origin xyz="5.0388580281e-20 -5.0000002375e-04 -2.0596424901e-20" rpy="0 0 0" />
@@ -233,5 +233,5 @@
     <origin xyz="-0.000216235 0.178108 -0.0547417" rpy="0 0.00174763 3.14159" />
     <parent link="rightfinger" />
-    <child link="arm_end_side" />
+    <child link="arm_end_side_optical" />
     <axis xyz="0 0 1" />
     <limit effort="10" velocity="10" />
@@ -295,5 +295,5 @@
     <limit effort="10" velocity="10" lower="-1.22125e-15" upper="0.055" />
   </joint>
-  <link name="arm_end_finger">
+  <link name="arm_end_finger_optical">
     <inertial>
       <origin xyz="5.0388580281e-20 -5.0000002375e-04 -2.0596424901e-20" rpy="0 0 0" />
@@ -320,5 +320,5 @@
     <origin xyz="1.96205e-05 -0.0711415 -0.0299814" rpy="-3.14152 ${radians(180) + 1.52166} -1.5708" />
     <parent link="leftfinger" />
-    <child link="arm_end_finger" />
+    <child link="arm_end_finger_optical" />
     <axis xyz="0 0 1" />
     <limit effort="10" velocity="10" />
@@ -331,5 +331,5 @@
     <limit effort="10" velocity="10" lower="0" upper="0.084" />
   </joint>
-  <link name="arm_end_top">
+  <link name="arm_end_top_optical">
     <inertial>
       <origin xyz="5.0388580281e-20 -5.0000002375e-04 -2.0596424901e-20" rpy="0 0 0" />
@@ -356,9 +356,9 @@
     <origin xyz="-6.33269e-14 0.10042 0.231753" rpy="1.5708 ${-1.56853 - radians(90)} 0" />
     <parent link="eebase" />
-    <child link="arm_end_top" />
+    <child link="arm_end_top_optical" />
     <axis xyz="0 0 1" />
     <limit effort="10" velocity="10" />
   </joint>
-  <link name="arm_end_periscope">
+  <link name="arm_end_periscope_optical">
     <inertial>
       <origin xyz="5.0388580281e-20 -5.0000002375e-04 -2.0596424901e-20" rpy="0 0 0" />
@@ -385,14 +385,14 @@
      <origin xyz="-0.00015 -0.0378336 0.0594947" rpy="-3.14159 -3.14159 0" />
     <parent link="eebase" />
-    <child link="arm_end_periscope" />
+    <child link="arm_end_periscope_optical" />
     <axis xyz="0 0 1" />
     <limit effort="10" velocity="10" />
   </joint>
-  <joint name="J6" type="continuous">
+  <joint name="J6" type="revolute">
     <origin xyz="5.64652e-16 -0.1945 0.05075" rpy="1.5708 -1.48145e-14 2.12503e-17" />
     <parent link="j6" />
     <child link="eebase" />
     <axis xyz="0 0 1" />
-    <limit effort="10" velocity="10" />
+    <limit effort="10" velocity="10" lower="0" upper="0"/>
   </joint>
   <joint name="J5" type="revolute">
@@ -401,5 +401,5 @@
     <child link="j6" />
     <axis xyz="0 0 1" />
-    <limit effort="10" velocity="10" lower="-1.5708" upper="1.91986" />
+    <limit effort="10" velocity="10" lower="0" upper="0" />
   </joint>
   <joint name="J4" type="revolute">
@@ -408,12 +408,12 @@
     <child link="j5" />
     <axis xyz="0 0 1" />
-    <limit effort="10" velocity="10" lower="-1.5708" upper="1.5708" />
-  </joint>
-  <joint name="l1a_tp" type="continuous">
+    <limit effort="10" velocity="10" lower="0" upper="0" />
+  </joint>
+  <joint name="l1a_tp" type="revolute">
     <origin xyz="7.73032e-10 -0.5 0.0239" rpy="5.57224e-15 1.15529e-15 1.5708" />
     <parent link="l1" />
     <child link="l2" />
     <axis xyz="0 0 1" />
-    <limit effort="10" velocity="10" />
+    <limit effort="10" velocity="10" lower="0" upper="0"/>
     <mimic joint="J3" multiplier="1" offset="0"/>
   </joint>
@@ -423,5 +423,5 @@
     <child link="l1" />
     <axis xyz="0 0 1" />
-    <limit effort="10" velocity="10" lower="-3.141592653589793" upper="3.141592653589793" />
+    <limit effort="10" velocity="10" lower="0" upper="0" />
   </joint>
   <link name="l2prime">
@@ -491,17 +491,17 @@
     </collision>
   </link>
-  <joint name="l1b_tp" type="continuous">
+  <joint name="l1b_tp" type="revolute">
     <origin xyz="3.05311e-16 -0.5 5.77479e-16" rpy="-1.0988e-15 4.62615e-16 0.648016" />
     <parent link="l1prime" />
     <child link="l2cam" />
     <axis xyz="0 0 1" />
-    <limit effort="10" velocity="10" />
-  </joint>
-  <joint name="l1b_bp" type="continuous">
+    <limit effort="10" velocity="10" lower="0" upper="0"/>
+  </joint>
+  <joint name="l1b_bp" type="revolute">
     <origin xyz="0.0797283 -0.0603606 -0.006" rpy="-1.08371e-22 -4.6005e-22 -0.648016" />
     <parent link="l2prime" />
     <child link="l1prime" />
     <axis xyz="0 0 1" />
-    <limit effort="10" velocity="10" />
+    <limit effort="10" velocity="10" lower="0" upper="0"/>
   </joint>
   <joint name="J3" type="revolute">
@@ -510,12 +510,12 @@
     <child link="l2prime" />
     <axis xyz="0 0 1" />
-    <limit effort="10" velocity="10" lower="-3.141592653589793" upper="3.141592653589793" />
-  </joint>
-  <joint name="J1" type="continuous">
+    <limit effort="10" velocity="10" lower="0" upper="0" />
+  </joint>
+  <joint name="J1" type="revolute">
     <origin xyz="-2.45166e-16 -1.77636e-15 -0.062" rpy="3.14159 -0 -7.70285e-39" />
     <parent link="gearbox" />
     <child link="linkagedrive" />
     <axis xyz="0 0 1" />
-    <limit effort="10" velocity="10" />
+    <limit effort="10" velocity="10" lower="0" upper="0"/>
   </joint>
   <joint name="base_to_gearbox" type="fixed">
