Commit message: Self intersection checks in `nova_twistmapper` (#446)
Signed-off-by: Bailey Chessum <bailey.chessum1@gmail.com>

File: src/ros/rover/rover_description/banksia_arm/urdf/arm.urdf.xacro (robot description, xacro)
@@ -25,8 +25,14 @@
       </material>
     </visual>
-    <collision>
-      <origin xyz="-0.0671788 0.129712 -0.183721" rpy="-1.88173e-16 -1.99729e-09 -1.5708" />
-      <geometry>
-        <mesh filename="file://$(find rover_description)/banksia_arm/meshes/armmount.stl" />
+<!--    <collision>-->
+<!--      <origin xyz="-0.0671788 0.129712 -0.183721" rpy="-1.88173e-16 -1.99729e-09 -1.5708" />-->
+<!--      <geometry>-->
+<!--        <mesh filename="file://$(find rover_description)/banksia_arm/meshes/armmount.stl" />-->
+<!--      </geometry>-->
+<!--    </collision>-->
+    <collision>
+      <origin xyz="0 0 -0.085" rpy="0 0 0" />
+      <geometry>
+        <box size="0.34 0.27 0.19"/>
       </geometry>
     </collision>
@@ -49,7 +55,7 @@
     <collision>
       <origin xyz="-9.93063e-18 0 5.55112e-17" rpy="3.14159 -0 -7.70285e-39" />
-      <geometry>
-        <mesh filename="file://$(find rover_description)/banksia_arm/meshes/gearbox.stl" />
-      </geometry>
+<!--      <geometry>-->
+<!--        <mesh filename="file://$(find rover_description)/banksia_arm/meshes/gearbox.stl" />-->
+<!--      </geometry>-->
     </collision>
   </link>
@@ -69,8 +75,20 @@
       </material>
     </visual>
-    <collision>
-      <origin xyz="-1.58901e-15 -1.36391e-16 -5.55112e-17" rpy="6.68673e-23 -1.0222e-22 2.39693e-07" />
-      <geometry>
-        <mesh filename="file://$(find rover_description)/banksia_arm/meshes/linkagedrive.stl" />
+<!--    <collision>-->
+<!--      <origin xyz="-1.58901e-15 -1.36391e-16 -5.55112e-17" rpy="6.68673e-23 -1.0222e-22 2.39693e-07" />-->
+<!--      <geometry>-->
+<!--        <mesh filename="file://$(find rover_description)/banksia_arm/meshes/linkagedrive.stl" />-->
+<!--      </geometry>-->
+<!--    </collision>-->
+    <collision>
+      <origin xyz="0 0 0.065" rpy="0 0 0" />
+      <geometry>
+        <box size="0.17 0.13 0.13"/>
+      </geometry>
+    </collision>
+    <collision>
+      <origin xyz="0 0 0.13" rpy="0 1.5708 0" />
+      <geometry>
+        <cylinder length="0.33" radius="0.065"/>
       </geometry>
     </collision>
@@ -91,8 +109,14 @@
       </material>
     </visual>
-    <collision>
-      <origin xyz="3.1979e-15 -6.85563e-15 0.0239" rpy="1.5708 1.5708 0" />
-      <geometry>
-        <mesh filename="file://$(find rover_description)/banksia_arm/meshes/l1.stl" />
+<!--    <collision>-->
+<!--      <origin xyz="3.1979e-15 -6.85563e-15 0.0239" rpy="1.5708 1.5708 0" />-->
+<!--      <geometry>-->
+<!--        <mesh filename="file://$(find rover_description)/banksia_arm/meshes/l1.stl" />-->
+<!--      </geometry>-->
+<!--    </collision>-->
+    <collision>
+      <origin xyz="0 -0.255 0.024" rpy="0 0 0" />
+      <geometry>
+        <box size="0.043 0.53 0.1125"/>
       </geometry>
     </collision>
@@ -113,8 +137,50 @@
       </material>
     </visual>
-    <collision>
-      <origin xyz="0.398641 0.301803 6.48063e-16" rpy="2.49358 1.5708 0" />
-      <geometry>
-        <mesh filename="file://$(find rover_description)/banksia_arm/meshes/l2.stl" />
+<!--    <collision>-->
+<!--      <origin xyz="0.398641 0.301803 6.48063e-16" rpy="2.49358 1.5708 0" />-->
+<!--      <geometry>-->
+<!--        <mesh filename="file://$(find rover_description)/banksia_arm/meshes/l2.stl" />-->
+<!--      </geometry>-->
+<!--    </collision>-->
+    <collision>
+      <origin xyz="0 0.11 0" rpy="0 0 0" />
+      <geometry>
+        <box size="0.04 0.44 0.028"/>
+      </geometry>
+    </collision>
+    <collision>
+      <origin xyz="0 0.33 0.0065" rpy="0 0 0" />
+      <geometry>
+        <box size="0.026 0.013 0.123"/>
+      </geometry>
+    </collision>
+    <collision>
+      <origin xyz="0 0.379 0.065" rpy="0 0 0" />
+      <geometry>
+        <box size="0.026 0.11 0.01"/>
+      </geometry>
+    </collision>
+    <collision>
+      <origin xyz="0 0.379 -0.05" rpy="0 0 0" />
+      <geometry>
+        <box size="0.026 0.11 0.01"/>
+      </geometry>
+    </collision>
+    <collision>
+      <origin xyz="0 0.349 -0.072" rpy="0 0 0" />
+      <geometry>
+        <box size="0.041 0.185 0.03"/>
+      </geometry>
+    </collision>
+    <collision>
+      <origin xyz="0 0.3635 -0.072" rpy="0 0 0" />
+      <geometry>
+        <box size="0.07 0.02 0.03"/>
+      </geometry>
+    </collision>
+    <collision>
+      <origin xyz="0 0.275 -0.0025" rpy="0 0 0" />
+      <geometry>
+        <cylinder length="0.082" radius="0.045"/>
       </geometry>
     </collision>
@@ -135,10 +201,10 @@
       </material>
     </visual>
-    <collision>
-      <origin xyz="1.94289e-15 0.05075 -0.0795" rpy="1.5708 1.5708 0" />
-      <geometry>
-        <mesh filename="file://$(find rover_description)/banksia_arm/meshes/j5.stl" />
-      </geometry>
-    </collision>
+<!--    <collision>-->
+<!--      <origin xyz="1.94289e-15 0.05075 -0.0795" rpy="1.5708 1.5708 0" />-->
+<!--      <geometry>-->
+<!--        <mesh filename="file://$(find rover_description)/banksia_arm/meshes/j5.stl" />-->
+<!--      </geometry>-->
+<!--    </collision>-->
   </link>
   <link name="j6">
@@ -157,8 +223,32 @@
       </material>
     </visual>
-    <collision>
-      <origin xyz="5.80265e-16 -0.1945 0.05075" rpy="-1.5708 -1.48145e-14 -7.47144e-23" />
-      <geometry>
-        <mesh filename="file://$(find rover_description)/banksia_arm/meshes/j6.stl" />
+<!--    <collision>-->
+<!--      <origin xyz="5.80265e-16 -0.1945 0.05075" rpy="-1.5708 -1.48145e-14 -7.47144e-23" />-->
+<!--      <geometry>-->
+<!--        <mesh filename="file://$(find rover_description)/banksia_arm/meshes/j6.stl" />-->
+<!--      </geometry>-->
+<!--    </collision>-->
+    <collision>
+      <origin xyz="0 -0.09 0.1" rpy="0 0 0" />
+      <geometry>
+        <box size="0.06 0.2 0.01"/>
+      </geometry>
+    </collision>
+    <collision>
+      <origin xyz="0 -0.09 0" rpy="0 0 0" />
+      <geometry>
+        <box size="0.06 0.2 0.01"/>
+      </geometry>
+    </collision>
+    <collision>
+      <origin xyz="0 -0.145 0.05" rpy="0 0 0" />
+      <geometry>
+        <box size="0.06 0.09 0.1"/>
+      </geometry>
+    </collision>
+    <collision>
+      <origin xyz="0 -0.169 0.05" rpy="1.5708 0 0" />
+      <geometry>
+        <cylinder length="0.025" radius="0.045"/>
       </geometry>
     </collision>
@@ -179,8 +269,14 @@
       </material>
     </visual>
-    <collision>
-      <origin xyz="0.00775 0.013 0.0215" rpy="-6.15694e-07 4.61983e-15 3.14159" />
-      <geometry>
-        <mesh filename="file://$(find rover_description)/banksia_arm/meshes/eebase.stl" />
+<!--    <collision>-->
+<!--      <origin xyz="0.00775 0.013 0.0215" rpy="-6.15694e-07 4.61983e-15 3.14159" />-->
+<!--      <geometry>-->
+<!--        <mesh filename="file://$(find rover_description)/banksia_arm/meshes/eebase.stl" />-->
+<!--      </geometry>-->
+<!--    </collision>-->
+    <collision>
+      <origin xyz="0 0.02 0.0675" rpy="0 0 0" />
+      <geometry>
+        <box size="0.25 0.08 0.075"/>
       </geometry>
     </collision>
@@ -201,10 +297,10 @@
       </material>
     </visual>
-    <collision>
-      <origin xyz="-3.64856e-05 0.115305 0.0109" rpy="-3.14159 -6.60532e-30 2.57948e-23" />
-      <geometry>
-        <mesh filename="file://$(find rover_description)/banksia_arm/meshes/rightfinger.stl" />
-      </geometry>
-    </collision>
+<!--    <collision>-->
+<!--      <origin xyz="-3.64856e-05 0.115305 0.0109" rpy="-3.14159 -6.60532e-30 2.57948e-23" />-->
+<!--      <geometry>-->
+<!--        <mesh filename="file://$(find rover_description)/banksia_arm/meshes/rightfinger.stl" />-->
+<!--      </geometry>-->
+<!--    </collision>-->
   </link>
   <link name="arm_end_side_optical">
@@ -223,10 +319,10 @@
       </material>
     </visual>
-    <collision>
-      <origin xyz="0 0 0" rpy="1.5708 1.86776e-19 -2.0576e-24" />
-      <geometry>
-        <mesh filename="file://$(find rover_description)/banksia_arm/meshes/arm_end_side.stl" />
-      </geometry>
-    </collision>
+<!--    <collision>-->
+<!--      <origin xyz="0 0 0" rpy="1.5708 1.86776e-19 -2.0576e-24" />-->
+<!--      <geometry>-->
+<!--        <mesh filename="file://$(find rover_description)/banksia_arm/meshes/arm_end_side.stl" />-->
+<!--      </geometry>-->
+<!--    </collision>-->
   </link>
   <joint name="camera_ee_side" type="fixed">
@@ -259,10 +355,10 @@
       </material>
     </visual>
-    <collision>
-      <origin xyz="-8.71485e-06 -0.115251 0.0109" rpy="-3.14159 4.996e-15 -5.80744e-23" />
-      <geometry>
-        <mesh filename="file://$(find rover_description)/banksia_arm/meshes/leftfinger.stl" />
-      </geometry>
-    </collision>
+<!--    <collision>-->
+<!--      <origin xyz="-8.71485e-06 -0.115251 0.0109" rpy="-3.14159 4.996e-15 -5.80744e-23" />-->
+<!--      <geometry>-->
+<!--        <mesh filename="file://$(find rover_description)/banksia_arm/meshes/leftfinger.stl" />-->
+<!--      </geometry>-->
+<!--    </collision>-->
   </link>
   <link name="actuator">
@@ -281,10 +377,10 @@
       </material>
     </visual>
-    <collision>
-      <origin xyz="-1.38778e-17 0 -0.058" rpy="3.11287e-20 2.12505e-23 1.99292e-27" />
-      <geometry>
-        <mesh filename="file://$(find rover_description)/banksia_arm/meshes/actuator.stl" />
-      </geometry>
-    </collision>
+<!--    <collision>-->
+<!--      <origin xyz="-1.38778e-17 0 -0.058" rpy="3.11287e-20 2.12505e-23 1.99292e-27" />-->
+<!--      <geometry>-->
+<!--        <mesh filename="file://$(find rover_description)/banksia_arm/meshes/actuator.stl" />-->
+<!--      </geometry>-->
+<!--    </collision>-->
   </link>
   <joint name="actuator_head" type="prismatic">
@@ -310,10 +406,10 @@
       </material>
     </visual>
-    <collision>
-      <origin xyz="2.77556e-17 0 -1.11022e-16" rpy="1.5708 -2.87448e-18 1.5822e-23" />
-      <geometry>
-        <mesh filename="file://$(find rover_description)/banksia_arm/meshes/arm_end_finger.stl" />
-      </geometry>
-    </collision>
+<!--    <collision>-->
+<!--      <origin xyz="2.77556e-17 0 -1.11022e-16" rpy="1.5708 -2.87448e-18 1.5822e-23" />-->
+<!--      <geometry>-->
+<!--        <mesh filename="file://$(find rover_description)/banksia_arm/meshes/arm_end_finger.stl" />-->
+<!--      </geometry>-->
+<!--    </collision>-->
   </link>
   <joint name="camera_ee_finger" type="fixed">
@@ -346,10 +442,10 @@
       </material>
     </visual>
-    <collision>
-      <origin xyz="1.11022e-16 0 0" rpy="1.5708 -2.5589e-20 3.89707e-23" />
-      <geometry>
-        <mesh filename="file://$(find rover_description)/banksia_arm/meshes/arm_end_top.stl" />
-      </geometry>
-    </collision>
+<!--    <collision>-->
+<!--      <origin xyz="1.11022e-16 0 0" rpy="1.5708 -2.5589e-20 3.89707e-23" />-->
+<!--      <geometry>-->
+<!--        <mesh filename="file://$(find rover_description)/banksia_arm/meshes/arm_end_top.stl" />-->
+<!--      </geometry>-->
+<!--    </collision>-->
   </link>
   <joint name="camera_ee_top" type="fixed">
@@ -375,10 +471,10 @@
       </material>
     </visual>
-    <collision>
-      <origin xyz="0 0 0" rpy="1.5708 -1.12386e-23 -2.15772e-29" />
-      <geometry>
-        <mesh filename="file://$(find rover_description)/banksia_arm/meshes/arm_end_periscope.stl" />
-      </geometry>
-    </collision>
+<!--    <collision>-->
+<!--      <origin xyz="0 0 0" rpy="1.5708 -1.12386e-23 -2.15772e-29" />-->
+<!--      <geometry>-->
+<!--        <mesh filename="file://$(find rover_description)/banksia_arm/meshes/arm_end_periscope.stl" />-->
+<!--      </geometry>-->
+<!--    </collision>-->
   </link>
   <joint name="camera_ee_periscope" type="fixed">
@@ -440,10 +536,10 @@
       </material>
     </visual>
-    <collision>
-      <origin xyz="2.77556e-17 0 -0.006" rpy="1.5708 1.5708 0" />
-      <geometry>
-        <mesh filename="file://$(find rover_description)/banksia_arm/meshes/l2prime.stl" />
-      </geometry>
-    </collision>
+<!--    <collision>-->
+<!--      <origin xyz="2.77556e-17 0 -0.006" rpy="1.5708 1.5708 0" />-->
+<!--      <geometry>-->
+<!--        <mesh filename="file://$(find rover_description)/banksia_arm/meshes/l2prime.stl" />-->
+<!--      </geometry>-->
+<!--    </collision>-->
   </link>
   <link name="l1prime">
@@ -464,7 +560,7 @@
     <collision>
       <origin xyz="-0.0797283 0.0603606 1.05415e-16" rpy="1.5708 1.5708 0" />
-      <geometry>
-        <mesh filename="file://$(find rover_description)/banksia_arm/meshes/l1prime.stl" />
-      </geometry>
+<!--      <geometry>-->
+<!--        <mesh filename="file://$(find rover_description)/banksia_arm/meshes/l1prime.stl" />-->
+<!--      </geometry>-->
     </collision>
   </link>
@@ -486,7 +582,7 @@
     <collision>
       <origin xyz="-0.0797283 0.560361 2.48639e-16" rpy="1.5708 1.5708 0" />
-      <geometry>
-        <mesh filename="file://$(find rover_description)/banksia_arm/meshes/l2cam.stl" />
-      </geometry>
+<!--      <geometry>-->
+<!--        <mesh filename="file://$(find rover_description)/banksia_arm/meshes/l2cam.stl" />-->
+<!--      </geometry>-->
     </collision>
   </link>

Commit message: feat: remove unused collisions in arm urdf

File: src/ros/rover/rover_description/banksia_arm/urdf/arm.urdf.xacro (robot description, xacro)
@@ -25,10 +25,4 @@
       </material>
     </visual>
-<!--    <collision>-->
-<!--      <origin xyz="-0.0671788 0.129712 -0.183721" rpy="-1.88173e-16 -1.99729e-09 -1.5708" />-->
-<!--      <geometry>-->
-<!--        <mesh filename="file://$(find rover_description)/banksia_arm/meshes/armmount.stl" />-->
-<!--      </geometry>-->
-<!--    </collision>-->
     <collision>
       <origin xyz="0 0 -0.085" rpy="0 0 0" />
@@ -53,10 +47,4 @@
       </material>
     </visual>
-    <collision>
-      <origin xyz="-9.93063e-18 0 5.55112e-17" rpy="3.14159 -0 -7.70285e-39" />
-<!--      <geometry>-->
-<!--        <mesh filename="file://$(find rover_description)/banksia_arm/meshes/gearbox.stl" />-->
-<!--      </geometry>-->
-    </collision>
   </link>
   <link name="linkagedrive">
@@ -75,10 +63,4 @@
       </material>
     </visual>
-<!--    <collision>-->
-<!--      <origin xyz="-1.58901e-15 -1.36391e-16 -5.55112e-17" rpy="6.68673e-23 -1.0222e-22 2.39693e-07" />-->
-<!--      <geometry>-->
-<!--        <mesh filename="file://$(find rover_description)/banksia_arm/meshes/linkagedrive.stl" />-->
-<!--      </geometry>-->
-<!--    </collision>-->
     <collision>
       <origin xyz="0 0 0.065" rpy="0 0 0" />
@@ -109,10 +91,4 @@
       </material>
     </visual>
-<!--    <collision>-->
-<!--      <origin xyz="3.1979e-15 -6.85563e-15 0.0239" rpy="1.5708 1.5708 0" />-->
-<!--      <geometry>-->
-<!--        <mesh filename="file://$(find rover_description)/banksia_arm/meshes/l1.stl" />-->
-<!--      </geometry>-->
-<!--    </collision>-->
     <collision>
       <origin xyz="0 -0.255 0.024" rpy="0 0 0" />
@@ -137,10 +113,4 @@
       </material>
     </visual>
-<!--    <collision>-->
-<!--      <origin xyz="0.398641 0.301803 6.48063e-16" rpy="2.49358 1.5708 0" />-->
-<!--      <geometry>-->
-<!--        <mesh filename="file://$(find rover_description)/banksia_arm/meshes/l2.stl" />-->
-<!--      </geometry>-->
-<!--    </collision>-->
     <collision>
       <origin xyz="0 0.11 0" rpy="0 0 0" />
@@ -201,10 +171,4 @@
       </material>
     </visual>
-<!--    <collision>-->
-<!--      <origin xyz="1.94289e-15 0.05075 -0.0795" rpy="1.5708 1.5708 0" />-->
-<!--      <geometry>-->
-<!--        <mesh filename="file://$(find rover_description)/banksia_arm/meshes/j5.stl" />-->
-<!--      </geometry>-->
-<!--    </collision>-->
   </link>
   <link name="j6">
@@ -223,10 +187,4 @@
       </material>
     </visual>
-<!--    <collision>-->
-<!--      <origin xyz="5.80265e-16 -0.1945 0.05075" rpy="-1.5708 -1.48145e-14 -7.47144e-23" />-->
-<!--      <geometry>-->
-<!--        <mesh filename="file://$(find rover_description)/banksia_arm/meshes/j6.stl" />-->
-<!--      </geometry>-->
-<!--    </collision>-->
     <collision>
       <origin xyz="0 -0.09 0.1" rpy="0 0 0" />
@@ -269,10 +227,4 @@
       </material>
     </visual>
-<!--    <collision>-->
-<!--      <origin xyz="0.00775 0.013 0.0215" rpy="-6.15694e-07 4.61983e-15 3.14159" />-->
-<!--      <geometry>-->
-<!--        <mesh filename="file://$(find rover_description)/banksia_arm/meshes/eebase.stl" />-->
-<!--      </geometry>-->
-<!--    </collision>-->
     <collision>
       <origin xyz="0 0.02 0.0675" rpy="0 0 0" />
@@ -297,10 +249,4 @@
       </material>
     </visual>
-<!--    <collision>-->
-<!--      <origin xyz="-3.64856e-05 0.115305 0.0109" rpy="-3.14159 -6.60532e-30 2.57948e-23" />-->
-<!--      <geometry>-->
-<!--        <mesh filename="file://$(find rover_description)/banksia_arm/meshes/rightfinger.stl" />-->
-<!--      </geometry>-->
-<!--    </collision>-->
   </link>
   <link name="arm_end_side_optical">
@@ -319,10 +265,4 @@
       </material>
     </visual>
-<!--    <collision>-->
-<!--      <origin xyz="0 0 0" rpy="1.5708 1.86776e-19 -2.0576e-24" />-->
-<!--      <geometry>-->
-<!--        <mesh filename="file://$(find rover_description)/banksia_arm/meshes/arm_end_side.stl" />-->
-<!--      </geometry>-->
-<!--    </collision>-->
   </link>
   <joint name="camera_ee_side" type="fixed">
@@ -355,10 +295,4 @@
       </material>
     </visual>
-<!--    <collision>-->
-<!--      <origin xyz="-8.71485e-06 -0.115251 0.0109" rpy="-3.14159 4.996e-15 -5.80744e-23" />-->
-<!--      <geometry>-->
-<!--        <mesh filename="file://$(find rover_description)/banksia_arm/meshes/leftfinger.stl" />-->
-<!--      </geometry>-->
-<!--    </collision>-->
   </link>
   <link name="actuator">
@@ -377,10 +311,4 @@
       </material>
     </visual>
-<!--    <collision>-->
-<!--      <origin xyz="-1.38778e-17 0 -0.058" rpy="3.11287e-20 2.12505e-23 1.99292e-27" />-->
-<!--      <geometry>-->
-<!--        <mesh filename="file://$(find rover_description)/banksia_arm/meshes/actuator.stl" />-->
-<!--      </geometry>-->
-<!--    </collision>-->
   </link>
   <joint name="actuator_head" type="prismatic">
@@ -406,10 +334,4 @@
       </material>
     </visual>
-<!--    <collision>-->
-<!--      <origin xyz="2.77556e-17 0 -1.11022e-16" rpy="1.5708 -2.87448e-18 1.5822e-23" />-->
-<!--      <geometry>-->
-<!--        <mesh filename="file://$(find rover_description)/banksia_arm/meshes/arm_end_finger.stl" />-->
-<!--      </geometry>-->
-<!--    </collision>-->
   </link>
   <joint name="camera_ee_finger" type="fixed">
@@ -442,10 +364,4 @@
       </material>
     </visual>
-<!--    <collision>-->
-<!--      <origin xyz="1.11022e-16 0 0" rpy="1.5708 -2.5589e-20 3.89707e-23" />-->
-<!--      <geometry>-->
-<!--        <mesh filename="file://$(find rover_description)/banksia_arm/meshes/arm_end_top.stl" />-->
-<!--      </geometry>-->
-<!--    </collision>-->
   </link>
   <joint name="camera_ee_top" type="fixed">
@@ -471,10 +387,4 @@
       </material>
     </visual>
-<!--    <collision>-->
-<!--      <origin xyz="0 0 0" rpy="1.5708 -1.12386e-23 -2.15772e-29" />-->
-<!--      <geometry>-->
-<!--        <mesh filename="file://$(find rover_description)/banksia_arm/meshes/arm_end_periscope.stl" />-->
-<!--      </geometry>-->
-<!--    </collision>-->
   </link>
   <joint name="camera_ee_periscope" type="fixed">
@@ -536,10 +446,4 @@
       </material>
     </visual>
-<!--    <collision>-->
-<!--      <origin xyz="2.77556e-17 0 -0.006" rpy="1.5708 1.5708 0" />-->
-<!--      <geometry>-->
-<!--        <mesh filename="file://$(find rover_description)/banksia_arm/meshes/l2prime.stl" />-->
-<!--      </geometry>-->
-<!--    </collision>-->
   </link>
   <link name="l1prime">
@@ -558,10 +462,4 @@
       </material>
     </visual>
-    <collision>
-      <origin xyz="-0.0797283 0.0603606 1.05415e-16" rpy="1.5708 1.5708 0" />
-<!--      <geometry>-->
-<!--        <mesh filename="file://$(find rover_description)/banksia_arm/meshes/l1prime.stl" />-->
-<!--      </geometry>-->
-    </collision>
   </link>
   <link name="l2cam">
@@ -580,10 +478,4 @@
       </material>
     </visual>
-    <collision>
-      <origin xyz="-0.0797283 0.560361 2.48639e-16" rpy="1.5708 1.5708 0" />
-<!--      <geometry>-->
-<!--        <mesh filename="file://$(find rover_description)/banksia_arm/meshes/l2cam.stl" />-->
-<!--      </geometry>-->
-    </collision>
   </link>
   <joint name="l1b_tp" type="revolute">

Commit message: feat: added l1a_tp_j2_mimic_joint to mimic J2 movement in the elbow

File: src/ros/rover/rover_description/banksia_arm/urdf/arm.urdf.xacro (robot description, xacro)
@@ -416,8 +416,17 @@
     <limit effort="10" velocity="10" lower="0" upper="0" />
   </joint>
+  <!-- Enables proper 4 bar linkage kinematics -->
+  <link name="l1a_tp_j2_mimic"/>
+  <joint name="l1a_tp_j2_mimic_joint" type="revolute">
+    <!-- before rotating to match IK function expected 0: 1.5707963 0.0 1.5707963 -->
+    <origin xyz="0 0 0" rpy="0.0 0.0 0.0" />
+    <parent link="l1a_tp_j2_mimic" />
+    <child link="l2" />
+    <mimic joint="J2" multiplier="1" offset="0"/>
+  </joint>
   <joint name="l1a_tp" type="revolute">
     <origin xyz="7.73032e-10 -0.5 0.0239" rpy="5.57224e-15 1.15529e-15 1.5708" />
     <parent link="l1" />
-    <child link="l2" />
+    <child link="l1a_tp_j2_mimic" />
     <axis xyz="0 0 1" />
     <limit effort="10" velocity="10" lower="0" upper="0"/>

Commit message: feat: add limit tag to l1a_tp_j2_mimic_joint

File: src/ros/rover/rover_description/banksia_arm/urdf/arm.urdf.xacro (robot description, xacro)
@@ -423,4 +423,5 @@
     <parent link="l1a_tp_j2_mimic" />
     <child link="l2" />
+    <limit effort="10" velocity="10" lower="-3.14" upper="3.14"/>
     <mimic joint="J2" multiplier="1" offset="0"/>
   </joint>
