Commit message: Revert "feat: remove unused collisions in arm urdf"
This reverts commit 4bd8c5678d7b596f211c26c566a8410883bf7bbb.

File: src/ros/rover/rover_description/banksia_arm/urdf/arm.urdf.xacro (robot description, xacro)
@@ -25,4 +25,10 @@
       </material>
     </visual>
+<!--    <collision>-->
+<!--      <origin xyz="-0.0671788 0.129712 -0.183721" rpy="-1.88173e-16 -1.99729e-09 -1.5708" />-->
+<!--      <geometry>-->
+<!--        <mesh filename="file://$(find rover_description)/banksia_arm/meshes/armmount.stl" />-->
+<!--      </geometry>-->
+<!--    </collision>-->
     <collision>
       <origin xyz="0 0 -0.085" rpy="0 0 0" />
@@ -47,4 +53,10 @@
       </material>
     </visual>
+    <collision>
+      <origin xyz="-9.93063e-18 0 5.55112e-17" rpy="3.14159 -0 -7.70285e-39" />
+<!--      <geometry>-->
+<!--        <mesh filename="file://$(find rover_description)/banksia_arm/meshes/gearbox.stl" />-->
+<!--      </geometry>-->
+    </collision>
   </link>
   <link name="linkagedrive">
@@ -63,4 +75,10 @@
       </material>
     </visual>
+<!--    <collision>-->
+<!--      <origin xyz="-1.58901e-15 -1.36391e-16 -5.55112e-17" rpy="6.68673e-23 -1.0222e-22 2.39693e-07" />-->
+<!--      <geometry>-->
+<!--        <mesh filename="file://$(find rover_description)/banksia_arm/meshes/linkagedrive.stl" />-->
+<!--      </geometry>-->
+<!--    </collision>-->
     <collision>
       <origin xyz="0 0 0.065" rpy="0 0 0" />
@@ -91,4 +109,10 @@
       </material>
     </visual>
+<!--    <collision>-->
+<!--      <origin xyz="3.1979e-15 -6.85563e-15 0.0239" rpy="1.5708 1.5708 0" />-->
+<!--      <geometry>-->
+<!--        <mesh filename="file://$(find rover_description)/banksia_arm/meshes/l1.stl" />-->
+<!--      </geometry>-->
+<!--    </collision>-->
     <collision>
       <origin xyz="0 -0.255 0.024" rpy="0 0 0" />
@@ -113,4 +137,10 @@
       </material>
     </visual>
+<!--    <collision>-->
+<!--      <origin xyz="0.398641 0.301803 6.48063e-16" rpy="2.49358 1.5708 0" />-->
+<!--      <geometry>-->
+<!--        <mesh filename="file://$(find rover_description)/banksia_arm/meshes/l2.stl" />-->
+<!--      </geometry>-->
+<!--    </collision>-->
     <collision>
       <origin xyz="0 0.11 0" rpy="0 0 0" />
@@ -171,4 +201,10 @@
       </material>
     </visual>
+<!--    <collision>-->
+<!--      <origin xyz="1.94289e-15 0.05075 -0.0795" rpy="1.5708 1.5708 0" />-->
+<!--      <geometry>-->
+<!--        <mesh filename="file://$(find rover_description)/banksia_arm/meshes/j5.stl" />-->
+<!--      </geometry>-->
+<!--    </collision>-->
   </link>
   <link name="j6">
@@ -187,4 +223,10 @@
       </material>
     </visual>
+<!--    <collision>-->
+<!--      <origin xyz="5.80265e-16 -0.1945 0.05075" rpy="-1.5708 -1.48145e-14 -7.47144e-23" />-->
+<!--      <geometry>-->
+<!--        <mesh filename="file://$(find rover_description)/banksia_arm/meshes/j6.stl" />-->
+<!--      </geometry>-->
+<!--    </collision>-->
     <collision>
       <origin xyz="0 -0.09 0.1" rpy="0 0 0" />
@@ -227,4 +269,10 @@
       </material>
     </visual>
+<!--    <collision>-->
+<!--      <origin xyz="0.00775 0.013 0.0215" rpy="-6.15694e-07 4.61983e-15 3.14159" />-->
+<!--      <geometry>-->
+<!--        <mesh filename="file://$(find rover_description)/banksia_arm/meshes/eebase.stl" />-->
+<!--      </geometry>-->
+<!--    </collision>-->
     <collision>
       <origin xyz="0 0.02 0.0675" rpy="0 0 0" />
@@ -249,4 +297,10 @@
       </material>
     </visual>
+<!--    <collision>-->
+<!--      <origin xyz="-3.64856e-05 0.115305 0.0109" rpy="-3.14159 -6.60532e-30 2.57948e-23" />-->
+<!--      <geometry>-->
+<!--        <mesh filename="file://$(find rover_description)/banksia_arm/meshes/rightfinger.stl" />-->
+<!--      </geometry>-->
+<!--    </collision>-->
   </link>
   <link name="arm_end_side_optical">
@@ -265,4 +319,10 @@
       </material>
     </visual>
+<!--    <collision>-->
+<!--      <origin xyz="0 0 0" rpy="1.5708 1.86776e-19 -2.0576e-24" />-->
+<!--      <geometry>-->
+<!--        <mesh filename="file://$(find rover_description)/banksia_arm/meshes/arm_end_side.stl" />-->
+<!--      </geometry>-->
+<!--    </collision>-->
   </link>
   <joint name="camera_ee_side" type="fixed">
@@ -295,4 +355,10 @@
       </material>
     </visual>
+<!--    <collision>-->
+<!--      <origin xyz="-8.71485e-06 -0.115251 0.0109" rpy="-3.14159 4.996e-15 -5.80744e-23" />-->
+<!--      <geometry>-->
+<!--        <mesh filename="file://$(find rover_description)/banksia_arm/meshes/leftfinger.stl" />-->
+<!--      </geometry>-->
+<!--    </collision>-->
   </link>
   <link name="actuator">
@@ -311,4 +377,10 @@
       </material>
     </visual>
+<!--    <collision>-->
+<!--      <origin xyz="-1.38778e-17 0 -0.058" rpy="3.11287e-20 2.12505e-23 1.99292e-27" />-->
+<!--      <geometry>-->
+<!--        <mesh filename="file://$(find rover_description)/banksia_arm/meshes/actuator.stl" />-->
+<!--      </geometry>-->
+<!--    </collision>-->
   </link>
   <joint name="actuator_head" type="prismatic">
@@ -334,4 +406,10 @@
       </material>
     </visual>
+<!--    <collision>-->
+<!--      <origin xyz="2.77556e-17 0 -1.11022e-16" rpy="1.5708 -2.87448e-18 1.5822e-23" />-->
+<!--      <geometry>-->
+<!--        <mesh filename="file://$(find rover_description)/banksia_arm/meshes/arm_end_finger.stl" />-->
+<!--      </geometry>-->
+<!--    </collision>-->
   </link>
   <joint name="camera_ee_finger" type="fixed">
@@ -364,4 +442,10 @@
       </material>
     </visual>
+<!--    <collision>-->
+<!--      <origin xyz="1.11022e-16 0 0" rpy="1.5708 -2.5589e-20 3.89707e-23" />-->
+<!--      <geometry>-->
+<!--        <mesh filename="file://$(find rover_description)/banksia_arm/meshes/arm_end_top.stl" />-->
+<!--      </geometry>-->
+<!--    </collision>-->
   </link>
   <joint name="camera_ee_top" type="fixed">
@@ -387,4 +471,10 @@
       </material>
     </visual>
+<!--    <collision>-->
+<!--      <origin xyz="0 0 0" rpy="1.5708 -1.12386e-23 -2.15772e-29" />-->
+<!--      <geometry>-->
+<!--        <mesh filename="file://$(find rover_description)/banksia_arm/meshes/arm_end_periscope.stl" />-->
+<!--      </geometry>-->
+<!--    </collision>-->
   </link>
   <joint name="camera_ee_periscope" type="fixed">
@@ -456,4 +546,10 @@
       </material>
     </visual>
+<!--    <collision>-->
+<!--      <origin xyz="2.77556e-17 0 -0.006" rpy="1.5708 1.5708 0" />-->
+<!--      <geometry>-->
+<!--        <mesh filename="file://$(find rover_description)/banksia_arm/meshes/l2prime.stl" />-->
+<!--      </geometry>-->
+<!--    </collision>-->
   </link>
   <link name="l1prime">
@@ -472,4 +568,10 @@
       </material>
     </visual>
+    <collision>
+      <origin xyz="-0.0797283 0.0603606 1.05415e-16" rpy="1.5708 1.5708 0" />
+<!--      <geometry>-->
+<!--        <mesh filename="file://$(find rover_description)/banksia_arm/meshes/l1prime.stl" />-->
+<!--      </geometry>-->
+    </collision>
   </link>
   <link name="l2cam">
@@ -488,4 +590,10 @@
       </material>
     </visual>
+    <collision>
+      <origin xyz="-0.0797283 0.560361 2.48639e-16" rpy="1.5708 1.5708 0" />
+<!--      <geometry>-->
+<!--        <mesh filename="file://$(find rover_description)/banksia_arm/meshes/l2cam.stl" />-->
+<!--      </geometry>-->
+    </collision>
   </link>
   <joint name="l1b_tp" type="revolute">

Commit message: feat: fixed 4 bar linkage forward kinematics to match real arm with another mimic joint

File: src/ros/rover/rover_description/banksia_arm/urdf/arm.urdf.xacro (robot description, xacro)
@@ -509,10 +509,10 @@
   <link name="l1a_tp_j2_mimic"/>
   <joint name="l1a_tp_j2_mimic_joint" type="revolute">
-    <!-- before rotating to match IK function expected 0: 1.5707963 0.0 1.5707963 -->
     <origin xyz="0 0 0" rpy="0.0 0.0 0.0" />
     <parent link="l1a_tp_j2_mimic" />
     <child link="l2" />
+    <axis xyz="0 0 1" />
     <limit effort="10" velocity="10" lower="-3.14" upper="3.14"/>
-    <mimic joint="J2" multiplier="1" offset="0"/>
+    <mimic joint="J2" multiplier="-1" offset="0"/>
   </joint>
   <joint name="l1a_tp" type="revolute">

Commit message: feat: fixed 4 bar linkage inverse kinematics

File: src/ros/rover/rover_description/banksia_arm/urdf/arm.urdf.xacro (robot description, xacro)
@@ -25,10 +25,4 @@
       </material>
     </visual>
-<!--    <collision>-->
-<!--      <origin xyz="-0.0671788 0.129712 -0.183721" rpy="-1.88173e-16 -1.99729e-09 -1.5708" />-->
-<!--      <geometry>-->
-<!--        <mesh filename="file://$(find rover_description)/banksia_arm/meshes/armmount.stl" />-->
-<!--      </geometry>-->
-<!--    </collision>-->
     <collision>
       <origin xyz="0 0 -0.085" rpy="0 0 0" />
@@ -53,10 +47,4 @@
       </material>
     </visual>
-    <collision>
-      <origin xyz="-9.93063e-18 0 5.55112e-17" rpy="3.14159 -0 -7.70285e-39" />
-<!--      <geometry>-->
-<!--        <mesh filename="file://$(find rover_description)/banksia_arm/meshes/gearbox.stl" />-->
-<!--      </geometry>-->
-    </collision>
   </link>
   <link name="linkagedrive">
@@ -75,10 +63,4 @@
       </material>
     </visual>
-<!--    <collision>-->
-<!--      <origin xyz="-1.58901e-15 -1.36391e-16 -5.55112e-17" rpy="6.68673e-23 -1.0222e-22 2.39693e-07" />-->
-<!--      <geometry>-->
-<!--        <mesh filename="file://$(find rover_description)/banksia_arm/meshes/linkagedrive.stl" />-->
-<!--      </geometry>-->
-<!--    </collision>-->
     <collision>
       <origin xyz="0 0 0.065" rpy="0 0 0" />
@@ -109,10 +91,4 @@
       </material>
     </visual>
-<!--    <collision>-->
-<!--      <origin xyz="3.1979e-15 -6.85563e-15 0.0239" rpy="1.5708 1.5708 0" />-->
-<!--      <geometry>-->
-<!--        <mesh filename="file://$(find rover_description)/banksia_arm/meshes/l1.stl" />-->
-<!--      </geometry>-->
-<!--    </collision>-->
     <collision>
       <origin xyz="0 -0.255 0.024" rpy="0 0 0" />
@@ -137,10 +113,4 @@
       </material>
     </visual>
-<!--    <collision>-->
-<!--      <origin xyz="0.398641 0.301803 6.48063e-16" rpy="2.49358 1.5708 0" />-->
-<!--      <geometry>-->
-<!--        <mesh filename="file://$(find rover_description)/banksia_arm/meshes/l2.stl" />-->
-<!--      </geometry>-->
-<!--    </collision>-->
     <collision>
       <origin xyz="0 0.11 0" rpy="0 0 0" />
@@ -201,10 +171,4 @@
       </material>
     </visual>
-<!--    <collision>-->
-<!--      <origin xyz="1.94289e-15 0.05075 -0.0795" rpy="1.5708 1.5708 0" />-->
-<!--      <geometry>-->
-<!--        <mesh filename="file://$(find rover_description)/banksia_arm/meshes/j5.stl" />-->
-<!--      </geometry>-->
-<!--    </collision>-->
   </link>
   <link name="j6">
@@ -223,10 +187,4 @@
       </material>
     </visual>
-<!--    <collision>-->
-<!--      <origin xyz="5.80265e-16 -0.1945 0.05075" rpy="-1.5708 -1.48145e-14 -7.47144e-23" />-->
-<!--      <geometry>-->
-<!--        <mesh filename="file://$(find rover_description)/banksia_arm/meshes/j6.stl" />-->
-<!--      </geometry>-->
-<!--    </collision>-->
     <collision>
       <origin xyz="0 -0.09 0.1" rpy="0 0 0" />
@@ -269,10 +227,4 @@
       </material>
     </visual>
-<!--    <collision>-->
-<!--      <origin xyz="0.00775 0.013 0.0215" rpy="-6.15694e-07 4.61983e-15 3.14159" />-->
-<!--      <geometry>-->
-<!--        <mesh filename="file://$(find rover_description)/banksia_arm/meshes/eebase.stl" />-->
-<!--      </geometry>-->
-<!--    </collision>-->
     <collision>
       <origin xyz="0 0.02 0.0675" rpy="0 0 0" />
@@ -297,10 +249,4 @@
       </material>
     </visual>
-<!--    <collision>-->
-<!--      <origin xyz="-3.64856e-05 0.115305 0.0109" rpy="-3.14159 -6.60532e-30 2.57948e-23" />-->
-<!--      <geometry>-->
-<!--        <mesh filename="file://$(find rover_description)/banksia_arm/meshes/rightfinger.stl" />-->
-<!--      </geometry>-->
-<!--    </collision>-->
   </link>
   <link name="arm_end_side_optical">
@@ -319,10 +265,4 @@
       </material>
     </visual>
-<!--    <collision>-->
-<!--      <origin xyz="0 0 0" rpy="1.5708 1.86776e-19 -2.0576e-24" />-->
-<!--      <geometry>-->
-<!--        <mesh filename="file://$(find rover_description)/banksia_arm/meshes/arm_end_side.stl" />-->
-<!--      </geometry>-->
-<!--    </collision>-->
   </link>
   <joint name="camera_ee_side" type="fixed">
@@ -355,10 +295,4 @@
       </material>
     </visual>
-<!--    <collision>-->
-<!--      <origin xyz="-8.71485e-06 -0.115251 0.0109" rpy="-3.14159 4.996e-15 -5.80744e-23" />-->
-<!--      <geometry>-->
-<!--        <mesh filename="file://$(find rover_description)/banksia_arm/meshes/leftfinger.stl" />-->
-<!--      </geometry>-->
-<!--    </collision>-->
   </link>
   <link name="actuator">
@@ -377,10 +311,4 @@
       </material>
     </visual>
-<!--    <collision>-->
-<!--      <origin xyz="-1.38778e-17 0 -0.058" rpy="3.11287e-20 2.12505e-23 1.99292e-27" />-->
-<!--      <geometry>-->
-<!--        <mesh filename="file://$(find rover_description)/banksia_arm/meshes/actuator.stl" />-->
-<!--      </geometry>-->
-<!--    </collision>-->
   </link>
   <joint name="actuator_head" type="prismatic">
@@ -406,10 +334,4 @@
       </material>
     </visual>
-<!--    <collision>-->
-<!--      <origin xyz="2.77556e-17 0 -1.11022e-16" rpy="1.5708 -2.87448e-18 1.5822e-23" />-->
-<!--      <geometry>-->
-<!--        <mesh filename="file://$(find rover_description)/banksia_arm/meshes/arm_end_finger.stl" />-->
-<!--      </geometry>-->
-<!--    </collision>-->
   </link>
   <joint name="camera_ee_finger" type="fixed">
@@ -442,10 +364,4 @@
       </material>
     </visual>
-<!--    <collision>-->
-<!--      <origin xyz="1.11022e-16 0 0" rpy="1.5708 -2.5589e-20 3.89707e-23" />-->
-<!--      <geometry>-->
-<!--        <mesh filename="file://$(find rover_description)/banksia_arm/meshes/arm_end_top.stl" />-->
-<!--      </geometry>-->
-<!--    </collision>-->
   </link>
   <joint name="camera_ee_top" type="fixed">
@@ -471,10 +387,4 @@
       </material>
     </visual>
-<!--    <collision>-->
-<!--      <origin xyz="0 0 0" rpy="1.5708 -1.12386e-23 -2.15772e-29" />-->
-<!--      <geometry>-->
-<!--        <mesh filename="file://$(find rover_description)/banksia_arm/meshes/arm_end_periscope.stl" />-->
-<!--      </geometry>-->
-<!--    </collision>-->
   </link>
   <joint name="camera_ee_periscope" type="fixed">
@@ -546,10 +456,4 @@
       </material>
     </visual>
-<!--    <collision>-->
-<!--      <origin xyz="2.77556e-17 0 -0.006" rpy="1.5708 1.5708 0" />-->
-<!--      <geometry>-->
-<!--        <mesh filename="file://$(find rover_description)/banksia_arm/meshes/l2prime.stl" />-->
-<!--      </geometry>-->
-<!--    </collision>-->
   </link>
   <link name="l1prime">
@@ -568,10 +472,4 @@
       </material>
     </visual>
-    <collision>
-      <origin xyz="-0.0797283 0.0603606 1.05415e-16" rpy="1.5708 1.5708 0" />
-<!--      <geometry>-->
-<!--        <mesh filename="file://$(find rover_description)/banksia_arm/meshes/l1prime.stl" />-->
-<!--      </geometry>-->
-    </collision>
   </link>
   <link name="l2cam">
@@ -590,24 +488,38 @@
       </material>
     </visual>
-    <collision>
-      <origin xyz="-0.0797283 0.560361 2.48639e-16" rpy="1.5708 1.5708 0" />
-<!--      <geometry>-->
-<!--        <mesh filename="file://$(find rover_description)/banksia_arm/meshes/l2cam.stl" />-->
-<!--      </geometry>-->
-    </collision>
-  </link>
+  </link>
+  <link name="l2cam_mimic"/>
+  <joint name="l2cam_mimic_joint" type="revolute">
+    <origin xyz="0 0 0" rpy="0.0 0.0 0.0" />
+    <parent link="l2cam_mimic" />
+    <child link="l2cam" />
+    <axis xyz="0 0 1" />
+    <limit effort="10" velocity="10" lower="-3.14" upper="3.14"/>
+    <mimic joint="J3" multiplier="1" offset="0"/>
+  </joint>
   <joint name="l1b_tp" type="revolute">
     <origin xyz="3.05311e-16 -0.5 5.77479e-16" rpy="-1.0988e-15 4.62615e-16 0.648016" />
     <parent link="l1prime" />
-    <child link="l2cam" />
+    <child link="l2cam_mimic" />
     <axis xyz="0 0 1" />
     <limit effort="10" velocity="10" lower="0" upper="0"/>
+    <mimic joint="J2" multiplier="-1" offset="0"/>
+  </joint>
+  <link name="l1prime_mimic"/>
+  <joint name="l1prime_mimic_joint" type="revolute">
+    <origin xyz="0 0 0" rpy="0.0 0.0 0.0" />
+    <parent link="l1prime_mimic" />
+    <child link="l1prime" />
+    <axis xyz="0 0 1" />
+    <limit effort="10" velocity="10" lower="-3.14" upper="3.14"/>
+    <mimic joint="J3" multiplier="-1" offset="0"/>
   </joint>
   <joint name="l1b_bp" type="revolute">
     <origin xyz="0.0797283 -0.0603606 -0.006" rpy="-1.08371e-22 -4.6005e-22 -0.648016" />
     <parent link="l2prime" />
-    <child link="l1prime" />
+    <child link="l1prime_mimic" />
     <axis xyz="0 0 1" />
     <limit effort="10" velocity="10" lower="0" upper="0"/>
+    <mimic joint="J2" multiplier="1" offset="0"/>
   </joint>
   <joint name="J3" type="revolute">
