Commit message: simple attempt to populate all values for velocity control on the arm, PLEASE RUN AT A REALLY LOW SPEED FOR THE FIRST TIME

File: src/ros/rover/rover_description/banksia_arm/urdf/arm.ros2_control.xacro (robot description, xacro)
@@ -101,51 +101,57 @@
 					<param name="candevice">can1</param>
 					<param name="canid">3</param>
-					<param name="resolver_reduction">1.33333333333</param>
-					<param name="clock_rate">100000000</param>
-					<param name="revolution_pulses">8192</param>
-					<param name="min_interval">122</param>
-					<param name="gear_ratio">36.0</param>
-					<param name="mock">true</param>
-					<param name="reversed">true</param>
+					<param name="resolver_reduction">5.375</param>
+					<param name="clock_rate">100000000</param>
+					<param name="revolution_pulses">8192</param>
+					<param name="min_interval">1728</param>
+					<param name="gear_ratio">100.0</param>
+					<param name="mock">true</param>
+					<param name="reversed">false</param>
+					<param name="integrate_velocity">false</param>
+					<param name="max_position">12.5663706144 / 5.375</param>
+					<param name="position_offset">0.0</param>
+					<param name="max_velocity">292.444791136 / 100</param>
+				</hardware>
+			</xacro:unless>
+			<xacro:if value="${use_mock_hardware}">
+				<hardware>
+					<plugin>mock_components/GenericSystem</plugin>
+					<param name="calculate_dynamics">true</param>
+				</hardware>
+			</xacro:if>
+			<joint name="J3">
+				<command_interface name="velocity">
+					<param name="max">292.444791137</param>
+				</command_interface>
+				<command_interface name="position">
+					<param name="max">12.5663706144</param>
+				</command_interface>
+				<state_interface name="velocity">
+					<param name="max">292.444791137</param>
+					<param name="initial_value">0.0</param>
+				</state_interface>
+				<state_interface name="position">
+					<param name="max">12.5663706144</param>
+					<param name="initial_value">0.0</param>
+				</state_interface>
+			</joint>
+		</ros2_control>
+		<ros2_control name="arm_J4" type="system">
+			<xacro:unless value="${use_mock_hardware}">
+				<hardware>
+					<plugin>blcmd_hardware/BLCMDHardware</plugin>
+					<param name="candevice">can1</param>
+					<param name="canid">4</param>
+					<param name="resolver_reduction">15</param>
+					<param name="clock_rate">100000000</param>
+					<param name="revolution_pulses">8192</param>
+					<param name="min_interval">1728</param>
+					<param name="gear_ratio">15.0</param>
+					<param name="mock">true</param>
+					<param name="reversed">false</param>
 					<param name="integrate_velocity">true</param>
-				</hardware>
-			</xacro:unless>
-			<xacro:if value="${use_mock_hardware}">
-				<hardware>
-					<plugin>mock_components/GenericSystem</plugin>
-					<param name="calculate_dynamics">true</param>
-				</hardware>
-			</xacro:if>
-			<joint name="J3">
-				<command_interface name="velocity">
-					<param name="max">292.444791137</param>
-				</command_interface>
-				<command_interface name="position">
-					<param name="max">12.5663706144</param>
-				</command_interface>
-				<state_interface name="velocity">
-					<param name="max">292.444791137</param>
-					<param name="initial_value">0.0</param>
-				</state_interface>
-				<state_interface name="position">
-					<param name="max">12.5663706144</param>
-					<param name="initial_value">0.0</param>
-				</state_interface>
-			</joint>
-		</ros2_control>
-		<ros2_control name="arm_J4" type="system">
-			<xacro:unless value="${use_mock_hardware}">
-				<hardware>
-					<plugin>blcmd_hardware/BLCMDHardware</plugin>
-					<param name="candevice">can1</param>
-					<param name="canid">4</param>
-					<param name="resolver_reduction">1.33333333333</param>
-					<param name="clock_rate">100000000</param>
-					<param name="revolution_pulses">8192</param>
-					<param name="min_interval">122</param>
-					<param name="gear_ratio">36.0</param>
-					<param name="mock">true</param>
-					<param name="reversed">true</param>
-					<param name="integrate_velocity">true</param>
+					<param name="max_position">12.5663706144</param>
+					<param name="position_offset">0.0</param>
+					<param name="max_velocity">292.444791136 / 15</param>
 				</hardware>
 			</xacro:unless>
@@ -179,12 +185,15 @@
 					<param name="candevice">can1</param>
 					<param name="canid">5</param>
-					<param name="resolver_reduction">1.33333333333</param>
-					<param name="clock_rate">100000000</param>
-					<param name="revolution_pulses">8192</param>
-					<param name="min_interval">122</param>
-					<param name="gear_ratio">36.0</param>
-					<param name="mock">true</param>
-					<param name="reversed">true</param>
-					<param name="integrate_velocity">true</param>
+					<param name="resolver_reduction">1.0</param>
+					<param name="clock_rate">100000000</param>
+					<param name="revolution_pulses">8192</param>
+          			<param name="min_interval">1792</param>
+					<param name="gear_ratio">1.0</param>
+					<param name="mock">true</param>
+					<param name="reversed">false</param>
+					<param name="integrate_velocity">false</param>
+					<param name="max_position">12.5663706144</param>
+					<param name="position_offset">3.14159265359</param>
+					<param name="max_velocity">292.444791136</param>
 				</hardware>
 			</xacro:unless>

Commit message: wip: teleop joint space mode left stick control

File: src/ros/rover/rover_description/banksia_arm/urdf/arm.ros2_control.xacro (robot description, xacro)
@@ -299,4 +299,36 @@
       </joint>
     -->
+	 <ros2_control name="arm_actuator_head" type="system">
+		<xacro:unless value="${use_mock_hardware}">
+			<hardware>
+				<plugin>cmd_hardware/CMDHardware</plugin>
+				<param name="candevice">can1</param>
+				<param name="canid">5</param> <!-- TODO: Get CAN id, resolver id should be that *4 -->
+				<param name="resolver_id">20</param>
+				<param name="resolver_reduction">1.0</param>
+				<param name="reversed">false</param>
+				<param name="reverse_velocity">true</param>
+				<param name="max_velocity">0.365109712045</param>
+				<param name="max_effort">1</param>
+			</hardware>
+		</xacro:unless>
+		<xacro:if value="${use_mock_hardware}">
+			<hardware>
+				<plugin>mock_components/GenericSystem</plugin>
+				<param name="calculate_dynamics">true</param>
+			</hardware>
+		</xacro:if>
+		<joint name="actuator_head">
+			<command_interface name="velocity">
+			<param name="max">1</param>
+			</command_interface>
+			<state_interface name="velocity">
+			<param name="initial_value">0.0</param>
+			</state_interface>
+			<state_interface name="position">
+			<param name="initial_value">0.0</param>
+			</state_interface>
+		</joint>
+	</ros2_control>
 	</xacro:macro>
 </robot>

Commit message: fix: renamed joints to be consistent with preexisting urdf

File: src/ros/rover/rover_description/banksia_arm/urdf/arm.ros2_control.xacro (robot description, xacro)
@@ -264,39 +264,4 @@
 			</joint>
 		</ros2_control>
-		<!--
-    <joint name="rf_slide">
-		<command_interface name="velocity">
-		  <param name="max">1</param>
-		</command_interface>
-		<state_interface name="velocity">
-		  <param name="initial_value">0.0</param>
-		</state_interface>
-		<state_interface name="position">
-		  <param name="initial_value">0.0</param>
-		</state_interface>
-      </joint>
-	  <joint name="lf_slide">
-		<command_interface name="velocity">
-		  <param name="max">1</param>
-		</command_interface>
-		<state_interface name="velocity">
-		  <param name="initial_value">0.0</param>
-		</state_interface>
-		<state_interface name="position">
-		  <param name="initial_value">0.0</param>
-		</state_interface>
-      </joint>
-	  <joint name="actuator_head">
-		<command_interface name="velocity">
-		  <param name="max">1</param>
-		</command_interface>
-		<state_interface name="velocity">
-		  <param name="initial_value">0.0</param>
-		</state_interface>
-		<state_interface name="position">
-		  <param name="initial_value">0.0</param>
-		</state_interface>
-      </joint>
-    -->
 	 <ros2_control name="arm_actuator_head" type="system">
 		<xacro:unless value="${use_mock_hardware}">
@@ -331,4 +296,68 @@
 		</joint>
 	</ros2_control>
+  <ros2_control name="arm_right_slide" type="system">
+		<xacro:unless value="${use_mock_hardware}">
+			<hardware>
+				<plugin>cmd_hardware/CMDHardware</plugin>
+				<param name="candevice">can1</param>
+				<param name="canid">5</param> <!-- TODO: Get CAN id, resolver id should be that *4 -->
+				<param name="resolver_id">20</param>
+				<param name="resolver_reduction">1.0</param>
+				<param name="reversed">false</param>
+				<param name="reverse_velocity">true</param>
+				<param name="max_velocity">0.365109712045</param>
+				<param name="max_effort">1</param>
+			</hardware>
+		</xacro:unless>
+		<xacro:if value="${use_mock_hardware}">
+			<hardware>
+				<plugin>mock_components/GenericSystem</plugin>
+				<param name="calculate_dynamics">true</param>
+			</hardware>
+		</xacro:if>
+    <joint name="right_slide">
+      <command_interface name="velocity">
+        <param name="max">1</param>
+      </command_interface>
+      <state_interface name="velocity">
+        <param name="initial_value">0.0</param>
+      </state_interface>
+      <state_interface name="position">
+        <param name="initial_value">0.0</param>
+      </state_interface>
+    </joint>
+	</ros2_control>
+  <ros2_control name="arm_left_slide" type="system">
+		<xacro:unless value="${use_mock_hardware}">
+			<hardware>
+				<plugin>cmd_hardware/CMDHardware</plugin>
+				<param name="candevice">can1</param>
+				<param name="canid">5</param> <!-- TODO: Get CAN id, resolver id should be that *4 -->
+				<param name="resolver_id">20</param>
+				<param name="resolver_reduction">1.0</param>
+				<param name="reversed">false</param>
+				<param name="reverse_velocity">true</param>
+				<param name="max_velocity">0.365109712045</param>
+				<param name="max_effort">1</param>
+			</hardware>
+		</xacro:unless>
+		<xacro:if value="${use_mock_hardware}">
+			<hardware>
+				<plugin>mock_components/GenericSystem</plugin>
+				<param name="calculate_dynamics">true</param>
+			</hardware>
+		</xacro:if>
+	  <joint name="left_slide">
+      <command_interface name="velocity">
+        <param name="max">1</param>
+      </command_interface>
+      <state_interface name="velocity">
+        <param name="initial_value">0.0</param>
+      </state_interface>
+      <state_interface name="position">
+        <param name="initial_value">0.0</param>
+      </state_interface>
+    </joint>
+	</ros2_control>
 	</xacro:macro>
 </robot>
