Commit message: fixed sim gps

File: src/ros/rover/rover_description/banksia/urdf/gps.xacro (robot description, xacro)
@@ -8,5 +8,5 @@
     <parent link="base_link"/>
     <child link="gps"/>
-    <origin xyz="0.04 -0.26 0.614" rpy="0 0 0"/>
+    <origin xyz="0 0 0" rpy="0 0 0"/>
   </joint>
   <gazebo reference="gps">
