Commit message: feat: Added cameras to gazebo (unsure if correct positions or fov)

File: src/ros/rover/rover_description/banksia/urdf/gz_ros2_control.xacro (robot description, xacro)
@@ -228,18 +228,18 @@
       </state_interface>
     </joint>
-    <joint name="rf_slide">
-      <command_interface name="velocity">
-        <param name="max">1</param>
-      </command_interface>
-      <command_interface name="position">
-      </command_interface>
-      <state_interface name="velocity">
-        <param name="initial_value">0.0</param>
-      </state_interface>
-      <state_interface name="position">
-        <param name="initial_value">0.0</param>
-      </state_interface>
-    </joint>
-    <joint name="lf_slide">
+    <joint name="right_slide">
+      <command_interface name="velocity">
+        <param name="max">1</param>
+      </command_interface>
+      <command_interface name="position">
+      </command_interface>
+      <state_interface name="velocity">
+        <param name="initial_value">0.0</param>
+      </state_interface>
+      <state_interface name="position">
+        <param name="initial_value">0.0</param>
+      </state_interface>
+    </joint>
+    <joint name="left_slide">
       <command_interface name="velocity">
         <param name="max">1</param>

File: src/ros/rover/rover_description/banksia/urdf/rover.urdf.xacro (robot description, xacro)
@@ -704,5 +704,5 @@
         </joint> -->
         <!-- Banksia's arm -->
-        <xacro:include filename="$(find rover_description)/banksia_arm/urdf/arm.urdf.xacro" />
+        <xacro:include filename="/home/nova/nova/src/ros/rover/rover_description/banksia_arm/urdf/arm.urdf.xacro" />
         <joint name="chassis_to_arm_base" type="fixed">
             <origin xyz="0.234 -0.001 0.116750" rpy="0 0 1.5708"/>
@@ -725,4 +725,3 @@
     <xacro:include filename="$(find rover_description)/banksia/urdf/odom.xacro"/>
     <xacro:include filename="$(find rover_description)/banksia/urdf/gps.xacro"/>
-    <xacro:include filename="$(find rover_description)/banksia/urdf/joint_states.xacro"/>
 </robot>

File: src/ros/rover/rover_description/banksia_arm/urdf/arm.urdf.xacro (robot description, xacro)
@@ -383,5 +383,5 @@
   </link>
   <joint name="camera_ee_periscope" type="fixed">
-    <origin xyz="-0.00015 -0.0378336 0.0594947" rpy="-3.14159 6.15694e-07 -1.5708" />
+    <origin xyz="-0.00015 -0.0378336 0.0594947" rpy="-3.14159 -1.5708 1.5708" />
     <parent link="eebase" />
     <child link="arm_end_periscope" />
@@ -555,4 +555,5 @@
   <xacro:if value="$(arg gazebo)">
     <xacro:include filename="$(find rover_description)/banksia_arm/urdf/arm.gz_ros2_control.xacro" />
+    <xacro:include filename="/home/nova/nova/src/ros/rover/rover_description/banksia_arm/urdf/arm_sensors.xacro"/>
   </xacro:if>
   <xacro:unless value="$(arg gazebo)">
