Commit message: [WIP] Merge `arm-master` (#425)
Signed-off-by: Bailey Chessum <bailey.chessum1@gmail.com>
Co-authored-by: RohitPilakkat <rohit.pilakkat@gmail.com>
Co-authored-by: arbabf <arbab.fahm@gmail.com>
Co-authored-by: Orlando Chamberlain <ocha0025@student.monash.edu>
Co-authored-by: Felicity Matthews <felicitymatthews30@gmail.com>
Co-authored-by: Monash Nova Rover <novaroverteam@monash.edu>
Co-authored-by: Anthony Lew <anthony@v01dbreaker.cc>
Co-authored-by: Victor Bartlinski <vicbart08@gmail.com>
Co-authored-by: Orlando Chamberlain <orlandoch.dev@gmail.com>
Co-authored-by: hacker1024 <jlei0014@student.monash.edu>
Co-authored-by: arbabf <34561149+arbabf@users.noreply.github.com>
Co-authored-by: Anthony Lew <ant87518@gmail.com>

File: src/ros/rover/rover_description/banksia/urdf/gz_ros2_control.xacro (robot description, xacro)
@@ -117,4 +117,154 @@
       </state_interface>
     </joint>
+    <joint name="J1">
+      <command_interface name="velocity">
+        <param name="max">1</param>
+      </command_interface>
+      <command_interface name="position">
+      </command_interface>
+      <state_interface name="velocity">
+        <param name="initial_value">0.0</param>
+      </state_interface>
+      <state_interface name="position">
+        <param name="initial_value">0.0</param>
+      </state_interface>
+    </joint>
+    <joint name="J2">
+      <command_interface name="velocity">
+        <param name="max">1</param>
+      </command_interface>
+      <command_interface name="position">
+      </command_interface>
+      <state_interface name="velocity">
+        <param name="initial_value">0.0</param>
+      </state_interface>
+      <state_interface name="position">
+        <param name="initial_value">0.0</param>
+      </state_interface>
+    </joint>
+    <joint name="J3">
+      <command_interface name="velocity">
+        <param name="max">1</param>
+      </command_interface>
+      <command_interface name="position">
+      </command_interface>
+      <state_interface name="velocity">
+        <param name="initial_value">0.0</param>
+      </state_interface>
+      <state_interface name="position">
+        <param name="initial_value">0.0</param>
+      </state_interface>
+    </joint>
+    <!-- <joint name="l1b_bp">
+		<command_interface name="velocity">
+		  <param name="max">1</param>
+		</command_interface>
+		<state_interface name="velocity">
+		  <param name="initial_value">0.0</param>
+		</state_interface>
+		<state_interface name="position">
+		  <param name="initial_value">0.0</param>
+		</state_interface>
+      </joint>
+	  <joint name="l1b_tp">
+		<command_interface name="velocity">
+		  <param name="max">1</param>
+		</command_interface>
+		<state_interface name="velocity">
+		  <param name="initial_value">0.0</param>
+		</state_interface>
+		<state_interface name="position">
+		  <param name="initial_value">0.0</param>
+		</state_interface>
+      </joint>
+	  <joint name="l1a_tp">
+		<command_interface name="velocity">
+		  <param name="max">1</param>
+		</command_interface>
+		<state_interface name="velocity">
+		  <param name="initial_value">0.0</param>
+		</state_interface>
+		<state_interface name="position">
+		  <param name="initial_value">0.0</param>
+		</state_interface>
+      </joint> -->
+    <joint name="J4">
+      <command_interface name="velocity">
+        <param name="max">1</param>
+      </command_interface>
+      <command_interface name="position">
+      </command_interface>
+      <state_interface name="velocity">
+        <param name="initial_value">0.0</param>
+      </state_interface>
+      <state_interface name="position">
+        <param name="initial_value">0.0</param>
+      </state_interface>
+    </joint>
+    <joint name="J5">
+      <command_interface name="velocity">
+        <param name="max">1</param>
+      </command_interface>
+      <command_interface name="position">
+      </command_interface>
+      <state_interface name="velocity">
+        <param name="initial_value">0.0</param>
+      </state_interface>
+      <state_interface name="position">
+        <param name="initial_value">0.0</param>
+      </state_interface>
+    </joint>
+    <joint name="J6">
+      <command_interface name="velocity">
+        <param name="max">1</param>
+      </command_interface>
+      <command_interface name="position">
+      </command_interface>
+      <state_interface name="velocity">
+        <param name="initial_value">0.0</param>
+      </state_interface>
+      <state_interface name="position">
+        <param name="initial_value">0.0</param>
+      </state_interface>
+    </joint>
+    <joint name="right_slide">
+      <command_interface name="velocity">
+        <param name="max">1</param>
+      </command_interface>
+      <command_interface name="position">
+      </command_interface>
+      <state_interface name="velocity">
+        <param name="initial_value">0.0</param>
+      </state_interface>
+      <state_interface name="position">
+        <param name="initial_value">0.0</param>
+      </state_interface>
+    </joint>
+    <joint name="left_slide">
+      <command_interface name="velocity">
+        <param name="max">1</param>
+      </command_interface>
+      <command_interface name="position">
+      </command_interface>
+      <state_interface name="velocity">
+        <param name="initial_value">0.0</param>
+      </state_interface>
+      <state_interface name="position">
+        <param name="initial_value">0.0</param>
+      </state_interface>
+    </joint>
+    <joint name="actuator_head">
+      <command_interface name="velocity">
+        <param name="max">1</param>
+      </command_interface>
+      <command_interface name="position">
+      </command_interface>
+      <state_interface name="velocity">
+        <param name="initial_value">0.0</param>
+      </state_interface>
+      <state_interface name="position">
+        <param name="initial_value">0.0</param>
+      </state_interface>
+    </joint>
   </ros2_control>
   <gazebo>

File: src/ros/rover/rover_description/banksia/urdf/ros2_control.xacro (robot description, xacro)
@@ -155,5 +155,5 @@
                     <plugin>blcmd_hardware/BLCMDHardware</plugin>
                     <param name="candevice">can0</param>
-                    <param name="canid">5</param>
+                    <param name="canid">3F1</param>
 		            <param name="resolver_reduction">1.33333333333</param>
                     <param name="clock_rate">100000000</param>

File: src/ros/rover/rover_description/banksia/urdf/rover.urdf.xacro (robot description, xacro)
@@ -10,4 +10,5 @@
     <xacro:arg name="use_mock_hardware" default="false"/>
     <xacro:arg name="arm" default="false"/>
+    <xacro:arg name="old_arm" default="false"/>
     <xacro:arg name="auto_camera" default="true"/>
     <xacro:arg name="robot_name" default="Banksia"/>
@@ -715,4 +716,12 @@
         <xacro:include filename="$(find rover_description)/banksia/urdf/joint_states.xacro"/>
     </xacro:unless>
+    <xacro:if value="$(arg old_arm)">
+        <xacro:include filename="$(find rover_description)/waratah_arm/urdf/arm.urdf.xacro" />
+        <joint name="chassis_to_arm_base" type="fixed">
+            <origin xyz="0.2 0 -0.06" rpy="0 0 0"/>
+            <parent link="chassis" />
+            <child link="arm_link" />
+        </joint>
+    </xacro:if>
     <xacro:unless value="$(arg gazebo)">
         <xacro:include filename="$(find rover_description)/banksia/urdf/ros2_control.xacro" />
@@ -725,4 +734,3 @@
     <xacro:include filename="$(find rover_description)/banksia/urdf/odom.xacro"/>
     <xacro:include filename="$(find rover_description)/banksia/urdf/gps.xacro"/>
-    <xacro:include filename="$(find rover_description)/banksia/urdf/joint_states.xacro"/>
 </robot>

File: src/ros/rover/rover_description/banksia_arm/urdf/arm.gz_ros2_control.xacro (robot description, xacro)
@@ -116,5 +116,5 @@
 		</state_interface>
       </joint>
-	  <joint name="rf_slide">
+	  <joint name="right_slide">
 		<command_interface name="velocity">
 		  <param name="max">1</param>
@@ -129,5 +129,5 @@
 		</state_interface>
       </joint>
-	  <joint name="lf_slide">
+	  <joint name="left_slide">
 		<command_interface name="velocity">
 		  <param name="max">1</param>

File: src/ros/rover/rover_description/banksia_arm/urdf/arm.ros2_control.xacro (robot description, xacro)
@@ -9,13 +9,16 @@
 					<plugin>blcmd_hardware/BLCMDHardware</plugin>
 					<param name="candevice">can1</param>
-					<param name="canid">4F1</param>
-					<param name="resolver_reduction">1.33333333333</param>
-					<param name="clock_rate">100000000</param>
-					<param name="revolution_pulses">8192</param>
-					<param name="min_interval">122</param>
-					<param name="gear_ratio">36.0</param>
-					<param name="mock">true</param>
-					<param name="reversed">true</param>
-					<param name="integrate_velocity">true</param>
+					<param name="canid">1</param>
+					<param name="resolver_reduction">4</param>
+					<param name="clock_rate">100000000</param>
+					<param name="revolution_pulses">8192</param>
+					<param name="min_interval">1728</param>
+					<param name="gear_ratio">100.0</param>
+					<param name="mock">true</param>
+					<param name="reversed">false</param>
+					<param name="integrate_velocity">false</param>
+					<param name="max_position">12.5663706144 / 4</param>
+					<param name="position_offset">0.0</param>
+					<param name="max_velocity">292.444791136 / 100</param>
 				</hardware>
 			</xacro:unless>
@@ -34,12 +37,16 @@
 			<joint name="J1">
 				<command_interface name="velocity">
-					<param name="max">1</param>
-				</command_interface>
-				<command_interface name="position">
-				</command_interface>
-				<state_interface name="velocity">
-					<param name="initial_value">0.0</param>
-				</state_interface>
-				<state_interface name="position">
+					<param name="max">292.444791137</param>
+					<param name="max">1.0</param>
+				</command_interface>
+				<command_interface name="position">
+					<param name="max">12.5663706144</param>
+				</command_interface>
+				<state_interface name="velocity">
+					<param name="max">292.444791137</param>
+					<param name="initial_value">0.0</param>
+				</state_interface>
+				<state_interface name="position">
+					<param name="max">12.5663706144</param>
 					<param name="initial_value">0.0</param>
 				</state_interface>
@@ -51,85 +58,100 @@
 					<plugin>blcmd_hardware/BLCMDHardware</plugin>
 					<param name="candevice">can1</param>
-					<param name="canid">4F2</param>
-					<param name="resolver_reduction">1.33333333333</param>
-					<param name="clock_rate">100000000</param>
-					<param name="revolution_pulses">8192</param>
-					<param name="min_interval">122</param>
-					<param name="gear_ratio">36.0</param>
+					<param name="canid">2</param>
+					<param name="resolver_reduction">5.375</param>
+					<param name="clock_rate">100000000</param>
+					<param name="revolution_pulses">8192</param>
+					<param name="min_interval">1728</param>
+					<param name="gear_ratio">100.0</param>
 					<param name="mock">true</param>
 					<param name="reversed">true</param>
+					<param name="integrate_velocity">false</param>
+					<param name="max_position">12.5663706144 / 5.375</param>
+					<param name="position_offset">0.0</param>
+					<param name="max_velocity">292.444791136 / 100</param>
+				</hardware>
+			</xacro:unless>
+			<xacro:if value="${use_mock_hardware}">
+				<hardware>
+					<plugin>mock_components/GenericSystem</plugin>
+					<param name="calculate_dynamics">true</param>
+				</hardware>
+			</xacro:if>
+			<joint name="J2">
+				<command_interface name="velocity">
+					<param name="max">292.444791137</param>
+				</command_interface>
+				<command_interface name="position">
+					<param name="max">12.5663706144</param>
+				</command_interface>
+				<state_interface name="velocity">
+					<param name="max">292.444791137</param>
+					<param name="initial_value">0.0</param>
+				</state_interface>
+				<state_interface name="position">
+					<param name="max">12.5663706144</param>
+					<param name="initial_value">0.0</param>
+				</state_interface>
+			</joint>
+		</ros2_control>
+		<ros2_control name="arm_J3" type="system">
+			<xacro:unless value="${use_mock_hardware}">
+				<hardware>
+					<plugin>blcmd_hardware/BLCMDHardware</plugin>
+					<param name="candevice">can1</param>
+					<param name="canid">3</param>
+					<param name="resolver_reduction">5.375</param>
+					<param name="clock_rate">100000000</param>
+					<param name="revolution_pulses">8192</param>
+					<param name="min_interval">1728</param>
+					<param name="gear_ratio">100.0</param>
+					<param name="mock">true</param>
+					<param name="reversed">false</param>
+					<param name="integrate_velocity">false</param>
+					<param name="max_position">12.5663706144 / 5.375</param>
+					<param name="position_offset">0.0</param>
+					<param name="max_velocity">292.444791136 / 100</param>
+				</hardware>
+			</xacro:unless>
+			<xacro:if value="${use_mock_hardware}">
+				<hardware>
+					<plugin>mock_components/GenericSystem</plugin>
+					<param name="calculate_dynamics">true</param>
+				</hardware>
+			</xacro:if>
+			<joint name="J3">
+				<command_interface name="velocity">
+					<param name="max">292.444791137</param>
+				</command_interface>
+				<command_interface name="position">
+					<param name="max">12.5663706144</param>
+				</command_interface>
+				<state_interface name="velocity">
+					<param name="max">292.444791137</param>
+					<param name="initial_value">0.0</param>
+				</state_interface>
+				<state_interface name="position">
+					<param name="max">12.5663706144</param>
+					<param name="initial_value">0.0</param>
+				</state_interface>
+			</joint>
+		</ros2_control>
+		<ros2_control name="arm_J4" type="system">
+			<xacro:unless value="${use_mock_hardware}">
+				<hardware>
+					<plugin>blcmd_hardware/BLCMDHardware</plugin>
+					<param name="candevice">can1</param>
+					<param name="canid">4</param>
+					<param name="resolver_reduction">15</param>
+					<param name="clock_rate">100000000</param>
+					<param name="revolution_pulses">8192</param>
+					<param name="min_interval">1728</param>
+					<param name="gear_ratio">15.0</param>
+					<param name="mock">true</param>
+					<param name="reversed">false</param>
 					<param name="integrate_velocity">true</param>
-				</hardware>
-			</xacro:unless>
-			<xacro:if value="${use_mock_hardware}">
-				<hardware>
-					<plugin>mock_components/GenericSystem</plugin>
-					<param name="calculate_dynamics">true</param>
-				</hardware>
-			</xacro:if>
-			<joint name="J2">
-				<command_interface name="velocity">
-					<param name="max">1</param>
-				</command_interface>
-				<command_interface name="position">
-				</command_interface>
-				<state_interface name="velocity">
-					<param name="initial_value">0.0</param>
-				</state_interface>
-				<state_interface name="position">
-					<param name="initial_value">0.0</param>
-				</state_interface>
-			</joint>
-		</ros2_control>
-		<ros2_control name="arm_J3" type="system">
-			<xacro:unless value="${use_mock_hardware}">
-				<hardware>
-					<plugin>blcmd_hardware/BLCMDHardware</plugin>
-					<param name="candevice">can1</param>
-					<param name="canid">4F3</param>
-					<param name="resolver_reduction">1.33333333333</param>
-					<param name="clock_rate">100000000</param>
-					<param name="revolution_pulses">8192</param>
-					<param name="min_interval">122</param>
-					<param name="gear_ratio">36.0</param>
-					<param name="mock">true</param>
-					<param name="reversed">true</param>
-					<param name="integrate_velocity">true</param>
-				</hardware>
-			</xacro:unless>
-			<xacro:if value="${use_mock_hardware}">
-				<hardware>
-					<plugin>mock_components/GenericSystem</plugin>
-					<param name="calculate_dynamics">true</param>
-				</hardware>
-			</xacro:if>
-			<joint name="J3">
-				<command_interface name="velocity">
-					<param name="max">1</param>
-				</command_interface>
-				<command_interface name="position">
-				</command_interface>
-				<state_interface name="velocity">
-					<param name="initial_value">0.0</param>
-				</state_interface>
-				<state_interface name="position">
-					<param name="initial_value">0.0</param>
-				</state_interface>
-			</joint>
-		</ros2_control>
-		<ros2_control name="arm_J4" type="system">
-			<xacro:unless value="${use_mock_hardware}">
-				<hardware>
-					<plugin>blcmd_hardware/BLCMDHardware</plugin>
-					<param name="candevice">can1</param>
-					<param name="canid">4F4</param>
-					<param name="resolver_reduction">1.33333333333</param>
-					<param name="clock_rate">100000000</param>
-					<param name="revolution_pulses">8192</param>
-					<param name="min_interval">122</param>
-					<param name="gear_ratio">36.0</param>
-					<param name="mock">true</param>
-					<param name="reversed">true</param>
-					<param name="integrate_velocity">true</param>
+					<param name="max_position">12.5663706144</param>
+					<param name="position_offset">0.0</param>
+					<param name="max_velocity">292.444791136 / 15</param>
 				</hardware>
 			</xacro:unless>
@@ -142,12 +164,15 @@
 			<joint name="J4">
 				<command_interface name="velocity">
-					<param name="max">1</param>
-				</command_interface>
-				<command_interface name="position">
-				</command_interface>
-				<state_interface name="velocity">
-					<param name="initial_value">0.0</param>
-				</state_interface>
-				<state_interface name="position">
+					<param name="max">292.444791137</param>
+				</command_interface>
+				<command_interface name="position">
+					<param name="max">12.5663706144</param>
+				</command_interface>
+				<state_interface name="velocity">
+					<param name="max">292.444791137</param>
+					<param name="initial_value">0.0</param>
+				</state_interface>
+				<state_interface name="position">
+					<param name="max">12.5663706144</param>
 					<param name="initial_value">0.0</param>
 				</state_interface>
@@ -159,13 +184,16 @@
 					<plugin>blcmd_hardware/BLCMDHardware</plugin>
 					<param name="candevice">can1</param>
-					<param name="canid">4F5</param>
-					<param name="resolver_reduction">1.33333333333</param>
-					<param name="clock_rate">100000000</param>
-					<param name="revolution_pulses">8192</param>
-					<param name="min_interval">122</param>
-					<param name="gear_ratio">36.0</param>
-					<param name="mock">true</param>
-					<param name="reversed">true</param>
-					<param name="integrate_velocity">true</param>
+					<param name="canid">5</param>
+					<param name="resolver_reduction">1.0</param>
+					<param name="clock_rate">100000000</param>
+					<param name="revolution_pulses">8192</param>
+          			<param name="min_interval">1792</param>
+					<param name="gear_ratio">1.0</param>
+					<param name="mock">true</param>
+					<param name="reversed">false</param>
+					<param name="integrate_velocity">false</param>
+					<param name="max_position">12.5663706144</param>
+					<param name="position_offset">3.14159265359</param>
+					<param name="max_velocity">292.444791136</param>
 				</hardware>
 			</xacro:unless>
@@ -178,12 +206,15 @@
 			<joint name="J5">
 				<command_interface name="velocity">
-					<param name="max">1</param>
-				</command_interface>
-				<command_interface name="position">
-				</command_interface>
-				<state_interface name="velocity">
-					<param name="initial_value">0.0</param>
-				</state_interface>
-				<state_interface name="position">
+					<param name="max">292.444791137</param>
+				</command_interface>
+				<command_interface name="position">
+					<param name="max">12.5663706144</param>
+				</command_interface>
+				<state_interface name="velocity">
+					<param name="max">292.444791137</param>
+					<param name="initial_value">0.0</param>
+				</state_interface>
+				<state_interface name="position">
+					<param name="max">12.5663706144</param>
 					<param name="initial_value">0.0</param>
 				</state_interface>
@@ -195,13 +226,17 @@
 					<plugin>blcmd_hardware/BLCMDHardware</plugin>
 					<param name="candevice">can1</param>
-					<param name="canid">4F6</param>
-					<param name="resolver_reduction">1.33333333333</param>
-					<param name="clock_rate">100000000</param>
-					<param name="revolution_pulses">8192</param>
-					<param name="min_interval">122</param>
-					<param name="gear_ratio">36.0</param>
-					<param name="mock">true</param>
-					<param name="reversed">true</param>
-					<param name="integrate_velocity">true</param>
+					<param name="canid">6</param>
+					<param name="resolver_reduction">1.0</param>
+					<param name="clock_rate">100000000</param>
+					<param name="revolution_pulses">8192</param>
+          			<param name="min_interval">1792</param>
+					<param name="gear_ratio">1.0</param>
+					<param name="mock">true</param>
+					<param name="reversed">false</param>
+					<param name="integrate_velocity">false</param>
+					<param name="max_position">12.5663706144</param>
+					<param name="position_offset">3.14159265359</param>
+					<!-- <param name="max_velocity">146.222395568</param> -->
+					<param name="max_velocity">292.444791136</param>
 				</hardware>
 			</xacro:unless>
@@ -214,13 +249,16 @@
 			<joint name="J6">
 				<command_interface name="velocity">
-					<param name="max">1</param>
-				</command_interface>
-				<command_interface name="position">
-				</command_interface>
-				<state_interface name="velocity">
-					<param name="initial_value">0.0</param>
-				</state_interface>
-				<state_interface name="position">
-					<param name="initial_value">0.0</param>
+					<param name="max">292.444791137</param>
+				</command_interface>
+				<command_interface name="position">
+					<param name="max">12.5663706144</param>
+				</command_interface>
+				<state_interface name="velocity">
+					<param name="max">292.444791137</param>
+					<param name="initial_value">0.0</param>
+				</state_interface>
+				<state_interface name="position">
+					<param name="initial_value">0.0</param>
+					<param name="max">12.5663706144</param>
 				</state_interface>
 			</joint>
