Commit message: [WIP] Merge `arm-master` (#425)
Signed-off-by: Bailey Chessum <bailey.chessum1@gmail.com>
Co-authored-by: RohitPilakkat <rohit.pilakkat@gmail.com>
Co-authored-by: arbabf <arbab.fahm@gmail.com>
Co-authored-by: Orlando Chamberlain <ocha0025@student.monash.edu>
Co-authored-by: Felicity Matthews <felicitymatthews30@gmail.com>
Co-authored-by: Monash Nova Rover <novaroverteam@monash.edu>
Co-authored-by: Anthony Lew <anthony@v01dbreaker.cc>
Co-authored-by: Victor Bartlinski <vicbart08@gmail.com>
Co-authored-by: Orlando Chamberlain <orlandoch.dev@gmail.com>
Co-authored-by: hacker1024 <jlei0014@student.monash.edu>
Co-authored-by: arbabf <34561149+arbabf@users.noreply.github.com>
Co-authored-by: Anthony Lew <ant87518@gmail.com>

File: src/ros/rover/rover_description/banksia_arm/urdf/arm.urdf.xacro (robot description, xacro)
@@ -26,7 +26,7 @@
     </visual>
     <collision>
-      <origin xyz="-0.0671788 0.129712 -0.183721" rpy="-1.88173e-16 -1.99729e-09 -1.5708" />
-      <geometry>
-        <mesh filename="file://$(find rover_description)/banksia_arm/meshes/armmount.stl" />
+      <origin xyz="0 0 -0.085" rpy="0 0 0" />
+      <geometry>
+        <box size="0.34 0.27 0.19"/>
       </geometry>
     </collision>
@@ -47,10 +47,4 @@
       </material>
     </visual>
-    <collision>
-      <origin xyz="-9.93063e-18 0 5.55112e-17" rpy="3.14159 -0 -7.70285e-39" />
-      <geometry>
-        <mesh filename="file://$(find rover_description)/banksia_arm/meshes/gearbox.stl" />
-      </geometry>
-    </collision>
   </link>
   <link name="linkagedrive">
@@ -70,7 +64,13 @@
     </visual>
     <collision>
-      <origin xyz="-1.58901e-15 -1.36391e-16 -5.55112e-17" rpy="6.68673e-23 -1.0222e-22 2.39693e-07" />
-      <geometry>
-        <mesh filename="file://$(find rover_description)/banksia_arm/meshes/linkagedrive.stl" />
+      <origin xyz="0 0 0.065" rpy="0 0 0" />
+      <geometry>
+        <box size="0.17 0.13 0.13"/>
+      </geometry>
+    </collision>
+    <collision>
+      <origin xyz="0 0 0.13" rpy="0 1.5708 0" />
+      <geometry>
+        <cylinder length="0.33" radius="0.065"/>
       </geometry>
     </collision>
@@ -92,7 +92,7 @@
     </visual>
     <collision>
-      <origin xyz="3.1979e-15 -6.85563e-15 0.0239" rpy="1.5708 1.5708 0" />
-      <geometry>
-        <mesh filename="file://$(find rover_description)/banksia_arm/meshes/l1.stl" />
+      <origin xyz="0 -0.255 0.024" rpy="0 0 0" />
+      <geometry>
+        <box size="0.043 0.53 0.1125"/>
       </geometry>
     </collision>
@@ -114,7 +114,43 @@
     </visual>
     <collision>
-      <origin xyz="0.398641 0.301803 6.48063e-16" rpy="2.49358 1.5708 0" />
-      <geometry>
-        <mesh filename="file://$(find rover_description)/banksia_arm/meshes/l2.stl" />
+      <origin xyz="0 0.11 0" rpy="0 0 0" />
+      <geometry>
+        <box size="0.04 0.44 0.028"/>
+      </geometry>
+    </collision>
+    <collision>
+      <origin xyz="0 0.33 0.0065" rpy="0 0 0" />
+      <geometry>
+        <box size="0.026 0.013 0.123"/>
+      </geometry>
+    </collision>
+    <collision>
+      <origin xyz="0 0.379 0.065" rpy="0 0 0" />
+      <geometry>
+        <box size="0.026 0.11 0.01"/>
+      </geometry>
+    </collision>
+    <collision>
+      <origin xyz="0 0.379 -0.05" rpy="0 0 0" />
+      <geometry>
+        <box size="0.026 0.11 0.01"/>
+      </geometry>
+    </collision>
+    <collision>
+      <origin xyz="0 0.349 -0.072" rpy="0 0 0" />
+      <geometry>
+        <box size="0.041 0.185 0.03"/>
+      </geometry>
+    </collision>
+    <collision>
+      <origin xyz="0 0.3635 -0.072" rpy="0 0 0" />
+      <geometry>
+        <box size="0.07 0.02 0.03"/>
+      </geometry>
+    </collision>
+    <collision>
+      <origin xyz="0 0.275 -0.0025" rpy="0 0 0" />
+      <geometry>
+        <cylinder length="0.082" radius="0.045"/>
       </geometry>
     </collision>
@@ -135,10 +171,4 @@
       </material>
     </visual>
-    <collision>
-      <origin xyz="1.94289e-15 0.05075 -0.0795" rpy="1.5708 1.5708 0" />
-      <geometry>
-        <mesh filename="file://$(find rover_description)/banksia_arm/meshes/j5.stl" />
-      </geometry>
-    </collision>
   </link>
   <link name="j6">
@@ -158,7 +188,25 @@
     </visual>
     <collision>
-      <origin xyz="5.80265e-16 -0.1945 0.05075" rpy="-1.5708 -1.48145e-14 -7.47144e-23" />
-      <geometry>
-        <mesh filename="file://$(find rover_description)/banksia_arm/meshes/j6.stl" />
+      <origin xyz="0 -0.09 0.1" rpy="0 0 0" />
+      <geometry>
+        <box size="0.06 0.2 0.01"/>
+      </geometry>
+    </collision>
+    <collision>
+      <origin xyz="0 -0.09 0" rpy="0 0 0" />
+      <geometry>
+        <box size="0.06 0.2 0.01"/>
+      </geometry>
+    </collision>
+    <collision>
+      <origin xyz="0 -0.145 0.05" rpy="0 0 0" />
+      <geometry>
+        <box size="0.06 0.09 0.1"/>
+      </geometry>
+    </collision>
+    <collision>
+      <origin xyz="0 -0.169 0.05" rpy="1.5708 0 0" />
+      <geometry>
+        <cylinder length="0.025" radius="0.045"/>
       </geometry>
     </collision>
@@ -180,7 +228,7 @@
     </visual>
     <collision>
-      <origin xyz="0.00775 0.013 0.0215" rpy="-6.15694e-07 4.61983e-15 3.14159" />
-      <geometry>
-        <mesh filename="file://$(find rover_description)/banksia_arm/meshes/eebase.stl" />
+      <origin xyz="0 0.02 0.0675" rpy="0 0 0" />
+      <geometry>
+        <box size="0.25 0.08 0.075"/>
       </geometry>
     </collision>
@@ -201,12 +249,6 @@
       </material>
     </visual>
-    <collision>
-      <origin xyz="-3.64856e-05 0.115305 0.0109" rpy="-3.14159 -6.60532e-30 2.57948e-23" />
-      <geometry>
-        <mesh filename="file://$(find rover_description)/banksia_arm/meshes/rightfinger.stl" />
-      </geometry>
-    </collision>
-  </link>
-  <link name="arm_end_side">
+  </link>
+  <link name="arm_end_side_optical">
     <inertial>
       <origin xyz="5.0388580281e-20 -5.0000002375e-04 -2.0596424901e-20" rpy="0 0 0" />
@@ -223,15 +265,9 @@
       </material>
     </visual>
-    <collision>
-      <origin xyz="0 0 0" rpy="1.5708 1.86776e-19 -2.0576e-24" />
-      <geometry>
-        <mesh filename="file://$(find rover_description)/banksia_arm/meshes/arm_end_side.stl" />
-      </geometry>
-    </collision>
   </link>
   <joint name="camera_ee_side" type="fixed">
-    <origin xyz="-0.000216235 0.178108 -0.0547417" rpy="3.14159 0.00174763 1.5708" />
+    <origin xyz="-0.000216235 0.178108 -0.0547417" rpy="0 0.00174763 3.14159" />
     <parent link="rightfinger" />
-    <child link="arm_end_side" />
+    <child link="arm_end_side_optical" />
     <axis xyz="0 0 1" />
     <limit effort="10" velocity="10" />
@@ -259,10 +295,4 @@
       </material>
     </visual>
-    <collision>
-      <origin xyz="-8.71485e-06 -0.115251 0.0109" rpy="-3.14159 4.996e-15 -5.80744e-23" />
-      <geometry>
-        <mesh filename="file://$(find rover_description)/banksia_arm/meshes/leftfinger.stl" />
-      </geometry>
-    </collision>
   </link>
   <link name="actuator">
@@ -281,10 +311,4 @@
       </material>
     </visual>
-    <collision>
-      <origin xyz="-1.38778e-17 0 -0.058" rpy="3.11287e-20 2.12505e-23 1.99292e-27" />
-      <geometry>
-        <mesh filename="file://$(find rover_description)/banksia_arm/meshes/actuator.stl" />
-      </geometry>
-    </collision>
   </link>
   <joint name="actuator_head" type="prismatic">
@@ -295,5 +319,5 @@
     <limit effort="10" velocity="10" lower="-1.22125e-15" upper="0.055" />
   </joint>
-  <link name="arm_end_finger">
+  <link name="arm_end_finger_optical">
     <inertial>
       <origin xyz="5.0388580281e-20 -5.0000002375e-04 -2.0596424901e-20" rpy="0 0 0" />
@@ -310,15 +334,9 @@
       </material>
     </visual>
-    <collision>
-      <origin xyz="2.77556e-17 0 -1.11022e-16" rpy="1.5708 -2.87448e-18 1.5822e-23" />
-      <geometry>
-        <mesh filename="file://$(find rover_description)/banksia_arm/meshes/arm_end_finger.stl" />
-      </geometry>
-    </collision>
   </link>
   <joint name="camera_ee_finger" type="fixed">
-    <origin xyz="1.96205e-05 -0.0711415 -0.0299814" rpy="-3.14152 1.52166 -1.5708" />
+    <origin xyz="1.96205e-05 -0.0711415 -0.0299814" rpy="-3.14152 ${radians(180) + 1.52166} -1.5708" />
     <parent link="leftfinger" />
-    <child link="arm_end_finger" />
+    <child link="arm_end_finger_optical" />
     <axis xyz="0 0 1" />
     <limit effort="10" velocity="10" />
@@ -331,5 +349,5 @@
     <limit effort="10" velocity="10" lower="0" upper="0.084" />
   </joint>
-  <link name="arm_end_top">
+  <link name="arm_end_top_optical">
     <inertial>
       <origin xyz="5.0388580281e-20 -5.0000002375e-04 -2.0596424901e-20" rpy="0 0 0" />
@@ -346,19 +364,13 @@
       </material>
     </visual>
-    <collision>
-      <origin xyz="1.11022e-16 0 0" rpy="1.5708 -2.5589e-20 3.89707e-23" />
-      <geometry>
-        <mesh filename="file://$(find rover_description)/banksia_arm/meshes/arm_end_top.stl" />
-      </geometry>
-    </collision>
   </link>
   <joint name="camera_ee_top" type="fixed">
-    <origin xyz="-6.33269e-14 0.10042 0.231753" rpy="3.14159 -1.56853 1.5708" />
+    <origin xyz="-6.33269e-14 0.10042 0.231753" rpy="1.5708 ${-1.56853 - radians(90)} 0" />
     <parent link="eebase" />
-    <child link="arm_end_top" />
+    <child link="arm_end_top_optical" />
     <axis xyz="0 0 1" />
     <limit effort="10" velocity="10" />
   </joint>
-  <link name="arm_end_periscope">
+  <link name="arm_end_periscope_optical">
     <inertial>
       <origin xyz="5.0388580281e-20 -5.0000002375e-04 -2.0596424901e-20" rpy="0 0 0" />
@@ -375,24 +387,18 @@
       </material>
     </visual>
-    <collision>
-      <origin xyz="0 0 0" rpy="1.5708 -1.12386e-23 -2.15772e-29" />
-      <geometry>
-        <mesh filename="file://$(find rover_description)/banksia_arm/meshes/arm_end_periscope.stl" />
-      </geometry>
-    </collision>
   </link>
   <joint name="camera_ee_periscope" type="fixed">
-    <origin xyz="-0.00015 -0.0378336 0.0594947" rpy="-3.14159 6.15694e-07 -1.5708" />
+     <origin xyz="-0.00015 -0.0378336 0.0594947" rpy="-3.14159 -3.14159 0" />
     <parent link="eebase" />
-    <child link="arm_end_periscope" />
+    <child link="arm_end_periscope_optical" />
     <axis xyz="0 0 1" />
     <limit effort="10" velocity="10" />
   </joint>
-  <joint name="J6" type="continuous">
+  <joint name="J6" type="revolute">
     <origin xyz="5.64652e-16 -0.1945 0.05075" rpy="1.5708 -1.48145e-14 2.12503e-17" />
     <parent link="j6" />
     <child link="eebase" />
     <axis xyz="0 0 1" />
-    <limit effort="10" velocity="10" />
+    <limit effort="10" velocity="10" lower="0" upper="0"/>
   </joint>
   <joint name="J5" type="revolute">
@@ -401,5 +407,5 @@
     <child link="j6" />
     <axis xyz="0 0 1" />
-    <limit effort="10" velocity="10" lower="-1.5708" upper="1.91986" />
+    <limit effort="10" velocity="10" lower="0" upper="0" />
   </joint>
   <joint name="J4" type="revolute">
@@ -408,12 +414,23 @@
     <child link="j5" />
     <axis xyz="0 0 1" />
-    <limit effort="10" velocity="10" lower="-1.5708" upper="1.5708" />
-  </joint>
-  <joint name="l1a_tp" type="continuous">
+    <limit effort="10" velocity="10" lower="0" upper="0" />
+  </joint>
+  <!-- Enables proper 4 bar linkage kinematics -->
+  <link name="l1a_tp_j2_mimic"/>
+  <joint name="l1a_tp_j2_mimic_joint" type="revolute">
+    <origin xyz="0 0 0" rpy="0.0 0.0 0.0" />
+    <parent link="l1a_tp_j2_mimic" />
+    <child link="l2" />
+    <axis xyz="0 0 1" />
+    <limit effort="10" velocity="10" lower="-3.14" upper="3.14"/>
+    <mimic joint="J2" multiplier="-1" offset="0"/>
+  </joint>
+  <joint name="l1a_tp" type="revolute">
     <origin xyz="7.73032e-10 -0.5 0.0239" rpy="5.57224e-15 1.15529e-15 1.5708" />
     <parent link="l1" />
-    <child link="l2" />
-    <axis xyz="0 0 1" />
-    <limit effort="10" velocity="10" />
+    <child link="l1a_tp_j2_mimic" />
+    <axis xyz="0 0 1" />
+    <limit effort="10" velocity="10" lower="0" upper="0"/>
+    <mimic joint="J3" multiplier="1" offset="0"/>
   </joint>
   <joint name="J2" type="revolute">
@@ -422,5 +439,5 @@
     <child link="l1" />
     <axis xyz="0 0 1" />
-    <limit effort="10" velocity="10" lower="-3.141592653589793" upper="3.141592653589793" />
+    <limit effort="10" velocity="10" lower="0" upper="0" />
   </joint>
   <link name="l2prime">
@@ -439,10 +456,4 @@
       </material>
     </visual>
-    <collision>
-      <origin xyz="2.77556e-17 0 -0.006" rpy="1.5708 1.5708 0" />
-      <geometry>
-        <mesh filename="file://$(find rover_description)/banksia_arm/meshes/l2prime.stl" />
-      </geometry>
-    </collision>
   </link>
   <link name="l1prime">
@@ -461,10 +472,4 @@
       </material>
     </visual>
-    <collision>
-      <origin xyz="-0.0797283 0.0603606 1.05415e-16" rpy="1.5708 1.5708 0" />
-      <geometry>
-        <mesh filename="file://$(find rover_description)/banksia_arm/meshes/l1prime.stl" />
-      </geometry>
-    </collision>
   </link>
   <link name="l2cam">
@@ -483,24 +488,38 @@
       </material>
     </visual>
-    <collision>
-      <origin xyz="-0.0797283 0.560361 2.48639e-16" rpy="1.5708 1.5708 0" />
-      <geometry>
-        <mesh filename="file://$(find rover_description)/banksia_arm/meshes/l2cam.stl" />
-      </geometry>
-    </collision>
-  </link>
-  <joint name="l1b_tp" type="continuous">
+  </link>
+  <link name="l2cam_mimic"/>
+  <joint name="l2cam_mimic_joint" type="revolute">
+    <origin xyz="0 0 0" rpy="0.0 0.0 0.0" />
+    <parent link="l2cam_mimic" />
+    <child link="l2cam" />
+    <axis xyz="0 0 1" />
+    <limit effort="10" velocity="10" lower="-3.14" upper="3.14"/>
+    <mimic joint="J3" multiplier="1" offset="0"/>
+  </joint>
+  <joint name="l1b_tp" type="revolute">
     <origin xyz="3.05311e-16 -0.5 5.77479e-16" rpy="-1.0988e-15 4.62615e-16 0.648016" />
     <parent link="l1prime" />
-    <child link="l2cam" />
-    <axis xyz="0 0 1" />
-    <limit effort="10" velocity="10" />
-  </joint>
-  <joint name="l1b_bp" type="continuous">
+    <child link="l2cam_mimic" />
+    <axis xyz="0 0 1" />
+    <limit effort="10" velocity="10" lower="0" upper="0"/>
+    <mimic joint="J2" multiplier="-1" offset="0"/>
+  </joint>
+  <link name="l1prime_mimic"/>
+  <joint name="l1prime_mimic_joint" type="revolute">
+    <origin xyz="0 0 0" rpy="0.0 0.0 0.0" />
+    <parent link="l1prime_mimic" />
+    <child link="l1prime" />
+    <axis xyz="0 0 1" />
+    <limit effort="10" velocity="10" lower="-3.14" upper="3.14"/>
+    <mimic joint="J3" multiplier="-1" offset="0"/>
+  </joint>
+  <joint name="l1b_bp" type="revolute">
     <origin xyz="0.0797283 -0.0603606 -0.006" rpy="-1.08371e-22 -4.6005e-22 -0.648016" />
     <parent link="l2prime" />
-    <child link="l1prime" />
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
File: src/ros/rover/rover_description/banksia_arm/urdf/arm_joints.xacro (robot description, xacro)
@@ -4,5 +4,6 @@
      <gazebo>
           <plugin filename="gz-sim-joint-state-publisher-system" name="gz::sim::systems::JointStatePublisher">
-               <topic>arm_joints</topic>
+               <topic>joint_states</topic>
+               <joint_name>arm_kinematics_origin_joint</joint_name>
                <joint_name>J1</joint_name>
                <joint_name>J2</joint_name>

File: src/ros/rover/rover_description/banksia_arm/urdf/joint_states_with_arm.xacro (robot description, xacro)
@@ -4,5 +4,5 @@
     <gazebo>
         <plugin filename="gz-sim-joint-state-publisher-system" name="gz::sim::systems::JointStatePublisher">
-            <topic>dynamic_joints</topic>
+            <topic>joint_states</topic>
             <joint_name>blp</joint_name>
             <joint_name>brp</joint_name>

File: src/ros/rover/rover_description/waratah_arm/urdf/arm.urdf.xacro (robot description, xacro)
@@ -100,6 +100,6 @@
       xyz="0 1 0" />
     <limit
-      lower="0"
-      upper="0"
+      lower="-2"
+      upper="2"
       effort="0"
       velocity="0" />
@@ -443,8 +443,24 @@
       xyz="0 0 1" />
     <limit
-      lower="0"
-      upper="0"
-      effort="0"
-      velocity="0" />
-  </joint>
+      lower="-1.57079632679"
+      upper="1.57079632679"
+      effort="0"
+      velocity="0" />
+  </joint>
+  <!-- Kinematics -->
+  <link name="arm_kinematics_origin"/>
+  <joint name="arm_kinematics_origin_joint" type="fixed">
+    <origin xyz="0.0 0.0 0.0" rpy="0.0 0.0 0.0" />
+    <parent link="$(arg prefix)_link" />
+    <child link="arm_kinematics_origin" />
+  </joint>
+  <link name="endeffector_kinematics"/>
+  <joint name="endeffector_kinematics_joint" type="fixed">
+    <!-- before rotating to match IK function expected 0: 1.5707963 0.0 1.5707963 -->
+    <origin xyz="0.0067503 -0.0012 0.2225" rpy="-1.57079632679 -1.57079632679 0.0" />
+    <parent link="$(arg prefix)_j6_to_ee" />
+    <child link="endeffector_kinematics" />
+  </joint>
+  <xacro:include filename="$(find rover_description)/waratah_arm/urdf/arm.ros2_control.xacro" />
+  <xacro:arm_ros2_control use_mock_hardware="$(arg use_mock_hardware)"/>
 </robot>

Commit message: fixing arm issues

File: src/ros/rover/rover_description/banksia/urdf/gz_ros2_control.xacro (robot description, xacro)
@@ -117,154 +117,4 @@
       </state_interface>
     </joint>
-    <joint name="J1">
-      <command_interface name="velocity">
-        <param name="max">1</param>
-      </command_interface>
-      <command_interface name="position">
-      </command_interface>
-      <state_interface name="velocity">
-        <param name="initial_value">0.0</param>
-      </state_interface>
-      <state_interface name="position">
-        <param name="initial_value">0.0</param>
-      </state_interface>
-    </joint>
-    <joint name="J2">
-      <command_interface name="velocity">
-        <param name="max">1</param>
-      </command_interface>
-      <command_interface name="position">
-      </command_interface>
-      <state_interface name="velocity">
-        <param name="initial_value">0.0</param>
-      </state_interface>
-      <state_interface name="position">
-        <param name="initial_value">0.0</param>
-      </state_interface>
-    </joint>
-    <joint name="J3">
-      <command_interface name="velocity">
-        <param name="max">1</param>
-      </command_interface>
-      <command_interface name="position">
-      </command_interface>
-      <state_interface name="velocity">
-        <param name="initial_value">0.0</param>
-      </state_interface>
-      <state_interface name="position">
-        <param name="initial_value">0.0</param>
-      </state_interface>
-    </joint>
-    <!-- <joint name="l1b_bp">
-		<command_interface name="velocity">
-		  <param name="max">1</param>
-		</command_interface>
-		<state_interface name="velocity">
-		  <param name="initial_value">0.0</param>
-		</state_interface>
-		<state_interface name="position">
-		  <param name="initial_value">0.0</param>
-		</state_interface>
-      </joint>
-	  <joint name="l1b_tp">
-		<command_interface name="velocity">
-		  <param name="max">1</param>
-		</command_interface>
-		<state_interface name="velocity">
-		  <param name="initial_value">0.0</param>
-		</state_interface>
-		<state_interface name="position">
-		  <param name="initial_value">0.0</param>
-		</state_interface>
-      </joint>
-	  <joint name="l1a_tp">
-		<command_interface name="velocity">
-		  <param name="max">1</param>
-		</command_interface>
-		<state_interface name="velocity">
-		  <param name="initial_value">0.0</param>
-		</state_interface>
-		<state_interface name="position">
-		  <param name="initial_value">0.0</param>
-		</state_interface>
-      </joint> -->
-    <joint name="J4">
-      <command_interface name="velocity">
-        <param name="max">1</param>
-      </command_interface>
-      <command_interface name="position">
-      </command_interface>
-      <state_interface name="velocity">
-        <param name="initial_value">0.0</param>
-      </state_interface>
-      <state_interface name="position">
-        <param name="initial_value">0.0</param>
-      </state_interface>
-    </joint>
-    <joint name="J5">
-      <command_interface name="velocity">
-        <param name="max">1</param>
-      </command_interface>
-      <command_interface name="position">
-      </command_interface>
-      <state_interface name="velocity">
-        <param name="initial_value">0.0</param>
-      </state_interface>
-      <state_interface name="position">
-        <param name="initial_value">0.0</param>
-      </state_interface>
-    </joint>
-    <joint name="J6">
-      <command_interface name="velocity">
-        <param name="max">1</param>
-      </command_interface>
-      <command_interface name="position">
-      </command_interface>
-      <state_interface name="velocity">
-        <param name="initial_value">0.0</param>
-      </state_interface>
-      <state_interface name="position">
-        <param name="initial_value">0.0</param>
-      </state_interface>
-    </joint>
-    <joint name="right_slide">
-      <command_interface name="velocity">
-        <param name="max">1</param>
-      </command_interface>
-      <command_interface name="position">
-      </command_interface>
-      <state_interface name="velocity">
-        <param name="initial_value">0.0</param>
-      </state_interface>
-      <state_interface name="position">
-        <param name="initial_value">0.0</param>
-      </state_interface>
-    </joint>
-    <joint name="left_slide">
-      <command_interface name="velocity">
-        <param name="max">1</param>
-      </command_interface>
-      <command_interface name="position">
-      </command_interface>
-      <state_interface name="velocity">
-        <param name="initial_value">0.0</param>
-      </state_interface>
-      <state_interface name="position">
-        <param name="initial_value">0.0</param>
-      </state_interface>
-    </joint>
-    <joint name="actuator_head">
-      <command_interface name="velocity">
-        <param name="max">1</param>
-      </command_interface>
-      <command_interface name="position">
-      </command_interface>
-      <state_interface name="velocity">
-        <param name="initial_value">0.0</param>
-      </state_interface>
-      <state_interface name="position">
-        <param name="initial_value">0.0</param>
-      </state_interface>
-    </joint>
   </ros2_control>
   <gazebo>
