Commit message: feat: Update banksia urdf with parallel wheels as zero pivots. Also update rviz with local meshes.

File: src/ros/rover/rover_description/banksia/urdf/ckc.xacro (robot description, xacro)
@@ -22,5 +22,5 @@
         </plugin>
     </gazebo>
-    <!-- Ball joint for top left on diff bar-->
+    <!-- Ball joint for top left on diff bar
     <link name="tl_ball">
         <inertial>
@@ -54,5 +54,5 @@
         <limit effort="20" velocity="20" />
     </joint>
-    <!-- Ball joint for bottom left on diff bar-->
+    Ball joint for bottom left on diff bar
     <link name="bl_ball">
         <inertial>
@@ -86,5 +86,5 @@
         <limit effort="20" velocity="20" />
     </joint>
-        <!-- Ball joint for top right on diff bar-->
+        Ball joint for top right on diff bar
     <link name="tr_ball">
         <inertial>
@@ -118,5 +118,5 @@
         <limit effort="20" velocity="20" />
     </joint>
-    <!-- Ball joint for bottom right on diff bar-->
+    Ball joint for bottom right on diff bar
     <link name="br_ball">
         <inertial>
@@ -149,4 +149,4 @@
         <axis xyz="0 0 1"/>
         <limit effort="20" velocity="20" />
-    </joint>
+    </joint> -->
 </robot>

File: src/ros/rover/rover_description/banksia/urdf/joint_states.xacro (robot description, xacro)
@@ -16,16 +16,16 @@
             <joint_name>brw</joint_name>
             <joint_name>chassis_to_diffbar</joint_name>
-            <joint_name>tl_ball_roll</joint_name>
-            <joint_name>tl_ball_pitch</joint_name>
-            <joint_name>tl_ball_yaw</joint_name>
-            <joint_name>tr_ball_roll</joint_name>
-            <joint_name>tr_ball_pitch</joint_name>
-            <joint_name>tr_ball_yaw</joint_name>
-            <joint_name>bl_ball_roll</joint_name>
-            <joint_name>bl_ball_pitch</joint_name>
-            <joint_name>bl_ball_yaw</joint_name>
-            <joint_name>br_ball_roll</joint_name>
-            <joint_name>br_ball_pitch</joint_name>
-            <joint_name>br_ball_yaw</joint_name>
+            <joint_name>tl_ball_x</joint_name>
+            <joint_name>tl_ball_y</joint_name>
+            <joint_name>tl_ball_z</joint_name>
+            <joint_name>tr_ball_x</joint_name>
+            <joint_name>tr_ball_y</joint_name>
+            <joint_name>tr_ball_z</joint_name>
+            <joint_name>bl_ball_x</joint_name>
+            <joint_name>bl_ball_y</joint_name>
+            <joint_name>bl_ball_z</joint_name>
+            <joint_name>br_ball_x</joint_name>
+            <joint_name>br_ball_y</joint_name>
+            <joint_name>br_ball_z</joint_name>
         </plugin>
     </gazebo>
