Commit message: Remove dummy stls

File: src/ros/rover/rover_description/banksia/urdf/rover.urdf (robot description, URDF)
Before this commit: robot Banksia, 24 links, 23 joints
Links:
- link left_diffend_dummy: geometry 
- link right_diffend_dummy: geometry 

Commit message: Fix balls to stop gazebo crashing

File: src/ros/rover/rover_description/banksia/urdf/rover.urdf (robot description, URDF)
Before this commit: robot Banksia, 24 links, 23 joints
Links:
- link bl_ball_link_x: mass 1e-09 -> 0.00001
- link bl_ball_link_y: mass 1e-09 -> 0.00001
- link br_ball_link_x: mass 1e-09 -> 0.00001
- link br_ball_link_y: mass 1e-09 -> 0.00001
- link tl_ball_link_x: mass 1e-09 -> 0.00001
- link tl_ball_link_y: mass 1e-09 -> 0.00001
- link tr_ball_link_x: mass 1e-09 -> 0.00001
- link tr_ball_link_y: mass 1e-09 -> 0.00001

Commit message: update urdf with cocad simple convex meshes

File: src/ros/rover/rover_description/banksia/urdf/rover.urdf (robot description, URDF)
Before this commit: robot Banksia, 24 links, 23 joints
Links:
- link bl_ankle: geometry collision mesh filename=file://$(arg rover_description_dir)/banksia/meshes/convex_d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; collision mesh filename=file://$(arg rover_description_dir)/banksia/meshes/convex_d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
- link bl_ball_link_x: mass 0.00001 -> 1e-09
- link bl_ball_link_y: mass 0.00001 -> 1e-09
- link bl_wheel: geometry collision mesh filename=file://$(arg rover_description_dir)/banksia/meshes/convex_d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; collision mesh filename=file://$(arg rover_description_dir)/banksia/meshes/convex_d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
- link br_ankle: geometry collision mesh filename=file://$(arg rover_description_dir)/banksia/meshes/convex_d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; collision mesh filename=file://$(arg rover_description_dir)/banksia/meshes/convex_d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
- link br_wheel: geometry collision mesh filename=file://$(arg rover_description_dir)/banksia/meshes/convex_d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; collision mesh filename=file://$(arg rover_description_dir)/banksia/meshes/convex_d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
- link chassis: geometry collision mesh filename=file://$(arg rover_description_dir)/banksia/meshes/convex_d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; collision mesh filename=file://$(arg rover_description_dir)/banksia/meshes/convex_d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
- link diffbar: geometry collision mesh filename=file://$(arg rover_description_dir)/banksia/meshes/convex_d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; collision mesh filename=file://$(arg rover_description_dir)/banksia/meshes/convex_d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
- link fl_ankle: geometry collision mesh filename=file://$(arg rover_description_dir)/banksia/meshes/convex_d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; collision mesh filename=file://$(arg rover_description_dir)/banksia/meshes/convex_d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
- link fl_wheel: geometry collision mesh filename=file://$(arg rover_description_dir)/banksia/meshes/convex_d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; collision mesh filename=file://$(arg rover_description_dir)/banksia/meshes/convex_d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
- link fr_ankle: geometry collision mesh filename=file://$(arg rover_description_dir)/banksia/meshes/convex_d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; collision mesh filename=file://$(arg rover_description_dir)/banksia/meshes/convex_d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
- link fr_wheel: geometry collision mesh filename=file://$(arg rover_description_dir)/banksia/meshes/convex_d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; collision mesh filename=file://$(arg rover_description_dir)/banksia/meshes/convex_d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
- link left_diffend_dummy: geometry collision mesh filename=file://$(arg rover_description_dir)/banksia/meshes/convex_d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; collision mesh filename=file://$(arg rover_description_dir)/banksia/meshes/convex_d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
- link left_difflink: geometry collision mesh filename=file://$(arg rover_description_dir)/banksia/meshes/convex_d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; collision mesh filename=file://$(arg rover_description_dir)/banksia/meshes/convex_d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
- link left_leg: geometry collision mesh filename=file://$(arg rover_description_dir)/banksia/meshes/convex_d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; collision mesh filename=file://$(arg rover_description_dir)/banksia/meshes/convex_d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
- link right_diffend_dummy: geometry collision mesh filename=file://$(arg rover_description_dir)/banksia/meshes/convex_d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; collision mesh filename=file://$(arg rover_description_dir)/banksia/meshes/convex_d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
- link right_difflink: geometry collision mesh filename=file://$(arg rover_description_dir)/banksia/meshes/convex_d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; collision mesh filename=file://$(arg rover_description_dir)/banksia/meshes/convex_d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
- link right_leg: geometry collision mesh filename=file://$(arg rover_description_dir)/banksia/meshes/convex_d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; collision mesh filename=file://$(arg rover_description_dir)/banksia/meshes/convex_d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
- link tr_ball_link_x: mass 0.00001 -> 1e-09
- link tr_ball_link_y: mass 0.00001 -> 1e-09
Joints:
- joint chassis_to_diffbar: limit lower=2.10084e-09 upper=2.10084e-09 effort=10 velocity=10 -> effort=10 velocity=10

Commit message: rover urdf changes

File: src/ros/rover/rover_description/banksia/urdf/rover.urdf (robot description, URDF)
Before this commit: robot Banksia, 24 links, 23 joints
Links:
- link bl_ball_link_x: mass 1e-09 -> 0.00001
- link bl_ball_link_y: mass 1e-09 -> 0.00001
- link left_diffend_dummy: geometry 
- link right_diffend_dummy: geometry 
- link tr_ball_link_x: mass 1e-09 -> 0.00001
- link tr_ball_link_y: mass 1e-09 -> 0.00001
