Commit message: (WIP) Feat: URDF collisions rendering in test/urdf, warning: very messy

File: src/ros/rover/rover_description/banksia/urdf/rover.urdf (robot description, URDF)
Before this commit: robot Banksia, 24 links, 23 joints
Links:
- link bl_ankle: geometry collision box size=0.012 0.03 0.06; collision box size=0.012 0.076 0.06
- link bl_wheel: geometry collision cylinder length=0.16 radius=0.157; visual mesh filename=/rover_description/banksia/meshes/bl_wheel.stl
- link br_ankle: geometry collision box size=0.012 0.03 0.06; collision box size=0.012 0.076 0.06
- link br_wheel: geometry collision cylinder length=0.16 radius=0.157; visual mesh filename=/rover_description/banksia/meshes/br_wheel.stl
- link chassis: geometry collision box size=0.48 0.545 0.175; visual mesh filename=/rover_description/banksia/meshes/chassis.stl
- link diffbar: geometry collision cylinder length=0.41 radius=0.01; collision cylinder length=0.41 radius=0.01
- link fl_ankle: geometry collision box size=0.012 0.03 0.06; collision box size=0.012 0.076 0.06
- link fl_wheel: geometry collision cylinder length=0.16 radius=0.157; visual mesh filename=/rover_description/banksia/meshes/fl_wheel.stl
- link fr_ankle: geometry collision box size=0.012 0.03 0.06; collision box size=0.012 0.076 0.06
- link fr_wheel: geometry collision cylinder length=0.16 radius=0.157; visual mesh filename=/rover_description/banksia/meshes/fr_wheel.stl
- link left_difflink: geometry visual mesh filename=/rover_description/banksia/meshes/left_difflink.stl
- link left_leg: geometry collision box size=0.106 0.065 0.077; collision box size=0.107 0.065 0.077
- link right_difflink: geometry visual mesh filename=/rover_description/banksia/meshes/right_difflink.stl
- link right_leg: geometry collision box size=0.106 0.065 0.077; collision box size=0.107 0.065 0.077
