Commit message: Rename to old_arm and taipan

File: src/ros/rover/rover_description/old_arm/urdf/improved.arm.urdf.xacro (robot description, xacro)
@@ -30,19 +30,19 @@
       <geometry>
         <mesh
-          filename="file://$(arg rover_description_dir)/waratah_arm/meshes/arm_base.stl" />
-      </geometry>
-      <material
-        name="">
-        <color
-          rgba="0.792156862745098 0.819607843137255 0.933333333333333 1" />
-      </material>
-    </visual>
-    <collision>
-      <origin
-        xyz="0 0 0"
-        rpy="0 0 0" />
-      <geometry>
-        <mesh
-          filename="file://$(arg rover_description_dir)/waratah_arm/meshes/arm_base.stl" />
+          filename="file://$(arg rover_description_dir)/old_arm/meshes/arm_base.stl" />
+      </geometry>
+      <material
+        name="">
+        <color
+          rgba="0.792156862745098 0.819607843137255 0.933333333333333 1" />
+      </material>
+    </visual>
+    <collision>
+      <origin
+        xyz="0 0 0"
+        rpy="0 0 0" />
+      <geometry>
+        <mesh
+          filename="file://$(arg rover_description_dir)/old_arm/meshes/arm_base.stl" />
       </geometry>
     </collision>
@@ -70,19 +70,19 @@
       <geometry>
         <mesh
-          filename="file://$(arg rover_description_dir)/waratah_arm/meshes/base_to_j1.stl" />
-      </geometry>
-      <material
-        name="">
-        <color
-          rgba="0.792156862745098 0.819607843137255 0.933333333333333 1" />
-      </material>
-    </visual>
-    <collision>
-      <origin
-        xyz="0 0 0"
-        rpy="0 0 0" />
-      <geometry>
-        <mesh
-          filename="file://$(arg rover_description_dir)/waratah_arm/meshes/base_to_j1.stl" />
+          filename="file://$(arg rover_description_dir)/old_arm/meshes/base_to_j1.stl" />
+      </geometry>
+      <material
+        name="">
+        <color
+          rgba="0.792156862745098 0.819607843137255 0.933333333333333 1" />
+      </material>
+    </visual>
+    <collision>
+      <origin
+        xyz="0 0 0"
+        rpy="0 0 0" />
+      <geometry>
+        <mesh
+          filename="file://$(arg rover_description_dir)/old_arm/meshes/base_to_j1.stl" />
       </geometry>
     </collision>
@@ -128,19 +128,19 @@
       <geometry>
         <mesh
-          filename="file://$(arg rover_description_dir)/waratah_arm/meshes/j2_to_link1.stl" />
-      </geometry>
-      <material
-        name="">
-        <color
-          rgba="0.792156862745098 0.819607843137255 0.933333333333333 1" />
-      </material>
-    </visual>
-    <collision>
-      <origin
-        xyz="0 0 0"
-        rpy="0 0 0" />
-      <geometry>
-        <mesh
-          filename="file://$(arg rover_description_dir)/waratah_arm/meshes/j2_to_link1.stl" />
+          filename="file://$(arg rover_description_dir)/old_arm/meshes/j2_to_link1.stl" />
+      </geometry>
+      <material
+        name="">
+        <color
+          rgba="0.792156862745098 0.819607843137255 0.933333333333333 1" />
+      </material>
+    </visual>
+    <collision>
+      <origin
+        xyz="0 0 0"
+        rpy="0 0 0" />
+      <geometry>
+        <mesh
+          filename="file://$(arg rover_description_dir)/old_arm/meshes/j2_to_link1.stl" />
       </geometry>
     </collision>
@@ -186,19 +186,19 @@
       <geometry>
         <mesh
-          filename="file://$(arg rover_description_dir)/waratah_arm/meshes/j3_to_link2.stl" />
-      </geometry>
-      <material
-        name="">
-        <color
-          rgba="0.792156862745098 0.819607843137255 0.933333333333333 1" />
-      </material>
-    </visual>
-    <collision>
-      <origin
-        xyz="0 0 0"
-        rpy="0 0 0" />
-      <geometry>
-        <mesh
-          filename="file://$(arg rover_description_dir)/waratah_arm/meshes/j3_to_link2.stl" />
+          filename="file://$(arg rover_description_dir)/old_arm/meshes/j3_to_link2.stl" />
+      </geometry>
+      <material
+        name="">
+        <color
+          rgba="0.792156862745098 0.819607843137255 0.933333333333333 1" />
+      </material>
+    </visual>
+    <collision>
+      <origin
+        xyz="0 0 0"
+        rpy="0 0 0" />
+      <geometry>
+        <mesh
+          filename="file://$(arg rover_description_dir)/old_arm/meshes/j3_to_link2.stl" />
       </geometry>
     </collision>
@@ -244,19 +244,19 @@
       <geometry>
         <mesh
-          filename="file://$(arg rover_description_dir)/waratah_arm/meshes/link2_to_fixed_j4.stl" />
-      </geometry>
-      <material
-        name="">
-        <color
-          rgba="0.792156862745098 0.819607843137255 0.933333333333333 1" />
-      </material>
-    </visual>
-    <collision>
-      <origin
-        xyz="0 0 0"
-        rpy="0 0 0" />
-      <geometry>
-        <mesh
-          filename="file://$(arg rover_description_dir)/waratah_arm/meshes/link2_to_fixed_j4.stl" />
+          filename="file://$(arg rover_description_dir)/old_arm/meshes/link2_to_fixed_j4.stl" />
+      </geometry>
+      <material
+        name="">
+        <color
+          rgba="0.792156862745098 0.819607843137255 0.933333333333333 1" />
+      </material>
+    </visual>
+    <collision>
+      <origin
+        xyz="0 0 0"
+        rpy="0 0 0" />
+      <geometry>
+        <mesh
+          filename="file://$(arg rover_description_dir)/old_arm/meshes/link2_to_fixed_j4.stl" />
       </geometry>
     </collision>
@@ -297,19 +297,19 @@
       <geometry>
         <mesh
-          filename="file://$(arg rover_description_dir)/waratah_arm/meshes/j4_to_j5.stl" />
-      </geometry>
-      <material
-        name="">
-        <color
-          rgba="0.792156862745098 0.819607843137255 0.933333333333333 1" />
-      </material>
-    </visual>
-    <collision>
-      <origin
-        xyz="0 0 0"
-        rpy="0 0 0" />
-      <geometry>
-        <mesh
-          filename="file://$(arg rover_description_dir)/waratah_arm/meshes/j4_to_j5.stl" />
+          filename="file://$(arg rover_description_dir)/old_arm/meshes/j4_to_j5.stl" />
+      </geometry>
+      <material
+        name="">
+        <color
+          rgba="0.792156862745098 0.819607843137255 0.933333333333333 1" />
+      </material>
+    </visual>
+    <collision>
+      <origin
+        xyz="0 0 0"
+        rpy="0 0 0" />
+      <geometry>
+        <mesh
+          filename="file://$(arg rover_description_dir)/old_arm/meshes/j4_to_j5.stl" />
       </geometry>
     </collision>
@@ -355,19 +355,19 @@
       <geometry>
         <mesh
-          filename="file://$(arg rover_description_dir)/waratah_arm/meshes/j5_to_j6.stl" />
-      </geometry>
-      <material
-        name="">
-        <color
-          rgba="0.792156862745098 0.819607843137255 0.933333333333333 1" />
-      </material>
-    </visual>
-    <collision>
-      <origin
-        xyz="0 0 0"
-        rpy="0 0 0" />
-      <geometry>
-        <mesh
-          filename="file://$(arg rover_description_dir)/waratah_arm/meshes/j5_to_j6.stl" />
+          filename="file://$(arg rover_description_dir)/old_arm/meshes/j5_to_j6.stl" />
+      </geometry>
+      <material
+        name="">
+        <color
+          rgba="0.792156862745098 0.819607843137255 0.933333333333333 1" />
+      </material>
+    </visual>
+    <collision>
+      <origin
+        xyz="0 0 0"
+        rpy="0 0 0" />
+      <geometry>
+        <mesh
+          filename="file://$(arg rover_description_dir)/old_arm/meshes/j5_to_j6.stl" />
       </geometry>
     </collision>
@@ -377,12 +377,12 @@
     type="revolute">
     <origin
-      xyz="0.00022562 0.10236 0.020578"
-      rpy="0 1.5708 0" />
-    <parent
-      link="$(arg prefix)_j4_to_j5" />
+      xyz="0.00022562 -0.020578 0.10236"
+      rpy="1.5708 0 1.5708" />
+    <parent
+      link="j5_fixer" />
     <child
       link="$(arg prefix)_j5_to_j6" />
     <axis
-      xyz="0 1 0" />
+      xyz="0 0 1" />
     <limit
       lower="-1.88"
@@ -413,19 +413,19 @@
       <geometry>
         <mesh
-          filename="file://$(arg rover_description_dir)/waratah_arm/meshes/j6_to_ee.stl" />
-      </geometry>
-      <material
-        name="">
-        <color
-          rgba="0.792156862745098 0.819607843137255 0.933333333333333 1" />
-      </material>
-    </visual>
-    <collision>
-      <origin
-        xyz="0 0 0"
-        rpy="0 0 0" />
-      <geometry>
-        <mesh
-          filename="file://$(arg rover_description_dir)/waratah_arm/meshes/j6_to_ee.stl" />
+          filename="file://$(arg rover_description_dir)/old_arm/meshes/j6_to_ee.stl" />
+      </geometry>
+      <material
+        name="">
+        <color
+          rgba="0.792156862745098 0.819607843137255 0.933333333333333 1" />
+      </material>
+    </visual>
+    <collision>
+      <origin
+        xyz="0 0 0"
+        rpy="0 0 0" />
+      <geometry>
+        <mesh
+          filename="file://$(arg rover_description_dir)/old_arm/meshes/j6_to_ee.stl" />
       </geometry>
     </collision>
@@ -449,49 +449,11 @@
       velocity="0" />
   </joint>
-  <!-- Replace all this with a end effector xacro file that is shared across waratah_arm and banksia_arm-->
-  <!-- EEbase to Actuator transform for auto typing -->
-  <link name="actuator"> <!-- Actuator head position when unextended but fingers are fully open-->
-    <inertial>
-      <origin xyz="-2.0984526232e-09 -1.7951021237e-09 3.6197018104e-02" rpy="0 0 0" />
-      <mass value="0.00499493" />
-      <inertia ixx="1.9746052847e-06" ixy="3.2584721895e-14" ixz="3.1261224204e-13" iyy="1.9775524756e-06" iyz="2.6609843251e-13" izz="7.2954357931e-08" />
-    </inertial>
-  </link>
-  <joint name="actuator_j" type="fixed">
-    <origin xyz="-0.006287977 0.159 -0.0075" rpy="0 1.5708 1.57072" />
-    <parent link="rightfinger" />
-    <child link="actuator" />
-    <axis xyz="0 0 1" />
-  </joint>
-  <link name="rightfinger">
-    <inertial>
-      <origin xyz="-3.0820093691e-05 -2.4076955607e-02 1.7779582954e-02" rpy="0 0 0" />
-      <mass value="0.259097" />
-      <inertia ixx="8.0113158332e-04" ixy="-2.1276248523e-07" ixz="1.9237282265e-07" iyy="7.8712513524e-05" iyz="5.1221559668e-05" izz="8.1168195146e-04" />
-    </inertial>
-  </link>
-  <joint name="right_slide" type="fixed">
-    <origin xyz="-0.0953625 -2.37042e-08 0.0635" rpy="1.5708 -6.15694e-07 1.5708" />
-    <parent link="$(arg prefix)_j6_to_ee" />
-    <child link="rightfinger" />
-    <axis xyz="0 0 1" />
-    <limit effort="10" velocity="10"/>
-  </joint>
-  <!-- EEbase to arm_end_periscope for auto typing-->
-  <link name="arm_end_periscope_optical">
-    <inertial>
-      <origin xyz="5.0388580281e-20 -5.0000002375e-04 -2.0596424901e-20" rpy="0 0 0" />
-      <mass value="1e-09" />
-      <inertia ixx="6.3254056983e-15" ixy="-1.2661721154e-31" ixz="-1.4456719139e-31" iyy="1.2484144714e-14" iyz="7.0639301518e-32" izz="6.3254056983e-15" />
-    </inertial>
-  </link>
-  <joint name="camera_ee_periscope" type="fixed">
-     <origin xyz="-0.00015 0.0378336 0.0594947" rpy="0 0 0" />
-    <parent link="$(arg prefix)_j6_to_ee" />
-    <child link="arm_end_periscope_optical" />
-    <axis xyz="0 0 1" />
-    <limit effort="10" velocity="10" />
-  </joint>
   <!-- Kinematics -->
+  <link name="j5_fixer"/>
+  <joint name="j5_fixer_joint" type="fixed">
+    <origin xyz="0.0 0.0 0.0" rpy="-1.5708 0.0 0.0" />
+    <parent link="$(arg prefix)_j4_to_j5" />
+    <child link="j5_fixer" />
+  </joint>
   <link name="arm_kinematics_origin"/>
   <joint name="arm_kinematics_origin_joint" type="fixed">
@@ -507,5 +469,5 @@
     <child link="endeffector_kinematics" />
   </joint>
-  <xacro:include filename="$(arg rover_description_dir)/waratah_arm/urdf/arm.ros2_control.xacro" />
+  <xacro:include filename="$(arg rover_description_dir)/old_arm/urdf/arm.ros2_control.xacro" />
   <xacro:arm_ros2_control use_mock_hardware="$(arg use_mock_hardware)"/>
 </robot>

File: src/ros/rover/rover_description/taipan/urdf/arm.urdf.xacro (robot description, xacro)
@@ -20,5 +20,5 @@
       <origin xyz="-0.0671788 0.129712 -0.183721" rpy="-1.88173e-16 -1.99729e-09 -1.5708" />
       <geometry>
-        <mesh filename="file://$(arg rover_description_dir)/banksia_arm/meshes/armmount.stl" />
+        <mesh filename="file://$(arg rover_description_dir)/taipan/meshes/armmount.stl" />
       </geometry>
       <material name="armmount_material">
@@ -42,5 +42,5 @@
       <origin xyz="-9.93063e-18 0 5.55112e-17" rpy="3.14159 -0 -7.70285e-39" />
       <geometry>
-        <mesh filename="file://$(arg rover_description_dir)/banksia_arm/meshes/gearbox.stl" />
+        <mesh filename="file://$(arg rover_description_dir)/taipan/meshes/gearbox.stl" />
       </geometry>
       <material name="gearbox_material">
@@ -58,5 +58,5 @@
       <origin xyz="-1.58901e-15 -1.36391e-16 -5.55112e-17" rpy="6.68673e-23 -1.0222e-22 2.39693e-07" />
       <geometry>
-        <mesh filename="file://$(arg rover_description_dir)/banksia_arm/meshes/linkagedrive.stl" />
+        <mesh filename="file://$(arg rover_description_dir)/taipan/meshes/linkagedrive.stl" />
       </geometry>
       <material name="linkagedrive_material">
@@ -86,5 +86,5 @@
       <origin xyz="3.1979e-15 -6.85563e-15 0.0239" rpy="1.5708 1.5708 0" />
       <geometry>
-        <mesh filename="file://$(arg rover_description_dir)/banksia_arm/meshes/l1.stl" />
+        <mesh filename="file://$(arg rover_description_dir)/taipan/meshes/l1.stl" />
       </geometry>
       <material name="l1_material">
@@ -108,5 +108,5 @@
       <origin xyz="0.398641 0.301803 6.48063e-16" rpy="2.49358 1.5708 0" />
       <geometry>
-        <mesh filename="file://$(arg rover_description_dir)/banksia_arm/meshes/l2.stl" />
+        <mesh filename="file://$(arg rover_description_dir)/taipan/meshes/l2.stl" />
       </geometry>
       <material name="l2_material">
@@ -166,5 +166,5 @@
       <origin xyz="1.94289e-15 0.05075 -0.0795" rpy="1.5708 1.5708 0" />
       <geometry>
-        <mesh filename="file://$(arg rover_description_dir)/banksia_arm/meshes/j5.stl" />
+        <mesh filename="file://$(arg rover_description_dir)/taipan/meshes/j5.stl" />
       </geometry>
       <material name="j5_material">
@@ -182,5 +182,5 @@
       <origin xyz="5.80265e-16 -0.1945 0.05075" rpy="-1.5708 -1.48145e-14 -7.47144e-23" />
       <geometry>
-        <mesh filename="file://$(arg rover_description_dir)/banksia_arm/meshes/j6.stl" />
+        <mesh filename="file://$(arg rover_description_dir)/taipan/meshes/j6.stl" />
       </geometry>
       <material name="j6_material">
@@ -222,5 +222,5 @@
       <origin xyz="0.00775 0.013 0.0215" rpy="-6.15694e-07 4.61983e-15 3.14159" />
       <geometry>
-        <mesh filename="file://$(arg rover_description_dir)/banksia_arm/meshes/eebase.stl" />
+        <mesh filename="file://$(arg rover_description_dir)/taipan/meshes/eebase.stl" />
       </geometry>
       <material name="eebase_material">
@@ -244,5 +244,5 @@
       <origin xyz="-3.64856e-05 0.115305 0.0109" rpy="-3.14159 -6.60532e-30 2.57948e-23" />
       <geometry>
-        <mesh filename="file://$(arg rover_description_dir)/banksia_arm/meshes/rightfinger.stl" />
+        <mesh filename="file://$(arg rover_description_dir)/taipan/meshes/rightfinger.stl" />
       </geometry>
       <material name="rightfinger_material">
@@ -260,5 +260,5 @@
       <origin xyz="0 0 0" rpy="1.5708 1.86776e-19 -2.0576e-24" />
       <geometry>
-        <mesh filename="file://$(arg rover_description_dir)/banksia_arm/meshes/arm_end_side.stl" />
+        <mesh filename="file://$(arg rover_description_dir)/taipan/meshes/arm_end_side.stl" />
       </geometry>
       <material name="arm_end_side_material">
@@ -291,5 +291,5 @@
       <origin xyz="-8.71485e-06 -0.115251 0.0109" rpy="-3.14159 4.996e-15 -5.80744e-23" />
       <geometry>
-        <mesh filename="file://$(arg rover_description_dir)/banksia_arm/meshes/leftfinger.stl" />
+        <mesh filename="file://$(arg rover_description_dir)/taipan/meshes/leftfinger.stl" />
       </geometry>
       <material name="leftfinger_material">
@@ -307,5 +307,5 @@
       <origin xyz="-1.38778e-17 0 -0.058" rpy="3.11287e-20 2.12505e-23 1.99292e-27" />
       <geometry>
-        <mesh filename="file://$(arg rover_description_dir)/banksia_arm/meshes/actuator.stl" />
+        <mesh filename="file://$(arg rover_description_dir)/taipan/meshes/actuator.stl" />
       </geometry>
       <material name="actuator_material">
@@ -330,5 +330,5 @@
       <origin xyz="2.77556e-17 0 -1.11022e-16" rpy="1.5708 -2.87448e-18 1.5822e-23" />
       <geometry>
-        <mesh filename="file://$(arg rover_description_dir)/banksia_arm/meshes/arm_end_finger.stl" />
+        <mesh filename="file://$(arg rover_description_dir)/taipan/meshes/arm_end_finger.stl" />
       </geometry>
       <material name="arm_end_finger_material">
@@ -360,5 +360,5 @@
       <origin xyz="1.11022e-16 0 0" rpy="1.5708 -2.5589e-20 3.89707e-23" />
       <geometry>
-        <mesh filename="file://$(arg rover_description_dir)/banksia_arm/meshes/arm_end_top.stl" />
+        <mesh filename="file://$(arg rover_description_dir)/taipan/meshes/arm_end_top.stl" />
       </geometry>
       <material name="arm_end_top_material">
@@ -383,5 +383,5 @@
       <origin xyz="0 0 0" rpy="1.5708 -1.12386e-23 -2.15772e-29" />
       <geometry>
-        <mesh filename="file://$(arg rover_description_dir)/banksia_arm/meshes/arm_end_periscope.stl" />
+        <mesh filename="file://$(arg rover_description_dir)/taipan/meshes/arm_end_periscope.stl" />
       </geometry>
       <material name="arm_end_periscope_material">
@@ -452,5 +452,5 @@
       <origin xyz="2.77556e-17 0 -0.006" rpy="1.5708 1.5708 0" />
       <geometry>
-        <mesh filename="file://$(arg rover_description_dir)/banksia_arm/meshes/l2prime.stl" />
+        <mesh filename="file://$(arg rover_description_dir)/taipan/meshes/l2prime.stl" />
       </geometry>
       <material name="l2prime_material">
@@ -468,5 +468,5 @@
       <origin xyz="-0.0797283 0.0603606 1.05415e-16" rpy="1.5708 1.5708 0" />
       <geometry>
-        <mesh filename="file://$(arg rover_description_dir)/banksia_arm/meshes/l1prime.stl" />
+        <mesh filename="file://$(arg rover_description_dir)/taipan/meshes/l1prime.stl" />
       </geometry>
       <material name="l1prime_material">
@@ -484,5 +484,5 @@
       <origin xyz="-0.0797283 0.560361 2.48639e-16" rpy="1.5708 1.5708 0" />
       <geometry>
-        <mesh filename="file://$(arg rover_description_dir)/banksia_arm/meshes/l2cam.stl" />
+        <mesh filename="file://$(arg rover_description_dir)/taipan/meshes/l2cam.stl" />
       </geometry>
       <material name="l2cam_material">
@@ -572,14 +572,12 @@
   <!--    forward 0.012512-->
   <!-- Gazebo / IRL Control -->
-  <xacro:include filename="$(arg rover_description_dir)/banksia_arm/urdf/arm_ckc.xacro"/>
-  <xacro:if value="$(arg arm_control)">
-    <xacro:if value="$(arg gazebo)">
-      <xacro:include filename="$(arg rover_description_dir)/banksia_arm/urdf/arm.gz_ros2_control.xacro" />
-      <xacro:include filename="$(arg rover_description_dir)/banksia_arm/urdf/arm_sensors.xacro"/>
-    </xacro:if>
-    <xacro:unless value="$(arg gazebo)">
-      <xacro:include filename="$(arg rover_description_dir)/banksia_arm/urdf/arm.ros2_control.xacro" />
-      <xacro:arm_ros2_control use_mock_hardware="$(arg use_mock_hardware)"/>
-    </xacro:unless>
+  <xacro:include filename="$(arg rover_description_dir)/taipan/urdf/arm_ckc.xacro"/>
+  <xacro:if value="$(arg gazebo)">
+    <xacro:include filename="$(arg rover_description_dir)/taipan/urdf/arm.gz_ros2_control.xacro" />
+    <xacro:include filename="$(arg rover_description_dir)/taipan/urdf/arm_sensors.xacro"/>
   </xacro:if>
+  <xacro:unless value="$(arg gazebo)">
+    <xacro:include filename="$(arg rover_description_dir)/taipan/urdf/arm.ros2_control.xacro" />
+    <xacro:arm_ros2_control use_mock_hardware="$(arg use_mock_hardware)"/>
+  </xacro:unless>
 </robot>

File: src/ros/rover/rover_description/waratah/urdf/rover.urdf.xacro (robot description, xacro)
@@ -446,5 +446,5 @@
   <xacro:if value="$(arg arm)">
         <!-- Attaches waratah's arm -->
-        <xacro:include filename="$(arg rover_description_dir)/waratah_arm/urdf/arm.urdf.xacro" />
+        <xacro:include filename="$(arg rover_description_dir)/old_arm/urdf/arm.urdf.xacro" />
         <joint name="chassis_to_arm_base" type="fixed">
             <origin xyz="0 0.15 -0.06" rpy="0 0 1.57" />
