Commit message: drive compat

File: src/ros/rover/rover_description/banksia/urdf/ros2_control.xacro (robot description, xacro)
@@ -8,12 +8,7 @@
                     <param name="candevice">can0</param>
                     <param name="canid">1</param>
-                    <param name="resolver_reduction">1.33333333333</param>
-                    <param name="clock_rate">100000000</param>
-                    <param name="revolution_pulses">8192</param>
-                    <param name="min_interval">122</param>
-                    <param name="gear_ratio">15.0</param>
-                    <param name="mock">true</param>
-                    <param name="reversed">true</param>
-                    <param name="integrate_velocity">true</param>
+                    <param name="gear_ratio">15.0</param>
+                    <param name="max_input_vel">626.66</param>
+                    <param name="reversed">true</param>
                 </hardware>
             </xacro:unless>
@@ -25,14 +20,14 @@
             </xacro:if>
             <joint name="flw">
-		        <command_interface name="velocity">
-                    <param name="max">1</param>
-                </command_interface>
-                <command_interface name="effort">
-                    <param name="max">1</param>
-                </command_interface>
-                <state_interface name="velocity">
-                    <param name="initial_value">0.0</param>
-                </state_interface>
-                <state_interface name="position">
+		            <command_interface name="velocity">
+                    <param name="max">1</param>
+                </command_interface>
+                <command_interface name="effort">
+                    <param name="max">1</param>
+                </command_interface>
+                <state_interface name="velocity">
+                    <param name="initial_value">0.0</param>
+                </state_interface>
+                <state_interface name="effort">
                     <param name="initial_value">0.0</param>
                 </state_interface>
@@ -45,12 +40,7 @@
                     <param name="candevice">can0</param>
                     <param name="canid">2</param>
-                    <param name="resolver_reduction">1.33333333333</param>
-                    <param name="clock_rate">100000000</param>
-                    <param name="revolution_pulses">8192</param>
-                    <param name="min_interval">122</param>
-                    <param name="gear_ratio">15.0</param>
-                    <param name="mock">true</param>
-                    <param name="reversed">true</param>
-                    <param name="integrate_velocity">true</param>
+                    <param name="gear_ratio">15.0</param>
+                    <param name="max_input_vel">626.66</param>
+                    <param name="reversed">true</param>
                 </hardware>
             </xacro:unless>
@@ -62,14 +52,14 @@
             </xacro:if>
             <joint name="blw">
-                <command_interface name="velocity">
-                    <param name="max">1</param>
-                </command_interface>
-                <command_interface name="effort">
-                    <param name="max">1</param>
-                </command_interface>
-                <state_interface name="velocity">
-                    <param name="initial_value">0.0</param>
-                </state_interface>
-                <state_interface name="position">
+		            <command_interface name="velocity">
+                    <param name="max">1</param>
+                </command_interface>
+                <command_interface name="effort">
+                    <param name="max">1</param>
+                </command_interface>
+                <state_interface name="velocity">
+                    <param name="initial_value">0.0</param>
+                </state_interface>
+                <state_interface name="effort">
                     <param name="initial_value">0.0</param>
                 </state_interface>
@@ -82,12 +72,7 @@
                     <param name="candevice">can0</param>
                     <param name="canid">3</param>
-                    <param name="resolver_reduction">1.33333333333</param>
-                    <param name="clock_rate">100000000</param>
-                    <param name="revolution_pulses">8192</param>
-                    <param name="min_interval">122</param>
-                    <param name="gear_ratio">15.0</param>
-	                <param name="mock">true</param>
-                    <param name="reversed">false</param>
-                    <param name="integrate_velocity">true</param>
+                    <param name="gear_ratio">15.0</param>
+                    <param name="max_input_vel">626.66</param>
+                    <param name="reversed">true</param>
                 </hardware>
             </xacro:unless>
@@ -99,14 +84,14 @@
             </xacro:if>
             <joint name="brw">
-                <command_interface name="velocity">
-                    <param name="max">1</param>
-                </command_interface>
-                <command_interface name="effort">
-                    <param name="max">1</param>
-                </command_interface>
-                <state_interface name="velocity">
-                    <param name="initial_value">0.0</param>
-                </state_interface>
-                <state_interface name="position">
+		            <command_interface name="velocity">
+                    <param name="max">1</param>
+                </command_interface>
+                <command_interface name="effort">
+                    <param name="max">1</param>
+                </command_interface>
+                <state_interface name="velocity">
+                    <param name="initial_value">0.0</param>
+                </state_interface>
+                <state_interface name="effort">
                     <param name="initial_value">0.0</param>
                 </state_interface>
@@ -119,12 +104,7 @@
                     <param name="candevice">can0</param>
                     <param name="canid">4</param>
-                    <param name="resolver_reduction">1.33333333333</param>
-                    <param name="clock_rate">100000000</param>
-                    <param name="revolution_pulses">8192</param>
-                    <param name="min_interval">122</param>
-                    <param name="gear_ratio">15.0</param>
-	                <param name="mock">true</param>
-                    <param name="reversed">false</param>
-                    <param name="integrate_velocity">true</param>
+                    <param name="gear_ratio">15.0</param>
+                    <param name="max_input_vel">626.66</param>
+                    <param name="reversed">true</param>
                 </hardware>
             </xacro:unless>
@@ -136,14 +116,14 @@
             </xacro:if>
             <joint name="frw">
-                <command_interface name="velocity">
-                    <param name="max">1</param>
-                </command_interface>
-                <command_interface name="effort">
-                    <param name="max">1</param>
-                </command_interface>
-                <state_interface name="velocity">
-                    <param name="initial_value">0.0</param>
-                </state_interface>
-                <state_interface name="position">
+		            <command_interface name="velocity">
+                    <param name="max">1</param>
+                </command_interface>
+                <command_interface name="effort">
+                    <param name="max">1</param>
+                </command_interface>
+                <state_interface name="velocity">
+                    <param name="initial_value">0.0</param>
+                </state_interface>
+                <state_interface name="effort">
                     <param name="initial_value">0.0</param>
                 </state_interface>
@@ -156,12 +136,10 @@
                     <param name="candevice">can0</param>
                     <param name="canid">5</param>
-		            <param name="resolver_reduction">1.33333333333</param>
-                    <param name="clock_rate">100000000</param>
-                    <param name="revolution_pulses">8192</param>
-                    <param name="min_interval">233</param>
-                    <param name="gear_ratio">36.0</param>
-	                <param name="mock">true</param>
-                    <param name="reversed">true</param>
-                    <param name="position_offset">-0.70554839</param>
+		                <param name="resolver_reduction">1.33333333333</param>
+                    <param name="home_offset">14717</param>
+                    <param name="res_ticks_per_rev">98304</param>
+                    <param name="max_input_vel">328.12</param>
+                    <param name="gear_ratio">36.0</param>
+                    <param name="reversed">true</param>
                 </hardware>
             </xacro:unless>
@@ -182,4 +160,7 @@
                     <param name="max">1</param>
                 </command_interface>
+                <state_interface name="effort">
+                    <param name="initial_value">0.0</param>
+                </state_interface>
                 <state_interface name="velocity">
                     <param name="initial_value">0.0</param>
@@ -187,5 +168,4 @@
                 <state_interface name="position">
                     <param name="inital_value">0.0</param>
-                    <param name="max">1.57079632679</param>
                 </state_interface>
             </joint>
@@ -198,11 +178,8 @@
                     <param name="canid">6</param>
                     <param name="resolver_reduction">1.33333333333</param>
-                    <param name="clock_rate">100000000</param>
-                    <param name="revolution_pulses">8192</param>
-                    <param name="min_interval">233</param>
-                    <param name="gear_ratio">36.0</param>
-                    <param name="revolution_pulses">8192</param>
-                    <param name="mock">true</param>
-                    <param name="position_offset">-0.70554839</param>
+                    <param name="home_offset">14717</param>
+                    <param name="res_ticks_per_rev">98304</param>
+                    <param name="max_input_vel">328.12</param>
+                    <param name="gear_ratio">36.0</param>
                 </hardware>
             </xacro:unless>
@@ -239,11 +216,9 @@
                     <param name="canid">7</param>
                     <param name="resolver_reduction">1.33333333333</param>
-                    <param name="clock_rate">100000000</param>
-                    <param name="revolution_pulses">8192</param>
-                    <param name="min_interval">233</param>
-                    <param name="gear_ratio">36.0</param>
-	                <param name="mock">true</param>
-                    <param name="reversed">true</param>
-                    <param name="position_offset">-0.70554839</param>
+                    <param name="home_offset">14717</param>
+                    <param name="res_ticks_per_rev">98304</param>
+                    <param name="max_input_vel">328.12</param>
+                    <param name="gear_ratio">36.0</param>
+                    <param name="reversed">true</param>
                 </hardware>
             </xacro:unless>
@@ -280,10 +255,10 @@
                     <param name="canid">8</param>
                     <param name="resolver_reduction">1.33333333333</param>
-                    <param name="clock_rate">100000000</param>
-                    <param name="revolution_pulses">8192</param>
-                    <param name="min_interval">233</param>
-                    <param name="gear_ratio">36.0</param>
-	                <param name="mock">true</param>
-                    <param name="position_offset">-0.70554839</param>
+                    <param name="home_offset">14717</param>
+                    <!-- This seems wrong, it should be 2^16, but this is the value that
+                    preserves old behaviour. Maybe the resolver reduction is incorrect? -->
+                    <param name="res_ticks_per_rev">98304</param>
+                    <param name="max_input_vel">328.12</param>
+                    <param name="gear_ratio">36.0</param>
                 </hardware>
             </xacro:unless>
@@ -299,5 +274,5 @@
                 </command_interface>
                 <command_interface name="velocity">
-                    <param name="max">1.0</param>
+                    <param name="max">1</param>
                 </command_interface>
                 <command_interface name="effort">
