Commit message: feat: working new arm path planning

File: src/ros/rover/rover_description/waratah_arm/urdf/arm.ros2_control.xacro (robot description, xacro)
@@ -75,5 +75,5 @@
         <state_interface name="position">
           <param name="max">12.5663706144</param>
-          <param name="initial_value">0.0</param>
+          <param name="initial_value">0.523</param>
         </state_interface>
       </joint>
@@ -109,5 +109,5 @@
         <state_interface name="position">
           <param name="max">12.5663706144</param>
-          <param name="initial_value">0.0</param>
+          <param name="initial_value">-1.57</param>
         </state_interface>
       </joint>
@@ -143,5 +143,5 @@
         <state_interface name="position">
           <param name="max">12.5663706144</param>
-          <param name="initial_value">0.0</param>
+          <param name="initial_value">-0.785</param>
         </state_interface>
       </joint>

File: src/ros/rover/rover_description/waratah_arm/urdf/arm.urdf.xacro (robot description, xacro)
@@ -376,12 +376,12 @@
     type="revolute">
     <origin
-      xyz="0.00022562 0.10236 0.020578"
-      rpy="0 1.5708 0" />
-    <parent
-      link="$(arg prefix)_j4_to_j5" />
+      xyz="0.00022562 -0.020578 0.10236"
+      rpy="1.5708 0 1.5708" />
+    <parent
+      link="j5_fixer" />
     <child
       link="$(arg prefix)_j5_to_j6" />
     <axis
-      xyz="0 1 0" />
+      xyz="0 0 1" />
     <limit
       lower="-1.88"
@@ -449,4 +449,10 @@
   </joint>
   <!-- Kinematics -->
+  <link name="j5_fixer"/>
+  <joint name="j5_fixer_joint" type="fixed">
+    <origin xyz="0.0 0.0 0.0" rpy="-1.5708 0.0 0.0" />
+    <parent link="$(arg prefix)_j4_to_j5" />
+    <child link="j5_fixer" />
+  </joint>
   <link name="arm_kinematics_origin"/>
   <joint name="arm_kinematics_origin_joint" type="fixed">
