Commit message: feat: added configuration to make KDL somewhat usable

File: src/ros/rover/rover_description/waratah_arm/urdf/arm.urdf.xacro (robot description, xacro)
@@ -100,6 +100,6 @@
       xyz="0 1 0" />
     <limit
-      lower="0"
-      upper="0"
+      lower="-2"
+      upper="2"
       effort="0"
       velocity="0" />
@@ -443,8 +443,22 @@
       xyz="0 0 1" />
     <limit
-      lower="0"
-      upper="0"
-      effort="0"
-      velocity="0" />
+      lower="-1.57079632679"
+      upper="1.57079632679"
+      effort="0"
+      velocity="0" />
+  </joint>
+  <!-- Kinematics -->
+  <link name="arm_kinematics_origin"/>
+  <joint name="arm_kinematics_origin_joint" type="fixed">
+    <origin xyz="0.0 0.0 0.0" rpy="0.0 0.0 0.0" />
+    <parent link="$(arg prefix)_link" />
+    <child link="arm_kinematics_origin" />
+  </joint>
+  <link name="endeffector_kinematics"/>
+  <joint name="endeffector_kinematics_joint" type="fixed">
+    <!-- before rotating to match IK function expected 0: 1.5707963 0.0 1.5707963 -->
+    <origin xyz="0.0067503 -0.0012 0.2225" rpy="-1.57079632679 -1.57079632679 0.0" />
+    <parent link="$(arg prefix)_j6_to_ee" />
+    <child link="endeffector_kinematics" />
   </joint>
   <xacro:include filename="$(find rover_description)/waratah_arm/urdf/arm.ros2_control.xacro" />

Commit message: feat: add actuator to old arm urdf

File: src/ros/rover/rover_description/waratah_arm/urdf/arm.urdf.xacro (robot description, xacro)
@@ -448,4 +448,32 @@
       velocity="0" />
   </joint>
+  <!-- EEbase to Actuator transform for auto typing -->
+  <link name="actuator_frame"> <!-- Actuator head position when unextended but fingers are fully open-->
+    <inertial>
+      <origin xyz="-2.0984526232e-09 -1.7951021237e-09 3.6197018104e-02" rpy="0 0 0" />
+      <mass value="0.00499493" />
+      <inertia ixx="1.9746052847e-06" ixy="3.2584721895e-14" ixz="3.1261224204e-13" iyy="1.9775524756e-06" iyz="2.6609843251e-13" izz="7.2954357931e-08" />
+    </inertial>
+  </link>
+  <joint name="actuator" type="fixed">
+    <origin xyz="-0.006287977 0.159 -0.0075" rpy="0 1.5708 1.57072" />
+    <parent link="rightfinger" />
+    <child link="actuator_frame" />
+    <axis xyz="0 0 1" />
+  </joint>
+  <link name="rightfinger">
+    <inertial>
+      <origin xyz="-3.0820093691e-05 -2.4076955607e-02 1.7779582954e-02" rpy="0 0 0" />
+      <mass value="0.259097" />
+      <inertia ixx="8.0113158332e-04" ixy="-2.1276248523e-07" ixz="1.9237282265e-07" iyy="7.8712513524e-05" iyz="5.1221559668e-05" izz="8.1168195146e-04" />
+    </inertial>
+  </link>
+  <joint name="right_slide" type="fixed">
+    <origin xyz="-0.0953625 -2.37042e-08 0.0635" rpy="1.5708 -6.15694e-07 1.5708" />
+    <parent link="$(arg prefix)_j6_to_ee" />
+    <child link="rightfinger" />
+    <axis xyz="0 0 1" />
+    <limit effort="10" velocity="10"/>
+  </joint>
   <!-- Kinematics -->
   <link name="arm_kinematics_origin"/>

Commit message: feat: add periscope optical frame to old arm

File: src/ros/rover/rover_description/waratah_arm/urdf/arm.urdf.xacro (robot description, xacro)
@@ -448,4 +448,5 @@
       velocity="0" />
   </joint>
+  <!-- Replace all this with a end effector xacro file that is shared across waratah_arm and banksia_arm-->
   <!-- EEbase to Actuator transform for auto typing -->
   <link name="actuator_frame"> <!-- Actuator head position when unextended but fingers are fully open-->
@@ -476,4 +477,19 @@
     <limit effort="10" velocity="10"/>
   </joint>
+  <!-- EEbase to arm_end_periscope for auto typing-->
+  <link name="arm_end_periscope_optical">
+    <inertial>
+      <origin xyz="5.0388580281e-20 -5.0000002375e-04 -2.0596424901e-20" rpy="0 0 0" />
+      <mass value="1e-09" />
+      <inertia ixx="6.3254056983e-15" ixy="-1.2661721154e-31" ixz="-1.4456719139e-31" iyy="1.2484144714e-14" iyz="7.0639301518e-32" izz="6.3254056983e-15" />
+    </inertial>
+  </link>
+  <joint name="camera_ee_periscope" type="fixed">
+     <origin xyz="-0.00015 0.0378336 0.0594947" rpy="0 0 0" />
+    <parent link="$(arg prefix)_j6_to_ee" />
+    <child link="arm_end_periscope_optical" />
+    <axis xyz="0 0 1" />
+    <limit effort="10" velocity="10" />
+  </joint>
   <!-- Kinematics -->
   <link name="arm_kinematics_origin"/>

Commit message: fix: various auto_typing things

File: src/ros/rover/rover_description/waratah_arm/urdf/arm.urdf.xacro (robot description, xacro)
@@ -450,5 +450,5 @@
   <!-- Replace all this with a end effector xacro file that is shared across waratah_arm and banksia_arm-->
   <!-- EEbase to Actuator transform for auto typing -->
-  <link name="actuator_frame"> <!-- Actuator head position when unextended but fingers are fully open-->
+  <link name="actuator"> <!-- Actuator head position when unextended but fingers are fully open-->
     <inertial>
       <origin xyz="-2.0984526232e-09 -1.7951021237e-09 3.6197018104e-02" rpy="0 0 0" />
@@ -457,5 +457,5 @@
     </inertial>
   </link>
-  <joint name="actuator" type="fixed">
+  <joint name="actuator_j" type="fixed">
     <origin xyz="-0.006287977 0.159 -0.0075" rpy="0 1.5708 1.57072" />
     <parent link="rightfinger" />

Commit message: random fixes

File: src/ros/rover/rover_description/waratah_arm/urdf/arm.urdf.xacro (robot description, xacro)
@@ -460,5 +460,5 @@
     <origin xyz="-0.006287977 0.159 -0.0075" rpy="0 1.5708 1.57072" />
     <parent link="rightfinger" />
-    <child link="actuator_frame" />
+    <child link="actuator" />
     <axis xyz="0 0 1" />
   </joint>

Commit message: Integrates pokey action node into the auto typing sequencer. (#554)

File: src/ros/rover/rover_description/waratah_arm/urdf/arm.urdf.xacro (robot description, xacro)
@@ -450,5 +450,5 @@
   <!-- Replace all this with a end effector xacro file that is shared across waratah_arm and banksia_arm-->
   <!-- EEbase to Actuator transform for auto typing -->
-  <link name="actuator_frame"> <!-- Actuator head position when unextended but fingers are fully open-->
+  <link name="actuator"> <!-- Actuator head position when unextended but fingers are fully open-->
     <inertial>
       <origin xyz="-2.0984526232e-09 -1.7951021237e-09 3.6197018104e-02" rpy="0 0 0" />
@@ -457,8 +457,8 @@
     </inertial>
   </link>
-  <joint name="actuator" type="fixed">
+  <joint name="actuator_j" type="fixed">
     <origin xyz="-0.006287977 0.159 -0.0075" rpy="0 1.5708 1.57072" />
     <parent link="rightfinger" />
-    <child link="actuator_frame" />
+    <child link="actuator" />
     <axis xyz="0 0 1" />
   </joint>
