Commit message: add new taipan urdf

File: src/ros/rover/rover_description/taipan/urdf/arm.gz_ros2_control.xacro (robot description, xacro)
@@ -5,5 +5,5 @@
       <plugin>gz_ros2_control/GazeboSimSystem</plugin>
     </hardware>
-    <joint name="J1">
+    <joint name="j1">
 		<command_interface name="velocity">
 		  <param name="max">1</param>
@@ -18,5 +18,5 @@
 		</state_interface>
       </joint>
-	  <joint name="J2">
+	  <joint name="j2">
 		<command_interface name="velocity">
 		  <param name="max">1</param>
@@ -31,5 +31,5 @@
 		</state_interface>
       </joint>
-	  <joint name="J3">
+	  <joint name="j3">
 		<command_interface name="velocity">
 		  <param name="max">1</param>
@@ -44,38 +44,5 @@
 		</state_interface>
       </joint>
-	  <!-- <joint name="l1b_bp">
-		<command_interface name="velocity">
-		  <param name="max">1</param>
-		</command_interface>
-		<state_interface name="velocity">
-		  <param name="initial_value">0.0</param>
-		</state_interface>
-		<state_interface name="position">
-		  <param name="initial_value">0.0</param>
-		</state_interface>
-      </joint>
-	  <joint name="l1b_tp">
-		<command_interface name="velocity">
-		  <param name="max">1</param>
-		</command_interface>
-		<state_interface name="velocity">
-		  <param name="initial_value">0.0</param>
-		</state_interface>
-		<state_interface name="position">
-		  <param name="initial_value">0.0</param>
-		</state_interface>
-      </joint>
-	  <joint name="l1a_tp">
-		<command_interface name="velocity">
-		  <param name="max">1</param>
-		</command_interface>
-		<state_interface name="velocity">
-		  <param name="initial_value">0.0</param>
-		</state_interface>
-		<state_interface name="position">
-		  <param name="initial_value">0.0</param>
-		</state_interface>
-      </joint> -->
-	  <joint name="J4">
+	  <joint name="j4">
 		<command_interface name="velocity">
 		  <param name="max">1</param>
@@ -90,5 +57,5 @@
 		</state_interface>
       </joint>
-	  <joint name="J5">
+	  <joint name="j5">
 		<command_interface name="velocity">
 		  <param name="max">1</param>
@@ -103,5 +70,5 @@
 		</state_interface>
       </joint>
-	  <joint name="J6">
+	  <joint name="j6">
 		<command_interface name="velocity">
 		  <param name="max">1</param>
@@ -116,5 +83,5 @@
 		</state_interface>
       </joint>
-	  <joint name="left_slide">
+	  <joint name="lead_left">
 		<command_interface name="velocity">
 		  <param name="max">1</param>
@@ -129,5 +96,5 @@
 		</state_interface>
       </joint>
-	  <joint name="actuator_head">
+	  <joint name="la_prismatic">
 		<command_interface name="velocity">
 		  <param name="max">1</param>

File: src/ros/rover/rover_description/taipan/urdf/arm.ros2_control.xacro (robot description, xacro)
@@ -35,5 +35,5 @@
 	  </hardware>
 	  -->
-			<joint name="J1">
+			<joint name="j1">
 				<command_interface name="velocity">
 					<param name="max">292.444791137</param>
@@ -78,5 +78,5 @@
 				</hardware>
 			</xacro:if>
-			<joint name="J2">
+			<joint name="j2">
 				<command_interface name="velocity">
 					<param name="max">292.444791137</param>
@@ -120,5 +120,5 @@
 				</hardware>
 			</xacro:if>
-			<joint name="J3">
+			<joint name="j3">
 				<command_interface name="velocity">
 					<param name="max">292.444791137</param>
@@ -162,5 +162,5 @@
 				</hardware>
 			</xacro:if>
-			<joint name="J4">
+			<joint name="j4">
 				<command_interface name="velocity">
 					<param name="max">292.444791137</param>
@@ -204,5 +204,5 @@
 				</hardware>
 			</xacro:if>
-			<joint name="J5">
+			<joint name="j5">
 				<command_interface name="velocity">
 					<param name="max">292.444791137</param>
@@ -247,22 +247,22 @@
 				</hardware>
 			</xacro:if>
-			<joint name="J6">
-				<command_interface name="velocity">
-					<param name="max">292.444791137</param>
-				</command_interface>
-				<command_interface name="position">
-					<param name="max">12.5663706144</param>
-				</command_interface>
-				<state_interface name="velocity">
-					<param name="max">292.444791137</param>
-					<param name="initial_value">0.0</param>
-				</state_interface>
-				<state_interface name="position">
-					<param name="initial_value">0.0</param>
-					<param name="max">12.5663706144</param>
-				</state_interface>
-			</joint>
-		</ros2_control>
-	 <ros2_control name="arm_actuator_head" type="system">
+			<joint name="j6">
+				<command_interface name="velocity">
+					<param name="max">292.444791137</param>
+				</command_interface>
+				<command_interface name="position">
+					<param name="max">12.5663706144</param>
+				</command_interface>
+				<state_interface name="velocity">
+					<param name="max">292.444791137</param>
+					<param name="initial_value">0.0</param>
+				</state_interface>
+				<state_interface name="position">
+					<param name="initial_value">0.0</param>
+					<param name="max">12.5663706144</param>
+				</state_interface>
+			</joint>
+		</ros2_control>
+	 <ros2_control name="arm_la_prismatic" type="system">
 		<xacro:unless value="${use_mock_hardware}">
 			<hardware>
@@ -282,5 +282,5 @@
 			</hardware>
 		</xacro:if>
-		<joint name="actuator_head">
+		<joint name="la_prismatic">
 			<command_interface name="velocity">
 			<param name="max">1</param>
@@ -291,37 +291,5 @@
 		</joint>
 	</ros2_control>
-  <!-- <ros2_control name="arm_right_slide" type="system">
-		<xacro:unless value="${use_mock_hardware}">
-			<hardware>
-				<plugin>cmd_hardware/CMDHardware</plugin>
-				<param name="candevice">can1</param>
-				<param name="canid">0C2</param>
-				<param name="resolver_id">308</param>
-				<param name="resolver_reduction">1.0</param>
-				<param name="reversed">false</param>
-				<param name="reverse_velocity">true</param>
-				<param name="max_velocity">0.365109712045</param>
-				<param name="max_effort">1</param>
-			</hardware>
-		</xacro:unless>
-		<xacro:if value="${use_mock_hardware}">
-			<hardware>
-				<plugin>mock_components/GenericSystem</plugin>
-				<param name="calculate_dynamics">true</param>
-			</hardware>
-		</xacro:if>
-    <joint name="right_slide">
-      <command_interface name="velocity">
-        <param name="max">1</param>
-      </command_interface>
-      <state_interface name="velocity">
-        <param name="initial_value">0.0</param>
-      </state_interface>
-      <state_interface name="position">
-        <param name="initial_value">0.0</param>
-      </state_interface>
-    </joint>
-	</ros2_control> -->
-  <ros2_control name="arm_left_slide" type="system">
+  <ros2_control name="arm_lead_left" type="system">
 		<xacro:unless value="${use_mock_hardware}">
 			<hardware>
@@ -343,5 +311,5 @@
 			</hardware>
 		</xacro:if>
-	  <joint name="left_slide">
+	  <joint name="lead_left">
       <command_interface name="velocity">
         <param name="max">1</param>

File: src/ros/rover/rover_description/taipan/urdf/arm.urdf.xacro (robot description, xacro)
@@ -4,551 +4,5 @@
   xmlns:xacro="http://www.ros.org/wiki/xacro">
   <xacro:arg name="rover_description_dir" default="$(find rover_description)" />
-  <link name="arm_link">
-    <inertial>
-      <origin xyz="0 0 0" rpy="0 0 0" />
-      <mass value="0" />
-      <inertia ixx="0" ixy="0" ixz="0" iyy="0" iyz="0" izz="0" />
-    </inertial>
-  </link>
-  <link name="armmount">
-    <inertial>
-      <origin xyz="1.0026735487e-01 6.7184838502e-02 1.0892448810e-01" rpy="0 0 0" />
-      <mass value="2.89989" />
-      <inertia ixx="4.9625273465e-02" ixy="-5.5273266406e-07" ixz="-1.7120308592e-03" iyy="3.1308984541e-02" iyz="1.0530224090e-06" izz="5.6564003946e-02" />
-    </inertial>
-    <visual>
-      <origin xyz="-0.0671788 0.129712 -0.183721" rpy="-1.88173e-16 -1.99729e-09 -1.5708" />
-      <geometry>
-        <mesh filename="file://$(arg rover_description_dir)/taipan/meshes/armmount.stl" />
-      </geometry>
-      <material name="armmount_material">
-        <color rgba="0.866667 0.0745098 0.32549 1.0" />
-      </material>
-    </visual>
-    <collision>
-      <origin xyz="0 0 -0.085" rpy="0 0 0" />
-      <geometry>
-        <box size="0.34 0.27 0.19"/>
-      </geometry>
-    </collision>
-  </link>
-  <link name="gearbox">
-    <inertial>
-      <origin xyz="1.5517995279e-06 -1.5436967725e-05 2.9196698911e-02" rpy="0 0 0" />
-      <mass value="1.14385" />
-      <inertia ixx="1.6613733657e-03" ixy="-2.7401017167e-11" ixz="2.3220558636e-08" iyy="1.6613736356e-03" iyz="-2.1472923963e-07" izz="2.6570870533e-03" />
-    </inertial>
-    <visual>
-      <origin xyz="-9.93063e-18 0 5.55112e-17" rpy="3.14159 -0 -7.70285e-39" />
-      <geometry>
-        <mesh filename="file://$(arg rover_description_dir)/taipan/meshes/gearbox.stl" />
-      </geometry>
-      <material name="gearbox_material">
-        <color rgba="0.866667 0.0745098 0.32549 1.0" />
-      </material>
-    </visual>
-  </link>
-  <link name="linkagedrive">
-    <inertial>
-      <origin xyz="-1.2655758715e-03 4.4726798551e-03 9.3524916551e-02" rpy="0 0 0" />
-      <mass value="3.93358" />
-      <inertia ixx="1.5664196707e-02" ixy="3.0028427663e-04" ixz="-2.1300499897e-04" iyy="3.4406324873e-02" iyz="7.6758448878e-04" izz="2.7092109586e-02" />
-    </inertial>
-    <visual>
-      <origin xyz="-1.58901e-15 -1.36391e-16 -5.55112e-17" rpy="6.68673e-23 -1.0222e-22 2.39693e-07" />
-      <geometry>
-        <mesh filename="file://$(arg rover_description_dir)/taipan/meshes/linkagedrive.stl" />
-      </geometry>
-      <material name="linkagedrive_material">
-        <color rgba="0.866667 0.0745098 0.32549 1.0" />
-      </material>
-    </visual>
-    <collision>
-      <origin xyz="0 0 0.065" rpy="0 0 0" />
-      <geometry>
-        <box size="0.17 0.13 0.13"/>
-      </geometry>
-    </collision>
-    <collision>
-      <origin xyz="0 0 0.13" rpy="0 1.5708 0" />
-      <geometry>
-        <cylinder length="0.33" radius="0.065"/>
-      </geometry>
-    </collision>
-  </link>
-  <link name="l1">
-    <inertial>
-      <origin xyz="9.8617717772e-05 -2.5902167046e-04 2.6363294133e-01" rpy="0 0 0" />
-      <mass value="1.03818" />
-      <inertia ixx="3.4637121821e-02" ixy="2.7028859609e-08" ixz="2.9471387302e-05" iyy="3.5662964589e-02" iyz="-2.3126360649e-07" izz="1.4733017478e-03" />
-    </inertial>
-    <visual>
-      <origin xyz="3.1979e-15 -6.85563e-15 0.0239" rpy="1.5708 1.5708 0" />
-      <geometry>
-        <mesh filename="file://$(arg rover_description_dir)/taipan/meshes/l1.stl" />
-      </geometry>
-      <material name="l1_material">
-        <color rgba="0.866667 0.0745098 0.32549 1.0" />
-      </material>
-    </visual>
-    <collision>
-      <origin xyz="0 -0.255 0.024" rpy="0 0 0" />
-      <geometry>
-        <box size="0.043 0.53 0.1125"/>
-      </geometry>
-    </collision>
-  </link>
-  <link name="l2">
-    <inertial>
-      <origin xyz="3.9958382695e-03 -2.0455304076e-01 3.4576652668e-01" rpy="0 0 0" />
-      <mass value="1.28299" />
-      <inertia ixx="1.2195242198e-02" ixy="6.2402565899e-04" ixz="4.7783495683e-04" iyy="6.1811297654e-03" iyz="-5.5062214849e-03" izz="9.1557193257e-03" />
-    </inertial>
-    <visual>
-      <origin xyz="0.398641 0.301803 6.48063e-16" rpy="2.49358 1.5708 0" />
-      <geometry>
-        <mesh filename="file://$(arg rover_description_dir)/taipan/meshes/l2.stl" />
-      </geometry>
-      <material name="l2_material">
-        <color rgba="0.866667 0.0745098 0.32549 1.0" />
-      </material>
-    </visual>
-    <collision>
-      <origin xyz="0 0.11 0" rpy="0 0 0" />
-      <geometry>
-        <box size="0.04 0.44 0.028"/>
-      </geometry>
-    </collision>
-    <collision>
-      <origin xyz="0 0.33 0.0065" rpy="0 0 0" />
-      <geometry>
-        <box size="0.026 0.013 0.123"/>
-      </geometry>
-    </collision>
-    <collision>
-      <origin xyz="0 0.379 0.065" rpy="0 0 0" />
-      <geometry>
-        <box size="0.026 0.11 0.01"/>
-      </geometry>
-    </collision>
-    <collision>
-      <origin xyz="0 0.379 -0.05" rpy="0 0 0" />
-      <geometry>
-        <box size="0.026 0.11 0.01"/>
-      </geometry>
-    </collision>
-    <collision>
-      <origin xyz="0 0.349 -0.072" rpy="0 0 0" />
-      <geometry>
-        <box size="0.041 0.185 0.03"/>
-      </geometry>
-    </collision>
-    <collision>
-      <origin xyz="0 0.3635 -0.072" rpy="0 0 0" />
-      <geometry>
-        <box size="0.07 0.02 0.03"/>
-      </geometry>
-    </collision>
-    <collision>
-      <origin xyz="0 0.275 -0.0025" rpy="0 0 0" />
-      <geometry>
-        <cylinder length="0.082" radius="0.045"/>
-      </geometry>
-    </collision>
-  </link>
-  <link name="j5">
-    <inertial>
-      <origin xyz="1.6304453499e-04 1.3310885204e-04 4.9429943641e-02" rpy="0 0 0" />
-      <mass value="0.632837" />
-      <inertia ixx="4.2793037045e-04" ixy="-2.8799099692e-06" ixz="-1.2787619925e-06" iyy="5.5653102600e-04" iyz="5.1247237439e-06" izz="7.8687161656e-04" />
-    </inertial>
-    <visual>
-      <origin xyz="1.94289e-15 0.05075 -0.0795" rpy="1.5708 1.5708 0" />
-      <geometry>
-        <mesh filename="file://$(arg rover_description_dir)/taipan/meshes/j5.stl" />
-      </geometry>
-      <material name="j5_material">
-        <color rgba="0.866667 0.0745098 0.32549 1.0" />
-      </material>
-    </visual>
-  </link>
-  <link name="j6">
-    <inertial>
-      <origin xyz="1.1883033288e-04 4.2174023459e-04 4.5350143681e-02" rpy="0 0 0" />
-      <mass value="0.768628" />
-      <inertia ixx="1.9985920161e-03" ixy="-1.6005592251e-07" ixz="4.0364224668e-07" iyy="1.4889297725e-03" iyz="-8.2877165939e-06" izz="1.0636569880e-03" />
-    </inertial>
-    <visual>
-      <origin xyz="5.80265e-16 -0.1945 0.05075" rpy="-1.5708 -1.48145e-14 -7.47144e-23" />
-      <geometry>
-        <mesh filename="file://$(arg rover_description_dir)/taipan/meshes/j6.stl" />
-      </geometry>
-      <material name="j6_material">
-        <color rgba="0.866667 0.0745098 0.32549 1.0" />
-      </material>
-    </visual>
-    <collision>
-      <origin xyz="0 -0.09 0.1" rpy="0 0 0" />
-      <geometry>
-        <box size="0.06 0.2 0.01"/>
-      </geometry>
-    </collision>
-    <collision>
-      <origin xyz="0 -0.09 0" rpy="0 0 0" />
-      <geometry>
-        <box size="0.06 0.2 0.01"/>
-      </geometry>
-    </collision>
-    <collision>
-      <origin xyz="0 -0.145 0.05" rpy="0 0 0" />
-      <geometry>
-        <box size="0.06 0.09 0.1"/>
-      </geometry>
-    </collision>
-    <collision>
-      <origin xyz="0 -0.169 0.05" rpy="1.5708 0 0" />
-      <geometry>
-        <cylinder length="0.025" radius="0.045"/>
-      </geometry>
-    </collision>
-  </link>
-  <link name="eebase">
-    <inertial>
-      <origin xyz="4.2518858921e-02 -1.3680332624e-02 5.1489918726e-02" rpy="0 0 0" />
-      <mass value="0.964685" />
-      <inertia ixx="3.9819443378e-03" ixy="-7.7314319464e-05" ixz="2.7737204681e-04" iyy="7.8827897449e-03" iyz="1.4686739679e-03" izz="6.8055990755e-03" />
-    </inertial>
-    <visual>
-      <origin xyz="0.00775 0.013 0.0215" rpy="-6.15694e-07 4.61983e-15 3.14159" />
-      <geometry>
-        <mesh filename="file://$(arg rover_description_dir)/taipan/meshes/eebase.stl" />
-      </geometry>
-      <material name="eebase_material">
-        <color rgba="0.866667 0.0745098 0.32549 1.0" />
-      </material>
-    </visual>
-    <collision>
-      <origin xyz="0 0.02 0.0675" rpy="0 0 0" />
-      <geometry>
-        <box size="0.25 0.08 0.075"/>
-      </geometry>
-    </collision>
-  </link>
-  <link name="rightfinger">
-    <inertial>
-      <origin xyz="1.8050558411e-05 7.3968039193e-03 2.8621961810e-02" rpy="0 0 0" />
-      <mass value="0.299805" />
-      <inertia ixx="1.1544859455e-03" ixy="3.3371529469e-07" ixz="-2.2265830694e-07" iyy="2.2126179923e-04" iyz="1.4057271751e-04" izz="1.0316786208e-03" />
-    </inertial>
-    <visual>
-      <origin xyz="-3.64856e-05 0.115305 0.0109" rpy="-3.14159 -6.60532e-30 2.57948e-23" />
-      <geometry>
-        <mesh filename="file://$(arg rover_description_dir)/taipan/meshes/rightfinger.stl" />
-      </geometry>
-      <material name="rightfinger_material">
-        <color rgba="0.866667 0.0745098 0.32549 1.0" />
-      </material>
-    </visual>
-  </link>
-  <link name="arm_end_side_optical">
-    <inertial>
-      <origin xyz="5.0388580281e-20 -5.0000002375e-04 -2.0596424901e-20" rpy="0 0 0" />
-      <mass value="1e-09" />
-      <inertia ixx="6.3254056983e-15" ixy="-1.2661721154e-31" ixz="-1.4456719139e-31" iyy="1.2484144714e-14" iyz="7.0639301518e-32" izz="6.3254056983e-15" />
-    </inertial>
-    <visual>
-      <origin xyz="0 0 0" rpy="1.5708 1.86776e-19 -2.0576e-24" />
-      <geometry>
-        <mesh filename="file://$(arg rover_description_dir)/taipan/meshes/arm_end_side.stl" />
-      </geometry>
-      <material name="arm_end_side_material">
-        <color rgba="0.866667 0.0745098 0.32549 1.0" />
-      </material>
-    </visual>
-  </link>
-  <joint name="camera_ee_side" type="fixed">
-    <origin xyz="-0.000216235 0.178108 -0.0547417" rpy="0 0.00174763 3.14159" />
-    <parent link="rightfinger" />
-    <child link="arm_end_side_optical" />
-    <axis xyz="0 0 1" />
-    <limit effort="10" velocity="10" />
-  </joint>
-  <joint name="right_slide" type="prismatic">
-    <origin xyz="-0.0953625 -2.37042e-08 0.0635" rpy="1.5708 -6.15694e-07 1.5708" />
-    <parent link="eebase" />
-    <child link="rightfinger" />
-    <axis xyz="0 0 1" />
-    <limit effort="10" velocity="10" lower="0" upper="0.084" />
-    <mimic joint="left_slide" multiplier="1" offset="0"/>
-  </joint>
-  <link name="leftfinger">
-    <inertial>
-      <origin xyz="-3.0820093691e-05 -2.4076955607e-02 1.7779582954e-02" rpy="0 0 0" />
-      <mass value="0.259097" />
-      <inertia ixx="8.0113158332e-04" ixy="-2.1276248523e-07" ixz="1.9237282265e-07" iyy="7.8712513524e-05" iyz="5.1221559668e-05" izz="8.1168195146e-04" />
-    </inertial>
-    <visual>
-      <origin xyz="-8.71485e-06 -0.115251 0.0109" rpy="-3.14159 4.996e-15 -5.80744e-23" />
-      <geometry>
-        <mesh filename="file://$(arg rover_description_dir)/taipan/meshes/leftfinger.stl" />
-      </geometry>
-      <material name="leftfinger_material">
-        <color rgba="0.866667 0.0745098 0.32549 1.0" />
-      </material>
-    </visual>
-  </link>
-  <link name="actuator">
-    <inertial>
-      <origin xyz="-2.0984526232e-09 -1.7951021237e-09 3.6197018104e-02" rpy="0 0 0" />
-      <mass value="0.00499493" />
-      <inertia ixx="1.9746052847e-06" ixy="3.2584721895e-14" ixz="3.1261224204e-13" iyy="1.9775524756e-06" iyz="2.6609843251e-13" izz="7.2954357931e-08" />
-    </inertial>
-    <visual>
-      <origin xyz="-1.38778e-17 0 -0.058" rpy="3.11287e-20 2.12505e-23 1.99292e-27" />
-      <geometry>
-        <mesh filename="file://$(arg rover_description_dir)/taipan/meshes/actuator.stl" />
-      </geometry>
-      <material name="actuator_material">
-        <color rgba="0.866667 0.0745098 0.32549 1.0" />
-      </material>
-    </visual>
-  </link>
-  <joint name="actuator_head" type="prismatic">
-    <origin xyz="-1.2023e-05 -0.159 -0.0075" rpy="1.57072 -1.5708 0" />
-    <parent link="leftfinger" />
-    <child link="actuator" />
-    <axis xyz="0 0 1" />
-    <limit effort="10" velocity="10" lower="-1.22125e-15" upper="0.055" />
-  </joint>
-  <link name="arm_end_finger_optical">
-    <inertial>
-      <origin xyz="5.0388580281e-20 -5.0000002375e-04 -2.0596424901e-20" rpy="0 0 0" />
-      <mass value="1e-09" />
-      <inertia ixx="6.3254056983e-15" ixy="-1.2661721154e-31" ixz="-1.4456719139e-31" iyy="1.2484144714e-14" iyz="7.0639301518e-32" izz="6.3254056983e-15" />
-    </inertial>
-    <visual>
-      <origin xyz="2.77556e-17 0 -1.11022e-16" rpy="1.5708 -2.87448e-18 1.5822e-23" />
-      <geometry>
-        <mesh filename="file://$(arg rover_description_dir)/taipan/meshes/arm_end_finger.stl" />
-      </geometry>
-      <material name="arm_end_finger_material">
-        <color rgba="0.866667 0.0745098 0.32549 1.0" />
-      </material>
-    </visual>
-  </link>
-  <joint name="camera_ee_finger" type="fixed">
-    <origin xyz="1.96205e-05 -0.0711415 -0.0299814" rpy="-3.14152 ${radians(180) + 1.52166} -1.5708" />
-    <parent link="leftfinger" />
-    <child link="arm_end_finger_optical" />
-    <axis xyz="0 0 1" />
-    <limit effort="10" velocity="10" />
-  </joint>
-  <joint name="left_slide" type="prismatic">
-    <origin xyz="0.0951 -2.37042e-08 0.0635" rpy="-1.5708 -6.15694e-07 1.5708" />
-    <parent link="eebase" />
-    <child link="leftfinger" />
-    <axis xyz="0 0 1" />
-    <limit effort="10" velocity="10" lower="0" upper="0.084" />
-  </joint>
-  <link name="arm_end_top_optical">
-    <inertial>
-      <origin xyz="5.0388580281e-20 -5.0000002375e-04 -2.0596424901e-20" rpy="0 0 0" />
-      <mass value="1e-09" />
-      <inertia ixx="6.3254056983e-15" ixy="-1.2661721154e-31" ixz="-1.4456719139e-31" iyy="1.2484144714e-14" iyz="7.0639301518e-32" izz="6.3254056983e-15" />
-    </inertial>
-    <visual>
-      <origin xyz="1.11022e-16 0 0" rpy="1.5708 -2.5589e-20 3.89707e-23" />
-      <geometry>
-        <mesh filename="file://$(arg rover_description_dir)/taipan/meshes/arm_end_top.stl" />
-      </geometry>
-      <material name="arm_end_top_material">
-        <color rgba="0.866667 0.0745098 0.32549 1.0" />
-      </material>
-    </visual>
-  </link>
-  <joint name="camera_ee_top" type="fixed">
-    <origin xyz="-6.33269e-14 0.10042 0.231753" rpy="1.5708 ${-1.56853 - radians(90)} 0" />
-    <parent link="eebase" />
-    <child link="arm_end_top_optical" />
-    <axis xyz="0 0 1" />
-    <limit effort="10" velocity="10" />
-  </joint>
-  <link name="arm_end_periscope_optical">
-    <inertial>
-      <origin xyz="5.0388580281e-20 -5.0000002375e-04 -2.0596424901e-20" rpy="0 0 0" />
-      <mass value="1e-09" />
-      <inertia ixx="6.3254056983e-15" ixy="-1.2661721154e-31" ixz="-1.4456719139e-31" iyy="1.2484144714e-14" iyz="7.0639301518e-32" izz="6.3254056983e-15" />
-    </inertial>
-    <visual>
-      <origin xyz="0 0 0" rpy="1.5708 -1.12386e-23 -2.15772e-29" />
-      <geometry>
-        <mesh filename="file://$(arg rover_description_dir)/taipan/meshes/arm_end_periscope.stl" />
-      </geometry>
-      <material name="arm_end_periscope_material">
-        <color rgba="0.866667 0.0745098 0.32549 1.0" />
-      </material>
-    </visual>
-  </link>
-  <joint name="camera_ee_periscope" type="fixed">
-     <origin xyz="-0.00015 -0.0378336 0.0594947" rpy="-3.14159 -3.14159 0" />
-    <parent link="eebase" />
-    <child link="arm_end_periscope_optical" />
-    <axis xyz="0 0 1" />
-    <limit effort="10" velocity="10" />
-  </joint>
-  <joint name="J6" type="revolute">
-    <origin xyz="5.64652e-16 -0.1945 0.05075" rpy="1.5708 -1.48145e-14 2.12503e-17" />
-    <parent link="j6" />
-    <child link="eebase" />
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