Commit message: add new taipan urdf

File: src/ros/rover/rover_description/taipan/urdf/arm_joints.xacro (robot description, xacro)
@@ -6,16 +6,16 @@
                <topic>joint_states</topic>
                <joint_name>arm_kinematics_origin_joint</joint_name>
-               <joint_name>J1</joint_name>
-               <joint_name>J2</joint_name>
-               <joint_name>J3</joint_name>
-               <joint_name>l1b_bp</joint_name>
-               <joint_name>l1b_tp</joint_name>
-               <joint_name>l1a_tp</joint_name>
-               <joint_name>J4</joint_name>
-               <joint_name>J5</joint_name>
-               <joint_name>J6</joint_name>
-               <joint_name>left_slide</joint_name>
-               <joint_name>right_slide</joint_name>
-               <joint_name>actuator_head</joint_name>
+               <joint_name>j1</joint_name>
+               <joint_name>j2</joint_name>
+               <joint_name>j3</joint_name>
+               <joint_name>l1_p_lower</joint_name>
+               <joint_name>l1_p_upper</joint_name>
+               <joint_name>l1_l2_pivot</joint_name>
+               <joint_name>j4</joint_name>
+               <joint_name>j5</joint_name>
+               <joint_name>j6</joint_name>
+               <joint_name>lead_left</joint_name>
+               <joint_name>lead_right</joint_name>
+               <joint_name>la_prismatic</joint_name>
           </plugin>
      </gazebo>

File: src/ros/rover/rover_description/taipan/urdf/joint_states_with_arm.xacro (robot description, xacro)
@@ -30,15 +30,15 @@
             <joint_name>br_ball_yaw</joint_name>
             <!-- Arm joints -->
-            <joint_name>J1</joint_name>
-            <joint_name>J2</joint_name>
-            <joint_name>J3</joint_name>
-            <joint_name>l1b_bp</joint_name>
-            <joint_name>l1b_tp</joint_name>
-            <joint_name>l1a_tp</joint_name>
-            <joint_name>J4</joint_name>
-            <joint_name>J5</joint_name>
-            <joint_name>J6</joint_name>
-            <joint_name>left_slide</joint_name>
-            <joint_name>actuator_head</joint_name>
+            <joint_name>j1</joint_name>
+            <joint_name>j2</joint_name>
+            <joint_name>j3</joint_name>
+            <joint_name>l1_p_lower</joint_name>
+            <joint_name>l1_p_upper</joint_name>
+            <joint_name>l1_l2_pivot</joint_name>
+            <joint_name>j4</joint_name>
+            <joint_name>j5</joint_name>
+            <joint_name>j6</joint_name>
+            <joint_name>lead_left</joint_name>
+            <joint_name>la_prismatic</joint_name>
         </plugin>
     </gazebo>
