Commit message: fix some small bugs

File: src/ros/rover/rover_description/taipan/urdf/arm.urdf (robot description, URDF)
Before this commit: robot Arm, 17 links, 13 joints
Joints:
- added joint l1_l2_pivot_mimic: type revolute, parent l1_l2_pivot_j2_mimic, child l2, origin xyz=0 0 0 rpy=0 0 0, axis 0 0 1, limit lower=-3.141592653589793 upper=3.141592653589793 effort=10 velocity=10, mimic joint=j2 multiplier=-1 offset=0
- added joint l1_p_lower_mimic: type revolute, parent l1_p_lower_j3_mimic, child l1_prime_fake, origin xyz=0 0 0 rpy=0 0 0, axis 0 0 1, limit lower=-3.141592653589793 upper=3.141592653589793 effort=10 velocity=10, mimic joint=j3 multiplier=-1 offset=0
- added joint l1_p_upper_mimic: type revolute, parent l1_p_upper_j3_mimic, child l1_prime, origin xyz=0 0 0 rpy=0 0 0, axis 0 0 1, limit lower=-3.141592653589793 upper=3.141592653589793 effort=10 velocity=10, mimic joint=j3 multiplier=1 offset=0
- joint l1_l2_pivot: child l2 -> l1_l2_pivot_j2_mimic; mimic joint=j2 multiplier=-1 offset=0 -> joint=j3 multiplier=1 offset=0; origin xyz=0 0 0 rpy=0 0 0 -> xyz=-2.18226e-15 0.5 -0.0457 rpy=-3.14159 2.98806e-14 -1.5708; parent l1_l2_pivot_j2_mimic -> l1
- joint l1_p_lower: child l1_prime_fake -> l1_p_lower_j3_mimic; mimic joint=j3 multiplier=-1 offset=0 -> joint=j2 multiplier=1 offset=0; origin xyz=0 0 0 rpy=0 0 0 -> xyz=0.1 -2.77556e-17 0 rpy=-3.14159 1.22432e-16 1.5708
- joint l1_p_upper: child l1_prime -> l1_p_upper_j3_mimic; mimic joint=j3 multiplier=1 offset=0 -> joint=j2 multiplier=-1 offset=0; origin xyz=0 0 0 rpy=0 0 0 -> xyz=1.87628e-14 -0.1 0.006 rpy=3.14159 -2.86493e-15 -1.5708; parent l1_p_upper_j2_mimic -> l2

File: src/ros/rover/rover_description/taipan/urdf/arm.urdf.xacro (robot description, xacro)
@@ -6,9 +6,10 @@
   <xacro:include filename="$(arg rover_description_dir)/taipan/urdf/arm.urdf"/>
   <!-- Kinematics -->
+  <!-- THESE NEED FIXING 4/02/2026 !!! -->
   <!-- Origin of arm for IK. Should align with J1, but not -->
   <link name="arm_kinematics_origin"/>
   <joint name="arm_kinematics_origin_joint" type="fixed">
     <origin xyz="0.0 0.0 0.196" rpy="0.0 0.0 -1.57079632679" />
-    <parent link="armmount" />
+    <parent link="arm_link" />
     <child link="arm_kinematics_origin" />
   </joint>
@@ -18,5 +19,5 @@
     <!-- before rotating to match IK function expected 0: 1.5707963 0.0 1.5707963 -->
     <origin xyz="0.0067503 -0.0012 0.2225" rpy="-1.57079632679 -1.57079632679 0.0" />
-    <parent link="eebase" />
+    <parent link="ee_base" />
     <child link="endeffector_kinematics" />
   </joint>

Commit message: fix l2 prime

File: src/ros/rover/rover_description/taipan/urdf/arm.urdf (robot description, URDF)
Before this commit: robot Arm, 17 links, 16 joints
Joints:
- joint l1_l2_pivot: mimic joint=j3 multiplier=1 offset=0 -> joint=j3 multiplier=-1 offset=0
- joint l1_p_lower_mimic: mimic joint=j3 multiplier=-1 offset=0 -> joint=j3 multiplier=1 offset=0
- joint l1_p_upper_mimic: mimic joint=j3 multiplier=1 offset=0 -> joint=j3 multiplier=-1 offset=0

Commit message: fix 4 bar linkage mimics

File: src/ros/rover/rover_description/taipan/urdf/arm.urdf (robot description, URDF)
Before this commit: robot Arm, 18 links, 14 joints
Joints:
- joint l1_l2_pivot_mimic: mimic joint=j2 multiplier=-1 offset=0 -> joint=j2 multiplier=1 offset=0
- joint l1_p_upper: mimic joint=j2 multiplier=-1 offset=0 -> joint=j2 multiplier=1 offset=0
- joint l2_p_j2_mimic: mimic joint=j2 multiplier=2 offset=0 -> joint=j2 multiplier=0 offset=0

Commit message: taipan: limits
i was able to get it stuck with l2' and l1' colliding and it not letting
me move away from that collision but i changed the boxes a bit and
didn't get it again so idk if its still an issue.

blcmd_hardware: ensure pitch commands are same direction as feedback
nova_arm_controller: pramaterise if we collect position/velocity
feedback
arm_bringup: reenable position and collision limits for nova arm
controller
rover_description: taipan: add collider for l2', extend collider for l1'
teleop_arm: swap wrist pitch direction as I think the change to blcmd
hardware will have swapped it.

File: src/ros/rover/rover_description/taipan/urdf/arm.urdf (robot description, URDF)
Before this commit: robot Arm, 18 links, 16 joints
Links:
- link l1_prime: geometry collision box size=0.019 0.41 0.019; visual mesh filename=file://$(arg rover_description_dir)/taipan/meshes/elbow_joi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
- link l2_prime: geometry collision box size=0.17 0.03 0.05; visual mesh filename=file://$(arg rover_description_dir)/taipan/meshes/base_cam_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
Joints:
- joint j5: origin xyz=0.04071 -4.09672e-14 -0.45 rpy=1.5708 -0.611293 1.5708 -> xyz=0.04071 -4.09672e-14 -0.45 rpy=1.5708 -1.5708 1.5708

Commit message: position limits for 4 bar linkage
Ended up very sloppy implementation but there are params to
enable/disable it and change the limits.

This means that it won't let you crunch the 4 bar linkage as it limits
the angle j2-j3 which controls the angle of the two joints of L1' that
can crunch.

Self collision limits didn't work well for this as it would get stuck
in the collider, but with this implementation it knows that moving from
an illegal position closer to a legal position is ok so it doesn't get
stuck.

It may still be able to get stuck in the collider tho

File: src/ros/rover/rover_description/taipan/urdf/arm.urdf (robot description, URDF)
Before this commit: robot Arm, 18 links, 16 joints
Links:
- link l1_prime: geometry collision box size=0.019 0.51 0.019; visual mesh filename=file://$(arg rover_description_dir)/taipan/meshes/elbow_joi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

Commit message: urdf tipan
remove l2' collider. The position limit for J3 ensures that l2 does not
hit the base. The 4 bar limit ensures it does not hit l1', so it does
not need the manually added collider anymore

shorted l1' collider a bit so that it doesn't hit arm base (it
physically cannot do this)

File: src/ros/rover/rover_description/taipan/urdf/arm.urdf (robot description, URDF)
Before this commit: robot Arm, 18 links, 16 joints
Links:
- link l1_prime: geometry collision box size=0.019 0.45 0.019; visual mesh filename=file://$(arg rover_description_dir)/taipan/meshes/elbow_joi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
- link l2_prime: geometry visual mesh filename=file://$(arg rover_description_dir)/taipan/meshes/base_cam_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

Commit message: taipan: limits (#946)
Co-authored-by: Jackson <83764855+jacksonmacc@users.noreply.github.com>

File: src/ros/rover/rover_description/taipan/urdf/arm.urdf (robot description, URDF)
Before this commit: robot Arm, 18 links, 16 joints
Links:
- link l1_prime: geometry collision box size=0.019 0.45 0.019; visual mesh filename=file://$(arg rover_description_dir)/taipan/meshes/elbow_joi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
Joints:
- joint j5: origin xyz=0.04071 -4.09672e-14 -0.45 rpy=1.5708 -0.611293 1.5708 -> xyz=0.04071 -4.09672e-14 -0.45 rpy=1.5708 -1.5708 1.5708

Commit message: arm fixes
remind me to put this on a seperate branch

File: src/ros/rover/rover_description/taipan/urdf/arm.urdf (robot description, URDF)
Before this commit: robot Arm, 18 links, 16 joints
Joints:
- joint j6: axis 0 0 1 -> 0 0 -1

Commit message: fix: better error message for mimic joints with a multiplier of 0

File: src/ros/rover/rover_description/taipan/urdf/arm.urdf (robot description, URDF)
Before this commit: robot Arm, 18 links, 16 joints
Joints:
- joint l2_p_j2_mimic: axis 0 0 1 -> (none); limit lower=-3.141592653589793 upper=3.141592653589793 effort=10 velocity=10 -> (none); mimic joint=j2 multiplier=0 offset=0 -> (none); type revolute -> fixed
