Commit message: made end effector joints fixed when running mock hardware

File: src/ros/rover/rover_description/taipan/urdf/arm.ros2_control.xacro (robot description, xacro)
@@ -264,33 +264,33 @@
 			</joint>
 		</ros2_control>
-	 <ros2_control name="arm_la_prismatic" type="system">
 		<xacro:unless value="${use_mock_hardware}">
-			<hardware>
-				<plugin>qcmd_hardware/QCMDHardware</plugin>
-				<param name="candevice">can1</param>
-				<param name="canid">0C1</param> <!-- TODO: Get CAN id, resolver id should be that *4 -->
-				<!-- <param name="reversed">false</param> -->
-				<!-- <param name="reverse_velocity">true</param> -->
-				<!-- <param name="max_velocity">0.365109712045</param> -->
-				<param name="max_effort">1</param>
-			</hardware>
+			<ros2_control name="arm_la_prismatic" type="system">
+					<hardware>
+						<plugin>qcmd_hardware/QCMDHardware</plugin>
+						<param name="candevice">can1</param>
+						<param name="canid">0C1</param> <!-- TODO: Get CAN id, resolver id should be that *4 -->
+						<!-- <param name="reversed">false</param> -->
+						<!-- <param name="reverse_velocity">true</param> -->
+						<!-- <param name="max_velocity">0.365109712045</param> -->
+						<param name="max_effort">1</param>
+					</hardware>
+				<xacro:if value="${use_mock_hardware}">
+					<hardware>
+						<plugin>mock_components/GenericSystem</plugin>
+						<param name="calculate_dynamics">true</param>
+					</hardware>
+				</xacro:if>
+				<joint name="la_prismatic">
+					<command_interface name="velocity">
+					<param name="max">1</param>
+					</command_interface>
+					<state_interface name="velocity">
+					<param name="initial_value">0.0</param>
+					</state_interface>
+				</joint>
+			</ros2_control>
 		</xacro:unless>
-		<xacro:if value="${use_mock_hardware}">
-			<hardware>
-				<plugin>mock_components/GenericSystem</plugin>
-				<param name="calculate_dynamics">true</param>
-			</hardware>
-		</xacro:if>
-		<joint name="la_prismatic">
-			<command_interface name="velocity">
-			<param name="max">1</param>
-			</command_interface>
-			<state_interface name="velocity">
-			<param name="initial_value">0.0</param>
-			</state_interface>
-		</joint>
-	</ros2_control>
-  <ros2_control name="arm_lead_left" type="system">
-		<xacro:unless value="${use_mock_hardware}">
+	<xacro:unless value="${use_mock_hardware}">
+		<ros2_control name="arm_lead_left" type="system">
 			<hardware>
 				<plugin>qcmd_hardware/QCMDHardware</plugin>
@@ -304,20 +304,20 @@
 				<param name="max_effort">1</param>
 			</hardware>
-		</xacro:unless>
-		<xacro:if value="${use_mock_hardware}">
-			<hardware>
-				<plugin>mock_components/GenericSystem</plugin>
-				<param name="calculate_dynamics">true</param>
-			</hardware>
-		</xacro:if>
-	  <joint name="lead_left">
-      <command_interface name="velocity">
-        <param name="max">1</param>
-      </command_interface>
-      <state_interface name="velocity">
-        <param name="initial_value">0.0</param>
-      </state_interface>
-    </joint>
-	</ros2_control>
+			<xacro:if value="${use_mock_hardware}">
+				<hardware>
+					<plugin>mock_components/GenericSystem</plugin>
+					<param name="calculate_dynamics">true</param>
+				</hardware>
+			</xacro:if>
+			<joint name="lead_left">
+				<command_interface name="velocity">
+					<param name="max">1</param>
+				</command_interface>
+				<state_interface name="velocity">
+					<param name="initial_value">0.0</param>
+				</state_interface>
+			</joint>
+		</ros2_control>
+	</xacro:unless>
 	</xacro:macro>
 </robot>

File: src/ros/rover/rover_description/taipan/urdf/arm.urdf (robot description, URDF)
Before this commit: robot Arm, 17 links, 16 joints
Links:
- added link ee_base_l2_prime_mimic
Joints:
- added joint l2_p_j2_mimic: type revolute, parent base_frame, child ee_base_l2_prime_mimic, origin xyz=0.006 -9.18923e-17 0.131 rpy=1.5708 7.26102e-16 1.5708, axis 0 0 1, limit lower=-3.141592653589793 upper=3.141592653589793 effort=10 velocity=10, mimic joint=j2 multiplier=2 offset=0
- joint j3: origin xyz=0.006 -9.18923e-17 0.131 rpy=1.5708 7.26102e-16 1.5708 -> (none); parent base_frame -> ee_base_l2_prime_mimic
- joint la_prismatic: type prismatic -> fixed
- joint lead_left: type prismatic -> fixed
- joint lead_right: mimic joint=lead_left multiplier=1 offset=0 -> (none); type prismatic -> fixed

File: src/ros/rover/rover_description/taipan/urdf/arm_joints.xacro (robot description, xacro)
@@ -15,7 +15,9 @@
                <joint_name>j5</joint_name>
                <joint_name>j6</joint_name>
-               <joint_name>lead_left</joint_name>
-               <joint_name>lead_right</joint_name>
-               <joint_name>la_prismatic</joint_name>
+		     <xacro:unless value="${use_mock_hardware}">
+                    <joint_name>lead_left</joint_name>
+                    <joint_name>lead_right</joint_name>
+                    <joint_name>la_prismatic</joint_name>
+               </xacro:unless>
           </plugin>
      </gazebo>

Commit message: updated blcmd hardware to take lists of canids

File: src/ros/rover/rover_description/taipan/urdf/arm.ros2_control.xacro (robot description, xacro)
@@ -179,10 +179,10 @@
 			</joint>
 		</ros2_control>
-		<ros2_control name="arm_J5" type="system">
-			<xacro:unless value="${use_mock_hardware}">
-				<hardware>
-					<plugin>blcmd_hardware2/BLCMDHardware</plugin>
-					<param name="candevice">can1</param>
-					<param name="canid">5</param>
+		<ros2_control name="arm_diff_wrist" type="system">
+			<xacro:unless value="${use_mock_hardware}">
+				<hardware>
+					<plugin>blcmd_hardware2/BLCMDHardware</plugin>
+					<param name="candevice">can1</param>
+					<param name="canid">5 6</param>
 					<param name="resolver_reduction">1.0</param>
 					<param name="clock_rate">100000000</param>
@@ -220,6 +220,71 @@
 				</state_interface>
 			</joint>
-		</ros2_control>
-		<ros2_control name="arm_J6" type="system">
+			<joint name="j6">
+				<command_interface name="velocity">
+					<param name="max">292.444791137</param>
+				</command_interface>
+				<command_interface name="position">
+					<param name="max">12.5663706144</param>
+				</command_interface>
+				<state_interface name="velocity">
+					<param name="max">292.444791137</param>
+					<param name="initial_value">0.0</param>
+				</state_interface>
+				<state_interface name="position">
+					<param name="max">12.5663706144</param>
+					<param name="initial_value">0.0</param>
+				</state_interface>
+			</joint>
+			<!-- <transmission name="diff_wrist_transmission">
+				<plugin>transmission_interface/DifferentialTransmission</plugin>
+				<actuator name="arm_J5" role="actuator1"/>
+				<actuator name="arm_J6" role="actuator2"/>
+				<joint name="j5" role="joint1"/>
+				<joint name="j6" role="joint2"/>
+			</transmission> -->
+		</ros2_control>
+		<!-- <ros2_control name="arm_J5" type="system">
+			<xacro:unless value="${use_mock_hardware}">
+				<hardware>
+					<plugin>blcmd_hardware2/BLCMDHardware</plugin>
+					<param name="candevice">can1</param>
+					<param name="canid">5</param>
+					<param name="resolver_reduction">1.0</param>
+					<param name="clock_rate">100000000</param>
+					<param name="revolution_pulses">8192</param>
+          			<param name="min_interval">1792</param>
+					<param name="gear_ratio">1.0</param>
+					<param name="mock">true</param>
+					<param name="reversed">false</param>
+					<param name="integrate_velocity">false</param>
+					<param name="max_position">12.5663706144</param>
+					<param name="position_offset">3.14159265359</param>
+					<param name="max_velocity">292.444791136</param>
+				</hardware>
+			</xacro:unless>
+			<xacro:if value="${use_mock_hardware}">
+				<hardware>
+					<plugin>mock_components/GenericSystem</plugin>
+					<param name="calculate_dynamics">true</param>
+				</hardware>
+			</xacro:if>
+			<joint name="j5">
+				<command_interface name="velocity">
+					<param name="max">292.444791137</param>
+				</command_interface>
+				<command_interface name="position">
+					<param name="max">12.5663706144</param>
+				</command_interface>
+				<state_interface name="velocity">
+					<param name="max">292.444791137</param>
+					<param name="initial_value">0.0</param>
+				</state_interface>
+				<state_interface name="position">
+					<param name="max">12.5663706144</param>
+					<param name="initial_value">0.0</param>
+				</state_interface>
+			</joint>
+		</ros2_control> -->
+		<!-- <ros2_control name="arm_J6" type="system">
 			<xacro:unless value="${use_mock_hardware}">
 				<hardware>
@@ -237,5 +302,5 @@
 					<param name="max_position">12.5663706144</param>
 					<param name="position_offset">3.14159265359</param>
-					<!-- <param name="max_velocity">146.222395568</param> -->
+					<!-/- <param name="max_velocity">146.222395568</param> -/->
 					<param name="max_velocity">292.444791136</param>
 				</hardware>
@@ -263,5 +328,5 @@
 				</state_interface>
 			</joint>
-		</ros2_control>
+		</ros2_control> -->
 		<xacro:unless value="${use_mock_hardware}">
 			<ros2_control name="arm_la_prismatic" type="system">

File: src/ros/rover/rover_description/taipan/urdf/arm.urdf (robot description, URDF)
Before this commit: robot Arm, 18 links, 17 joints
Joints:
- removed joint la_prismatic
- removed joint lead_left
- removed joint lead_right

Commit message: test on hardware
tested position feedback only, not position commands.
issues:

wrist roll is backwards
mimic joints for 4 bar link is wrong - same issue as last time. when j2
moves the wrist should stay paralell to what it was.

wrist pitch offset might be wrong.

File: src/ros/rover/rover_description/taipan/urdf/arm.ros2_control.xacro (robot description, xacro)
@@ -64,4 +64,86 @@
 					<param name="gear_ratio">100.0</param>
 					<param name="mock">true</param>
+					<param name="reversed">false</param>
+					<param name="integrate_velocity">false</param>
+          <param name="res_ticks_per_rev">4096</param> <!-- 0x1000 is proportional to 2pi -->
+          <param name="zero_offset">7792</param> <!-- electrical's "home" is 0x2000 -->
+				</hardware>
+			</xacro:unless>
+			<xacro:if value="${use_mock_hardware}">
+				<hardware>
+					<plugin>mock_components/GenericSystem</plugin>
+					<param name="calculate_dynamics">true</param>
+				</hardware>
+			</xacro:if>
+			<joint name="j2">
+				<command_interface name="velocity">
+					<param name="max">292.444791137</param>
+				</command_interface>
+				<command_interface name="position">
+					<param name="max">12.5663706144</param>
+				</command_interface>
+				<state_interface name="velocity">
+					<param name="max">292.444791137</param>
+					<param name="initial_value">0.0</param>
+				</state_interface>
+				<state_interface name="position">
+					<param name="max">12.5663706144</param>
+					<param name="initial_value">0.0</param>
+				</state_interface>
+			</joint>
+		</ros2_control>
+		<ros2_control name="arm_J3" type="system">
+			<xacro:unless value="${use_mock_hardware}">
+				<hardware>
+					<plugin>blcmd_hardware2/BLCMDHardware</plugin>
+					<param name="candevice">can1</param>
+					<param name="canid">3</param>
+					<param name="resolver_reduction">5.375</param>
+					<param name="clock_rate">100000000</param>
+					<param name="revolution_pulses">8192</param>
+					<param name="min_interval">233</param>
+					<param name="gear_ratio">100.0</param>
+					<param name="mock">true</param>
+					<param name="reversed">true</param>
+					<param name="integrate_velocity">false</param>
+          <param name="res_ticks_per_rev">4096</param> <!-- 0x1000 is proportional to 2pi -->
+          <param name="zero_offset">8210</param> <!-- electrical's "home" is 0x2000 -->
+				</hardware>
+			</xacro:unless>
+			<xacro:if value="${use_mock_hardware}">
+				<hardware>
+					<plugin>mock_components/GenericSystem</plugin>
+					<param name="calculate_dynamics">true</param>
+				</hardware>
+			</xacro:if>
+			<joint name="j3">
+				<command_interface name="velocity">
+					<param name="max">292.444791137</param>
+				</command_interface>
+				<command_interface name="position">
+					<param name="max">12.5663706144</param>
+				</command_interface>
+				<state_interface name="velocity">
+					<param name="max">292.444791137</param>
+					<param name="initial_value">0.0</param>
+				</state_interface>
+				<state_interface name="position">
+					<param name="max">12.5663706144</param>
+					<param name="initial_value">0.0</param>
+				</state_interface>
+			</joint>
+		</ros2_control>
+		<ros2_control name="arm_J4" type="system">
+			<xacro:unless value="${use_mock_hardware}">
+				<hardware>
+					<plugin>blcmd_hardware2/BLCMDHardware</plugin>
+					<param name="candevice">can1</param>
+					<param name="canid">4</param>
+					<param name="resolver_reduction">4</param>
+					<param name="clock_rate">100000000</param>
+					<param name="revolution_pulses">8192</param>
+					<param name="min_interval">122</param>
+					<param name="gear_ratio">8.0</param>
+					<param name="mock">true</param>
 					<param name="reversed">true</param>
 					<param name="integrate_velocity">false</param>
@@ -76,86 +158,4 @@
 				</hardware>
 			</xacro:if>
-			<joint name="j2">
-				<command_interface name="velocity">
-					<param name="max">292.444791137</param>
-				</command_interface>
-				<command_interface name="position">
-					<param name="max">12.5663706144</param>
-				</command_interface>
-				<state_interface name="velocity">
-					<param name="max">292.444791137</param>
-					<param name="initial_value">0.0</param>
-				</state_interface>
-				<state_interface name="position">
-					<param name="max">12.5663706144</param>
-					<param name="initial_value">0.0</param>
-				</state_interface>
-			</joint>
-		</ros2_control>
-		<ros2_control name="arm_J3" type="system">
-			<xacro:unless value="${use_mock_hardware}">
-				<hardware>
-					<plugin>blcmd_hardware2/BLCMDHardware</plugin>
-					<param name="candevice">can1</param>
-					<param name="canid">3</param>
-					<param name="resolver_reduction">5.375</param>
-					<param name="clock_rate">100000000</param>
-					<param name="revolution_pulses">8192</param>
-					<param name="min_interval">233</param>
-					<param name="gear_ratio">100.0</param>
-					<param name="mock">true</param>
-					<param name="reversed">false</param>
-					<param name="integrate_velocity">false</param>
-          <param name="res_ticks_per_rev">4096</param> <!-- 0x1000 is proportional to 2pi -->
-          <param name="zero_offset">8192</param> <!-- electrical's "home" is 0x2000 -->
-				</hardware>
-			</xacro:unless>
-			<xacro:if value="${use_mock_hardware}">
-				<hardware>
-					<plugin>mock_components/GenericSystem</plugin>
-					<param name="calculate_dynamics">true</param>
-				</hardware>
-			</xacro:if>
-			<joint name="j3">
-				<command_interface name="velocity">
-					<param name="max">292.444791137</param>
-				</command_interface>
-				<command_interface name="position">
-					<param name="max">12.5663706144</param>
-				</command_interface>
-				<state_interface name="velocity">
-					<param name="max">292.444791137</param>
-					<param name="initial_value">0.0</param>
-				</state_interface>
-				<state_interface name="position">
-					<param name="max">12.5663706144</param>
-					<param name="initial_value">0.0</param>
-				</state_interface>
-			</joint>
-		</ros2_control>
-		<ros2_control name="arm_J4" type="system">
-			<xacro:unless value="${use_mock_hardware}">
-				<hardware>
-					<plugin>blcmd_hardware2/BLCMDHardware</plugin>
-					<param name="candevice">can1</param>
-					<param name="canid">4</param>
-					<param name="resolver_reduction">4</param>
-					<param name="clock_rate">100000000</param>
-					<param name="revolution_pulses">8192</param>
-					<param name="min_interval">122</param>
-					<param name="gear_ratio">8.0</param>
-					<param name="mock">true</param>
-					<param name="reversed">true</param>
-					<param name="integrate_velocity">false</param>
-          <param name="res_ticks_per_rev">4096</param> <!-- 0x1000 is proportional to 2pi -->
-          <param name="zero_offset">8192</param> <!-- electrical's "home" is 0x2000 -->
-				</hardware>
-			</xacro:unless>
-			<xacro:if value="${use_mock_hardware}">
-				<hardware>
-					<plugin>mock_components/GenericSystem</plugin>
-					<param name="calculate_dynamics">true</param>
-				</hardware>
-			</xacro:if>
 			<joint name="j4">
 				<command_interface name="velocity">
@@ -186,5 +186,5 @@
 					<param name="integrate_velocity">false</param>
 					<param name="res_ticks_per_rev">4096</param> <!-- 0x1000 is proportional to 2pi -->
-					<param name="zero_offset">8192</param> <!-- electrical's "home" is 0x2000 -->
+					<param name="zero_offset">7785</param> <!-- electrical's "home" is 0x2000 -->
 					<param name="diff_wrist">true</param>
 				</hardware>

Commit message: rover desc: taipan: fix urdf for mock.launch.py

File: src/ros/rover/rover_description/taipan/urdf/arm.ros2_control.xacro (robot description, xacro)
@@ -321,6 +321,6 @@
 			</joint>
 		</ros2_control> -->
-		<xacro:unless value="${use_mock_hardware}">
 			<ros2_control name="arm_la_prismatic" type="system">
+        <xacro:unless value="${use_mock_hardware}">
 					<hardware>
 						<plugin>qcmd_hardware/QCMDHardware</plugin>
@@ -329,4 +329,5 @@
 						<param name="max_effort">1</param>
 					</hardware>
+        </xacro:unless>
 				<xacro:if value="${use_mock_hardware}">
 					<hardware>
@@ -344,7 +345,6 @@
 				</joint>
 			</ros2_control>
-		</xacro:unless>
-	<xacro:unless value="${use_mock_hardware}">
 		<ros2_control name="arm_lead_left" type="system">
+	  <xacro:unless value="${use_mock_hardware}">
 			<hardware>
 				<plugin>qcmd_hardware/QCMDHardware</plugin>
@@ -353,10 +353,11 @@
 				<param name="max_effort">1</param>
 			</hardware>
-			<xacro:if value="${use_mock_hardware}">
-				<hardware>
-					<plugin>mock_components/GenericSystem</plugin>
-					<param name="calculate_dynamics">true</param>
-				</hardware>
-			</xacro:if>
+    </xacro:unless>
+    <xacro:if value="${use_mock_hardware}">
+      <hardware>
+        <plugin>mock_components/GenericSystem</plugin>
+        <param name="calculate_dynamics">true</param>
+      </hardware>
+    </xacro:if>
 			<joint name="lead_left">
 				<command_interface name="velocity">
@@ -368,5 +369,4 @@
 			</joint>
 		</ros2_control>
-	</xacro:unless>
 	</xacro:macro>
 </robot>

File: src/ros/rover/rover_description/taipan/urdf/arm.urdf (robot description, URDF)
Before this commit: robot Arm, 18 links, 14 joints
Joints:
- added joint la_prismatic: type prismatic, parent left_finger, child linear_actuator, origin xyz=-0.0001 -0.1175 -0.0125 rpy=-1.5708 -1.57652e-14 2.52817e-15, axis 0 0 1, limit lower=-0.05 upper=8.5652e-17 effort=10 velocity=10
- added joint lead_left: type prismatic, parent ee_base, child left_finger, origin xyz=-0.11253 -0.0301524 -0.1035 rpy=1.5708 -1.43108e-14 -1.309, axis 0 0 1, limit lower=-0.0855 upper=0 effort=10 velocity=10

File: src/ros/rover/rover_description/taipan/urdf/arm.urdf.xacro (robot description, xacro)
@@ -18,5 +18,5 @@
   <joint name="endeffector_kinematics_joint" type="fixed">
     <!-- before rotating to match IK function expected 0: 1.5707963 0.0 1.5707963 -->
-    <origin xyz="0.0067503 -0.0012 0.2225" rpy="-1.57079632679 -1.57079632679 0.0" />
+    <origin xyz="0.0067503 -0.0012 -0.2225" rpy="0.0 1.5707963 1.5707963" />
     <parent link="ee_base" />
     <child link="endeffector_kinematics" />

Commit message: add image frame to urdf and fixed finger/actuator positions for mock

File: src/ros/rover/rover_description/taipan/urdf/arm.ros2_control.xacro (robot description, xacro)
@@ -381,4 +381,9 @@
 					<param name="initial_value">0.0</param>
 					</state_interface>
+					<xacro:if value="${use_mock_hardware}">
+					<state_interface name="position">
+					<param name="initial_value">0.0</param>
+					</state_interface>
+					</xacro:if>
 				</joint>
 			</ros2_control>
@@ -405,4 +410,9 @@
 					<param name="initial_value">0.0</param>
 				</state_interface>
+				<xacro:if value="${use_mock_hardware}">
+				<state_interface name="position">
+				<param name="initial_value">0.0</param>
+				</state_interface>
+				</xacro:if>
 			</joint>
 		</ros2_control>

File: src/ros/rover/rover_description/taipan/urdf/arm.urdf.xacro (robot description, xacro)
@@ -36,4 +36,11 @@
   <!--    up 0.0138-->
   <!--    forward 0.012512-->
+  <!-- Periscope camera frame for auto-typing -->
+  <link name="image_frame"/>
+  <joint name="camera_ee_periscope" type="fixed">
+    <origin xyz="0.0001 -0.014 0.013" rpy="1.5708 1.5708 0"/>
+    <parent link="diff_support"/>
+    <child link="image_frame"/>
+  </joint>
   <!-- Gazebo / IRL Control -->
   <xacro:include filename="$(arg rover_description_dir)/taipan/urdf/arm_ckc.xacro"/>
