Commit message: arm: make fingers fixed in rviz (#1057)

File: src/ros/rover/rover_description/taipan/urdf/arm.ros2_control.xacro (robot description, xacro)
@@ -336,5 +336,7 @@
 					</hardware>
 				</xacro:if>
-				<joint name="la_prismatic">
+        <!-- There is no position feedback so la_prismatic will be a fixed
+        joint that appears in rviz, and la_prismatic_ will be the joint ros2control uses-->
+				<joint name="la_prismatic_">
 					<command_interface name="velocity">
 					<param name="max">1</param>
@@ -360,5 +362,5 @@
       </hardware>
     </xacro:if>
-			<joint name="lead_left">
+			<joint name="lead_left_">
 				<command_interface name="velocity">
 					<param name="max">1</param>
@@ -369,4 +371,23 @@
 			</joint>
 		</ros2_control>
+  <!-- fake joints with no visual for ros2control to use. -->
+  <joint name="la_prismatic_" type="prismatic">
+    <origin xyz="-0.0001 -0.1175 -0.0125" rpy="-1.5708 -1.57652e-14 2.52817e-15"/>
+    <parent link="left_finger"/>
+    <child link="linear_actuator_"/>
+    <axis xyz="0 0 1"/>
+    <limit effort="10" velocity="10" lower="-0.05" upper="8.5652e-17"/>
+  </joint>
+  <joint name="lead_left_" type="prismatic">
+    <origin xyz="-0.11253 -0.0301524 -0.1035" rpy="1.5708 -1.43108e-14 -1.309"/>
+    <parent link="ee_base"/>
+    <child link="left_finger_"/>
+    <axis xyz="0 0 1"/>
+    <limit effort="10" velocity="10" lower="-0.0855" upper="0"/>
+  </joint>
+  <link name="linear_actuator_">
+  </link>
+  <link name="left_finger_">
+  </link>
 	</xacro:macro>
 </robot>

File: src/ros/rover/rover_description/taipan/urdf/arm.urdf (robot description, URDF)
Before this commit: robot Arm, 18 links, 16 joints
Joints:
- added joint lead_right: type fixed, parent ee_base, child right_finger, origin xyz=-3.0892e-14 -5.32907e-15 -0.1035 rpy=-2.87979 -1.5708 0, axis 0 0 1, limit lower=-0.0855 upper=0 effort=10 velocity=10
- joint la_prismatic: type prismatic -> fixed
- joint lead_left: type prismatic -> fixed

File: src/ros/rover/rover_description/taipan/urdf/arm_joints.xacro (robot description, xacro)
@@ -15,9 +15,7 @@
                <joint_name>j5</joint_name>
                <joint_name>j6</joint_name>
-		     <xacro:unless value="${use_mock_hardware}">
-                    <joint_name>lead_left</joint_name>
-                    <joint_name>lead_right</joint_name>
-                    <joint_name>la_prismatic</joint_name>
-               </xacro:unless>
+               <joint_name>lead_left</joint_name>
+               <joint_name>lead_right</joint_name>
+               <joint_name>la_prismatic</joint_name>
           </plugin>
      </gazebo>
