Commit message: urdf: taipan: line up ee kinematics roll correctly

File: src/ros/rover/rover_description/taipan/urdf/arm.urdf.xacro (robot description, xacro)
@@ -18,5 +18,5 @@
   <joint name="endeffector_kinematics_joint" type="fixed">
     <!-- before rotating to match IK function expected 0: 1.5707963 0.0 1.5707963 -->
-    <origin xyz="0.0067503 -0.0012 -0.2225" rpy="0.0 1.5707963 1.5707963" />
+    <origin xyz="0.0 0.0 -0.2225" rpy="0.0 1.5707963 1.833" />
     <parent link="ee_base" />
     <child link="endeffector_kinematics" />

Commit message: feat: add ducket

File: src/ros/rover/rover_description/taipan/urdf/arm.urdf.xacro (robot description, xacro)
@@ -4,5 +4,15 @@
   xmlns:xacro="http://www.ros.org/wiki/xacro">
   <xacro:arg name="rover_description_dir" default="$(find rover_description)" />
+  <xacro:arg name="ducket" default="true"/>
   <xacro:include filename="$(arg rover_description_dir)/taipan/urdf/arm.urdf"/>
+  <xacro:if value="$(arg ducket)">
+    <xacro:include filename="$(arg rover_description_dir)/ducket/ducket.urdf.xacro"/>
+    <joint name="armbox_to_ducket" type="fixed">
+        <origin xyz="-0.0354798 -0.151628 -0.122841" rpy="-7.71583e-15 8.81621e-38 -4.38974e-37" />
+        <axis xyz="0 -0.707107 -0.707107" />
+        <parent link="arm_box" />
+        <child link="ducket_link" />
+    </joint>
+  </xacro:if>
   <!-- Kinematics -->
   <!-- THESE NEED FIXING 4/02/2026 !!! -->

Commit message: fix image frame position and add actuator frame

File: src/ros/rover/rover_description/taipan/urdf/arm.urdf.xacro (robot description, xacro)
@@ -36,9 +36,16 @@
   <!--    up 0.0138-->
   <!--    forward 0.012512-->
+  <!-- Linear actuator tip frame for auto-typing -->
+  <link name="actuator"/>
+  <joint name="actuator_tip_joint" type="fixed">
+    <origin xyz="0 0 -0.05" rpy="3.14159 0 0"/>
+    <parent link="linear_actuator"/>
+    <child link="actuator"/>
+  </joint>
   <!-- Periscope camera frame for auto-typing -->
   <link name="image_frame"/>
   <joint name="camera_ee_periscope" type="fixed">
-    <origin xyz="0.0001 -0.014 0.013" rpy="1.5708 1.5708 0"/>
-    <parent link="diff_support"/>
+    <origin xyz="0.0097 -0.037 -0.055" rpy="-3.14159 0 0.2618"/>
+    <parent link="ee_base"/>
     <child link="image_frame"/>
   </joint>

Commit message: fix actuator spacing, and yaw to match key tfs

File: src/ros/rover/rover_description/taipan/urdf/arm.urdf.xacro (robot description, xacro)
@@ -39,5 +39,5 @@
   <link name="actuator"/>
   <joint name="actuator_tip_joint" type="fixed">
-    <origin xyz="0 0 -0.05" rpy="3.14159 0 0"/>
+    <origin xyz="0 0 -0.016" rpy="3.14159 0 1.5707"/>
     <parent link="linear_actuator"/>
     <child link="actuator"/>

Commit message: fix: use arm end finger

File: src/ros/rover/rover_description/taipan/urdf/arm.urdf.xacro (robot description, xacro)
@@ -46,6 +46,6 @@
   <link name="image_frame"/>
   <joint name="camera_ee_periscope" type="fixed">
-    <origin xyz="0.0097 -0.037 -0.055" rpy="-3.14159 0 0.2618"/>
-    <parent link="ee_base"/>
+    <origin xyz="-0.063 0 0.017" rpy="3.14159 0 -1.5707"/>
+    <parent link="linear_actuator"/>
     <child link="image_frame"/>
   </joint>

Commit message: rename periscope to finger

File: src/ros/rover/rover_description/taipan/urdf/arm.urdf.xacro (robot description, xacro)
@@ -45,5 +45,5 @@
   <!-- Periscope camera frame for auto-typing -->
   <link name="image_frame"/>
-  <joint name="camera_ee_periscope" type="fixed">
+  <joint name="camera_ee_finger" type="fixed">
     <origin xyz="-0.063 0 0.017" rpy="3.14159 0 -1.5707"/>
     <parent link="linear_actuator"/>

Commit message: fix: add limit switch offset

File: src/ros/rover/rover_description/taipan/urdf/arm.urdf.xacro (robot description, xacro)
@@ -39,5 +39,5 @@
   <link name="actuator"/>
   <joint name="actuator_tip_joint" type="fixed">
-    <origin xyz="0 0 -0.016" rpy="3.14159 0 1.5707"/>
+    <origin xyz="0 0.0104 -0.016" rpy="3.14159 0 1.5707"/>
     <parent link="linear_actuator"/>
     <child link="actuator"/>

Commit message: feat: rotate ee 90deg

File: src/ros/rover/rover_description/taipan/urdf/arm.urdf.xacro (robot description, xacro)
@@ -39,5 +39,5 @@
   <link name="actuator"/>
   <joint name="actuator_tip_joint" type="fixed">
-    <origin xyz="0 0.0104 -0.016" rpy="3.14159 0 1.5707"/>
+    <origin xyz="0 0.0104 -0.016" rpy="3.1415926 0 -3.1415926"/>
     <parent link="linear_actuator"/>
     <child link="actuator"/>
@@ -46,5 +46,5 @@
   <link name="image_frame"/>
   <joint name="camera_ee_finger" type="fixed">
-    <origin xyz="-0.063 0 0.017" rpy="3.14159 0 -1.5707"/>
+    <origin xyz="-0.063 0 0.017" rpy="3.1415926 0 -1.5707963"/>
     <parent link="linear_actuator"/>
     <child link="image_frame"/>

Commit message: stuff

File: src/ros/rover/rover_description/taipan/urdf/arm.urdf.xacro (robot description, xacro)
@@ -39,12 +39,19 @@
   <link name="actuator"/>
   <joint name="actuator_tip_joint" type="fixed">
-    <origin xyz="0 0.0104 -0.016" rpy="3.1415926 0 -3.1415926"/>
+    <origin xyz="0 0.0104 -0.016" rpy="0 3.1415926 1.5707963"/>
     <parent link="linear_actuator"/>
     <child link="actuator"/>
+  </joint>
+  <!-- Linear actuator tip frame for auto-typing -->
+  <link name="old_actuator"/>
+  <joint name="a" type="fixed">
+    <origin xyz="0 0.0104 -0.016" rpy="0 3.1415926 0"/>
+    <parent link="linear_actuator"/>
+    <child link="old_actuator"/>
   </joint>
   <!-- Periscope camera frame for auto-typing -->
   <link name="image_frame"/>
   <joint name="camera_ee_finger" type="fixed">
-    <origin xyz="-0.063 0 0.017" rpy="3.1415926 0 -1.5707963"/>
+    <origin xyz="0 0 0" rpy="1.5707963 3.1415926 0"/>
     <parent link="linear_actuator"/>
     <child link="image_frame"/>

Commit message: feat: add back periscope camera for usbc

File: src/ros/rover/rover_description/taipan/urdf/arm.urdf.xacro (robot description, xacro)
@@ -36,5 +36,5 @@
   <!--    up 0.0138-->
   <!--    forward 0.012512-->
-  <!-- Linear actuator tip frame for auto-typing -->
+  <!-- Linear actuator tip frame -->
   <link name="actuator"/>
   <joint name="actuator_tip_joint" type="fixed">
@@ -43,5 +43,12 @@
     <child link="actuator"/>
   </joint>
-  <!-- Periscope camera frame for auto-typing -->
+  <!-- Periscope camera frame -->
+  <link name="arm_end_periscope_optical"/>
+  <joint name="camera_ee_periscope" type="fixed">
+    <origin xyz="0.0097 -0.037 -0.055" rpy="-3.14159 0 0.2618"/>
+    <parent link="ee_base"/>
+    <child link="arm_end_periscope_optical"/>
+  </joint>
+  <!-- Finger camera frame -->
   <link name="image_frame"/>
   <joint name="camera_ee_finger" type="fixed">
