Commit message: wip: more progress on can description

File: src/other/can_description/blcmd.kcd.xacro (robot description, xacro)
@@ -1,4 +1,4 @@
 <?xml version="1.0" encoding="utf-8" ?>
-<wrapper xmlns:xacro="http://www.ros.org/wiki/xacro">
+<wrapper xmlns:xacro="http://www.ros.org/wiki/xacro" xmlns:xsi="http://www.w3.org/2001/XMLSchema-instance" xmlns="http://kayak.2codeornot2code.org/1.0" xsi:noNamespaceSchemaLocation="schemas/kcd-macro.xsd">
     <xacro:macro name="blcmd_messages" params="
     blcmd_id
@@ -7,10 +7,38 @@
     position_multiplier:=${None}
     position_offset:=${None}
-    raw_values:=false
     blcmd_node_id:=${None}
     orin_node_id:=0
+    raw_velocity:=false
+    raw_position:=false
+    raw_effort:=false
     ">
+        <!-- variables -->
         <xacro:property name="limit_16_bit_signed_integer" value="${2**15 - 1}"/>
-        <xacro:property name="blcmd_node_id_" value="${blcmd_id if blcmd_node_id is None else blcmd_node_id}"/>
+        <xacro:property name="blcmd_node_id" value="${blcmd_id if blcmd_node_id is None else blcmd_node_id}" lazy_eval="false"/>
+        <xacro:property name="velocity_multiplier" value="${max_velocity / limit_16_bit_signed_integer}"/>
+        <xacro:property name="effort_multiplier" value="${1 / limit_16_bit_signed_integer}"/>
+        <!-- output raw values (if requested) by modifying variables -->
+        <xacro:if value="${raw_velocity}">
+            <xacro:property name="velocity_multiplier" value="1" lazy_eval="false"/>
+        </xacro:if>
+        <xacro:if value="${raw_position or position_multiplier is None or position_offset is None}">
+            <xacro:property name="position_multiplier" value="1" lazy_eval="false"/>
+            <xacro:property name="position_offset" value="0" lazy_eval="false"/>
+        </xacro:if>
+        <xacro:if value="${raw_effort}">
+            <xacro:property name="effort_multiplier" value="1" lazy_eval="false"/>
+        </xacro:if>
+        <!-- messages sent from orin to blcmd -->
+        <!-- macros for repetitive consumer/producer tags -->
+        <xacro:macro name="consumer_blcmd">
+            <Consumer>
+                <NodeRef id="${blcmd_node_id}"/>
+            </Consumer>
+        </xacro:macro>
+        <xacro:macro name="producer_orin">
+            <Producer>
+                <NodeRef id="${orin_node_id}"/>
+            </Producer>
+        </xacro:macro>
         <Message id="0x0${blcmd_id}0" name="${joint_name}_all_stop">
             <Producer>
@@ -19,5 +47,5 @@
             <Signal name="all_stop_requested" offset="0">
                 <Consumer>
-                    <NodeRef id="${blcmd_node_id_}"/>
+                    <NodeRef id="${blcmd_node_id}"/>
                 </Consumer>
             </Signal>
@@ -29,5 +57,5 @@
             <Signal name="twitch_forward_requested" offset="0">
                 <Consumer>
-                    <NodeRef id="${blcmd_node_id_}"/>
+                    <NodeRef id="${blcmd_node_id}"/>
                 </Consumer>
             </Signal>
@@ -39,5 +67,5 @@
             <Signal name="twitch_backward_requested" offset="0">
                 <Consumer>
-                    <NodeRef id="${blcmd_node_id_}"/>
+                    <NodeRef id="${blcmd_node_id}"/>
                 </Consumer>
             </Signal>
@@ -47,19 +75,11 @@
                 <NodeRef id="${orin_node_id}"/>
             </Producer>
-            <xacro:unless value="${raw_values}">
-                <Signal name="velocity_requested" offset="0" length="16" endianess="big">
-                    <Notes>Target velocity (radians per second)</Notes>
-                    <Consumer>
-                        <NodeRef id="${blcmd_node_id_}"/>
-                    </Consumer>
-                    <Value type="signed" unit="rad/s" slope="${max_velocity / limit_16_bit_signed_integer}"/>
-                </Signal>
-            </xacro:unless>
-            <xacro:if value="${raw_values}">
-                <Signal name="velocity_requested_raw" offset="0" length="16" endianess="big">
-                    <Notes>Target velocity (signed value sent on CAN bus)</Notes>
-                    <Value type="signed"/>
-                </Signal>
-            </xacro:if>
+            <Signal name="velocity_requested" offset="0" length="16" endianess="big">
+                <Notes>Target velocity (radians per second)</Notes>
+                <Consumer>
+                    <NodeRef id="${blcmd_node_id}"/>
+                </Consumer>
+                <Value type="signed" unit="rad/s" slope="${velocity_multiplier}"/>
+            </Signal>
         </Message>
         <Message id="0x0${blcmd_id}4" name="${joint_name}_drive_to_position">
@@ -67,22 +87,11 @@
                 <NodeRef id="${orin_node_id}"/>
             </Producer>
-            <!-- decide whether to calculate position or just provide raw values -->
-            <xacro:property name="raw_position" value="${raw_values
-            or position_multiplier is None or position_offset is None}"/>
-            <xacro:unless value="${raw_position}">
-                <Signal name="position_requested" offset="0" length="16" endianess="big">
-                    <Notes>Target position (radians from zero)</Notes>
-                    <Consumer>
-                        <NodeRef id="${blcmd_node_id_}"/>
-                    </Consumer>
-                    <Value type="signed" unit="rad" slope="${position_multiplier}" intercept="${position_offset}"/>
-                </Signal>
-            </xacro:unless>
-            <xacro:if value="${raw_position}">
-                <Signal name="position_requested_raw" offset="0" length="16" endianess="big">
-                    <Notes>Target position (signed value sent on CAN bus)</Notes>
-                    <Value type="signed"/>
-                </Signal>
-            </xacro:if>
+            <Signal name="position_requested" offset="0" length="16" endianess="big">
+                <Notes>Target position (radians from zero)</Notes>
+                <Consumer>
+                    <NodeRef id="${blcmd_node_id}"/>
+                </Consumer>
+                <Value type="signed" unit="rad" slope="${position_multiplier}" intercept="${position_offset}"/>
+            </Signal>
         </Message>
         <Message id="0x0${blcmd_id}5" name="${joint_name}_drive_at_current">
@@ -90,19 +99,11 @@
                 <NodeRef id="${orin_node_id}"/>
             </Producer>
-            <xacro:unless value="${raw_values}">
-                <Signal name="effort_requested" offset="0" length="16" endianess="big">
-                    <Notes>Target effort (proportion of max effort)</Notes>
-                    <Consumer>
-                        <NodeRef id="${blcmd_node_id_}"/>
-                    </Consumer>
-                    <Value type="signed" unit="1" slope="${1 / limit_16_bit_signed_integer}"/>
-                </Signal>
-            </xacro:unless>
-            <xacro:if value="${raw_values}">
-                <Signal name="effort_requested_raw" offset="0" length="16" endianess="big">
-                    <Notes>Target effort (signed value sent on CAN bus)</Notes>
-                    <Value type="signed"/>
-                </Signal>
-            </xacro:if>
+            <Signal name="effort_requested" offset="0" length="16" endianess="big">
+                <Notes>Target effort (proportion of max effort)</Notes>
+                <Consumer>
+                    <NodeRef id="${blcmd_node_id}"/>
+                </Consumer>
+                <Value type="signed" unit="1" slope="${effort_multiplier}"/>
+            </Signal>
         </Message>
         <Message id="0x0${blcmd_id}6" name="${joint_name}_drive_open_loop">
@@ -113,5 +114,5 @@
             <Signal name="open_loop_current_requested_raw" offset="0" length="16" endianess="big">
                 <Consumer>
-                    <NodeRef id="${blcmd_node_id_}"/>
+                    <NodeRef id="${blcmd_node_id}"/>
                 </Consumer>
                 <Value type="signed"/>
@@ -119,5 +120,5 @@
             <Signal name="open_loop_velocity_requested_raw" offset="16" length="16" endianess="big">
                 <Consumer>
-                    <NodeRef id="${blcmd_node_id_}"/>
+                    <NodeRef id="${blcmd_node_id}"/>
                 </Consumer>
                 <Value type="signed"/>
@@ -130,15 +131,15 @@
             <Signal name="home_rotor_requested" offset="0">
                 <Consumer>
-                    <NodeRef id="${blcmd_node_id_}"/>
-                </Consumer>
-            </Signal>
-        </Message>
-        <Message id="0x0${blcmd_id}8" name="${joint_name}_set_resolver_zero_flag">
-            <Producer>
-                <NodeRef id="${orin_node_id}"/>
-            </Producer>
-            <Signal name="set_resolver_zero_flag_requested" offset="0">
-                <Consumer>
-                    <NodeRef id="${blcmd_node_id_}"/>
+                    <NodeRef id="${blcmd_node_id}"/>
+                </Consumer>
+            </Signal>
+        </Message>
+        <Message id="0x0${blcmd_id}8" name="${joint_name}_zero_resolver">
+            <Producer>
+                <NodeRef id="${orin_node_id}"/>
+            </Producer>
+            <Signal name="zero_resolver_requested" offset="0">
+                <Consumer>
+                    <NodeRef id="${blcmd_node_id}"/>
                 </Consumer>
             </Signal>
@@ -150,5 +151,5 @@
             <Signal name="configuration_requested" offset="0" length="8" endianess="big">
                 <Consumer>
-                    <NodeRef id="${blcmd_node_id_}"/>
+                    <NodeRef id="${blcmd_node_id}"/>
                 </Consumer>
                 <Value type="signed"/>
@@ -172,5 +173,138 @@
             </Signal>
         </Message>
-        <!-- TODO: REST -->
+        <Message id="0x0${blcmd_id}A" name="${joint_name}_set_configuration">
+            <Producer>
+                <NodeRef id="${orin_node_id}"/>
+            </Producer>
+            <!-- set configuration is "multiplexed" (so value of first byte determines what remaining bytes mean) -->
+            <Multiplex name="configuration_set" offset="0" length="8" endianess="big">
+                <Consumer>
+                    <NodeRef id="${blcmd_node_id}"/>
+                </Consumer>
+                <Value type="signed"/>
+                <LabelSet>
+                    <Label name="has_resolver" value="0"/>
+                    <Label name="current_kp" value="1"/>
+                    <Label name="current_ki" value="2"/>
+                    <Label name="max_current_threshold" value="3"/>
+                    <Label name="velocity_kp" value="4"/>
+                    <Label name="velocity_ki" value="5"/>
+                    <Label name="max_velocity_threshold" value="6"/>
+                    <Label name="min_interval" value="7"/>
+                    <Label name="position_kp" value="8"/>
+                    <Label name="position_ki" value="9"/>
+                    <Label name="max_position_threshold" value="10"/>
+                    <Label name="telemetry_packet_1_speed" value="11"/>
+                    <Label name="telemetry_packet_2_speed" value="12"/>
+                    <Label name="telemetry_packet_3_speed" value="13"/>
+                    <Label name="telemetry_packet_4_speed" value="14"/>
+                </LabelSet>
+                <!-- signals for has_resolver -->
+                <MuxGroup count="0">
+                    <Signal name="value" offset="8" length="8" endianess="big">
+                        <LabelSet>
+                            <Label name="false" value="0"/>
+                            <Label name="true" value="1"/>
+                        </LabelSet>
+                    </Signal>
+                </MuxGroup>
+                <!-- signals for current_kp and current_ki -->
+                <MuxGroup count="1">
+                    <Signal name="fractional" offset="8" length="16" endianess="big"/>
+                    <Signal name="shift_amount" offset="24" length="8" endianess="big"/>
+                </MuxGroup>
+                <MuxGroup count="2">
+                    <Signal name="fractional" offset="8" length="16" endianess="big"/>
+                    <Signal name="shift_amount" offset="24" length="8" endianess="big"/>
+                </MuxGroup>
+                <!-- signals for max_current_threshold -->
+                <MuxGroup count="3">
+                    <Signal name="max_current" offset="8" length="16" endianess="big"/>
+                </MuxGroup>
+                <!-- signals for velocity_kp and velocity_ki -->
+                <MuxGroup count="4">
+                    <Signal name="fractional" offset="8" length="16" endianess="big"/>
+                    <Signal name="shift_amount" offset="24" length="8" endianess="big"/>
+                </MuxGroup>
+                <MuxGroup count="5">
+                    <Signal name="fractional" offset="8" length="16" endianess="big"/>
+                    <Signal name="shift_amount" offset="24" length="8" endianess="big"/>
+                </MuxGroup>
+                <!-- signals for max_velocity_threshold -->
+                <MuxGroup count="6">
+                    <Signal name="max_velocity" offset="8" length="16" endianess="big"/>
+                </MuxGroup>
+                <!-- signals for min_interval -->
+                <MuxGroup count="7">
+                    <!-- WARNING: in blcmd firmware, this value appears not to be used -->
+                    <Signal name="min_interval" offset="8" length="16" endianess="big"/>
+                </MuxGroup>
+                <!-- signals for position_kp and position_ki-->
+                <MuxGroup count="8">
+                    <Signal name="fractional" offset="8" length="16" endianess="big"/>
+                    <Signal name="shift_amount" offset="24" length="8" endianess="big"/>
+                </MuxGroup>
+                <MuxGroup count="9">
+                    <Signal name="fractional" offset="8" length="16" endianess="big"/>
+                    <Signal name="shift_amount" offset="24" length="8" endianess="big"/>
+                </MuxGroup>
+                <!-- signals for max_position_threshold -->
+                <MuxGroup count="10">
+                    <Signal name="max_position" offset="8" length="16" endianess="big"/>
+                </MuxGroup>
+                <!-- signals for telemetry_packet_1_speed, telemetry_packet_2_speed
+                telemetry_packet_3_speed and telemetry_packet_4_speed -->
+                <MuxGroup count="11">
+                    <Signal name="speed" offset="8" length="8" endianess="big"/>
+                </MuxGroup>
+                <MuxGroup count="12">
+                    <Signal name="speed" offset="8" length="8" endianess="big"/>
+                </MuxGroup>
+                <MuxGroup count="13">
+                    <Signal name="speed" offset="8" length="8" endianess="big"/>
+                </MuxGroup>
+                <MuxGroup count="14">
+                    <Signal name="speed" offset="8" length="8" endianess="big"/>
+                </MuxGroup>
+            </Multiplex>
+        </Message>
+        <Message id="0x0${blcmd_id}B" name="${joint_name}_reset_blcmd">
+            <xacro:producer_orin/>
+            <Signal name="reset_blcmd_requested" offset="0">
+                <xacro:consumer_blcmd/>
+            </Signal>
+        </Message>
+        <Message id="0x0${blcmd_id}C" name="${joint_name}_reset_resolver">
+            <xacro:producer_orin/>
+            <Signal name="reset_resolver_requested" offset="0">
+                <xacro:consumer_blcmd/>
+            </Signal>
+        </Message>
+        <Message id="0x0${blcmd_id}D" name="${joint_name}_read_gate_driver_fault">
+            <xacro:producer_orin/>
+            <Signal name="read_gate_driver_fault_requested" offset="0">
+                <xacro:consumer_blcmd/>
+            </Signal>
+        </Message>
+        <!-- messages sent from blcmd to orin -->
+        <!-- macros for repetitive consumer/producer tags -->
+        <xacro:macro name="consumer_orin">
+            <Consumer>
+                <NodeRef id="${orin_node_id}"/>
+            </Consumer>
+        </xacro:macro>
+        <xacro:macro name="producer_blcmd">
+            <Producer>
+                <NodeRef id="${blcmd_node_id}"/>
+            </Producer>
+        </xacro:macro>
+        <Message id="0x4${blcmd_id}1" name="${joint_name}_telemetry_packet_1">
+            <xacro:producer_blcmd/>
+            <Signal name="velocity" offset="0" length="16" endianess="big">
+                <Notes>Velocity (radians per second)</Notes>
+                <xacro:consumer_orin/>
+                <Value type="signed" unit="rad/s" slope="${velocity_multiplier}"/>
+            </Signal>
+        </Message>
     </xacro:macro>
 </wrapper>
