Commit message: feat: don't convert dynamics to si units, add more telemetry packets

File: src/other/can_description/blcmd.kcd.xacro (robot description, xacro)
@@ -4,29 +4,23 @@
     blcmd_id
     joint_name
-    max_velocity
-    position_multiplier:=${None}
-    position_offset:=${None}
     blcmd_node_id:=${None}
     orin_node_id:=0
-    raw_velocity:=false
-    raw_position:=false
-    raw_effort:=false
     ">
         <!-- variables -->
-        <xacro:property name="limit_16_bit_signed_integer" value="${2**15 - 1}"/>
+<!--        <xacro:property name="limit_16_bit_signed_integer" value="${2**15 - 1}"/>-->
         <xacro:property name="blcmd_node_id" value="${blcmd_id if blcmd_node_id is None else blcmd_node_id}" lazy_eval="false"/>
-        <xacro:property name="velocity_multiplier" value="${max_velocity / limit_16_bit_signed_integer}"/>
-        <xacro:property name="effort_multiplier" value="${1 / limit_16_bit_signed_integer}"/>
+<!--        <xacro:property name="velocity_multiplier" value="${max_velocity / limit_16_bit_signed_integer}"/>-->
+<!--        <xacro:property name="effort_multiplier" value="${1 / limit_16_bit_signed_integer}"/>-->
         <!-- output raw values (if requested) by modifying variables -->
-        <xacro:if value="${raw_velocity}">
-            <xacro:property name="velocity_multiplier" value="1" lazy_eval="false"/>
-        </xacro:if>
-        <xacro:if value="${raw_position or position_multiplier is None or position_offset is None}">
-            <xacro:property name="position_multiplier" value="1" lazy_eval="false"/>
-            <xacro:property name="position_offset" value="0" lazy_eval="false"/>
-        </xacro:if>
-        <xacro:if value="${raw_effort}">
-            <xacro:property name="effort_multiplier" value="1" lazy_eval="false"/>
-        </xacro:if>
+<!--        <xacro:if value="${raw_velocity}">-->
+<!--            <xacro:property name="velocity_multiplier" value="1" lazy_eval="false"/>-->
+<!--        </xacro:if>-->
+<!--        <xacro:if value="${raw_position or position_multiplier is None or position_offset is None}">-->
+<!--            <xacro:property name="position_multiplier" value="1" lazy_eval="false"/>-->
+<!--            <xacro:property name="position_offset" value="0" lazy_eval="false"/>-->
+<!--        </xacro:if>-->
+<!--        <xacro:if value="${raw_effort}">-->
+<!--            <xacro:property name="effort_multiplier" value="1" lazy_eval="false"/>-->
+<!--        </xacro:if>-->
         <!-- messages sent from orin to blcmd -->
         <!-- macros for repetitive consumer/producer tags -->
@@ -62,7 +56,6 @@
             <xacro:producer_orin/>
             <Signal name="velocity_requested" offset="0" length="16" endianess="big">
-                <Notes>Target velocity (radians per second)</Notes>
-                <xacro:consumer_blcmd/>
-                <Value type="signed" unit="rad/s" slope="${velocity_multiplier}"/>
+                <xacro:consumer_blcmd/>
+                <Value type="signed"/>
             </Signal>
         </Message>
@@ -70,7 +63,6 @@
             <xacro:producer_orin/>
             <Signal name="position_requested" offset="0" length="16" endianess="big">
-                <Notes>Target position (radians from zero)</Notes>
-                <xacro:consumer_blcmd/>
-                <Value type="signed" unit="rad" slope="${position_multiplier}" intercept="${position_offset}"/>
+                <xacro:consumer_blcmd/>
+                <Value type="signed"/>
             </Signal>
         </Message>
@@ -78,7 +70,6 @@
             <xacro:producer_orin/>
             <Signal name="effort_requested" offset="0" length="16" endianess="big">
-                <Notes>Target effort (proportion of max effort)</Notes>
-                <xacro:consumer_blcmd/>
-                <Value type="signed" unit="1" slope="${effort_multiplier}"/>
+                <xacro:consumer_blcmd/>
+                <Value type="signed"/>
             </Signal>
         </Message>
@@ -86,9 +77,9 @@
             <xacro:producer_orin/>
             <!-- not implemented in blcmd firmware, so only raw values provided -->
-            <Signal name="open_loop_current_requested_raw" offset="0" length="16" endianess="big">
-                <xacro:consumer_blcmd/>
-                <Value type="signed"/>
-            </Signal>
-            <Signal name="open_loop_velocity_requested_raw" offset="16" length="16" endianess="big">
+            <Signal name="open_loop_current_requested" offset="0" length="16" endianess="big">
+                <xacro:consumer_blcmd/>
+                <Value type="signed"/>
+            </Signal>
+            <Signal name="open_loop_velocity_requested" offset="16" length="16" endianess="big">
                 <xacro:consumer_blcmd/>
                 <Value type="signed"/>
@@ -256,7 +247,51 @@
             <xacro:producer_blcmd/>
             <Signal name="velocity" offset="0" length="16" endianess="big">
-                <Notes>Velocity (radians per second)</Notes>
-                <xacro:consumer_orin/>
-                <Value type="signed" unit="rad/s" slope="${velocity_multiplier}"/>
+                <xacro:consumer_orin/>
+                <Value type="signed"/>
+            </Signal>
+            <Signal name="q_current" offset="16" length="16" endianess="big">
+                <xacro:consumer_orin/>
+                <Value type="signed"/>
+            </Signal>
+        </Message>
+        <Message id="0x4${blcmd_id}2" name="${joint_name}_telemetry_packet_2">
+            <xacro:producer_blcmd/>
+            <Signal name="interval" offset="0" length="16" endianess="big">
+                <xacro:consumer_orin/>
+                <Value type="signed"/>
+            </Signal>
+            <Signal name="d_current" offset="16" length="16" endianess="big">
+                <xacro:consumer_orin/>
+                <Value type="signed"/>
+            </Signal>
+        </Message>
+        <Message id="0x4${blcmd_id}3" name="${joint_name}_telemetry_packet_3">
+            <xacro:producer_blcmd/>
+            <Signal name="resolver_position" offset="0" length="16" endianess="big">
+                <xacro:consumer_orin/>
+                <Value type="signed"/>
+            </Signal>
+            <Signal name="resolver_velocity" offset="16" length="16" endianess="big">
+                <xacro:consumer_orin/>
+                <Value type="signed"/>
+            </Signal>
+        </Message>
+        <Message id="0x4${blcmd_id}4" name="${joint_name}_telemetry_packet_4">
+            <xacro:producer_blcmd/>
+            <Signal name="power" offset="0" length="16" endianess="big">
+                <xacro:consumer_orin/>
+                <Value type="signed"/>
+            </Signal>
+            <Signal name="voltage" offset="16" length="16" endianess="big">
+                <xacro:consumer_orin/>
+                <Value type="signed"/>
+            </Signal>
+            <Signal name="temperature" offset="32" length="16" endianess="big">
+                <xacro:consumer_orin/>
+                <Value type="signed"/>
+            </Signal>
+            <Signal name="current" offset="48" length="16" endianess="big">
+                <xacro:consumer_orin/>
+                <Value type="signed"/>
             </Signal>
         </Message>

File: src/other/can_description/drive.kcd.xacro (robot description, xacro)
@@ -27,44 +27,12 @@
 	<xacro:property name="pivot_position_offset" value="${ -1 * zero_offset * pivot_position_multiplier }"/>
 	<Bus name="can0" baudrate="250000">
-		<xacro:blcmd_messages
-				blcmd_id="1"
-				joint_name="flw"
-				max_velocity="${wheel_max_velocity}"/>
-		<xacro:blcmd_messages
-				blcmd_id="2"
-				joint_name="blw"
-				max_velocity="${wheel_max_velocity}"/>
-		<xacro:blcmd_messages
-				blcmd_id="3"
-				joint_name="brw"
-				max_velocity="${wheel_max_velocity}"/>
-		<xacro:blcmd_messages
-				blcmd_id="4"
-				joint_name="frw"
-				max_velocity="${wheel_max_velocity}"/>
-		<xacro:blcmd_messages
-				blcmd_id="5"
-				joint_name="flp"
-				max_velocity="${pivot_max_velocity}"
-				position_multiplier="${-1 * pivot_position_multiplier}"
-				position_offset="${-1 * pivot_position_offset}"/>
-		<xacro:blcmd_messages
-				blcmd_id="6"
-				joint_name="blp"
-				max_velocity="${pivot_max_velocity}"
-				position_multiplier="${pivot_position_multiplier}"
-				position_offset="${pivot_position_offset}"/>
-		<xacro:blcmd_messages
-				blcmd_id="7"
-				joint_name="brp"
-				max_velocity="${pivot_max_velocity}"
-				position_multiplier="${-1 * pivot_position_multiplier}"
-				position_offset="${-1 * pivot_position_offset}"/>
-		<xacro:blcmd_messages
-				blcmd_id="8"
-				joint_name="frp"
-				max_velocity="${pivot_max_velocity}"
-				position_multiplier="${pivot_position_multiplier}"
-				position_offset="${pivot_position_offset}"/>
+		<xacro:blcmd_messages blcmd_id="1" joint_name="flw"/>
+		<xacro:blcmd_messages blcmd_id="2" joint_name="blw"/>
+		<xacro:blcmd_messages blcmd_id="3" joint_name="brw"/>
+		<xacro:blcmd_messages blcmd_id="4" joint_name="frw"/>
+		<xacro:blcmd_messages blcmd_id="5" joint_name="flp"/>
+		<xacro:blcmd_messages blcmd_id="6" joint_name="blp"/>
+		<xacro:blcmd_messages blcmd_id="7" joint_name="brp"/>
+		<xacro:blcmd_messages blcmd_id="8" joint_name="frp"/>
 	</Bus>
 </NetworkDefinition>

Commit message: feat: blcmd configuration reply

File: src/other/can_description/blcmd.kcd.xacro (robot description, xacro)
@@ -98,120 +98,115 @@
             </Signal>
         </Message>
+        <!-- labels for configuration signal/multiplex (i.e. associates configuration id with name) -->
+        <xacro:macro name="configuration_labels">
+            <LabelSet>
+                <Label name="has_resolver" value="0"/>
+                <Label name="current_kp" value="1"/>
+                <Label name="current_ki" value="2"/>
+                <Label name="max_current_threshold" value="3"/>
+                <Label name="velocity_kp" value="4"/>
+                <Label name="velocity_ki" value="5"/>
+                <Label name="max_velocity_threshold" value="6"/>
+                <Label name="min_interval" value="7"/>
+                <Label name="position_kp" value="8"/>
+                <Label name="position_ki" value="9"/>
+                <Label name="max_position_threshold" value="10"/>
+                <Label name="telemetry_packet_1_speed" value="11"/>
+                <Label name="telemetry_packet_2_speed" value="12"/>
+                <Label name="telemetry_packet_3_speed" value="13"/>
+                <Label name="telemetry_packet_4_speed" value="14"/>
+            </LabelSet>
+        </xacro:macro>
         <Message id="0x0${blcmd_id}9" name="${joint_name}_get_configuration">
             <xacro:producer_orin/>
-            <Signal name="configuration_requested" offset="0" length="8" endianess="big">
-                <xacro:consumer_blcmd/>
-                <Value type="signed"/>
-                <LabelSet>
-                    <Label name="has_resolver" value="0"/>
-                    <Label name="current_kp" value="1"/>
-                    <Label name="current_ki" value="2"/>
-                    <Label name="max_current_threshold" value="3"/>
-                    <Label name="velocity_kp" value="4"/>
-                    <Label name="velocity_ki" value="5"/>
-                    <Label name="max_velocity_threshold" value="6"/>
-                    <Label name="min_interval" value="7"/>
-                    <Label name="position_kp" value="8"/>
-                    <Label name="position_ki" value="9"/>
-                    <Label name="max_position_threshold" value="10"/>
-                    <Label name="telemetry_packet_1_speed" value="11"/>
-                    <Label name="telemetry_packet_2_speed" value="12"/>
-                    <Label name="telemetry_packet_3_speed" value="13"/>
-                    <Label name="telemetry_packet_4_speed" value="14"/>
-                </LabelSet>
-            </Signal>
-        </Message>
-        <Message id="0x0${blcmd_id}A" name="${joint_name}_set_configuration">
-            <xacro:producer_orin/>
-            <!-- set configuration is "multiplexed" (so value of first byte determines what remaining bytes mean) -->
-            <Multiplex name="configuration_set" offset="0" length="8" endianess="big">
-                <xacro:consumer_blcmd/>
-                <Value type="signed"/>
-                <LabelSet>
-                    <Label name="has_resolver" value="0"/>
-                    <Label name="current_kp" value="1"/>
-                    <Label name="current_ki" value="2"/>
-                    <Label name="max_current_threshold" value="3"/>
-                    <Label name="velocity_kp" value="4"/>
-                    <Label name="velocity_ki" value="5"/>
-                    <Label name="max_velocity_threshold" value="6"/>
-                    <Label name="min_interval" value="7"/>
-                    <Label name="position_kp" value="8"/>
-                    <Label name="position_ki" value="9"/>
-                    <Label name="max_position_threshold" value="10"/>
-                    <Label name="telemetry_packet_1_speed" value="11"/>
-                    <Label name="telemetry_packet_2_speed" value="12"/>
-                    <Label name="telemetry_packet_3_speed" value="13"/>
-                    <Label name="telemetry_packet_4_speed" value="14"/>
-                </LabelSet>
-                <!-- signals for has_resolver -->
-                <MuxGroup count="0">
-                    <Signal name="value" offset="8" length="8" endianess="big">
-                        <LabelSet>
-                            <Label name="false" value="0"/>
-                            <Label name="true" value="1"/>
-                        </LabelSet>
-                    </Signal>
-                </MuxGroup>
-                <!-- signals for current_kp and current_ki -->
-                <MuxGroup count="1">
-                    <Signal name="fractional" offset="8" length="16" endianess="big"/>
-                    <Signal name="shift_amount" offset="24" length="8" endianess="big"/>
-                </MuxGroup>
-                <MuxGroup count="2">
-                    <Signal name="fractional" offset="8" length="16" endianess="big"/>
-                    <Signal name="shift_amount" offset="24" length="8" endianess="big"/>
-                </MuxGroup>
-                <!-- signals for max_current_threshold -->
-                <MuxGroup count="3">
-                    <Signal name="max_current" offset="8" length="16" endianess="big"/>
-                </MuxGroup>
-                <!-- signals for velocity_kp and velocity_ki -->
-                <MuxGroup count="4">
-                    <Signal name="fractional" offset="8" length="16" endianess="big"/>
-                    <Signal name="shift_amount" offset="24" length="8" endianess="big"/>
-                </MuxGroup>
-                <MuxGroup count="5">
-                    <Signal name="fractional" offset="8" length="16" endianess="big"/>
-                    <Signal name="shift_amount" offset="24" length="8" endianess="big"/>
-                </MuxGroup>
-                <!-- signals for max_velocity_threshold -->
-                <MuxGroup count="6">
-                    <Signal name="max_velocity" offset="8" length="16" endianess="big"/>
-                </MuxGroup>
-                <!-- signals for min_interval -->
-                <MuxGroup count="7">
-                    <!-- WARNING: in blcmd firmware, this value appears not to be used -->
-                    <Signal name="min_interval" offset="8" length="16" endianess="big"/>
-                </MuxGroup>
-                <!-- signals for position_kp and position_ki-->
-                <MuxGroup count="8">
-                    <Signal name="fractional" offset="8" length="16" endianess="big"/>
-                    <Signal name="shift_amount" offset="24" length="8" endianess="big"/>
-                </MuxGroup>
-                <MuxGroup count="9">
-                    <Signal name="fractional" offset="8" length="16" endianess="big"/>
-                    <Signal name="shift_amount" offset="24" length="8" endianess="big"/>
-                </MuxGroup>
-                <!-- signals for max_position_threshold -->
-                <MuxGroup count="10">
-                    <Signal name="max_position" offset="8" length="16" endianess="big"/>
-                </MuxGroup>
-                <!-- signals for telemetry_packet_1_speed, telemetry_packet_2_speed
-                telemetry_packet_3_speed and telemetry_packet_4_speed -->
-                <MuxGroup count="11">
-                    <Signal name="speed" offset="8" length="8" endianess="big"/>
-                </MuxGroup>
-                <MuxGroup count="12">
-                    <Signal name="speed" offset="8" length="8" endianess="big"/>
-                </MuxGroup>
-                <MuxGroup count="13">
-                    <Signal name="speed" offset="8" length="8" endianess="big"/>
-                </MuxGroup>
-                <MuxGroup count="14">
-                    <Signal name="speed" offset="8" length="8" endianess="big"/>
-                </MuxGroup>
-            </Multiplex>
-        </Message>
+            <Signal name="configuration" offset="0" length="8" endianess="big">
+                <xacro:consumer_blcmd/>
+                <Value type="signed"/>
+                <xacro:configuration_labels/>
+            </Signal>
+        </Message>
+        <!-- message macro for both set_configuration (from orin to blcmd)
+        and current_configuration (from blcmd to orin) -->
+        <xacro:macro name="configuration_messages" params="id name *producer_block *consumer_block">
+            <Message id="${id}" name="${name}">
+                <xacro:insert_block name="producer_block"/>
+                <!-- set configuration is "multiplexed" (so value of first byte determines what remaining bytes mean) -->
+                <Multiplex name="configuration" offset="0" length="8" endianess="big">
+                    <xacro:insert_block name="consumer_block"/>
+                    <xacro:configuration_labels/>
+                    <!-- signals for has_resolver -->
+                    <MuxGroup count="0">
+                        <Signal name="value" offset="8" length="8" endianess="big">
+                            <LabelSet>
+                                <Label name="false" value="0"/>
+                                <Label name="true" value="1"/>
+                            </LabelSet>
+                        </Signal>
+                    </MuxGroup>
+                    <!-- signals for current_kp and current_ki -->
+                    <MuxGroup count="1">
+                        <Signal name="fractional" offset="8" length="16" endianess="big"/>
+                        <Signal name="shift_amount" offset="24" length="8" endianess="big"/>
+                    </MuxGroup>
+                    <MuxGroup count="2">
+                        <Signal name="fractional" offset="8" length="16" endianess="big"/>
+                        <Signal name="shift_amount" offset="24" length="8" endianess="big"/>
+                    </MuxGroup>
+                    <!-- signals for max_current_threshold -->
+                    <MuxGroup count="3">
+                        <Signal name="max_current" offset="8" length="16" endianess="big"/>
+                    </MuxGroup>
+                    <!-- signals for velocity_kp and velocity_ki -->
+                    <MuxGroup count="4">
+                        <Signal name="fractional" offset="8" length="16" endianess="big"/>
+                        <Signal name="shift_amount" offset="24" length="8" endianess="big"/>
+                    </MuxGroup>
+                    <MuxGroup count="5">
+                        <Signal name="fractional" offset="8" length="16" endianess="big"/>
+                        <Signal name="shift_amount" offset="24" length="8" endianess="big"/>
+                    </MuxGroup>
+                    <!-- signals for max_velocity_threshold -->
+                    <MuxGroup count="6">
+                        <Signal name="max_velocity" offset="8" length="16" endianess="big"/>
+                    </MuxGroup>
+                    <!-- signals for min_interval -->
+                    <MuxGroup count="7">
+                        <!-- WARNING: in blcmd firmware, this value appears not to be used -->
+                        <Signal name="min_interval" offset="8" length="16" endianess="big"/>
+                    </MuxGroup>
+                    <!-- signals for position_kp and position_ki-->
+                    <MuxGroup count="8">
+                        <Signal name="fractional" offset="8" length="16" endianess="big"/>
+                        <Signal name="shift_amount" offset="24" length="8" endianess="big"/>
+                    </MuxGroup>
+                    <MuxGroup count="9">
+                        <Signal name="fractional" offset="8" length="16" endianess="big"/>
+                        <Signal name="shift_amount" offset="24" length="8" endianess="big"/>
+                    </MuxGroup>
+                    <!-- signals for max_position_threshold -->
+                    <MuxGroup count="10">
+                        <Signal name="max_position" offset="8" length="16" endianess="big"/>
+                    </MuxGroup>
+                    <!-- signals for telemetry_packet_1_speed, telemetry_packet_2_speed
+                    telemetry_packet_3_speed and telemetry_packet_4_speed -->
+                    <MuxGroup count="11">
+                        <Signal name="speed" offset="8" length="8" endianess="big"/>
+                    </MuxGroup>
+                    <MuxGroup count="12">
+                        <Signal name="speed" offset="8" length="8" endianess="big"/>
+                    </MuxGroup>
+                    <MuxGroup count="13">
+                        <Signal name="speed" offset="8" length="8" endianess="big"/>
+                    </MuxGroup>
+                    <MuxGroup count="14">
+                        <Signal name="speed" offset="8" length="8" endianess="big"/>
+                    </MuxGroup>
+                </Multiplex>
+            </Message>
+        </xacro:macro>
+        <xacro:configuration_messages id="0x0${blcmd_id}A" name="${joint_name}_set_configuration">
+            <xacro:producer_orin/>
+            <xacro:consumer_blcmd/>
+        </xacro:configuration_messages>
         <Message id="0x0${blcmd_id}B" name="${joint_name}_reset_blcmd">
             <xacro:producer_orin/>
@@ -359,4 +354,8 @@
             </Multiplex>
         </Message>
+        <xacro:configuration_messages id="0x4${blcmd_id}9" name="${joint_name}_current_configuration">
+            <xacro:producer_blcmd/>
+            <xacro:consumer_orin/>
+        </xacro:configuration_messages>
     </xacro:macro>
 </wrapper>
