Commit message: feat: Refactored rover description, renamed arm to waratah_arm (to prepare for banksia_arm), renamed rover7 to banksia, fixed nova_bringup urdf.launch to load both waratah and banksia with waratah_arm and disable rviz, also now launches with banksia chassis and waratah arm

File: src/ros/rover/rover_description/auto_mount/urdf/auto_camera.xacro (robot description, xacro)
@@ -2,4 +2,5 @@
 <!--This is a file for the depth camera plugin for the rover in gazebo. This file is referenced at the bottom of rover.urdf.xacro,
 which is how it gets added to the gazebo sim. Edited by: Victor Bartlinski, Kabi Velmurugan Sujatha -->
+<!-- Auto mount is also appended to the top, however it has no simplified collisions -->
 <robot xmlns:xacro="http://www.ros.org/wiki/xacro">
   <xacro:macro name="auto_cam" params="angle">
@@ -14,5 +15,5 @@
             <origin xyz="0.138856 0.281 0.00511278" rpy="3.14159 -0.00348764 3.3577e-34" />
             <geometry>
-                <mesh filename="file://$(find rover_description)/rover7/auto/meshes/clam.stl" />
+                <mesh filename="file://$(find rover_description)/auto_mount/meshes/clam.stl" />
             </geometry>
             <material name="clam_material">
@@ -23,5 +24,5 @@
             <origin xyz="0.138856 0.281 0.00511278" rpy="3.14159 -0.00348764 3.3577e-34" />
             <geometry>
-                <mesh filename="file://$(find rover_description)/rover7/auto/meshes/clam.stl" />
+                <mesh filename="file://$(find rover_description)/auto_mount/meshes/clam.stl" />
             </geometry>
         </collision>
@@ -36,5 +37,5 @@
             <origin xyz="0.081 0.000713936 -0.025" rpy="4.93038e-32 6.86401e-31 -3.70732e-33" />
             <geometry>
-                <mesh filename="file://$(find rover_description)/rover7/auto/meshes/mount.stl" />
+                <mesh filename="file://$(find rover_description)/auto_mount/meshes/mount.stl" />
             </geometry>
             <material name="mount_material">
@@ -45,5 +46,5 @@
             <origin xyz="0.081 0.000713936 -0.025" rpy="4.93038e-32 6.86401e-31 -3.70732e-33" />
             <geometry>
-                <mesh filename="file://$(find rover_description)/rover7/auto/meshes/mount.stl" />
+                <mesh filename="file://$(find rover_description)/auto_mount/meshes/mount.stl" />
             </geometry>
         </collision>
@@ -58,5 +59,5 @@
             <origin xyz="-0.075 5.55112e-17 0.06" rpy="-1.5708 -1.5708 0" />
             <geometry>
-                <mesh filename="file://$(find rover_description)/rover7/auto/meshes/camera_holder.stl" />
+                <mesh filename="file://$(find rover_description)/auto_mount/meshes/camera_holder.stl" />
             </geometry>
             <material name="camera_holder_front_material">
@@ -67,5 +68,5 @@
             <origin xyz="-0.075 5.55112e-17 0.06" rpy="-1.5708 -1.5708 0" />
             <geometry>
-                <mesh filename="file://$(find rover_description)/rover7/auto/meshes/camera_holder.stl" />
+                <mesh filename="file://$(find rover_description)/auto_mount/meshes/camera_holder.stl" />
             </geometry>
         </collision>
@@ -86,5 +87,5 @@
             <origin xyz="-0.075 0 0.06" rpy="1.5708 1.5708 0" />
             <geometry>
-                <mesh filename="file://$(find rover_description)/rover7/auto/meshes/camera_holder.stl" />
+                <mesh filename="file://$(find rover_description)/auto_mount/meshes/camera_holder.stl" />
             </geometry>
             <material name="camera_holder_back_material">
@@ -95,5 +96,5 @@
             <origin xyz="-0.075 0 0.06" rpy="1.5708 1.5708 0" />
             <geometry>
-                <mesh filename="file://$(find rover_description)/rover7/auto/meshes/camera_holder.stl" />
+                <mesh filename="file://$(find rover_description)/auto_mount/meshes/camera_holder.stl" />
             </geometry>
         </collision>

File: src/ros/rover/rover_description/banksia/urdf/rover.urdf.xacro (robot description, xacro)
@@ -5,5 +5,5 @@
            Therefore if exported from onshape, don't forget to add a negative sign to the z of the axis tag on each pivot
      Note 2: Exporting from onshape has _continuous at the end of continuous joint names these have been removed post-export -->
-<robot name="rover"  xmlns:xacro="http://www.ros.org/wiki/xacro" >
+<robot name="banksia"  xmlns:xacro="http://www.ros.org/wiki/xacro" >
     <!-- Loading args -->
     <xacro:arg name="gazebo" default="false"/>
@@ -11,5 +11,5 @@
     <xacro:arg name="arm" default="false"/>
     <xacro:arg name="auto_camera" default="true"/>
-    <xacro:arg name="robot_name" default="rover"/>
+    <xacro:arg name="robot_name" default="banksia"/>
     <xacro:arg name="angle" default="0"/>
     <!-- Robot properties-->
@@ -28,5 +28,5 @@
             <origin xyz="0 0 0" rpy="3.26128e-16 -1.01395e-15 1.5708" />
             <geometry>
-                <mesh filename="file://$(find rover_description)/rover7/meshes/chassis.stl" />
+                <mesh filename="file://$(find rover_description)/banksia/meshes/chassis.stl" />
             </geometry>
             <material name="chassis_material">
@@ -45,5 +45,5 @@
             <origin xyz="-1.3078806732583218725e-20 8.6736173798840354721e-19 -0.021000000000000518252" rpy="-3.141592653589793116 6.2280032059897877693e-19 -4.1232880706353110482e-18" />
             <geometry>
-                <mesh filename="file://$(find rover_description)/rover7/meshes/left_leg.stl"/>
+                <mesh filename="file://$(find rover_description)/banksia/meshes/left_leg.stl"/>
             </geometry>
             <material name="left_leg_material">
@@ -116,5 +116,5 @@
             <origin xyz="-0.12415341931613717297 2.2204460492503130808e-16 -0.1250000000000002498" rpy="-1.570796326794896558 -0.13351607992219349796 -5.9804098682663148249e-17" />
             <geometry>
-                <mesh filename="file://$(find rover_description)/rover7/meshes/fl_ankle.stl"/>
+                <mesh filename="file://$(find rover_description)/banksia/meshes/fl_ankle.stl"/>
             </geometry>
             <material name="fl_ankle_material">
@@ -175,5 +175,5 @@
             <origin xyz="5.5511151231257827021e-17 0 5.963111948670274387e-18" rpy="7.279848939407052303e-17 1.0638440422271473935e-16 -6.3914183266779029169e-20" />
             <geometry>
-                <mesh filename="file://$(find rover_description)/rover7/meshes/fl_wheel.stl"/>
+                <mesh filename="file://$(find rover_description)/banksia/meshes/fl_wheel.stl"/>
             </geometry>
             <material name="fl_wheel_material">
@@ -198,5 +198,5 @@
             <origin xyz="-0.12415341931613714521 2.2204460492503130808e-16 -0.1250000000000002498" rpy="-1.570796326794896558 -0.13351607992219349796 -7.1088909477657821376e-17" />
             <geometry>
-                <mesh filename="file://$(find rover_description)/rover7/meshes/bl_ankle.stl"/>
+                <mesh filename="file://$(find rover_description)/banksia/meshes/bl_ankle.stl"/>
             </geometry>
             <material name="bl_ankle_material">
@@ -257,5 +257,5 @@
             <origin xyz="0 1.1102230246251565404e-16 1.7780915628762272718e-17" rpy="4.6040217445536182725e-17 1.0513492286565858337e-16 2.3412503191653332746e-19" />
             <geometry>
-                <mesh filename="file://$(find rover_description)/rover7/meshes/bl_wheel.stl"/>
+                <mesh filename="file://$(find rover_description)/banksia/meshes/bl_wheel.stl"/>
             </geometry>
             <material name="bl_wheel_material">
@@ -280,5 +280,5 @@
             <origin xyz="-7.9461177221465168975e-19 -7.2858385990954703269e-20 -0.020999999999999519051" rpy="3.141592653589793116 3.7838655819744092421e-17 -5.8406613147999892266e-19" />
             <geometry>
-                <mesh filename="file://$(find rover_description)/rover7/meshes/right_leg.stl"/>
+                <mesh filename="file://$(find rover_description)/banksia/meshes/right_leg.stl"/>
             </geometry>
             <material name="right_leg_material">
@@ -351,5 +351,5 @@
             <origin xyz="0.12415341931613695092 -2.2204460492503130808e-16 -0.12500000000000027756" rpy="-1.57079632679489678 0.13351607992219352572 9.9507186100571649487e-18" />
             <geometry>
-                <mesh filename="file://$(find rover_description)/rover7/meshes/fr_ankle.stl"/>
+                <mesh filename="file://$(find rover_description)/banksia/meshes/fr_ankle.stl"/>
             </geometry>
             <material name="fr_ankle_material">
@@ -410,5 +410,5 @@
             <origin xyz="5.5511151231257827021e-17 -1.1102230246251565404e-16 -3.0791341698588325926e-17" rpy="-3.6194812825998444115e-17 1.0511409763610977507e-16 -2.2325341479697011877e-19" />
             <geometry>
-                <mesh filename="file://$(find rover_description)/rover7/meshes/fr_wheel.stl"/>
+                <mesh filename="file://$(find rover_description)/banksia/meshes/fr_wheel.stl"/>
             </geometry>
             <material name="fr_wheel_material">
@@ -433,5 +433,5 @@
             <origin xyz="0.12415341931613720072 -2.2204460492503130808e-16 -0.12500000000000027756" rpy="-1.57079632679489678 0.13351607992219349796 -6.7670245197813334123e-17" />
             <geometry>
-                <mesh filename="file://$(find rover_description)/rover7/meshes/br_ankle.stl"/>
+                <mesh filename="file://$(find rover_description)/banksia/meshes/br_ankle.stl"/>
             </geometry>
             <material name="br_ankle_material">
@@ -492,5 +492,5 @@
             <origin xyz="5.5511151231257827021e-17 0 5.8763757748714340323e-17" rpy="1.4537948349788456791e-16 1.0501738044156386319e-16 -7.6074648532850333807e-21" />
             <geometry>
-                <mesh filename="file://$(find rover_description)/rover7/meshes/br_wheel.stl"/>
+                <mesh filename="file://$(find rover_description)/banksia/meshes/br_wheel.stl"/>
             </geometry>
             <material name="br_wheel_material">
@@ -515,5 +515,5 @@
             <origin xyz="4.9770590769729886024e-14 -0.00015426611885745872277 -0.010000000000000730527" rpy="1.570796326794896558 -3.0512890594788867116e-34 0" />
             <geometry>
-                <mesh filename="file://$(find rover_description)/rover7/meshes/diffbar.stl"/>
+                <mesh filename="file://$(find rover_description)/banksia/meshes/diffbar.stl"/>
             </geometry>
             <material name="diffbar_material">
@@ -544,5 +544,5 @@
             <origin xyz="-2.7755575615628913511e-15 -0.057750000000000162315 3.3306690738754696213e-16" rpy="1.5707963267948350516 -1.5127867282353739675 -3.1415926535897926719" />
             <geometry>
-                <mesh filename="file://$(find rover_description)/rover7/meshes/left_difflink.stl"/>
+                <mesh filename="file://$(find rover_description)/banksia/meshes/left_difflink.stl"/>
             </geometry>
             <material name="left_difflink_material">
@@ -567,5 +567,5 @@
             <origin xyz="6.2172489379008766264e-15 -0.057749999999999454547 -2.4424906541753443889e-15" rpy="1.5707963267948286123 1.512786629442331332 3.141592653589793116" />
             <geometry>
-                <mesh filename="file://$(find rover_description)/rover7/meshes/right_difflink.stl"/>
+                <mesh filename="file://$(find rover_description)/banksia/meshes/right_difflink.stl"/>
             </geometry>
             <material name="right_difflink_material">
@@ -682,14 +682,14 @@
     <!-- End of Generated URDF -->
     <!-- Include additional xacro files-->
-    <xacro:include filename="$(find rover_description)/rover7/urdf/ckc.xacro"/>
+    <xacro:include filename="$(find rover_description)/banksia/urdf/ckc.xacro"/>
     <xacro:if value="$(arg auto_camera)">
-        <xacro:include filename="$(find rover_description)/rover7/auto/auto_camera.xacro"/>
+        <xacro:include filename="$(find rover_description)/auto_mount/urdf/auto_camera.xacro"/>
         <xacro:auto_cam angle="$(arg angle)"></xacro:auto_cam>
     </xacro:if>
     <xacro:if value="$(arg arm)">
-        <!-- Needs to be updated for new arm-->
-        <xacro:include filename="$(find rover_description)/arm/urdf/arm.urdf.xacro" />
+        <!-- Currently attaches waratah's arm, add banksia arm after ARCh-->
+        <xacro:include filename="/home/nova/nova/src/ros/rover/rover_description/waratah_arm/urdf/arm.urdf.xacro" />
         <joint name="chassis_to_arm_base" type="fixed">
-            <origin xyz="0.18 0 -0.03" rpy="0 0 0"/>
+            <origin xyz="0.2 0 -0.06" rpy="0 0 0"/>
             <parent link="chassis" />
             <child link="arm_link" />
@@ -697,13 +697,13 @@
     </xacro:if>
     <xacro:unless value="$(arg gazebo)">
-        <xacro:include filename="$(find rover_description)/rover7/urdf/ros2_control.xacro" />
+        <xacro:include filename="$(find rover_description)/banksia/urdf/ros2_control.xacro" />
         <xacro:rover_ros2_control use_mock_hardware="$(arg use_mock_hardware)"/>
     </xacro:unless>
     <xacro:if value="$(arg gazebo)">
-        <xacro:include filename="$(find rover_description)/rover7/urdf/gz_ros2_control.xacro" />
+        <xacro:include filename="$(find rover_description)/banksia/urdf/gz_ros2_control.xacro" />
     </xacro:if>
-    <xacro:include filename="$(find rover_description)/rover7/urdf/p3d.xacro"/>
-    <xacro:include filename="$(find rover_description)/rover7/urdf/odom.xacro"/>
-    <xacro:include filename="$(find rover_description)/rover7/urdf/gps.xacro"/>
-    <xacro:include filename="$(find rover_description)/rover7/urdf/joint_states.xacro"/>
+    <xacro:include filename="$(find rover_description)/banksia/urdf/p3d.xacro"/>
+    <xacro:include filename="$(find rover_description)/banksia/urdf/odom.xacro"/>
+    <xacro:include filename="$(find rover_description)/banksia/urdf/gps.xacro"/>
+    <xacro:include filename="$(find rover_description)/banksia/urdf/joint_states.xacro"/>
 </robot>
