Commit message: removed sensor stuff temporarily to stop URDF from crashing

File: src/ros/rover/rover_description/auto_mount/urdf/auto_camera.xacro (robot description, xacro)
@@ -123,10 +123,4 @@
     <link name="camera_link"/>
     <link name="bootie_link"/> <!-- KABI OR SOMEONE ADD BOOTIE CAM GAZEBO SENSORS!!! -->
-  <!-- Add camera directly to chassis
-    <joint name="camera_joint" type="fixed">
-      <origin xyz="0.8 0 0.525" rpy="0 ${angle*(pi/180)} 0"/>
-      <parent link="chassis"/>
-      <child link="camera_link"/>
-    </joint> -->
     <joint name="oak_to_mount" type="fixed">
       <origin xyz="-0.120 0.004 0.039" rpy="1.5708 0 3.14159" />
@@ -173,190 +167,4 @@
       <child link="camera_link_optical"/>
     </joint>
-    <!-- Front Oak Depth Camera for Gazebo-->
-    <gazebo reference="camera_link">
-      <sensor name="oak" type="rgbd_camera">
-        <gz_frame_id>camera_link_optical</gz_frame_id>
-        <!-- Link that corresponds to the Depth Point Clouds -->
-        <optical_frame_id>camera_link</optical_frame_id>
-        <topic>oak</topic>
-        <visualize>true</visualize>
-        <update_rate>30</update_rate>
-        <always_on>1</always_on>
-        <camera name="oak">
-          <horizontal_fov>${radians(82)}</horizontal_fov>
-          <image>
-            <width>1280</width>
-            <height>900</height>
-          </image>
-          <clip>
-            <near>0.4</near>
-            <far>10.0</far>
-          </clip>
-        </camera>
-        <plugin name="gz::sim::systems::Sensors" filename="gz-sim-sensors-system">
-          <frame_name>camera_link_optical</frame_name>
-        </plugin>
-      </sensor>
-    </gazebo>
-    <!-- Bootie Rear Depth Camera for Gazebo-->
-    <gazebo reference="bootie_link">
-      <sensor name="bootie" type="rgbd_camera">
-        <gz_frame_id>bootie_link_optical</gz_frame_id>
-        <!-- Link that corresponds to the Depth Point Clouds -->
-        <optical_frame_id>bootie_link</optical_frame_id>
-        <topic>bootie</topic>
-        <visualize>true</visualize>
-        <update_rate>30</update_rate>
-        <always_on>1</always_on>
-        <camera name="bootie">
-          <horizontal_fov>${radians(82)}</horizontal_fov>
-          <image>
-            <width>1280</width>
-            <height>900</height>
-          </image>
-          <clip>
-            <near>0.4</near>
-            <far>10.0</far>
-          </clip>
-        </camera>
-        <plugin name="gz::sim::systems::Sensors" filename="gz-sim-sensors-system">
-          <frame_name>bootie_link_optical</frame_name>
-        </plugin>
-      </sensor>
-    </gazebo>
-    <!-- Front IMU for Gazebo-->
-    <gazebo reference="oak_imu_frame">
-      <sensor name="imu_sensor" type="imu">
-        <topic>oak/imu</topic>
-        <plugin filename="gz-sim-imu-system" name="gz::sim::systems::Imu">
-          <frame_name>oak_imu_frame</frame_name>
-          <initial_orientation_as_reference>false</initial_orientation_as_reference>
-        </plugin>
-        <always_on>true</always_on>
-        <update_rate>200</update_rate>
-        <visualize>true</visualize>
-        <imu>
-          <angular_velocity>
-            <x>
-              <noise type="gaussian">
-                <mean>0.0</mean>
-                <stddev>2e-4</stddev>
-                <bias_mean>0.0000075</bias_mean>
-                <bias_stddev>0.0000008</bias_stddev>
-              </noise>
-            </x>
-            <y>
-              <noise type="gaussian">
-                <mean>0.0</mean>
-                <stddev>2e-4</stddev>
-                <bias_mean>0.0000075</bias_mean>
-                <bias_stddev>0.0000008</bias_stddev>
-              </noise>
-            </y>
-            <z>
-              <noise type="gaussian">
-                <mean>0.0</mean>
-                <stddev>2e-4</stddev>
-                <bias_mean>0.0000075</bias_mean>
-                <bias_stddev>0.0000008</bias_stddev>
-              </noise>
-            </z>
-          </angular_velocity>
-          <linear_acceleration>
-            <x>
-              <noise type="gaussian">
-                <mean>0.0</mean>
-                <stddev>1.7e-2</stddev>
-                <bias_mean>0.1</bias_mean>
-                <bias_stddev>0.001</bias_stddev>
-              </noise>
-            </x>
-            <y>
-              <noise type="gaussian">
-                <mean>0.0</mean>
-                <stddev>1.7e-2</stddev>
-                <bias_mean>0.1</bias_mean>
-                <bias_stddev>0.001</bias_stddev>
-              </noise>
-            </y>
-            <z>
-              <noise type="gaussian">
-                <mean>0.0</mean>
-                <stddev>1.7e-2</stddev>
-                <bias_mean>0.1</bias_mean>
-                <bias_stddev>0.001</bias_stddev>
-              </noise>
-            </z>
-          </linear_acceleration>
-        </imu>
-      </sensor>
-    </gazebo>
-    <!-- Bootie for Gazebo-->
-    <gazebo reference="bootie_imu_frame">
-      <sensor name="bootie_imu_sensor" type="imu">
-        <topic>bootie/imu</topic>
-        <plugin filename="gz-sim-imu-system" name="gz::sim::systems::Imu">
-          <frame_name>bootie_imu_frame</frame_name>
-          <initial_orientation_as_reference>false</initial_orientation_as_reference>
-        </plugin>
-        <always_on>true</always_on>
-        <update_rate>200</update_rate>
-        <visualize>true</visualize>
-        <imu>
-          <angular_velocity>
-            <x>
-              <noise type="gaussian">
-                <mean>0.0</mean>
-                <stddev>2e-4</stddev>
-                <bias_mean>0.0000075</bias_mean>
-                <bias_stddev>0.0000008</bias_stddev>
-              </noise>
-            </x>
-            <y>
-              <noise type="gaussian">
-                <mean>0.0</mean>
-                <stddev>2e-4</stddev>
-                <bias_mean>0.0000075</bias_mean>
-                <bias_stddev>0.0000008</bias_stddev>
-              </noise>
-            </y>
-            <z>
-              <noise type="gaussian">
-                <mean>0.0</mean>
-                <stddev>2e-4</stddev>
-                <bias_mean>0.0000075</bias_mean>
-                <bias_stddev>0.0000008</bias_stddev>
-              </noise>
-            </z>
-          </angular_velocity>
-          <linear_acceleration>
-            <x>
-              <noise type="gaussian">
-                <mean>0.0</mean>
-                <stddev>1.7e-2</stddev>
-                <bias_mean>0.1</bias_mean>
-                <bias_stddev>0.001</bias_stddev>
-              </noise>
-            </x>
-            <y>
-              <noise type="gaussian">
-                <mean>0.0</mean>
-                <stddev>1.7e-2</stddev>
-                <bias_mean>0.1</bias_mean>
-                <bias_stddev>0.001</bias_stddev>
-              </noise>
-            </y>
-            <z>
-              <noise type="gaussian">
-                <mean>0.0</mean>
-                <stddev>1.7e-2</stddev>
-                <bias_mean>0.1</bias_mean>
-                <bias_stddev>0.001</bias_stddev>
-              </noise>
-            </z>
-          </linear_acceleration>
-        </imu>
-      </sensor>
-    </gazebo>
   </xacro:macro>
 </robot>

File: src/ros/rover/rover_description/rover7/urdf/rover.urdf.xacro (robot description, xacro)
@@ -5,5 +5,5 @@
            Therefore if exported from onshape, don't forget to add a negative sign to the z of the axis tag on each pivot
      Note 2: Exporting from onshape has _continuous at the end of continuous joint names these have been removed post-export -->
-<robot name="banksia"  xmlns:xacro="http://www.ros.org/wiki/xacro" >
+<robot name="rover7"  xmlns:xacro="http://www.ros.org/wiki/xacro" >
     <!-- Loading args -->
     <xacro:arg name="gazebo" default="false"/>
@@ -11,5 +11,5 @@
     <xacro:arg name="arm" default="false"/>
     <xacro:arg name="auto_camera" default="true"/>
-    <xacro:arg name="robot_name" default="banksia"/>
+    <xacro:arg name="robot_name" default="rover7"/>
     <xacro:arg name="angle" default="0"/>
     <!-- Robot properties-->
@@ -28,5 +28,5 @@
             <origin xyz="0 0 0" rpy="3.26128e-16 -1.01395e-15 1.5708" />
             <geometry>
-                <mesh filename="file://$(find rover_description)/banksia/meshes/chassis.stl" />
+                <mesh filename="file://$(find rover_description)/rover7/meshes/chassis.stl" />
             </geometry>
             <material name="chassis_material">
@@ -45,5 +45,5 @@
             <origin xyz="-1.3078806732583218725e-20 8.6736173798840354721e-19 -0.021000000000000518252" rpy="-3.141592653589793116 6.2280032059897877693e-19 -4.1232880706353110482e-18" />
             <geometry>
-                <mesh filename="file://$(find rover_description)/banksia/meshes/left_leg.stl"/>
+                <mesh filename="file://$(find rover_description)/rover7/meshes/left_leg.stl"/>
             </geometry>
             <material name="left_leg_material">
@@ -116,5 +116,5 @@
             <origin xyz="-0.12415341931613717297 2.2204460492503130808e-16 -0.1250000000000002498" rpy="-1.570796326794896558 -0.13351607992219349796 -5.9804098682663148249e-17" />
             <geometry>
-                <mesh filename="file://$(find rover_description)/banksia/meshes/fl_ankle.stl"/>
+                <mesh filename="file://$(find rover_description)/rover7/meshes/fl_ankle.stl"/>
             </geometry>
             <material name="fl_ankle_material">
@@ -175,5 +175,5 @@
             <origin xyz="5.5511151231257827021e-17 0 5.963111948670274387e-18" rpy="7.279848939407052303e-17 1.0638440422271473935e-16 -6.3914183266779029169e-20" />
             <geometry>
-                <mesh filename="file://$(find rover_description)/banksia/meshes/fl_wheel.stl"/>
+                <mesh filename="file://$(find rover_description)/rover7/meshes/fl_wheel.stl"/>
             </geometry>
             <material name="fl_wheel_material">
@@ -198,5 +198,5 @@
             <origin xyz="-0.12415341931613714521 2.2204460492503130808e-16 -0.1250000000000002498" rpy="-1.570796326794896558 -0.13351607992219349796 -7.1088909477657821376e-17" />
             <geometry>
-                <mesh filename="file://$(find rover_description)/banksia/meshes/bl_ankle.stl"/>
+                <mesh filename="file://$(find rover_description)/rover7/meshes/bl_ankle.stl"/>
             </geometry>
             <material name="bl_ankle_material">
@@ -257,5 +257,5 @@
             <origin xyz="0 1.1102230246251565404e-16 1.7780915628762272718e-17" rpy="4.6040217445536182725e-17 1.0513492286565858337e-16 2.3412503191653332746e-19" />
             <geometry>
-                <mesh filename="file://$(find rover_description)/banksia/meshes/bl_wheel.stl"/>
+                <mesh filename="file://$(find rover_description)/rover7/meshes/bl_wheel.stl"/>
             </geometry>
             <material name="bl_wheel_material">
@@ -280,5 +280,5 @@
             <origin xyz="-7.9461177221465168975e-19 -7.2858385990954703269e-20 -0.020999999999999519051" rpy="3.141592653589793116 3.7838655819744092421e-17 -5.8406613147999892266e-19" />
             <geometry>
-                <mesh filename="file://$(find rover_description)/banksia/meshes/right_leg.stl"/>
+                <mesh filename="file://$(find rover_description)/rover7/meshes/right_leg.stl"/>
             </geometry>
             <material name="right_leg_material">
@@ -351,5 +351,5 @@
             <origin xyz="0.12415341931613695092 -2.2204460492503130808e-16 -0.12500000000000027756" rpy="-1.57079632679489678 0.13351607992219352572 9.9507186100571649487e-18" />
             <geometry>
-                <mesh filename="file://$(find rover_description)/banksia/meshes/fr_ankle.stl"/>
+                <mesh filename="file://$(find rover_description)/rover7/meshes/fr_ankle.stl"/>
             </geometry>
             <material name="fr_ankle_material">
@@ -410,5 +410,5 @@
             <origin xyz="5.5511151231257827021e-17 -1.1102230246251565404e-16 -3.0791341698588325926e-17" rpy="-3.6194812825998444115e-17 1.0511409763610977507e-16 -2.2325341479697011877e-19" />
             <geometry>
-                <mesh filename="file://$(find rover_description)/banksia/meshes/fr_wheel.stl"/>
+                <mesh filename="file://$(find rover_description)/rover7/meshes/fr_wheel.stl"/>
             </geometry>
             <material name="fr_wheel_material">
@@ -433,5 +433,5 @@
             <origin xyz="0.12415341931613720072 -2.2204460492503130808e-16 -0.12500000000000027756" rpy="-1.57079632679489678 0.13351607992219349796 -6.7670245197813334123e-17" />
             <geometry>
-                <mesh filename="file://$(find rover_description)/banksia/meshes/br_ankle.stl"/>
+                <mesh filename="file://$(find rover_description)/rover7/meshes/br_ankle.stl"/>
             </geometry>
             <material name="br_ankle_material">
@@ -492,5 +492,5 @@
             <origin xyz="5.5511151231257827021e-17 0 5.8763757748714340323e-17" rpy="1.4537948349788456791e-16 1.0501738044156386319e-16 -7.6074648532850333807e-21" />
             <geometry>
-                <mesh filename="file://$(find rover_description)/banksia/meshes/br_wheel.stl"/>
+                <mesh filename="file://$(find rover_description)/rover7/meshes/br_wheel.stl"/>
             </geometry>
             <material name="br_wheel_material">
@@ -515,5 +515,5 @@
             <origin xyz="4.9770590769729886024e-14 -0.00015426611885745872277 -0.010000000000000730527" rpy="1.570796326794896558 -3.0512890594788867116e-34 0" />
             <geometry>
-                <mesh filename="file://$(find rover_description)/banksia/meshes/diffbar.stl"/>
+                <mesh filename="file://$(find rover_description)/rover7/meshes/diffbar.stl"/>
             </geometry>
             <material name="diffbar_material">
@@ -544,5 +544,5 @@
             <origin xyz="-2.7755575615628913511e-15 -0.057750000000000162315 3.3306690738754696213e-16" rpy="1.5707963267948350516 -1.5127867282353739675 -3.1415926535897926719" />
             <geometry>
-                <mesh filename="file://$(find rover_description)/banksia/meshes/left_difflink.stl"/>
+                <mesh filename="file://$(find rover_description)/rover7/meshes/left_difflink.stl"/>
             </geometry>
             <material name="left_difflink_material">
@@ -567,5 +567,5 @@
             <origin xyz="6.2172489379008766264e-15 -0.057749999999999454547 -2.4424906541753443889e-15" rpy="1.5707963267948286123 1.512786629442331332 3.141592653589793116" />
             <geometry>
-                <mesh filename="file://$(find rover_description)/banksia/meshes/right_difflink.stl"/>
+                <mesh filename="file://$(find rover_description)/rover7/meshes/right_difflink.stl"/>
             </geometry>
             <material name="right_difflink_material">
@@ -682,5 +682,5 @@
     <!-- End of Generated URDF -->
     <!-- Include additional xacro files-->
-    <xacro:include filename="$(find rover_description)/banksia/urdf/ckc.xacro"/>
+    <xacro:include filename="$(find rover_description)/rover7/urdf/ckc.xacro"/>
     <xacro:if value="$(arg auto_camera)">
         <xacro:include filename="$(find rover_description)/auto_mount/urdf/auto_camera.xacro"/>
@@ -688,5 +688,5 @@
     </xacro:if>
     <xacro:if value="$(arg arm)">
-        <!-- Currently attaches waratah's arm, add banksia arm after ARCh-->
+        <!-- Currently attaches waratah's arm, add rover7 arm after ARCh-->
         <xacro:include filename="$(find rover_description)/waratah_arm/urdf/arm.urdf.xacro" />
         <joint name="chassis_to_arm_base" type="fixed">
@@ -697,13 +697,13 @@
     </xacro:if>
     <xacro:unless value="$(arg gazebo)">
-        <xacro:include filename="$(find rover_description)/banksia/urdf/ros2_control.xacro" />
+        <xacro:include filename="$(find rover_description)/rover7/urdf/ros2_control.xacro" />
         <xacro:rover_ros2_control use_mock_hardware="$(arg use_mock_hardware)"/>
     </xacro:unless>
     <xacro:if value="$(arg gazebo)">
-        <xacro:include filename="$(find rover_description)/banksia/urdf/gz_ros2_control.xacro" />
+        <xacro:include filename="$(find rover_description)/rover7/urdf/gz_ros2_control.xacro" />
     </xacro:if>
-    <xacro:include filename="$(find rover_description)/banksia/urdf/p3d.xacro"/>
-    <xacro:include filename="$(find rover_description)/banksia/urdf/odom.xacro"/>
-    <xacro:include filename="$(find rover_description)/banksia/urdf/gps.xacro"/>
-    <xacro:include filename="$(find rover_description)/banksia/urdf/joint_states.xacro"/>
+    <xacro:include filename="$(find rover_description)/rover7/urdf/p3d.xacro"/>
+    <xacro:include filename="$(find rover_description)/rover7/urdf/odom.xacro"/>
+    <xacro:include filename="$(find rover_description)/rover7/urdf/gps.xacro"/>
+    <xacro:include filename="$(find rover_description)/rover7/urdf/joint_states.xacro"/>
 </robot>

Commit message: fixed oak/bootie camera sensor plugins for gz; auto sim works

File: src/ros/rover/rover_description/auto_mount/urdf/auto_camera.xacro (robot description, xacro)
@@ -5,5 +5,4 @@
 <robot xmlns:xacro="http://www.ros.org/wiki/xacro">
   <xacro:macro name="auto_cam" params="angle">
-    <!-- Auto Mount start -->
     <link name="clam">
         <inertial>
@@ -120,7 +119,6 @@
         <limit effort="10" velocity="10" />
     </joint>
-    <!-- Auto Mount stop -->
     <link name="camera_link"/>
-    <link name="bootie_link"/> <!-- KABI OR SOMEONE ADD BOOTIE CAM GAZEBO SENSORS!!! -->
+    <link name="bootie_link"/>
     <joint name="oak_to_mount" type="fixed">
       <origin xyz="-0.120 0.004 0.039" rpy="1.5708 0 3.14159" />
@@ -161,4 +159,5 @@
       cam_yaw="0.0"
     />
+    <!-- EVERYTHING BELOW IS FOR SENSOR PLUGINS! REMOVE IF CAUSING PROBLEMS IRL -->
     <link name="camera_link_optical"/>
     <joint name="camera_optical_joint" type="fixed">
@@ -167,4 +166,60 @@
       <child link="camera_link_optical"/>
     </joint>
+    <link name="bootie_link_optical"/>
+    <joint name="bootie_optical_joint" type="fixed">
+      <origin xyz="0.0 0 0.0" rpy="${-pi/2} 0 ${-pi/2}"/>
+      <parent link="bootie_link"/>
+      <child link="bootie_link_optical"/>
+    </joint>
+    <!-- Oak Depth Camera for Gazebo-->
+    <gazebo reference="camera_link">
+      <sensor name="oak" type="rgbd_camera">
+        <plugin name="gz::sim::systems::Sensors" filename="gz-sim-sensors-system">
+          <frame_name>camera_link_optical</frame_name>
+        </plugin>
+        <gz_frame_id>camera_link_optical</gz_frame_id>
+        <optical_frame_id>camera_link</optical_frame_id>
+        <topic>oak</topic>
+        <visualize>true</visualize>
+        <update_rate>30</update_rate>
+        <always_on>1</always_on>
+        <camera name="oak">
+          <horizontal_fov>${radians(82)}</horizontal_fov>
+          <image>
+            <width>1280</width>
+            <height>900</height>
+          </image>
+          <clip>
+            <near>0.4</near>
+            <far>10.0</far>
+          </clip>
+        </camera>
+      </sensor>
+    </gazebo>
+    <!-- Bootie Depth Camera for Gazebo-->
+    <gazebo reference="bootie_link">
+      <sensor name="bootie" type="rgbd_camera">
+        <!-- <plugin name="gz::sim::systems::Sensors" filename="gz-sim-sensors-system">
+          <frame_name>bootie_link_optical</frame_name>
+        </plugin> -->
+        <gz_frame_id>bootie_link_optical</gz_frame_id>
+        <optical_frame_id>bootie_link</optical_frame_id>
+        <topic>bootie</topic>
+        <visualize>true</visualize>
+        <update_rate>30</update_rate>
+        <always_on>1</always_on>
+        <camera name="bootie">
+          <horizontal_fov>${radians(82)}</horizontal_fov>
+          <image>
+            <width>1280</width>
+            <height>900</height>
+          </image>
+          <clip>
+            <near>0.4</near>
+            <far>10.0</far>
+          </clip>
+        </camera>
+      </sensor>
+    </gazebo>
   </xacro:macro>
 </robot>

Commit message: feat: Simplified collisions for auto_mount

File: src/ros/rover/rover_description/auto_mount/urdf/auto_camera.xacro (robot description, xacro)
@@ -21,7 +21,31 @@
         </visual>
         <collision>
-            <origin xyz="0.138856 0.281 0.00511278" rpy="3.14159 -0.00348764 3.3577e-34" />
-            <geometry>
-                <mesh filename="file://$(find rover_description)/auto_mount/meshes/clam.stl" />
+            <origin xyz="0.138821 0.291 0.0151127" rpy="3.14159 -0.00348764 3.3577e-34"/>
+            <geometry>
+                <box size="0.3 0.02 0.06"/>
+            </geometry>
+        </collision>
+        <collision>
+            <origin xyz="0.278786 0.171 0.0256009" rpy="3.14159 -0.00348764 3.3577e-34"/>
+            <geometry>
+                <box size="0.02 0.25 0.04"/>
+            </geometry>
+        </collision>
+        <collision>
+            <origin xyz="-0.00121269 0.171 0.0246244" rpy="3.14159 -0.00348764 3.3577e-34"/>
+            <geometry>
+                <box size="0.02 0.25 0.04"/>
+            </geometry>
+        </collision>
+        <collision>
+            <origin xyz="0.0650716 0.3285 -0.200146" rpy="3.14159 3.01669e-06 -4.11764e-18"/>
+            <geometry>
+                <cylinder length="0.5" radius="0.013"/>
+            </geometry>
+        </collision>
+        <collision>
+            <origin xyz="0.226671 0.3285 -0.199582" rpy="3.14159 3.01669e-06 -4.11764e-18"/>
+            <geometry>
+                <cylinder length="0.5" radius="0.013"/>
             </geometry>
         </collision>
@@ -43,7 +67,7 @@
         </visual>
         <collision>
-            <origin xyz="0.081 0.000713936 -0.025" rpy="4.93038e-32 6.86401e-31 -3.70732e-33" />
-            <geometry>
-                <mesh filename="file://$(find rover_description)/auto_mount/meshes/mount.stl" />
+            <origin xyz="0.081 0.000713936 -0.025" rpy="4.93038e-32 6.86401e-31 -3.70732e-33"/>
+            <geometry>
+                <box size="0.2 0.04 0.05"/>
             </geometry>
         </collision>
@@ -65,7 +89,7 @@
         </visual>
         <collision>
-            <origin xyz="-0.075 5.55112e-17 0.06" rpy="-1.5708 -1.5708 0" />
-            <geometry>
-                <mesh filename="file://$(find rover_description)/auto_mount/meshes/camera_holder.stl" />
+            <origin xyz="-0.04 5.55112e-17 0.06" rpy="-1.5708 -1.5708 0"/>
+            <geometry>
+                <box size="0.143 0.086 0.05"/>
             </geometry>
         </collision>
@@ -93,7 +117,7 @@
         </visual>
         <collision>
-            <origin xyz="-0.075 0 0.06" rpy="1.5708 1.5708 0" />
-            <geometry>
-                <mesh filename="file://$(find rover_description)/auto_mount/meshes/camera_holder.stl" />
+            <origin xyz="-0.04 8.62817e-34 0.06" rpy="1.5708 1.5708 0"/>
+            <geometry>
+                <box size="0.143 0.086 0.05"/>
             </geometry>
         </collision>
