Commit message: Add local_path param to xacro

File: src/ros/rover/rover_description/rover7/urdf/rover.urdf.xacro (robot description, xacro)
@@ -13,8 +13,17 @@
     <xacro:arg name="robot_name" default="rover7"/>
     <xacro:arg name="angle" default="0"/>
+    <xacro:arg name="use_local_mesh" default="false"/>
     <!-- Robot properties-->
     <gazebo>
         <self_collide>false</self_collide>
     </gazebo>
+    <!-- Variables -->
+    <xacro:if value="$(arg use_local_mesh)">
+        <xacro:property name="mesh_path" value="file://home/nova/nova/src/ros/rover/rover_description" />
+    </xacro:if>
+    <xacro:unless value="$(arg use_local_mesh)">
+        <xacro:property name="mesh_path" value="file://$(find rover_description)" />
+    </xacro:unless>
+    <xacro:property name="angle" value="$(arg angle)" />
     <!-- Generated URDF -->
     <link name="base_link"></link>
@@ -28,5 +37,5 @@
             <origin xyz="0 0 0" rpy="3.26128e-16 -1.01395e-15 1.5708" />
             <geometry>
-                <mesh filename="file://$(find rover_description)/rover7/meshes/chassis.stl" />
+                <mesh filename="${mesh_path}/rover7/meshes/chassis.stl" />
             </geometry>
             <material name="chassis_material">
@@ -45,5 +54,5 @@
             <origin xyz="-1.3078806732583218725e-20 8.6736173798840354721e-19 -0.021000000000000518252" rpy="-3.141592653589793116 6.2280032059897877693e-19 -4.1232880706353110482e-18" />
             <geometry>
-                <mesh filename="file://$(find rover_description)/rover7/meshes/left_leg.stl"/>
+                <mesh filename="${mesh_path}/rover7/meshes/left_leg.stl"/>
             </geometry>
             <material name="left_leg_material">
@@ -116,5 +125,5 @@
             <origin xyz="-0.12415341931613717297 2.2204460492503130808e-16 -0.1250000000000002498" rpy="-1.570796326794896558 -0.13351607992219349796 -5.9804098682663148249e-17" />
             <geometry>
-                <mesh filename="file://$(find rover_description)/rover7/meshes/fl_ankle.stl"/>
+                <mesh filename="${mesh_path}/rover7/meshes/fl_ankle.stl"/>
             </geometry>
             <material name="fl_ankle_material">
@@ -175,5 +184,5 @@
             <origin xyz="5.5511151231257827021e-17 0 5.963111948670274387e-18" rpy="7.279848939407052303e-17 1.0638440422271473935e-16 -6.3914183266779029169e-20" />
             <geometry>
-                <mesh filename="file://$(find rover_description)/rover7/meshes/fl_wheel.stl"/>
+                <mesh filename="${mesh_path}/rover7/meshes/fl_wheel.stl"/>
             </geometry>
             <material name="fl_wheel_material">
@@ -198,5 +207,5 @@
             <origin xyz="-0.12415341931613714521 2.2204460492503130808e-16 -0.1250000000000002498" rpy="-1.570796326794896558 -0.13351607992219349796 -7.1088909477657821376e-17" />
             <geometry>
-                <mesh filename="file://$(find rover_description)/rover7/meshes/bl_ankle.stl"/>
+                <mesh filename="${mesh_path}/rover7/meshes/bl_ankle.stl"/>
             </geometry>
             <material name="bl_ankle_material">
@@ -257,5 +266,5 @@
             <origin xyz="0 1.1102230246251565404e-16 1.7780915628762272718e-17" rpy="4.6040217445536182725e-17 1.0513492286565858337e-16 2.3412503191653332746e-19" />
             <geometry>
-                <mesh filename="file://$(find rover_description)/rover7/meshes/bl_wheel.stl"/>
+                <mesh filename="${mesh_path}/rover7/meshes/bl_wheel.stl"/>
             </geometry>
             <material name="bl_wheel_material">
@@ -280,5 +289,5 @@
             <origin xyz="-7.9461177221465168975e-19 -7.2858385990954703269e-20 -0.020999999999999519051" rpy="3.141592653589793116 3.7838655819744092421e-17 -5.8406613147999892266e-19" />
             <geometry>
-                <mesh filename="file://$(find rover_description)/rover7/meshes/right_leg.stl"/>
+                <mesh filename="${mesh_path}/rover7/meshes/right_leg.stl"/>
             </geometry>
             <material name="right_leg_material">
@@ -351,5 +360,5 @@
             <origin xyz="0.12415341931613695092 -2.2204460492503130808e-16 -0.12500000000000027756" rpy="-1.57079632679489678 0.13351607992219352572 9.9507186100571649487e-18" />
             <geometry>
-                <mesh filename="file://$(find rover_description)/rover7/meshes/fr_ankle.stl"/>
+                <mesh filename="${mesh_path}/rover7/meshes/fr_ankle.stl"/>
             </geometry>
             <material name="fr_ankle_material">
@@ -410,5 +419,5 @@
             <origin xyz="5.5511151231257827021e-17 -1.1102230246251565404e-16 -3.0791341698588325926e-17" rpy="-3.6194812825998444115e-17 1.0511409763610977507e-16 -2.2325341479697011877e-19" />
             <geometry>
-                <mesh filename="file://$(find rover_description)/rover7/meshes/fr_wheel.stl"/>
+                <mesh filename="${mesh_path}/rover7/meshes/fr_wheel.stl"/>
             </geometry>
             <material name="fr_wheel_material">
@@ -433,5 +442,5 @@
             <origin xyz="0.12415341931613720072 -2.2204460492503130808e-16 -0.12500000000000027756" rpy="-1.57079632679489678 0.13351607992219349796 -6.7670245197813334123e-17" />
             <geometry>
-                <mesh filename="file://$(find rover_description)/rover7/meshes/br_ankle.stl"/>
+                <mesh filename="${mesh_path}/rover7/meshes/br_ankle.stl"/>
             </geometry>
             <material name="br_ankle_material">
@@ -492,5 +501,5 @@
             <origin xyz="5.5511151231257827021e-17 0 5.8763757748714340323e-17" rpy="1.4537948349788456791e-16 1.0501738044156386319e-16 -7.6074648532850333807e-21" />
             <geometry>
-                <mesh filename="file://$(find rover_description)/rover7/meshes/br_wheel.stl"/>
+                <mesh filename="${mesh_path}/rover7/meshes/br_wheel.stl"/>
             </geometry>
             <material name="br_wheel_material">
@@ -515,5 +524,5 @@
             <origin xyz="4.9770590769729886024e-14 -0.00015426611885745872277 -0.010000000000000730527" rpy="1.570796326794896558 -3.0512890594788867116e-34 0" />
             <geometry>
-                <mesh filename="file://$(find rover_description)/rover7/meshes/diffbar.stl"/>
+                <mesh filename="${mesh_path}/rover7/meshes/diffbar.stl"/>
             </geometry>
             <material name="diffbar_material">
@@ -544,5 +553,5 @@
             <origin xyz="-2.7755575615628913511e-15 -0.057750000000000162315 3.3306690738754696213e-16" rpy="1.5707963267948350516 -1.5127867282353739675 -3.1415926535897926719" />
             <geometry>
-                <mesh filename="file://$(find rover_description)/rover7/meshes/left_difflink.stl"/>
+                <mesh filename="${mesh_path}/rover7/meshes/left_difflink.stl"/>
             </geometry>
             <material name="left_difflink_material">
@@ -567,5 +576,5 @@
             <origin xyz="6.2172489379008766264e-15 -0.057749999999999454547 -2.4424906541753443889e-15" rpy="1.5707963267948286123 1.512786629442331332 3.141592653589793116" />
             <geometry>
-                <mesh filename="file://$(find rover_description)/rover7/meshes/right_difflink.stl"/>
+                <mesh filename="${mesh_path}/rover7/meshes/right_difflink.stl"/>
             </geometry>
             <material name="right_difflink_material">
@@ -684,6 +693,5 @@
     <xacro:include filename="$(find rover_description)/rover7/urdf/ckc.xacro"/>
     <xacro:if value="$(arg auto_camera)">
-        <xacro:include filename="$(find rover_description)/auto_mount/urdf/auto_camera.xacro"/>
-        <xacro:auto_cam angle="$(arg angle)"></xacro:auto_cam>
+        <xacro:include filename="/home/nova/nova/src/ros/rover/rover_description/auto_mount/urdf/auto_camera.xacro"/>
     </xacro:if>
     <xacro:if value="$(arg arm)">

Commit message: fix: gazebo sensor cameras and add frame for pointcloud transform using custom node to change header frame_id

File: src/ros/rover/rover_description/auto_mount/urdf/auto_camera.xacro (robot description, xacro)
@@ -195,12 +195,23 @@
     <child link="bootie_link_optical"/>
   </joint>
+  <!-- Used in conjuction with gz_header_republisher to fix pointcloud frame transform-->
+  <link name="camera_link_gz_pointcloud"/>
+  <link name="bootie_link_gz_pointcloud"/>
+  <joint name="camera_pointcloud_joint" type="fixed">
+    <origin xyz="0 0 0" rpy="0 ${-pi/2} 0"/>
+    <parent link="camera_link_optical"/>
+    <child link="camera_link_gz_pointcloud"/>
+  </joint>
+  <joint name="bootie_pointcloud_joint" type="fixed">
+    <origin xyz="0 0 0" rpy="0 ${-pi/2} 0"/>
+    <parent link="bootie_link_optical"/>
+    <child link="bootie_link_gz_pointcloud"/>
+  </joint>
   <!-- Oak Depth Camera for Gazebo-->
-  <gazebo reference="camera_link">
+  <gazebo reference="camera_link_optical">
     <sensor name="oak" type="rgbd_camera">
-      <plugin name="gz::sim::systems::Sensors" filename="gz-sim-sensors-system">
-        <frame_name>camera_link_optical</frame_name>
-      </plugin>
+      <pose> 0 0 0 0 ${-pi/2} 0 </pose> <!-- Get camera facing correct way in optical frame -->
+      <plugin name="gz::sim::systems::Sensors" filename="gz-sim-sensors-system"></plugin>
       <gz_frame_id>camera_link_optical</gz_frame_id>
-      <optical_frame_id>camera_link</optical_frame_id>
       <topic>oak</topic>
       <visualize>true</visualize>
@@ -221,11 +232,11 @@
   </gazebo>
   <!-- Bootie Depth Camera for Gazebo-->
-  <gazebo reference="bootie_link">
+  <gazebo reference="bootie_link_optical">
     <sensor name="bootie" type="rgbd_camera">
+      <pose> 0 0 0 0 ${-pi/2} 0 </pose> <!-- Get camera facing correct way in optical frame -->
       <!-- <plugin name="gz::sim::systems::Sensors" filename="gz-sim-sensors-system">
         <frame_name>bootie_link_optical</frame_name>
       </plugin> -->
       <gz_frame_id>bootie_link_optical</gz_frame_id>
-      <optical_frame_id>bootie_link</optical_frame_id>
       <topic>bootie</topic>
       <visualize>true</visualize>

Commit message: fix: Gazebo sensor cameras rotated + add point cloud topics to nav2_urc

File: src/ros/rover/rover_description/auto_mount/urdf/auto_camera.xacro (robot description, xacro)
@@ -199,10 +199,10 @@
   <link name="bootie_link_gz_pointcloud"/>
   <joint name="camera_pointcloud_joint" type="fixed">
-    <origin xyz="0 0 0" rpy="0 ${-pi/2} 0"/>
+    <origin xyz="0 0 0" rpy="0 ${-pi/2} ${pi/2}"/>
     <parent link="camera_link_optical"/>
     <child link="camera_link_gz_pointcloud"/>
   </joint>
   <joint name="bootie_pointcloud_joint" type="fixed">
-    <origin xyz="0 0 0" rpy="0 ${-pi/2} 0"/>
+    <origin xyz="0 0 0" rpy="0 ${-pi/2} ${pi/2}"/>
     <parent link="bootie_link_optical"/>
     <child link="bootie_link_gz_pointcloud"/>
@@ -211,5 +211,5 @@
   <gazebo reference="camera_link_optical">
     <sensor name="oak" type="rgbd_camera">
-      <pose> 0 0 0 0 ${-pi/2} 0 </pose> <!-- Get camera facing correct way in optical frame -->
+      <pose> 0 0 0 0 ${-pi/2} ${pi/2} </pose> <!-- Get camera facing correct way in optical frame -->
       <plugin name="gz::sim::systems::Sensors" filename="gz-sim-sensors-system"></plugin>
       <gz_frame_id>camera_link_optical</gz_frame_id>
@@ -234,5 +234,5 @@
   <gazebo reference="bootie_link_optical">
     <sensor name="bootie" type="rgbd_camera">
-      <pose> 0 0 0 0 ${-pi/2} 0 </pose> <!-- Get camera facing correct way in optical frame -->
+      <pose> 0 0 0 0 ${-pi/2} ${pi/2} </pose> <!-- Get camera facing correct way in optical frame -->
       <!-- <plugin name="gz::sim::systems::Sensors" filename="gz-sim-sensors-system">
         <frame_name>bootie_link_optical</frame_name>

Commit message: Adding STVL to Nav2 (#462)
Co-authored-by: Victor Bartlinski <vicbart08@gmail.com>

File: src/ros/rover/rover_description/auto_mount/urdf/auto_camera.xacro (robot description, xacro)
@@ -195,12 +195,23 @@
     <child link="bootie_link_optical"/>
   </joint>
+  <!-- Used in conjuction with gz_header_republisher to fix pointcloud frame transform-->
+  <link name="camera_link_gz_pointcloud"/>
+  <link name="bootie_link_gz_pointcloud"/>
+  <joint name="camera_pointcloud_joint" type="fixed">
+    <origin xyz="0 0 0" rpy="0 ${-pi/2} ${pi/2}"/>
+    <parent link="camera_link_optical"/>
+    <child link="camera_link_gz_pointcloud"/>
+  </joint>
+  <joint name="bootie_pointcloud_joint" type="fixed">
+    <origin xyz="0 0 0" rpy="0 ${-pi/2} ${pi/2}"/>
+    <parent link="bootie_link_optical"/>
+    <child link="bootie_link_gz_pointcloud"/>
+  </joint>
   <!-- Oak Depth Camera for Gazebo-->
-  <gazebo reference="camera_link">
+  <gazebo reference="camera_link_optical">
     <sensor name="oak" type="rgbd_camera">
-      <plugin name="gz::sim::systems::Sensors" filename="gz-sim-sensors-system">
-        <frame_name>camera_link_optical</frame_name>
-      </plugin>
+      <pose> 0 0 0 0 ${-pi/2} ${pi/2} </pose> <!-- Get camera facing correct way in optical frame -->
+      <plugin name="gz::sim::systems::Sensors" filename="gz-sim-sensors-system"></plugin>
       <gz_frame_id>camera_link_optical</gz_frame_id>
-      <optical_frame_id>camera_link</optical_frame_id>
       <topic>oak</topic>
       <visualize>true</visualize>
@@ -221,11 +232,11 @@
   </gazebo>
   <!-- Bootie Depth Camera for Gazebo-->
-  <gazebo reference="bootie_link">
+  <gazebo reference="bootie_link_optical">
     <sensor name="bootie" type="rgbd_camera">
+      <pose> 0 0 0 0 ${-pi/2} ${pi/2} </pose> <!-- Get camera facing correct way in optical frame -->
       <!-- <plugin name="gz::sim::systems::Sensors" filename="gz-sim-sensors-system">
         <frame_name>bootie_link_optical</frame_name>
       </plugin> -->
       <gz_frame_id>bootie_link_optical</gz_frame_id>
-      <optical_frame_id>bootie_link</optical_frame_id>
       <topic>bootie</topic>
       <visualize>true</visualize>

Commit message: getting gps integrated with auto, WIP, rover currently flies away when using GPS

File: src/ros/rover/rover_description/auto_mount/urdf/auto_camera.xacro (robot description, xacro)
@@ -256,3 +256,130 @@
     </sensor>
   </gazebo>
+  <gazebo reference="base_link">
+    <sensor name="oak_imu_sensor" type="imu">
+      <topic>oak/imu</topic>
+      <plugin filename="gz-sim-imu-system" name="gz::sim::systems::Imu"></plugin>
+      <gz_frame_id>base_link</gz_frame_id>
+      <always_on>true</always_on>
+      <update_rate>200</update_rate>
+      <visualize>true</visualize>
+      <imu>
+        <angular_velocity>
+          <x>
+            <noise type="gaussian">
+              <mean>0.0</mean>
+              <stddev>0.0</stddev>
+              <bias_mean>0.0</bias_mean>
+              <bias_stddev>0.0</bias_stddev>
+            </noise>
+          </x>
+          <y>
+            <noise type="gaussian">
+              <mean>0.0</mean>
+              <stddev>0.0</stddev>
+              <bias_mean>0.0</bias_mean>
+              <bias_stddev>0.0</bias_stddev>
+            </noise>
+          </y>
+          <z>
+            <noise type="gaussian">
+              <mean>0.0</mean>
+              <stddev>0.0</stddev>
+              <bias_mean>0.0</bias_mean>
+              <bias_stddev>0.0</bias_stddev>
+            </noise>
+          </z>
+        </angular_velocity>
+        <linear_acceleration>
+          <x>
+            <noise type="gaussian">
+              <mean>0.0</mean>
+              <stddev>0.0</stddev>
+              <bias_mean>0.0</bias_mean>
+              <bias_stddev>0.0</bias_stddev>
+            </noise>
+          </x>
+          <y>
+            <noise type="gaussian">
+              <mean>0.0</mean>
+              <stddev>0.0</stddev>
+              <bias_mean>0.0</bias_mean>
+              <bias_stddev>0.0</bias_stddev>
+            </noise>
+          </y>
+          <z>
+            <noise type="gaussian">
+              <mean>0.0</mean>
+              <stddev>0.0</stddev>
+              <bias_mean>0.0</bias_mean>
+              <bias_stddev>0.0</bias_stddev>
+            </noise>
+          </z>
+        </linear_acceleration>
+      </imu>
+    </sensor>
+  </gazebo>
+  <gazebo reference="base_link">
+    <sensor name="bootie_imu_sensor" type="imu">
+      <topic>bootie/imu</topic>
+      <gz_frame_id>base_link</gz_frame_id>
+      <always_on>true</always_on>
+      <update_rate>200</update_rate>
+      <visualize>true</visualize>
+      <imu>
+        <angular_velocity>
+          <x>
+            <noise type="gaussian">
+              <mean>0.0</mean>
+              <stddev>0.0</stddev>
+              <bias_mean>0.0</bias_mean>
+              <bias_stddev>0.0</bias_stddev>
+            </noise>
+          </x>
+          <y>
+            <noise type="gaussian">
+              <mean>0.0</mean>
+              <stddev>0.0</stddev>
+              <bias_mean>0.0</bias_mean>
+              <bias_stddev>0.0</bias_stddev>
+            </noise>
+          </y>
+          <z>
+            <noise type="gaussian">
+              <mean>0.0</mean>
+              <stddev>0.0</stddev>
+              <bias_mean>0.0</bias_mean>
+              <bias_stddev>0.0</bias_stddev>
+            </noise>
+          </z>
+        </angular_velocity>
+        <linear_acceleration>
+          <x>
+            <noise type="gaussian">
+              <mean>0.0</mean>
+              <stddev>0.0</stddev>
+              <bias_mean>0.0</bias_mean>
+              <bias_stddev>0.0</bias_stddev>
+            </noise>
+          </x>
+          <y>
+            <noise type="gaussian">
+              <mean>0.0</mean>
+              <stddev>0.0</stddev>
+              <bias_mean>0.0</bias_mean>
+              <bias_stddev>0.0</bias_stddev>
+            </noise>
+          </y>
+          <z>
+            <noise type="gaussian">
+              <mean>0.0</mean>
+              <stddev>0.0</stddev>
+              <bias_mean>0.0</bias_mean>
+              <bias_stddev>0.0</bias_stddev>
+            </noise>
+          </z>
+        </linear_acceleration>
+      </imu>
+    </sensor>
+  </gazebo>
 </robot>

File: src/ros/rover/rover_description/banksia/urdf/gps.xacro (robot description, xacro)
@@ -4,19 +4,4 @@
 <robot xmlns:xacro="http://www.ros.org/wiki/xacro" >
   <link name="gps">
-    <!--
-    <inertial>
-      <pose>-0.052 0 0.111 0 0 0</pose>
-      <inertia>
-        <mass>0.001</mass>
-        <ixx>0.001</ixx>
-        <ixy>0.000</ixy>
-        <ixz>0.000</ixz>
-        <iyy>0.001</iyy>
-        <iyz>0.000</iyz>
-        <izz>0.001</izz>
-      </inertia>
-      <mass>0.125</mass>
-    </inertial>
-    -->
   </link>
   <joint name="gps_joint" type="fixed">
@@ -26,5 +11,5 @@
   </joint>
   <gazebo reference="gps">
-    <sensor name="skytraq_gps" type="gps">
+    <sensor name="gps_rover" type="navsat">
       <topic>gps</topic>
       <plugin
@@ -32,6 +17,7 @@
         name="gz::sim::systems::NavSat">
       </plugin>
+      <gz_frame_id>gps</gz_frame_id>
       <always_on>true</always_on>
-      <update_rate>1</update_rate>
+      <update_rate>30</update_rate>
       <gps>
         <position_sensing>
@@ -39,5 +25,5 @@
             <noise type="gaussian">
               <mean>0.0</mean>
-              <stddev>0.01</stddev>
+              <stddev>0.0</stddev>
             </noise>
           </horizontal>
@@ -45,8 +31,22 @@
             <noise type="gaussian">
               <mean>0.0</mean>
-              <stddev>0.01</stddev>
+              <stddev>0.0</stddev>
             </noise>
           </vertical>
         </position_sensing>
+        <velocity_sensing>
+          <horizontal>
+            <noise type="gaussian">
+              <mean>0.0</mean>
+              <stddev>0.0</stddev>
+            </noise>
+          </horizontal>
+          <vertical>
+            <noise type="gaussian">
+              <mean>0.0</mean>
+              <stddev>0.0</stddev>
+            </noise>
+          </vertical>
+        </velocity_sensing>
       </gps>
     </sensor>

Commit message: Fixed GPS (#505)
Co-authored-by: Monash Nova Rover <novaroverteam@monash.edu>
Co-authored-by: Anthony Lew <anthony@v01dbreaker.cc>

File: src/ros/rover/rover_description/auto_mount/urdf/auto_camera.xacro (robot description, xacro)
@@ -256,3 +256,22 @@
     </sensor>
   </gazebo>
+  <gazebo reference="base_link">
+    <sensor name="oak_imu_sensor" type="imu">
+      <topic>oak/imu</topic>
+      <plugin filename="gz-sim-imu-system" name="gz::sim::systems::Imu"></plugin>
+      <gz_frame_id>base_link</gz_frame_id>
+      <always_on>true</always_on>
+      <update_rate>100</update_rate>
+      <visualize>true</visualize>
+    </sensor>
+  </gazebo>
+  <gazebo reference="base_link">
+    <sensor name="bootie_imu_sensor" type="imu">
+      <topic>bootie/imu</topic>
+      <gz_frame_id>base_link</gz_frame_id>
+      <always_on>true</always_on>
+      <update_rate>100</update_rate>
+      <visualize>true</visualize>
+    </sensor>
+  </gazebo>
 </robot>

File: src/ros/rover/rover_description/banksia/urdf/gps.xacro (robot description, xacro)
@@ -4,27 +4,12 @@
 <robot xmlns:xacro="http://www.ros.org/wiki/xacro" >
   <link name="gps">
-    <!--
-    <inertial>
-      <pose>-0.052 0 0.111 0 0 0</pose>
-      <inertia>
-        <mass>0.001</mass>
-        <ixx>0.001</ixx>
-        <ixy>0.000</ixy>
-        <ixz>0.000</ixz>
-        <iyy>0.001</iyy>
-        <iyz>0.000</iyz>
-        <izz>0.001</izz>
-      </inertia>
-      <mass>0.125</mass>
-    </inertial>
-    -->
   </link>
   <joint name="gps_joint" type="fixed">
     <parent link="base_link"/>
     <child link="gps"/>
-    <origin xyz="0.04 -0.26 0.614" rpy="0 0 0"/>
+    <origin xyz="0 0 0" rpy="0 0 0"/>
   </joint>
   <gazebo reference="gps">
-    <sensor name="skytraq_gps" type="gps">
+    <sensor name="gps_rover" type="navsat">
       <topic>gps</topic>
       <plugin
@@ -32,6 +17,7 @@
         name="gz::sim::systems::NavSat">
       </plugin>
+      <gz_frame_id>gps</gz_frame_id>
       <always_on>true</always_on>
-      <update_rate>1</update_rate>
+      <update_rate>30</update_rate>
       <gps>
         <position_sensing>
@@ -39,5 +25,5 @@
             <noise type="gaussian">
               <mean>0.0</mean>
-              <stddev>0.01</stddev>
+              <stddev>0.0</stddev>
             </noise>
           </horizontal>
@@ -45,8 +31,22 @@
             <noise type="gaussian">
               <mean>0.0</mean>
-              <stddev>0.01</stddev>
+              <stddev>0.0</stddev>
             </noise>
           </vertical>
         </position_sensing>
+        <velocity_sensing>
+          <horizontal>
+            <noise type="gaussian">
+              <mean>0.0</mean>
+              <stddev>0.0</stddev>
+            </noise>
+          </horizontal>
+          <vertical>
+            <noise type="gaussian">
+              <mean>0.0</mean>
+              <stddev>0.0</stddev>
+            </noise>
+          </vertical>
+        </velocity_sensing>
       </gps>
     </sensor>
