Commit message: added magnetometers and changed all camera references to oak

File: src/ros/rover/rover_description/auto_mount/urdf/auto_camera.xacro (robot description, xacro)
@@ -142,10 +142,10 @@
       <limit effort="10" velocity="10" />
   </joint>
-  <link name="camera_link"/>
+  <link name="oak_link"/>
   <link name="bootie_link"/>
   <joint name="oak_to_mount" type="fixed">
     <origin xyz="-0.120 0.004 0.039" rpy="1.5708 0 3.14159" />
     <parent link="camera_holder_front" />
-    <child link="camera_link" />
+    <child link="oak_link" />
     <axis xyz="0 0 1" />
   </joint>
@@ -159,5 +159,5 @@
   <xacro:depthai_camera
     camera_name="oak"
-    parent="camera_link"
+    parent="oak_link"
     camera_model="OAK-D-LR"
     base_frame="oak-base-frame"
@@ -183,9 +183,9 @@
   />
   <!-- EVERYTHING BELOW IS FOR SENSOR PLUGINS! REMOVE IF CAUSING PROBLEMS IRL -->
-  <link name="camera_link_optical"/>
-  <joint name="camera_optical_joint" type="fixed">
+  <link name="oak_link_optical"/>
+  <joint name="oak_optical_joint" type="fixed">
     <origin xyz="0.0 0 0.0" rpy="${-pi/2} 0 ${-pi/2}"/>
-    <parent link="camera_link"/>
-    <child link="camera_link_optical"/>
+    <parent link="oak_link"/>
+    <child link="oak_link_optical"/>
   </joint>
   <link name="bootie_link_optical"/>
@@ -196,11 +196,11 @@
   </joint>
   <!-- Used in conjuction with gz_header_republisher to fix pointcloud frame transform-->
-  <link name="camera_link_gz_pointcloud"/>
+  <link name="oak_link_gz_pointcloud"/>
+  <joint name="oak_pointcloud_joint" type="fixed">
+    <origin xyz="0 0 0" rpy="0 ${-pi/2} ${pi/2}"/>
+    <parent link="oak_link_optical"/>
+    <child link="oak_link_gz_pointcloud"/>
+  </joint>
   <link name="bootie_link_gz_pointcloud"/>
-  <joint name="camera_pointcloud_joint" type="fixed">
-    <origin xyz="0 0 0" rpy="0 ${-pi/2} ${pi/2}"/>
-    <parent link="camera_link_optical"/>
-    <child link="camera_link_gz_pointcloud"/>
-  </joint>
   <joint name="bootie_pointcloud_joint" type="fixed">
     <origin xyz="0 0 0" rpy="0 ${-pi/2} ${pi/2}"/>
@@ -209,9 +209,9 @@
   </joint>
   <!-- Oak Depth Camera for Gazebo-->
-  <gazebo reference="camera_link_optical">
+  <gazebo reference="oak_link_optical">
     <sensor name="oak" type="rgbd_camera">
       <pose> 0 0 0 0 ${-pi/2} ${pi/2} </pose> <!-- Get camera facing correct way in optical frame -->
       <plugin name="gz::sim::systems::Sensors" filename="gz-sim-sensors-system"></plugin>
-      <gz_frame_id>camera_link_optical</gz_frame_id>
+      <gz_frame_id>oak_link_optical</gz_frame_id>
       <topic>oak</topic>
       <visualize>true</visualize>

File: src/ros/rover/rover_description/waratah/urdf/auto_camera.xacro (robot description, xacro)
@@ -3,12 +3,12 @@
 which is how it gets added to the gazebo sim. Author/s: Victor Bartlinski-->
 <robot xmlns:xacro="http://www.ros.org/wiki/xacro" >
-  <link name='camera_link'></link>
+  <link name='oak_link'></link>
   <joint name="camera_joint" type="fixed">
     <origin xyz="0.49 0 0.48" rpy="0 0 0" />
     <parent link="base_link" />
-    <child link="camera_link" />
+    <child link="oak_link" />
   </joint>
   <xacro:include filename="$(find depthai_descriptions)/urdf/include/depthai_macro.urdf.xacro"/>
-  <xacro:depthai_camera camera_name = "oak" parent = "camera_link" camera_model = "OAK-D-LR"
+  <xacro:depthai_camera camera_name = "oak" parent = "oak_link" camera_model = "OAK-D-LR"
    base_frame = "oak-d_frame" cam_pos_x = "0.0" cam_pos_y = "0.0" cam_pos_z = "0.0"
    cam_roll = "0.0" cam_pitch = "0.0" cam_yaw = "0.0"/>
@@ -16,5 +16,5 @@
     <sensor name="oak/stereo" type="depth_camera">
       <topic>oak/depth</topic>
-      <gz_frame_id>camera_link</gz_frame_id> <!-- Sets the frame_id so that rviz2 correctly transforms it -->
+      <gz_frame_id>oak_link</gz_frame_id> <!-- Sets the frame_id so that rviz2 correctly transforms it -->
       <visualize>true</visualize>
       <update_rate>30</update_rate>

Commit message: Remove use_local_mesh (It didn't work). Add camera disable option for gazebo

File: src/ros/rover/rover_description/auto_mount/urdf/auto_camera.xacro (robot description, xacro)
@@ -13,5 +13,5 @@
           <origin xyz="0.138856 0.281 0.00511278" rpy="3.14159 -0.00348764 3.3577e-34" />
           <geometry>
-              <mesh filename="${mesh_path}/auto_mount/meshes/clam.stl" />
+              <mesh filename="file://$(find rover_description)/auto_mount/meshes/clam.stl" />
           </geometry>
           <material name="clam_material">
@@ -59,5 +59,5 @@
           <origin xyz="0.081 0.000713936 -0.025" rpy="4.93038e-32 6.86401e-31 -3.70732e-33" />
           <geometry>
-              <mesh filename="${mesh_path}/auto_mount/meshes/mount.stl" />
+              <mesh filename="file://$(find rover_description)/auto_mount/meshes/mount.stl" />
           </geometry>
           <material name="mount_material">
@@ -81,5 +81,5 @@
           <origin xyz="-0.075 5.55112e-17 0.06" rpy="-1.5708 -1.5708 0" />
           <geometry>
-              <mesh filename="${mesh_path}/auto_mount/meshes/camera_holder.stl" />
+              <mesh filename="file://$(find rover_description)/auto_mount/meshes/camera_holder.stl" />
           </geometry>
           <material name="camera_holder_front_material">
@@ -109,5 +109,5 @@
           <origin xyz="-0.075 0 0.06" rpy="1.5708 1.5708 0" />
           <geometry>
-              <mesh filename="${mesh_path}/auto_mount/meshes/camera_holder.stl" />
+              <mesh filename="file://$(find rover_description)/auto_mount/meshes/camera_holder.stl" />
           </geometry>
           <material name="camera_holder_back_material">

File: src/ros/rover/rover_description/banksia/urdf/rover.urdf.xacro (robot description, xacro)
@@ -14,5 +14,4 @@
     <xacro:arg name="robot_name" default="Banksia"/>
     <xacro:arg name="angle" default="0"/>
-    <xacro:arg name="use_local_mesh" default="false"/>
     <!-- Robot properties-->
     <gazebo>
@@ -20,10 +19,4 @@
     </gazebo>
     <!-- Variables -->
-    <xacro:if value="$(arg use_local_mesh)">
-        <xacro:property name="mesh_path" value="file://home/nova/nova/src/ros/rover/rover_description" />
-    </xacro:if>
-    <xacro:unless value="$(arg use_local_mesh)">
-        <xacro:property name="mesh_path" value="file://$(find rover_description)" />
-    </xacro:unless>
     <xacro:property name="angle" value="$(arg angle)" />
     <!-- Generated URDF -->
@@ -38,5 +31,5 @@
             <origin xyz="0 0 0" rpy="3.26128e-16 -1.01395e-15 1.5708" />
             <geometry>
-                <mesh filename="${mesh_path}/banksia/meshes/chassis.stl" />
+                <mesh filename="file://$(find rover_description)/banksia/meshes/chassis.stl" />
             </geometry>
             <material name="chassis_material">
@@ -55,5 +48,5 @@
             <origin xyz="-1.3078806732583218725e-20 8.6736173798840354721e-19 -0.021000000000000518252" rpy="-3.141592653589793116 6.2280032059897877693e-19 -4.1232880706353110482e-18" />
             <geometry>
-                <mesh filename="${mesh_path}/banksia/meshes/left_leg.stl"/>
+                <mesh filename="file://$(find rover_description)/banksia/meshes/left_leg.stl"/>
             </geometry>
             <material name="left_leg_material">
@@ -126,5 +119,5 @@
             <origin xyz="-0.12415341931613717297 2.2204460492503130808e-16 -0.1250000000000002498" rpy="-1.570796326794896558 -0.13351607992219349796 -5.9804098682663148249e-17" />
             <geometry>
-                <mesh filename="${mesh_path}/banksia/meshes/fl_ankle.stl"/>
+                <mesh filename="file://$(find rover_description)/banksia/meshes/fl_ankle.stl"/>
             </geometry>
             <material name="fl_ankle_material">
@@ -185,5 +178,5 @@
             <origin xyz="5.5511151231257827021e-17 0 5.963111948670274387e-18" rpy="7.279848939407052303e-17 1.0638440422271473935e-16 -6.3914183266779029169e-20" />
             <geometry>
-                <mesh filename="${mesh_path}/banksia/meshes/fl_wheel.stl"/>
+                <mesh filename="file://$(find rover_description)/banksia/meshes/fl_wheel.stl"/>
             </geometry>
             <material name="fl_wheel_material">
@@ -208,5 +201,5 @@
             <origin xyz="-0.12415341931613714521 2.2204460492503130808e-16 -0.1250000000000002498" rpy="-1.570796326794896558 -0.13351607992219349796 -7.1088909477657821376e-17" />
             <geometry>
-                <mesh filename="${mesh_path}/banksia/meshes/bl_ankle.stl"/>
+                <mesh filename="file://$(find rover_description)/banksia/meshes/bl_ankle.stl"/>
             </geometry>
             <material name="bl_ankle_material">
@@ -267,5 +260,5 @@
             <origin xyz="0 1.1102230246251565404e-16 1.7780915628762272718e-17" rpy="4.6040217445536182725e-17 1.0513492286565858337e-16 2.3412503191653332746e-19" />
             <geometry>
-                <mesh filename="${mesh_path}/banksia/meshes/bl_wheel.stl"/>
+                <mesh filename="file://$(find rover_description)/banksia/meshes/bl_wheel.stl"/>
             </geometry>
             <material name="bl_wheel_material">
@@ -290,5 +283,5 @@
             <origin xyz="-7.9461177221465168975e-19 -7.2858385990954703269e-20 -0.020999999999999519051" rpy="3.141592653589793116 3.7838655819744092421e-17 -5.8406613147999892266e-19" />
             <geometry>
-                <mesh filename="${mesh_path}/banksia/meshes/right_leg.stl"/>
+                <mesh filename="file://$(find rover_description)/banksia/meshes/right_leg.stl"/>
             </geometry>
             <material name="right_leg_material">
@@ -361,5 +354,5 @@
             <origin xyz="0.12415341931613695092 -2.2204460492503130808e-16 -0.12500000000000027756" rpy="-1.57079632679489678 0.13351607992219352572 9.9507186100571649487e-18" />
             <geometry>
-                <mesh filename="${mesh_path}/banksia/meshes/fr_ankle.stl"/>
+                <mesh filename="file://$(find rover_description)/banksia/meshes/fr_ankle.stl"/>
             </geometry>
             <material name="fr_ankle_material">
@@ -420,5 +413,5 @@
             <origin xyz="5.5511151231257827021e-17 -1.1102230246251565404e-16 -3.0791341698588325926e-17" rpy="-3.6194812825998444115e-17 1.0511409763610977507e-16 -2.2325341479697011877e-19" />
             <geometry>
-                <mesh filename="${mesh_path}/banksia/meshes/fr_wheel.stl"/>
+                <mesh filename="file://$(find rover_description)/banksia/meshes/fr_wheel.stl"/>
             </geometry>
             <material name="fr_wheel_material">
@@ -443,5 +436,5 @@
             <origin xyz="0.12415341931613720072 -2.2204460492503130808e-16 -0.12500000000000027756" rpy="-1.57079632679489678 0.13351607992219349796 -6.7670245197813334123e-17" />
             <geometry>
-                <mesh filename="${mesh_path}/banksia/meshes/br_ankle.stl"/>
+                <mesh filename="file://$(find rover_description)/banksia/meshes/br_ankle.stl"/>
             </geometry>
             <material name="br_ankle_material">
@@ -502,5 +495,5 @@
             <origin xyz="5.5511151231257827021e-17 0 5.8763757748714340323e-17" rpy="1.4537948349788456791e-16 1.0501738044156386319e-16 -7.6074648532850333807e-21" />
             <geometry>
-                <mesh filename="${mesh_path}/banksia/meshes/br_wheel.stl"/>
+                <mesh filename="file://$(find rover_description)/banksia/meshes/br_wheel.stl"/>
             </geometry>
             <material name="br_wheel_material">
@@ -525,5 +518,5 @@
             <origin xyz="4.9770590769729886024e-14 -0.00015426611885745872277 -0.010000000000000730527" rpy="1.570796326794896558 -3.0512890594788867116e-34 0" />
             <geometry>
-                <mesh filename="${mesh_path}/banksia/meshes/diffbar.stl"/>
+                <mesh filename="file://$(find rover_description)/banksia/meshes/diffbar.stl"/>
             </geometry>
             <material name="diffbar_material">
@@ -554,5 +547,5 @@
             <origin xyz="-2.7755575615628913511e-15 -0.057750000000000162315 3.3306690738754696213e-16" rpy="1.5707963267948350516 -1.5127867282353739675 -3.1415926535897926719" />
             <geometry>
-                <mesh filename="${mesh_path}/banksia/meshes/left_difflink.stl"/>
+                <mesh filename="file://$(find rover_description)/banksia/meshes/left_difflink.stl"/>
             </geometry>
             <material name="left_difflink_material">
@@ -577,5 +570,5 @@
             <origin xyz="6.2172489379008766264e-15 -0.057749999999999454547 -2.4424906541753443889e-15" rpy="1.5707963267948286123 1.512786629442331332 3.141592653589793116" />
             <geometry>
-                <mesh filename="${mesh_path}/banksia/meshes/right_difflink.stl"/>
+                <mesh filename="file://$(find rover_description)/banksia/meshes/right_difflink.stl"/>
             </geometry>
             <material name="right_difflink_material">

Commit message: new lidar angle, 36 degrees

File: src/ros/rover/rover_description/auto_mount/urdf/auto_camera.xacro (robot description, xacro)
@@ -130,5 +130,5 @@
   </joint>
   <joint name="clam_to_mount" type="fixed">
-      <origin xyz="0.2269 0.3285 -0.436186" rpy="3.14159 5.13507e-14 3.14159" />
+      <origin xyz="0.2269 0.3285 -0.3531" rpy="3.14159 5.13507e-14 3.14159" />
       <parent link="clam" />
       <child link="mount" />

File: src/ros/rover/rover_description/auto_mount/urdf/livox.xacro (robot description, xacro)
@@ -1,6 +1,3 @@
 <?xml version="1.0" encoding="utf-8" ?>
-<!--This is a file for the depth camera plugin for the rover in gazebo. This file is referenced at the bottom of rover.urdf.xacro,
-which is how it gets added to the gazebo sim. Edited by: Victor Bartlinski, Kabi Velmurugan Sujatha -->
-<!-- Auto mount is also appended to the top, however it has no simplified collisions -->
 <robot xmlns:xacro="http://www.ros.org/wiki/xacro">
   <link name="livox_frame">
@@ -15,5 +12,5 @@
   </link>
   <joint name="base_link_to_livox" type="fixed">
-    <origin xyz="0.53 0 0.79" rpy=" 3.14 0.0377 0" />
+    <origin xyz="0.53 0 0.85" rpy=" 0 -0.605 0" />
     <parent link="base_link" />
     <child link="livox_frame" />

Commit message: fixes to previous commit!

File: src/ros/rover/rover_description/auto_mount/urdf/auto_camera.xacro (robot description, xacro)
@@ -183,96 +183,98 @@
     cam_yaw="0.0"
   />
-  <!-- EVERYTHING BELOW IS FOR SENSOR PLUGINS! REMOVE IF CAUSING PROBLEMS IRL -->
-  <link name="oak_link_optical"/>
-  <joint name="oak_optical_joint" type="fixed">
-    <origin xyz="0.0 0 0.0" rpy="${-pi/2} 0 ${-pi/2}"/>
-    <parent link="oak_link"/>
-    <child link="oak_link_optical"/>
-  </joint>
-  <link name="bootie_link_optical"/>
-  <joint name="bootie_optical_joint" type="fixed">
-    <origin xyz="0.0 0 0.0" rpy="${-pi/2} 0 ${-pi/2}"/>
-    <parent link="bootie_link"/>
-    <child link="bootie_link_optical"/>
-  </joint>
-  <!-- Used in conjuction with gz_header_republisher to fix pointcloud frame transform-->
-  <link name="oak_link_gz_pointcloud"/>
-  <joint name="oak_pointcloud_joint" type="fixed">
-    <origin xyz="0 0 0" rpy="0 ${-pi/2} ${pi/2}"/>
-    <parent link="oak_link_optical"/>
-    <child link="oak_link_gz_pointcloud"/>
-  </joint>
-  <link name="bootie_link_gz_pointcloud"/>
-  <joint name="bootie_pointcloud_joint" type="fixed">
-    <origin xyz="0 0 0" rpy="0 ${-pi/2} ${pi/2}"/>
-    <parent link="bootie_link_optical"/>
-    <child link="bootie_link_gz_pointcloud"/>
-  </joint>
-  <!-- Oak Depth Camera for Gazebo-->
-  <gazebo reference="oak_link_optical">
-    <sensor name="oak" type="rgbd_camera">
-      <pose> 0 0 0 0 ${-pi/2} ${pi/2} </pose> <!-- Get camera facing correct way in optical frame -->
-      <plugin name="gz::sim::systems::Sensors" filename="gz-sim-sensors-system"></plugin>
-      <gz_frame_id>oak_link_optical</gz_frame_id>
-      <topic>oak</topic>
-      <visualize>true</visualize>
-      <update_rate>30</update_rate>
-      <always_on>1</always_on>
-      <camera name="oak">
-        <horizontal_fov>${radians(82)}</horizontal_fov>
-        <image>
-          <width>1280</width>
-          <height>900</height>
-        </image>
-        <clip>
-          <near>0.4</near>
-          <far>10.0</far>
-        </clip>
-      </camera>
-    </sensor>
-  </gazebo>
-  <!-- Bootie Depth Camera for Gazebo-->
-  <gazebo reference="bootie_link_optical">
-    <sensor name="bootie" type="rgbd_camera">
-      <pose> 0 0 0 0 ${-pi/2} ${pi/2} </pose> <!-- Get camera facing correct way in optical frame -->
-      <!-- <plugin name="gz::sim::systems::Sensors" filename="gz-sim-sensors-system">
-        <frame_name>bootie_link_optical</frame_name>
-      </plugin> -->
-      <gz_frame_id>bootie_link_optical</gz_frame_id>
-      <topic>bootie</topic>
-      <visualize>true</visualize>
-      <update_rate>30</update_rate>
-      <always_on>1</always_on>
-      <camera name="bootie">
-        <horizontal_fov>${radians(82)}</horizontal_fov>
-        <image>
-          <width>1280</width>
-          <height>900</height>
-        </image>
-        <clip>
-          <near>0.4</near>
-          <far>10.0</far>
-        </clip>
-      </camera>
-    </sensor>
-  </gazebo>
-  <gazebo reference="base_link">
-    <sensor name="oak_imu_sensor" type="imu">
-      <topic>oak/imu</topic>
-      <plugin filename="gz-sim-imu-system" name="gz::sim::systems::Imu"></plugin>
-      <gz_frame_id>base_link</gz_frame_id>
-      <always_on>true</always_on>
-      <update_rate>100</update_rate>
-      <visualize>true</visualize>
-    </sensor>
-  </gazebo>
-  <gazebo reference="base_link">
-    <sensor name="bootie_imu_sensor" type="imu">
-      <topic>bootie/imu</topic>
-      <gz_frame_id>base_link</gz_frame_id>
-      <always_on>true</always_on>
-      <update_rate>100</update_rate>
-      <visualize>true</visualize>
-    </sensor>
-  </gazebo>
+  <xacro:unless value="$(arg hitl_camera)">
+    <!-- EVERYTHING BELOW IS FOR SENSOR PLUGINS! REMOVE IF CAUSING PROBLEMS IRL -->
+    <link name="oak_link_optical"/>
+    <joint name="oak_optical_joint" type="fixed">
+      <origin xyz="0.0 0 0.0" rpy="${-pi/2} 0 ${-pi/2}"/>
+      <parent link="oak_link"/>
+      <child link="oak_link_optical"/>
+    </joint>
+    <link name="bootie_link_optical"/>
+    <joint name="bootie_optical_joint" type="fixed">
+      <origin xyz="0.0 0 0.0" rpy="${-pi/2} 0 ${-pi/2}"/>
+      <parent link="bootie_link"/>
+      <child link="bootie_link_optical"/>
+    </joint>
+    <!-- Used in conjuction with gz_header_republisher to fix pointcloud frame transform-->
+    <link name="oak_link_gz_pointcloud"/>
+    <joint name="oak_pointcloud_joint" type="fixed">
+      <origin xyz="0 0 0" rpy="0 ${-pi/2} ${pi/2}"/>
+      <parent link="oak_link_optical"/>
+      <child link="oak_link_gz_pointcloud"/>
+    </joint>
+    <link name="bootie_link_gz_pointcloud"/>
+    <joint name="bootie_pointcloud_joint" type="fixed">
+      <origin xyz="0 0 0" rpy="0 ${-pi/2} ${pi/2}"/>
+      <parent link="bootie_link_optical"/>
+      <child link="bootie_link_gz_pointcloud"/>
+    </joint>
+    <!-- Oak Depth Camera for Gazebo-->
+    <gazebo reference="oak_link_optical">
+      <sensor name="oak" type="rgbd_camera">
+        <pose> 0 0 0 0 ${-pi/2} ${pi/2} </pose> <!-- Get camera facing correct way in optical frame -->
+        <plugin name="gz::sim::systems::Sensors" filename="gz-sim-sensors-system"></plugin>
+        <gz_frame_id>oak_link_optical</gz_frame_id>
+        <topic>oak</topic>
+        <visualize>true</visualize>
+        <update_rate>30</update_rate>
+        <always_on>1</always_on>
+        <camera name="oak">
+          <horizontal_fov>${radians(82)}</horizontal_fov>
+          <image>
+            <width>1280</width>
+            <height>900</height>
+          </image>
+          <clip>
+            <near>0.4</near>
+            <far>10.0</far>
+          </clip>
+        </camera>
+      </sensor>
+    </gazebo>
+    <!-- Bootie Depth Camera for Gazebo-->
+    <gazebo reference="bootie_link_optical">
+      <sensor name="bootie" type="rgbd_camera">
+        <pose> 0 0 0 0 ${-pi/2} ${pi/2} </pose> <!-- Get camera facing correct way in optical frame -->
+        <!-- <plugin name="gz::sim::systems::Sensors" filename="gz-sim-sensors-system">
+          <frame_name>bootie_link_optical</frame_name>
+        </plugin> -->
+        <gz_frame_id>bootie_link_optical</gz_frame_id>
+        <topic>bootie</topic>
+        <visualize>true</visualize>
+        <update_rate>30</update_rate>
+        <always_on>1</always_on>
+        <camera name="bootie">
+          <horizontal_fov>${radians(82)}</horizontal_fov>
+          <image>
+            <width>1280</width>
+            <height>900</height>
+          </image>
+          <clip>
+            <near>0.4</near>
+            <far>10.0</far>
+          </clip>
+        </camera>
+      </sensor>
+    </gazebo>
+    <gazebo reference="base_link">
+      <sensor name="oak_imu_sensor" type="imu">
+        <topic>oak/imu</topic>
+        <plugin filename="gz-sim-imu-system" name="gz::sim::systems::Imu"></plugin>
+        <gz_frame_id>base_link</gz_frame_id>
+        <always_on>true</always_on>
+        <update_rate>100</update_rate>
+        <visualize>true</visualize>
+      </sensor>
+    </gazebo>
+    <gazebo reference="base_link">
+      <sensor name="bootie_imu_sensor" type="imu">
+        <topic>bootie/imu</topic>
+        <gz_frame_id>base_link</gz_frame_id>
+        <always_on>true</always_on>
+        <update_rate>100</update_rate>
+        <visualize>true</visualize>
+      </sensor>
+    </gazebo>
+  </xacro:unless>
 </robot>

File: src/ros/rover/rover_description/banksia/urdf/rover.urdf.xacro (robot description, xacro)
@@ -8,4 +8,5 @@
     <xacro:arg name="use_mock_hardware" default="false"/>
     <xacro:arg name="arm" default="false"/>
+    <xacro:arg name="hitl_camera" default="false" />
     <xacro:arg name="old_arm" default="false"/>
     <xacro:arg name="auto_camera" default="true"/>
@@ -19,4 +20,5 @@
     <!-- Variables -->
     <xacro:property name="angle" value="$(arg angle)" />
+    <xacro:property name="hitl_camera" value="$(arg hitl_camera)" />
     <link name="base_link"></link>
     <joint name="base_link_to_chassis" type="fixed">
