Commit message: Fix/auto-urdf (#863)

File: src/ros/rover/rover_description/auto_mount/urdf/auto_camera.xacro (robot description, xacro)
@@ -125,33 +125,17 @@
     </visual>
   </link>
-  <!-- Link lidar_camera_approx -->
-  <link name="lidar_camera_approx">
-    <inertial>
-      <origin xyz="0 0 0" rpy="0 0 0"/>
-      <mass value="1e-09"/>
-      <inertia ixx="1e-09" ixy="0" ixz="0" iyy="1e-09" iyz="0" izz="1e-09"/>
-    </inertial>
-    <!-- Part lidar_camera_approx -->
-    <visual>
-      <origin xyz="0.024 0.018 -0.01975" rpy="-3.14159 9.70415e-18 6.97585e-19"/>
-      <geometry>
-        <mesh filename="file://$(arg rover_description_dir)/auto_mount/meshes/lidar_camera_approx.stl"/>
-      </geometry>
-      <material name="lidar_camera_approx_material">
-        <color rgba="0.439216 0.47451 0.501961 0"/>
-      </material>
-    </visual>
-  </link>
-  <!-- Joint from lidar_holder to lidar_camera_approx -->
+  <!-- livox_frame -->
+  <xacro:include
+        filename="$(find rover_description)/auto_mount/urdf/livox.xacro"
+    />
+  <!-- Joint from lidar_holder to livox_frame -->
   <joint name="lidar_mate" type="fixed">
-    <origin xyz="-0.114 -0.005 0.06" rpy="-1.5708 4.26348e-17 -4.99937e-17"/>
+    <origin xyz="-0.09 -0.03 0.0375" rpy="1.5708 0 0"/>
     <parent link="lidar_holder"/>
-    <child link="lidar_camera_approx"/>
-    <axis xyz="0 0 1"/>
-    <limit effort="10" velocity="10"/>
+    <child link="livox_frame"/>
   </joint>
   <!-- Joint from mount to lidar_holder -->
   <joint name="mount_to_lidar" type="fixed">
-    <origin xyz="0.123 -0.0775 0.0124231" rpy="-1.5708 0.0662646 1.5708"/>
+    <origin xyz="0.123 -0.0775 0.0124231" rpy="-1.5708 -1.5708 1.5708"/>
     <parent link="mount"/>
     <child link="lidar_rotator"/>
@@ -160,5 +144,5 @@
     <link name="lidar_rotator"/>
   <joint name="lidar_rotator_offset" type="fixed">
-    <origin rpy="0 0 ${lidar_angle+90*(pi/180)}"/>
+    <origin rpy="0 0 ${-lidar_angle*(pi/180)}"/>
     <parent link="lidar_rotator"/>
     <child link="lidar_holder"/>

File: src/ros/rover/rover_description/auto_mount/urdf/livox.xacro (robot description, xacro)
@@ -5,16 +5,8 @@
         <origin xyz="0 0 0" rpy="0 0 0" />
         <geometry>
-            <mesh
-                    filename="file://$(find rover_description)/auto_mount/meshes/mid-360-asm.stl"
-                />
+            <mesh filename="file://$(find rover_description)/auto_mount/meshes/mid-360-asm.stl"/>
         </geometry>
     </visual>
   </link>
-  <joint name="lidar_camera_approx_to_livox" type="fixed">
-    <origin xyz="0.023 0.023 -0.025" rpy=" 3.14159 0 0" />
-    <parent link="lidar_camera_approx" />
-    <child link="livox_frame" />
-    <axis xyz="1 0 0" />
-  </joint>
   <gazebo reference="livox_frame">
         <sensor name="gpu_lidar" type="gpu_lidar">

File: src/ros/rover/rover_description/banksia/urdf/rover.urdf.xacro (robot description, xacro)
@@ -37,7 +37,4 @@
         <xacro:include filename="$(arg rover_description_dir)/auto_mount/urdf/auto_camera.xacro"/>
     </xacro:if>
-    <xacro:include
-        filename="$(find rover_description)/auto_mount/urdf/livox.xacro"
-    />
     <xacro:if value="$(arg arm)">
         <!-- Waratah's arm

Commit message: fix urdf (again), lidar was facing backwards AHHHH

File: src/ros/rover/rover_description/auto_mount/urdf/auto_camera.xacro (robot description, xacro)
@@ -131,5 +131,5 @@
   <!-- Joint from lidar_holder to livox_frame -->
   <joint name="lidar_mate" type="fixed">
-    <origin xyz="-0.09 -0.03 0.0375" rpy="1.5708 0 0"/>
+    <origin xyz="-0.09 -0.03 0.045" rpy="1.5708 3.14159 0"/>
     <parent link="lidar_holder"/>
     <child link="livox_frame"/>

Commit message: added aft_mapped (dummy livox_frame) to tf tree

File: src/ros/rover/rover_description/auto_mount/urdf/auto_camera.xacro (robot description, xacro)
@@ -132,4 +132,11 @@
     <parent link="lidar_holder"/>
     <child link="livox_frame"/>
+  </joint>
+  <!-- Joint from aft_mapped to livox_frame (for FAST-LIVO2) -->
+  <link name="aft_mapped" />
+  <joint name="livox_frame_to_aft_mapped" type="fixed">
+      <parent link="livox_frame" />
+      <child link="aft_mapped" />
+      <origin rpy="0 0 0" xyz="0 0 0" />
   </joint>
   <!-- Joint from mount to lidar_holder -->

Commit message: Ready to test on stack

File: src/ros/rover/rover_description/auto_mount/urdf/auto_camera.xacro (robot description, xacro)
@@ -132,11 +132,4 @@
     <parent link="lidar_holder"/>
     <child link="livox_frame"/>
-  </joint>
-  <!-- Joint from aft_mapped to livox_frame (for FAST-LIVO2) -->
-  <link name="aft_mapped" />
-  <joint name="livox_frame_to_aft_mapped" type="fixed">
-      <parent link="livox_frame" />
-      <child link="aft_mapped" />
-      <origin rpy="0 0 0" xyz="0 0 0" />
   </joint>
   <!-- Joint from mount to lidar_holder -->

Commit message: realsense urdf WIP

File: src/ros/rover/rover_description/auto_mount/urdf/auto_camera.xacro (robot description, xacro)
@@ -126,10 +126,8 @@
   </link>
   <!-- livox_frame -->
-  <xacro:include
-        filename="$(find rover_description)/auto_mount/urdf/livox.xacro"
-    />
+  <xacro:include filename="$(find rover_description)/auto_mount/urdf/livox.xacro"/>
   <!-- Joint from lidar_holder to livox_frame -->
   <joint name="lidar_mate" type="fixed">
-    <origin xyz="-0.09 -0.03 0.045" rpy="1.5708 3.14159 0"/>
+    <origin xyz="-0.09 -0.03 0.0435" rpy="1.5708 3.14159 0"/>
     <parent link="lidar_holder"/>
     <child link="livox_frame"/>
@@ -223,6 +221,24 @@
     <child link="oak_link"/>
     <axis xyz="0 0 1"/>
-    <limit effort="10" velocity="10"/>
-  </joint>
+  </joint>
+  <!-- realsense d415 -->
+  <xacro:include filename="$(find realsense2_description)/urdf/_d415.urdf.xacro"/>
+  <xacro:sensor_d415 parent="camera_holder_2" name="d415">
+    <origin xyz="-0.08 0 -0.058" rpy="-1.5708 0 3.14159" />
+  </xacro:sensor_d415>
+  <!-- Joint from camera_holder_2 to realsense d415 -->
+  <!-- <xacro:include filename="$(find rover_description)/auto_mount/urdf/rs_d415.xacro"/>
+  <joint name="d415_to_mount" type="fixed">
+    <origin xyz="0 0 0" rpy="0 0 0" />
+    <parent link="camera_holder_2"/>
+    <child link="d415_link"/>
+    <axis xyz="0 0 1"/>
+  </joint>
+  <joint name="d415_to_mount" type="fixed">
+    <origin xyz="-0.08 0 -0.058" rpy="-1.5708 0 3.14159" />
+    <parent link="camera_holder_2"/>
+    <child link="d415_link"/>
+    <axis xyz="0 0 1"/>
+  </joint> -->
   <!-- Joint from mount to camera_holder_2 -->
   <joint name="mount_to_front" type="fixed">

File: src/ros/rover/rover_description/auto_mount/urdf/livox.xacro (robot description, xacro)
@@ -3,5 +3,5 @@
   <link name="livox_frame">
     <visual>
-        <origin xyz="0 0 0" rpy="0 0 0" />
+        <origin xyz="0 0.0055 0" rpy="0 0 3.14159" />
         <geometry>
             <mesh filename="file://$(find rover_description)/auto_mount/meshes/mid-360-asm.stl"/>

Commit message: set origin to screw hole to position properly

File: src/ros/rover/rover_description/auto_mount/urdf/auto_camera.xacro (robot description, xacro)
@@ -225,16 +225,10 @@
   <xacro:include filename="$(find realsense2_description)/urdf/_d415.urdf.xacro"/>
   <xacro:sensor_d415 parent="camera_holder_2" name="d415">
-    <origin xyz="-0.08 0 -0.058" rpy="-1.5708 0 3.14159" />
+    <origin xyz="-0.09 0.0115 -0.058" rpy="-1.5708 0 3.14159" />
   </xacro:sensor_d415>
   <!-- Joint from camera_holder_2 to realsense d415 -->
   <!-- <xacro:include filename="$(find rover_description)/auto_mount/urdf/rs_d415.xacro"/>
   <joint name="d415_to_mount" type="fixed">
-    <origin xyz="0 0 0" rpy="0 0 0" />
-    <parent link="camera_holder_2"/>
-    <child link="d415_link"/>
-    <axis xyz="0 0 1"/>
-  </joint>
-  <joint name="d415_to_mount" type="fixed">
-    <origin xyz="-0.08 0 -0.058" rpy="-1.5708 0 3.14159" />
+    <origin xyz="-0.09 0.0115 -0.058" rpy="-1.5708 0 3.14159" />
     <parent link="camera_holder_2"/>
     <child link="d415_link"/>

File: src/ros/rover/rover_description/auto_mount/urdf/rs_d415.xacro (robot description, xacro)
@@ -3,5 +3,5 @@
   <link name="d415_link">
     <visual>
-        <origin xyz="0 -0.0377 0" rpy="3.14159 0 1.5708" />
+        <origin xyz="-0.01 -0.0377 0.0115" rpy="3.14159 0 1.5708" />
         <geometry>
             <mesh filename="file://$(find rover_description)/auto_mount/meshes/intel_d415.stl"/>
@@ -11,5 +11,5 @@
   <link name="d415_rgb_camera_frame"/>
   <joint name="d415_link_to_rgb" type="fixed">
-    <origin xyz="0.02 0.036 0" rpy="0 0 0" />
+    <origin xyz="0.01 0.036 0.0115" rpy="0 0 0" />
     <parent link="d415_link"/>
     <child link="d415_rgb_camera_frame"/>

Commit message: cleanup

File: src/ros/rover/rover_description/auto_mount/urdf/auto_camera.xacro (robot description, xacro)
@@ -227,12 +227,4 @@
     <origin xyz="-0.09 0.0115 -0.058" rpy="-1.5708 0 3.14159" />
   </xacro:sensor_d415>
-  <!-- Joint from camera_holder_2 to realsense d415 -->
-  <!-- <xacro:include filename="$(find rover_description)/auto_mount/urdf/rs_d415.xacro"/>
-  <joint name="d415_to_mount" type="fixed">
-    <origin xyz="-0.09 0.0115 -0.058" rpy="-1.5708 0 3.14159" />
-    <parent link="camera_holder_2"/>
-    <child link="d415_link"/>
-    <axis xyz="0 0 1"/>
-  </joint> -->
   <!-- Joint from mount to camera_holder_2 -->
   <joint name="mount_to_front" type="fixed">

Commit message: Feat/auto-cameras (#921)
Co-authored-by: Monash Nova Rover <novaroverteam@monash.edu>

File: src/ros/rover/rover_description/auto_mount/urdf/auto_camera.xacro (robot description, xacro)
@@ -126,10 +126,8 @@
   </link>
   <!-- livox_frame -->
-  <xacro:include
-        filename="$(find rover_description)/auto_mount/urdf/livox.xacro"
-    />
+  <xacro:include filename="$(find rover_description)/auto_mount/urdf/livox.xacro"/>
   <!-- Joint from lidar_holder to livox_frame -->
   <joint name="lidar_mate" type="fixed">
-    <origin xyz="-0.09 -0.03 0.045" rpy="1.5708 3.14159 0"/>
+    <origin xyz="-0.09 -0.03 0.0435" rpy="1.5708 3.14159 0"/>
     <parent link="lidar_holder"/>
     <child link="livox_frame"/>
@@ -223,6 +221,10 @@
     <child link="oak_link"/>
     <axis xyz="0 0 1"/>
-    <limit effort="10" velocity="10"/>
-  </joint>
+  </joint>
+  <!-- realsense d415 -->
+  <xacro:include filename="$(find realsense2_description)/urdf/_d415.urdf.xacro"/>
+  <xacro:sensor_d415 parent="camera_holder_2" name="d415">
+    <origin xyz="-0.09 0.0115 -0.058" rpy="-1.5708 0 3.14159" />
+  </xacro:sensor_d415>
   <!-- Joint from mount to camera_holder_2 -->
   <joint name="mount_to_front" type="fixed">

Commit message: feat: Add cut auto mount

File: src/ros/rover/rover_description/auto_mount/urdf/auto_camera.xacro (robot description, xacro)
@@ -249,5 +249,5 @@
   </joint>
   <joint name="auto_mount_to_chassis" type="fixed">
-      <origin xyz="-0.137 0 -0.063" rpy="0 -1.01333e-15 0" />
+      <origin xyz="-0.348 0 -0.063" rpy="0 -1.01333e-15 0" />
       <parent link="chassis" />
       <child link="clam" />
