Commit message: fix : rename livox_link -> livox_frame

File: src/ros/rover/rover_description/auto_mount/urdf/livox.xacro (robot description, xacro)
@@ -4,5 +4,5 @@
 <!-- Auto mount is also appended to the top, however it has no simplified collisions -->
 <robot xmlns:xacro="http://www.ros.org/wiki/xacro">
-  <link name="livox_link">
+  <link name="livox_frame">
     <visual>
         <origin xyz="0 0 0" rpy="0 0 0" />
@@ -17,12 +17,12 @@
     <origin xyz="0.53 0 0.79" rpy=" 3.14 0 0" />
     <parent link="base_link" />
-    <child link="livox_link" />
+    <child link="livox_frame" />
     <axis xyz="1 0 0" />
   </joint>
-  <gazebo reference="livox_link">
+  <gazebo reference="livox_frame">
         <sensor name="gpu_lidar" type="gpu_lidar">
             <update_rate>10</update_rate>
             <topic>livox/lidar</topic>
-            <gz_frame_id>livox_link</gz_frame_id>
+            <gz_frame_id>livox_frame</gz_frame_id>
             <update_rate>10</update_rate>
             <ray>

Commit message: fix : angle tilt on the mount

File: src/ros/rover/rover_description/auto_mount/urdf/livox.xacro (robot description, xacro)
@@ -15,5 +15,5 @@
   </link>
   <joint name="base_link_to_livox" type="fixed">
-    <origin xyz="0.53 0 0.79" rpy=" 3.14 0 0" />
+    <origin xyz="0.53 0 0.79" rpy=" 3.14 0.0754 0" />
     <parent link="base_link" />
     <child link="livox_frame" />

Commit message: changing pitch

File: src/ros/rover/rover_description/auto_mount/urdf/livox.xacro (robot description, xacro)
@@ -15,5 +15,5 @@
   </link>
   <joint name="base_link_to_livox" type="fixed">
-    <origin xyz="0.53 0 0.79" rpy=" 3.14 0.0754 0" />
+    <origin xyz="0.53 0 0.79" rpy=" 3.14 0.0377 0" />
     <parent link="base_link" />
     <child link="livox_frame" />

Commit message: fix : pitch is positive?

File: src/ros/rover/rover_description/auto_mount/urdf/livox.xacro (robot description, xacro)
@@ -12,5 +12,5 @@
   </link>
   <joint name="base_link_to_livox" type="fixed">
-    <origin xyz="0.53 0 0.85" rpy=" 0 -0.605 0" />
+    <origin xyz="0.53 0 0.85" rpy=" 0 0.605 0" />
     <parent link="base_link" />
     <child link="livox_frame" />

Commit message: fixed lidar angle calculation

File: src/ros/rover/rover_description/auto_mount/urdf/livox.xacro (robot description, xacro)
@@ -9,4 +9,10 @@
     </visual>
   </link>
+  <joint name="lidar_camera_approx_to_livox" type="fixed">
+    <origin xyz="0.023 0.023 -0.026" rpy=" 3.14159 0 0" />
+    <parent link="lidar_camera_approx" />
+    <child link="livox_frame" />
+    <axis xyz="1 0 0" />
+  </joint>
   <gazebo reference="livox_frame">
         <sensor name="gpu_lidar" type="gpu_lidar">

Commit message: remove lidar approx and include livox_frame in auto_camera.xacro

File: src/ros/rover/rover_description/auto_mount/urdf/livox.xacro (robot description, xacro)
@@ -9,10 +9,4 @@
     </visual>
   </link>
-  <joint name="lidar_camera_approx_to_livox" type="fixed">
-    <origin xyz="0.023 0.023 -0.026" rpy=" 3.14159 0 0" />
-    <parent link="lidar_camera_approx" />
-    <child link="livox_frame" />
-    <axis xyz="1 0 0" />
-  </joint>
   <gazebo reference="livox_frame">
         <sensor name="gpu_lidar" type="gpu_lidar">

Commit message: clean up URDFs

File: src/ros/rover/rover_description/auto_mount/urdf/livox.xacro (robot description, xacro)
@@ -1,47 +1,49 @@
 <?xml version="1.0" encoding="utf-8" ?>
 <robot xmlns:xacro="http://www.ros.org/wiki/xacro">
-  <link name="livox_frame">
-    <visual>
-        <origin xyz="0 0.0055 0" rpy="0 0 3.14159" />
-        <geometry>
-            <mesh filename="file://$(find rover_description)/auto_mount/meshes/mid-360-asm.stl"/>
-        </geometry>
-    </visual>
-  </link>
-  <gazebo reference="livox_frame">
-        <sensor name="gpu_lidar" type="gpu_lidar">
-            <update_rate>10</update_rate>
-            <topic>livox/lidar</topic>
-            <gz_frame_id>livox_frame</gz_frame_id>
-            <update_rate>10</update_rate>
-            <ray>
-              <scan>
-                <horizontal>
-                  <samples>720</samples>      <!-- MID-360 0.5° resolution -->
-                  <resolution>1</resolution>
-                  <!-- MID-360 HFOV = 360° -->
-                  <min_angle>-3.14156</min_angle>
-                  <max_angle>3.14156</max_angle>
-                </horizontal>
-                <vertical>
-                  <samples
-                        >40</samples>       <!-- MID-360 point cloud density -->
-                  <resolution>1</resolution>
-                  <!-- MID-360 VFOV = 59° -->
-                  <min_angle>0</min_angle>
-                  <max_angle>0.9774</max_angle>
-                </vertical>
-              </scan>
-              <range>
-                <min
-                    >0.01</min>                 <!-- MID-360 min. detection range -->
-                <max
-                    >40.0</max>                 <!-- MID-360 max. detection range -->
-                <resolution>0.01</resolution>
-              </range>
-            </ray>
-            <always_on>1</always_on>
-            <visualize>true</visualize>
-        </sensor>
-  </gazebo>
+    <link name="livox_frame">
+        <visual>
+            <origin xyz="0 0.0055 0" rpy="0 0 3.14159" />
+            <geometry>
+                <mesh filename="file://$(arg rover_description_dir)/auto_mount/meshes/mid-360-asm.stl"/>
+            </geometry>
+            <visibility_flags>0x02</visibility_flags> <!-- Bit 1 -->
+        </visual>
+    </link>
+    <!-- Gazebo sensor plugin for the Livox MID-360 LiDAR (does not affect IRL) -->
+    <xacro:if value="$(arg gazebo)">
+        <gazebo reference="livox_frame">
+            <sensor name="gpu_lidar" type="gpu_lidar">
+                <update_rate>10</update_rate>
+                <topic>livox/lidar</topic>
+                <gz_frame_id>livox_frame</gz_frame_id>
+                <update_rate>10</update_rate>
+                <ray>
+                    <scan>
+                        <horizontal>
+                            <samples>720</samples>      <!-- MID-360 0.5° resolution -->
+                            <resolution>0.01</resolution>
+                            <!-- MID-360 HFOV = 360° -->
+                            <min_angle>-3.14156</min_angle>
+                            <max_angle>3.14156</max_angle>
+                        </horizontal>
+                        <vertical>
+                            <samples>40</samples>       <!-- MID-360 point cloud density -->
+                            <resolution>0.01</resolution>
+                            <!-- MID-360 VFOV = 59° -->
+                            <min_angle>-0.122173</min_angle>
+                            <max_angle>0.907571</max_angle>
+                        </vertical>
+                    </scan>
+                    <range>
+                        <min>0.01</min>                 <!-- MID-360 min. detection range -->
+                        <max>40.0</max>                 <!-- MID-360 max. detection range -->
+                        <resolution>0.01</resolution>
+                    </range>
+                    <visibility_mask>0xFFFFFFFD</visibility_mask> <!-- All bits except bit 1 -->
+                </ray>
+                <always_on>1</always_on>
+                <visualize>false</visualize>
+            </sensor>
+        </gazebo>
+    </xacro:if>
 </robot>

File: src/ros/rover/rover_description/banksia/urdf/rover.urdf.xacro (robot description, xacro)
@@ -9,9 +9,7 @@
     <xacro:arg name="arm" default="false"/>
     <xacro:arg name="old_arm" default="false"/>
-    <xacro:arg name="auto_camera" default="true"/>
+    <xacro:arg name="auto_mount" default="false"/>
+    <xacro:arg name="shortened_auto_mount" default="true"/>
     <xacro:arg name="robot_name" default="Banksia"/>
-    <xacro:arg name="oak_angle" default="15"/>
-    <xacro:arg name="bootie_angle" default="15"/>
-    <xacro:arg name="lidar_angle" default="40"/>
     <xacro:arg name="rover_description_dir" default="$(find rover_description)" />
     <!-- Needed to prevent arm control from launching hardware interfaces for the wheels/pivots -->
@@ -22,8 +20,4 @@
         <self_collide>false</self_collide>
     </gazebo>
-    <!-- Variables -->
-    <xacro:property name="oak_angle" value="$(arg oak_angle)" />
-    <xacro:property name="bootie_angle" value="$(arg bootie_angle)" />
-    <xacro:property name="lidar_angle" value="$(arg lidar_angle)" />
     <link name="base_link" />
     <joint name="base_link_to_chassis" type="fixed">
@@ -37,6 +31,6 @@
     <!-- Include additional xacro files-->
     <xacro:include filename="$(arg rover_description_dir)/banksia/urdf/ckc.xacro"/>
-    <xacro:if value="$(arg auto_camera)">
-        <xacro:include filename="$(arg rover_description_dir)/auto_mount/urdf/auto_camera.xacro"/>
+    <xacro:if value="$(arg auto_mount)">
+        <xacro:include filename="$(arg rover_description_dir)/auto_mount/urdf/auto_mount.xacro"/>
     </xacro:if>
     <xacro:if value="$(arg arm)">
