Commit message: feat: optional arbitrary multipliers for blcmd interpretation because it is all fucked

File: src/other/can_database/banksia/boards/blcmd_interpreted.kcd.xacro (robot description, xacro)
@@ -26,6 +26,14 @@
         <!-- all calculations are derived from blcmd_hardware2.cpp -->
         <!-- constants -->
+        <!-- to experimentally determine as theoretical values appear to be wrong :( -->
+        <xacro:property name="velocity_command_slope_multiplier" value="1"/>
+        <xacro:property name="velocity_telemetry_slope_multiplier" value="1"/>
+        <xacro:property name="position_command_slope_multiplier" value="1"/>
+        <xacro:property name="position_command_intercept_multiplier" value="1"/>
+        <xacro:property name="position_telemetry_slope_multiplier" value="1"/>
+        <xacro:property name="position_telemetry_intercept_multiplier" value="1"/>
         <xacro:property name="signed_16_bit_integer_limit" value="${2**15 - 1}"/>
         <xacro:property name="reversed_multiplier" value="${-1 if reversed else 1}"/>
+        <!-- calculations -->
         <!-- display radians or degrees -->
         <xacro:if value="${unit_radians}">
@@ -61,13 +69,13 @@
                 drive_at_current_slope="${effort_slope}"
                 telemetry_packet_1_effort_slope="${effort_slope}"
-                drive_at_speed_slope="${velocity_command_slope}"
+                drive_at_speed_slope="${velocity_command_slope * velocity_command_slope_multiplier}"
                 drive_at_speed_unit="${angular_velocity_unit}"
-                telemetry_packet_1_velocity_slope="${velocity_telemetry_slope}"
+                telemetry_packet_1_velocity_slope="${velocity_telemetry_slope * velocity_telemetry_slope_multiplier}"
                 telemetry_packet_1_velocity_unit="${angular_velocity_unit}"
-                drive_to_position_intercept="${position_intercept}"
-                drive_to_position_slope="${position_slope}"
+                drive_to_position_intercept="${position_intercept * position_command_intercept_multiplier}"
+                drive_to_position_slope="${position_slope * position_command_slope_multiplier}"
                 drive_to_position_unit="${angle_unit}"
-                telemetry_packet_3_resolver_position_intercept="${position_intercept}"
-                telemetry_packet_3_resolver_position_slope="${position_slope}"
+                telemetry_packet_3_resolver_position_intercept="${position_intercept * position_telemetry_intercept_multiplier}"
+                telemetry_packet_3_resolver_position_slope="${position_slope * position_telemetry_slope_multiplier}"
                 telemetry_packet_3_resolver_position_unit="${angle_unit}"
         />

Commit message: fix: allow arbitrary slope multipliers to be passed in blcmd interepreted's params

File: src/other/can_database/banksia/boards/blcmd_interpreted.kcd.xacro (robot description, xacro)
@@ -23,14 +23,13 @@
     resolver_reduction:=None
     res_ticks_per_rev:=None
-    zero_offset:=None">
+    zero_offset:=None
+    velocity_command_slope_multiplier:=1
+    velocity_telemetry_slope_multiplier:=1
+    position_command_slope_multiplier:=1
+    position_command_intercept_multiplier:=1
+    position_telemetry_slope_multiplier:=1
+    position_telemetry_intercept_multiplier:=1">
         <!-- all calculations are derived from blcmd_hardware2.cpp -->
         <!-- constants -->
-        <!-- to experimentally determine as theoretical values appear to be wrong :( -->
-        <xacro:property name="velocity_command_slope_multiplier" value="1"/>
-        <xacro:property name="velocity_telemetry_slope_multiplier" value="1"/>
-        <xacro:property name="position_command_slope_multiplier" value="1"/>
-        <xacro:property name="position_command_intercept_multiplier" value="1"/>
-        <xacro:property name="position_telemetry_slope_multiplier" value="1"/>
-        <xacro:property name="position_telemetry_intercept_multiplier" value="1"/>
         <xacro:property name="signed_16_bit_integer_limit" value="${2**15 - 1}"/>
         <xacro:property name="reversed_multiplier" value="${-1 if reversed else 1}"/>

Commit message: feat: move strange adjustment of velocity telemetry to system instead of board level for blcmds

File: src/other/can_database/banksia/boards/blcmd_interpreted.kcd.xacro (robot description, xacro)
@@ -51,5 +51,5 @@
         <xacro:property name="max_velocity" value="${ (clock_rate) / (min_interval * revolution_pulses * gear_ratio) * 2 * pi }"/>
         <xacro:property name="velocity_command_slope" value="${ max_velocity / signed_16_bit_integer_limit * reversed_multiplier * conversion_multiplier}"/>
-        <xacro:property name="velocity_telemetry_slope" value="${ (max_velocity * -1 * 0.5) / signed_16_bit_integer_limit * reversed_multiplier * conversion_multiplier}"/>
+        <xacro:property name="velocity_telemetry_slope" value="${ max_velocity / signed_16_bit_integer_limit * reversed_multiplier * conversion_multiplier}"/>
         <!-- position -->
         <xacro:if value="${interpret_position}">

File: src/other/can_database/banksia/systems/drive_interpreted.kcd.xacro (robot description, xacro)
@@ -6,4 +6,7 @@
 	<xacro:macro name="drive_interpreted_system">
 		<!-- from ros2_control.xacro: -->
+		<!-- constants for all blcmds -->
+		<!-- whyyyyyy electrical why is this needed -->
+		<xacro:property name="velocity_telemetry_slope_adjustment" value="${-1 * 0.5}"/>
 		<!-- constants for wheels -->
 		<xacro:property name="wheel_clock_rate" value="100000000"/>
@@ -25,5 +28,6 @@
 		   revolution_pulses="${wheel_revolution_pulses}"
 		   min_interval="${wheel_min_interval}"
-		   gear_ratio="${wheel_gear_ratio}"/>
+		   gear_ratio="${wheel_gear_ratio}"
+		   velocity_telemetry_slope_multiplier="${velocity_telemetry_slope_adjustment}"/>
 		<xacro:blcmd_interpreted_board blcmd_id="2" blcmd_node_id="${BLW_BLCMD_NODE_ID}" joint_name="blw"
 		   reversed="True"
@@ -31,5 +35,6 @@
 		   revolution_pulses="${wheel_revolution_pulses}"
 		   min_interval="${wheel_min_interval}"
-		   gear_ratio="${wheel_gear_ratio}"/>
+		   gear_ratio="${wheel_gear_ratio}"
+		   velocity_telemetry_slope_multiplier="${velocity_telemetry_slope_adjustment}"/>
 		<xacro:blcmd_interpreted_board blcmd_id="3" blcmd_node_id="${BRW_BLCMD_NODE_ID}" joint_name="brw"
 		   reversed="False"
@@ -37,5 +42,6 @@
 		   revolution_pulses="${wheel_revolution_pulses}"
 		   min_interval="${wheel_min_interval}"
-		   gear_ratio="${wheel_gear_ratio}"/>
+		   gear_ratio="${wheel_gear_ratio}"
+		   velocity_telemetry_slope_multiplier="${velocity_telemetry_slope_adjustment}"/>
 		<xacro:blcmd_interpreted_board blcmd_id="4" blcmd_node_id="${FRW_BLCMD_NODE_ID}" joint_name="frw"
 		   reversed="False"
@@ -43,5 +49,6 @@
 		   revolution_pulses="${wheel_revolution_pulses}"
 		   min_interval="${wheel_min_interval}"
-		   gear_ratio="${wheel_gear_ratio}"/>
+		   gear_ratio="${wheel_gear_ratio}"
+		   velocity_telemetry_slope_multiplier="${velocity_telemetry_slope_adjustment}"/>
 		<xacro:blcmd_interpreted_board blcmd_id="5" blcmd_node_id="${FLP_BLCMD_NODE_ID}" joint_name="flp"
 		   reversed="True"
@@ -50,4 +57,5 @@
 		   min_interval="${pivot_min_interval}"
 		   gear_ratio="${pivot_gear_ratio}"
+		   velocity_telemetry_slope_multiplier="${velocity_telemetry_slope_adjustment}"
 		   interpret_position="True"
 		   resolver_reduction="${resolver_reduction}"
@@ -60,4 +68,5 @@
 		   min_interval="${pivot_min_interval}"
 		   gear_ratio="${pivot_gear_ratio}"
+		   velocity_telemetry_slope_multiplier="${velocity_telemetry_slope_adjustment}"
 		   interpret_position="True"
 		   resolver_reduction="${resolver_reduction}"
@@ -70,4 +79,5 @@
 		   min_interval="${pivot_min_interval}"
 		   gear_ratio="${pivot_gear_ratio}"
+		   velocity_telemetry_slope_multiplier="${velocity_telemetry_slope_adjustment}"
 		   interpret_position="True"
 		   resolver_reduction="${resolver_reduction}"
@@ -80,4 +90,5 @@
 		   min_interval="${pivot_min_interval}"
 		   gear_ratio="${pivot_gear_ratio}"
+		   velocity_telemetry_slope_multiplier="${velocity_telemetry_slope_adjustment}"
 		   interpret_position="True"
 		   resolver_reduction="${resolver_reduction}"
