Commit message: fix: renamed ducket_link map to correct stl

File: src/ros/rover/rover_description/ducket/ducket.urdf.xacro (robot description, xacro)
@@ -26,5 +26,5 @@
             <origin xyz="0.0354798 0.116628 -0.0371589" rpy="0 -0 0" />
             <geometry>
-                <mesh filename="file://$(arg rover_description_dir)/ducket/meshes/ducket_link.stl" scale="1 1 1" />
+                <mesh filename="file://$(arg rover_description_dir)/ducket/meshes/Arm_Mount_Connector__Mirror_.stl" scale="1 1 1" />
             </geometry>
             <material name="0.301961_0.301961_0.301961_0.000000_0.000000">
