Commit message: fix: new drive min interval

File: src/other/can_database/banksia/systems/drive_interpreted.kcd.xacro (robot description, xacro)
@@ -12,5 +12,5 @@
 		<xacro:property name="wheel_clock_rate" value="100000000"/>
 		<xacro:property name="wheel_revolution_pulses" value="8192"/>
-		<xacro:property name="wheel_min_interval" value="122"/>
+		<xacro:property name="wheel_min_interval" value="233"/>
 		<xacro:property name="wheel_gear_ratio" value="15.0"/>
 		<!-- constants for pivots -->

Commit message: fix: remove 0.5 multiplier from can database

File: src/other/can_database/banksia/systems/drive_interpreted.kcd.xacro (robot description, xacro)
@@ -8,5 +8,5 @@
 		<!-- constants for all blcmds -->
 		<!-- whyyyyyy electrical why is this needed -->
-		<xacro:property name="velocity_telemetry_slope_adjustment" value="${-1 * 0.5}"/>
+		<xacro:property name="velocity_telemetry_slope_adjustment" value="${-1}"/>
 		<!-- constants for wheels -->
 		<xacro:property name="wheel_clock_rate" value="100000000"/>
