Commit message: add: Automount for arch26 and urc26 can be chosen from launch and from comp env variable

File: src/ros/rover/rover_description/auto_mount_arch/urdf/auto_mount.xacro (robot description, xacro)
@@ -42,10 +42,5 @@
             <origin xyz="0.542061 -0.00202068 0.0980872" rpy="-1.61388e-15 0.00348764 1.5708"/>
             <geometry>
-                <xacro:if value="$(arg shortened_auto_mount)">
-                    <mesh filename="file://$(arg rover_description_dir)/auto_mount/meshes/clam.stl"/>
-                </xacro:if>
-                <xacro:unless value="$(arg shortened_auto_mount)">
-                    <mesh filename="file://$(arg rover_description_dir)/auto_mount/meshes/clam_old.stl"/>
-                </xacro:unless>
+                <mesh filename="file://$(arg rover_description_dir)/auto_mount_arch/meshes/clam.stl"/>
             </geometry>
             <material name="clam_material">
@@ -95,5 +90,5 @@
             <origin xyz="0.081 0.0375 -0.0275769" rpy="1.5708 2.97004e-16 -8.22153e-19"/>
             <geometry>
-                <mesh filename="file://$(arg rover_description_dir)/auto_mount/meshes/mount.stl"/>
+                <mesh filename="file://$(arg rover_description_dir)/auto_mount_arch/meshes/mount.stl"/>
             </geometry>
             <material name="mount_material">
@@ -119,5 +114,5 @@
             <origin xyz="-0.065 0.115 0.042" rpy="1.5708 1.5708 0"/>
             <geometry>
-                <mesh filename="file://$(arg rover_description_dir)/auto_mount/meshes/lidar_holder.stl"/>
+                <mesh filename="file://$(arg rover_description_dir)/auto_mount_arch/meshes/lidar_holder.stl"/>
             </geometry>
             <material name="lidar_holder_material">
@@ -127,5 +122,5 @@
     </link>
     <!-- livox_frame -->
-    <xacro:include filename="$(arg rover_description_dir)/auto_mount/urdf/livox.xacro"/>
+    <xacro:include filename="$(arg rover_description_dir)/auto_mount_arch/urdf/livox.xacro"/>
     <!-- Joint from lidar_holder to livox_frame -->
     <joint name="lidar_mate" type="fixed">
@@ -164,5 +159,5 @@
             <origin xyz="-0.005 0.025 -0.06" rpy="1.5708 1.5708 0"/>
             <geometry>
-                <mesh filename="file://$(arg rover_description_dir)/auto_mount/meshes/camera_holder.stl"/>
+                <mesh filename="file://$(arg rover_description_dir)/auto_mount_arch/meshes/camera_holder.stl"/>
             </geometry>
             <material name="camera_holder_material">
@@ -201,5 +196,5 @@
             <origin xyz="-0.005 0.025 -0.06" rpy="1.5708 1.5708 0"/>
             <geometry>
-                <mesh filename="file://$(arg rover_description_dir)/auto_mount/meshes/camera_holder.stl"/>
+                <mesh filename="file://$(arg rover_description_dir)/auto_mount_arch/meshes/camera_holder.stl"/>
             </geometry>
             <material name="camera_holder_2_material">
@@ -209,5 +204,5 @@
     </link>
     <!-- realsense d415 -->
-    <xacro:include filename="$(arg rover_description_dir)/auto_mount/urdf/realsense.xacro"/>
+    <xacro:include filename="$(arg rover_description_dir)/auto_mount_arch/urdf/realsense.xacro"/>
     <xacro:sensor_d415 parent="camera_holder_2" name="d415" use_nominal_extrinsics="$(arg gazebo)">
         <origin xyz="-0.09 0.0115 -0.058" rpy="-1.5708 0 3.14159" />
@@ -234,11 +229,6 @@
         <limit effort="10" velocity="10"/>
     </joint>
-    <joint name="auto_mount_to_chassis" type="fixed">
-        <xacro:if value="$(arg shortened_auto_mount)">
-            <origin xyz="-0.348 0 -0.063" rpy="0 -1.01333e-15 0" />
-        </xacro:if>
-        <xacro:unless value="$(arg shortened_auto_mount)">
-            <origin xyz="-0.137 0 -0.063" rpy="0 -1.01333e-15 0" />
-        </xacro:unless>
+    <joint name="auto_mount_arch_to_chassis" type="fixed">
+        <origin xyz="-0.348 0 -0.063" rpy="0 -1.01333e-15 0" />
         <parent link="chassis" />
         <child link="clam" />

File: src/ros/rover/rover_description/auto_mount_arch/urdf/livox.xacro (robot description, xacro)
@@ -5,5 +5,5 @@
             <origin xyz="0 0.0055 0" rpy="0 0 3.14159" />
             <geometry>
-                <mesh filename="file://$(arg rover_description_dir)/auto_mount/meshes/mid-360-asm.stl"/>
+                <mesh filename="file://$(arg rover_description_dir)/auto_mount_arch/meshes/mid-360-asm.stl"/>
             </geometry>
             <visibility_flags>0x02</visibility_flags> <!-- Bit 1 -->

File: src/ros/rover/rover_description/auto_mount_urc/urdf/auto_mount.xacro (robot description, xacro)
@@ -36,5 +36,5 @@
             <origin xyz="0.542061 -0.00202068 0.0980872" rpy="0 0 1.5708"/>
             <geometry>
-                <mesh filename="file://$(arg rover_description_dir)/auto_mount/meshes/clam.stl"/>
+                <mesh filename="file://$(arg rover_description_dir)/auto_mount_urc/meshes/clam.stl"/>
             </geometry>
             <material name="clam_material">
@@ -55,5 +55,5 @@
             <origin xyz="0.078 0.0285 0.0124231" rpy="1.5708 0 0" />
             <geometry>
-                <mesh filename="file://$(arg rover_description_dir)/auto_mount/meshes/mount.stl" scale="1 1 1"/>
+                <mesh filename="file://$(arg rover_description_dir)/auto_mount_urc/meshes/mount.stl" scale="1 1 1"/>
             </geometry>
             <material name="0.874510_0.568627_0.745098_0.000000_0.000000">
@@ -71,10 +71,10 @@
     </joint>
     <!-- realsense d415 -->
-    <xacro:include filename="$(arg rover_description_dir)/auto_mount/urdf/realsense.xacro"/>
+    <xacro:include filename="$(arg rover_description_dir)/auto_mount_urc/urdf/realsense.xacro"/>
     <xacro:sensor_d415 parent="mount" name="d415" use_nominal_extrinsics="${('$(arg gazebo)' == 'true') or ('$(arg sim)' == 'true')}">
         <origin xyz="0.07835 0.02469 -0.04" rpy="1.5708 1.5708 0" />
     </xacro:sensor_d415>
     <!-- livox mid-360 -->
-    <xacro:include filename="$(arg rover_description_dir)/auto_mount/urdf/livox.xacro"/>
+    <xacro:include filename="$(arg rover_description_dir)/auto_mount_urc/urdf/livox.xacro"/>
     <xacro:sensor_livox parent="mount">
         <origin xyz="0.078 0.0285 0" rpy="-1.5708 1.5708 0" />

File: src/ros/rover/rover_description/auto_mount_urc/urdf/livox.xacro (robot description, xacro)
@@ -6,5 +6,5 @@
                 <origin xyz="0 0.0055 0" rpy="0 0 3.14159" />
                 <geometry>
-                    <mesh filename="file://$(arg rover_description_dir)/auto_mount/meshes/mid-360-asm.stl"/>
+                    <mesh filename="file://$(arg rover_description_dir)/auto_mount_urc/meshes/mid-360-asm.stl"/>
                 </geometry>
                 <visibility_flags>0x02</visibility_flags> <!-- Bit 1 -->

File: src/ros/rover/rover_description/banksia/urdf/rover.urdf.xacro (robot description, xacro)
@@ -12,4 +12,5 @@
     <xacro:arg name="auto_mount" default="false"/>
     <xacro:arg name="robot_name" default="Banksia"/>
+    <xacro:arg name="comp" default ="arch"/>
     <xacro:arg name="rover_description_dir" default="$(find rover_description)" />
     <!-- Needed to prevent arm control from launching hardware interfaces for the wheels/pivots -->
@@ -32,5 +33,10 @@
     <xacro:include filename="$(arg rover_description_dir)/banksia/urdf/ckc.xacro"/>
     <xacro:if value="$(arg auto_mount)">
-        <xacro:include filename="$(arg rover_description_dir)/auto_mount/urdf/auto_mount.xacro"/>
+        <xacro:if value="${'$(arg comp)' == 'urc'}">
+            <xacro:include filename="$(arg rover_description_dir)/auto_mount_urc/urdf/auto_mount.xacro"/>
+        </xacro:if>
+        <xacro:if value="${'$(arg comp)' == 'arch'}">
+            <xacro:include filename="$(arg rover_description_dir)/auto_mount_arch/urdf/auto_mount.xacro"/>
+        </xacro:if>
     </xacro:if>
     <xacro:if value="$(arg arm)">

File: src/ros/rover/rover_description/waratah/urdf/rover.urdf.xacro (robot description, xacro)
@@ -10,5 +10,5 @@
   <xacro:arg name="rover_description_dir" default="$(find rover_description)" />
   <xacro:include
-        filename="$(find rover_description)/auto_mount/urdf/livox.xacro"
+        filename="$(find rover_description)/auto_mount_arch/urdf/livox.xacro"
     />
   <!-- Manually added links-->
