Commit message: refactor: removed duplicate urdfs of the livox and realsense.

File: src/ros/rover/rover_description/auto_mount/arch/urdf/auto_mount.xacro (robot description, xacro)
@@ -42,5 +42,5 @@
             <origin xyz="0.542061 -0.00202068 0.0980872" rpy="-1.61388e-15 0.00348764 1.5708"/>
             <geometry>
-                <mesh filename="file://$(arg rover_description_dir)/auto_mount_arch/meshes/clam.stl"/>
+                <mesh filename="file://$(arg rover_description_dir)/auto_mount/arch/meshes/clam.stl"/>
             </geometry>
             <material name="clam_material">
@@ -90,5 +90,5 @@
             <origin xyz="0.081 0.0375 -0.0275769" rpy="1.5708 2.97004e-16 -8.22153e-19"/>
             <geometry>
-                <mesh filename="file://$(arg rover_description_dir)/auto_mount_arch/meshes/mount.stl"/>
+                <mesh filename="file://$(arg rover_description_dir)/auto_mount/arch/meshes/mount.stl"/>
             </geometry>
             <material name="mount_material">
@@ -114,5 +114,5 @@
             <origin xyz="-0.065 0.115 0.042" rpy="1.5708 1.5708 0"/>
             <geometry>
-                <mesh filename="file://$(arg rover_description_dir)/auto_mount_arch/meshes/lidar_holder.stl"/>
+                <mesh filename="file://$(arg rover_description_dir)/auto_mount/arch/meshes/lidar_holder.stl"/>
             </geometry>
             <material name="lidar_holder_material">
@@ -122,11 +122,9 @@
     </link>
     <!-- livox_frame -->
-    <xacro:include filename="$(arg rover_description_dir)/auto_mount_arch/urdf/livox.xacro"/>
-    <!-- Joint from lidar_holder to livox_frame -->
-    <joint name="lidar_mate" type="fixed">
+    <xacro:include filename="$(arg rover_description_dir)/auto_mount/shared/urdf/livox.xacro"/>
+    <!-- Livox mounted on lidar_holder -->
+    <xacro:sensor_livox parent="lidar_holder">
         <origin xyz="-0.09 -0.03 0.0435" rpy="1.5708 3.14159 0"/>
-        <parent link="lidar_holder"/>
-        <child link="livox_frame"/>
-    </joint>
+    </xacro:sensor_livox>
     <!-- Joint from mount to lidar_holder -->
     <joint name="mount_to_lidar" type="fixed">
@@ -159,5 +157,5 @@
             <origin xyz="-0.005 0.025 -0.06" rpy="1.5708 1.5708 0"/>
             <geometry>
-                <mesh filename="file://$(arg rover_description_dir)/auto_mount_arch/meshes/camera_holder.stl"/>
+                <mesh filename="file://$(arg rover_description_dir)/auto_mount/arch/meshes/camera_holder.stl"/>
             </geometry>
             <material name="camera_holder_material">
@@ -196,5 +194,5 @@
             <origin xyz="-0.005 0.025 -0.06" rpy="1.5708 1.5708 0"/>
             <geometry>
-                <mesh filename="file://$(arg rover_description_dir)/auto_mount_arch/meshes/camera_holder.stl"/>
+                <mesh filename="file://$(arg rover_description_dir)/auto_mount/arch/meshes/camera_holder.stl"/>
             </geometry>
             <material name="camera_holder_2_material">
@@ -204,5 +202,5 @@
     </link>
     <!-- realsense d415 -->
-    <xacro:include filename="$(arg rover_description_dir)/auto_mount_arch/urdf/realsense.xacro"/>
+    <xacro:include filename="$(arg rover_description_dir)/auto_mount/shared/urdf/realsense.xacro"/>
     <xacro:sensor_d415 parent="camera_holder_2" name="d415" use_nominal_extrinsics="$(arg gazebo)">
         <origin xyz="-0.09 0.0115 -0.058" rpy="-1.5708 0 3.14159" />

File: src/ros/rover/rover_description/auto_mount/shared/urdf/livox.xacro (robot description, xacro)
@@ -1,13 +1,20 @@
 <?xml version="1.0" encoding="utf-8" ?>
 <robot xmlns:xacro="http://www.ros.org/wiki/xacro">
-    <link name="livox_frame">
-        <visual>
-            <origin xyz="0 0.0055 0" rpy="0 0 3.14159" />
-            <geometry>
-                <mesh filename="file://$(arg rover_description_dir)/auto_mount_arch/meshes/mid-360-asm.stl"/>
-            </geometry>
-            <visibility_flags>0x02</visibility_flags> <!-- Bit 1 -->
-        </visual>
-    </link>
+    <xacro:macro name="sensor_livox" params="parent *origin">
+        <link name="livox_frame">
+            <visual>
+                <origin xyz="0 0.0055 0" rpy="0 0 3.14159" />
+                <geometry>
+                    <mesh filename="file://$(arg rover_description_dir)/auto_mount/shared/meshes/mid-360-asm.stl"/>
+                </geometry>
+                <visibility_flags>0x02</visibility_flags> <!-- Bit 1 -->
+            </visual>
+        </link>
+        <joint name="livox_joint" type="fixed">
+            <xacro:insert_block name="origin" />
+            <parent link="${parent}" />
+            <child link="livox_frame" />
+        </joint>
+    </xacro:macro>
     <!-- Gazebo sensor plugin for the Livox MID-360 LiDAR (does not affect IRL) -->
     <xacro:if value="$(arg gazebo)">
@@ -15,5 +22,5 @@
             <visibility_flags>0x02</visibility_flags>
             <sensor name="mid360" type="gpu_lidar">
-                <update_rate>10</update_rate>
+                <update_rate>20</update_rate>
                 <topic>livox/lidar</topic>
                 <gz_frame_id>livox_frame</gz_frame_id>
@@ -51,4 +58,16 @@
                 <always_on>1</always_on>
                 <visualize>false</visualize>
+                <imu>
+                    <angular_velocity>
+                        <x><noise type="gaussian"><mean>0.0</mean><stddev>2e-4</stddev></noise></x>
+                        <y><noise type="gaussian"><mean>0.0</mean><stddev>2e-4</stddev></noise></y>
+                        <z><noise type="gaussian"><mean>0.0</mean><stddev>2e-4</stddev></noise></z>
+                    </angular_velocity>
+                    <linear_acceleration>
+                        <x><noise type="gaussian"><mean>0.0</mean><stddev>1.7e-2</stddev></noise></x>
+                        <y><noise type="gaussian"><mean>0.0</mean><stddev>1.7e-2</stddev></noise></y>
+                        <z><noise type="gaussian"><mean>0.0</mean><stddev>1.7e-2</stddev></noise></z>
+                    </linear_acceleration>
+                </imu>
             </sensor>
         </gazebo>

File: src/ros/rover/rover_description/auto_mount/urc/urdf/auto_mount.xacro (robot description, xacro)
@@ -36,5 +36,5 @@
             <origin xyz="0.542061 -0.00202068 0.0980872" rpy="0 0 1.5708"/>
             <geometry>
-                <mesh filename="file://$(arg rover_description_dir)/auto_mount_urc/meshes/clam.stl"/>
+                <mesh filename="file://$(arg rover_description_dir)/auto_mount/urc/meshes/clam.stl"/>
             </geometry>
             <material name="clam_material">
@@ -55,5 +55,5 @@
             <origin xyz="0.078 0.0285 0.0124231" rpy="1.5708 0 0" />
             <geometry>
-                <mesh filename="file://$(arg rover_description_dir)/auto_mount_urc/meshes/mount.stl" scale="1 1 1"/>
+                <mesh filename="file://$(arg rover_description_dir)/auto_mount/urc/meshes/mount.stl" scale="1 1 1"/>
             </geometry>
             <material name="0.874510_0.568627_0.745098_0.000000_0.000000">
@@ -71,10 +71,10 @@
     </joint>
     <!-- realsense d415 -->
-    <xacro:include filename="$(arg rover_description_dir)/auto_mount_urc/urdf/realsense.xacro"/>
+    <xacro:include filename="$(arg rover_description_dir)/auto_mount/shared/urdf/realsense.xacro"/>
     <xacro:sensor_d415 parent="mount" name="d415" use_nominal_extrinsics="${('$(arg gazebo)' == 'true') or ('$(arg sim)' == 'true')}">
         <origin xyz="0.07835 0.02469 -0.04" rpy="1.5708 1.5708 0" />
     </xacro:sensor_d415>
     <!-- livox mid-360 -->
-    <xacro:include filename="$(arg rover_description_dir)/auto_mount_urc/urdf/livox.xacro"/>
+    <xacro:include filename="$(arg rover_description_dir)/auto_mount/shared/urdf/livox.xacro"/>
     <xacro:sensor_livox parent="mount">
         <origin xyz="0.078 0.0285 0" rpy="-1.5708 1.5708 0" />

File: src/ros/rover/rover_description/banksia/urdf/rover.urdf.xacro (robot description, xacro)
@@ -34,8 +34,8 @@
     <xacro:if value="$(arg auto_mount)">
         <xacro:if value="${'$(arg comp)' == 'urc'}">
-            <xacro:include filename="$(arg rover_description_dir)/auto_mount_urc/urdf/auto_mount.xacro"/>
+            <xacro:include filename="$(arg rover_description_dir)/auto_mount/urc/urdf/auto_mount.xacro"/>
         </xacro:if>
         <xacro:if value="${'$(arg comp)' == 'arch'}">
-            <xacro:include filename="$(arg rover_description_dir)/auto_mount_arch/urdf/auto_mount.xacro"/>
+            <xacro:include filename="$(arg rover_description_dir)/auto_mount/arch/urdf/auto_mount.xacro"/>
         </xacro:if>
     </xacro:if>
