Commit message: Auto mount comp conditional URDF launching, and other comp demo additions. (#1256)
Co-authored-by: Monash Nova Rover <novaroverteam@monash.edu>
Co-authored-by: hhoverall <hove0001@student.monash.edu>

File: src/ros/rover/rover_description/auto_mount/shared/urdf/livox.xacro (robot description, xacro)
@@ -6,5 +6,5 @@
                 <origin xyz="0 0.0055 0" rpy="0 0 3.14159" />
                 <geometry>
-                    <mesh filename="file://$(arg rover_description_dir)/auto_mount/meshes/mid-360-asm.stl"/>
+                    <mesh filename="file://$(arg rover_description_dir)/auto_mount/shared/meshes/mid-360-asm.stl"/>
                 </geometry>
                 <visibility_flags>0x02</visibility_flags> <!-- Bit 1 -->

File: src/ros/rover/rover_description/auto_mount/urc/urdf/auto_mount.xacro (robot description, xacro)
@@ -36,5 +36,5 @@
             <origin xyz="0.542061 -0.00202068 0.0980872" rpy="0 0 1.5708"/>
             <geometry>
-                <mesh filename="file://$(arg rover_description_dir)/auto_mount/meshes/clam.stl"/>
+                <mesh filename="file://$(arg rover_description_dir)/auto_mount/urc/meshes/clam.stl"/>
             </geometry>
             <material name="clam_material">
@@ -55,5 +55,5 @@
             <origin xyz="0.078 0.0285 0.0124231" rpy="1.5708 0 0" />
             <geometry>
-                <mesh filename="file://$(arg rover_description_dir)/auto_mount/meshes/mount.stl" scale="1 1 1"/>
+                <mesh filename="file://$(arg rover_description_dir)/auto_mount/urc/meshes/mount.stl" scale="1 1 1"/>
             </geometry>
             <material name="0.874510_0.568627_0.745098_0.000000_0.000000">
@@ -71,10 +71,10 @@
     </joint>
     <!-- realsense d415 -->
-    <xacro:include filename="$(arg rover_description_dir)/auto_mount/urdf/realsense.xacro"/>
+    <xacro:include filename="$(arg rover_description_dir)/auto_mount/shared/urdf/realsense.xacro"/>
     <xacro:sensor_d415 parent="mount" name="d415" use_nominal_extrinsics="${('$(arg gazebo)' == 'true') or ('$(arg sim)' == 'true')}">
         <origin xyz="0.07835 0.02469 -0.04" rpy="1.5708 1.5708 0" />
     </xacro:sensor_d415>
     <!-- livox mid-360 -->
-    <xacro:include filename="$(arg rover_description_dir)/auto_mount/urdf/livox.xacro"/>
+    <xacro:include filename="$(arg rover_description_dir)/auto_mount/shared/urdf/livox.xacro"/>
     <xacro:sensor_livox parent="mount">
         <origin xyz="0.078 0.0285 0" rpy="-1.5708 1.5708 0" />

File: src/ros/rover/rover_description/banksia/urdf/rover.urdf.xacro (robot description, xacro)
@@ -12,4 +12,5 @@
     <xacro:arg name="auto_mount" default="false"/>
     <xacro:arg name="robot_name" default="Banksia"/>
+    <xacro:arg name="comp" default ="arch"/>
     <xacro:arg name="rover_description_dir" default="$(find rover_description)" />
     <!-- Needed to prevent arm control from launching hardware interfaces for the wheels/pivots -->
@@ -32,5 +33,10 @@
     <xacro:include filename="$(arg rover_description_dir)/banksia/urdf/ckc.xacro"/>
     <xacro:if value="$(arg auto_mount)">
-        <xacro:include filename="$(arg rover_description_dir)/auto_mount/urdf/auto_mount.xacro"/>
+        <xacro:if value="${'$(arg comp)' == 'urc'}">
+            <xacro:include filename="$(arg rover_description_dir)/auto_mount/urc/urdf/auto_mount.xacro"/>
+        </xacro:if>
+        <xacro:if value="${'$(arg comp)' == 'arch'}">
+            <xacro:include filename="$(arg rover_description_dir)/auto_mount/arch/urdf/auto_mount.xacro"/>
+        </xacro:if>
     </xacro:if>
     <xacro:if value="$(arg arm)">
